Commit message: started urdf reorganization:
helicopter.gazebo.urdf now instantiates the heli "mechanics" first, as these usually do not change. Then, we create links and attach sensors / plugins according to the current task. Hope that makes sense...

File: mav_description/urdf/firefly.gazebo.xacro (robot description, xacro)
@@ -1,4 +1,88 @@
 <?xml version="1.0"?>
 <robot name="firefly" xmlns:xacro="http://ros.org/wiki/xacro">
-    <xacro:include filename="$(find mav_description)/urdf/firefly.urdf.xacro" />
+  <xacro:property name="namespace" value="firefly" />
+	<xacro:property name="enable_bag_plugin" value="false" />
+	<!-- Instantiate firefly "mechanics" -->
+	<xacro:include filename="$(find mav_description)/urdf/firefly.urdf.xacro" />
+	<!-- Create link and joint for a sensor -->
+	<link name="pose_sensor1_link">
+		<inertial>
+			<inertia ixx="0.001" ixy="0.0" ixz="0.0" iyy="0.001" iyz="0.0"
+				izz="0.001" />
+			<mass value="0.01" />  <!-- [kg] -->
+		</inertial>
+	</link>
+	<joint name="pose_sensor1_joint" type="revolute">
+		<parent link="base_link" />
+		<origin xyz="0 0 0" rpy="0 0 0" />
+		<child link="pose_sensor1_link" />
+		<limit upper="0" lower="0" effort="0" velocity="0" />
+	</joint>
+  <!-- Mount an IMU -->
+  <gazebo>
+    <!-- IMU -->
+    <plugin filename="libhector_gazebo_ros_imu.so" name="imu_ros">
+      <!-- parameters according to http://wiki.ros.org/hector_gazebo_plugins#GazeboRosImu -->
+      <robotNamespace>${namespace}</robotNamespace>
+      <bodyName>imu_link</bodyName> <!-- (string, required): name of the body which holds the IMU sensor -->
+      <topicName>imu</topicName> <!-- (string): name of the sensor output topic and prefix of service names (defaults to imu) -->
+      <accelOffset>0.0 0.0 0.0</accelOffset> <!-- (Vector3): constant acceleration offset -->
+      <accelDrift>0.0 0.0 0.0</accelDrift> <!-- (Vector3): standard deviation of the acceleration drift error -->
+      <accelDriftFrequency>${1.0/3600.0} ${1.0/3600.0} ${1.0/3600.0}</accelDriftFrequency> <!-- (Vector3): mean frequency of the acceleration drift -->
+      <accelGaussianNoise>0.0 0.0 0.0</accelGaussianNoise> <!-- (Vector3): standard deviation of the additive Gaussian acceleration noise -->
+      <rateOffset>0.0 0.0 0.0</rateOffset> <!-- (Vector3): constant rate offset -->
+      <rateDrift>0.0 0.0 0.0</rateDrift> <!-- (Vector3): standard deviation of the rate drift error -->
+      <rateDriftFrequency>${1.0/3600.0} ${1.0/3600.0} ${1.0/3600.0}</rateDriftFrequency> <!-- (Vector3): mean frequency of the rate drift -->
+      <rateGaussianNoise>0.0 0.0 0.0</rateGaussianNoise> <!-- (Vector3): standard deviation of the additive Gaussian rate noise -->
+      <headingOffset>0.0</headingOffset> <!-- (double): constant heading offset -->
+      <headingDrift>0.0</headingDrift> <!-- (double): standard deviation of the heading drift error -->
+      <headingDriftFrequency>${1.0/3600.0}</headingDriftFrequency> <!-- (double): mean frequency of the heading drift -->
+      <headingGaussianNoise>0.0</headingGaussianNoise> <!-- (double): standard deviation of the heading additive Gaussian noise -->
+      <rpyOffsets>0.0 0.0 0.0</rpyOffsets> <!-- (Vector3): if non-zero, used to calculate accelOffset and headingOffset so that resulting roll, pitch and yaw errors correspond to this values when the platform is leveled (for compatibility with gazebo_plugins) -->
+    </plugin>
+  </gazebo>
+  <!-- Instantiate a controller -->
+	<gazebo>
+		<!-- Controller interface -->
+		<plugin name="controller_interface" filename="libmav_gazebo_controller_interface.so">
+			<robotNamespace>${namespace}</robotNamespace>
+			<commandTopicAttitude>mav_cmd_attitude</commandTopicAttitude>
+			<commandTopicRate>mav_cmd_rate</commandTopicRate>
+			<commandTopicMotor>mav_cmd_motor</commandTopicMotor>
+			<imuTopic>imu</imuTopic>
+			<poseTopic>pose</poseTopic>
+			<motorVelocityReferenceTopic>motor_vel_ref</motorVelocityReferenceTopic>
+		</plugin>
+	</gazebo>
+  <!-- Mount a generic pose sensor at link sensor1 -->
+  <gazebo>
+    <!-- Generic 6D pose sensor plugin -->
+    <plugin filename="libmav_gazebo_pose_plugin.so" name="pose_sensor1">
+      <linkName>pose_sensor1_link</linkName>
+      <robotNamespace>${namespace}</robotNamespace>
+      <poseTopic>sensors/pose1</poseTopic>
+      <measurementDivisor>7</measurementDivisor> <!-- only every (seq % measurementDivisor) == 0 measurement is published [int] -->
+      <measurementDelay>0</measurementDelay> <!-- time that measurement gets held back before it's published in [simulation cycles (int)] -->
+      <unknownDelay>0.0</unknownDelay> <!-- additional delay, that just gets added to the timestamp [s] -->
+      <noiseNormalP>0.005 0.005 0.005</noiseNormalP> <!-- standard deviation of additive white gaussian noise [m] -->
+      <noiseNormalQ>0.01 0.01 0.01</noiseNormalQ> <!-- standard deviation white gaussian noise [rad]: q_m = q*quaternionFromSmallAngleApproximation(noiseNormalQ) -->
+      <noiseUniformP>0 0 0</noiseUniformP> <!-- symmetric bounds of uniform noise [m] -->
+      <noiseUniformQ>0 0 0</noiseUniformQ> <!-- symmetric bounds of uniform noise [rad], computation see above -->
+    </plugin>
+  </gazebo>
+  <!-- Instantiate a logger -->
+  <gazebo>
+		<!-- ROS Bag Plugin -->
+		<xacro:if value="${enable_bag_plugin}">
+			<plugin filename="libmav_gazebo_bag_plugin.so" name="rosbag">
+				<robotNamespace>${namespace}</robotNamespace>
+				<bagFileName>${bag_file}</bagFileName>
+				<linkName>base_link</linkName>
+				<frameId>base_link</frameId>
+				<controlAttitudeThrustSubTopic>mav_cmd</controlAttitudeThrustSubTopic>
+				<controlAttitudeThrustPubTopic>mav_cmd</controlAttitudeThrustPubTopic>
+				<rotorVelocitySlowdownSim>${rotor_velocity_slowdown_sim}</rotorVelocitySlowdownSim>
+			</plugin>
+		</xacro:if>
+	</gazebo>
 </robot>

File: mav_description/urdf/firefly.urdf.xacro (robot description, xacro)
@@ -1,9 +1,6 @@
 <?xml version="1.0"?>
-<robot
-  name="firefly"
-  xmlns:xacro="http://ros.org/wiki/xacro"
->
+<robot name="firefly" xmlns:xacro="http://ros.org/wiki/xacro">
   <!-- Properties -->
-  <xacro:property name="namespace" value="firefly" />
+  <xacro:property name="rotor_velocity_slowdown_sim" value="10" />
   <xacro:property name="mesh_file" value="firefly.dae" />
   <xacro:property name="mass" value="1.5" /> <!-- [kg] -->
@@ -38,6 +35,5 @@
     body_height="${body_height}"
     mesh_file="${mesh_file}"
-    bag_file="firefly.bag"
-    enable_bag_plugin="false">
+    >
     <xacro:insert_block name="body_inertia" />
   </xacro:multirotor_base_macro>

File: mav_description/urdf/multirotor_base.urdf.xacro (robot description, xacro)
@@ -1,12 +1,12 @@
 <?xml version="1.0"?>
 <robot xmlns:xacro="http://ros.org/wiki/xacro">
-  <xacro:property name="rotor_velocity_slowdown_sim" value="10" />
   <!-- Main multirotor link -->
-  <xacro:macro name="multirotor_base_macro" params="robot_namespace mass body_width body_height mesh_file bag_file enable_bag_plugin *inertia">
+  <xacro:macro name="multirotor_base_macro"
+    params="robot_namespace mass body_width body_height mesh_file *inertia">
     <link name="base_link"></link>
     <joint name="base_joint" type="fixed">
       <origin xyz="0 0 0" rpy="0 0 0" />
-      <parent link="base_link"/>
-      <child link="base_link_inertia"/>
+      <parent link="base_link" />
+      <child link="base_link_inertia" />
     </joint>
     <link name="base_link_inertia">
@@ -19,5 +19,6 @@
         <origin xyz="0 0 0" rpy="0 0 0" />
         <geometry>
-          <mesh filename="package://mav_description/meshes/${mesh_file}" scale="1 1 1"/>
+          <mesh filename="package://mav_description/meshes/${mesh_file}"
+            scale="1 1 1" />
           <!-- <box size="${body_width} ${body_width} ${body_height}"/> --> <!-- [m] [m] [m] -->
         </geometry>
@@ -26,5 +27,5 @@
         <origin xyz="0 0 0" rpy="0 0 0" />
         <geometry>
-          <box size="${body_width} ${body_width} ${body_height}"/> <!-- [m] [m] [m] -->
+          <box size="${body_width} ${body_width} ${body_height}" /> <!-- [m] [m] [m] -->
         </geometry>
       </collision>
@@ -33,148 +34,17 @@
     <link name="imu_link">
       <inertial>
-        <inertia ixx="0.001" ixy="0.0" ixz="0.0" iyy="0.001" iyz="0.0" izz="0.001" />
+        <inertia ixx="0.001" ixy="0.0" ixz="0.0" iyy="0.001" iyz="0.0"
+          izz="0.001" />
         <mass value="0.01" />  <!-- [kg] -->
-        <origin xyz="0 0 0" rpy="0 0 0"/>
+        <origin xyz="0 0 0" rpy="0 0 0" />
       </inertial>
     </link>
     <!-- IMU joint -->
     <joint name="imu_joint" type="revolute">
-      <!--origin xyz="0 0 0" rpy="3.1416 0 0" /-->
-      <parent link="base_link"/>
-      <child link="imu_link"/>
-      <limit upper="0" lower="0" effort="0" velocity="0"/>
+      <!--origin xyz="0 0 0" rpy="3.1416 0 0" / -->
+      <parent link="base_link" />
+      <child link="imu_link" />
+      <limit upper="0" lower="0" effort="0" velocity="0" />
     </joint>
-    <!-- pose sensor1 -->
-    <link name="pose_sensor1_link" >
-      <inertial>
-        <inertia ixx="0.001" ixy="0.0" ixz="0.0" iyy="0.001" iyz="0.0" izz="0.001" />
-        <mass value="0.01" />  <!-- [kg] -->
-      </inertial>
-    </link>
-    <joint name="pose_sensor1_joint" type="revolute">
-    <parent link="base_link"/>
-      <origin xyz="0.1 0 0" rpy="0 ${3.14/4.0} 0" />
-      <child link="pose_sensor1_link"/>
-      <limit upper="0" lower="0" effort="0" velocity="0"/>
-    </joint>
-     <!-- pose sensor2 -->
-    <link name="pose_sensor2_link" >
-      <inertial>
-        <inertia ixx="0.001" ixy="0.0" ixz="0.0" iyy="0.001" iyz="0.0" izz="0.001" />
-        <mass value="0.01" />  <!-- [kg] -->
-      </inertial>
-    </link>
-    <joint name="pose_sensor2_joint" type="revolute">
-    <parent link="base_link"/>
-      <origin xyz="0.0 0.0 0.1" rpy="0.0 0.0 0.0" />
-      <child link="pose_sensor2_link"/>
-      <limit upper="0" lower="0" effort="0" velocity="0"/>
-    </joint>
-    <gazebo>
-      <!-- Controller interface -->
-      <plugin name="controller_interface"
-        filename="libmav_gazebo_controller_interface.so">
-        <robotNamespace>${robot_namespace}</robotNamespace>
-        <commandTopicAttitude>mav_cmd_attitude</commandTopicAttitude>
-        <commandTopicRate>mav_cmd_rate</commandTopicRate>
-        <commandTopicMotor>mav_cmd_motor</commandTopicMotor>
-        <imuTopic>imu</imuTopic>
-        <poseTopic>pose</poseTopic>
-        <motorVelocityReferenceTopic>motor_vel_ref</motorVelocityReferenceTopic>
-      </plugin>
-      <!-- IMU -->
-      <plugin filename="libhector_gazebo_ros_imu.so" name="imu_ros">
-        <!-- parameters according to http://wiki.ros.org/hector_gazebo_plugins#GazeboRosImu -->
-        <robotNamespace>${robot_namespace}</robotNamespace>
-        <bodyName>imu_link</bodyName> <!-- (string, required): name of the body which holds the IMU sensor -->
-        <topicName>imu</topicName> <!-- (string): name of the sensor output topic and prefix of service names (defaults to imu) -->
-        <accelOffset>0.0 0.0 0.0</accelOffset> <!-- (Vector3): constant acceleration offset -->
-        <accelDrift>0.0 0.0 0.0</accelDrift> <!-- (Vector3): standard deviation of the acceleration drift error -->
-        <accelDriftFrequency>${1.0/3600.0} ${1.0/3600.0} ${1.0/3600.0}</accelDriftFrequency> <!-- (Vector3): mean frequency of the acceleration drift -->
-        <accelGaussianNoise>0.0 0.0 0.0</accelGaussianNoise> <!-- (Vector3): standard deviation of the additive Gaussian acceleration noise -->
-        <rateOffset>0.0 0.0 0.0</rateOffset> <!-- (Vector3): constant rate offset -->
-        <rateDrift>0.0 0.0 0.0</rateDrift> <!-- (Vector3): standard deviation of the rate drift error -->
-        <rateDriftFrequency>${1.0/3600.0} ${1.0/3600.0} ${1.0/3600.0}</rateDriftFrequency> <!-- (Vector3): mean frequency of the rate drift -->
-        <rateGaussianNoise>0.0 0.0 0.0</rateGaussianNoise> <!-- (Vector3): standard deviation of the additive Gaussian rate noise -->
-        <headingOffset>0.0</headingOffset> <!-- (double): constant heading offset -->
-        <headingDrift>0.0</headingDrift> <!-- (double): standard deviation of the heading drift error -->
-        <headingDriftFrequency>${1.0/3600.0}</headingDriftFrequency> <!-- (double): mean frequency of the heading drift -->
-        <headingGaussianNoise>0.0</headingGaussianNoise> <!-- (double): standard deviation of the heading additive Gaussian noise -->
-        <rpyOffsets>0.0 0.0 0.0</rpyOffsets> <!-- (Vector3): if non-zero, used to calculate accelOffset and headingOffset so that resulting roll, pitch and yaw errors correspond to this values when the platform is leveled (for compatibility with gazebo_plugins) -->
-      </plugin>
-      <plugin filename="libhector_gazebo_ros_imu.so" name="imu_ros">
-        <robotNamespace>${robot_namespace}</robotNamespace>
-        <bodyName>imu_link</bodyName>
-        <topicName>ground_truth/imu</topicName>
-        <!-- everything defaults to zero, except drift frequency, let's do that for safety -->
-        <accelDriftFrequency>0.0 0.0 0.0</accelDriftFrequency>
-        <rateDriftFrequency>0.0 0.0 0.0</rateDriftFrequency>
-        <headingDriftFrequency>0.0</headingDriftFrequency>
-      </plugin>
-      <!-- ROS Bag Plugin -->
-      <xacro:if value="${enable_bag_plugin}">
-      <plugin filename="libmav_gazebo_bag_plugin.so" name="rosbag">
-        <robotNamespace>${robot_namespace}</robotNamespace>
-        <bagFileName>${bag_file}</bagFileName>
-        <linkName>base_link</linkName>
-        <frameId>base_link</frameId>
-        <controlAttitudeThrustSubTopic>mav_cmd</controlAttitudeThrustSubTopic>
-        <controlAttitudeThrustPubTopic>mav_cmd</controlAttitudeThrustPubTopic>
-        <rotorVelocitySlowdownSim>${rotor_velocity_slowdown_sim}</rotorVelocitySlowdownSim>
-      </plugin>
-      </xacro:if>
-      <plugin filename="libmav_gazebo_pose_plugin.so" name="ground_truth_pose">
-        <linkName>base_link</linkName>
-        <robotNamespace>${robot_namespace}</robotNamespace>
-        <poseTopic>ground_truth/pose</poseTopic>
-        <measurementDivisor>1</measurementDivisor>
-        <measurementDelay>0</measurementDelay>
-        <noiseNormalP>0 0 0</noiseNormalP>
-        <noiseNormalQ>0 0 0</noiseNormalQ>
-        <noiseUniformP>0 0 0</noiseUniformP>
-        <noiseUniformQ>0 0 0</noiseUniformQ>
-      </plugin>
-      <plugin filename="libmav_gazebo_pose_plugin.so" name="pose_sensor1">
-        <linkName>pose_sensor1_link</linkName>
-        <robotNamespace>${robot_namespace}</robotNamespace>
-        <poseTopic>sensors/pose1</poseTopic>
-        <measurementDivisor>7</measurementDivisor> <!-- only every (seq % measurementDivisor) == 0 measurement is published [int]-->
-        <measurementDelay>0</measurementDelay> <!-- time that measurement gets held back before it's published in [simulation cycles (int)] -->
-        <unknownDelay>0.0</unknownDelay> <!-- additional delay, that just gets added to the timestamp [s] -->
-        <noiseNormalP>0.01 0.01 0.01</noiseNormalP> <!-- standard deviation of additive white gaussian noise [m] -->
-        <noiseNormalQ>0.02 0.02 0.02</noiseNormalQ> <!-- standard deviation white gaussian noise [rad]: q_m = q*quaternionFromSmallAngleApproximation(noiseNormalQ)-->
-        <noiseUniformP>0 0 0</noiseUniformP> <!-- symmetric bounds of uniform noise [m] -->
-        <noiseUniformQ>0 0 0</noiseUniformQ> <!-- symmetric bounds of uniform noise [rad], computation see above -->
-        <covarianceImage>package://mav_gazebo/worlds/poseplugin_map1.bmp</covarianceImage>
-        <covarianceImageScale>0.1</covarianceImageScale>
-      </plugin>
-      <plugin filename="libmav_gazebo_pose_plugin.so" name="pose_sensor2">
-        <linkName>pose_sensor2_link</linkName>
-        <robotNamespace>${robot_namespace}</robotNamespace>
-        <poseTopic>sensors/pose2</poseTopic>
-        <measurementDivisor>5</measurementDivisor>
-        <measurementDelay>0</measurementDelay>
-        <unknownDelay>0.001</unknownDelay>
-        <noiseNormalP>0.01 0.01 0.01</noiseNormalP>
-        <noiseNormalQ>0.02 0.02 0.02</noiseNormalQ>
-        <noiseUniformP>0 0 0</noiseUniformP>
-        <noiseUniformQ>0 0 0</noiseUniformQ>
-        <covarianceImage>package://mav_gazebo/worlds/poseplugin_map2.bmp</covarianceImage>
-        <covarianceImageScale>0.1</covarianceImageScale>
-      </plugin>
-      <!-- Wind Plugin -->
-      <plugin filename="libmav_gazebo_wind_plugin.so" name="wind_plugin">
-        <frameId>base_link</frameId>
-        <linkName>base_link</linkName>
-        <robotNamespace>${robot_namespace}</robotNamespace>
-        <xyzOffset>0 0 0</xyzOffset> <!-- [m] [m] [m] -->
-        <windDirection>1 0 0</windDirection>
-        <windForceMean>0</windForceMean> <!-- [N] -->
-        <windGustDirection>0 1 0</windGustDirection>
-        <windGustDuration>2</windGustDuration> <!-- [s] -->
-        <windGustStart>10</windGustStart> <!-- [s] -->
-        <windGustForceMean>0</windGustForceMean> <!-- [N] -->
-      </plugin>
-    </gazebo>
   </xacro:macro>
   <!-- camera -->
@@ -183,26 +53,26 @@
     <joint name="camera_joint" type="fixed">
       <axis xyz="0 1 0" />
-      <origin xyz="0 0 0.2" rpy="0 0 0"/>
-      <parent link="base_link"/>
-      <child link="camera_link"/>
+      <origin xyz="0 0 0.2" rpy="0 0 0" />
+      <parent link="base_link" />
+      <child link="camera_link" />
     </joint>
     <!-- link -->
     <link name="camera_link">
       <collision>
-        <origin xyz="0 0 0" rpy="0 0 0"/>
+        <origin xyz="0 0 0" rpy="0 0 0" />
         <geometry>
-      <box size="0.1 0.1 0.1"/>
+          <box size="0.1 0.1 0.1" />
         </geometry>
       </collision>
       <visual>
-        <origin xyz="0 0 0" rpy="0 0 0"/>
+        <origin xyz="0 0 0" rpy="0 0 0" />
         <geometry>
-      <box size="0.1 0.1 0.1"/>
+          <box size="0.1 0.1 0.1" />
         </geometry>
-        <material name="red"/>
+        <material name="red" />
       </visual>
       <inertial>
         <mass value="1e-5" />
-        <origin xyz="0 0 0" rpy="0 0 0"/>
+        <origin xyz="0 0 0" rpy="0 0 0" />
         <inertia ixx="1e-6" ixy="0" ixz="0" iyy="1e-6" iyz="0" izz="1e-6" />
       </inertial>
@@ -246,5 +116,6 @@
   </xacro:macro>
   <!-- Rotor joint and link -->
-  <xacro:macro name="vertical_rotor" params="robot_namespace suffix direction motor_constant moment_constant parent mass_rotor radius_rotor time_constant max_rot_velocity motor_number rotor_drag_coefficient rolling_moment_coefficient color *origin *inertia">
+  <xacro:macro name="vertical_rotor"
+    params="robot_namespace suffix direction motor_constant moment_constant parent mass_rotor radius_rotor time_constant max_rot_velocity motor_number rotor_drag_coefficient rolling_moment_coefficient color *origin *inertia">
     <joint name="rotor_${motor_number}_joint" type="continuous">
       <xacro:insert_block name="origin" />
@@ -252,18 +123,10 @@
       <!-- TODO(ff): not currently set because it's not yet supported -->
       <!-- <limit effort="2000" velocity="${max_rot_velocity}" /> -->
-      <parent link="${parent}"/>
-      <child link="rotor_${motor_number}"/>
+      <parent link="${parent}" />
+      <child link="rotor_${motor_number}" />
     </joint>
     <!-- TODO(ff): not currently set because it's not yet supported -->
-    <!-- <gazebo reference="rotor_${motor_number}_joint">
-      <axis>
-        <xyz>0 0 1</xyz>
-        <limit>
-          <velocity>
-            ${max_rot_velocity}
-          </velocity>
-        </limit>
-      </axis>
-    </gazebo> -->
+    <!-- <gazebo reference="rotor_${motor_number}_joint"> <axis> <xyz>0 0 1</xyz>
+      <limit> <velocity> ${max_rot_velocity} </velocity> </limit> </axis> </gazebo> -->
     <link name="rotor_${motor_number}">
       <inertial>
@@ -274,5 +137,6 @@
         <geometry>
           <!-- <cylinder length="0.005" radius="${radius_rotor}"/> --> <!-- [m] -->
-          <mesh filename="package://mav_description/meshes/propeller_${direction}.dae" scale="0.001 0.001 0.001"/>
+          <mesh filename="package://mav_description/meshes/propeller_${direction}.dae"
+            scale="0.001 0.001 0.001" />
           <!-- <box size="${2*radius_rotor} 0.01 0.005"/> -->
         </geometry>
@@ -280,5 +144,5 @@
       <collision>
         <geometry>
-          <cylinder length="0.005" radius="${radius_rotor}"/> <!-- [m] -->
+          <cylinder length="0.005" radius="${radius_rotor}" /> <!-- [m] -->
         </geometry>
       </collision>

Commit message: added missing bagfilename parameter

File: mav_description/urdf/firefly.gazebo.xacro (robot description, xacro)
@@ -2,5 +2,6 @@
 <robot name="firefly" xmlns:xacro="http://ros.org/wiki/xacro">
   <xacro:property name="namespace" value="firefly" />
-	<xacro:property name="enable_bag_plugin" value="false" />
+  <xacro:property name="enable_bag_plugin" value="false" />
+  <xacro:property name="bag_file" value="firefly.bag" />
 	<!-- Instantiate firefly "mechanics" -->
 	<xacro:include filename="$(find mav_description)/urdf/firefly.urdf.xacro" />
