Commit message: added vi_sensor mesh

File: mav_description/urdf/vi_sensor.xacro (robot description, xacro)
@@ -16,7 +16,6 @@
       <origin xyz="0 0 0" rpy="0 0 0" />
       <geometry>
-        <box size="0.03 0.133 0.057" />
+        <mesh filename="package://mav_description/meshes/vi_sensor.dae" scale="1 1 1" />
       </geometry>
-      <material name="red" />
     </visual>
     <inertial>

Commit message: added mesh with texture for the vi_sensor

File: mav_description/urdf/vi_sensor.xacro (robot description, xacro)
@@ -33,5 +33,5 @@
       </geometry>
     </collision>
-    <visual>
+    <!-- <visual>
       <origin xyz="0 0 0" rpy="0 ${PI/2} 0" />
       <geometry>
@@ -39,5 +39,5 @@
       </geometry>
       <material name="red" />
-    </visual>
+    </visual> -->
     <inertial>
       <mass value="1e-5" />
@@ -54,5 +54,5 @@
       </geometry>
     </collision>
-    <visual>
+    <!-- <visual>
       <origin xyz="0 0 0" rpy="0 ${PI/2} 0" />
       <geometry>
@@ -60,5 +60,5 @@
       </geometry>
       <material name="red" />
-    </visual>
+    </visual> -->
     <inertial>
       <mass value="1e-5" />
@@ -75,5 +75,5 @@
       </geometry>
     </collision>
-    <visual>
+    <!-- <visual>
       <origin xyz="0 0 0" rpy="0 0 0" />
       <geometry>
@@ -81,5 +81,5 @@
       </geometry>
       <material name="red" />
-    </visual>
+    </visual> -->
     <inertial>
       <inertia ixx="0.001" ixy="0.0" ixz="0.0" iyy="0.001" iyz="0.0"
