Commit message: made bag plugin switchable by xacro fixed filenaming: if started with /, an absolute path is chosen

File: mav_description/urdf/firefly.urdf.xacro (robot description, xacro)
@@ -32,5 +32,12 @@
   <xacro:include filename="$(find mav_description)/urdf/multirotor_base.urdf.xacro" />
   <!-- Instantiate multirotor_base_macro once -->
-  <xacro:multirotor_base_macro robot_namespace="${namespace}" mass="${mass}" body_width="${body_width}" body_height="${body_height}" mesh_file="${mesh_file}">
+  <xacro:multirotor_base_macro
+    robot_namespace="${namespace}"
+    mass="${mass}"
+    body_width="${body_width}"
+    body_height="${body_height}"
+    mesh_file="${mesh_file}"
+    bag_file="firefly.bag"
+    enable_bag_plugin="true">
     <xacro:insert_block name="body_inertia" />
   </xacro:multirotor_base_macro>

File: mav_description/urdf/multirotor_base.urdf.xacro (robot description, xacro)
@@ -3,5 +3,5 @@
   <xacro:property name="rotor_velocity_slowdown_sim" value="10" />
   <!-- Main multirotor link -->
-  <xacro:macro name="multirotor_base_macro" params="robot_namespace mass body_width body_height mesh_file *inertia">
+  <xacro:macro name="multirotor_base_macro" params="robot_namespace mass body_width body_height mesh_file bag_file enable_bag_plugin *inertia">
     <link name="base_link"></link>
     <joint name="base_joint" type="fixed">
@@ -113,7 +113,8 @@
       </plugin>
       <!-- ROS Bag Plugin -->
+      <xacro:if value="${enable_bag_plugin}">
       <plugin filename="libmav_gazebo_bag_plugin.so" name="rosbag">
         <robotNamespace>${robot_namespace}</robotNamespace>
-        <bagFileName>firefly.bag</bagFileName>
+        <bagFileName>${bag_file}</bagFileName>
         <linkName>base_link</linkName>
         <frameId>base_link</frameId>
@@ -122,4 +123,5 @@
         <rotorVelocitySlowdownSim>${rotor_velocity_slowdown_sim}</rotorVelocitySlowdownSim>
       </plugin>
+      </xacro:if>
       <plugin filename="libmav_gazebo_pose_plugin.so" name="ground_truth_pose">
         <linkName>base_link</linkName>

Commit message: added (hopefully) correct inertia for rotor and compensated by rotor_slowdown_sim

File: mav_description/urdf/firefly.urdf.xacro (robot description, xacro)
@@ -7,9 +7,9 @@
   <xacro:property name="body_width" value="0.1" /> <!-- [m] -->
   <xacro:property name="body_height" value="0.16" /> <!-- [m] -->
-  <xacro:property name="mass_rotor" value="0.01" /> <!-- [kg] -->
+  <xacro:property name="mass_rotor" value="0.005" /> <!-- [kg] -->
   <xacro:property name="arm_length" value="0.215" /> <!-- [m] -->
   <xacro:property name="rotor_offset_top" value="0.037" /> <!-- [m] -->
-  <xacro:property name="radius_rotor" value="0.08" /> <!-- [m] -->
-  <xacro:property name="motor_constant" value="9.9865e-06" /> <!-- [kg·m/s^2] -->
+  <xacro:property name="radius_rotor" value="0.1" /> <!-- [m] -->
+  <xacro:property name="motor_constant" value="8.54858e-06" /> <!-- [kg·m/s^2] -->
   <xacro:property name="moment_constant" value="0.016" /> <!-- [m] -->
   <xacro:property name="time_constant" value="0.0125" /> <!-- [s] -->
@@ -17,12 +17,16 @@
   <xacro:property name="sin30" value="0.5" />
   <xacro:property name="cos30" value="0.866025403784" />
-  <xacro:property name="rotor_drag_coefficient" value="0.0001" />
+  <xacro:property name="rotor_drag_coefficient" value="8.06428e-05" />
   <xacro:property name="rolling_moment_coefficient" value="0.000001" />
   <!-- Property Blocks -->
   <xacro:property name="body_inertia">
-    <inertia ixx="0.0393" ixy="0.0" ixz="0.0" iyy="0.048" iyz="0.0" izz="0.0977" /> <!-- [kg·m^2] [kg·m^2] [kg·m^2] [kg·m^2] [kg·m^2] [kg·m^2] -->
+    <inertia ixx="0.0347563" ixy="0.0" ixz="0.0" iyy="0.0458929" iyz="0.0" izz="0.0977" /> <!-- [kg·m^2] [kg·m^2] [kg·m^2] [kg·m^2] [kg·m^2] [kg·m^2] -->
   </xacro:property>
   <xacro:property name="rotor_inertia">
-    <inertia ixx="0.0001" ixy="0.0" ixz="0.0" iyy="0.00001" iyz="0.0" izz="0.0000036" /> <!-- [kg·m^2] [kg·m^2] [kg·m^2] [kg·m^2] [kg·m^2] [kg·m^2] -->
+    <inertia
+    ixx="${1/12 * mass_rotor * (0.015 * 0.015 + 0.003 * 0.003) * rotor_velocity_slowdown_sim}"
+    iyy="${1/12 * mass_rotor * (4 * radius_rotor * radius_rotor + 0.003 * 0.003) * rotor_velocity_slowdown_sim}"
+    izz="${1/12 * mass_rotor * (4 * radius_rotor * radius_rotor + 0.015 * 0.015) * rotor_velocity_slowdown_sim}"
+    ixy="0.0" ixz="0.0"  iyz="0.0" /> <!-- [kg·m^2] [kg·m^2] [kg·m^2] [kg·m^2] [kg·m^2] [kg·m^2] -->
   </xacro:property>
   <!-- Included URDF Files -->

Commit message: Add 1st order system to rotor velocity. Fix the limit on velocity imposed by Gazebo.

File: mav_description/urdf/firefly.urdf.xacro (robot description, xacro)
@@ -2,5 +2,5 @@
 <robot name="firefly" xmlns:xacro="http://ros.org/wiki/xacro">
   <!-- Properties -->
-  <xacro:property name="rotor_velocity_slowdown_sim" value="10" />
+  <xacro:property name="rotor_velocity_slowdown_sim" value="1" />
   <xacro:property name="mesh_file" value="firefly.dae" />
   <xacro:property name="mass" value="1.5" /> <!-- [kg] -->
@@ -13,5 +13,6 @@
   <xacro:property name="motor_constant" value="8.54858e-06" /> <!-- [kg·m/s^2] -->
   <xacro:property name="moment_constant" value="0.016" /> <!-- [m] -->
-  <xacro:property name="time_constant" value="0.0125" /> <!-- [s] -->
+  <xacro:property name="time_constant_up" value="0.0125" /> <!-- [s] -->
+  <xacro:property name="time_constant_dwn" value="0.025" /> <!-- [s] -->
   <xacro:property name="max_rot_velocity" value="838" /> <!-- [rad/s] -->
   <xacro:property name="sin30" value="0.5" />
@@ -53,5 +54,6 @@
     mass_rotor="${mass_rotor}"
     radius_rotor="${radius_rotor}"
-    time_constant="${time_constant}"
+    time_constant_up="${time_constant_up}"
+    time_constant_dwn="${time_constant_dwn}"
     max_rot_velocity="${max_rot_velocity}"
     motor_number="0"
@@ -71,5 +73,6 @@
     mass_rotor="${mass_rotor}"
     radius_rotor="${radius_rotor}"
-    time_constant="${time_constant}"
+    time_constant_up="${time_constant_up}"
+    time_constant_dwn="${time_constant_dwn}"
     max_rot_velocity="${max_rot_velocity}"
     motor_number="1"
@@ -88,5 +91,6 @@
     mass_rotor="${mass_rotor}"
     radius_rotor="${radius_rotor}"
-    time_constant="${time_constant}"
+    time_constant_up="${time_constant_up}"
+    time_constant_dwn="${time_constant_dwn}"
     max_rot_velocity="${max_rot_velocity}"
     motor_number="2"
@@ -105,5 +109,6 @@
     mass_rotor="${mass_rotor}"
     radius_rotor="${radius_rotor}"
-    time_constant="${time_constant}"
+    time_constant_up="${time_constant_up}"
+    time_constant_dwn="${time_constant_dwn}"
     max_rot_velocity="${max_rot_velocity}"
     motor_number="3"
@@ -123,5 +128,6 @@
     mass_rotor="${mass_rotor}"
     radius_rotor="${radius_rotor}"
-    time_constant="${time_constant}"
+    time_constant_up="${time_constant_up}"
+    time_constant_dwn="${time_constant_dwn}"
     max_rot_velocity="${max_rot_velocity}"
     motor_number="4"
@@ -141,5 +147,6 @@
     mass_rotor="${mass_rotor}"
     radius_rotor="${radius_rotor}"
-    time_constant="${time_constant}"
+    time_constant_up="${time_constant_up}"
+    time_constant_dwn="${time_constant_dwn}"
     max_rot_velocity="${max_rot_velocity}"
     motor_number="5"

File: mav_description/urdf/multirotor_base.urdf.xacro (robot description, xacro)
@@ -125,5 +125,5 @@
   <!-- Rotor joint and link -->
   <xacro:macro name="vertical_rotor"
-    params="robot_namespace suffix direction motor_constant moment_constant parent mass_rotor radius_rotor time_constant max_rot_velocity motor_number rotor_drag_coefficient rolling_moment_coefficient color *origin *inertia">
+    params="robot_namespace suffix direction motor_constant moment_constant parent mass_rotor radius_rotor time_constant_up time_constant_dwn max_rot_velocity motor_number rotor_drag_coefficient rolling_moment_coefficient color *origin *inertia">
     <joint name="rotor_${motor_number}_joint" type="continuous">
       <xacro:insert_block name="origin" />
@@ -161,5 +161,6 @@
         <linkName>rotor_${motor_number}</linkName>
         <turningDirection>${direction}</turningDirection>
-        <timeConstant>${time_constant}</timeConstant>
+        <timeConstant_up>${time_constant_up}</timeConstant_up>
+        <timeConstant_dwn>${time_constant_dwn}</timeConstant_dwn>
         <maxRotVelocity>${max_rot_velocity}</maxRotVelocity>
         <motorConstant>${motor_constant}</motorConstant>

Commit message: 1st order system on rotors - running at 100 Hz.

File: mav_description/urdf/firefly.urdf.xacro (robot description, xacro)
@@ -2,5 +2,5 @@
 <robot name="firefly" xmlns:xacro="http://ros.org/wiki/xacro">
   <!-- Properties -->
-  <xacro:property name="rotor_velocity_slowdown_sim" value="1" />
+  <xacro:property name="rotor_velocity_slowdown_sim" value="10" />
   <xacro:property name="mesh_file" value="firefly.dae" />
   <xacro:property name="mass" value="1.5" /> <!-- [kg] -->
@@ -14,5 +14,5 @@
   <xacro:property name="moment_constant" value="0.016" /> <!-- [m] -->
   <xacro:property name="time_constant_up" value="0.0125" /> <!-- [s] -->
-  <xacro:property name="time_constant_dwn" value="0.025" /> <!-- [s] -->
+  <xacro:property name="time_constant_down" value="0.025" /> <!-- [s] -->
   <xacro:property name="max_rot_velocity" value="838" /> <!-- [rad/s] -->
   <xacro:property name="sin30" value="0.5" />
@@ -55,5 +55,5 @@
     radius_rotor="${radius_rotor}"
     time_constant_up="${time_constant_up}"
-    time_constant_dwn="${time_constant_dwn}"
+    time_constant_down="${time_constant_down}"
     max_rot_velocity="${max_rot_velocity}"
     motor_number="0"
@@ -74,5 +74,5 @@
     radius_rotor="${radius_rotor}"
     time_constant_up="${time_constant_up}"
-    time_constant_dwn="${time_constant_dwn}"
+    time_constant_down="${time_constant_down}"
     max_rot_velocity="${max_rot_velocity}"
     motor_number="1"
@@ -92,5 +92,5 @@
     radius_rotor="${radius_rotor}"
     time_constant_up="${time_constant_up}"
-    time_constant_dwn="${time_constant_dwn}"
+    time_constant_down="${time_constant_down}"
     max_rot_velocity="${max_rot_velocity}"
     motor_number="2"
@@ -110,5 +110,5 @@
     radius_rotor="${radius_rotor}"
     time_constant_up="${time_constant_up}"
-    time_constant_dwn="${time_constant_dwn}"
+    time_constant_down="${time_constant_down}"
     max_rot_velocity="${max_rot_velocity}"
     motor_number="3"
@@ -129,5 +129,5 @@
     radius_rotor="${radius_rotor}"
     time_constant_up="${time_constant_up}"
-    time_constant_dwn="${time_constant_dwn}"
+    time_constant_down="${time_constant_down}"
     max_rot_velocity="${max_rot_velocity}"
     motor_number="4"
@@ -148,5 +148,5 @@
     radius_rotor="${radius_rotor}"
     time_constant_up="${time_constant_up}"
-    time_constant_dwn="${time_constant_dwn}"
+    time_constant_down="${time_constant_down}"
     max_rot_velocity="${max_rot_velocity}"
     motor_number="5"

File: mav_description/urdf/multirotor_base.urdf.xacro (robot description, xacro)
@@ -125,5 +125,5 @@
   <!-- Rotor joint and link -->
   <xacro:macro name="vertical_rotor"
-    params="robot_namespace suffix direction motor_constant moment_constant parent mass_rotor radius_rotor time_constant_up time_constant_dwn max_rot_velocity motor_number rotor_drag_coefficient rolling_moment_coefficient color *origin *inertia">
+    params="robot_namespace suffix direction motor_constant moment_constant parent mass_rotor radius_rotor time_constant_up time_constant_down max_rot_velocity motor_number rotor_drag_coefficient rolling_moment_coefficient color *origin *inertia">
     <joint name="rotor_${motor_number}_joint" type="continuous">
       <xacro:insert_block name="origin" />
@@ -161,6 +161,6 @@
         <linkName>rotor_${motor_number}</linkName>
         <turningDirection>${direction}</turningDirection>
-        <timeConstant_up>${time_constant_up}</timeConstant_up>
-        <timeConstant_dwn>${time_constant_dwn}</timeConstant_dwn>
+        <timeConstantUp>${time_constant_up}</timeConstantUp>
+        <timeConstantDown>${time_constant_down}</timeConstantDown>
         <maxRotVelocity>${max_rot_velocity}</maxRotVelocity>
         <motorConstant>${motor_constant}</motorConstant>

Commit message: make base_link material and propeller mesh a parameter

File: mav_description/urdf/firefly.urdf.xacro (robot description, xacro)
@@ -4,4 +4,5 @@
   <xacro:property name="rotor_velocity_slowdown_sim" value="10" />
   <xacro:property name="mesh_file" value="firefly.dae" />
+  <xacro:property name="mesh_scale" value="1 1 1"/>
   <xacro:property name="mass" value="1.5" /> <!-- [kg] -->
   <xacro:property name="body_width" value="0.1" /> <!-- [m] -->
@@ -19,4 +20,5 @@
   <xacro:property name="rotor_drag_coefficient" value="8.06428e-05" />
   <xacro:property name="rolling_moment_coefficient" value="0.000001" />
+  <xacro:property name="color" value="White" />
   <!-- Property Blocks -->
   <xacro:property name="body_inertia">
@@ -40,4 +42,6 @@
     body_height="${body_height}"
     mesh_file="${mesh_file}"
+    mesh_scale="${mesh_scale}"
+    color="${color}"
     >
     <xacro:insert_block name="body_inertia" />
@@ -58,4 +62,5 @@
     rotor_drag_coefficient="${rotor_drag_coefficient}"
     rolling_moment_coefficient="${rolling_moment_coefficient}"
+    mesh="propeller"
     color="Red">
     <origin xyz="${cos30*arm_length} ${sin30*arm_length} ${rotor_offset_top}" rpy="0 0 0" />
@@ -76,4 +81,5 @@
     rotor_drag_coefficient="${rotor_drag_coefficient}"
     rolling_moment_coefficient="${rolling_moment_coefficient}"
+    mesh="propeller"
     color="Blue">
     <origin xyz="0 ${arm_length} ${rotor_offset_top}" rpy="0 0 0" />
@@ -93,4 +99,5 @@
     rotor_drag_coefficient="${rotor_drag_coefficient}"
     rolling_moment_coefficient="${rolling_moment_coefficient}"
+    mesh="propeller"
     color="Blue">
     <origin xyz="-${cos30*arm_length} ${sin30*arm_length} ${rotor_offset_top}" rpy="0 0 0" />
@@ -110,4 +117,5 @@
     rotor_drag_coefficient="${rotor_drag_coefficient}"
     rolling_moment_coefficient="${rolling_moment_coefficient}"
+    mesh="propeller"
     color="Blue">
     <origin xyz="-${cos30*arm_length} -${sin30*arm_length} ${rotor_offset_top}" rpy="0 0 0" />
@@ -128,4 +136,5 @@
     rotor_drag_coefficient="${rotor_drag_coefficient}"
     rolling_moment_coefficient="${rolling_moment_coefficient}"
+    mesh="propeller"
     color="Blue">
     <origin xyz="0 -${arm_length} ${rotor_offset_top}" rpy="0 0 0" />
@@ -146,4 +155,5 @@
     rotor_drag_coefficient="${rotor_drag_coefficient}"
     rolling_moment_coefficient="${rolling_moment_coefficient}"
+    mesh="propeller"
     color="Red">
     <origin xyz="${cos30*arm_length} -${sin30*arm_length} ${rotor_offset_top}" rpy="0 0 0" />

File: mav_description/urdf/multirotor_base.urdf.xacro (robot description, xacro)
@@ -3,6 +3,7 @@
   <!-- Main multirotor link -->
   <xacro:macro name="multirotor_base_macro"
-    params="robot_namespace mass body_width body_height mesh_file *inertia">
-    <link name="base_link"></link>
+    params="robot_namespace mass body_width body_height mesh_file mesh_scale color *inertia">
+    <link name="base_link">
+    </link>
     <joint name="base_joint" type="fixed">
       <origin xyz="0 0 0" rpy="0 0 0" />
@@ -20,5 +21,5 @@
         <geometry>
           <mesh filename="package://mav_description/meshes/${mesh_file}"
-            scale="1 1 1" />
+            scale="${mesh_scale}" />
           <!-- <box size="${body_width} ${body_width} ${body_height}"/> --> <!-- [m] [m] [m] -->
         </geometry>
@@ -54,4 +55,7 @@
         <rotorVelocitySlowdownSim>${rotor_velocity_slowdown_sim}</rotorVelocitySlowdownSim>
       </plugin>
+    </gazebo>
+    <gazebo reference="base_link">
+      <material>Gazebo/${color}</material>
     </gazebo>
   </xacro:macro>
@@ -125,5 +129,5 @@
   <!-- Rotor joint and link -->
   <xacro:macro name="vertical_rotor"
-    params="robot_namespace suffix direction motor_constant moment_constant parent mass_rotor radius_rotor time_constant max_rot_velocity motor_number rotor_drag_coefficient rolling_moment_coefficient color *origin *inertia">
+    params="robot_namespace suffix direction motor_constant moment_constant parent mass_rotor radius_rotor time_constant max_rot_velocity motor_number rotor_drag_coefficient rolling_moment_coefficient color mesh *origin *inertia">
     <joint name="rotor_${motor_number}_joint" type="continuous">
       <xacro:insert_block name="origin" />
@@ -145,5 +149,6 @@
         <geometry>
           <!-- <cylinder length="0.005" radius="${radius_rotor}"/> --> <!-- [m] -->
-          <mesh filename="package://mav_description/meshes/propeller_${direction}.dae"
+          <!-- <mesh filename="package://mav_description/meshes/propeller_${direction}.dae" -->
+          <mesh filename="package://mav_description/meshes/${mesh}_${direction}.dae"
             scale="0.001 0.001 0.001" />
           <!-- <box size="${2*radius_rotor} 0.01 0.005"/> -->

File: mav_description/urdf/pelican.urdf.xacro (robot description, xacro)
@@ -7,4 +7,5 @@
   <xacro:property name="namespace" value="pelican" />
   <xacro:property name="mesh_file" value="pelican.dae" />
+  <xacro:property name="mesh_scale" value="1 1 1"/>
   <xacro:property name="mass" value="0.6" /> <!-- [kg] -->
   <xacro:property name="body_width" value="0.1" /> <!-- [m] -->
@@ -20,4 +21,5 @@
   <xacro:property name="rotor_drag_coefficient" value="0.0001" />
   <xacro:property name="rolling_moment_coefficient" value="0.000001" />
+  <xacro:property name="color" value="White" />
   <!-- Property Blocks -->
   <xacro:property name="body_inertia">
@@ -36,4 +38,6 @@
     body_height="${body_height}"
     mesh_file="${mesh_file}"
+    mesh_scale="${mesh_scale}"
+    color="${color}"
     bag_file="pelican.bag"
     enable_bag_plugin="false">
@@ -54,4 +58,5 @@
     rotor_drag_coefficient="${rotor_drag_coefficient}"
     rolling_moment_coefficient="${rolling_moment_coefficient}"
+    mesh="propeller"
     color="Red">
     <origin xyz="${arm_length} 0 ${rotor_offset_top}" rpy="0 0 0" />
@@ -72,4 +77,5 @@
     rotor_drag_coefficient="${rotor_drag_coefficient}"
     rolling_moment_coefficient="${rolling_moment_coefficient}"
+    mesh="propeller"
     color="Blue">
     <origin xyz="0 ${arm_length} ${rotor_offset_top}" rpy="0 0 0" />
@@ -90,4 +96,5 @@
     rotor_drag_coefficient="${rotor_drag_coefficient}"
     rolling_moment_coefficient="${rolling_moment_coefficient}"
+    mesh="propeller"
     color="Blue">
     <origin xyz="-${arm_length} 0 ${rotor_offset_top}" rpy="0 0 0" />
@@ -108,4 +115,5 @@
     rotor_drag_coefficient="${rotor_drag_coefficient}"
     rolling_moment_coefficient="${rolling_moment_coefficient}"
+    mesh="propeller"
     color="Blue">
     <origin xyz="0 -${arm_length} ${rotor_offset_top}" rpy="0 0 0" />

File: mav_description/urdf/vtol.urdf.xacro (robot description, xacro)
@@ -4,4 +4,5 @@
   <xacro:property name="rotor_velocity_slowdown_sim" value="10" />
   <xacro:property name="mesh_file" value="firefly.dae" />
+  <xacro:property name="mesh_scale" value="1 1 1"/>
   <xacro:property name="mass" value="1.5" /> <!-- [kg] -->
   <xacro:property name="body_width" value="0.1" /> <!-- [m] -->
@@ -19,4 +20,5 @@
   <xacro:property name="rotor_drag_coefficient" value="8.06428e-05" />
   <xacro:property name="rolling_moment_coefficient" value="0.000001" />
+  <xacro:property name="color" value="White" />
   <!-- Property Blocks -->
   <xacro:property name="body_inertia">
@@ -41,4 +43,6 @@
     body_height="${body_height}"
     mesh_file="${mesh_file}"
+    mesh_scale="${mesh_scale}"
+    color="${color}"
     >
     <xacro:insert_block name="body_inertia" />
@@ -59,4 +63,5 @@
     rotor_drag_coefficient="${rotor_drag_coefficient}"
     rolling_moment_coefficient="${rolling_moment_coefficient}"
+    mesh="propeller"
     color="Red">
     <origin xyz="${arm_length} 0 ${rotor_offset_top}" rpy="0 0 0" />
@@ -77,4 +82,5 @@
     rotor_drag_coefficient="${rotor_drag_coefficient}"
     rolling_moment_coefficient="${rolling_moment_coefficient}"
+    mesh="propeller"
     color="Blue">
     <origin xyz="-${arm_length} 0 ${rotor_offset_top}" rpy="0 0 0" />
@@ -94,4 +100,5 @@
     rotor_drag_coefficient="${rotor_drag_coefficient}"
     rolling_moment_coefficient="${rolling_moment_coefficient}"
+    mesh="propeller"
     color="Blue">
     <origin xyz="0 ${arm_length} ${rotor_offset_top}" rpy="0 0 0" />
@@ -111,4 +118,5 @@
     rotor_drag_coefficient="${rotor_drag_coefficient}"
     rolling_moment_coefficient="${rolling_moment_coefficient}"
+    mesh="propeller"
     color="Blue">
     <origin xyz="0 -${arm_length} ${rotor_offset_top}" rpy="0 0 0" />
