Commit message: make spawning more than one static_camera possible, make them more static (still not really static)

File: mav_description/urdf/static_camera.gazebo.xacro (robot description, xacro)
@@ -1,5 +1,5 @@
 <?xml version="1.0"?>
 <robot name="static_camera" xmlns:xacro="http://ros.org/wiki/xacro">
-  <xacro:property name="namespace" value="observer" />
+  <xacro:property name="namespace" value="static_camera" />
   <xacro:property name="enable_bag_plugin" value="false" />
   <xacro:property name="bag_file" value="static_camera.bag" />

File: mav_description/urdf/static_camera.urdf.xacro (robot description, xacro)
@@ -5,7 +5,5 @@
   <xacro:property name="body_width" value="0.1" /> <!-- [m] -->
   <xacro:property name="body_height" value="0.16" /> <!-- [m] -->
-  <xacro:property name="rpy" value="0 -1.5707963267948966 0" />
-  <xacro:property name="pos" value="0 0 0" />
-  <xacro:property name="namespace" value="observer" />
+  <xacro:property name="namespace" value="static_camera" />
   <!-- Property Blocks -->
   <xacro:property name="body_inertia">
@@ -16,16 +14,16 @@
     params="robot_namespace mass body_width body_height *inertia">
     <link name="base_link">
-    </link>
-    <joint name="base_joint" type="fixed">
-      <origin xyz="0 0 0" rpy="0 0 0" />
-      <parent link="base_link" />
-      <child link="base_link_inertia" />
-    </joint>
-    <link name="base_link_inertia">
-      <inertial>
-        <mass value="${mass}" />  <!-- [kg] -->
-        <origin xyz="0 0 0" />
-        <xacro:insert_block name="inertia" />
-      </inertial>
+    <!-- </link> -->
+    <!-- <joint name="base_joint" type="fixed"> -->
+      <!-- <origin xyz="0 0 0" rpy="0 0 0" /> -->
+      <!-- <parent link="base_link" /> -->
+      <!-- <child link="base_link_inertia" /> -->
+    <!-- </joint> -->
+    <!-- <link name="base_link_inertia"> -->
+      <!-- <inertial> -->
+        <!-- <mass value="${mass}" />  [> [kg] <] -->
+        <!-- <origin xyz="0 0 0" /> -->
+        <!-- <xacro:insert_block name="inertia" /> -->
+      <!-- </inertial> -->
       <!-- <visual> -->
         <!-- <origin xyz="0 0 0" rpy="0 0 0" /> -->
@@ -43,4 +41,7 @@
       </collision>
     </link>
+    <gazebo reference="base_link">
+      <static>true</static>
+    </gazebo>
   </xacro:macro>
   <xacro:camera_base_macro
@@ -82,5 +83,4 @@
     </link>
     <gazebo reference="camera_link">
-      <static>true</static>
       <material>Gazebo/Red</material>
       <sensor type="camera" name="camera_static1">
@@ -118,4 +118,5 @@
         </plugin>
       </sensor>
+      <static>true</static>
     </gazebo>
   </xacro:macro>

Commit message: really make static cameras static

File: mav_description/urdf/static_camera.gazebo.xacro (robot description, xacro)
@@ -6,3 +6,6 @@
   <!-- Instantiate static_camera "mechanics" -->
   <xacro:include filename="$(find mav_description)/urdf/static_camera.urdf.xacro" />
+<gazebo>
+    <static>true</static>
+</gazebo>
 </robot>

File: mav_description/urdf/static_camera.urdf.xacro (robot description, xacro)
@@ -14,24 +14,4 @@
     params="robot_namespace mass body_width body_height *inertia">
     <link name="base_link">
-    <!-- </link> -->
-    <!-- <joint name="base_joint" type="fixed"> -->
-      <!-- <origin xyz="0 0 0" rpy="0 0 0" /> -->
-      <!-- <parent link="base_link" /> -->
-      <!-- <child link="base_link_inertia" /> -->
-    <!-- </joint> -->
-    <!-- <link name="base_link_inertia"> -->
-      <!-- <inertial> -->
-        <!-- <mass value="${mass}" />  [> [kg] <] -->
-        <!-- <origin xyz="0 0 0" /> -->
-        <!-- <xacro:insert_block name="inertia" /> -->
-      <!-- </inertial> -->
-      <!-- <visual> -->
-        <!-- <origin xyz="0 0 0" rpy="0 0 0" /> -->
-        <!-- <geometry> -->
-          <!-- <mesh filename="package://mav_description/meshes/${mesh_file}" -->
-            <!-- scale="${mesh_scale}" /> -->
-          <!-- [> <box size="${body_width} ${body_width} ${body_height}"/> [m] [m] [m] <] -->
-        <!-- </geometry> -->
-      <!-- </visual> -->
       <collision>
         <origin xyz="0 0 0" rpy="0 0 0" />
@@ -41,7 +21,4 @@
       </collision>
     </link>
-    <gazebo reference="base_link">
-      <static>true</static>
-    </gazebo>
   </xacro:macro>
   <xacro:camera_base_macro
@@ -118,5 +95,4 @@
         </plugin>
       </sensor>
-      <static>true</static>
     </gazebo>
   </xacro:macro>
