Commit message: mav_description: removed comments and added more params and its units
changes according to Simon and Michael A.:

removed useless comments as suggested by Simon
added units in comments in xacro files
renamed rotor to vertical_rotor
added more params for plugins

File: mav_description/urdf/multirotor_base.urdf.xacro (robot description, xacro)
@@ -5,5 +5,5 @@
     <link name="base_link">
       <inertial>
-        <mass value="${mass}" />
+        <mass value="${mass}" />  <!-- [kg] -->
         <origin xyz="0 0 0" />
         <xacro:insert_block name="inertia" />
@@ -12,5 +12,5 @@
         <origin xyz="0 0 0" rpy="0 0 0" />
         <geometry>
-          <box size="${body_width} ${body_width} ${body_height}"/>
+          <box size="${body_width} ${body_width} ${body_height}"/> <!-- [m] [m] [m] -->
         </geometry>
       </visual>
@@ -18,5 +18,5 @@
         <origin xyz="0 0 0" rpy="0 0 0" />
         <geometry>
-          <box size="${body_width} ${body_width} ${body_height}"/>
+          <box size="${body_width} ${body_width} ${body_height}"/> <!-- [m] [m] [m] -->
         </geometry>
       </collision>
@@ -24,5 +24,5 @@
   </xacro:macro>
   <!-- Rotor joint and link -->
-  <xacro:macro name="rotor" params="suffix parent mass_rotor radius_rotor *origin *inertia">
+  <xacro:macro name="vertical_rotor" params="suffix direction motor_constant moment_constant parent mass_rotor radius_rotor max_force *origin *inertia">
     <joint name="rotor_${suffix}_joint" type="continuous">
       <xacro:insert_block name="origin" />
@@ -33,15 +33,15 @@
     <link name="rotor_${suffix}">
       <inertial>
-        <mass value="${mass_rotor}" />
+        <mass value="${mass_rotor}" /> <!-- [kg] -->
         <xacro:insert_block name="inertia" />
       </inertial>
       <visual>
         <geometry>
-          <cylinder length="0.005" radius="${radius_rotor}"/>
+          <cylinder length="0.005" radius="${radius_rotor}"/> <!-- [m] -->
         </geometry>
       </visual>
       <collision>
         <geometry>
-          <cylinder length="0.005" radius="${radius_rotor}"/>
+          <cylinder length="0.005" radius="${radius_rotor}"/> <!-- [m] -->
         </geometry>
       </collision>

File: mav_description/urdf/pelican.urdf.xacro (robot description, xacro)
@@ -5,18 +5,19 @@
 >
   <!-- Properties -->
-  <xacro:property name="pi" value="3.1415926535897931" />
-  <xacro:property name="mass" value="1.477" />
-  <xacro:property name="body_width" value="0.1" />
-  <xacro:property name="body_height" value="0.2" />
-  <xacro:property name="mass_rotor" value="0.01" />
-  <xacro:property name="rotor_offset_side" value="0.15" />
-  <xacro:property name="rotor_offset_top" value="0.05" />
-  <xacro:property name="radius_rotor" value="0.08" />
+  <xacro:property name="mass" value="1.477" /> <!-- [kg] -->
+  <xacro:property name="body_width" value="0.1" /> <!-- [m] -->
+  <xacro:property name="body_height" value="0.2" /> <!-- [m] -->
+  <xacro:property name="mass_rotor" value="0.01" /> <!-- [kg] -->
+  <xacro:property name="arm_length" value="0.17" /> <!-- [m] -->
+  <xacro:property name="rotor_offset_top" value="0.05" /> <!-- [m] -->
+  <xacro:property name="radius_rotor" value="0.08" /> <!-- [m] -->
+  <xacro:property name="motor_constant" value="9.9865e-06" /> <!-- [kg·m/s^2] -->
+  <xacro:property name="moment_constant" value="0.016" /> <!-- [m] -->
   <!-- Property Blocks -->
   <xacro:property name="body_inertia">
-    <inertia ixx="0.01152" ixy="0.0" ixz="0.0" iyy="0.01152" iyz="0.0" izz="0.0218" />
+    <inertia ixx="0.01152" ixy="0.0" ixz="0.0" iyy="0.01152" iyz="0.0" izz="0.0218" /> <!-- [kg·m^2] [kg·m^2] [kg·m^2] [kg·m^2] [kg·m^2] [kg·m^2] -->
   </xacro:property>
   <xacro:property name="rotor_inertia">
-    <inertia ixx="0.01152" ixy="0.0" ixz="0.0" iyy="0.01152" iyz="0.0" izz="0.0218" />
+    <inertia ixx="0.01152" ixy="0.0" ixz="0.0" iyy="0.01152" iyz="0.0" izz="0.0218" /> <!-- [kg·m^2] [kg·m^2] [kg·m^2] [kg·m^2] [kg·m^2] [kg·m^2] -->
   </xacro:property>
   <!-- Included URDF Files -->
@@ -26,20 +27,20 @@
     <xacro:insert_block name="body_inertia" />
   </xacro:multirotor_base_macro>
-  <!-- Instantiate 4 rotors -->
-  <xacro:rotor suffix="front" parent="base_link" mass_rotor="${mass_rotor}" radius_rotor="${radius_rotor}">
-    <origin xyz="${rotor_offset_side} 0 ${rotor_offset_top}" rpy="0 0 0" />
+  <!-- Instantiate rotors -->
+  <xacro:vertical_rotor suffix="front" direction="ccw" motor_constant="${motor_constant}" moment_constant="${moment_constant}" parent="base_link" mass_rotor="${mass_rotor}" radius_rotor="${radius_rotor}" max_force="1">
+    <origin xyz="${arm_length} 0 ${rotor_offset_top}" rpy="0 0 0" />
     <xacro:insert_block name="rotor_inertia" />
-  </xacro:rotor>
-  <xacro:rotor suffix="left" parent="base_link" mass_rotor="${mass_rotor}" radius_rotor="${radius_rotor}">
-    <origin xyz="0 ${rotor_offset_side} ${rotor_offset_top}" rpy="0 0 0" />
+  </xacro:vertical_rotor>
+  <xacro:vertical_rotor suffix="left" direction="cw" motor_constant="${motor_constant}" moment_constant="${moment_constant}" parent="base_link" mass_rotor="${mass_rotor}" radius_rotor="${radius_rotor}" max_force="1">
+    <origin xyz="0 ${arm_length} ${rotor_offset_top}" rpy="0 0 0" />
     <xacro:insert_block name="rotor_inertia" />
-  </xacro:rotor>
-  <xacro:rotor suffix="back" parent="base_link" mass_rotor="${mass_rotor}" radius_rotor="${radius_rotor}">
-    <origin xyz="-${rotor_offset_side} 0 ${rotor_offset_top}" rpy="0 0 0" />
+  </xacro:vertical_rotor>
+  <xacro:vertical_rotor suffix="back" direction="ccw" motor_constant="${motor_constant}" moment_constant="${moment_constant}" parent="base_link" mass_rotor="${mass_rotor}" radius_rotor="${radius_rotor}" max_force="1">
+    <origin xyz="-${arm_length} 0 ${rotor_offset_top}" rpy="0 0 0" />
     <xacro:insert_block name="rotor_inertia" />
-  </xacro:rotor>
-  <xacro:rotor suffix="right" parent="base_link" mass_rotor="${mass_rotor}" radius_rotor="${radius_rotor}">
-    <origin xyz="0 -${rotor_offset_side} ${rotor_offset_top}" rpy="0 0 0" />
+  </xacro:vertical_rotor>
+  <xacro:vertical_rotor suffix="right" direction="cw" motor_constant="${motor_constant}" moment_constant="${moment_constant}" parent="base_link" mass_rotor="${mass_rotor}" radius_rotor="${radius_rotor}" max_force="1">
+    <origin xyz="0 -${arm_length} ${rotor_offset_top}" rpy="0 0 0" />
     <xacro:insert_block name="rotor_inertia" />
-  </xacro:rotor>
+  </xacro:vertical_rotor>
 </robot>

Commit message: mav_gazebo_plugins: added topic names to the plugin
From here on there is only one topic where reference motor velocities
are published on and each motor has to name a motor number to which he
is assigned to.

File: mav_description/urdf/multirotor_base.urdf.xacro (robot description, xacro)
@@ -25,9 +25,13 @@
       <plugin name="controller_interface"
         filename="libmav_gazebo_controller_interface.so">
+        <commandTopic>mav_cmd</commandTopic>
+        <imuTopic>imu</imuTopic>
+        <poseTopic>pose</poseTopic>
+        <motorVelocityReferenceTopic>motor_vel_ref</motorVelocityReferenceTopic>
       </plugin>
     </gazebo>
   </xacro:macro>
   <!-- Rotor joint and link -->
-  <xacro:macro name="vertical_rotor" params="suffix direction motor_constant moment_constant parent mass_rotor radius_rotor max_force *origin *inertia">
+  <xacro:macro name="vertical_rotor" params="suffix direction motor_constant moment_constant parent mass_rotor radius_rotor max_force motor_number *origin *inertia">
     <joint name="rotor_${suffix}_joint" type="continuous">
       <xacro:insert_block name="origin" />
@@ -60,5 +64,6 @@
         <motorConstant>${motor_constant}</motorConstant>
         <momentConstant>${moment_constant}</momentConstant>
-        <commandTopic>cmd_${suffix}_motor_vel</commandTopic>
+        <commandTopic>motor_vel_ref</commandTopic>
+        <motorNumber>${motor_number}</motorNumber>
         <motorVelocityTopic>${suffix}_motor_vel</motorVelocityTopic>
       </plugin>

File: mav_description/urdf/pelican.urdf.xacro (robot description, xacro)
@@ -28,17 +28,17 @@
   </xacro:multirotor_base_macro>
   <!-- Instantiate rotors -->
-  <xacro:vertical_rotor suffix="front" direction="ccw" motor_constant="${motor_constant}" moment_constant="${moment_constant}" parent="base_link" mass_rotor="${mass_rotor}" radius_rotor="${radius_rotor}" max_force="1">
+  <xacro:vertical_rotor suffix="front" direction="ccw" motor_constant="${motor_constant}" moment_constant="${moment_constant}" parent="base_link" mass_rotor="${mass_rotor}" radius_rotor="${radius_rotor}" max_force="1" motor_number="0">
     <origin xyz="${arm_length} 0 ${rotor_offset_top}" rpy="0 0 0" />
     <xacro:insert_block name="rotor_inertia" />
   </xacro:vertical_rotor>
-  <xacro:vertical_rotor suffix="left" direction="cw" motor_constant="${motor_constant}" moment_constant="${moment_constant}" parent="base_link" mass_rotor="${mass_rotor}" radius_rotor="${radius_rotor}" max_force="1">
+  <xacro:vertical_rotor suffix="left" direction="cw" motor_constant="${motor_constant}" moment_constant="${moment_constant}" parent="base_link" mass_rotor="${mass_rotor}" radius_rotor="${radius_rotor}" max_force="1" motor_number="1">
     <origin xyz="0 ${arm_length} ${rotor_offset_top}" rpy="0 0 0" />
     <xacro:insert_block name="rotor_inertia" />
   </xacro:vertical_rotor>
-  <xacro:vertical_rotor suffix="back" direction="ccw" motor_constant="${motor_constant}" moment_constant="${moment_constant}" parent="base_link" mass_rotor="${mass_rotor}" radius_rotor="${radius_rotor}" max_force="1">
+  <xacro:vertical_rotor suffix="back" direction="ccw" motor_constant="${motor_constant}" moment_constant="${moment_constant}" parent="base_link" mass_rotor="${mass_rotor}" radius_rotor="${radius_rotor}" max_force="1" motor_number="2">
     <origin xyz="-${arm_length} 0 ${rotor_offset_top}" rpy="0 0 0" />
     <xacro:insert_block name="rotor_inertia" />
   </xacro:vertical_rotor>
-  <xacro:vertical_rotor suffix="right" direction="cw" motor_constant="${motor_constant}" moment_constant="${moment_constant}" parent="base_link" mass_rotor="${mass_rotor}" radius_rotor="${radius_rotor}" max_force="1">
+  <xacro:vertical_rotor suffix="right" direction="cw" motor_constant="${motor_constant}" moment_constant="${moment_constant}" parent="base_link" mass_rotor="${mass_rotor}" radius_rotor="${radius_rotor}" max_force="1" motor_number="3">
     <origin xyz="0 -${arm_length} ${rotor_offset_top}" rpy="0 0 0" />
     <xacro:insert_block name="rotor_inertia" />

Commit message: motor_model: updated with time_constant and max_rot_velocity
The joint friction is not yet implemented since it's not implemented in
gazebo at all, we should either do it ourselves or just use our own
model for the motors then.

File: mav_description/urdf/multirotor_base.urdf.xacro (robot description, xacro)
@@ -24,5 +24,5 @@
   </xacro:macro>
   <!-- Rotor joint and link -->
-  <xacro:macro name="vertical_rotor" params="suffix direction motor_constant moment_constant parent mass_rotor radius_rotor max_force *origin *inertia">
+  <xacro:macro name="vertical_rotor" params="suffix direction motor_constant moment_constant parent mass_rotor radius_rotor time_constant max_rot_velocity *origin *inertia">
     <joint name="rotor_${suffix}_joint" type="continuous">
       <xacro:insert_block name="origin" />
@@ -52,5 +52,6 @@
         <linkName>rotor_${suffix}</linkName>
         <turningDirection>${direction}</turningDirection>
-        <maxForce>${max_force}</maxForce>
+        <timeConstant>${time_constant}</timeConstant>
+        <maxRotVelocity>${max_rot_velocity}</maxRotVelocity>
         <motorConstant>${motor_constant}</motorConstant>
         <momentConstant>${moment_constant}</momentConstant>

File: mav_description/urdf/pelican.urdf.xacro (robot description, xacro)
@@ -28,17 +28,17 @@
   </xacro:multirotor_base_macro>
   <!-- Instantiate rotors -->
-  <xacro:vertical_rotor suffix="front" direction="ccw" motor_constant="${motor_constant}" moment_constant="${moment_constant}" parent="base_link" mass_rotor="${mass_rotor}" radius_rotor="${radius_rotor}" max_force="1">
+  <xacro:vertical_rotor suffix="front" direction="ccw" motor_constant="${motor_constant}" moment_constant="${moment_constant}" parent="base_link" mass_rotor="${mass_rotor}" radius_rotor="${radius_rotor}" time_constant="0.0125" max_rot_velocity="838">
     <origin xyz="${arm_length} 0 ${rotor_offset_top}" rpy="0 0 0" />
     <xacro:insert_block name="rotor_inertia" />
   </xacro:vertical_rotor>
-  <xacro:vertical_rotor suffix="left" direction="cw" motor_constant="${motor_constant}" moment_constant="${moment_constant}" parent="base_link" mass_rotor="${mass_rotor}" radius_rotor="${radius_rotor}" max_force="1">
+  <xacro:vertical_rotor suffix="left" direction="cw" motor_constant="${motor_constant}" moment_constant="${moment_constant}" parent="base_link" mass_rotor="${mass_rotor}" radius_rotor="${radius_rotor}" time_constant="0.0125" max_rot_velocity="838">
     <origin xyz="0 ${arm_length} ${rotor_offset_top}" rpy="0 0 0" />
     <xacro:insert_block name="rotor_inertia" />
   </xacro:vertical_rotor>
-  <xacro:vertical_rotor suffix="back" direction="ccw" motor_constant="${motor_constant}" moment_constant="${moment_constant}" parent="base_link" mass_rotor="${mass_rotor}" radius_rotor="${radius_rotor}" max_force="1">
+  <xacro:vertical_rotor suffix="back" direction="ccw" motor_constant="${motor_constant}" moment_constant="${moment_constant}" parent="base_link" mass_rotor="${mass_rotor}" radius_rotor="${radius_rotor}" time_constant="0.0125" max_rot_velocity="838">
     <origin xyz="-${arm_length} 0 ${rotor_offset_top}" rpy="0 0 0" />
     <xacro:insert_block name="rotor_inertia" />
   </xacro:vertical_rotor>
-  <xacro:vertical_rotor suffix="right" direction="cw" motor_constant="${motor_constant}" moment_constant="${moment_constant}" parent="base_link" mass_rotor="${mass_rotor}" radius_rotor="${radius_rotor}" max_force="1">
+  <xacro:vertical_rotor suffix="right" direction="cw" motor_constant="${motor_constant}" moment_constant="${moment_constant}" parent="base_link" mass_rotor="${mass_rotor}" radius_rotor="${radius_rotor}" time_constant="0.0125" max_rot_velocity="838">
     <origin xyz="0 -${arm_length} ${rotor_offset_top}" rpy="0 0 0" />
     <xacro:insert_block name="rotor_inertia" />

Commit message: mav_description: placed imu on pelican and added a robot namespace

File: mav_description/urdf/multirotor_base.urdf.xacro (robot description, xacro)
@@ -2,5 +2,5 @@
 <robot xmlns:xacro="http://ros.org/wiki/xacro">
   <!-- Main multirotor link -->
-  <xacro:macro name="multirotor_base_macro" params="mass body_width body_height *inertia">
+  <xacro:macro name="multirotor_base_macro" params="robot_namespace mass body_width body_height *inertia">
     <link name="base_link">
       <inertial>
@@ -25,8 +25,14 @@
       <plugin name="controller_interface"
         filename="libmav_gazebo_controller_interface.so">
+        <robotNamespace>${robot_namespace}</robotNamespace>
         <commandTopic>mav_cmd</commandTopic>
         <imuTopic>imu</imuTopic>
         <poseTopic>pose</poseTopic>
         <motorVelocityReferenceTopic>motor_vel_ref</motorVelocityReferenceTopic>
+      </plugin>
+      <plugin filename="libgazebo_ros_imu.so" name="imu_ros">
+        <bodyName>base_link</bodyName>
+        <robotNamespace>${robot_namespace}</robotNamespace>
+        <topicName>imu</topicName>
       </plugin>
     </gazebo>

File: mav_description/urdf/pelican.urdf.xacro (robot description, xacro)
@@ -5,4 +5,5 @@
 >
   <!-- Properties -->
+  <xacro:property name="namespace" value="pelican" />
   <xacro:property name="mass" value="1.477" /> <!-- [kg] -->
   <xacro:property name="body_width" value="0.1" /> <!-- [m] -->
@@ -24,5 +25,5 @@
   <xacro:include filename="$(find mav_description)/urdf/multirotor_base.urdf.xacro" />
   <!-- Instantiate multirotor_base_macro once -->
-  <xacro:multirotor_base_macro mass="${mass}" body_width="${body_width}" body_height="${body_height}">
+  <xacro:multirotor_base_macro robot_namespace="${namespace}" mass="${mass}" body_width="${body_width}" body_height="${body_height}">
     <xacro:insert_block name="body_inertia" />
   </xacro:multirotor_base_macro>

Commit message: mav_control: changed to mav_msgs/MotorSpeed and made everything work
Currently there is a hack for a limit joint velocity, which we can not
set, I will either fix this in gazebo or let them fix this. Please try
to fly if you want :).

File: mav_description/urdf/multirotor_base.urdf.xacro (robot description, xacro)
@@ -43,7 +43,20 @@
       <xacro:insert_block name="origin" />
       <axis xyz="0 0 1" />
+      <!-- TODO(ff): not currently set -->
+      <!-- <limit effort="2000" velocity="${max_rot_velocity}" /> -->
       <parent link="${parent}"/>
       <child link="rotor_${suffix}"/>
     </joint>
+    <!-- TODO(ff): not currently set -->
+    <!-- <gazebo reference="rotor_${suffix}_joint">
+      <axis>
+        <xyz>0 0 1</xyz>
+        <limit>
+          <velocity>
+            ${max_rot_velocity}
+          </velocity>
+        </limit>
+      </axis>
+    </gazebo> -->
     <link name="rotor_${suffix}">
       <inertial>
@@ -71,5 +84,5 @@
         <motorConstant>${motor_constant}</motorConstant>
         <momentConstant>${moment_constant}</momentConstant>
-        <commandTopic>motor_vel_ref</commandTopic>
+        <commandTopic>pelican/motor_vel_ref</commandTopic>
         <motorNumber>${motor_number}</motorNumber>
         <motorVelocityTopic>${suffix}_motor_vel</motorVelocityTopic>

File: mav_description/urdf/pelican.urdf.xacro (robot description, xacro)
@@ -6,5 +6,5 @@
   <!-- Properties -->
   <xacro:property name="namespace" value="pelican" />
-  <xacro:property name="mass" value="1.477" /> <!-- [kg] -->
+  <xacro:property name="mass" value="0.6" /> <!-- [kg] -->
   <xacro:property name="body_width" value="0.1" /> <!-- [m] -->
   <xacro:property name="body_height" value="0.2" /> <!-- [m] -->
@@ -19,8 +19,8 @@
   <!-- Property Blocks -->
   <xacro:property name="body_inertia">
-    <inertia ixx="0.01152" ixy="0.0" ixz="0.0" iyy="0.01152" iyz="0.0" izz="0.0218" /> <!-- [kg·m^2] [kg·m^2] [kg·m^2] [kg·m^2] [kg·m^2] [kg·m^2] -->
+    <inertia ixx="0.0056" ixy="0.0" ixz="0.0" iyy="0.0056" iyz="0.0" izz="0.0056" /> <!-- [kg·m^2] [kg·m^2] [kg·m^2] [kg·m^2] [kg·m^2] [kg·m^2] -->
   </xacro:property>
   <xacro:property name="rotor_inertia">
-    <inertia ixx="0.01152" ixy="0.0" ixz="0.0" iyy="0.01152" iyz="0.0" izz="0.0218" /> <!-- [kg·m^2] [kg·m^2] [kg·m^2] [kg·m^2] [kg·m^2] [kg·m^2] -->
+    <inertia ixx="0.0001" ixy="0.0" ixz="0.0" iyy="0.00001" iyz="0.0" izz="0.0000036" /> <!-- [kg·m^2] [kg·m^2] [kg·m^2] [kg·m^2] [kg·m^2] [kg·m^2] -->
   </xacro:property>
   <!-- Included URDF Files -->
@@ -31,17 +31,17 @@
   </xacro:multirotor_base_macro>
   <!-- Instantiate rotors -->
-  <xacro:vertical_rotor suffix="front" direction="ccw" motor_constant="${motor_constant}" moment_constant="${moment_constant}" parent="base_link" mass_rotor="${mass_rotor}" radius_rotor="${radius_rotor}" time_constant="${time_constant}" max_rot_velocity="${max_rot_velocity}" motor_number="0">
+  <xacro:vertical_rotor suffix="front" direction="cw" motor_constant="${motor_constant}" moment_constant="${moment_constant}" parent="base_link" mass_rotor="${mass_rotor}" radius_rotor="${radius_rotor}" time_constant="${time_constant}" max_rot_velocity="${max_rot_velocity}" motor_number="0">
     <origin xyz="${arm_length} 0 ${rotor_offset_top}" rpy="0 0 0" />
     <xacro:insert_block name="rotor_inertia" />
   </xacro:vertical_rotor>
-  <xacro:vertical_rotor suffix="left" direction="cw" motor_constant="${motor_constant}" moment_constant="${moment_constant}" parent="base_link" mass_rotor="${mass_rotor}" radius_rotor="${radius_rotor}" time_constant="${time_constant}" max_rot_velocity="${max_rot_velocity}" motor_number="1">
+  <xacro:vertical_rotor suffix="left" direction="ccw" motor_constant="${motor_constant}" moment_constant="${moment_constant}" parent="base_link" mass_rotor="${mass_rotor}" radius_rotor="${radius_rotor}" time_constant="${time_constant}" max_rot_velocity="${max_rot_velocity}" motor_number="3">
     <origin xyz="0 ${arm_length} ${rotor_offset_top}" rpy="0 0 0" />
     <xacro:insert_block name="rotor_inertia" />
   </xacro:vertical_rotor>
-  <xacro:vertical_rotor suffix="back" direction="ccw" motor_constant="${motor_constant}" moment_constant="${moment_constant}" parent="base_link" mass_rotor="${mass_rotor}" radius_rotor="${radius_rotor}" time_constant="${time_constant}" max_rot_velocity="${max_rot_velocity}" motor_number="2">
+  <xacro:vertical_rotor suffix="back" direction="cw" motor_constant="${motor_constant}" moment_constant="${moment_constant}" parent="base_link" mass_rotor="${mass_rotor}" radius_rotor="${radius_rotor}" time_constant="${time_constant}" max_rot_velocity="${max_rot_velocity}" motor_number="2">
     <origin xyz="-${arm_length} 0 ${rotor_offset_top}" rpy="0 0 0" />
     <xacro:insert_block name="rotor_inertia" />
   </xacro:vertical_rotor>
-  <xacro:vertical_rotor suffix="right" direction="cw" motor_constant="${motor_constant}" moment_constant="${moment_constant}" parent="base_link" mass_rotor="${mass_rotor}" radius_rotor="${radius_rotor}" time_constant="${time_constant}" max_rot_velocity="${max_rot_velocity}" motor_number="3">
+  <xacro:vertical_rotor suffix="right" direction="ccw" motor_constant="${motor_constant}" moment_constant="${moment_constant}" parent="base_link" mass_rotor="${mass_rotor}" radius_rotor="${radius_rotor}" time_constant="${time_constant}" max_rot_velocity="${max_rot_velocity}" motor_number="1">
     <origin xyz="0 -${arm_length} ${rotor_offset_top}" rpy="0 0 0" />
     <xacro:insert_block name="rotor_inertia" />
