Commit message: removed unneccessary comment in controller and fixed namespaces for launchfiles

File: mav_description/urdf/multirotor_base.urdf.xacro (robot description, xacro)
@@ -39,14 +39,14 @@
   </xacro:macro>
   <!-- Rotor joint and link -->
-  <xacro:macro name="vertical_rotor" params="suffix direction motor_constant moment_constant parent mass_rotor radius_rotor time_constant max_rot_velocity motor_number *origin *inertia">
+  <xacro:macro name="vertical_rotor" params="robot_namespace suffix direction motor_constant moment_constant parent mass_rotor radius_rotor time_constant max_rot_velocity motor_number *origin *inertia">
     <joint name="rotor_${suffix}_joint" type="continuous">
       <xacro:insert_block name="origin" />
       <axis xyz="0 0 1" />
-      <!-- TODO(ff): not currently set -->
+      <!-- TODO(ff): not currently set because it's not yet supported -->
       <!-- <limit effort="2000" velocity="${max_rot_velocity}" /> -->
       <parent link="${parent}"/>
       <child link="rotor_${suffix}"/>
     </joint>
-    <!-- TODO(ff): not currently set -->
+    <!-- TODO(ff): not currently set because it's not yet supported -->
     <!-- <gazebo reference="rotor_${suffix}_joint">
       <axis>
@@ -84,7 +84,7 @@
         <motorConstant>${motor_constant}</motorConstant>
         <momentConstant>${moment_constant}</momentConstant>
-        <commandTopic>pelican/motor_vel_ref</commandTopic>
+        <commandTopic>${robot_namespace}/motor_vel_ref</commandTopic>
         <motorNumber>${motor_number}</motorNumber>
-        <motorVelocityTopic>${suffix}_motor_vel</motorVelocityTopic>
+        <motorVelocityTopic>${robot_namespace}/${suffix}_motor_vel</motorVelocityTopic>
       </plugin>
     </gazebo>

File: mav_description/urdf/pelican.urdf.xacro (robot description, xacro)
@@ -31,17 +31,17 @@
   </xacro:multirotor_base_macro>
   <!-- Instantiate rotors -->
-  <xacro:vertical_rotor suffix="front" direction="cw" motor_constant="${motor_constant}" moment_constant="${moment_constant}" parent="base_link" mass_rotor="${mass_rotor}" radius_rotor="${radius_rotor}" time_constant="${time_constant}" max_rot_velocity="${max_rot_velocity}" motor_number="0">
+  <xacro:vertical_rotor robot_namespace="${namespace}" suffix="front" direction="cw" motor_constant="${motor_constant}" moment_constant="${moment_constant}" parent="base_link" mass_rotor="${mass_rotor}" radius_rotor="${radius_rotor}" time_constant="${time_constant}" max_rot_velocity="${max_rot_velocity}" motor_number="0">
     <origin xyz="${arm_length} 0 ${rotor_offset_top}" rpy="0 0 0" />
     <xacro:insert_block name="rotor_inertia" />
   </xacro:vertical_rotor>
-  <xacro:vertical_rotor suffix="left" direction="ccw" motor_constant="${motor_constant}" moment_constant="${moment_constant}" parent="base_link" mass_rotor="${mass_rotor}" radius_rotor="${radius_rotor}" time_constant="${time_constant}" max_rot_velocity="${max_rot_velocity}" motor_number="3">
+  <xacro:vertical_rotor robot_namespace="${namespace}" suffix="left" direction="ccw" motor_constant="${motor_constant}" moment_constant="${moment_constant}" parent="base_link" mass_rotor="${mass_rotor}" radius_rotor="${radius_rotor}" time_constant="${time_constant}" max_rot_velocity="${max_rot_velocity}" motor_number="3">
     <origin xyz="0 ${arm_length} ${rotor_offset_top}" rpy="0 0 0" />
     <xacro:insert_block name="rotor_inertia" />
   </xacro:vertical_rotor>
-  <xacro:vertical_rotor suffix="back" direction="cw" motor_constant="${motor_constant}" moment_constant="${moment_constant}" parent="base_link" mass_rotor="${mass_rotor}" radius_rotor="${radius_rotor}" time_constant="${time_constant}" max_rot_velocity="${max_rot_velocity}" motor_number="2">
+  <xacro:vertical_rotor robot_namespace="${namespace}" suffix="back" direction="cw" motor_constant="${motor_constant}" moment_constant="${moment_constant}" parent="base_link" mass_rotor="${mass_rotor}" radius_rotor="${radius_rotor}" time_constant="${time_constant}" max_rot_velocity="${max_rot_velocity}" motor_number="2">
     <origin xyz="-${arm_length} 0 ${rotor_offset_top}" rpy="0 0 0" />
     <xacro:insert_block name="rotor_inertia" />
   </xacro:vertical_rotor>
-  <xacro:vertical_rotor suffix="right" direction="ccw" motor_constant="${motor_constant}" moment_constant="${moment_constant}" parent="base_link" mass_rotor="${mass_rotor}" radius_rotor="${radius_rotor}" time_constant="${time_constant}" max_rot_velocity="${max_rot_velocity}" motor_number="1">
+  <xacro:vertical_rotor robot_namespace="${namespace}" suffix="right" direction="ccw" motor_constant="${motor_constant}" moment_constant="${moment_constant}" parent="base_link" mass_rotor="${mass_rotor}" radius_rotor="${radius_rotor}" time_constant="${time_constant}" max_rot_velocity="${max_rot_velocity}" motor_number="1">
     <origin xyz="0 -${arm_length} ${rotor_offset_top}" rpy="0 0 0" />
     <xacro:insert_block name="rotor_inertia" />

Commit message: controller is working while not rotating around the z-axis
To get the pose I created a gazebo_pose_publisher which calls the gazebo
service GetModelState to get the current pose of the helicopter and
publishes it over publish_topic.

File: mav_description/urdf/multirotor_base.urdf.xacro (robot description, xacro)
@@ -22,5 +22,20 @@
       </collision>
     </link>
+    <!-- IMU -->
+    <link name="imu_link">
+      <inertial>
+        <inertia ixx="0.001" ixy="0.0" ixz="0.0" iyy="0.001" iyz="0.0" izz="0.001" />
+        <mass value="0.01" />  <!-- [kg] -->
+        <origin xyz="0 0 0" rpy="0 0 0"/>
+      </inertial>
+    </link>
+    <!-- IMU joint -->
+    <joint name="imu_joint" type="fixed">
+      <origin xyz="0 0 0" rpy="3.1416 0 0" />
+      <parent link="base_link"/>
+      <child link="imu_link"/>
+    </joint>
     <gazebo>
+      <!-- Controller interface -->
       <plugin name="controller_interface"
         filename="libmav_gazebo_controller_interface.so">
@@ -31,13 +46,83 @@
         <motorVelocityReferenceTopic>motor_vel_ref</motorVelocityReferenceTopic>
       </plugin>
-      <plugin filename="libgazebo_ros_imu.so" name="imu_ros">
+      <!-- IMU -->
+      <plugin filename="libhector_gazebo_ros_imu.so" name="imu_ros">
         <bodyName>base_link</bodyName>
         <robotNamespace>${robot_namespace}</robotNamespace>
         <topicName>imu</topicName>
+        <updateRate>100.0</updateRate>
+        <gaussianNoise>0.0</gaussianNoise>
       </plugin>
     </gazebo>
   </xacro:macro>
+  <!-- camera -->
+  <xacro:macro name="camera_macro" params="robot_namespace">
+    <!-- joint -->
+    <joint name="camera_joint" type="fixed">
+      <axis xyz="0 1 0" />
+      <origin xyz="0 0 0.2" rpy="0 0 0"/>
+      <parent link="base_link"/>
+      <child link="camera_link"/>
+    </joint>
+    <!-- link -->
+    <link name="camera_link">
+      <collision>
+        <origin xyz="0 0 0" rpy="0 0 0"/>
+        <geometry>
+      <box size="0.1 0.1 0.1"/>
+        </geometry>
+      </collision>
+      <visual>
+        <origin xyz="0 0 0" rpy="0 0 0"/>
+        <geometry>
+      <box size="0.1 0.1 0.1"/>
+        </geometry>
+        <material name="red"/>
+      </visual>
+      <inertial>
+        <mass value="1e-5" />
+        <origin xyz="0 0 0" rpy="0 0 0"/>
+        <inertia ixx="1e-6" ixy="0" ixz="0" iyy="1e-6" iyz="0" izz="1e-6" />
+      </inertial>
+    </link>
+    <gazebo reference="camera_link">
+      <sensor type="camera" name="camera1">
+        <update_rate>30.0</update_rate>
+        <camera name="head">
+          <horizontal_fov>2</horizontal_fov>
+          <image>
+            <width>800</width>
+            <height>600</height>
+            <format>R8G8B8</format>
+          </image>
+          <clip>
+            <near>0.02</near>
+            <far>300</far>
+          </clip>
+          <noise>
+            <type>gaussian</type>
+            <mean>0.0</mean>
+            <stddev>0.007</stddev>
+          </noise>
+        </camera>
+        <plugin name="camera_controller" filename="libgazebo_ros_camera.so">
+          <alwaysOn>true</alwaysOn>
+          <updateRate>0.0</updateRate>
+          <cameraName>${robot_namespace}/camera1</cameraName>
+          <imageTopicName>image_raw</imageTopicName>
+          <cameraInfoTopicName>camera_info</cameraInfoTopicName>
+          <frameName>camera_link</frameName>
+          <hackBaseline>0.07</hackBaseline>
+          <distortionK1>-0.2</distortionK1>
+          <distortionK2>0.0</distortionK2>
+          <distortionK3>0.0</distortionK3>
+          <distortionT1>0.0</distortionT1>
+          <distortionT2>0.0</distortionT2>
+        </plugin>
+      </sensor>
+    </gazebo>
+  </xacro:macro>
   <!-- Rotor joint and link -->
-  <xacro:macro name="vertical_rotor" params="robot_namespace suffix direction motor_constant moment_constant parent mass_rotor radius_rotor time_constant max_rot_velocity motor_number *origin *inertia">
+  <xacro:macro name="vertical_rotor" params="robot_namespace suffix direction motor_constant moment_constant parent mass_rotor radius_rotor time_constant max_rot_velocity motor_number color *origin *inertia">
     <joint name="rotor_${suffix}_joint" type="continuous">
       <xacro:insert_block name="origin" />
@@ -89,4 +174,7 @@
       </plugin>
     </gazebo>
+    <gazebo reference="rotor_${suffix}">
+      <material>Gazebo/${color}</material>
+    </gazebo>
   </xacro:macro>
 </robot>

File: mav_description/urdf/pelican.urdf.xacro (robot description, xacro)
@@ -31,19 +31,21 @@
   </xacro:multirotor_base_macro>
   <!-- Instantiate rotors -->
-  <xacro:vertical_rotor robot_namespace="${namespace}" suffix="front" direction="cw" motor_constant="${motor_constant}" moment_constant="${moment_constant}" parent="base_link" mass_rotor="${mass_rotor}" radius_rotor="${radius_rotor}" time_constant="${time_constant}" max_rot_velocity="${max_rot_velocity}" motor_number="0">
+  <xacro:vertical_rotor robot_namespace="${namespace}" suffix="front" direction="cw" motor_constant="${motor_constant}" moment_constant="${moment_constant}" parent="base_link" mass_rotor="${mass_rotor}" radius_rotor="${radius_rotor}" time_constant="${time_constant}" max_rot_velocity="${max_rot_velocity}" motor_number="0" color="Red">
     <origin xyz="${arm_length} 0 ${rotor_offset_top}" rpy="0 0 0" />
     <xacro:insert_block name="rotor_inertia" />
   </xacro:vertical_rotor>
-  <xacro:vertical_rotor robot_namespace="${namespace}" suffix="left" direction="ccw" motor_constant="${motor_constant}" moment_constant="${moment_constant}" parent="base_link" mass_rotor="${mass_rotor}" radius_rotor="${radius_rotor}" time_constant="${time_constant}" max_rot_velocity="${max_rot_velocity}" motor_number="3">
+  <xacro:vertical_rotor robot_namespace="${namespace}" suffix="left" direction="ccw" motor_constant="${motor_constant}" moment_constant="${moment_constant}" parent="base_link" mass_rotor="${mass_rotor}" radius_rotor="${radius_rotor}" time_constant="${time_constant}" max_rot_velocity="${max_rot_velocity}" motor_number="1" color="Blue">
     <origin xyz="0 ${arm_length} ${rotor_offset_top}" rpy="0 0 0" />
     <xacro:insert_block name="rotor_inertia" />
   </xacro:vertical_rotor>
-  <xacro:vertical_rotor robot_namespace="${namespace}" suffix="back" direction="cw" motor_constant="${motor_constant}" moment_constant="${moment_constant}" parent="base_link" mass_rotor="${mass_rotor}" radius_rotor="${radius_rotor}" time_constant="${time_constant}" max_rot_velocity="${max_rot_velocity}" motor_number="2">
+  <xacro:vertical_rotor robot_namespace="${namespace}" suffix="back" direction="cw" motor_constant="${motor_constant}" moment_constant="${moment_constant}" parent="base_link" mass_rotor="${mass_rotor}" radius_rotor="${radius_rotor}" time_constant="${time_constant}" max_rot_velocity="${max_rot_velocity}" motor_number="2" color="Blue">
     <origin xyz="-${arm_length} 0 ${rotor_offset_top}" rpy="0 0 0" />
     <xacro:insert_block name="rotor_inertia" />
   </xacro:vertical_rotor>
-  <xacro:vertical_rotor robot_namespace="${namespace}" suffix="right" direction="ccw" motor_constant="${motor_constant}" moment_constant="${moment_constant}" parent="base_link" mass_rotor="${mass_rotor}" radius_rotor="${radius_rotor}" time_constant="${time_constant}" max_rot_velocity="${max_rot_velocity}" motor_number="1">
+  <xacro:vertical_rotor robot_namespace="${namespace}" suffix="right" direction="ccw" motor_constant="${motor_constant}" moment_constant="${moment_constant}" parent="base_link" mass_rotor="${mass_rotor}" radius_rotor="${radius_rotor}" time_constant="${time_constant}" max_rot_velocity="${max_rot_velocity}" motor_number="3" color="Blue">
     <origin xyz="0 -${arm_length} ${rotor_offset_top}" rpy="0 0 0" />
     <xacro:insert_block name="rotor_inertia" />
   </xacro:vertical_rotor>
+  <xacro:camera_macro robot_namespace="${namespace}">
+  </xacro:camera_macro>
 </robot>

Commit message: added a commented line for using a mesh instead of a box as the multirotor body

File: mav_description/urdf/multirotor_base.urdf.xacro (robot description, xacro)
@@ -2,5 +2,5 @@
 <robot xmlns:xacro="http://ros.org/wiki/xacro">
   <!-- Main multirotor link -->
-  <xacro:macro name="multirotor_base_macro" params="robot_namespace mass body_width body_height *inertia">
+  <xacro:macro name="multirotor_base_macro" params="robot_namespace mass body_width body_height mesh_file *inertia">
     <link name="base_link">
       <inertial>
@@ -12,4 +12,5 @@
         <origin xyz="0 0 0" rpy="0 0 0" />
         <geometry>
+          <!-- <mesh filename="package://mav_description/meshes/${mesh_file}" scale="0.001 0.001 0.001"/> -->
           <box size="${body_width} ${body_width} ${body_height}"/> <!-- [m] [m] [m] -->
         </geometry>

File: mav_description/urdf/pelican.urdf.xacro (robot description, xacro)
@@ -6,4 +6,5 @@
   <!-- Properties -->
   <xacro:property name="namespace" value="pelican" />
+  <xacro:property name="mesh_file" value="pelican.dae" />
   <xacro:property name="mass" value="0.6" /> <!-- [kg] -->
   <xacro:property name="body_width" value="0.1" /> <!-- [m] -->
@@ -27,5 +28,5 @@
   <xacro:include filename="$(find mav_description)/urdf/multirotor_base.urdf.xacro" />
   <!-- Instantiate multirotor_base_macro once -->
-  <xacro:multirotor_base_macro robot_namespace="${namespace}" mass="${mass}" body_width="${body_width}" body_height="${body_height}">
+  <xacro:multirotor_base_macro robot_namespace="${namespace}" mass="${mass}" body_width="${body_width}" body_height="${body_height}" mesh_file="${mesh_file}">
     <xacro:insert_block name="body_inertia" />
   </xacro:multirotor_base_macro>

Commit message: added firefly model with new params

File: mav_description/urdf/multirotor_base.urdf.xacro (robot description, xacro)
@@ -12,6 +12,6 @@
         <origin xyz="0 0 0" rpy="0 0 0" />
         <geometry>
-          <!-- <mesh filename="package://mav_description/meshes/${mesh_file}" scale="0.001 0.001 0.001"/> -->
-          <box size="${body_width} ${body_width} ${body_height}"/> <!-- [m] [m] [m] -->
+          <mesh filename="package://mav_description/meshes/${mesh_file}" scale="0.001 0.001 0.001"/>
+          <!-- <box size="${body_width} ${body_width} ${body_height}"/> --> <!-- [m] [m] [m] -->
         </geometry>
       </visual>
@@ -152,5 +152,6 @@
       <visual>
         <geometry>
-          <cylinder length="0.005" radius="${radius_rotor}"/> <!-- [m] -->
+          <!-- <cylinder length="0.005" radius="${radius_rotor}"/> --> <!-- [m] -->
+          <box size="${2*radius_rotor} 0.01 0.005"/>
         </geometry>
       </visual>

Commit message: added a cw and a ccw sample mesh for the propellers

File: mav_description/urdf/multirotor_base.urdf.xacro (robot description, xacro)
@@ -153,5 +153,6 @@
         <geometry>
           <!-- <cylinder length="0.005" radius="${radius_rotor}"/> --> <!-- [m] -->
-          <box size="${2*radius_rotor} 0.01 0.005"/>
+          <mesh filename="package://mav_description/meshes/propeller_${direction}.dae" scale="0.001 0.001 0.001"/>
+          <!-- <box size="${2*radius_rotor} 0.01 0.005"/> -->
         </geometry>
       </visual>

Commit message: gazebo_bag_plugin: added logging of the motors and the imu

File: mav_description/urdf/multirotor_base.urdf.xacro (robot description, xacro)
@@ -58,5 +58,5 @@
       <plugin filename="libmav_gazebo_bag_plugin.so" name="rosbag">
         <robotNamespace>${robot_namespace}</robotNamespace>
-        <bagFileName>test.bag</bagFileName>
+        <bagFileName>firefly.bag</bagFileName>
         <linkName>base_link</linkName>
         <frameId>base_link</frameId>
@@ -133,5 +133,5 @@
   <!-- Rotor joint and link -->
   <xacro:macro name="vertical_rotor" params="robot_namespace suffix direction motor_constant moment_constant parent mass_rotor radius_rotor time_constant max_rot_velocity motor_number rotor_drag_coefficient color *origin *inertia">
-    <joint name="rotor_${suffix}_joint" type="continuous">
+    <joint name="rotor_${motor_number}_joint" type="continuous">
       <xacro:insert_block name="origin" />
       <axis xyz="0 0 1" />
@@ -139,8 +139,8 @@
       <!-- <limit effort="2000" velocity="${max_rot_velocity}" /> -->
       <parent link="${parent}"/>
-      <child link="rotor_${suffix}"/>
+      <child link="rotor_${motor_number}"/>
     </joint>
     <!-- TODO(ff): not currently set because it's not yet supported -->
-    <!-- <gazebo reference="rotor_${suffix}_joint">
+    <!-- <gazebo reference="rotor_${motor_number}_joint">
       <axis>
         <xyz>0 0 1</xyz>
@@ -152,5 +152,5 @@
       </axis>
     </gazebo> -->
-    <link name="rotor_${suffix}">
+    <link name="rotor_${motor_number}">
       <inertial>
         <mass value="${mass_rotor}" /> <!-- [kg] -->
@@ -172,6 +172,6 @@
     <gazebo>
       <plugin name="${suffix}_motor_model" filename="libmav_gazebo_motor_model.so">
-        <jointName>rotor_${suffix}_joint</jointName>
-        <linkName>rotor_${suffix}</linkName>
+        <jointName>rotor_${motor_number}_joint</jointName>
+        <linkName>rotor_${motor_number}</linkName>
         <turningDirection>${direction}</turningDirection>
         <timeConstant>${time_constant}</timeConstant>
@@ -182,8 +182,8 @@
         <motorNumber>${motor_number}</motorNumber>
         <rotorDragCoefficient>${rotor_drag_coefficient}</rotorDragCoefficient>
-        <motorVelocityTopic>${robot_namespace}/${suffix}_motor_vel</motorVelocityTopic>
+        <motorVelocityTopic>${robot_namespace}/motor_vel/${motor_number}</motorVelocityTopic>
       </plugin>
     </gazebo>
-    <gazebo reference="rotor_${suffix}">
+    <gazebo reference="rotor_${motor_number}">
       <material>Gazebo/${color}</material>
     </gazebo>

Commit message: multirotor_base.urdf.xacro: added an additional base link containing the inertia

File: mav_description/urdf/multirotor_base.urdf.xacro (robot description, xacro)
@@ -3,5 +3,11 @@
   <!-- Main multirotor link -->
   <xacro:macro name="multirotor_base_macro" params="robot_namespace mass body_width body_height mesh_file *inertia">
-    <link name="base_link">
+    <link name="base_link"></link>
+    <joint name="base_joint" type="fixed">
+      <origin xyz="0 0 0" rpy="0 0 0" />
+      <parent link="base_link"/>
+      <child link="base_link_inertia"/>
+    </joint>
+    <link name="base_link_inertia">
       <inertial>
         <mass value="${mass}" />  <!-- [kg] -->

Commit message: gazebo_motor_model.cpp: Some style fixes and incorporated Markus' getSdfParam
The getSdfParam should be used for all params, but I will do this in a
separate pull request at a later stage and in all plugins.

File: mav_description/urdf/multirotor_base.urdf.xacro (robot description, xacro)
@@ -1,4 +1,5 @@
 <?xml version="1.0"?>
 <robot xmlns:xacro="http://ros.org/wiki/xacro">
+  <xacro:property name="rotor_velocity_slowdown_sim" value="10" />
   <!-- Main multirotor link -->
   <xacro:macro name="multirotor_base_macro" params="robot_namespace mass body_width body_height mesh_file *inertia">
@@ -220,4 +221,5 @@
         <rollingMomentCoefficient>${rolling_moment_coefficient}</rollingMomentCoefficient>
         <motorVelocityTopic>${robot_namespace}/motor_vel/${motor_number}</motorVelocityTopic>
+        <rotorVelocitySlowdownSim>${rotor_velocity_slowdown_sim}</rotorVelocitySlowdownSim>
       </plugin>
     </gazebo>
