Commit message: added full set of imu parameters and fixed imu link

File: mav_description/urdf/multirotor_base.urdf.xacro (robot description, xacro)
@@ -39,8 +39,9 @@
     </link>
     <!-- IMU joint -->
-    <joint name="imu_joint" type="fixed">
-      <origin xyz="0 0 0" rpy="3.1416 0 0" />
+    <joint name="imu_joint" type="revolute">
+      <!--origin xyz="0 0 0" rpy="3.1416 0 0" /-->
       <parent link="base_link"/>
       <child link="imu_link"/>
+      <limit upper="0" lower="0" effort="0" velocity="0"/>
     </joint>
     <gazebo>
@@ -58,9 +59,21 @@
       <!-- IMU -->
       <plugin filename="libhector_gazebo_ros_imu.so" name="imu_ros">
-        <bodyName>base_link</bodyName>
-        <robotNamespace>${robot_namespace}</robotNamespace>
-        <topicName>imu</topicName>
-        <updateRate>100.0</updateRate>
-        <gaussianNoise>0.0</gaussianNoise>
+        <!-- parameters according to http://wiki.ros.org/hector_gazebo_plugins#GazeboRosImu -->
+        <robotNamespace>${robot_namespace}</robotNamespace>
+        <bodyName>imu_link</bodyName> <!-- (string, required): name of the body which holds the IMU sensor -->
+        <topicName>imu</topicName> <!-- (string): name of the sensor output topic and prefix of service names (defaults to imu) -->
+        <accelOffset>0.0 0.0 0.0</accelOffset> <!-- (Vector3): constant acceleration offset -->
+        <accelDrift>0.0 0.0 0.0</accelDrift> <!-- (Vector3): standard deviation of the acceleration drift error -->
+        <accelDriftFrequency>${1.0/3600.0} ${1.0/3600.0} ${1.0/3600.0}</accelDriftFrequency> <!-- (Vector3): mean frequency of the acceleration drift -->
+        <accelGaussianNoise>0.0 0.0 0.0</accelGaussianNoise> <!-- (Vector3): standard deviation of the additive Gaussian acceleration noise -->
+        <rateOffset>0.0 0.0 0.0</rateOffset> <!-- (Vector3): constant rate offset -->
+        <rateDrift>0.0 0.0 0.0</rateDrift> <!-- (Vector3): standard deviation of the rate drift error -->
+        <rateDriftFrequency>${1.0/3600.0} ${1.0/3600.0} ${1.0/3600.0}</rateDriftFrequency> <!-- (Vector3): mean frequency of the rate drift -->
+        <rateGaussianNoise>0.0 0.0 0.0</rateGaussianNoise> <!-- (Vector3): standard deviation of the additive Gaussian rate noise -->
+        <headingOffset>0.0</headingOffset> <!-- (double): constant heading offset -->
+        <headingDrift>0.0</headingDrift> <!-- (double): standard deviation of the heading drift error -->
+        <headingDriftFrequency>${1.0/3600.0}</headingDriftFrequency> <!-- (double): mean frequency of the heading drift -->
+        <headingGaussianNoise>0.0</headingGaussianNoise> <!-- (double): standard deviation of the heading additive Gaussian noise -->
+        <rpyOffsets>0.0 0.0 0.0</rpyOffsets> <!-- (Vector3): if non-zero, used to calculate accelOffset and headingOffset so that resulting roll, pitch and yaw errors correspond to this values when the platform is leveled (for compatibility with gazebo_plugins) -->
       </plugin>
       <!-- ROS Bag Plugin -->

Commit message: cleanup in pose_plugin plugin takes vector parameters for noise added 2 frames and 2 pose sensors with some default params

File: mav_description/urdf/multirotor_base.urdf.xacro (robot description, xacro)
@@ -43,4 +43,30 @@
       <parent link="base_link"/>
       <child link="imu_link"/>
+      <limit upper="0" lower="0" effort="0" velocity="0"/>
+    </joint>
+    <!-- pose sensor1 -->
+    <link name="pose_sensor1_link" >
+      <inertial>
+        <inertia ixx="0.001" ixy="0.0" ixz="0.0" iyy="0.001" iyz="0.0" izz="0.001" />
+        <mass value="0.01" />  <!-- [kg] -->
+      </inertial>
+    </link>
+    <joint name="pose_sensor1_joint" type="revolute">
+    <parent link="base_link"/>
+      <origin xyz="0.05 0.1 0.15" rpy="0 ${3.14/4.0} 0" />
+      <child link="pose_sensor1_link"/>
+      <limit upper="0" lower="0" effort="0" velocity="0"/>
+    </joint>
+     <!-- pose sensor2 -->
+    <link name="pose_sensor2_link" >
+      <inertial>
+        <inertia ixx="0.001" ixy="0.0" ixz="0.0" iyy="0.001" iyz="0.0" izz="0.001" />
+        <mass value="0.01" />  <!-- [kg] -->
+      </inertial>
+    </link>
+    <joint name="pose_sensor2_joint" type="revolute">
+    <parent link="base_link"/>
+      <origin xyz="0.0 0.0 0.0" rpy="0.0 0.0 0.0" />
+      <child link="pose_sensor2_link"/>
       <limit upper="0" lower="0" effort="0" velocity="0"/>
     </joint>
@@ -87,16 +113,25 @@
         <rotorVelocitySlowdownSim>${rotor_velocity_slowdown_sim}</rotorVelocitySlowdownSim>
       </plugin>
-      <!-- Pose Plugin -->
-      <plugin filename="libmav_gazebo_pose_plugin.so" name="pose_plugin">
-        <frameId>base_link</frameId>
-        <linkName>base_link</linkName>
-        <robotNamespace>${robot_namespace}</robotNamespace>
-        <poseTopic>sensor_pose</poseTopic>
+      <plugin filename="libmav_gazebo_pose_plugin.so" name="pose_sensor1">
+        <linkName>pose_sensor1_link</linkName>
+        <robotNamespace>${robot_namespace}</robotNamespace>
+        <poseTopic>sensors/pose1</poseTopic>
         <measurementDivisor>1</measurementDivisor>
         <measurementDelay>0</measurementDelay>
-        <noiseNormalP>0.0</noiseNormalP>
-        <noiseNormalQ>0.0</noiseNormalQ>
-        <noiseUniformP>0.0</noiseUniformP>
-        <noiseUniformQ>0.0</noiseUniformQ>
+        <noiseNormalP>0.01 0.01 0.01</noiseNormalP>
+        <noiseNormalQ>0.02 0.02 0.02</noiseNormalQ>
+        <noiseUniformP>0 0 0</noiseUniformP>
+        <noiseUniformQ>0 0 0</noiseUniformQ>
+      </plugin>
+      <plugin filename="libmav_gazebo_pose_plugin.so" name="pose_sensor2">
+        <linkName>pose_sensor2_link</linkName>
+        <robotNamespace>${robot_namespace}</robotNamespace>
+        <poseTopic>sensors/pose2</poseTopic>
+        <measurementDivisor>1</measurementDivisor>
+        <measurementDelay>0</measurementDelay>
+        <noiseNormalP>0.01 0.01 0.01</noiseNormalP>
+        <noiseNormalQ>0.02 0.02 0.02</noiseNormalQ>
+        <noiseUniformP>0 0 0</noiseUniformP>
+        <noiseUniformQ>0 0 0</noiseUniformQ>
       </plugin>
       <!-- Wind Plugin -->

Commit message: added unknown delay to pose_plugin, which lets us play with how well the filter can handle unknown delay added some more interesting settings for the pose sensors documentation for the pose_plugin

File: mav_description/urdf/multirotor_base.urdf.xacro (robot description, xacro)
@@ -54,5 +54,5 @@
     <joint name="pose_sensor1_joint" type="revolute">
     <parent link="base_link"/>
-      <origin xyz="0.05 0.1 0.15" rpy="0 ${3.14/4.0} 0" />
+      <origin xyz="0.1 0 0" rpy="0 ${3.14/4.0} 0" />
       <child link="pose_sensor1_link"/>
       <limit upper="0" lower="0" effort="0" velocity="0"/>
@@ -67,5 +67,5 @@
     <joint name="pose_sensor2_joint" type="revolute">
     <parent link="base_link"/>
-      <origin xyz="0.0 0.0 0.0" rpy="0.0 0.0 0.0" />
+      <origin xyz="0.0 0.0 0.1" rpy="0.0 0.0 0.0" />
       <child link="pose_sensor2_link"/>
       <limit upper="0" lower="0" effort="0" velocity="0"/>
@@ -137,10 +137,11 @@
         <robotNamespace>${robot_namespace}</robotNamespace>
         <poseTopic>sensors/pose1</poseTopic>
-        <measurementDivisor>1</measurementDivisor>
-        <measurementDelay>0</measurementDelay>
-        <noiseNormalP>0.01 0.01 0.01</noiseNormalP>
-        <noiseNormalQ>0.02 0.02 0.02</noiseNormalQ>
-        <noiseUniformP>0 0 0</noiseUniformP>
-        <noiseUniformQ>0 0 0</noiseUniformQ>
+        <measurementDivisor>7</measurementDivisor> <!-- only every (seq % measurementDivisor) == 0 measurement is published [int]-->
+        <measurementDelay>0</measurementDelay> <!-- time that measurement gets held back before it's published in [simulation cycles (int)] -->
+        <unknownDelay>0.0</unknownDelay> <!-- additional delay, that just gets added to the timestamp [s] -->
+        <noiseNormalP>0.01 0.01 0.01</noiseNormalP> <!-- standard deviation of additive white gaussian noise [m] -->
+        <noiseNormalQ>0.02 0.02 0.02</noiseNormalQ> <!-- standard deviation white gaussian noise [rad]: q_m = q*quaternionFromSmallAngleApproximation(noiseNormalQ)-->
+        <noiseUniformP>0 0 0</noiseUniformP> <!-- symmetric bounds of uniform noise [m] -->
+        <noiseUniformQ>0 0 0</noiseUniformQ> <!-- symmetric bounds of uniform noise [rad], computation see above -->
       </plugin>
       <plugin filename="libmav_gazebo_pose_plugin.so" name="pose_sensor2">
@@ -148,6 +149,7 @@
         <robotNamespace>${robot_namespace}</robotNamespace>
         <poseTopic>sensors/pose2</poseTopic>
-        <measurementDivisor>1</measurementDivisor>
+        <measurementDivisor>5</measurementDivisor>
         <measurementDelay>0</measurementDelay>
+        <unknownDelay>0.001</unknownDelay>
         <noiseNormalP>0.01 0.01 0.01</noiseNormalP>
         <noiseNormalQ>0.02 0.02 0.02</noiseNormalQ>

Commit message: added kinect xacro macro

File: mav_description/urdf/multirotor_base.urdf.xacro (robot description, xacro)
@@ -177,3 +177,68 @@
     </gazebo>
   </xacro:macro>
+  <xacro:macro name="kinect_gazebo" params="frame_rate">
+    <joint name="vi_sensor_joint" type="fixed">
+      <axis xyz="0 1 0" />
+      <origin xyz="0.13 0 0" rpy="0 0 0" />
+      <parent link="base_link" />
+      <child link="vi_sensor_link" />
+    </joint>
+    <link name="vi_sensor_link">
+      <collision>
+        <origin xyz="0 0 0" rpy="0 0 0" />
+        <geometry>
+          <box size="0.1 0.1 0.1" />
+        </geometry>
+      </collision>
+      <visual>
+        <origin xyz="0 0 0" rpy="0 0 0" />
+        <geometry>
+          <box size="0.02 0.1 0.04" />
+        </geometry>
+        <material name="black" />
+      </visual>
+      <inertial>
+        <mass value="1e-5" />
+        <origin xyz="0 0 0" rpy="0 0 0" />
+        <inertia ixx="1e-6" ixy="0" ixz="0" iyy="1e-6" iyz="0" izz="1e-6" />
+      </inertial>
+    </link>
+    <gazebo reference="vi_sensor_link">
+	<sensor type="depth" name="vi_sensor">
+		<always_on>true</always_on>
+		<update_rate>20.0</update_rate>
+		<camera>
+			<horizontal_fov>2</horizontal_fov>
+			<image>
+				<format>L8</format>
+				<width>640</width>
+				<height>480</height>
+			</image>
+			<clip>
+				<near>0.01</near>
+				<far>100</far>
+			</clip>
+		</camera>
+		<plugin name="vi_sensor_link" filename="libgazebo_ros_openni_kinect.so">
+			<baseline>0.2</baseline>
+			<alwaysOn>true</alwaysOn>
+			<updateRate>20.0</updateRate>
+			<cameraName>vi_sensor</cameraName>
+			<imageTopicName>/vi_sensor/depth/image_raw</imageTopicName>
+			<cameraInfoTopicName>/vi_sensor/depth/camera_info</cameraInfoTopicName>
+			<depthImageTopicName>/vi_sensor/depth/image_raw</depthImageTopicName>
+			<depthImageInfoTopicName>/vi_sensor/depth/camera_info</depthImageInfoTopicName>
+			<pointCloudTopicName>/vi_sensor/depth/points</pointCloudTopicName>
+			<frameName>vi_sensor_link</frameName>
+			<pointCloudCutoff>0.5</pointCloudCutoff>
+			<distortionK1>0.00000001</distortionK1>
+			<distortionK2>0.00000001</distortionK2>
+			<distortionK3>0.00000001</distortionK3>
+			<distortionT1>0.00000001</distortionT1>
+			<distortionT2>0.00000001</distortionT2>
+		</plugin>
+	</sensor>
+	<material value="Gazebo/Red" />
+    </gazebo>
+  </xacro:macro>
 </robot>

Commit message: disable ugly camera visual

File: mav_description/urdf/multirotor_base.urdf.xacro (robot description, xacro)
@@ -77,11 +77,11 @@
         </geometry>
       </collision>
-      <visual>
-        <origin xyz="0 0 0" rpy="0 0 0" />
-        <geometry>
-          <box size="0.1 0.1 0.1" />
-        </geometry>
-        <material name="red" />
-      </visual>
+      <!-- <visual> -->
+        <!-- <origin xyz="0 0 0" rpy="0 0 0" /> -->
+        <!-- <geometry> -->
+          <!-- <box size="0.1 0.1 0.1" /> -->
+        <!-- </geometry> -->
+        <!-- <material name="red" /> -->
+      <!-- </visual> -->
       <inertial>
         <mass value="1e-5" />

Commit message: add laser scanner

File: mav_description/urdf/multirotor_base.urdf.xacro (robot description, xacro)
@@ -127,4 +127,71 @@
     </gazebo>
   </xacro:macro>
+  <!-- Laser -->
+  <xacro:macro name="laser_macro" params="robot_namespace">
+    <!-- joint -->
+    <joint name="laser_joint" type="fixed">
+      <axis xyz="0 1 0" />
+      <origin xyz="0 0 0.2" rpy="0 0 0" />
+      <parent link="base_link" />
+      <child link="laser_link" />
+    </joint>
+    <!-- link -->
+    <link name="laser_link">
+      <collision>
+        <origin xyz="0 0 0" rpy="0 0 0" />
+        <geometry>
+          <box size="0.1 0.1 0.1" />
+        </geometry>
+      </collision>
+      <!-- <visual> -->
+        <!-- <origin xyz="0 0 0" rpy="0 0 0" /> -->
+        <!-- <geometry> -->
+          <!-- <box size="0.1 0.1 0.1" /> -->
+        <!-- </geometry> -->
+        <!-- <material name="red" /> -->
+      <!-- </visual> -->
+      <!-- inertial-->
+      <inertial>
+        <mass value="1e-5" />
+        <origin xyz="0 0 0" rpy="0 0 0" />
+        <inertia ixx="1e-6" ixy="0" ixz="0" iyy="1e-6" iyz="0" izz="1e-6" />
+      </inertial>
+    </link>
+    <gazebo reference="laser_link">
+      <sensor type="gpu_ray" name="head_hokuyo_sensor">
+        <pose>0 0 0 0 0 0</pose>
+        <visualize>true</visualize>
+        <update_rate>40</update_rate>
+        <ray>
+          <scan>
+            <horizontal>
+              <samples>720</samples>
+              <resolution>1</resolution>
+              <min_angle>-1.570796</min_angle>
+              <max_angle>1.570796</max_angle>
+            </horizontal>
+          </scan>
+          <range>
+            <min>0.10</min>
+            <max>30.0</max>
+            <resolution>0.01</resolution>
+          </range>
+          <noise>
+            <type>gaussian</type>
+            <!-- Noise parameters based on published spec for Hokuyo laser
+               achieving "+-30mm" accuracy at range < 10m.  A mean of 0.0m and
+               stddev of 0.01m will put 99.7% of samples within 0.03m of the true
+               reading. -->
+          <mean>0.0</mean>
+          <stddev>0.01</stddev>
+        </noise>
+      </ray>
+      <plugin name="gazebo_ros_head_hokuyo_controller" filename="libgazebo_ros_gpu_laser.so">
+        <topicName>${robot_namespace}/laser1/scan</topicName>
+        <frameName>laser_link</frameName>
+      </plugin>
+    </sensor>
+  </gazebo>
+  </xacro:macro>
   <!-- Rotor joint and link -->
   <xacro:macro name="vertical_rotor"

Commit message: point laser downwards, simulate range finder

File: mav_description/urdf/multirotor_base.urdf.xacro (robot description, xacro)
@@ -132,5 +132,5 @@
     <joint name="laser_joint" type="fixed">
       <axis xyz="0 1 0" />
-      <origin xyz="0 0 0.2" rpy="0 0 0" />
+      <origin xyz="0 0 -0.2" rpy="0 1.5707963267948966 0" />
       <parent link="base_link" />
       <child link="laser_link" />
@@ -138,10 +138,10 @@
     <!-- link -->
     <link name="laser_link">
-      <collision>
-        <origin xyz="0 0 0" rpy="0 0 0" />
-        <geometry>
-          <box size="0.1 0.1 0.1" />
-        </geometry>
-      </collision>
+      <!-- <collision> -->
+        <!-- <origin xyz="0 0 0" rpy="0 0 0" /> -->
+        <!-- <geometry> -->
+          <!-- <box size="0.1 0.1 0.1" /> -->
+        <!-- </geometry> -->
+      <!-- </collision> -->
       <!-- <visual> -->
         <!-- <origin xyz="0 0 0" rpy="0 0 0" /> -->
@@ -161,18 +161,18 @@
       <sensor type="gpu_ray" name="head_hokuyo_sensor">
         <pose>0 0 0 0 0 0</pose>
-        <visualize>true</visualize>
+        <visualize>false</visualize>
         <update_rate>40</update_rate>
         <ray>
           <scan>
             <horizontal>
-              <samples>720</samples>
+              <samples>1</samples>
               <resolution>1</resolution>
-              <min_angle>-2.0943</min_angle>
-              <max_angle>2.0943</max_angle>
+              <min_angle>-0.1</min_angle>
+              <max_angle>0.1</max_angle>
             </horizontal>
           </scan>
           <range>
             <min>0.10</min>
-            <max>10.0</max>
+            <max>40.0</max>
             <resolution>0.01</resolution>
           </range>

Commit message: fix colors of sensor visuals

File: mav_description/urdf/multirotor_base.urdf.xacro (robot description, xacro)
@@ -82,5 +82,4 @@
           <!-- <box size="0.1 0.1 0.1" /> -->
         <!-- </geometry> -->
-        <!-- <material name="red" /> -->
       <!-- </visual> -->
       <inertial>
@@ -91,4 +90,5 @@
     </link>
     <gazebo reference="camera_link">
+      <material>Gazebo/Red</material>
       <sensor type="camera" name="camera1">
         <update_rate>30.0</update_rate>
@@ -149,5 +149,4 @@
           <!-- <box size="0.1 0.1 0.1" /> -->
         <!-- </geometry> -->
-        <!-- <material name="red" /> -->
       <!-- </visual> -->
       <!-- inertial-->
@@ -159,4 +158,5 @@
     </link>
     <gazebo reference="laser_link">
+      <material>Gazebo/Blue</material>
       <sensor type="gpu_ray" name="head_hokuyo_sensor">
         <pose>0 0 0 0 0 0</pose>

File: mav_description/urdf/static_camera.urdf.xacro (robot description, xacro)
@@ -74,5 +74,4 @@
           <box size="0.1 0.1 0.1" />
         </geometry>
-        <material name="red" />
       </visual>
       <inertial>
@@ -84,4 +83,5 @@
     <gazebo reference="camera_link">
       <static>true</static>
+      <material>Gazebo/Red</material>
       <sensor type="camera" name="camera_static1">
         <update_rate>30.0</update_rate>

Commit message: disable collision for onboard camera link

File: mav_description/urdf/multirotor_base.urdf.xacro (robot description, xacro)
@@ -71,10 +71,10 @@
     <!-- link -->
     <link name="camera_link">
-      <collision>
-        <origin xyz="0 0 0" rpy="0 0 0" />
-        <geometry>
-          <box size="0.1 0.1 0.1" />
-        </geometry>
-      </collision>
+      <!-- <collision> -->
+        <!-- <origin xyz="0 0 0" rpy="0 0 0" /> -->
+        <!-- <geometry> -->
+          <!-- <box size="0.1 0.1 0.1" /> -->
+        <!-- </geometry> -->
+      <!-- </collision> -->
       <!-- <visual> -->
         <!-- <origin xyz="0 0 0" rpy="0 0 0" /> -->
