Commit message: correct iris size

File: mav_description/urdf/iris.urdf.xacro (robot description, xacro)
@@ -7,6 +7,6 @@
   <xacro:property name="mesh_scale_prop" value="1 1 1"/>
   <xacro:property name="mass" value="1.5" /> <!-- [kg] -->
-  <xacro:property name="body_width" value="0.1" /> <!-- [m] -->
-  <xacro:property name="body_height" value="0.16" /> <!-- [m] -->
+  <xacro:property name="body_width" value="0.47" /> <!-- [m] -->
+  <xacro:property name="body_height" value="0.11" /> <!-- [m] -->
   <xacro:property name="mass_rotor" value="0.005" /> <!-- [kg] -->
   <xacro:property name="arm_length_front_x" value="0.13" /> <!-- [m] -->
