Commit message: parametrize propeller mesh scale

File: mav_description/urdf/ardrone.urdf.xacro (robot description, xacro)
@@ -5,4 +5,5 @@
   <xacro:property name="mesh_file" value="ardrone.dae"/>
   <xacro:property name="mesh_scale" value="0.001 0.001 0.001"/>
+  <xacro:property name="mesh_scale_prop" value="1 1 1"/>
   <xacro:property name="mass" value="1.5" /> <!-- [kg] -->
   <xacro:property name="body_width" value="0.1" /> <!-- [m] -->
@@ -67,4 +68,5 @@
     rolling_moment_coefficient="${rolling_moment_coefficient}"
     mesh="ardrone_prop"
+    mesh_scale="${mesh_scale_prop}"
     color="Red">
     <origin xyz="${sqrt2 * arm_length} -${sqrt2 * arm_length} ${rotor_offset_top}" rpy="0 0 0" />
@@ -87,4 +89,5 @@
     rolling_moment_coefficient="${rolling_moment_coefficient}"
     mesh="ardrone_prop"
+    mesh_scale="${mesh_scale_prop}"
     color="DarkGrey">
     <origin xyz="-${sqrt2 * arm_length} ${sqrt2 * arm_length} ${rotor_offset_top}" rpy="0 0 0" />
@@ -106,4 +109,5 @@
     rolling_moment_coefficient="${rolling_moment_coefficient}"
     mesh="ardrone_prop"
+    mesh_scale="${mesh_scale_prop}"
     color="Red">
     <origin xyz="${sqrt2 * arm_length} ${sqrt2 * arm_length} ${rotor_offset_top}" rpy="0 0 0" />
@@ -125,4 +129,5 @@
     rolling_moment_coefficient="${rolling_moment_coefficient}"
     mesh="ardrone_prop"
+    mesh_scale="${mesh_scale_prop}"
     color="DarkGrey">
     <origin xyz="-${sqrt2 * arm_length} -${sqrt2 * arm_length} ${rotor_offset_top}" rpy="0 0 0" />

File: mav_description/urdf/firefly.urdf.xacro (robot description, xacro)
@@ -12,4 +12,5 @@
   <xacro:property name="rotor_offset_top" value="0.037" /> <!-- [m] -->
   <xacro:property name="radius_rotor" value="0.1" /> <!-- [m] -->
+  <xacro:property name="mesh_scale_prop" value="${radius_rotor}"/>
   <xacro:property name="motor_constant" value="8.54858e-06" /> <!-- [kg·m/s^2] -->
   <xacro:property name="moment_constant" value="0.016" /> <!-- [m] -->
@@ -65,4 +66,5 @@
     rolling_moment_coefficient="${rolling_moment_coefficient}"
     mesh="propeller"
+    mesh_scale="${mesh_scale_prop}"
     color="Red">
     <origin xyz="${cos30*arm_length} ${sin30*arm_length} ${rotor_offset_top}" rpy="0 0 0" />
@@ -85,4 +87,5 @@
     rolling_moment_coefficient="${rolling_moment_coefficient}"
     mesh="propeller"
+    mesh_scale="${mesh_scale_prop}"
     color="Blue">
     <origin xyz="0 ${arm_length} ${rotor_offset_top}" rpy="0 0 0" />
@@ -104,4 +107,5 @@
     rolling_moment_coefficient="${rolling_moment_coefficient}"
     mesh="propeller"
+    mesh_scale="${mesh_scale_prop}"
     color="Blue">
     <origin xyz="-${cos30*arm_length} ${sin30*arm_length} ${rotor_offset_top}" rpy="0 0 0" />
@@ -123,4 +127,5 @@
     rolling_moment_coefficient="${rolling_moment_coefficient}"
     mesh="propeller"
+    mesh_scale="${mesh_scale_prop}"
     color="Blue">
     <origin xyz="-${cos30*arm_length} -${sin30*arm_length} ${rotor_offset_top}" rpy="0 0 0" />
@@ -143,4 +148,5 @@
     rolling_moment_coefficient="${rolling_moment_coefficient}"
     mesh="propeller"
+    mesh_scale="${mesh_scale_prop}"
     color="Blue">
     <origin xyz="0 -${arm_length} ${rotor_offset_top}" rpy="0 0 0" />
@@ -163,4 +169,5 @@
     rolling_moment_coefficient="${rolling_moment_coefficient}"
     mesh="propeller"
+    mesh_scale="${mesh_scale_prop}"
     color="Red">
     <origin xyz="${cos30*arm_length} -${sin30*arm_length} ${rotor_offset_top}" rpy="0 0 0" />

File: mav_description/urdf/multirotor_base.urdf.xacro (robot description, xacro)
@@ -196,5 +196,5 @@
   <!-- Rotor joint and link -->
   <xacro:macro name="vertical_rotor"
-    params="robot_namespace suffix direction motor_constant moment_constant parent mass_rotor radius_rotor time_constant_up time_constant_down max_rot_velocity motor_number rotor_drag_coefficient rolling_moment_coefficient color mesh *origin *inertia">
+    params="robot_namespace suffix direction motor_constant moment_constant parent mass_rotor radius_rotor time_constant_up time_constant_down max_rot_velocity motor_number rotor_drag_coefficient rolling_moment_coefficient color mesh mesh_scale *origin *inertia">
     <joint name="rotor_${motor_number}_joint" type="continuous">
       <xacro:insert_block name="origin" />
@@ -218,5 +218,5 @@
           <!-- <mesh filename="package://mav_description/meshes/propeller_${direction}.dae" -->
           <mesh filename="package://mav_description/meshes/${mesh}_${direction}.dae"
-            scale="0.001 0.001 0.001" /> <!-- The propeller meshes have a radius of 1m -->
+            scale="${mesh_scale}" />
           <!-- <box size="${2*radius_rotor} 0.01 0.005"/> -->
         </geometry>

File: mav_description/urdf/pelican.urdf.xacro (robot description, xacro)
@@ -14,4 +14,5 @@
   <xacro:property name="arm_length" value="0.17" /> <!-- [m] -->
   <xacro:property name="rotor_offset_top" value="0.05" /> <!-- [m] -->
+  <xacro:property name="mesh_scale_prop" value="${radius_rotor}"/>
   <xacro:property name="radius_rotor" value="0.08" /> <!-- [m] -->
   <xacro:property name="motor_constant" value="9.9865e-06" /> <!-- [kg·m/s^2] -->
@@ -59,4 +60,5 @@
     rolling_moment_coefficient="${rolling_moment_coefficient}"
     mesh="propeller"
+    mesh_scale="${mesh_scale}"
     color="Red">
     <origin xyz="${arm_length} 0 ${rotor_offset_top}" rpy="0 0 0" />
@@ -78,4 +80,5 @@
     rolling_moment_coefficient="${rolling_moment_coefficient}"
     mesh="propeller"
+    mesh_scale="${mesh_scale}"
     color="Blue">
     <origin xyz="0 ${arm_length} ${rotor_offset_top}" rpy="0 0 0" />
@@ -97,4 +100,5 @@
     rolling_moment_coefficient="${rolling_moment_coefficient}"
     mesh="propeller"
+    mesh_scale="${mesh_scale}"
     color="Blue">
     <origin xyz="-${arm_length} 0 ${rotor_offset_top}" rpy="0 0 0" />
@@ -116,4 +120,5 @@
     rolling_moment_coefficient="${rolling_moment_coefficient}"
     mesh="propeller"
+    mesh_scale="${mesh_scale}"
     color="Blue">
     <origin xyz="0 -${arm_length} ${rotor_offset_top}" rpy="0 0 0" />

Commit message: fix ardrone propeller scale

File: mav_description/urdf/ardrone.urdf.xacro (robot description, xacro)
@@ -5,5 +5,5 @@
   <xacro:property name="mesh_file" value="ardrone.dae"/>
   <xacro:property name="mesh_scale" value="0.001 0.001 0.001"/>
-  <xacro:property name="mesh_scale_prop" value="1 1 1"/>
+  <xacro:property name="mesh_scale_prop" value="0.001 0.001 0.001"/>
   <xacro:property name="mass" value="1.5" /> <!-- [kg] -->
   <xacro:property name="body_width" value="0.1" /> <!-- [m] -->

Commit message: change ardrone size

File: mav_description/urdf/ardrone.urdf.xacro (robot description, xacro)
@@ -7,5 +7,5 @@
   <xacro:property name="mesh_scale_prop" value="0.001 0.001 0.001"/>
   <xacro:property name="mass" value="1.5" /> <!-- [kg] -->
-  <xacro:property name="body_width" value="0.1" /> <!-- [m] -->
+  <xacro:property name="body_width" value="0.3" /> <!-- [m] -->
   <xacro:property name="body_height" value="0.16" /> <!-- [m] -->
   <xacro:property name="mass_rotor" value="0.005" /> <!-- [kg] -->
