Commit message: mav_description & mav_gazebo: updated the launch files and xacro properties

File: mav_description/urdf/firefly.xacro (robot description, xacro)
@@ -2,4 +2,5 @@
 <robot name="firefly" xmlns:xacro="http://ros.org/wiki/xacro">
   <!-- Properties -->
+  <xacro:property name="namespace" value="firefly" />
   <xacro:property name="rotor_velocity_slowdown_sim" value="10" />
   <xacro:property name="mesh_file" value="firefly.dae" />

Commit message: fix merge errors, make firefly spawn again

File: mav_description/urdf/firefly.xacro (robot description, xacro)
@@ -13,5 +13,5 @@
   <xacro:property name="rotor_offset_top" value="0.037" /> <!-- [m] -->
   <xacro:property name="radius_rotor" value="0.1" /> <!-- [m] -->
-  <xacro:property name="mesh_scale_prop" value="${radius_rotor}"/>
+  <xacro:property name="mesh_scale_prop" value="${radius_rotor} ${radius_rotor} ${radius_rotor}"/>
   <xacro:property name="motor_constant" value="8.54858e-06" /> <!-- [kg·m/s^2] -->
   <xacro:property name="moment_constant" value="0.016" /> <!-- [m] -->

File: mav_description/urdf/multirotor_base.xacro (robot description, xacro)
@@ -3,15 +3,6 @@
   <!-- Main multirotor link -->
   <xacro:macro name="multirotor_base_macro"
-<<<<<<< HEAD:mav_description/urdf/multirotor_base.urdf.xacro
     params="robot_namespace mass body_width body_height mesh_file mesh_scale color *inertia">
-    <link name="base_link">
-    </link>
-||||||| merged common ancestors
-    params="robot_namespace mass body_width body_height mesh_file *inertia">
     <link name="base_link"></link>
-=======
-    params="robot_namespace mass body_width body_height mesh_file *inertia">
-    <link name="base_link"></link>
->>>>>>> origin/master:mav_description/urdf/multirotor_base.xacro
     <joint name="base_joint" type="fixed">
       <origin xyz="0 0 0" rpy="0 0 0" />
@@ -63,16 +54,17 @@
     <!-- link -->
     <link name="camera_link">
-      <!-- <collision> -->
-        <!-- <origin xyz="0 0 0" rpy="0 0 0" /> -->
-        <!-- <geometry> -->
-          <!-- <box size="0.1 0.1 0.1" /> -->
-        <!-- </geometry> -->
-      <!-- </collision> -->
-      <!-- <visual> -->
-        <!-- <origin xyz="0 0 0" rpy="0 0 0" /> -->
-        <!-- <geometry> -->
-          <!-- <box size="0.1 0.1 0.1" /> -->
-        <!-- </geometry> -->
-      <!-- </visual> -->
+      <collision>
+        <origin xyz="0 0 0" rpy="0 0 0" />
+        <geometry>
+          <box size="0.1 0.1 0.1" />
+        </geometry>
+      </collision>
+      <visual>
+        <origin xyz="0 0 0" rpy="0 0 0" />
+        <geometry>
+          <box size="0.1 0.1 0.1" />
+        </geometry>
+        <material name="red" />
+      </visual>
       <inertial>
         <mass value="1e-5" />

File: mav_description/urdf/pelican.xacro (robot description, xacro)
@@ -14,5 +14,5 @@
   <xacro:property name="arm_length" value="0.17" /> <!-- [m] -->
   <xacro:property name="rotor_offset_top" value="0.05" /> <!-- [m] -->
-  <xacro:property name="mesh_scale_prop" value="${radius_rotor}"/>
+  <xacro:property name="mesh_scale_prop" value="${radius_rotor} ${radius_rotor} ${radius_rotor}"/>
   <xacro:property name="radius_rotor" value="0.08" /> <!-- [m] -->
   <xacro:property name="motor_constant" value="9.9865e-06" /> <!-- [kg·m/s^2] -->
@@ -60,5 +60,5 @@
     rolling_moment_coefficient="${rolling_moment_coefficient}"
     mesh="propeller"
-    mesh_scale="${mesh_scale}"
+    mesh_scale="${mesh_scale_prop}"
     color="Red">
     <origin xyz="${arm_length} 0 ${rotor_offset_top}" rpy="0 0 0" />
@@ -80,5 +80,5 @@
     rolling_moment_coefficient="${rolling_moment_coefficient}"
     mesh="propeller"
-    mesh_scale="${mesh_scale}"
+    mesh_scale="${mesh_scale_prop}"
     color="Blue">
     <origin xyz="0 ${arm_length} ${rotor_offset_top}" rpy="0 0 0" />
@@ -100,5 +100,5 @@
     rolling_moment_coefficient="${rolling_moment_coefficient}"
     mesh="propeller"
-    mesh_scale="${mesh_scale}"
+    mesh_scale="${mesh_scale_prop}"
     color="Blue">
     <origin xyz="-${arm_length} 0 ${rotor_offset_top}" rpy="0 0 0" />
@@ -120,5 +120,5 @@
     rolling_moment_coefficient="${rolling_moment_coefficient}"
     mesh="propeller"
-    mesh_scale="${mesh_scale}"
+    mesh_scale="${mesh_scale_prop}"
     color="Blue">
     <origin xyz="0 -${arm_length} ${rotor_offset_top}" rpy="0 0 0" />
