Commit message: removed more annoying tabs

File: mav_description/urdf/component_snippets.xacro (robot description, xacro)
@@ -1,15 +1,15 @@
 <!-- pose sensor2 -->
 <link name="pose_sensor2_link">
-	<inertial>
-		<inertia ixx="0.001" ixy="0.0" ixz="0.0" iyy="0.001" iyz="0.0"
-			izz="0.001" />
-		<mass value="0.01" />  <!-- [kg] -->
-	</inertial>
+  <inertial>
+    <inertia ixx="0.001" ixy="0.0" ixz="0.0" iyy="0.001" iyz="0.0"
+      izz="0.001" />
+    <mass value="0.01" />  <!-- [kg] -->
+  </inertial>
 </link>
 <joint name="pose_sensor2_joint" type="revolute">
-	<parent link="base_link" />
-	<origin xyz="0.0 0.0 0.1" rpy="0.0 0.0 0.0" />
-	<child link="pose_sensor2_link" />
-	<limit upper="0" lower="0" effort="0" velocity="0" />
+  <parent link="base_link" />
+  <origin xyz="0.0 0.0 0.1" rpy="0.0 0.0 0.0" />
+  <child link="pose_sensor2_link" />
+  <limit upper="0" lower="0" effort="0" velocity="0" />
 </joint>
 <gazebo>

File: mav_description/urdf/firefly.gazebo.xacro (robot description, xacro)
@@ -4,20 +4,20 @@
   <xacro:property name="enable_bag_plugin" value="false" />
   <xacro:property name="bag_file" value="firefly.bag" />
-	<!-- Instantiate firefly "mechanics" -->
-	<xacro:include filename="$(find mav_description)/urdf/firefly.urdf.xacro" />
-	<!-- Create link and joint for a sensor -->
-	<link name="pose_sensor1_link">
-		<inertial>
-			<inertia ixx="0.001" ixy="0.0" ixz="0.0" iyy="0.001" iyz="0.0"
-				izz="0.001" />
-			<mass value="0.01" />  <!-- [kg] -->
-		</inertial>
-	</link>
-	<joint name="pose_sensor1_joint" type="revolute">
-		<parent link="base_link" />
-		<origin xyz="0 0 0" rpy="0 0 0" />
-		<child link="pose_sensor1_link" />
-		<limit upper="0" lower="0" effort="0" velocity="0" />
-	</joint>
+  <!-- Instantiate firefly "mechanics" -->
+  <xacro:include filename="$(find mav_description)/urdf/firefly.urdf.xacro" />
+  <!-- Create link and joint for a sensor -->
+  <link name="pose_sensor1_link">
+    <inertial>
+      <inertia ixx="0.001" ixy="0.0" ixz="0.0" iyy="0.001" iyz="0.0"
+        izz="0.001" />
+      <mass value="0.01" />  <!-- [kg] -->
+    </inertial>
+  </link>
+  <joint name="pose_sensor1_joint" type="revolute">
+    <parent link="base_link" />
+    <origin xyz="0 0 0" rpy="0 0 0" />
+    <child link="pose_sensor1_link" />
+    <limit upper="0" lower="0" effort="0" velocity="0" />
+  </joint>
   <!-- Mount an IMU -->
   <gazebo>
@@ -44,16 +44,16 @@
   </gazebo>
   <!-- Instantiate a controller -->
-	<gazebo>
-		<!-- Controller interface -->
-		<plugin name="controller_interface" filename="libmav_gazebo_controller_interface.so">
-			<robotNamespace>${namespace}</robotNamespace>
-			<commandTopicAttitude>mav_cmd_attitude</commandTopicAttitude>
-			<commandTopicRate>mav_cmd_rate</commandTopicRate>
-			<commandTopicMotor>mav_cmd_motor</commandTopicMotor>
-			<imuTopic>imu</imuTopic>
-			<poseTopic>pose</poseTopic>
-			<motorVelocityReferenceTopic>motor_vel_ref</motorVelocityReferenceTopic>
-		</plugin>
-	</gazebo>
+  <gazebo>
+    <!-- Controller interface -->
+    <plugin name="controller_interface" filename="libmav_gazebo_controller_interface.so">
+      <robotNamespace>${namespace}</robotNamespace>
+      <commandTopicAttitude>mav_cmd_attitude</commandTopicAttitude>
+      <commandTopicRate>mav_cmd_rate</commandTopicRate>
+      <commandTopicMotor>mav_cmd_motor</commandTopicMotor>
+      <imuTopic>imu</imuTopic>
+      <poseTopic>pose</poseTopic>
+      <motorVelocityReferenceTopic>motor_vel_ref</motorVelocityReferenceTopic>
+    </plugin>
+  </gazebo>
   <!-- Mount a generic pose sensor at link sensor1 -->
   <gazebo>
@@ -74,16 +74,16 @@
   <!-- Instantiate a logger -->
   <gazebo>
-		<!-- ROS Bag Plugin -->
-		<xacro:if value="${enable_bag_plugin}">
-			<plugin filename="libmav_gazebo_bag_plugin.so" name="rosbag">
-				<robotNamespace>${namespace}</robotNamespace>
-				<bagFileName>${bag_file}</bagFileName>
-				<linkName>base_link</linkName>
-				<frameId>base_link</frameId>
-				<controlAttitudeThrustSubTopic>mav_cmd</controlAttitudeThrustSubTopic>
-				<controlAttitudeThrustPubTopic>mav_cmd</controlAttitudeThrustPubTopic>
-				<rotorVelocitySlowdownSim>${rotor_velocity_slowdown_sim}</rotorVelocitySlowdownSim>
-			</plugin>
-		</xacro:if>
-	</gazebo>
+    <!-- ROS Bag Plugin -->
+    <xacro:if value="${enable_bag_plugin}">
+      <plugin filename="libmav_gazebo_bag_plugin.so" name="rosbag">
+        <robotNamespace>${namespace}</robotNamespace>
+        <bagFileName>${bag_file}</bagFileName>
+        <linkName>base_link</linkName>
+        <frameId>base_link</frameId>
+        <controlAttitudeThrustSubTopic>mav_cmd</controlAttitudeThrustSubTopic>
+        <controlAttitudeThrustPubTopic>mav_cmd</controlAttitudeThrustPubTopic>
+        <rotorVelocitySlowdownSim>${rotor_velocity_slowdown_sim}</rotorVelocitySlowdownSim>
+      </plugin>
+    </xacro:if>
+  </gazebo>
 </robot>
