Commit message: mav_description: created macros for all plugins and cleaned up xacro files

File: mav_description/urdf/component_snippets.xacro (robot description, xacro)
@@ -1,154 +1,186 @@
-<!-- pose sensor2 -->
-<link name="pose_sensor2_link">
-  <inertial>
-    <inertia ixx="0.001" ixy="0.0" ixz="0.0" iyy="0.001" iyz="0.0"
-      izz="0.001" />
-    <mass value="0.01" />  <!-- [kg] -->
-  </inertial>
-</link>
-<joint name="pose_sensor2_joint" type="revolute">
-  <parent link="base_link" />
-  <origin xyz="0.0 0.0 0.1" rpy="0.0 0.0 0.0" />
-  <child link="pose_sensor2_link" />
-  <limit upper="0" lower="0" effort="0" velocity="0" />
-</joint>
-<gazebo>
-  <!-- Controller interface -->
-  <plugin name="controller_interface" filename="libmav_gazebo_controller_interface.so">
-    <robotNamespace>${namespace}</robotNamespace>
-    <commandAttitudeThrustSubTopic>command/attitude</commandAttitudeThrustSubTopic>
-    <commandRateThrustSubTopic>command/rate</commandRateThrustSubTopic>
-    <commandMotorSpeedSubTopic>command/motors</commandMotorSpeedSubTopic>
-    <imuSubTopic>imu</imuSubTopic>
-    <poseTopic>pose</poseTopic>
-    <motorVelocityCommandPubTopic>motor_velocity_reference</motorVelocityCommandPubTopic>
-  </plugin>
-</gazebo>
-<!-- Mount our IMU -->
-<gazebo>
-  <!-- IMU -->
-  <plugin filename="libmav_gazebo_imu_plugin.so" name="mav_gazebo_imu_plugin">
-	<!-- A good description of the IMU parameters can be found in the kalibr documentation:
-	     https://github.com/ethz-asl/kalibr/wiki/IMU-Noise-Model-and-Intrinsics -->
-    <robotNamespace>${namespace}</robotNamespace> <!-- (string, required): ros namespace in which the messages are published -->
-    <linkName>imu_link</linkName> <!-- (string, required): name of the body which holds the IMU sensor -->
-    <imuTopic>imu</imuTopic> <!-- (string): name of the sensor output topic and prefix of service names (defaults to imu) -->
-    <gyroscopeNoiseDensity>0.0003394</gyroscopeNoiseDensity> <!-- Gyroscope noise density (two-sided spectrum) [rad/s/sqrt(Hz)] -->
-    <gyroscopeRandomWalk>0.000038785</gyroscopeRandomWalk> <!-- Gyroscope bias random walk [rad/s/s/sqrt(Hz)] -->
-    <gyroscopeBiasCorrelationTime>1000.0</gyroscopeBiasCorrelationTime> <!-- Gyroscope bias correlation time constant [s] -->
-    <gyroscopeTurnOnBiasSigma>0.0087</gyroscopeTurnOnBiasSigma> <!-- Gyroscope turn on bias standard deviation [rad/s] -->
-    <accelerometerNoiseDensity>0.004</accelerometerNoiseDensity> <!-- Accelerometer noise density (two-sided spectrum) [m/s^2/sqrt(Hz)] -->
-    <accelerometerRandomWalk>0.006</accelerometerRandomWalk> <!-- Accelerometer bias random walk. [m/s^2/s/sqrt(Hz)] -->
-    <accelerometerBiasCorrelationTime>300.0</accelerometerBiasCorrelationTime> <!-- Accelerometer bias correlation time constant [s] -->
-    <accelerometerTurnOnBiasSigma>0.1960</accelerometerTurnOnBiasSigma> <!-- Accelerometer turn on bias standard deviation [m/s^2] -->
-  </plugin>
-</gazebo>
-<gazebo>
-  <!-- Hector IMU -->
-  <plugin filename="libhector_gazebo_ros_imu.so" name="imu_ros">
-    <!-- parameters according to http://wiki.ros.org/hector_gazebo_plugins#GazeboRosImu -->
-    <robotNamespace>${namespace}</robotNamespace>
-    <bodyName>imu_link</bodyName> <!-- (string, required): name of the body which holds the IMU sensor -->
-    <topicName>imu</topicName> <!-- (string): name of the sensor output topic and prefix of service names (defaults to imu) -->
-    <accelOffset>0.0 0.0 0.0</accelOffset> <!-- (Vector3): constant acceleration offset -->
-    <accelDrift>0.0 0.0 0.0</accelDrift> <!-- (Vector3): standard deviation of the acceleration drift error -->
-    <accelDriftFrequency>${1.0/3600.0} ${1.0/3600.0} ${1.0/3600.0}</accelDriftFrequency> <!-- (Vector3): mean frequency of the acceleration drift -->
-    <accelGaussianNoise>0.0 0.0 0.0</accelGaussianNoise> <!-- (Vector3): standard deviation of the additive Gaussian acceleration noise -->
-    <rateOffset>0.0 0.0 0.0</rateOffset> <!-- (Vector3): constant rate offset -->
-    <rateDrift>0.0 0.0 0.0</rateDrift> <!-- (Vector3): standard deviation of the rate drift error -->
-    <rateDriftFrequency>${1.0/3600.0} ${1.0/3600.0} ${1.0/3600.0}</rateDriftFrequency> <!-- (Vector3): mean frequency of the rate drift -->
-    <rateGaussianNoise>0.0 0.0 0.0</rateGaussianNoise> <!-- (Vector3): standard deviation of the additive Gaussian rate noise -->
-    <headingOffset>0.0</headingOffset> <!-- (double): constant heading offset -->
-    <headingDrift>0.0</headingDrift> <!-- (double): standard deviation of the heading drift error -->
-    <headingDriftFrequency>${1.0/3600.0}</headingDriftFrequency> <!-- (double): mean frequency of the heading drift -->
-    <headingGaussianNoise>0.0</headingGaussianNoise> <!-- (double): standard deviation of the heading additive Gaussian noise -->
-    <rpyOffsets>0.0 0.0 0.0</rpyOffsets> <!-- (Vector3): if non-zero, used to calculate accelOffset and headingOffset so that resulting roll, pitch and yaw errors correspond to this values when the platform is leveled (for compatibility with gazebo_plugins) -->
-   </plugin>
-</gazebo>
-<gazebo>
-   <plugin filename="libhector_gazebo_ros_imu.so" name="imu_ros">
-     <robotNamespace>${namespace}</robotNamespace>
-     <bodyName>imu_link</bodyName>
-     <topicName>ground_truth/imu</topicName>
-     <!-- everything defaults to zero, except drift frequency, let's do that
-      for safety -->
-    <accelDriftFrequency>0.0 0.0 0.0</accelDriftFrequency>
-    <rateDriftFrequency>0.0 0.0 0.0</rateDriftFrequency>
-    <headingDriftFrequency>0.0</headingDriftFrequency>
-  </plugin>
-</gazebo>
-<gazebo>
-  <!-- ROS Bag Plugin -->
-  <xacro:if value="${enable_bag_plugin}">
-    <plugin filename="libmav_gazebo_bag_plugin.so" name="rosbag">
-      <robotNamespace>${namespace}</robotNamespace>
-      <bagFileName>${bag_file}</bagFileName>
-      <linkName>base_link</linkName>
-      <frameId>base_link</frameId>
-      <commandAttitudeThrustSubTopic>command/attitude</commandAttitudeThrustSubTopic>
-      <commandAttitudeThrustPubTopic>command/attitude</commandAttitudeThrustPubTopic>
-      <rotorVelocitySlowdownSim>${rotor_velocity_slowdown_sim}</rotorVelocitySlowdownSim>
-      <excludeFloorLinkFromCollisionCheck>${exclude_floor_link_from_collision_check}</excludeFloorLinkFromCollisionCheck>
-    </plugin>
-  </xacro:if>
-</gazebo>
-<gazebo>
-  <plugin filename="libmav_gazebo_pose_plugin.so" name="ground_truth_pose">
-    <linkName>base_link</linkName>
-    <robotNamespace>${namespace}</robotNamespace>
-    <poseTopic>ground_truth/pose</poseTopic>
-    <measurementDivisor>1</measurementDivisor>
-    <measurementDelay>0</measurementDelay>
-    <noiseNormalPosition>0 0 0</noiseNormalPosition>
-    <noiseNormalQuaternion>0 0 0</noiseNormalQuaternion>
-    <noiseUniformPosition>0 0 0</noiseUniformPosition>
-    <noiseUniformQuaternion>0 0 0</noiseUniformQuaternion>
-  </plugin>
-</gazebo>
-<gazebo>
-  <plugin filename="libmav_gazebo_pose_plugin.so" name="pose_sensor1">
-    <linkName>pose_sensor1_link</linkName>
-    <robotNamespace>${namespace}</robotNamespace>
-    <poseTopic>sensors/pose1</poseTopic>
-    <measurementDivisor>7</measurementDivisor> <!-- only every (seq % measurementDivisor) == 0 measurement is published [int] -->
-    <measurementDelay>0</measurementDelay> <!-- time that measurement gets held back before it's published in [simulation cycles (int)] -->
-    <unknownDelay>0.0</unknownDelay> <!-- additional delay, that just gets added to the timestamp [s] -->
-    <noiseNormalPosition>0.01 0.01 0.01</noiseNormalPosition> <!-- standard deviation of additive white gaussian noise [m] -->
-    <noiseNormalQuaternion>0.02 0.02 0.02</noiseNormalQuaternion> <!-- standard deviation white gaussian noise [rad]: q_m = q*quaternionFromSmallAngleApproximation(noiseNormalQ) -->
-    <noiseUniformPosition>0 0 0</noiseUniformPosition> <!-- symmetric bounds of uniform noise [m] -->
-    <noiseUniformQuaternion>0 0 0</noiseUniformQuaternion> <!-- symmetric bounds of uniform noise [rad], computation see above -->
-    <covarianceImage>package://mav_gazebo/resource/example_poseplugin_map1.bmp</covarianceImage>
-    <covarianceImageScale>0.1</covarianceImageScale>
-  </plugin>
-</gazebo>
-<gazebo>
-  <plugin filename="libmav_gazebo_pose_plugin.so" name="pose_sensor2">
-    <linkName>pose_sensor2_link</linkName>
-    <robotNamespace>${namespace}</robotNamespace>
-    <poseTopic>sensors/pose2</poseTopic>
-    <measurementDivisor>5</measurementDivisor>
-    <measurementDelay>0</measurementDelay>
-    <unknownDelay>0.001</unknownDelay>
-    <noiseNormalPosition>0.01 0.01 0.01</noiseNormalPosition>
-    <noiseNormalQuaternion>0.02 0.02 0.02</noiseNormalQuaternion>
-    <noiseUniformPosition>0 0 0</noiseUniformPosition>
-    <noiseUniformQuaternion>0 0 0</noiseUniformQuaternion>
-    <covarianceImage>package://mav_gazebo/resource/example_poseplugin_map2.bmp</covarianceImage>
-    <covarianceImageScale>0.1</covarianceImageScale>
-  </plugin>
-</gazebo>
-<gazebo>
-  <!-- Wind Plugin -->
-  <plugin filename="libmav_gazebo_wind_plugin.so" name="wind_plugin">
-    <frameId>base_link</frameId>
-    <linkName>base_link</linkName>
-    <robotNamespace>${namespace}</robotNamespace>
-    <xyzOffset>0 0 0</xyzOffset> <!-- [m] [m] [m] -->
-    <windDirection>1 0 0</windDirection>
-    <windForceMean>0</windForceMean> <!-- [N] -->
-    <windGustDirection>0 1 0</windGustDirection>
-    <windGustDuration>2</windGustDuration> <!-- [s] -->
-    <windGustStart>10</windGustStart> <!-- [s] -->
-    <windGustForceMean>0</windGustForceMean> <!-- [N] -->
-  </plugin>
-</gazebo>
+<robot xmlns:xacro="http://ros.org/wiki/xacro">
+  <!-- Macro to add logging to a bag file. -->
+  <xacro:macro name="bag_plugin_macro" params="namespace bag_file rotor_velocity_slowdown_sim">
+    <gazebo>
+      <plugin filename="libmav_gazebo_bag_plugin.so" name="rosbag">
+        <robotNamespace>${namespace}</robotNamespace>
+        <bagFileName>${bag_file}</bagFileName>
+        <linkName>base_link</linkName>
+        <frameId>base_link</frameId>
+        <commandAttitudeThrustSubTopic>command/attitude</commandAttitudeThrustSubTopic>
+        <commandAttitudeThrustPubTopic>command/attitude</commandAttitudeThrustPubTopic>
+        <rotorVelocitySlowdownSim>${rotor_velocity_slowdown_sim}</rotorVelocitySlowdownSim>
+      </plugin>
+    </gazebo>
+  </xacro:macro>
+  <!-- Macro to add a camera. -->
+  <xacro:macro name="camera_macro" params="namespace camera_number update_rate horizontal_fov image_width image_height image_format *origin">
+    <!-- Camera joint -->
+    <joint name="camera${camera_number}_joint" type="fixed">
+      <axis xyz="0 1 0" />
+      <xacro:insert_block name="origin" />
+      <parent link="base_link" />
+      <child link="camera${camera_number}_link" />
+    </joint>
+    <!-- Camera link -->
+    <link name="camera${camera_number}_link">
+      <collision>
+        <origin xyz="0 0 0" rpy="0 0 0" />
+        <geometry>
+          <box size="0.1 0.1 0.1" />
+        </geometry>
+      </collision>
+      <visual>
+        <origin xyz="0 0 0" rpy="0 0 0" />
+        <geometry>
+          <box size="0.1 0.1 0.1" />
+        </geometry>
+        <material name="red" />
+      </visual>
+      <inertial>
+        <mass value="1e-5" />
+        <origin xyz="0 0 0" rpy="0 0 0" />
+        <inertia ixx="1e-6" ixy="0" ixz="0" iyy="1e-6" iyz="0" izz="1e-6" />
+      </inertial>
+    </link>
+    <gazebo reference="camera${camera_number}_link">
+      <sensor type="camera" name="camera${camera_number}">
+        <update_rate>${update_rate}</update_rate>
+        <camera name="head">
+          <horizontal_fov>${horizontal_fov}</horizontal_fov>
+          <image>
+            <width>${image_width}</width>
+            <height>${image_height}</height>
+            <format>${image_format}</format>
+          </image>
+          <clip>
+            <near>0.02</near>
+            <far>300</far>
+          </clip>
+          <noise>
+            <type>gaussian</type>
+            <mean>0.0</mean>
+            <stddev>0.007</stddev>
+          </noise>
+        </camera>
+        <plugin name="camera${camera_number}_controller" filename="libgazebo_ros_camera.so">
+          <alwaysOn>true</alwaysOn>
+          <updateRate>0.0</updateRate>
+          <cameraName>${namespace}/camera${camera_number}</cameraName>
+          <imageTopicName>image_raw</imageTopicName>
+          <cameraInfoTopicName>camera_info</cameraInfoTopicName>
+          <frameName>camera${camera_number}_link</frameName>
+          <hackBaseline>0.0</hackBaseline>
+          <distortionK1>0.0</distortionK1>
+          <distortionK2>0.0</distortionK2>
+          <distortionK3>0.0</distortionK3>
+          <distortionT1>0.0</distortionT1>
+          <distortionT2>0.0</distortionT2>
+        </plugin>
+      </sensor>
+    </gazebo>
+  </xacro:macro>
+  <!-- Macro to add the controller interface. -->
+  <xacro:macro name="controller_plugin_macro" params="namespace imu_sub_topic pose_topic">
+    <gazebo>
+      <plugin name="controller_interface" filename="libmav_gazebo_controller_interface.so">
+        <robotNamespace>${namespace}</robotNamespace>
+        <commandAttitudeThrustSubTopic>command/attitude</commandAttitudeThrustSubTopic>
+        <commandRateThrustSubTopic>command/rate</commandRateThrustSubTopic>
+        <commandMotorSpeedSubTopic>command/motors</commandMotorSpeedSubTopic>
+        <imuSubTopic>${imu_sub_topic}</imuSubTopic>
+        <poseTopic>${pose_topic}</poseTopic>
+        <motorVelocityCommandPubTopic>motor_velocity_reference</motorVelocityCommandPubTopic>
+      </plugin>
+    </gazebo>
+  </xacro:macro>
+  <!-- Macro to add an IMU. -->
+  <xacro:macro name="imu_plugin_macro" params="namespace imu_suffix gyroscope_noise_density gyroscopoe_random_walk gyroscope_bias_correlation_time gyroscope_turn_on_bias_sigma accelerometer_noise_density accelerometer_random_walk accelerometer_bias_correlation_time accelerometer_turn_on_bias_sigma *origin">
+    <!-- IMU link -->
+    <link name="imu${imu_suffix}_link">
+      <inertial>
+        <inertia ixx="0.001" ixy="0.0" ixz="0.0" iyy="0.001" iyz="0.0"
+          izz="0.001" />
+        <mass value="0.01" />  <!-- [kg] -->
+        <origin xyz="0 0 0" rpy="0 0 0" />
+      </inertial>
+    </link>
+    <!-- IMU joint -->
+    <joint name="imu${imu_suffix}_joint" type="revolute">
+      <xacro:insert_block name="origin" />
+      <parent link="base_link" />
+      <child link="imu${imu_suffix}_link" />
+      <limit upper="0" lower="0" effort="0" velocity="0" />
+    </joint>
+    <gazebo>
+      <plugin filename="libmav_gazebo_imu_plugin.so" name="mav_gazebo_imu${imu_suffix}_plugin">
+      <!-- A good description of the IMU parameters can be found in the kalibr documentation:
+           https://github.com/ethz-asl/kalibr/wiki/IMU-Noise-Model-and-Intrinsics -->
+        <robotNamespace>${namespace}</robotNamespace> <!-- (string, required): ros namespace in which the messages are published -->
+        <linkName>imu${imu_suffix}_link</linkName> <!-- (string, required): name of the body which holds the IMU sensor -->
+        <imuTopic>imu${imu_suffix}</imuTopic> <!-- (string): name of the sensor output topic and prefix of service names (defaults to imu) -->
+        <gyroscopeNoiseDensity>${gyroscope_noise_density}</gyroscopeNoiseDensity> <!-- Gyroscope noise density (two-sided spectrum) [rad/s/sqrt(Hz)] -->
+        <gyroscopeRandomWalk>${gyroscopoe_random_walk}</gyroscopeRandomWalk> <!-- Gyroscope bias random walk [rad/s/s/sqrt(Hz)] -->
+        <gyroscopeBiasCorrelationTime>${gyroscope_bias_correlation_time}</gyroscopeBiasCorrelationTime> <!-- Gyroscope bias correlation time constant [s] -->
+        <gyroscopeTurnOnBiasSigma>${gyroscope_turn_on_bias_sigma}</gyroscopeTurnOnBiasSigma> <!-- Gyroscope turn on bias standard deviation [rad/s] -->
+        <accelerometerNoiseDensity>${accelerometer_noise_density}</accelerometerNoiseDensity> <!-- Accelerometer noise density (two-sided spectrum) [m/s^2/sqrt(Hz)] -->
+        <accelerometerRandomWalk>${accelerometer_random_walk}</accelerometerRandomWalk> <!-- Accelerometer bias random walk. [m/s^2/s/sqrt(Hz)] -->
+        <accelerometerBiasCorrelationTime>${accelerometer_bias_correlation_time}</accelerometerBiasCorrelationTime> <!-- Accelerometer bias correlation time constant [s] -->
+        <accelerometerTurnOnBiasSigma>${accelerometer_turn_on_bias_sigma}</accelerometerTurnOnBiasSigma> <!-- Accelerometer turn on bias standard deviation [m/s^2] -->
+      </plugin>
+    </gazebo>
+  </xacro:macro>
+  <!-- Macro to add a generic pose sensor. -->
+  <xacro:macro name="pose_plugin_macro" params="namespace pose_sensor_suffix measurement_divisor measurement_delay unknown_delay noise_normal_position noise_normal_quaternion noise_uniform_position noise_uniform_quaternion enable_pose_map pose_map image_scale *origin">
+    <!-- Pose link -->
+    <link name="pose_sensor${pose_sensor_suffix}_link">
+      <inertial>
+        <inertia ixx="0.001" ixy="0.0" ixz="0.0" iyy="0.001" iyz="0.0"
+          izz="0.001" />
+        <mass value="0.01" />  <!-- [kg] -->
+      </inertial>
+    </link>
+    <!-- Pose joint -->
+    <joint name="pose_sensor${pose_sensor_suffix}_joint" type="revolute">
+      <parent link="base_link" />
+      <xacro:insert_block name="origin" />
+      <child link="pose_sensor${pose_sensor_suffix}_link" />
+      <limit upper="0" lower="0" effort="0" velocity="0" />
+    </joint>
+    <gazebo>
+      <plugin filename="libmav_gazebo_pose_plugin.so" name="pose_sensor${pose_sensor_suffix}">
+        <linkName>pose_sensor${pose_sensor_suffix}_link</linkName>
+        <robotNamespace>${namespace}</robotNamespace>
+        <poseTopic>pose${pose_sensor_suffix}</poseTopic>
+        <measurementDivisor>${measurement_divisor}</measurementDivisor> <!-- only every (seq % measurementDivisor) == 0 measurement is published [int] -->
+        <measurementDelay>${measurement_delay}</measurementDelay> <!-- time that measurement gets held back before it's published in [simulation cycles (int)] -->
+        <unknownDelay>${unknown_delay}</unknownDelay> <!-- additional delay, that just gets added to the timestamp [s] -->
+        <noiseNormalPosition>${noise_normal_position}</noiseNormalPosition> <!-- standard deviation of additive white gaussian noise [m] -->
+        <noiseNormalQuaternion>${noise_normal_quaternion}</noiseNormalQuaternion> <!-- standard deviation white gaussian noise [rad]: q_m = q*quaternionFromSmallAngleApproximation(noiseNormalQ) -->
+        <noiseUniformPosition>${noise_uniform_position}</noiseUniformPosition> <!-- symmetric bounds of uniform noise [m] -->
+        <noiseUniformQuaternion>${noise_uniform_quaternion}</noiseUniformQuaternion> <!-- symmetric bounds of uniform noise [rad], computation see above -->
+        <xacro:if value="${enable_pose_map}">
+          <covarianceImage>package://mav_gazebo/resource/${pose_map}</covarianceImage>
+          <covarianceImageScale>${image_scale}</covarianceImageScale>
+        </xacro:if>
+      </plugin>
+    </gazebo>
+  </xacro:macro>
+  <!-- Macro to add the wind plugin. -->
+  <xacro:macro name="wind_plugin_macro" params="namespace xyz_offset wind_direction wind_force_mean wind_gust_direction wind_gust_duration wind_gust_start wind_gust_force_mean">
+    <gazebo>
+      <plugin filename="libmav_gazebo_wind_plugin.so" name="wind_plugin">
+        <frameId>base_link</frameId>
+        <linkName>base_link</linkName>
+        <robotNamespace>${namespace}</robotNamespace>
+        <xyzOffset>${xyz_offset}</xyzOffset> <!-- [m] [m] [m] -->
+        <windDirection>${wind_direction}</windDirection>
+        <windForceMean>${wind_force_mean}</windForceMean> <!-- [N] -->
+        <windGustDirection>${wind_gust_direction}</windGustDirection>
+        <windGustDuration>${wind_gust_duration}</windGustDuration> <!-- [s] -->
+        <windGustStart>${wind_gust_start}</windGustStart> <!-- [s] -->
+        <windGustForceMean>${wind_gust_force_mean}</windGustForceMean> <!-- [N] -->
+      </plugin>
+    </gazebo>
+  </xacro:macro>
+</robot>

File: mav_description/urdf/firefly.xacro (robot description, xacro)
@@ -33,5 +33,5 @@
   </xacro:property>
   <!-- Included URDF Files -->
-  <xacro:include filename="$(find mav_description)/urdf/multirotor_base.urdf.xacro" />
+  <xacro:include filename="$(find mav_description)/urdf/multirotor_base.xacro" />
   <!-- Instantiate multirotor_base_macro once -->
   <xacro:multirotor_base_macro
@@ -157,5 +157,3 @@
     <xacro:insert_block name="rotor_inertia" />
   </xacro:vertical_rotor>
-  <!-- <xacro:camera_macro robot_namespace="${namespace}">
-  </xacro:camera_macro> -->
 </robot>
