Commit message: mav_description: created macros for all plugins and cleaned up xacro files

File: mav_description/urdf/firefly_base.xacro (robot description, xacro)
@@ -1,98 +1,71 @@
 <?xml version="1.0"?>
 <robot name="firefly" xmlns:xacro="http://ros.org/wiki/xacro">
+  <xacro:include filename="$(find mav_description)/urdf/component_snippets.xacro" />
   <!-- Instantiate firefly "mechanics" -->
-  <xacro:include filename="$(find mav_description)/urdf/firefly.urdf.xacro" />
-  <!-- Create link and joint for a sensor -->
-  <link name="pose_sensor1_link">
-    <inertial>
-      <inertia ixx="0.001" ixy="0.0" ixz="0.0" iyy="0.001" iyz="0.0"
-        izz="0.001" />
-      <mass value="0.01" />  <!-- [kg] -->
-    </inertial>
-  </link>
-  <joint name="pose_sensor1_joint" type="revolute">
-    <parent link="base_link" />
-    <origin xyz="0.03 -0.07 0.1" rpy="0.2 -0.1 0.3" />
-    <child link="pose_sensor1_link" />
-    <limit upper="0" lower="0" effort="0" velocity="0" />
-  </joint>
-  <gazebo>
-    <!-- IMU -->
-    <plugin filename="libmav_gazebo_imu_plugin.so" name="mav_gazebo_imu_plugin">
-  	<!-- A good description of the IMU parameters can be found in the kalibr documentation:
-  	     https://github.com/ethz-asl/kalibr/wiki/IMU-Noise-Model-and-Intrinsics -->
-      <robotNamespace>${namespace}</robotNamespace> <!-- (string, required): ros namespace in which the messages are published -->
-      <linkName>imu_link</linkName> <!-- (string, required): name of the body which holds the IMU sensor -->
-      <imuTopic>imu</imuTopic> <!-- (string): name of the sensor output topic and prefix of service names (defaults to imu) -->
-      <gyroscopeNoiseDensity>0.0003394</gyroscopeNoiseDensity> <!-- Gyroscope noise density (two-sided spectrum) [rad/s/sqrt(Hz)] -->
-      <gyroscopeRandomWalk>0.000038785</gyroscopeRandomWalk> <!-- Gyroscope bias random walk [rad/s/s/sqrt(Hz)] -->
-      <gyroscopeBiasCorrelationTime>1000.0</gyroscopeBiasCorrelationTime> <!-- Gyroscope bias correlation time constant [s] -->
-      <gyroscopeTurnOnBiasSigma>0.0087</gyroscopeTurnOnBiasSigma> <!-- Gyroscope turn on bias standard deviation [rad/s] -->
-      <accelerometerNoiseDensity>0.004</accelerometerNoiseDensity> <!-- Accelerometer noise density (two-sided spectrum) [m/s^2/sqrt(Hz)] -->
-      <accelerometerRandomWalk>0.006</accelerometerRandomWalk> <!-- Accelerometer bias random walk. [m/s^2/s/sqrt(Hz)] -->
-      <accelerometerBiasCorrelationTime>300.0</accelerometerBiasCorrelationTime> <!-- Accelerometer bias correlation time constant [s] -->
-      <accelerometerTurnOnBiasSigma>0.1960</accelerometerTurnOnBiasSigma> <!-- Accelerometer turn on bias standard deviation [m/s^2] -->
-    </plugin>
-  </gazebo>
-  <!-- Ground truth IMU Data. Will be removed for final evaluation. -->
+  <xacro:include filename="$(find mav_description)/urdf/firefly.xacro" />
+  <!-- Instantiate a controller. -->
+  <xacro:controller_plugin_macro
+    namespace="${namespace}"
+    imu_sub_topic="imu"
+    pose_topic="pose1"
+    >
+  </xacro:controller_plugin_macro>
+  <!-- Mount an ADIS16448 IMU. -->
+  <xacro:imu_plugin_macro
+    namespace="${namespace}"
+    imu_suffix=""
+    gyroscope_noise_density="0.0003394"
+    gyroscopoe_random_walk="0.000038785"
+    gyroscope_bias_correlation_time="1000.0"
+    gyroscope_turn_on_bias_sigma="0.0087"
+    accelerometer_noise_density="0.004"
+    accelerometer_random_walk="0.006"
+    accelerometer_bias_correlation_time="300.0"
+    accelerometer_turn_on_bias_sigma="0.1960"
+  >
+    <origin xyz="0 0 0" rpy="0 0 0" />
+  </xacro:imu_plugin_macro>
   <xacro:if value="$(arg enable_ground_truth)">
-    <gazebo>
-      <plugin filename="libhector_gazebo_ros_imu.so" name="imu_ros">
-        <robotNamespace>${namespace}</robotNamespace>
-        <bodyName>imu_link</bodyName>
-        <topicName>ground_truth/imu</topicName>
-        <!-- everything defaults to zero, except drift frequency, let's do that for safety -->
-        <accelDriftFrequency>0.0 0.0 0.0</accelDriftFrequency>
-        <rateDriftFrequency>0.0 0.0 0.0</rateDriftFrequency>
-        <headingDriftFrequency>0.0</headingDriftFrequency>
-      </plugin>
-    </gazebo>
+    <!-- Mount an IMU providing ground truth. -->
+    <xacro:imu_plugin_macro
+      namespace="${namespace}"
+      imu_suffix="gt"
+      gyroscope_noise_density="0.0"
+      gyroscopoe_random_walk="0.0"
+      gyroscope_bias_correlation_time="1000.0"
+      gyroscope_turn_on_bias_sigma="0.0"
+      accelerometer_noise_density="0.0"
+      accelerometer_random_walk="0.0"
+      accelerometer_bias_correlation_time="300.0"
+      accelerometer_turn_on_bias_sigma="0.0"
+    >
+      <origin xyz="0 0 0" rpy="0 0 0" />
+    </xacro:imu_plugin_macro>
+    <!-- Mount a generic pose sensor providing ground truth. -->
+    <xacro:pose_plugin_macro
+      namespace="${namespace}"
+      pose_sensor_suffix="gt"
+      measurement_divisor="1"
+      measurement_delay="0"
+      unknown_delay="0.0"
+      noise_normal_position="0 0 0"
+      noise_normal_quaternion="0 0 0"
+      noise_uniform_position="0 0 0"
+      noise_uniform_quaternion="0 0 0"
+      enable_pose_map="false"
+      pose_map=""
+      image_scale=""
+    >
+      <origin xyz="0 0 0" rpy="0 0 0" />
+    </xacro:pose_plugin_macro>
   </xacro:if>
-  <!-- Instantiate a controller -->
-  <gazebo>
-    <!-- Controller interface -->
-    <plugin name="controller_interface" filename="libmav_gazebo_controller_interface.so">
-      <robotNamespace>${namespace}</robotNamespace>
-      <commandAttitudeThrustSubTopic>command/attitude</commandAttitudeThrustSubTopic>
-      <commandRateThrustSubTopic>command/rate</commandRateThrustSubTopic>
-      <commandMotorSpeedSubTopic>command/motors</commandMotorSpeedSubTopic>
-      <imuSubTopic>imu</imuSubTopic>
-      <poseTopic>pose</poseTopic>
-      <motorVelocityCommandPubTopic>motor_velocity_reference</motorVelocityCommandPubTopic>
-    </plugin>
-  </gazebo>
-  <!-- Mount a generic pose sensor providing ground truth. Will be removed for final evaluation. -->
-  <xacro:if value="$(arg enable_ground_truth)">
-    <gazebo>
-      <!-- Generic 6D pose sensor plugin -->
-      <plugin filename="libmav_gazebo_pose_plugin.so" name="pose_sensor1">
-        <linkName>base_link</linkName>
-        <robotNamespace>${namespace}</robotNamespace>
-        <poseTopic>ground_truth/pose</poseTopic>
-        <measurementDivisor>1</measurementDivisor> <!-- only every (seq % measurementDivisor) == 0 measurement is published [int] -->
-        <measurementDelay>0</measurementDelay> <!-- time that measurement gets held back before it's published in [simulation cycles (int)] -->
-        <unknownDelay>0.0</unknownDelay> <!-- additional delay, that just gets added to the timestamp [s] -->
-        <noiseNormalPosition>0 0 0</noiseNormalPosition> <!-- standard deviation of additive white gaussian noise [m] -->
-        <noiseNormalQuaternion>0 0 0</noiseNormalQuaternion> <!-- standard deviation white gaussian noise [rad]: q_m = q*quaternionFromSmallAngleApproximation(noiseNormalQ) -->
-        <noiseUniformPosition>0 0 0</noiseUniformPosition> <!-- symmetric bounds of uniform noise [m] -->
-        <noiseUniformQuaternion>0 0 0</noiseUniformQuaternion> <!-- symmetric bounds of uniform noise [rad], computation see above -->
-      </plugin>
-    </gazebo>
+  <xacro:if value="$(arg enable_logging)">
+    <!-- Instantiate a logger -->
+    <xacro:bag_plugin_macro
+      namespace="${namespace}"
+      bag_file="$(arg log_file)"
+      rotor_velocity_slowdown_sim="${rotor_velocity_slowdown_sim}"
+    >
+    </xacro:bag_plugin_macro>
   </xacro:if>
-  <!-- Instantiate a logger -->
-  <gazebo>
-    <!-- ROS Bag Plugin -->
-    <xacro:if value="$(arg enable_logging)">
-      <plugin filename="libmav_gazebo_bag_plugin.so" name="rosbag">
-        <robotNamespace>${namespace}</robotNamespace>
-        <bagFileName>$(arg log_file)</bagFileName>
-        <linkName>base_link</linkName>
-        <frameId>base_link</frameId>
-        <commandAttitudeThrustSubTopic>command/attitude</commandAttitudeThrustSubTopic>
-        <commandAttitudeThrustPubTopic>command/attitude</commandAttitudeThrustPubTopic>
-        <rotorVelocitySlowdownSim>${rotor_velocity_slowdown_sim}</rotorVelocitySlowdownSim>
-        <excludeFloorLinkFromCollisionCheck>$(arg exclude_floor_link_from_collision_check)</excludeFloorLinkFromCollisionCheck>
-      </plugin>
-    </xacro:if>
-  </gazebo>
 </robot>

File: mav_description/urdf/multirotor_base.xacro (robot description, xacro)
@@ -31,20 +31,4 @@
       </collision>
     </link>
-    <!-- IMU -->
-    <link name="imu_link">
-      <inertial>
-        <inertia ixx="0.001" ixy="0.0" ixz="0.0" iyy="0.001" iyz="0.0"
-          izz="0.001" />
-        <mass value="0.01" />  <!-- [kg] -->
-        <origin xyz="0 0 0" rpy="0 0 0" />
-      </inertial>
-    </link>
-    <!-- IMU joint -->
-    <joint name="imu_joint" type="revolute">
-      <!--origin xyz="0 0 0" rpy="3.1416 0 0" / -->
-      <parent link="base_link" />
-      <child link="imu_link" />
-      <limit upper="0" lower="0" effort="0" velocity="0" />
-    </joint>
     <!-- attach multirotor_base_plugin to the base_link -->
     <gazebo>

File: mav_description/urdf/pelican.xacro (robot description, xacro)
@@ -28,5 +28,5 @@
   </xacro:property>
   <!-- Included URDF Files -->
-  <xacro:include filename="$(find mav_description)/urdf/multirotor_base.urdf.xacro" />
+  <xacro:include filename="$(find mav_description)/urdf/multirotor_base.xacro" />
   <!-- Instantiate multirotor_base_macro once -->
   <xacro:multirotor_base_macro

Commit message: mav_description: added topic names for pose and imu + minor fixes

File: mav_description/urdf/component_snippets.xacro (robot description, xacro)
@@ -82,5 +82,5 @@
   </xacro:macro>
   <!-- Macro to add the controller interface. -->
-  <xacro:macro name="controller_plugin_macro" params="namespace imu_sub_topic pose_topic">
+  <xacro:macro name="controller_plugin_macro" params="namespace imu_sub_topic">
     <gazebo>
       <plugin name="controller_interface" filename="libmav_gazebo_controller_interface.so">
@@ -90,5 +90,4 @@
         <commandMotorSpeedSubTopic>command/motors</commandMotorSpeedSubTopic>
         <imuSubTopic>${imu_sub_topic}</imuSubTopic>
-        <poseTopic>${pose_topic}</poseTopic>
         <motorVelocityCommandPubTopic>motor_velocity_reference</motorVelocityCommandPubTopic>
       </plugin>
@@ -96,5 +95,5 @@
   </xacro:macro>
   <!-- Macro to add an IMU. -->
-  <xacro:macro name="imu_plugin_macro" params="namespace imu_suffix gyroscope_noise_density gyroscopoe_random_walk gyroscope_bias_correlation_time gyroscope_turn_on_bias_sigma accelerometer_noise_density accelerometer_random_walk accelerometer_bias_correlation_time accelerometer_turn_on_bias_sigma *origin">
+  <xacro:macro name="imu_plugin_macro" params="namespace imu_suffix imu_topic gyroscope_noise_density gyroscopoe_random_walk gyroscope_bias_correlation_time gyroscope_turn_on_bias_sigma accelerometer_noise_density accelerometer_random_walk accelerometer_bias_correlation_time accelerometer_turn_on_bias_sigma *origin">
     <!-- IMU link -->
     <link name="imu${imu_suffix}_link">
@@ -119,5 +118,5 @@
         <robotNamespace>${namespace}</robotNamespace> <!-- (string, required): ros namespace in which the messages are published -->
         <linkName>imu${imu_suffix}_link</linkName> <!-- (string, required): name of the body which holds the IMU sensor -->
-        <imuTopic>imu${imu_suffix}</imuTopic> <!-- (string): name of the sensor output topic and prefix of service names (defaults to imu) -->
+        <imuTopic>${imu_topic}</imuTopic> <!-- (string): name of the sensor output topic and prefix of service names (defaults to imu) -->
         <gyroscopeNoiseDensity>${gyroscope_noise_density}</gyroscopeNoiseDensity> <!-- Gyroscope noise density (two-sided spectrum) [rad/s/sqrt(Hz)] -->
         <gyroscopeRandomWalk>${gyroscopoe_random_walk}</gyroscopeRandomWalk> <!-- Gyroscope bias random walk [rad/s/s/sqrt(Hz)] -->
@@ -132,5 +131,5 @@
   </xacro:macro>
   <!-- Macro to add a generic pose sensor. -->
-  <xacro:macro name="pose_plugin_macro" params="namespace pose_sensor_suffix measurement_divisor measurement_delay unknown_delay noise_normal_position noise_normal_quaternion noise_uniform_position noise_uniform_quaternion enable_pose_map pose_map image_scale *origin">
+  <xacro:macro name="pose_plugin_macro" params="namespace pose_sensor_suffix pose_topic measurement_divisor measurement_delay unknown_delay noise_normal_position noise_normal_quaternion noise_uniform_position noise_uniform_quaternion enable_pose_map pose_map image_scale *origin">
     <!-- Pose link -->
     <link name="pose_sensor${pose_sensor_suffix}_link">
@@ -152,5 +151,5 @@
         <linkName>pose_sensor${pose_sensor_suffix}_link</linkName>
         <robotNamespace>${namespace}</robotNamespace>
-        <poseTopic>pose${pose_sensor_suffix}</poseTopic>
+        <poseTopic>${pose_topic}</poseTopic>
         <measurementDivisor>${measurement_divisor}</measurementDivisor> <!-- only every (seq % measurementDivisor) == 0 measurement is published [int] -->
         <measurementDelay>${measurement_delay}</measurementDelay> <!-- time that measurement gets held back before it's published in [simulation cycles (int)] -->

File: mav_description/urdf/firefly_base.xacro (robot description, xacro)
@@ -8,5 +8,4 @@
     namespace="${namespace}"
     imu_sub_topic="imu"
-    pose_topic="pose1"
     >
   </xacro:controller_plugin_macro>
@@ -15,4 +14,5 @@
     namespace="${namespace}"
     imu_suffix=""
+    imu_topic="imu"
     gyroscope_noise_density="0.0003394"
     gyroscopoe_random_walk="0.000038785"
@@ -31,4 +31,5 @@
       namespace="${namespace}"
       imu_suffix="gt"
+      imu_topic="ground_truth/imu"
       gyroscope_noise_density="0.0"
       gyroscopoe_random_walk="0.0"
@@ -46,4 +47,5 @@
       namespace="${namespace}"
       pose_sensor_suffix="gt"
+      pose_topic="ground_truth/pose"
       measurement_divisor="1"
       measurement_delay="0"

Commit message: firefly_generic_pose_sensor: set the origin of the pose sensor not to zero

File: mav_description/urdf/component_snippets.xacro (robot description, xacro)
@@ -99,6 +99,5 @@
     <link name="imu${imu_suffix}_link">
       <inertial>
-        <inertia ixx="0.001" ixy="0.0" ixz="0.0" iyy="0.001" iyz="0.0"
-          izz="0.001" />
+        <inertia ixx="0.001" ixy="0.0" ixz="0.0" iyy="0.001" iyz="0.0" izz="0.001" />
         <mass value="0.01" />  <!-- [kg] -->
         <origin xyz="0 0 0" rpy="0 0 0" />

Commit message: mav_description: made mass and inertia params and set to smallest, gazebo acceptable, values (except for ADIS16448 set to 15g according to datasheet)

File: mav_description/urdf/component_snippets.xacro (robot description, xacro)
@@ -95,10 +95,10 @@
   </xacro:macro>
   <!-- Macro to add an IMU. -->
-  <xacro:macro name="imu_plugin_macro" params="namespace imu_suffix imu_topic gyroscope_noise_density gyroscopoe_random_walk gyroscope_bias_correlation_time gyroscope_turn_on_bias_sigma accelerometer_noise_density accelerometer_random_walk accelerometer_bias_correlation_time accelerometer_turn_on_bias_sigma *origin">
+  <xacro:macro name="imu_plugin_macro" params="namespace imu_suffix imu_topic mass_imu_sensor gyroscope_noise_density gyroscopoe_random_walk gyroscope_bias_correlation_time gyroscope_turn_on_bias_sigma accelerometer_noise_density accelerometer_random_walk accelerometer_bias_correlation_time accelerometer_turn_on_bias_sigma *inertia *origin">
     <!-- IMU link -->
     <link name="imu${imu_suffix}_link">
       <inertial>
-        <inertia ixx="0.001" ixy="0.0" ixz="0.0" iyy="0.001" iyz="0.0" izz="0.001" />
-        <mass value="0.01" />  <!-- [kg] -->
+        <xacro:insert_block name="inertia" />
+        <mass value="${mass_imu_sensor}" />  <!-- [kg] -->
         <origin xyz="0 0 0" rpy="0 0 0" />
       </inertial>
@@ -130,11 +130,10 @@
   </xacro:macro>
   <!-- Macro to add a generic pose sensor. -->
-  <xacro:macro name="pose_plugin_macro" params="namespace pose_sensor_suffix pose_topic measurement_divisor measurement_delay unknown_delay noise_normal_position noise_normal_quaternion noise_uniform_position noise_uniform_quaternion enable_pose_map pose_map image_scale *origin">
+  <xacro:macro name="pose_plugin_macro" params="namespace pose_sensor_suffix pose_topic mass_pose_sensor measurement_divisor measurement_delay unknown_delay noise_normal_position noise_normal_quaternion noise_uniform_position noise_uniform_quaternion enable_pose_map pose_map image_scale *inertia *origin">
     <!-- Pose link -->
     <link name="pose_sensor${pose_sensor_suffix}_link">
       <inertial>
-        <inertia ixx="0.001" ixy="0.0" ixz="0.0" iyy="0.001" iyz="0.0"
-          izz="0.001" />
-        <mass value="0.01" />  <!-- [kg] -->
+        <xacro:insert_block name="inertia" />
+        <mass value="${mass_pose_sensor}" />  <!-- [kg] -->
       </inertial>
     </link>

File: mav_description/urdf/firefly_base.xacro (robot description, xacro)
@@ -15,4 +15,5 @@
     imu_suffix=""
     imu_topic="imu"
+    mass_imu_sensor="0.015"
     gyroscope_noise_density="0.0003394"
     gyroscopoe_random_walk="0.000038785"
@@ -24,4 +25,5 @@
     accelerometer_turn_on_bias_sigma="0.1960"
   >
+    <inertia ixx="0.00001" ixy="0.0" ixz="0.0" iyy="0.00001" iyz="0.0" izz="0.00001" />
     <origin xyz="0 0 0" rpy="0 0 0" />
   </xacro:imu_plugin_macro>
@@ -32,4 +34,5 @@
       imu_suffix="gt"
       imu_topic="ground_truth/imu"
+      mass_imu_sensor="0.00001"
       gyroscope_noise_density="0.0"
       gyroscopoe_random_walk="0.0"
@@ -41,4 +44,5 @@
       accelerometer_turn_on_bias_sigma="0.0"
     >
+      <inertia ixx="0.00001" ixy="0.0" ixz="0.0" iyy="0.00001" iyz="0.0" izz="0.00001" />
       <origin xyz="0 0 0" rpy="0 0 0" />
     </xacro:imu_plugin_macro>
@@ -48,4 +52,5 @@
       pose_sensor_suffix="gt"
       pose_topic="ground_truth/pose"
+      mass_pose_sensor="0.00001"
       measurement_divisor="1"
       measurement_delay="0"
@@ -59,4 +64,5 @@
       image_scale=""
     >
+      <inertia ixx="0.00001" ixy="0.0" ixz="0.0" iyy="0.00001" iyz="0.0" izz="0.00001" /> <!-- [kg·m^2] [kg·m^2] [kg·m^2] [kg·m^2] [kg·m^2] [kg·m^2] -->
       <origin xyz="0 0 0" rpy="0 0 0" />
     </xacro:pose_plugin_macro>

Commit message: mav_gazebo: added hovering example with ground truth odometry

File: mav_description/urdf/component_snippets.xacro (robot description, xacro)
@@ -129,4 +129,43 @@
     </gazebo>
   </xacro:macro>
+<!-- Macro to add a generic odometry sensor. -->
+  <xacro:macro name="odometry_plugin_macro" params="namespace odometry_sensor_suffix odometry_topic mass_odometry_sensor measurement_divisor measurement_delay unknown_delay noise_normal_position noise_normal_quaternion noise_normal_linear noise_normal_angular noise_uniform_position noise_uniform_quaternion noise_uniform_linear noise_uniform_angular enable_odometry_map odometry_map image_scale *inertia *origin">
+    <!-- odometry link -->
+    <link name="odometry_sensor${odometry_sensor_suffix}_link">
+      <inertial>
+        <xacro:insert_block name="inertia" />
+        <mass value="${mass_odometry_sensor}" />  <!-- [kg] -->
+      </inertial>
+    </link>
+    <!-- odometry joint -->
+    <joint name="odometry_sensor${odometry_sensor_suffix}_joint" type="revolute">
+      <parent link="base_link" />
+      <xacro:insert_block name="origin" />
+      <child link="odometry_sensor${odometry_sensor_suffix}_link" />
+      <limit upper="0" lower="0" effort="0" velocity="0" />
+    </joint>
+    <gazebo>
+      <plugin filename="libmav_gazebo_odometry_plugin.so" name="odometry_sensor${odometry_sensor_suffix}">
+        <linkName>odometry_sensor${odometry_sensor_suffix}_link</linkName>
+        <robotNamespace>${namespace}</robotNamespace>
+        <odometryTopic>${odometry_topic}</odometryTopic>
+        <measurementDivisor>${measurement_divisor}</measurementDivisor> <!-- only every (seq % measurementDivisor) == 0 measurement is published [int] -->
+        <measurementDelay>${measurement_delay}</measurementDelay> <!-- time that measurement gets held back before it's published in [simulation cycles (int)] -->
+        <unknownDelay>${unknown_delay}</unknownDelay> <!-- additional delay, that just gets added to the timestamp [s] -->
+        <noiseNormalPosition>${noise_normal_position}</noiseNormalPosition> <!-- standard deviation of additive white gaussian noise [m] -->
+        <noiseNormalQuaternion>${noise_normal_quaternion}</noiseNormalQuaternion> <!-- standard deviation white gaussian noise [rad]: q_m = q*quaternionFromSmallAngleApproximation(noiseNormalQ) -->
+        <noiseNormalLinearVelocity>${noise_normal_linear}</noiseNormalLinearVelocity> <!-- standard deviation of additive white gaussian noise [m/s] -->
+        <noiseNormalAngularVelocity>${noise_normal_angular}</noiseNormalAngularVelocity> <!-- standard deviation of additive white gaussian noise [rad/s] -->
+        <noiseUniformPosition>${noise_uniform_position}</noiseUniformPosition> <!-- symmetric bounds of uniform noise [m] -->
+        <noiseUniformQuaternion>${noise_uniform_quaternion}</noiseUniformQuaternion> <!-- symmetric bounds of uniform noise [rad], computation see above -->
+        <noiseUniformLinearVelocity>${noise_uniform_linear}</noiseUniformLinearVelocity>  <!-- symmetric bounds of uniform noise [m/s] -->
+        <noiseUniformAngularVelocity>${noise_uniform_angular}</noiseUniformAngularVelocity>  <!-- symmetric bounds of uniform noise [rad/s] -->
+        <xacro:if value="${enable_odometry_map}">
+          <covarianceImage>package://mav_gazebo/resource/${odometry_map}</covarianceImage>
+          <covarianceImageScale>${image_scale}</covarianceImageScale>
+        </xacro:if>
+      </plugin>
+    </gazebo>
+  </xacro:macro>
   <!-- Macro to add a generic pose sensor. -->
   <xacro:macro name="pose_plugin_macro" params="namespace pose_sensor_suffix pose_topic mass_pose_sensor measurement_divisor measurement_delay unknown_delay noise_normal_position noise_normal_quaternion noise_uniform_position noise_uniform_quaternion enable_pose_map pose_map image_scale *inertia *origin">
