Commit message: gazebo_odometry_plugin: converted plugin to be able to publish various topics
Now you can publish Pose, PoseWithCovariance, Point, Transform, tf,
Odometry msgs.

File: mav_description/urdf/component_snippets.xacro (robot description, xacro)
@@ -130,5 +130,5 @@
   </xacro:macro>
 <!-- Macro to add a generic odometry sensor. -->
-  <xacro:macro name="odometry_plugin_macro" params="namespace odometry_sensor_suffix odometry_topic mass_odometry_sensor measurement_divisor measurement_delay unknown_delay noise_normal_position noise_normal_quaternion noise_normal_linear noise_normal_angular noise_uniform_position noise_uniform_quaternion noise_uniform_linear noise_uniform_angular enable_odometry_map odometry_map image_scale *inertia *origin">
+  <xacro:macro name="odometry_plugin_macro" params="namespace odometry_sensor_suffix pose_topic pose_with_covariance_topic position_topic transform_topic odometry_topic tf_frame mass_odometry_sensor measurement_divisor measurement_delay unknown_delay noise_normal_position noise_normal_quaternion noise_normal_linear noise_normal_angular noise_uniform_position noise_uniform_quaternion noise_uniform_linear noise_uniform_angular enable_odometry_map odometry_map image_scale *inertia *origin">
     <!-- odometry link -->
     <link name="odometry_sensor${odometry_sensor_suffix}_link">
@@ -149,5 +149,10 @@
         <linkName>odometry_sensor${odometry_sensor_suffix}_link</linkName>
         <robotNamespace>${namespace}</robotNamespace>
+        <poseTopic>${pose_topic}</poseTopic>
+        <poseWithCovarianceTopic>${pose_with_covariance_topic}</poseWithCovarianceTopic>
+        <positionTopic>${position_topic}</positionTopic>
+        <transformTopic>${transform_topic}</transformTopic>
         <odometryTopic>${odometry_topic}</odometryTopic>
+        <tfFrame>${tf_frame}</tfFrame>
         <measurementDivisor>${measurement_divisor}</measurementDivisor> <!-- only every (seq % measurementDivisor) == 0 measurement is published [int] -->
         <measurementDelay>${measurement_delay}</measurementDelay> <!-- time that measurement gets held back before it's published in [simulation cycles (int)] -->

Commit message: gazebo_odometry_plugin: replaced linear by linear_velocity and angular by angular_velocity

File: mav_description/urdf/component_snippets.xacro (robot description, xacro)
@@ -130,5 +130,5 @@
   </xacro:macro>
 <!-- Macro to add a generic odometry sensor. -->
-  <xacro:macro name="odometry_plugin_macro" params="namespace odometry_sensor_suffix pose_topic pose_with_covariance_topic position_topic transform_topic odometry_topic tf_frame mass_odometry_sensor measurement_divisor measurement_delay unknown_delay noise_normal_position noise_normal_quaternion noise_normal_linear noise_normal_angular noise_uniform_position noise_uniform_quaternion noise_uniform_linear noise_uniform_angular enable_odometry_map odometry_map image_scale *inertia *origin">
+  <xacro:macro name="odometry_plugin_macro" params="namespace odometry_sensor_suffix pose_topic pose_with_covariance_topic position_topic transform_topic odometry_topic tf_frame mass_odometry_sensor measurement_divisor measurement_delay unknown_delay noise_normal_position noise_normal_quaternion noise_normal_linear_velocity noise_normal_angular_velocity noise_uniform_position noise_uniform_quaternion noise_uniform_linear_velocity noise_uniform_angular_velocity enable_odometry_map odometry_map image_scale *inertia *origin">
     <!-- odometry link -->
     <link name="odometry_sensor${odometry_sensor_suffix}_link">
@@ -160,10 +160,10 @@
         <noiseNormalPosition>${noise_normal_position}</noiseNormalPosition> <!-- standard deviation of additive white gaussian noise [m] -->
         <noiseNormalQuaternion>${noise_normal_quaternion}</noiseNormalQuaternion> <!-- standard deviation white gaussian noise [rad]: q_m = q*quaternionFromSmallAngleApproximation(noiseNormalQ) -->
-        <noiseNormalLinearVelocity>${noise_normal_linear}</noiseNormalLinearVelocity> <!-- standard deviation of additive white gaussian noise [m/s] -->
-        <noiseNormalAngularVelocity>${noise_normal_angular}</noiseNormalAngularVelocity> <!-- standard deviation of additive white gaussian noise [rad/s] -->
+        <noiseNormalLinearVelocity>${noise_normal_linear_velocity}</noiseNormalLinearVelocity> <!-- standard deviation of additive white gaussian noise [m/s] -->
+        <noiseNormalAngularVelocity>${noise_normal_angular_velocity}</noiseNormalAngularVelocity> <!-- standard deviation of additive white gaussian noise [rad/s] -->
         <noiseUniformPosition>${noise_uniform_position}</noiseUniformPosition> <!-- symmetric bounds of uniform noise [m] -->
         <noiseUniformQuaternion>${noise_uniform_quaternion}</noiseUniformQuaternion> <!-- symmetric bounds of uniform noise [rad], computation see above -->
-        <noiseUniformLinearVelocity>${noise_uniform_linear}</noiseUniformLinearVelocity>  <!-- symmetric bounds of uniform noise [m/s] -->
-        <noiseUniformAngularVelocity>${noise_uniform_angular}</noiseUniformAngularVelocity>  <!-- symmetric bounds of uniform noise [rad/s] -->
+        <noiseUniformLinearVelocity>${noise_uniform_linear_velocity}</noiseUniformLinearVelocity>  <!-- symmetric bounds of uniform noise [m/s] -->
+        <noiseUniformAngularVelocity>${noise_uniform_angular_velocity}</noiseUniformAngularVelocity>  <!-- symmetric bounds of uniform noise [rad/s] -->
         <xacro:if value="${enable_odometry_map}">
           <covarianceImage>package://mav_gazebo/resource/${odometry_map}</covarianceImage>

Commit message: removed gazebo_pose_plugin

File: mav_description/urdf/component_snippets.xacro (robot description, xacro)
@@ -173,39 +173,4 @@
     </gazebo>
   </xacro:macro>
-  <!-- Macro to add a generic pose sensor. -->
-  <xacro:macro name="pose_plugin_macro" params="namespace pose_sensor_suffix pose_topic mass_pose_sensor measurement_divisor measurement_delay unknown_delay noise_normal_position noise_normal_quaternion noise_uniform_position noise_uniform_quaternion enable_pose_map pose_map image_scale *inertia *origin">
-    <!-- Pose link -->
-    <link name="pose_sensor${pose_sensor_suffix}_link">
-      <inertial>
-        <xacro:insert_block name="inertia" />
-        <mass value="${mass_pose_sensor}" />  <!-- [kg] -->
-      </inertial>
-    </link>
-    <!-- Pose joint -->
-    <joint name="pose_sensor${pose_sensor_suffix}_joint" type="revolute">
-      <parent link="base_link" />
-      <xacro:insert_block name="origin" />
-      <child link="pose_sensor${pose_sensor_suffix}_link" />
-      <limit upper="0" lower="0" effort="0" velocity="0" />
-    </joint>
-    <gazebo>
-      <plugin filename="libmav_gazebo_pose_plugin.so" name="pose_sensor${pose_sensor_suffix}">
-        <linkName>pose_sensor${pose_sensor_suffix}_link</linkName>
-        <robotNamespace>${namespace}</robotNamespace>
-        <poseTopic>${pose_topic}</poseTopic>
-        <measurementDivisor>${measurement_divisor}</measurementDivisor> <!-- only every (seq % measurementDivisor) == 0 measurement is published [int] -->
-        <measurementDelay>${measurement_delay}</measurementDelay> <!-- time that measurement gets held back before it's published in [simulation cycles (int)] -->
-        <unknownDelay>${unknown_delay}</unknownDelay> <!-- additional delay, that just gets added to the timestamp [s] -->
-        <noiseNormalPosition>${noise_normal_position}</noiseNormalPosition> <!-- standard deviation of additive white gaussian noise [m] -->
-        <noiseNormalQuaternion>${noise_normal_quaternion}</noiseNormalQuaternion> <!-- standard deviation white gaussian noise [rad]: q_m = q*quaternionFromSmallAngleApproximation(noiseNormalQ) -->
-        <noiseUniformPosition>${noise_uniform_position}</noiseUniformPosition> <!-- symmetric bounds of uniform noise [m] -->
-        <noiseUniformQuaternion>${noise_uniform_quaternion}</noiseUniformQuaternion> <!-- symmetric bounds of uniform noise [rad], computation see above -->
-        <xacro:if value="${enable_pose_map}">
-          <covarianceImage>package://mav_gazebo/resource/${pose_map}</covarianceImage>
-          <covarianceImageScale>${image_scale}</covarianceImageScale>
-        </xacro:if>
-      </plugin>
-    </gazebo>
-  </xacro:macro>
   <!-- Macro to add the wind plugin. -->
   <xacro:macro name="wind_plugin_macro" params="namespace xyz_offset wind_direction wind_force_mean wind_gust_direction wind_gust_duration wind_gust_start wind_gust_force_mean">

File: mav_description/urdf/firefly_base.xacro (robot description, xacro)
@@ -47,10 +47,15 @@
       <origin xyz="0 0 0" rpy="0 0 0" />
     </xacro:imu_plugin_macro>
-    <!-- Mount a generic pose sensor providing ground truth. -->
-    <xacro:pose_plugin_macro
+    <!-- Mount a generic odometry sensor providing ground truth. -->
+    <xacro:odometry_plugin_macro
       namespace="${namespace}"
-      pose_sensor_suffix="gt"
-      pose_topic="ground_truth/pose"
-      mass_pose_sensor="0.00001"
+      odometry_sensor_suffix="gt"
+      pose_topic=""
+      pose_with_covariance_topic="ground_truth/pose"
+      position_topic=""
+      transform_topic=""
+      odometry_topic="ground_truth/odometry"
+      tf_frame="ground_truth/firefly"
+      mass_odometry_sensor="0.00001"
       measurement_divisor="1"
       measurement_delay="0"
@@ -58,13 +63,17 @@
       noise_normal_position="0 0 0"
       noise_normal_quaternion="0 0 0"
+      noise_normal_linear_velocity="0 0 0"
+      noise_normal_angular_velocity="0 0 0"
       noise_uniform_position="0 0 0"
       noise_uniform_quaternion="0 0 0"
-      enable_pose_map="false"
-      pose_map=""
+      noise_uniform_linear_velocity="0 0 0"
+      noise_uniform_angular_velocity="0 0 0"
+      enable_odometry_map="false"
+      odometry_map=""
       image_scale=""
     >
       <inertia ixx="0.00001" ixy="0.0" ixz="0.0" iyy="0.00001" iyz="0.0" izz="0.00001" /> <!-- [kg·m^2] [kg·m^2] [kg·m^2] [kg·m^2] [kg·m^2] [kg·m^2] -->
-      <origin xyz="0 0 0" rpy="0 0 0" />
-    </xacro:pose_plugin_macro>
+      <origin xyz="0.0 0.0 0.0" rpy="0.0 0.0 0.0" />
+    </xacro:odometry_plugin_macro>
   </xacro:if>
   <xacro:if value="$(arg enable_logging)">

Commit message: gazebo_odometry_plugin: removed tf_frame and always publish if there are subscribers on topic

File: mav_description/urdf/component_snippets.xacro (robot description, xacro)
@@ -130,5 +130,5 @@
   </xacro:macro>
 <!-- Macro to add a generic odometry sensor. -->
-  <xacro:macro name="odometry_plugin_macro" params="namespace odometry_sensor_suffix pose_topic pose_with_covariance_topic position_topic transform_topic odometry_topic tf_frame mass_odometry_sensor measurement_divisor measurement_delay unknown_delay noise_normal_position noise_normal_quaternion noise_normal_linear_velocity noise_normal_angular_velocity noise_uniform_position noise_uniform_quaternion noise_uniform_linear_velocity noise_uniform_angular_velocity enable_odometry_map odometry_map image_scale *inertia *origin">
+  <xacro:macro name="odometry_plugin_macro" params="namespace odometry_sensor_suffix pose_topic pose_with_covariance_topic position_topic transform_topic odometry_topic mass_odometry_sensor measurement_divisor measurement_delay unknown_delay noise_normal_position noise_normal_quaternion noise_normal_linear_velocity noise_normal_angular_velocity noise_uniform_position noise_uniform_quaternion noise_uniform_linear_velocity noise_uniform_angular_velocity enable_odometry_map odometry_map image_scale *inertia *origin">
     <!-- odometry link -->
     <link name="odometry_sensor${odometry_sensor_suffix}_link">
@@ -154,5 +154,4 @@
         <transformTopic>${transform_topic}</transformTopic>
         <odometryTopic>${odometry_topic}</odometryTopic>
-        <tfFrame>${tf_frame}</tfFrame>
         <measurementDivisor>${measurement_divisor}</measurementDivisor> <!-- only every (seq % measurementDivisor) == 0 measurement is published [int] -->
         <measurementDelay>${measurement_delay}</measurementDelay> <!-- time that measurement gets held back before it's published in [simulation cycles (int)] -->

File: mav_description/urdf/firefly_base.xacro (robot description, xacro)
@@ -49,12 +49,11 @@
     <!-- Mount a generic odometry sensor providing ground truth. -->
     <xacro:odometry_plugin_macro
-      namespace="${namespace}"
+      namespace="${namespace}/ground_truth"
       odometry_sensor_suffix="gt"
-      pose_topic=""
-      pose_with_covariance_topic="ground_truth/pose"
-      position_topic=""
-      transform_topic=""
-      odometry_topic="ground_truth/odometry"
-      tf_frame="ground_truth/firefly"
+      pose_topic="pose"
+      pose_with_covariance_topic="pose_with_covariance"
+      position_topic="position"
+      transform_topic="transform"
+      odometry_topic="odometry"
       mass_odometry_sensor="0.00001"
       measurement_divisor="1"

Commit message: gazebo_odometry_plugin: added the possibility to have odometry sensors relative to a parent_link

File: mav_description/urdf/component_snippets.xacro (robot description, xacro)
@@ -130,5 +130,5 @@
   </xacro:macro>
 <!-- Macro to add a generic odometry sensor. -->
-  <xacro:macro name="odometry_plugin_macro" params="namespace odometry_sensor_suffix pose_topic pose_with_covariance_topic position_topic transform_topic odometry_topic mass_odometry_sensor measurement_divisor measurement_delay unknown_delay noise_normal_position noise_normal_quaternion noise_normal_linear_velocity noise_normal_angular_velocity noise_uniform_position noise_uniform_quaternion noise_uniform_linear_velocity noise_uniform_angular_velocity enable_odometry_map odometry_map image_scale *inertia *origin">
+  <xacro:macro name="odometry_plugin_macro" params="namespace odometry_sensor_suffix pose_topic pose_with_covariance_topic position_topic transform_topic odometry_topic parent_frame_id mass_odometry_sensor measurement_divisor measurement_delay unknown_delay noise_normal_position noise_normal_quaternion noise_normal_linear_velocity noise_normal_angular_velocity noise_uniform_position noise_uniform_quaternion noise_uniform_linear_velocity noise_uniform_angular_velocity enable_odometry_map odometry_map image_scale *inertia *origin">
     <!-- odometry link -->
     <link name="odometry_sensor${odometry_sensor_suffix}_link">
@@ -154,4 +154,5 @@
         <transformTopic>${transform_topic}</transformTopic>
         <odometryTopic>${odometry_topic}</odometryTopic>
+        <parentFrameId>${parent_frame_id}</parentFrameId>  <!-- Use the scoped link name here. e.g. Model::link. -->
         <measurementDivisor>${measurement_divisor}</measurementDivisor> <!-- only every (seq % measurementDivisor) == 0 measurement is published [int] -->
         <measurementDelay>${measurement_delay}</measurementDelay> <!-- time that measurement gets held back before it's published in [simulation cycles (int)] -->

File: mav_description/urdf/firefly_base.xacro (robot description, xacro)
@@ -56,4 +56,5 @@
       transform_topic="transform"
       odometry_topic="odometry"
+      parent_frame_id="world"
       mass_odometry_sensor="0.00001"
       measurement_divisor="1"

Commit message: component_snippets.xacro: added line breaks in macros for params

File: mav_description/urdf/component_snippets.xacro (robot description, xacro)
@@ -1,5 +1,6 @@
 <robot xmlns:xacro="http://ros.org/wiki/xacro">
   <!-- Macro to add logging to a bag file. -->
-  <xacro:macro name="bag_plugin_macro" params="namespace bag_file rotor_velocity_slowdown_sim">
+  <xacro:macro name="bag_plugin_macro"
+    params="namespace bag_file rotor_velocity_slowdown_sim">
     <gazebo>
       <plugin filename="libmav_gazebo_bag_plugin.so" name="rosbag">
@@ -15,5 +16,7 @@
   </xacro:macro>
   <!-- Macro to add a camera. -->
-  <xacro:macro name="camera_macro" params="namespace camera_number update_rate horizontal_fov image_width image_height image_format *origin">
+  <xacro:macro name="camera_macro"
+    params="namespace camera_number update_rate
+      horizontal_fov image_width image_height image_format *origin">
     <!-- Camera joint -->
     <joint name="camera${camera_number}_joint" type="fixed">
@@ -95,5 +98,11 @@
   </xacro:macro>
   <!-- Macro to add an IMU. -->
-  <xacro:macro name="imu_plugin_macro" params="namespace imu_suffix imu_topic mass_imu_sensor gyroscope_noise_density gyroscopoe_random_walk gyroscope_bias_correlation_time gyroscope_turn_on_bias_sigma accelerometer_noise_density accelerometer_random_walk accelerometer_bias_correlation_time accelerometer_turn_on_bias_sigma *inertia *origin">
+  <xacro:macro name="imu_plugin_macro"
+    params="namespace imu_suffix imu_topic
+      mass_imu_sensor gyroscope_noise_density gyroscopoe_random_walk
+      gyroscope_bias_correlation_time gyroscope_turn_on_bias_sigma
+      accelerometer_noise_density accelerometer_random_walk
+      accelerometer_bias_correlation_time accelerometer_turn_on_bias_sigma
+      *inertia *origin">
     <!-- IMU link -->
     <link name="imu${imu_suffix}_link">
@@ -130,5 +139,14 @@
   </xacro:macro>
 <!-- Macro to add a generic odometry sensor. -->
-  <xacro:macro name="odometry_plugin_macro" params="namespace odometry_sensor_suffix pose_topic pose_with_covariance_topic position_topic transform_topic odometry_topic parent_frame_id mass_odometry_sensor measurement_divisor measurement_delay unknown_delay noise_normal_position noise_normal_quaternion noise_normal_linear_velocity noise_normal_angular_velocity noise_uniform_position noise_uniform_quaternion noise_uniform_linear_velocity noise_uniform_angular_velocity enable_odometry_map odometry_map image_scale *inertia *origin">
+  <xacro:macro name="odometry_plugin_macro"
+    params="
+      namespace odometry_sensor_suffix pose_topic pose_with_covariance_topic
+      position_topic transform_topic odometry_topic parent_frame_id
+      mass_odometry_sensor measurement_divisor measurement_delay unknown_delay
+      noise_normal_position noise_normal_quaternion noise_normal_linear_velocity
+      noise_normal_angular_velocity noise_uniform_position
+      noise_uniform_quaternion noise_uniform_linear_velocity
+      noise_uniform_angular_velocity enable_odometry_map odometry_map
+      image_scale *inertia *origin">
     <!-- odometry link -->
     <link name="odometry_sensor${odometry_sensor_suffix}_link">
@@ -174,5 +192,8 @@
   </xacro:macro>
   <!-- Macro to add the wind plugin. -->
-  <xacro:macro name="wind_plugin_macro" params="namespace xyz_offset wind_direction wind_force_mean wind_gust_direction wind_gust_duration wind_gust_start wind_gust_force_mean">
+  <xacro:macro name="wind_plugin_macro"
+    params="namespace xyz_offset wind_direction wind_force_mean
+      wind_gust_direction wind_gust_duration wind_gust_start
+      wind_gust_force_mean">
     <gazebo>
       <plugin filename="libmav_gazebo_wind_plugin.so" name="wind_plugin">
