Commit message: ardrone and iris: update from pose to odometry plugin

File: mav_description/urdf/ardrone_base.xacro (robot description, xacro)
@@ -47,10 +47,15 @@
       <origin xyz="0 0 0" rpy="0 0 0" />
     </xacro:imu_plugin_macro>
-    <!-- Mount a generic pose sensor providing ground truth. -->
-    <xacro:pose_plugin_macro
+    <!-- Mount a generic odometry sensor providing ground truth. -->
+    <xacro:odometry_plugin_macro
       namespace="${namespace}"
-      pose_sensor_suffix="gt"
-      pose_topic="ground_truth/pose"
-      mass_pose_sensor="0.00001"
+      odometry_sensor_suffix="gt"
+      pose_topic=""
+      pose_with_covariance_topic="ground_truth/pose"
+      position_topic=""
+      transform_topic=""
+      odometry_topic="ground_truth/odometry"
+      tf_frame="ground_truth/firefly"
+      mass_odometry_sensor="0.00001"
       measurement_divisor="1"
       measurement_delay="0"
@@ -58,13 +63,17 @@
       noise_normal_position="0 0 0"
       noise_normal_quaternion="0 0 0"
+      noise_normal_linear_velocity="0 0 0"
+      noise_normal_angular_velocity="0 0 0"
       noise_uniform_position="0 0 0"
       noise_uniform_quaternion="0 0 0"
-      enable_pose_map="false"
-      pose_map=""
+      noise_uniform_linear_velocity="0 0 0"
+      noise_uniform_angular_velocity="0 0 0"
+      enable_odometry_map="false"
+      odometry_map=""
       image_scale=""
     >
       <inertia ixx="0.00001" ixy="0.0" ixz="0.0" iyy="0.00001" iyz="0.0" izz="0.00001" /> <!-- [kg·m^2] [kg·m^2] [kg·m^2] [kg·m^2] [kg·m^2] [kg·m^2] -->
-      <origin xyz="0 0 0" rpy="0 0 0" />
-    </xacro:pose_plugin_macro>
+      <origin xyz="0.0 0.0 0.0" rpy="0.0 0.0 0.0" />
+    </xacro:odometry_plugin_macro>
   </xacro:if>
   <xacro:if value="$(arg enable_logging)">

File: mav_description/urdf/iris_base.xacro (robot description, xacro)
@@ -47,10 +47,15 @@
       <origin xyz="0 0 0" rpy="0 0 0" />
     </xacro:imu_plugin_macro>
-    <!-- Mount a generic pose sensor providing ground truth. -->
-    <xacro:pose_plugin_macro
+    <!-- Mount a generic odometry sensor providing ground truth. -->
+    <xacro:odometry_plugin_macro
       namespace="${namespace}"
-      pose_sensor_suffix="gt"
-      pose_topic="ground_truth/pose"
-      mass_pose_sensor="0.00001"
+      odometry_sensor_suffix="gt"
+      pose_topic=""
+      pose_with_covariance_topic="ground_truth/pose"
+      position_topic=""
+      transform_topic=""
+      odometry_topic="ground_truth/odometry"
+      tf_frame="ground_truth/firefly"
+      mass_odometry_sensor="0.00001"
       measurement_divisor="1"
       measurement_delay="0"
@@ -58,13 +63,17 @@
       noise_normal_position="0 0 0"
       noise_normal_quaternion="0 0 0"
+      noise_normal_linear_velocity="0 0 0"
+      noise_normal_angular_velocity="0 0 0"
       noise_uniform_position="0 0 0"
       noise_uniform_quaternion="0 0 0"
-      enable_pose_map="false"
-      pose_map=""
+      noise_uniform_linear_velocity="0 0 0"
+      noise_uniform_angular_velocity="0 0 0"
+      enable_odometry_map="false"
+      odometry_map=""
       image_scale=""
     >
       <inertia ixx="0.00001" ixy="0.0" ixz="0.0" iyy="0.00001" iyz="0.0" izz="0.00001" /> <!-- [kg·m^2] [kg·m^2] [kg·m^2] [kg·m^2] [kg·m^2] [kg·m^2] -->
-      <origin xyz="0 0 0" rpy="0 0 0" />
-    </xacro:pose_plugin_macro>
+      <origin xyz="0.0 0.0 0.0" rpy="0.0 0.0 0.0" />
+    </xacro:odometry_plugin_macro>
   </xacro:if>
   <xacro:if value="$(arg enable_logging)">
