Commit message: removed some annoying tabs

File: euroc_simulation_server/urdf/firefly_t3_1.gazebo.xacro (robot description, xacro)
@@ -2,8 +2,8 @@
 <robot name="firefly" xmlns:xacro="http://ros.org/wiki/xacro">
   <xacro:property name="namespace" value="firefly" />
-	<xacro:property name="enable_bag_plugin" value="true" />
+  <xacro:property name="enable_bag_plugin" value="true" />
   <xacro:property name="bag_file" value="firefly_t3_1.bag" />
-	<!-- Instantiate default firefly-->
-	<xacro:include filename="$(find euroc_simulation_server)/urdf/firefly_base.urdf.xacro" />
+  <!-- Instantiate default firefly-->
+  <xacro:include filename="$(find euroc_simulation_server)/urdf/firefly_base.urdf.xacro" />
   <!-- Mount Pose sensor at pose_sensor1_link -->
   <gazebo>

File: euroc_simulation_server/urdf/firefly_t3_2.gazebo.xacro (robot description, xacro)
@@ -2,8 +2,8 @@
 <robot name="firefly" xmlns:xacro="http://ros.org/wiki/xacro">
   <xacro:property name="namespace" value="firefly" />
-	<xacro:property name="enable_bag_plugin" value="true" />
+  <xacro:property name="enable_bag_plugin" value="true" />
   <xacro:property name="bag_file" value="firefly_t3_2.bag" />
-	<!-- Instantiate default firefly-->
-	<xacro:include filename="$(find euroc_simulation_server)/urdf/firefly_base.urdf.xacro" />
+  <!-- Instantiate default firefly-->
+  <xacro:include filename="$(find euroc_simulation_server)/urdf/firefly_base.urdf.xacro" />
   <!-- Mount Pose sensor at pose_sensor1_link -->
   <gazebo>

File: euroc_simulation_server/urdf/firefly_t3_3.gazebo.xacro (robot description, xacro)
@@ -2,8 +2,8 @@
 <robot name="firefly" xmlns:xacro="http://ros.org/wiki/xacro">
   <xacro:property name="namespace" value="firefly" />
-	<xacro:property name="enable_bag_plugin" value="true" />
+  <xacro:property name="enable_bag_plugin" value="true" />
   <xacro:property name="bag_file" value="firefly_t3_3.bag" />
-	<!-- Instantiate default firefly-->
-	<xacro:include filename="$(find euroc_simulation_server)/urdf/firefly_base.urdf.xacro" />
+  <!-- Instantiate default firefly-->
+  <xacro:include filename="$(find euroc_simulation_server)/urdf/firefly_base.urdf.xacro" />
   <!-- Mount Pose sensor at pose_sensor1_link -->
   <gazebo>

File: euroc_simulation_server/urdf/firefly_t4_1.gazebo.xacro (robot description, xacro)
@@ -2,8 +2,8 @@
 <robot name="firefly" xmlns:xacro="http://ros.org/wiki/xacro">
   <xacro:property name="namespace" value="firefly" />
-	<xacro:property name="enable_bag_plugin" value="true" />
+  <xacro:property name="enable_bag_plugin" value="true" />
   <xacro:property name="bag_file" value="firefly_t4_1.bag" />
-	<!-- Instantiate default firefly-->
-	<xacro:include filename="$(find euroc_simulation_server)/urdf/firefly_base.urdf.xacro" />
+  <!-- Instantiate default firefly-->
+  <xacro:include filename="$(find euroc_simulation_server)/urdf/firefly_base.urdf.xacro" />
   <!-- Mount Pose sensor at pose_sensor1_link -->
   <gazebo>

File: euroc_simulation_server/urdf/firefly_t4_2.gazebo.xacro (robot description, xacro)
@@ -2,8 +2,8 @@
 <robot name="firefly" xmlns:xacro="http://ros.org/wiki/xacro">
   <xacro:property name="namespace" value="firefly" />
-	<xacro:property name="enable_bag_plugin" value="true" />
+  <xacro:property name="enable_bag_plugin" value="true" />
   <xacro:property name="bag_file" value="firefly_t4_2.bag" />
-	<!-- Instantiate default firefly-->
-	<xacro:include filename="$(find euroc_simulation_server)/urdf/firefly_base.urdf.xacro" />
+  <!-- Instantiate default firefly-->
+  <xacro:include filename="$(find euroc_simulation_server)/urdf/firefly_base.urdf.xacro" />
   <!-- Create joint/link for pose sensor2 -->
   <link name="pose_sensor2_link">

File: euroc_simulation_server/urdf/firefly_t4_3.gazebo.xacro (robot description, xacro)
@@ -2,8 +2,8 @@
 <robot name="firefly" xmlns:xacro="http://ros.org/wiki/xacro">
   <xacro:property name="namespace" value="firefly" />
-	<xacro:property name="enable_bag_plugin" value="true" />
+  <xacro:property name="enable_bag_plugin" value="true" />
   <xacro:property name="bag_file" value="firefly_t4_3.bag" />
-	<!-- Instantiate default firefly-->
-	<xacro:include filename="$(find euroc_simulation_server)/urdf/firefly_base.urdf.xacro" />
+  <!-- Instantiate default firefly-->
+  <xacro:include filename="$(find euroc_simulation_server)/urdf/firefly_base.urdf.xacro" />
   <!-- Mount Pose sensor at pose_sensor1_link -->
   <gazebo>
