Commit message: funny argument passing: firefly xacro files now expect the following parameters that can be passed via launch files:  - enable_ground_truth: enables groundtruth plugins. true by default  - enable_logging: enables logging_plugin. false by default  - log_file: specifies a logfile. ~/.ros/firefly_DATE.bag by default

File: euroc_simulation_server/urdf/firefly_base.urdf.xacro (robot description, xacro)
@@ -2,5 +2,4 @@
 <robot name="firefly" xmlns:xacro="http://ros.org/wiki/xacro">
   <!-- Instantiate firefly "mechanics" -->
-  <xacro:property name="enable_ground_truth" value="true"/>
   <xacro:include filename="$(find mav_description)/urdf/firefly.urdf.xacro" />
   <!-- Create link and joint for a sensor -->
@@ -42,5 +41,5 @@
   </gazebo>
   <!-- Ground truth IMU Data. Will be removed for final evaluation. -->
-  <xacro:if value="${enable_ground_truth}">
+  <xacro:if value="$(arg enable_ground_truth)">
     <gazebo>
       <plugin filename="libhector_gazebo_ros_imu.so" name="imu_ros">
@@ -69,5 +68,5 @@
   </gazebo>
   <!-- Mount a generic pose sensor providing ground truth. Will be removed for final evaluation. -->
-  <xacro:if value="${enable_ground_truth}">
+  <xacro:if value="$(arg enable_ground_truth)">
     <gazebo>
       <!-- Generic 6D pose sensor plugin -->
@@ -89,8 +88,8 @@
   <gazebo>
     <!-- ROS Bag Plugin -->
-    <xacro:if value="${enable_bag_plugin}">
+    <xacro:if value="$(arg enable_logging)">
       <plugin filename="libmav_gazebo_bag_plugin.so" name="rosbag">
         <robotNamespace>${namespace}</robotNamespace>
-        <bagFileName>${bag_file}</bagFileName>
+        <bagFileName>$(arg log_file)</bagFileName>
         <linkName>base_link</linkName>
         <frameId>base_link</frameId>

File: euroc_simulation_server/urdf/firefly_t3_1.gazebo.xacro (robot description, xacro)
@@ -2,6 +2,4 @@
 <robot name="firefly" xmlns:xacro="http://ros.org/wiki/xacro">
   <xacro:property name="namespace" value="firefly" />
-  <xacro:property name="enable_bag_plugin" value="true" />
-  <xacro:property name="bag_file" value="firefly_t3_1.bag" />
   <!-- Instantiate default firefly-->
   <xacro:include filename="$(find euroc_simulation_server)/urdf/firefly_base.urdf.xacro" />

File: euroc_simulation_server/urdf/firefly_t3_2.gazebo.xacro (robot description, xacro)
@@ -2,6 +2,4 @@
 <robot name="firefly" xmlns:xacro="http://ros.org/wiki/xacro">
   <xacro:property name="namespace" value="firefly" />
-  <xacro:property name="enable_bag_plugin" value="true" />
-  <xacro:property name="bag_file" value="firefly_t3_2.bag" />
   <!-- Instantiate default firefly-->
   <xacro:include filename="$(find euroc_simulation_server)/urdf/firefly_base.urdf.xacro" />

File: euroc_simulation_server/urdf/firefly_t3_3.gazebo.xacro (robot description, xacro)
@@ -2,6 +2,4 @@
 <robot name="firefly" xmlns:xacro="http://ros.org/wiki/xacro">
   <xacro:property name="namespace" value="firefly" />
-  <xacro:property name="enable_bag_plugin" value="true" />
-  <xacro:property name="bag_file" value="firefly_t3_3.bag" />
   <!-- Instantiate default firefly-->
   <xacro:include filename="$(find euroc_simulation_server)/urdf/firefly_base.urdf.xacro" />

File: euroc_simulation_server/urdf/firefly_t4_1.gazebo.xacro (robot description, xacro)
@@ -2,6 +2,4 @@
 <robot name="firefly" xmlns:xacro="http://ros.org/wiki/xacro">
   <xacro:property name="namespace" value="firefly" />
-  <xacro:property name="enable_bag_plugin" value="true" />
-  <xacro:property name="bag_file" value="firefly_t4_1.bag" />
   <!-- Instantiate default firefly-->
   <xacro:include filename="$(find euroc_simulation_server)/urdf/firefly_base.urdf.xacro" />

File: euroc_simulation_server/urdf/firefly_t4_2.gazebo.xacro (robot description, xacro)
@@ -2,6 +2,4 @@
 <robot name="firefly" xmlns:xacro="http://ros.org/wiki/xacro">
   <xacro:property name="namespace" value="firefly" />
-  <xacro:property name="enable_bag_plugin" value="true" />
-  <xacro:property name="bag_file" value="firefly_t4_2.bag" />
   <!-- Instantiate default firefly-->
   <xacro:include filename="$(find euroc_simulation_server)/urdf/firefly_base.urdf.xacro" />

File: euroc_simulation_server/urdf/firefly_t4_3.gazebo.xacro (robot description, xacro)
@@ -2,6 +2,4 @@
 <robot name="firefly" xmlns:xacro="http://ros.org/wiki/xacro">
   <xacro:property name="namespace" value="firefly" />
-  <xacro:property name="enable_bag_plugin" value="true" />
-  <xacro:property name="bag_file" value="firefly_t4_3.bag" />
   <!-- Instantiate default firefly-->
   <xacro:include filename="$(find euroc_simulation_server)/urdf/firefly_base.urdf.xacro" />

File: mav_description/urdf/firefly.gazebo.xacro (robot description, xacro)
@@ -75,8 +75,8 @@
   <gazebo>
     <!-- ROS Bag Plugin -->
-    <xacro:if value="${enable_bag_plugin}">
+    <xacro:if value="$(arg enable_logging)">
       <plugin filename="libmav_gazebo_bag_plugin.so" name="rosbag">
         <robotNamespace>${namespace}</robotNamespace>
-        <bagFileName>${bag_file}</bagFileName>
+        <bagFileName>$(arg log_file)</bagFileName>
         <linkName>base_link</linkName>
         <frameId>base_link</frameId>

Commit message: changed sensor pose w.r.t. IMU, fixes #104

File: euroc_simulation_server/urdf/firefly_base.urdf.xacro (robot description, xacro)
@@ -13,5 +13,5 @@
   <joint name="pose_sensor1_joint" type="revolute">
     <parent link="base_link" />
-    <origin xyz="0 0 0" rpy="0 0 0" />
+    <origin xyz="0.03 -0.07 0.1" rpy="0.2 -0.1 0.3" />
     <child link="pose_sensor1_link" />
     <limit upper="0" lower="0" effort="0" velocity="0" />

File: euroc_simulation_server/urdf/firefly_t4_2.gazebo.xacro (robot description, xacro)
@@ -14,5 +14,5 @@
   <joint name="pose_sensor2_joint" type="revolute">
     <parent link="base_link" />
-    <origin xyz="0.0 0.0 0.1" rpy="0.0 0.0 0.0" />
+    <origin xyz="-0.05 0.08 0.1" rpy="-0.1 0.2 -0.3" />
     <child link="pose_sensor2_link" />
     <limit upper="0" lower="0" effort="0" velocity="0" />
