Commit message: renamed rotors_description

File: rotors_description/mav_description/urdf/hummingbird.xacro (robot description, xacro)
@@ -33,5 +33,5 @@
   </xacro:property>
   <!-- Included URDF Files -->
-  <xacro:include filename="$(find mav_description)/urdf/multirotor_base.xacro" />
+  <xacro:include filename="$(find rotors_description)/urdf/multirotor_base.xacro" />
   <!-- Instantiate multirotor_base_macro once -->
   <xacro:multirotor_base_macro

File: rotors_description/mav_description/urdf/hummingbird_base.xacro (robot description, xacro)
@@ -1,4 +1,4 @@
 <?xml version="1.0"?>
 <robot name="hummingbird" xmlns:xacro="http://ros.org/wiki/xacro">
-  <xacro:include filename="$(find mav_description)/urdf/hummingbird.xacro" />
+  <xacro:include filename="$(find rotors_description)/urdf/hummingbird.xacro" />
 </robot>

File: rotors_description/urdf/component_snippets.xacro (robot description, xacro)
@@ -21,5 +21,5 @@
     params="namespace bag_file rotor_velocity_slowdown_sim">
     <gazebo>
-      <plugin filename="libmav_gazebo_bag_plugin.so" name="rosbag">
+      <plugin filename="librotors_gazebo_bag_plugin.so" name="rosbag">
         <robotNamespace>${namespace}</robotNamespace>
         <bagFileName>${bag_file}</bagFileName>
@@ -104,5 +104,5 @@
   <xacro:macro name="controller_plugin_macro" params="namespace imu_sub_topic">
     <gazebo>
-      <plugin name="controller_interface" filename="libmav_gazebo_controller_interface.so">
+      <plugin name="controller_interface" filename="librotors_gazebo_controller_interface.so">
         <robotNamespace>${namespace}</robotNamespace>
         <commandAttitudeThrustSubTopic>command/attitude</commandAttitudeThrustSubTopic>
@@ -138,5 +138,5 @@
     </joint>
     <gazebo>
-      <plugin filename="libmav_gazebo_imu_plugin.so" name="mav_gazebo_imu${imu_suffix}_plugin">
+      <plugin filename="librotors_gazebo_imu_plugin.so" name="rotors_gazebo_imu${imu_suffix}_plugin">
       <!-- A good description of the IMU parameters can be found in the kalibr documentation:
            https://github.com/ethz-asl/kalibr/wiki/IMU-Noise-Model-and-Intrinsics -->
@@ -181,5 +181,5 @@
     </joint>
     <gazebo>
-      <plugin filename="libmav_gazebo_odometry_plugin.so" name="odometry_sensor${odometry_sensor_suffix}">
+      <plugin filename="librotors_gazebo_odometry_plugin.so" name="odometry_sensor${odometry_sensor_suffix}">
         <linkName>odometry_sensor${odometry_sensor_suffix}_link</linkName>
         <robotNamespace>${namespace}</robotNamespace>
@@ -202,5 +202,5 @@
         <noiseUniformAngularVelocity>${noise_uniform_angular_velocity}</noiseUniformAngularVelocity>  <!-- symmetric bounds of uniform noise [rad/s] -->
         <xacro:if value="${enable_odometry_map}">
-          <covarianceImage>package://mav_gazebo/resource/${odometry_map}</covarianceImage>
+          <covarianceImage>package://rotors_gazebo/resource/${odometry_map}</covarianceImage>
           <covarianceImageScale>${image_scale}</covarianceImageScale>
         </xacro:if>
@@ -214,5 +214,5 @@
       wind_gust_force_mean">
     <gazebo>
-      <plugin filename="libmav_gazebo_wind_plugin.so" name="wind_plugin">
+      <plugin filename="librotors_gazebo_wind_plugin.so" name="wind_plugin">
         <frameId>base_link</frameId>
         <linkName>base_link</linkName>

File: rotors_description/urdf/firefly.xacro (robot description, xacro)
@@ -50,5 +50,5 @@
   </xacro:property>
   <!-- Included URDF Files -->
-  <xacro:include filename="$(find mav_description)/urdf/multirotor_base.xacro" />
+  <xacro:include filename="$(find rotors_description)/urdf/multirotor_base.xacro" />
   <!-- Instantiate multirotor_base_macro once -->
   <xacro:multirotor_base_macro

File: rotors_description/urdf/firefly_base.xacro (robot description, xacro)
@@ -17,7 +17,7 @@
 -->
 <robot name="firefly" xmlns:xacro="http://ros.org/wiki/xacro">
-  <xacro:include filename="$(find mav_description)/urdf/component_snippets.xacro" />
+  <xacro:include filename="$(find rotors_description)/urdf/component_snippets.xacro" />
   <!-- Instantiate firefly "mechanics" -->
-  <xacro:include filename="$(find mav_description)/urdf/firefly.xacro" />
+  <xacro:include filename="$(find rotors_description)/urdf/firefly.xacro" />
   <!-- Instantiate a controller. -->
   <xacro:controller_plugin_macro

File: rotors_description/urdf/multirotor_base.xacro (robot description, xacro)
@@ -35,5 +35,5 @@
         <origin xyz="0 0 0" rpy="0 0 0" />
         <geometry>
-          <mesh filename="package://mav_description/meshes/${mesh_file}"
+          <mesh filename="package://rotors_description/meshes/${mesh_file}"
             scale="1 1 1" />
           <!-- <box size="${body_width} ${body_width} ${body_height}"/> --> <!-- [m] [m] [m] -->
@@ -49,5 +49,5 @@
     <!-- attach multirotor_base_plugin to the base_link -->
     <gazebo>
-      <plugin filename="libmav_gazebo_multirotor_base_plugin.so" name="rosbag">
+      <plugin filename="librotors_gazebo_multirotor_base_plugin.so" name="rosbag">
         <robotNamespace>${robot_namespace}</robotNamespace>
         <linkName>base_link</linkName>
@@ -145,5 +145,5 @@
         <geometry>
           <!-- <cylinder length="0.005" radius="${radius_rotor}"/> --> <!-- [m] -->
-          <mesh filename="package://mav_description/meshes/propeller_${direction}.dae"
+          <mesh filename="package://rotors_description/meshes/propeller_${direction}.dae"
             scale="${radius_rotor} ${radius_rotor} ${radius_rotor}" /> <!-- The propeller meshes have a radius of 1m -->
           <!-- <box size="${2*radius_rotor} 0.01 0.005"/> -->
@@ -157,5 +157,5 @@
     </link>
     <gazebo>
-      <plugin name="${suffix}_motor_model" filename="libmav_gazebo_motor_model.so">
+      <plugin name="${suffix}_motor_model" filename="librotors_gazebo_motor_model.so">
         <jointName>rotor_${motor_number}_joint</jointName>
         <linkName>rotor_${motor_number}</linkName>

File: rotors_description/urdf/pelican.xacro (robot description, xacro)
@@ -49,5 +49,5 @@
   </xacro:property>
   <!-- Included URDF Files -->
-  <xacro:include filename="$(find mav_description)/urdf/multirotor_base.xacro" />
+  <xacro:include filename="$(find rotors_description)/urdf/multirotor_base.xacro" />
   <!-- Instantiate multirotor_base_macro once -->
   <xacro:multirotor_base_macro

File: rotors_description/urdf/pelican_base.xacro (robot description, xacro)
@@ -17,4 +17,4 @@
 -->
 <robot name="pelican" xmlns:xacro="http://ros.org/wiki/xacro">
-  <xacro:include filename="$(find mav_description)/urdf/pelican.xacro" />
+  <xacro:include filename="$(find rotors_description)/urdf/pelican.xacro" />
 </robot>
