Commit message: update launch and xacro files to new names, update use of odometry plugin

File: rotors_description/urdf/ardrone.gazebo.xacro (robot description, xacro)
@@ -5,5 +5,5 @@
   <xacro:property name="bag_file" value="ardrone.bag" />
   <!-- Instantiate ardrone "mechanics" -->
-  <xacro:include filename="$(find mav_description)/urdf/ardrone.urdf.xacro" />
+  <xacro:include filename="$(find rotors_description)/urdf/ardrone.urdf.xacro" />
   <!-- Create link and joint for a sensor -->
   <link name="pose_sensor1_link">
@@ -23,5 +23,5 @@
   <gazebo>
     <!-- IMU -->
-    <plugin filename="libmav_gazebo_imu_plugin.so" name="mav_gazebo_imu_plugin">
+    <plugin filename="librotors_gazebo_imu_plugin.so" name="rotors_gazebo_imu_plugin">
   	<!-- A good description of the IMU parameters can be found in the kalibr documentation:
   	     https://github.com/ethz-asl/kalibr/wiki/IMU-Noise-Model-and-Intrinsics -->
@@ -42,5 +42,5 @@
   <gazebo>
     <!-- Controller interface -->
-    <plugin name="controller_interface" filename="libmav_gazebo_controller_interface.so">
+    <plugin name="controller_interface" filename="librotors_gazebo_controller_interface.so">
       <robotNamespace>${namespace}</robotNamespace>
       <commandAttitudeThrustSubTopic>command/attitude</commandAttitudeThrustSubTopic>
@@ -55,5 +55,5 @@
   <gazebo>
     <!-- Generic 6D pose sensor plugin -->
-    <plugin filename="libmav_gazebo_pose_plugin.so" name="pose_sensor1">
+    <plugin filename="librotors_gazebo_pose_plugin.so" name="pose_sensor1">
       <linkName>pose_sensor1_link</linkName>
       <robotNamespace>${namespace}</robotNamespace>
@@ -72,5 +72,5 @@
     <!-- ROS Bag Plugin -->
     <xacro:if value="$(arg enable_logging)">
-      <plugin filename="libmav_gazebo_bag_plugin.so" name="rosbag">
+      <plugin filename="librotors_gazebo_bag_plugin.so" name="rosbag">
         <robotNamespace>${namespace}</robotNamespace>
         <bagFileName>$(arg log_file)</bagFileName>
@@ -86,5 +86,5 @@
   <!-- attach wing plugin -->
   <gazebo>
-    <plugin filename="libmav_gazebo_wing_model_plugin.so" name="wing_plugin">
+    <plugin filename="librotors_gazebo_wing_model_plugin.so" name="wing_plugin">
       <robotNamespace>${namespace}</robotNamespace>
       <linkName>base_link</linkName>

File: rotors_description/urdf/ardrone.urdf.xacro (robot description, xacro)
@@ -37,6 +37,6 @@
   </xacro:property>
   <!-- Included URDF Files -->
-  <xacro:include filename="$(find mav_description)/urdf/multirotor_base.urdf.xacro" />
-  <!-- <xacro:include filename="$(find mav_description)/urdf/vtol_wing.urdf.xacro" /> -->
+  <xacro:include filename="$(find rotors_description)/urdf/multirotor_base.urdf.xacro" />
+  <!-- <xacro:include filename="$(find rotors_description)/urdf/vtol_wing.urdf.xacro" /> -->
   <!-- Instantiate multirotor_base_macro once -->
   <xacro:multirotor_base_macro

File: rotors_description/urdf/ardrone.xacro (robot description, xacro)
@@ -38,5 +38,5 @@
   </xacro:property>
   <!-- Included URDF Files -->
-  <xacro:include filename="$(find mav_description)/urdf/multirotor_base.xacro" />
+  <xacro:include filename="$(find rotors_description)/urdf/multirotor_base.xacro" />
   <!-- Instantiate multirotor_base_macro once -->
   <xacro:multirotor_base_macro

File: rotors_description/urdf/ardrone_base.xacro (robot description, xacro)
@@ -1,7 +1,7 @@
 <?xml version="1.0"?>
 <robot name="ardrone" xmlns:xacro="http://ros.org/wiki/xacro">
-  <xacro:include filename="$(find mav_description)/urdf/component_snippets.xacro" />
+  <xacro:include filename="$(find rotors_description)/urdf/component_snippets.xacro" />
   <!-- Instantiate ardrone "mechanics" -->
-  <xacro:include filename="$(find mav_description)/urdf/ardrone.xacro" />
+  <xacro:include filename="$(find rotors_description)/urdf/ardrone.xacro" />
   <!-- Instantiate a controller. -->
   <xacro:controller_plugin_macro
@@ -49,12 +49,12 @@
     <!-- Mount a generic odometry sensor providing ground truth. -->
     <xacro:odometry_plugin_macro
-      namespace="${namespace}"
+      namespace="${namespace}/ground_truth"
       odometry_sensor_suffix="gt"
-      pose_topic=""
-      pose_with_covariance_topic="ground_truth/pose"
-      position_topic=""
-      transform_topic=""
-      odometry_topic="ground_truth/odometry"
-      tf_frame="ground_truth/firefly"
+      pose_topic="pose"
+      pose_with_covariance_topic="pose_with_covariance"
+      position_topic="position"
+      transform_topic="transform"
+      odometry_topic="odometry"
+      parent_frame_id="world"
       mass_odometry_sensor="0.00001"
       measurement_divisor="1"
@@ -72,5 +72,5 @@
       odometry_map=""
       image_scale=""
-    >
+      >
       <inertia ixx="0.00001" ixy="0.0" ixz="0.0" iyy="0.00001" iyz="0.0" izz="0.00001" /> <!-- [kg·m^2] [kg·m^2] [kg·m^2] [kg·m^2] [kg·m^2] [kg·m^2] -->
       <origin xyz="0.0 0.0 0.0" rpy="0.0 0.0 0.0" />

File: rotors_description/urdf/iris.gazebo.xacro (robot description, xacro)
@@ -5,5 +5,5 @@
   <xacro:property name="bag_file" value="iris.bag" />
   <!-- Instantiate iris "mechanics" -->
-  <xacro:include filename="$(find mav_description)/urdf/iris.urdf.xacro" />
+  <xacro:include filename="$(find rotors_description)/urdf/iris.urdf.xacro" />
   <!-- Create link and joint for a sensor -->
   <link name="pose_sensor1_link">
@@ -23,5 +23,5 @@
   <gazebo>
     <!-- IMU -->
-    <plugin filename="libmav_gazebo_imu_plugin.so" name="mav_gazebo_imu_plugin">
+    <plugin filename="librotors_gazebo_imu_plugin.so" name="rotors_gazebo_imu_plugin">
   	<!-- A good description of the IMU parameters can be found in the kalibr documentation:
   	     https://github.com/ethz-asl/kalibr/wiki/IMU-Noise-Model-and-Intrinsics -->
@@ -42,5 +42,5 @@
   <gazebo>
     <!-- Controller interface -->
-    <plugin name="controller_interface" filename="libmav_gazebo_controller_interface.so">
+    <plugin name="controller_interface" filename="librotors_gazebo_controller_interface.so">
       <robotNamespace>${namespace}</robotNamespace>
       <commandAttitudeThrustSubTopic>command/attitude</commandAttitudeThrustSubTopic>
@@ -55,5 +55,5 @@
   <gazebo>
     <!-- Generic 6D pose sensor plugin -->
-    <plugin filename="libmav_gazebo_pose_plugin.so" name="pose_sensor1">
+    <plugin filename="librotors_gazebo_pose_plugin.so" name="pose_sensor1">
       <linkName>pose_sensor1_link</linkName>
       <robotNamespace>${namespace}</robotNamespace>
@@ -72,5 +72,5 @@
     <!-- ROS Bag Plugin -->
     <xacro:if value="$(arg enable_logging)">
-      <plugin filename="libmav_gazebo_bag_plugin.so" name="rosbag">
+      <plugin filename="librotors_gazebo_bag_plugin.so" name="rosbag">
         <robotNamespace>${namespace}</robotNamespace>
         <bagFileName>$(arg log_file)</bagFileName>
@@ -86,5 +86,5 @@
   <!-- attach wing plugin -->
   <gazebo>
-    <plugin filename="libmav_gazebo_wing_model_plugin.so" name="wing_plugin">
+    <plugin filename="librotors_gazebo_wing_model_plugin.so" name="wing_plugin">
       <robotNamespace>${namespace}</robotNamespace>
       <linkName>base_link</linkName>

File: rotors_description/urdf/iris.urdf.xacro (robot description, xacro)
@@ -40,6 +40,6 @@
   </xacro:property>
   <!-- Included URDF Files -->
-  <xacro:include filename="$(find mav_description)/urdf/multirotor_base.urdf.xacro" />
-  <!-- <xacro:include filename="$(find mav_description)/urdf/vtol_wing.urdf.xacro" /> -->
+  <xacro:include filename="$(find rotors_description)/urdf/multirotor_base.urdf.xacro" />
+  <!-- <xacro:include filename="$(find rotors_description)/urdf/vtol_wing.urdf.xacro" /> -->
   <!-- Instantiate multirotor_base_macro once -->
   <xacro:multirotor_base_macro

File: rotors_description/urdf/iris.xacro (robot description, xacro)
@@ -41,5 +41,5 @@
   </xacro:property>
   <!-- Included URDF Files -->
-  <xacro:include filename="$(find mav_description)/urdf/multirotor_base.xacro" />
+  <xacro:include filename="$(find rotors_description)/urdf/multirotor_base.xacro" />
   <!-- Instantiate multirotor_base_macro once -->
   <xacro:multirotor_base_macro

File: rotors_description/urdf/iris_base.xacro (robot description, xacro)
@@ -1,7 +1,7 @@
 <?xml version="1.0"?>
 <robot name="iris" xmlns:xacro="http://ros.org/wiki/xacro">
-  <xacro:include filename="$(find mav_description)/urdf/component_snippets.xacro" />
+  <xacro:include filename="$(find rotors_description)/urdf/component_snippets.xacro" />
   <!-- Instantiate iris "mechanics" -->
-  <xacro:include filename="$(find mav_description)/urdf/iris.xacro" />
+  <xacro:include filename="$(find rotors_description)/urdf/iris.xacro" />
   <!-- Instantiate a controller. -->
   <xacro:controller_plugin_macro
@@ -49,12 +49,12 @@
     <!-- Mount a generic odometry sensor providing ground truth. -->
     <xacro:odometry_plugin_macro
-      namespace="${namespace}"
+      namespace="${namespace}/ground_truth"
       odometry_sensor_suffix="gt"
-      pose_topic=""
-      pose_with_covariance_topic="ground_truth/pose"
-      position_topic=""
-      transform_topic=""
-      odometry_topic="ground_truth/odometry"
-      tf_frame="ground_truth/firefly"
+      pose_topic="pose"
+      pose_with_covariance_topic="pose_with_covariance"
+      position_topic="position"
+      transform_topic="transform"
+      odometry_topic="odometry"
+      parent_frame_id="world"
       mass_odometry_sensor="0.00001"
       measurement_divisor="1"

File: rotors_description/urdf/multirotor_base.xacro (robot description, xacro)
@@ -216,5 +216,5 @@
         <geometry>
           <!-- <cylinder length="0.005" radius="${radius_rotor}"/> --> <!-- [m] -->
-          <!-- <mesh filename="package://mav_description/meshes/propeller_${direction}.dae" -->
+          <!-- <mesh filename="package://rotors_description/meshes/propeller_${direction}.dae" -->
           <mesh filename="package://rotors_description/meshes/${mesh}_${direction}.dae"
             scale="${mesh_scale}" />

File: rotors_description/urdf/static_camera.gazebo.xacro (robot description, xacro)
@@ -5,5 +5,5 @@
   <xacro:property name="bag_file" value="static_camera.bag" />
   <!-- Instantiate static_camera "mechanics" -->
-  <xacro:include filename="$(find mav_description)/urdf/static_camera.urdf.xacro" />
+  <xacro:include filename="$(find rotors_description)/urdf/static_camera.urdf.xacro" />
 <gazebo>
     <static>true</static>

File: rotors_description/urdf/vtol.gazebo.xacro (robot description, xacro)
@@ -5,5 +5,5 @@
   <xacro:property name="bag_file" value="vtol.bag" />
   <!-- Instantiate vtol "mechanics" -->
-  <xacro:include filename="$(find mav_description)/urdf/vtol.urdf.xacro" />
+  <xacro:include filename="$(find rotors_description)/urdf/vtol.urdf.xacro" />
   <!-- Create link and joint for a sensor -->
   <link name="pose_sensor1_link">
@@ -46,5 +46,5 @@
   <gazebo>
     <!-- Controller interface -->
-    <plugin name="controller_interface" filename="libmav_gazebo_controller_interface.so">
+    <plugin name="controller_interface" filename="librotors_gazebo_controller_interface.so">
       <robotNamespace>${namespace}</robotNamespace>
       <commandTopicAttitude>command/attitude</commandTopicAttitude>
@@ -59,5 +59,5 @@
   <gazebo>
     <!-- Generic 6D pose sensor plugin -->
-    <plugin filename="libmav_gazebo_pose_plugin.so" name="pose_sensor1">
+    <plugin filename="librotors_gazebo_pose_plugin.so" name="pose_sensor1">
       <linkName>pose_sensor1_link</linkName>
       <robotNamespace>${namespace}</robotNamespace>
@@ -76,5 +76,5 @@
     <!-- ROS Bag Plugin -->
     <xacro:if value="$(arg enable_logging)">
-      <plugin filename="libmav_gazebo_bag_plugin.so" name="rosbag">
+      <plugin filename="librotors_gazebo_bag_plugin.so" name="rosbag">
         <robotNamespace>${namespace}</robotNamespace>
         <bagFileName>$(arg log_file)</bagFileName>
@@ -90,5 +90,5 @@
   <!-- attach wing plugin -->
   <gazebo>
-    <plugin filename="libmav_gazebo_wing_model_plugin.so" name="wing_plugin">
+    <plugin filename="librotors_gazebo_wing_model_plugin.so" name="wing_plugin">
       <robotNamespace>${namespace}</robotNamespace>
       <linkName>base_link</linkName>

File: rotors_description/urdf/vtol.urdf.xacro (robot description, xacro)
@@ -34,6 +34,6 @@
   </xacro:property>
   <!-- Included URDF Files -->
-  <xacro:include filename="$(find mav_description)/urdf/multirotor_base.urdf.xacro" />
-  <!-- <xacro:include filename="$(find mav_description)/urdf/vtol_wing.urdf.xacro" /> -->
+  <xacro:include filename="$(find rotors_description)/urdf/multirotor_base.urdf.xacro" />
+  <!-- <xacro:include filename="$(find rotors_description)/urdf/vtol_wing.urdf.xacro" /> -->
   <!-- Instantiate multirotor_base_macro once -->
   <xacro:multirotor_base_macro

File: rotors_description/urdf/vtol_wing.urdf.xacro (robot description, xacro)
@@ -11,5 +11,5 @@
   		</joint>
   		<gazebo>
-	      	<plugin name="gazebo_wing_model_plugin" filename="libmav_gazebo_wing_model_plugin.so">
+	      	<plugin name="gazebo_wing_model_plugin" filename="librotors_gazebo_wing_model_plugin.so">
 	      		<robotNamespace>${namespace}</robotNamespace>
 		        <linkName>base_link</linkName>
