Commit message: QP linear constraints structure modified

File: rotors_description/urdf/closed_chain_qp.xacro (robot description, xacro)
@@ -4,8 +4,8 @@
   <xacro:property name="r1_width" value="0.04"/>
   <xacro:property name="r1_height" value="0.008"/>
-  <xacro:property name="r1_length" value="0.24"/> <!-- 0.35 -->
+  <xacro:property name="r1_length" value="0.35"/> <!-- 0.24 vs 0.35 -->
   <xacro:property name="r2_width" value="0.04"/>
   <xacro:property name="r2_height" value="0.008"/>
-  <xacro:property name="r2_length" value="0.35"/> <!-- 0.40 -->
+  <xacro:property name="r2_length" value="0.40"/> <!-- 0.35 vs 0.40 -->
   <xacro:property name="r3_width" value="0.04"/>
   <xacro:property name="r3_height" value="0.0015"/>

Commit message: dynamic params + correct aerial manipulator model functions

File: rotors_description/urdf/closed_chain_qp.xacro (robot description, xacro)
@@ -4,12 +4,12 @@
   <xacro:property name="r1_width" value="0.04"/>
   <xacro:property name="r1_height" value="0.008"/>
-  <xacro:property name="r1_length" value="0.35"/> <!-- 0.24 vs 0.35 -->
+  <xacro:property name="r1_length" value="0.24"/> <!-- 0.24 vs 0.35 -->
   <xacro:property name="r2_width" value="0.04"/>
   <xacro:property name="r2_height" value="0.008"/>
-  <xacro:property name="r2_length" value="0.40"/> <!-- 0.35 vs 0.40 -->
+  <xacro:property name="r2_length" value="0.35"/> <!-- 0.35 vs 0.40 -->
   <xacro:property name="r3_width" value="0.04"/>
   <xacro:property name="r3_height" value="0.0015"/>
   <xacro:property name="r3_length" value="0.14"/>
-  <xacro:property name="center_to_center_length" value="0.12"/>
+  <xacro:property name="center_to_center_length" value="0.10"/> <!-- 0.10 vs 0.12 -->
   <xacro:property name="end_effector_length" value="0.12"/>
   <xacro:property name="end_effector_radius" value="0.03"/>
@@ -466,7 +466,7 @@
 					<config joint_name="pitching" initial_position="0.0"/>
 					<config joint_name="left_1"  initial_position="2.488"/>
-					<config joint_name="left_2"  initial_position="-1.676"/>
+					<config joint_name="left_2"  initial_position="${0.8127-2.488}"/>
 					<config joint_name="right_1" initial_position="0.653"/>
-					<config joint_name="right_2" initial_position="1.676"/>
+					<config joint_name="right_2" initial_position="${2.3284-0.653}"/>
 				</initial_configuration>
 				<loop_closure_joints>

Commit message: bug fixed in servo motor plugin + params updated

File: rotors_description/urdf/closed_chain_qp.xacro (robot description, xacro)
@@ -2,4 +2,6 @@
 <robot xmlns:xacro="http://ros.org/wiki/xacro">
   <xacro:include filename="$(find rotors_description)/urdf/manipulator_snippets.xacro" />
+	<xacro:property name="meas_delay" value="0"/>
+	<xacro:property name="angle_noise" value="0.0"/>
   <xacro:property name="r1_width" value="0.04"/>
   <xacro:property name="r1_height" value="0.008"/>
@@ -395,7 +397,7 @@
 			maxAngle="${PI}"
     	measurement_divisor="1"
-    	measurement_delay="0"
+    	measurement_delay="${meas_delay}"
     	unknown_delay="0.0"
-		  noise_normal_angle="0.0"
+		  noise_normal_angle="${angle_noise}"
 		  noise_normal_angular_velocity="0.0"
 		  noise_normal_torque="0.0"
@@ -423,7 +425,7 @@
 			maxAngle="${PI}"
     	measurement_divisor="1"
-    	measurement_delay="0"
+    	measurement_delay="${meas_delay}"
     	unknown_delay="0.0"
-		  noise_normal_angle="0.0"
+		  noise_normal_angle="${angle_noise}"
 		  noise_normal_angular_velocity="0.0"
 		  noise_normal_torque="0.0"
@@ -451,7 +453,7 @@
 			maxAngle="${PI}"
     	measurement_divisor="1"
-    	measurement_delay="0"
+    	measurement_delay="${meas_delay}"
     	unknown_delay="0.0"
-		  noise_normal_angle="0.0"
+		  noise_normal_angle="${angle_noise}"
 		  noise_normal_angular_velocity="0.0"
 		  noise_normal_torque="0.0"
