Commit message: changes in namespaces

File: rotors_description/urdf/closed_chain.xacro (robot description, xacro)
@@ -81,9 +81,19 @@
   <xacro:macro name="closed_chain_macro"
     params="namespace parent_link *origin">
-    <joint name="${namespace}/fixed_joint" type="fixed">
+    <xacro:revolute_joint_macro
+      namespace="${namespace}"
+      joint_name="${namespace}/pitching"
+      parent_link="${parent_link}"
+      child_link="${namespace}/r3"
+      axis="1 0 0"
+      friction="0"
+      damping="0.1">
+      <xacro:insert_block name="origin" />
+    </xacro:revolute_joint_macro>
+    <!-- <joint name="${namespace}/fixed_joint" type="fixed">
       <parent link="${parent_link}"/>
       <child  link="${namespace}/r3"/>
       <xacro:insert_block name="origin" />
-    </joint>
+    </joint> -->
   <!-- Here we define base link of closed kinematic chain -->
   <link name="${namespace}/r3">
@@ -174,7 +184,7 @@
   <xacro:revolute_joint_macro
     namespace="${namespace}"
-    joint_name="left_1"
-    parent_link="r3"
-    child_link="r1_left"
+    joint_name="${namespace}/left_1"
+    parent_link="${namespace}/r3"
+    child_link="${namespace}/r1_left"
     axis="0 0 1"
     friction="0"
@@ -184,7 +194,7 @@
   <xacro:revolute_joint_macro
     namespace="${namespace}"
-    joint_name="right_1"
-    parent_link="r3"
-    child_link="r1_right"
+    joint_name="${namespace}/right_1"
+    parent_link="${namespace}/r3"
+    child_link="${namespace}/r1_right"
     axis="0 0 1"
     friction="0"
@@ -194,7 +204,7 @@
   <xacro:revolute_joint_macro
     namespace="${namespace}"
-    joint_name="left_2"
-    parent_link="r1_left"
-    child_link="r2_left"
+    joint_name="${namespace}/left_2"
+    parent_link="${namespace}/r1_left"
+    child_link="${namespace}/r2_left"
     axis="0 0 1"
     friction="0"
@@ -204,7 +214,7 @@
   <xacro:revolute_joint_macro
     namespace="${namespace}"
-    joint_name="right_2"
-    parent_link="r1_right"
-    child_link="r2_right"
+    joint_name="${namespace}/right_2"
+    parent_link="${namespace}/r1_right"
+    child_link="${namespace}/r2_right"
     axis="0 0 1"
     friction="0"
@@ -214,7 +224,7 @@
   <xacro:gazebo_revolute_joint_macro
     namespace="${namespace}"
-    joint_name="closing"
-    parent_link="r2_left"
-    child_link="r2_right"
+    joint_name="${namespace}/closing"
+    parent_link="${namespace}/r2_left"
+    child_link="${namespace}/r2_right"
     pose="${r2_length} 0 0 0 0 0"
     axis="0 0 1"
@@ -227,17 +237,9 @@
     effort_limit="1000">
   </xacro:gazebo_revolute_joint_macro>
-  <!-- params="namespace suffix parent_link child_link *origin"> -->
-  <!-- <xacro:fixed_joint_macro
-    namespace="${namespace}"
-    suffix="end_effector"
-    parent_link="r2_left"
-    child_link="end_effector">
-    <origin xyz="${r2_length} 0 0" rpy="0 ${PI/2} 0"/>
-  </xacro:fixed_joint_macro> -->
-  <xacro:revolute_joint_macro
-    namespace="${namespace}"
-    joint_name="end_effector"
-    parent_link="r2_left"
-    child_link="end_effector"
+  <xacro:revolute_joint_macro
+    namespace="${namespace}"
+    joint_name="${namespace}/end_effector"
+    parent_link="${namespace}/r2_left"
+    child_link="${namespace}/end_effector"
     axis="0 0 1"
     friction="0"
@@ -256,7 +258,7 @@
  <xacro:servo_motor_macro
    namespace="${namespace}"
-   motor_name="left_motor"
-   parent_link="r3"
-   actuated_joint="left_1"
+   motor_name="motor_left"
+   parent_link="${namespace}/r3"
+   actuated_joint="${namespace}/left_1"
    motor_model="generic_servo1"
    maxTorque="3"
@@ -264,5 +266,5 @@
    Kp="30.0"
    Kd="0.05"
-   Ki="0.4"
+   Ki="0.40"
    minAngle="${-PI}"
    maxAngle="${PI}"
@@ -275,7 +277,7 @@
  <xacro:servo_motor_macro
    namespace="${namespace}"
-   motor_name="motor_right_1"
-   parent_link="r3"
-   actuated_joint="right_1"
+   motor_name="motor_right"
+   parent_link="${namespace}/r3"
+   actuated_joint="${namespace}/right_1"
    motor_model="generic_servo2"
    maxTorque="3"
@@ -283,5 +285,5 @@
    Kp="30.0"
    Kd="0.05"
-   Ki="0.4"
+   Ki="0.40"
    minAngle="${-PI}"
    maxAngle="${PI}"
@@ -295,6 +297,6 @@
    namespace="${namespace}"
    motor_name="motor_end_effector"
-   parent_link="r2_left"
-   actuated_joint="end_effector"
+   parent_link="${namespace}/r2_left"
+   actuated_joint="${namespace}/end_effector"
    motor_model="generic_servo3"
    maxTorque="0.8"
@@ -302,5 +304,5 @@
    Kp="10.0"
    Kd="0.05"
-   Ki="0.4"
+   Ki="0.40"
    minAngle="${-PI}"
    maxAngle="${PI}"
@@ -310,5 +312,25 @@
    <origin xyz="${r2_length} 0 0.02" rpy="-1.57 0 0"/>
    <xacro:insert_block name="generic_servo_inertial"/>
- </xacro:servo_motor_macro> >
+ </xacro:servo_motor_macro>
+ >
+ <xacro:servo_motor_macro
+   namespace="${namespace}"
+   motor_name="motor_pitching"
+   parent_link="${parent_link}"
+   actuated_joint="${namespace}/pitching"
+   motor_model="generic_servo0"
+   maxTorque="3"
+   noLoadSpeed="0.11"
+   Kp="30.0"
+   Kd="0.05"
+   Ki="0.40"
+   minAngle="${-PI}"
+   maxAngle="${PI}"
+   enable_visual="true"
+   visual_scale="1"
+   color="Red">
+   <origin xyz="0 0 0.02" rpy="0 0 0"/>
+   <xacro:insert_block name="generic_servo_inertial"/>
+ </xacro:servo_motor_macro>
 <!-- Initial configuration plugin -->
 <gazebo>
@@ -316,8 +338,9 @@
     <robotNamespace>${namespace}</robotNamespace>
  <initial_configuration>
-   <config joint_name="left_1" initial_position="0.3415"/>
-   <config joint_name="left_2" initial_position="2.2942"/>
+   <config joint_name="left_1"  initial_position="0.3415"/>
+   <config joint_name="left_2"  initial_position="2.2942"/>
    <config joint_name="right_1" initial_position="2.8001"/>
    <config joint_name="right_2" initial_position="-2.2942"/>
+   <config joint_name="pitching" initial_position="0"/>
  </initial_configuration>
  <loop_closure_joints>

File: rotors_description/urdf/manipulator_snippets.xacro (robot description, xacro)
@@ -26,8 +26,8 @@
             lower_limit upper_limit effort_limit">
     <gazebo>
-      <joint name="${namespace}/${joint_name}" type="revolute">
+      <joint name="${joint_name}" type="revolute">
         <pose>${pose}</pose>
-        <child>${namespace}/${child_link}</child>
-        <parent>${namespace}/${parent_link}</parent>
+        <child>${child_link}</child>
+        <parent>${parent_link}</parent>
         <axis>
           <xyz>${axis}</xyz>
@@ -50,7 +50,7 @@
   <xacro:macro name="fixed_joint_macro"
     params="namespace joint_name parent_link child_link *origin">
-            <joint name="${namespace}/${joint_name}" type="fixed">
-              <parent link="${namespace}/${parent_link}"/>
-              <child  link="${namespace}/${child_link}"/>
+            <joint name="${joint_name}" type="fixed">
+              <parent link="${parent_link}"/>
+              <child  link="${child_link}"/>
               <xacro:insert_block name="origin" />
             </joint>
@@ -59,7 +59,7 @@
   <xacro:macro name="revolute_joint_macro"
     params="namespace joint_name parent_link child_link axis friction damping *origin">
-            <joint name="${namespace}/${joint_name}" type="continuous">
-              <parent link="${namespace}/${parent_link}"/>
-              <child  link="${namespace}/${child_link}"/>
+            <joint name="${joint_name}" type="continuous">
+              <parent link="${parent_link}"/>
+              <child  link="${child_link}"/>
               <axis xyz="${axis}"/>
               <dynamics damping="${damping}"/>
@@ -73,7 +73,7 @@
     params="namespace joint_name parent_link child_link axis friction damping lower_limit upper_limit
             effort_limit velocity_limit *origin">
-            <joint name="${namespace}/${joint_name}" type="prismatic">
-              <parent link="${namespace}/${parent_link}"/>
-              <child link="${namespace}/${child_link}"/>
+            <joint name="${joint_name}" type="prismatic">
+              <parent link="${parent_link}"/>
+              <child link="${child_link}"/>
               <axis xyz="${axis}"/>
               <dynamics damping="${damping}"/>
@@ -101,5 +101,5 @@
             </gazebo>
             <joint name="${namespace}/${motor_name}" type="revolute">
-              <parent link="${namespace}/${parent_link}"/>
+              <parent link="${parent_link}"/>
               <child link="${namespace}/${motor_name}"/>
               <xacro:insert_block name="origin" />
@@ -109,5 +109,5 @@
               <plugin name="${namespace}/${motor_name}" filename="librotors_gazebo_servo_motor_plugin.so">
                 <robotNamespace>${namespace}</robotNamespace>
-                <jointName>${namespace}/${actuated_joint}</jointName>
+                <jointName>${actuated_joint}</jointName>
                 <motorModel>${motor_model}</motorModel>
                 <commandSubTopic>command/${motor_name}</commandSubTopic>

Commit message: add links meshes

File: rotors_description/urdf/closed_chain.xacro (robot description, xacro)
@@ -6,5 +6,5 @@
   <xacro:property name="r1_length" value="0.24"/>
   <xacro:property name="r2_width" value="0.05"/>
-  <xacro:property name="r2_height" value="0.01"/>
+  <xacro:property name="r2_height" value="0.008"/>
   <xacro:property name="r2_length" value="0.35"/>
   <xacro:property name="r3_width" value="0.05"/>
@@ -17,5 +17,5 @@
   </xacro:property>
   <xacro:property name="r3_inertial">
-    <mass value="0.02"/>
+    <mass value="0.002"/>
     <inertia ixx="0.0031" ixy="0.0" ixz="0.0"
     iyy="0.0061" iyz="0.0"
@@ -34,7 +34,7 @@
   </xacro:property>
   <xacro:property name="r2_inertial">
-    <mass value="0.02"/>
-    <inertia ixx="0.0031" ixy="0.0" ixz="0.0"
-    iyy="0.0061" iyz="0.0"
+    <mass value="0.0025"/>
+    <inertia ixx="0.0021" ixy="0.0" ixz="0.0"
+    iyy="0.0031" iyz="0.0"
     izz="0.0081"/>
   </xacro:property>
@@ -51,7 +51,7 @@
   </xacro:property>
   <xacro:property name="r1_inertial">
-    <mass value="0.02"/>
+    <mass value="0.0025"/>
     <inertia ixx="0.0031" ixy="0.0" ixz="0.0"
-    iyy="0.0051" iyz="0.0"
+    iyy="0.0031" iyz="0.0"
     izz="0.0081"/>
   </xacro:property>
@@ -117,6 +117,11 @@
     </collision>
     <visual>
-      <xacro:insert_block name="r1_frame"/>
-      <xacro:insert_block name="r1_geometry"/>
+      <!-- <xacro:insert_block name="r1_frame"/> -->
+      <!-- <xacro:insert_block name="r1_geometry"/> -->
+      <!-- <origin xyz="0.03 0.115 -0.005" rpy="1.57 0 -0.3"/> -->
+      <origin xyz="${r1_length/2} 0 -0.004" rpy="1.57 0 0"/>
+      <geometry>
+          <mesh filename="package://rotors_description/meshes/delta_arm_meshes/R1_v2.dae" scale="0.001 0.001 0.001" />
+      </geometry>
     </visual>
     <inertial>
@@ -131,6 +136,11 @@
     </collision>
     <visual>
-      <xacro:insert_block name="r1_frame"/>
-      <xacro:insert_block name="r1_geometry"/>
+      <!-- <xacro:insert_block name="r1_frame"/>
+      <xacro:insert_block name="r1_geometry"/> -->
+      <!-- <origin xyz="0.03 -0.115 0.008" rpy="-1.57 0 0.3"/> -->
+       <origin xyz="${r1_length/2} 0 0.012" rpy="-1.57 0 0"/>
+      <geometry>
+          <mesh filename="package://rotors_description/meshes/delta_arm_meshes/R1_v2.dae" scale="0.001 0.001 0.001" />
+      </geometry>
     </visual>
     <inertial>
@@ -145,6 +155,10 @@
     </collision>
     <visual>
-      <xacro:insert_block name="r2_frame"/>
-      <xacro:insert_block name="r2_geometry"/>
+      <!-- <xacro:insert_block name="r2_frame"/>
+      <xacro:insert_block name="r2_geometry"/> -->
+      <origin xyz="${r2_length/2} 0 -0.026" rpy="1.57 0 0"/>
+      <geometry>
+          <mesh filename="package://rotors_description/meshes/delta_arm_meshes/R2_v2.dae" scale="0.001 0.001 0.001" />
+      </geometry>
     </visual>
     <inertial>
@@ -159,6 +173,10 @@
     </collision>
     <visual>
-      <xacro:insert_block name="r2_frame"/>
-      <xacro:insert_block name="r2_geometry"/>
+      <!-- <xacro:insert_block name="r2_frame"/>
+      <xacro:insert_block name="r2_geometry"/> -->
+      <origin xyz="${r2_length/2} 0 -0.005" rpy="1.57 0 0"/>
+      <geometry>
+          <mesh filename="package://rotors_description/meshes/delta_arm_meshes/R2_v2.dae" scale="0.001 0.001 0.001" />
+      </geometry>
     </visual>
     <inertial>
@@ -173,6 +191,10 @@
     </collision>
     <visual>
-      <xacro:insert_block name="end_effector_frame"/>
-      <xacro:insert_block name="end_effector_geometry"/>
+      <!-- <xacro:insert_block name="end_effector_frame"/>
+      <xacro:insert_block name="end_effector_geometry"/> -->
+      <origin xyz="0 0 -0.015" rpy="1.57 0 1.2"/>
+      <geometry>
+          <mesh filename="package://rotors_description/meshes/delta_arm_meshes/end_effector_plate.dae" scale="0.001 0.001 0.001" />
+      </geometry>
     </visual>
     <inertial>
@@ -262,5 +284,5 @@
    actuated_joint="${namespace}/left_1"
    motor_model="generic_servo1"
-   maxTorque="3"
+   maxTorque="2"
    noLoadSpeed="0.11"
    Kp="30.0"
@@ -281,5 +303,5 @@
    actuated_joint="${namespace}/right_1"
    motor_model="generic_servo2"
-   maxTorque="3"
+   maxTorque="2"
    noLoadSpeed="0.11"
    Kp="30.0"
@@ -320,5 +342,5 @@
    actuated_joint="${namespace}/pitching"
    motor_model="generic_servo0"
-   maxTorque="3"
+   maxTorque="2"
    noLoadSpeed="0.11"
    Kp="30.0"
