Commit message: update manipulator model

File: rotors_description/urdf/closed_chain.xacro (robot description, xacro)
@@ -2,13 +2,14 @@
 <robot xmlns:xacro="http://ros.org/wiki/xacro">
   <xacro:include filename="$(find rotors_description)/urdf/manipulator_snippets.xacro" />
-  <xacro:property name="r1_width" value="0.05"/>
-  <xacro:property name="r1_height" value="0.01"/>
+  <xacro:property name="r1_width" value="0.04"/>
+  <xacro:property name="r1_height" value="0.008"/>
   <xacro:property name="r1_length" value="0.24"/>
-  <xacro:property name="r2_width" value="0.05"/>
+  <xacro:property name="r2_width" value="0.04"/>
   <xacro:property name="r2_height" value="0.008"/>
   <xacro:property name="r2_length" value="0.35"/>
-  <xacro:property name="r3_width" value="0.05"/>
-  <xacro:property name="r3_height" value="0.01"/>
-  <xacro:property name="r3_length" value="0.16"/>
+  <xacro:property name="r3_width" value="0.04"/>
+  <xacro:property name="r3_height" value="0.0015"/>
+  <xacro:property name="r3_length" value="0.14"/>
+  <xacro:property name="center_to_center_length" value="0.1"/>
   <xacro:property name="end_effector_length" value="0.12"/>
   <xacro:property name="end_effector_radius" value="0.03"/>
@@ -78,5 +79,7 @@
     </geometry>
   </xacro:property>
-<!-- macro used to define a closed chain -->
+<!-- ################################################################################################# -->
+<!-- #################################### Manipulator Macro ########################################## -->
+<!-- ################################################################################################# -->
   <xacro:macro name="closed_chain_macro"
     params="namespace parent_link *origin">
@@ -84,11 +87,17 @@
       namespace="${namespace}"
       joint_name="${namespace}/pitching"
-      parent_link="${parent_link}"
+      parent_link="${namespace}/r0"
       child_link="${namespace}/r3"
       axis="1 0 0"
       friction="0"
       damping="0.1">
-      <xacro:insert_block name="origin" />
+      <origin xyz="0 0 -0.05" rpy="0 0 0"/>
     </xacro:revolute_joint_macro>
+    <joint name="my_joint" type="floating">
+        <parent link="${parent_link}"/>
+        <child link="${namespace}/r0"/>
+        <xacro:insert_block name="origin" />
+        <dynamics damping="0.0" friction="0.0"/>
+     </joint>
     <!-- <joint name="${namespace}/fixed_joint" type="fixed">
       <parent link="${parent_link}"/>
@@ -97,12 +106,18 @@
     </joint> -->
   <!-- Here we define base link of closed kinematic chain -->
-  <link name="${namespace}/r3">
-   <collision>
-     <xacro:insert_block name="r3_frame"/>
-     <xacro:insert_block name="r3_geometry"/>
-    </collision>
-    <visual>
-      <xacro:insert_block name="r3_frame"/>
-      <xacro:insert_block name="r3_geometry"/>
+  <link name="${namespace}/r0">
+   <collision>
+     <!-- <xacro:insert_block name="r3_frame"/>
+     <xacro:insert_block name="r3_geometry"/> -->
+     <origin xyz="0 0 0" rpy="0 0 0"/>
+     <geometry>
+         <mesh filename="package://rotors_description/meshes/delta_arm_meshes/pitching_base.dae" scale="0.001 0.001 0.001" />
+     </geometry>
+    </collision>
+    <visual>
+        <origin xyz="0 0 0" rpy="0 0 0"/>
+        <geometry>
+            <mesh filename="package://rotors_description/meshes/delta_arm_meshes/pitching_base.dae" scale="0.001 0.001 0.001" />
+        </geometry>
     </visual>
     <inertial>
@@ -111,8 +126,32 @@
     </inertial>
   </link>
+  <link name="${namespace}/r3">
+   <collision>
+     <!-- <xacro:insert_block name="r3_frame"/>
+     <xacro:insert_block name="r3_geometry"/> -->
+     <origin xyz="0 0 0" rpy="0 0 0"/>
+     <geometry>
+         <mesh filename="package://rotors_description/meshes/delta_arm_meshes/pitching_base.dae" scale="0.001 0.001 0.001" />
+     </geometry>
+    </collision>
+    <visual>
+            <origin xyz="0 0 0" rpy="0 0 0"/>
+            <geometry>
+                <mesh filename="package://rotors_description/meshes/delta_arm_meshes/pitching_base.dae" scale="0.001 0.001 0.001" />
+            </geometry>
+    </visual>
+    <inertial>
+      <xacro:insert_block name="r3_frame"/>
+      <xacro:insert_block name="r3_inertial"/>
+    </inertial>
+  </link>
   <link name="${namespace}/r1_left">
    <collision>
-     <xacro:insert_block name="r1_frame"/>
-     <xacro:insert_block name="r1_geometry"/>
+     <!-- <xacro:insert_block name="r1_frame"/>
+     <xacro:insert_block name="r1_geometry"/> -->
+     <origin xyz="0 0 0" rpy="0 0 0"/>
+     <geometry>
+         <mesh filename="package://rotors_description/meshes/delta_arm_meshes/R1_v2_left.dae" scale="0.001 0.001 0.001" />
+     </geometry>
     </collision>
     <visual>
@@ -120,5 +159,28 @@
       <!-- <xacro:insert_block name="r1_geometry"/> -->
       <!-- <origin xyz="0.03 0.115 -0.005" rpy="1.57 0 -0.3"/> -->
-      <origin xyz="${r1_length/2} 0 -0.004" rpy="1.57 0 0"/>
+      <origin xyz="0 0 0" rpy="0 0 0"/>
+      <geometry>
+          <mesh filename="package://rotors_description/meshes/delta_arm_meshes/R1_v2_left.dae" scale="0.001 0.001 0.001" />
+      </geometry>
+    </visual>
+    <inertial>
+      <xacro:insert_block name="r1_frame"/>
+      <xacro:insert_block name="r1_inertial"/>
+    </inertial>
+  </link>
+  <link name="${namespace}/r1_right">
+   <collision>
+     <!-- <xacro:insert_block name="r1_frame"/>
+     <xacro:insert_block name="r1_geometry"/> -->
+     <origin xyz="0 0 0" rpy="0 0 0"/>
+    <geometry>
+        <mesh filename="package://rotors_description/meshes/delta_arm_meshes/R1_v2.dae" scale="0.001 0.001 0.001" />
+    </geometry>
+    </collision>
+    <visual>
+      <!-- <xacro:insert_block name="r1_frame"/>
+      <xacro:insert_block name="r1_geometry"/> -->
+      <!-- <origin xyz="0.03 -0.115 0.008" rpy="-1.57 0 0.3"/> -->
+       <origin xyz="0 0 0" rpy="0 0 0"/>
       <geometry>
           <mesh filename="package://rotors_description/meshes/delta_arm_meshes/R1_v2.dae" scale="0.001 0.001 0.001" />
@@ -130,32 +192,17 @@
     </inertial>
   </link>
-  <link name="${namespace}/r1_right">
-   <collision>
-     <xacro:insert_block name="r1_frame"/>
-     <xacro:insert_block name="r1_geometry"/>
-    </collision>
-    <visual>
-      <!-- <xacro:insert_block name="r1_frame"/>
-      <xacro:insert_block name="r1_geometry"/> -->
-      <!-- <origin xyz="0.03 -0.115 0.008" rpy="-1.57 0 0.3"/> -->
-       <origin xyz="${r1_length/2} 0 0.012" rpy="-1.57 0 0"/>
-      <geometry>
-          <mesh filename="package://rotors_description/meshes/delta_arm_meshes/R1_v2.dae" scale="0.001 0.001 0.001" />
-      </geometry>
-    </visual>
-    <inertial>
-      <xacro:insert_block name="r1_frame"/>
-      <xacro:insert_block name="r1_inertial"/>
-    </inertial>
-  </link>
   <link name="${namespace}/r2_left">
    <collision>
-     <xacro:insert_block name="r2_frame"/>
-     <xacro:insert_block name="r2_geometry"/>
+     <!-- <xacro:insert_block name="r2_frame"/>
+     <xacro:insert_block name="r2_geometry"/> -->
+     <origin xyz="0 0 0" rpy="0 0 0"/>
+     <geometry>
+         <mesh filename="package://rotors_description/meshes/delta_arm_meshes/R2_v2.dae" scale="0.001 0.001 0.001" />
+     </geometry>
     </collision>
     <visual>
       <!-- <xacro:insert_block name="r2_frame"/>
       <xacro:insert_block name="r2_geometry"/> -->
-      <origin xyz="${r2_length/2} 0 -0.026" rpy="1.57 0 0"/>
+      <origin xyz="0 0 0" rpy="0 0 0"/>
       <geometry>
           <mesh filename="package://rotors_description/meshes/delta_arm_meshes/R2_v2.dae" scale="0.001 0.001 0.001" />
@@ -169,11 +216,15 @@
   <link name="${namespace}/r2_right">
    <collision>
-     <xacro:insert_block name="r2_frame"/>
-     <xacro:insert_block name="r2_geometry"/>
+     <!-- <xacro:insert_block name="r2_frame"/>
+     <xacro:insert_block name="r2_geometry"/> -->
+     <origin xyz="0 0 0" rpy="0 0 0"/>
+     <geometry>
+         <mesh filename="package://rotors_description/meshes/delta_arm_meshes/R2_v2.dae" scale="0.001 0.001 0.001" />
+     </geometry>
     </collision>
     <visual>
       <!-- <xacro:insert_block name="r2_frame"/>
       <xacro:insert_block name="r2_geometry"/> -->
-      <origin xyz="${r2_length/2} 0 -0.005" rpy="1.57 0 0"/>
+      <origin xyz="0 0 0" rpy="0 0 0"/>
       <geometry>
           <mesh filename="package://rotors_description/meshes/delta_arm_meshes/R2_v2.dae" scale="0.001 0.001 0.001" />
@@ -187,11 +238,15 @@
   <link name="${namespace}/end_effector">
    <collision>
-     <xacro:insert_block name="end_effector_frame"/>
-     <xacro:insert_block name="end_effector_geometry"/>
+     <!-- <xacro:insert_block name="end_effector_frame"/>
+     <xacro:insert_block name="end_effector_geometry"/> -->
+     <origin xyz="0 0 -0.015" rpy="0 0 1.2"/>
+     <geometry>
+         <mesh filename="package://rotors_description/meshes/delta_arm_meshes/end_effector_plate.dae" scale="0.001 0.001 0.001" />
+     </geometry>
     </collision>
     <visual>
       <!-- <xacro:insert_block name="end_effector_frame"/>
       <xacro:insert_block name="end_effector_geometry"/> -->
-      <origin xyz="0 0 -0.015" rpy="1.57 0 1.2"/>
+      <origin xyz="0 0 -0.015" rpy="0 0 1.2"/>
       <geometry>
           <mesh filename="package://rotors_description/meshes/delta_arm_meshes/end_effector_plate.dae" scale="0.001 0.001 0.001" />
@@ -212,5 +267,5 @@
     friction="0"
     damping="0.1">
-    <origin xyz="${r3_length/2} 0 -0.01" rpy="0 0 0"/>
+    <origin xyz="${-center_to_center_length/2} 0 -0.005" rpy="0 0 0"/>
   </xacro:revolute_joint_macro>
   <xacro:revolute_joint_macro
@@ -222,5 +277,5 @@
     friction="0"
     damping="0.1">
-    <origin xyz="${-r3_length/2} 0 -0.015" rpy="0 0 0"/>
+    <origin xyz="${center_to_center_length/2} 0 -0.005" rpy="0 0 0"/>
   </xacro:revolute_joint_macro>
   <xacro:revolute_joint_macro
@@ -232,5 +287,5 @@
     friction="0"
     damping="0.1">
-    <origin xyz="${r1_length} 0 0.015" rpy="0 0 0"/>
+    <origin xyz="${r1_length} 0 0.01" rpy="0 0 0"/>
   </xacro:revolute_joint_macro>
   <xacro:revolute_joint_macro
@@ -242,5 +297,5 @@
     friction="0"
     damping="0.1">
-    <origin xyz="${r1_length} 0 0.015" rpy="0 0 0"/>
+    <origin xyz="${r1_length} 0 -0.01" rpy="0 0 0"/>
   </xacro:revolute_joint_macro>
   <xacro:gazebo_revolute_joint_macro
@@ -294,5 +349,5 @@
    visual_scale="1"
    color="Blue">
-   <origin xyz="${r3_length/2} 0 0.02" rpy="-1.57 0 0"/>
+   <origin xyz="${center_to_center_length/2} 0 0" rpy="0 0 0"/>
    <xacro:insert_block name="generic_servo_inertial"/>
  </xacro:servo_motor_macro>
@@ -313,5 +368,5 @@
    visual_scale="1"
    color="Red">
-   <origin xyz="${-r3_length/2} 0 0.02" rpy="-1.57 0 0"/>
+   <origin xyz="${-center_to_center_length/2} 0 0" rpy="0 0 0"/>
    <xacro:insert_block name="generic_servo_inertial"/>
  </xacro:servo_motor_macro>
@@ -339,5 +394,5 @@
    namespace="${namespace}"
    motor_name="motor_pitching"
-   parent_link="${parent_link}"
+   parent_link="${namespace}/r0"
    actuated_joint="${namespace}/pitching"
    motor_model="generic_servo0"
@@ -352,5 +407,5 @@
    visual_scale="1"
    color="Red">
-   <origin xyz="0 0 0.02" rpy="0 0 0"/>
+   <origin xyz="0 0.02 -0.02" rpy="1.57 1.57 0"/>
    <xacro:insert_block name="generic_servo_inertial"/>
  </xacro:servo_motor_macro>
@@ -360,9 +415,8 @@
     <robotNamespace>${namespace}</robotNamespace>
  <initial_configuration>
-   <config joint_name="left_1"  initial_position="0.3415"/>
-   <config joint_name="left_2"  initial_position="2.2942"/>
-   <config joint_name="right_1" initial_position="2.8001"/>
-   <config joint_name="right_2" initial_position="-2.2942"/>
-   <config joint_name="pitching" initial_position="0"/>
+   <config joint_name="left_1"  initial_position="2.488"/>
+   <config joint_name="left_2"  initial_position="-1.676"/>
+   <config joint_name="right_1" initial_position="0.653"/>
+   <config joint_name="right_2" initial_position="1.676"/>
  </initial_configuration>
  <loop_closure_joints>
@@ -371,4 +425,15 @@
  </plugin>
 </gazebo>
+<gazebo>
+  <plugin name="6dof_shock_absorber" filename="librotors_gazebo_six_dof_shock_absorber_plugin.so">
+    <robotNamespace>${namespace}</robotNamespace>
+    <ParentLinkName>${parent_link} </ParentLinkName>
+    <ChildLinkName>${namespace}/r0 </ChildLinkName>
+    <translational_spring_constant>20 20 100</translational_spring_constant>
+    <translational_damper_constant>5 5 20</translational_damper_constant>
+    <rotational_spring_constant>8 15 8</rotational_spring_constant>
+    <rotational_damper_constant>1 1 1</rotational_damper_constant>
+ </plugin>
+</gazebo>
 </xacro:macro>
 </robot>

Commit message: some bugs fixed + changed inertial params

File: rotors_description/urdf/closed_chain.xacro (robot description, xacro)
@@ -18,8 +18,8 @@
   </xacro:property>
   <xacro:property name="r3_inertial">
-    <mass value="0.002"/>
-    <inertia ixx="0.0031" ixy="0.0" ixz="0.0"
-    iyy="0.0061" iyz="0.0"
-    izz="0.0081"/>
+    <mass value="0.001"/>
+    <inertia ixx="0.0001" ixy="0.0" ixz="0.0"
+    iyy="0.0001" iyz="0.0"
+    izz="0.0001"/>
   </xacro:property>
   <xacro:property name="r3_geometry">
@@ -35,8 +35,8 @@
   </xacro:property>
   <xacro:property name="r2_inertial">
-    <mass value="0.0025"/>
-    <inertia ixx="0.0021" ixy="0.0" ixz="0.0"
-    iyy="0.0031" iyz="0.0"
-    izz="0.0081"/>
+    <mass value="0.0015"/>
+    <inertia ixx="0.00000229511" ixy="0.0" ixz="0.00000000098"
+    iyy="0.00018644679" iyz="0.0"
+    izz="0.00018419229"/>
   </xacro:property>
   <xacro:property name="r2_geometry">
@@ -52,8 +52,8 @@
   </xacro:property>
   <xacro:property name="r1_inertial">
-    <mass value="0.0025"/>
-    <inertia ixx="0.0031" ixy="0.0" ixz="0.0"
-    iyy="0.0031" iyz="0.0"
-    izz="0.0081"/>
+    <mass value="0.0012"/>
+    <inertia ixx="0.00000948062" ixy="0.0" ixz="-0.00001716204"
+    iyy="0.0000730949" iyz="0.0"
+    izz="0.00006364922"/>
   </xacro:property>
   <xacro:property name="r1_geometry">
@@ -69,8 +69,8 @@
   </xacro:property>
   <xacro:property name="end_effector_inertial">
-    <mass value="0.02"/>
-    <inertia ixx="0.0031" ixy="0.0" ixz="0.0"
-    iyy="0.0051" iyz="0.0"
-    izz="0.0081"/>
+    <mass value="0.001"/>
+    <inertia ixx="0.0001" ixy="0.0" ixz="0.0"
+    iyy="0.0001" iyz="0.0"
+    izz="0.0001"/>
   </xacro:property>
   <xacro:property name="end_effector_geometry">
@@ -314,5 +314,6 @@
     effort_limit="1000">
   </xacro:gazebo_revolute_joint_macro>
-  <xacro:revolute_joint_macro
+<!--
+	<xacro:revolute_joint_macro
     namespace="${namespace}"
     joint_name="${namespace}/end_effector"
@@ -324,8 +325,16 @@
     <origin xyz="${r2_length} 0 0" rpy="0 0 0"/>
   </xacro:revolute_joint_macro>
+-->
+  <xacro:fixed_joint_macro
+    namespace="${namespace}"
+    joint_name="${namespace}/end_effector"
+    parent_link="${namespace}/r2_left"
+    child_link="${namespace}/end_effector">
+    <origin xyz="${r2_length} 0 0" rpy="0 0 0"/>
+	</xacro:fixed_joint_macro>
   <!-- Attach actuators -->
   <xacro:property name="generic_servo_inertial">
     <inertial>
-    <mass value="0.02"/>
+    <mass value="0.070"/>
     <inertia ixx="0.001" ixy="0.0" ixz="0.0"
     iyy="0.001" iyz="0.0"
@@ -371,4 +380,5 @@
    <xacro:insert_block name="generic_servo_inertial"/>
  </xacro:servo_motor_macro>
+<!--
  <xacro:servo_motor_macro
    namespace="${namespace}"
@@ -390,4 +400,5 @@
    <xacro:insert_block name="generic_servo_inertial"/>
  </xacro:servo_motor_macro>
+-->
  >
  <xacro:servo_motor_macro

Commit message: debug in progress

File: rotors_description/urdf/closed_chain.xacro (robot description, xacro)
@@ -314,5 +314,4 @@
     effort_limit="1000">
   </xacro:gazebo_revolute_joint_macro>
-<!--
 	<xacro:revolute_joint_macro
     namespace="${namespace}"
@@ -325,5 +324,5 @@
     <origin xyz="${r2_length} 0 0" rpy="0 0 0"/>
   </xacro:revolute_joint_macro>
--->
+<!--
   <xacro:fixed_joint_macro
     namespace="${namespace}"
@@ -333,4 +332,5 @@
     <origin xyz="${r2_length} 0 0" rpy="0 0 0"/>
 	</xacro:fixed_joint_macro>
+-->
   <!-- Attach actuators -->
   <xacro:property name="generic_servo_inertial">
@@ -380,5 +380,4 @@
    <xacro:insert_block name="generic_servo_inertial"/>
  </xacro:servo_motor_macro>
-<!--
  <xacro:servo_motor_macro
    namespace="${namespace}"
@@ -400,5 +399,4 @@
    <xacro:insert_block name="generic_servo_inertial"/>
  </xacro:servo_motor_macro>
--->
  >
  <xacro:servo_motor_macro

File: rotors_description/urdf/firefly_qp.xacro (robot description, xacro)
@@ -22,5 +22,5 @@
   <xacro:property name="use_mesh_file" value="true" />
   <xacro:property name="mesh_file" value="package://rotors_description/meshes/firefly.dae" />
-  <xacro:property name="mass" value="2.6" /> <!-- [kg] --> <!-- Neo-like params -->
+  <xacro:property name="mass" value="2.77" /> <!-- [kg] --> <!-- Neo-like params -->
   <xacro:property name="body_width" value="0.1" /> <!-- [m] -->
   <xacro:property name="body_height" value="0.16" /> <!-- [m] -->
