Commit message: code clean up + comments added + name changed to neo + removed duplicates

File: rotors_description/urdf/closed_chain.xacro (robot description, xacro)
@@ -2,16 +2,21 @@
 <robot xmlns:xacro="http://ros.org/wiki/xacro">
   <xacro:include filename="$(find rotors_description)/urdf/manipulator_snippets.xacro" />
+	<xacro:property name="meas_delay" value="0"/>
+	<xacro:property name="angle_noise" value="0.0"/>
   <xacro:property name="r1_width" value="0.04"/>
   <xacro:property name="r1_height" value="0.008"/>
-  <xacro:property name="r1_length" value="0.24"/>
+  <xacro:property name="r1_length" value="0.24"/> <!-- 0.24 vs 0.35 -->
   <xacro:property name="r2_width" value="0.04"/>
   <xacro:property name="r2_height" value="0.008"/>
-  <xacro:property name="r2_length" value="0.35"/>
+  <xacro:property name="r2_length" value="0.35"/> <!-- 0.35 vs 0.40 -->
   <xacro:property name="r3_width" value="0.04"/>
   <xacro:property name="r3_height" value="0.0015"/>
   <xacro:property name="r3_length" value="0.14"/>
-  <xacro:property name="center_to_center_length" value="0.1"/>
+  <xacro:property name="center_to_center_length" value="0.10"/> <!-- 0.10 vs 0.12 -->
   <xacro:property name="end_effector_length" value="0.12"/>
   <xacro:property name="end_effector_radius" value="0.03"/>
+	<xacro:property name="use_mesh" value="true"/>
+	<xacro:property name="r1_scale" value="${r1_length/0.24*0.001} ${r1_length/0.24*0.001} 0.001"/>
+	<xacro:property name="r2_scale" value="${r2_length/0.35*0.001} ${r2_length/0.35*0.001} 0.001"/>
   <xacro:property name="r3_frame">
     <origin xyz="0 0 0" rpy="0 0 0"/>
@@ -35,5 +40,5 @@
   </xacro:property>
   <xacro:property name="r2_inertial">
-    <mass value="0.0015"/>
+    <mass value="0.015"/>
     <inertia ixx="0.00000229511" ixy="0.0" ixz="0.00000000098"
     iyy="0.00018644679" iyz="0.0"
@@ -52,5 +57,5 @@
   </xacro:property>
   <xacro:property name="r1_inertial">
-    <mass value="0.0012"/>
+    <mass value="0.012"/>
     <inertia ixx="0.00000948062" ixy="0.0" ixz="-0.00001716204"
     iyy="0.0000730949" iyz="0.0"
@@ -65,4 +70,5 @@
     <material name="orange"/>
   </xacro:property>
+<!--
   <xacro:property name="end_effector_frame">
     <origin xyz="${end_effector_length/2} 0 0" rpy="0 ${PI/2} 0"/>
@@ -79,405 +85,447 @@
     </geometry>
   </xacro:property>
+-->
 <!-- ################################################################################################# -->
 <!-- #################################### Manipulator Macro ########################################## -->
 <!-- ################################################################################################# -->
-  <xacro:macro name="closed_chain_macro"
-    params="namespace parent_link *origin">
-    <xacro:revolute_joint_macro
-      namespace="${namespace}"
-      joint_name="${namespace}/pitching"
-      parent_link="${namespace}/r0"
-      child_link="${namespace}/r3"
-      axis="1 0 0"
-      friction="0"
-      damping="0.1">
-      <origin xyz="0 0 -0.05" rpy="0 0 0"/>
-    </xacro:revolute_joint_macro>
-    <joint name="my_joint" type="floating">
-        <parent link="${parent_link}"/>
-        <child link="${namespace}/r0"/>
-        <xacro:insert_block name="origin" />
-        <dynamics damping="0.0" friction="0.0"/>
-     </joint>
-    <!-- <joint name="${namespace}/fixed_joint" type="fixed">
-      <parent link="${parent_link}"/>
-      <child  link="${namespace}/r3"/>
-      <xacro:insert_block name="origin" />
-    </joint> -->
+  <xacro:macro name="closed_chain_macro" params="namespace parent_link *origin">
+	<!-- Define how manipulator is attached to drone base -->
+		<!-- Uncomment this when using 6DOF shock-absorber -->
+<!--
+		<joint name="my_joint" type="floating">
+			<parent link="${parent_link}"/>
+			<child link="${namespace}/r0"/>
+			<xacro:insert_block name="origin" />
+			<dynamics damping="0.0" friction="0.0"/>
+		</joint>
+-->
+		<!-- Uncomment this for rigid connection -->
+		<joint name="${namespace}/fixed_joint" type="fixed">
+			<parent link="${parent_link}"/>
+			<child  link="${namespace}/r0"/>
+			<xacro:insert_block name="origin" />
+		</joint>
+		<!-- Additional pitching DoF -->
+		<xacro:revolute_joint_macro
+			namespace="${namespace}"
+			joint_name="${namespace}/pitching"
+			parent_link="${namespace}/r0"
+			child_link="${namespace}/r3"
+			axis="1 0 0"
+			friction="0"
+			damping="0.1">
+			<origin xyz="0 0 0" rpy="0 0 0"/>
+		</xacro:revolute_joint_macro>
   <!-- Here we define base link of closed kinematic chain -->
-  <link name="${namespace}/r0">
-   <collision>
-     <!-- <xacro:insert_block name="r3_frame"/>
-     <xacro:insert_block name="r3_geometry"/> -->
-     <origin xyz="0 0 0" rpy="0 0 0"/>
-     <geometry>
-         <mesh filename="package://rotors_description/meshes/delta_arm_meshes/pitching_base.dae" scale="0.001 0.001 0.001" />
-     </geometry>
-    </collision>
-    <visual>
-        <origin xyz="0 0 0" rpy="0 0 0"/>
-        <geometry>
-            <mesh filename="package://rotors_description/meshes/delta_arm_meshes/pitching_base.dae" scale="0.001 0.001 0.001" />
-        </geometry>
-    </visual>
-    <inertial>
-      <xacro:insert_block name="r3_frame"/>
-      <xacro:insert_block name="r3_inertial"/>
-    </inertial>
-  </link>
-  <link name="${namespace}/r3">
-   <collision>
-     <!-- <xacro:insert_block name="r3_frame"/>
-     <xacro:insert_block name="r3_geometry"/> -->
-     <origin xyz="0 0 0" rpy="0 0 0"/>
-     <geometry>
-         <mesh filename="package://rotors_description/meshes/delta_arm_meshes/pitching_base.dae" scale="0.001 0.001 0.001" />
-     </geometry>
-    </collision>
-    <visual>
-            <origin xyz="0 0 0" rpy="0 0 0"/>
-            <geometry>
-                <mesh filename="package://rotors_description/meshes/delta_arm_meshes/pitching_base.dae" scale="0.001 0.001 0.001" />
-            </geometry>
-    </visual>
-    <inertial>
-      <xacro:insert_block name="r3_frame"/>
-      <xacro:insert_block name="r3_inertial"/>
-    </inertial>
-  </link>
-  <link name="${namespace}/r1_left">
-   <collision>
-     <!-- <xacro:insert_block name="r1_frame"/>
-     <xacro:insert_block name="r1_geometry"/> -->
-     <origin xyz="0 0 0" rpy="0 0 0"/>
-     <geometry>
-         <mesh filename="package://rotors_description/meshes/delta_arm_meshes/R1_v2_left.dae" scale="0.001 0.001 0.001" />
-     </geometry>
-    </collision>
-    <visual>
-      <!-- <xacro:insert_block name="r1_frame"/> -->
-      <!-- <xacro:insert_block name="r1_geometry"/> -->
-      <!-- <origin xyz="0.03 0.115 -0.005" rpy="1.57 0 -0.3"/> -->
-      <origin xyz="0 0 0" rpy="0 0 0"/>
-      <geometry>
-          <mesh filename="package://rotors_description/meshes/delta_arm_meshes/R1_v2_left.dae" scale="0.001 0.001 0.001" />
-      </geometry>
-    </visual>
-    <inertial>
-      <xacro:insert_block name="r1_frame"/>
-      <xacro:insert_block name="r1_inertial"/>
-    </inertial>
-  </link>
-  <link name="${namespace}/r1_right">
-   <collision>
-     <!-- <xacro:insert_block name="r1_frame"/>
-     <xacro:insert_block name="r1_geometry"/> -->
-     <origin xyz="0 0 0" rpy="0 0 0"/>
-    <geometry>
-        <mesh filename="package://rotors_description/meshes/delta_arm_meshes/R1_v2.dae" scale="0.001 0.001 0.001" />
-    </geometry>
-    </collision>
-    <visual>
-      <!-- <xacro:insert_block name="r1_frame"/>
-      <xacro:insert_block name="r1_geometry"/> -->
-      <!-- <origin xyz="0.03 -0.115 0.008" rpy="-1.57 0 0.3"/> -->
-       <origin xyz="0 0 0" rpy="0 0 0"/>
-      <geometry>
-          <mesh filename="package://rotors_description/meshes/delta_arm_meshes/R1_v2.dae" scale="0.001 0.001 0.001" />
-      </geometry>
-    </visual>
-    <inertial>
-      <xacro:insert_block name="r1_frame"/>
-      <xacro:insert_block name="r1_inertial"/>
-    </inertial>
-  </link>
-  <link name="${namespace}/r2_left">
-   <collision>
-     <!-- <xacro:insert_block name="r2_frame"/>
-     <xacro:insert_block name="r2_geometry"/> -->
-     <origin xyz="0 0 0" rpy="0 0 0"/>
-     <geometry>
-         <mesh filename="package://rotors_description/meshes/delta_arm_meshes/R2_v2.dae" scale="0.001 0.001 0.001" />
-     </geometry>
-    </collision>
-    <visual>
-      <!-- <xacro:insert_block name="r2_frame"/>
-      <xacro:insert_block name="r2_geometry"/> -->
-      <origin xyz="0 0 0" rpy="0 0 0"/>
-      <geometry>
-          <mesh filename="package://rotors_description/meshes/delta_arm_meshes/R2_v2.dae" scale="0.001 0.001 0.001" />
-      </geometry>
-    </visual>
-    <inertial>
-      <xacro:insert_block name="r2_frame"/>
-      <xacro:insert_block name="r2_inertial"/>
-    </inertial>
-  </link>
-  <link name="${namespace}/r2_right">
-   <collision>
-     <!-- <xacro:insert_block name="r2_frame"/>
-     <xacro:insert_block name="r2_geometry"/> -->
-     <origin xyz="0 0 0" rpy="0 0 0"/>
-     <geometry>
-         <mesh filename="package://rotors_description/meshes/delta_arm_meshes/R2_v2.dae" scale="0.001 0.001 0.001" />
-     </geometry>
-    </collision>
-    <visual>
-      <!-- <xacro:insert_block name="r2_frame"/>
-      <xacro:insert_block name="r2_geometry"/> -->
-      <origin xyz="0 0 0" rpy="0 0 0"/>
-      <geometry>
-          <mesh filename="package://rotors_description/meshes/delta_arm_meshes/R2_v2.dae" scale="0.001 0.001 0.001" />
-      </geometry>
-    </visual>
-    <inertial>
-      <xacro:insert_block name="r2_frame"/>
-      <xacro:insert_block name="r2_inertial"/>
-    </inertial>
-  </link>
-  <link name="${namespace}/end_effector">
-   <collision>
-     <!-- <xacro:insert_block name="end_effector_frame"/>
-     <xacro:insert_block name="end_effector_geometry"/> -->
-     <origin xyz="0 0 -0.015" rpy="0 0 1.2"/>
-     <geometry>
-         <mesh filename="package://rotors_description/meshes/delta_arm_meshes/end_effector_plate.dae" scale="0.001 0.001 0.001" />
-     </geometry>
-    </collision>
-    <visual>
-      <!-- <xacro:insert_block name="end_effector_frame"/>
-      <xacro:insert_block name="end_effector_geometry"/> -->
-      <origin xyz="0 0 -0.015" rpy="0 0 1.2"/>
-      <geometry>
-          <mesh filename="package://rotors_description/meshes/delta_arm_meshes/end_effector_plate.dae" scale="0.001 0.001 0.001" />
-      </geometry>
-    </visual>
-    <inertial>
-      <xacro:insert_block name="end_effector_frame"/>
-      <xacro:insert_block name="end_effector_inertial"/>
-    </inertial>
-  </link>
-<!-- Define joints -->
-  <xacro:revolute_joint_macro
-    namespace="${namespace}"
-    joint_name="${namespace}/left_1"
-    parent_link="${namespace}/r3"
-    child_link="${namespace}/r1_left"
-    axis="0 0 1"
-    friction="0"
-    damping="0.1">
-    <origin xyz="${-center_to_center_length/2} 0 -0.005" rpy="0 0 0"/>
-  </xacro:revolute_joint_macro>
-  <xacro:revolute_joint_macro
-    namespace="${namespace}"
-    joint_name="${namespace}/right_1"
-    parent_link="${namespace}/r3"
-    child_link="${namespace}/r1_right"
-    axis="0 0 1"
-    friction="0"
-    damping="0.1">
-    <origin xyz="${center_to_center_length/2} 0 -0.005" rpy="0 0 0"/>
-  </xacro:revolute_joint_macro>
-  <xacro:revolute_joint_macro
-    namespace="${namespace}"
-    joint_name="${namespace}/left_2"
-    parent_link="${namespace}/r1_left"
-    child_link="${namespace}/r2_left"
-    axis="0 0 1"
-    friction="0"
-    damping="0.1">
-    <origin xyz="${r1_length} 0 0.01" rpy="0 0 0"/>
-  </xacro:revolute_joint_macro>
-  <xacro:revolute_joint_macro
-    namespace="${namespace}"
-    joint_name="${namespace}/right_2"
-    parent_link="${namespace}/r1_right"
-    child_link="${namespace}/r2_right"
-    axis="0 0 1"
-    friction="0"
-    damping="0.1">
-    <origin xyz="${r1_length} 0 -0.01" rpy="0 0 0"/>
-  </xacro:revolute_joint_macro>
-  <xacro:gazebo_revolute_joint_macro
-    namespace="${namespace}"
-    joint_name="${namespace}/closing"
-    parent_link="${namespace}/r2_left"
-    child_link="${namespace}/r2_right"
-    pose="${r2_length} 0 0 0 0 0"
-    axis="0 0 1"
-    friction="0"
-    damping="0.1"
-    spring_reference="0"
-    spring_stiffness="0"
-    lower_limit="-1e+16"
-    upper_limit="1e+16"
-    effort_limit="1000">
-  </xacro:gazebo_revolute_joint_macro>
-	<xacro:revolute_joint_macro
-    namespace="${namespace}"
-    joint_name="${namespace}/end_effector"
-    parent_link="${namespace}/r2_left"
-    child_link="${namespace}/end_effector"
-    axis="0 0 1"
-    friction="0"
-    damping="0.1">
-    <origin xyz="${r2_length} 0 0" rpy="0 0 0"/>
-  </xacro:revolute_joint_macro>
+		<link name="${namespace}/r0">
+			<collision>
+				<origin xyz="0 0 0" rpy="0 0 0"/>
+				<geometry>
+					<mesh filename="package://rotors_description/meshes/delta_arm_meshes/pitching_base.dae" scale="0.001 0.001 0.001" />
+				</geometry>
+			</collision>
+			<visual>
+				<origin xyz="0 0 0" rpy="0 0 0"/>
+				<geometry>
+					<mesh filename="package://rotors_description/meshes/delta_arm_meshes/pitching_base.dae" scale="0.001 0.001 0.001" />
+				</geometry>
+			</visual>
+			<inertial>
+				<xacro:insert_block name="r3_frame"/>
+				<mass value="0.00001"/>
+				<inertia ixx="0.00001" ixy="0.0" ixz="0.0"
+								 iyy="0.00001" iyz="0.0"
+								 izz="0.00001"/>
+			</inertial>
+		</link>
+		<link name="${namespace}/r3">
+			<collision>
+				<origin xyz="0 0 -0.05" rpy="0 0 0"/>
+				<geometry>
+					<mesh filename="package://rotors_description/meshes/delta_arm_meshes/pitching_base.dae" scale="0.001 0.001 0.001" />
+				</geometry>
+			</collision>
+			<visual>
+				<origin xyz="0 0 -0.05" rpy="0 0 0"/>
+				<geometry>
+					<mesh filename="package://rotors_description/meshes/delta_arm_meshes/pitching_base.dae" scale="0.001 0.001 0.001" />
+				</geometry>
+			</visual>
+			<inertial>
+				<origin xyz="0 0 -0.05" rpy="0 0 0"/>
+				<mass value="0.14"/>
+				<inertia ixx="0.00001" ixy="0.0" ixz="0.0"
+								 iyy="0.00035" iyz="0.0"
+								 izz="0.00035"/>
+			</inertial>
+		</link>
+		<link name="${namespace}/r1_left">
+			<collision>
+				<xacro:if value="${use_mesh == 'false'}">
+					<xacro:insert_block name="r1_frame"/>
+		   		<xacro:insert_block name="r1_geometry"/>
+				</xacro:if>
+				<xacro:if value="${use_mesh}">
+					<origin xyz="0 0 0" rpy="0 0 0"/>
+					<geometry>
+						<mesh filename="package://rotors_description/meshes/delta_arm_meshes/R1_v2_left.dae" scale="${r1_scale}" />
+					</geometry>
+				</xacro:if>
+			</collision>
+			<visual>
+				<xacro:if value="${use_mesh == 'false'}">
+					<xacro:insert_block name="r1_frame"/>
+		   		<xacro:insert_block name="r1_geometry"/>
+				</xacro:if>
+				<xacro:if value="${use_mesh}">
+					<origin xyz="0 0 0" rpy="0 0 0"/>
+					<geometry>
+						<mesh filename="package://rotors_description/meshes/delta_arm_meshes/R1_v2_left.dae" scale="${r1_scale}" />
+					</geometry>
+				</xacro:if>
+			</visual>
+			<inertial>
+				<xacro:insert_block name="r1_frame"/>
+				<xacro:insert_block name="r1_inertial"/>
+			</inertial>
+		</link>
+		<link name="${namespace}/r1_right">
+			<collision>
+				<xacro:if value="${use_mesh == 'false'}">
+					<xacro:insert_block name="r1_frame"/>
+		   		<xacro:insert_block name="r1_geometry"/>
+				</xacro:if>
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
File: rotors_description/urdf/neo.xacro (robot description, xacro)
@@ -6,4 +6,5 @@
   Copyright 2015 Janosch Nikolic, ASL, ETH Zurich, Switzerland
   Copyright 2015 Markus Achtelik, ASL, ETH Zurich, Switzerland
+  Copyright 2015 Simone Comari, ASL, ETH Zurich, Switzerland
   Licensed under the Apache License, Version 2.0 (the "License");
   you may not use this file except in compliance with the License.
@@ -16,10 +17,10 @@
   limitations under the License.
 -->
-<robot name="firefly" xmlns:xacro="http://ros.org/wiki/xacro">
+<robot name="neo" xmlns:xacro="http://ros.org/wiki/xacro">
   <!-- Properties -->
   <xacro:property name="namespace" value="$(arg mav_name)" />
   <xacro:property name="rotor_velocity_slowdown_sim" value="10" />
   <xacro:property name="use_mesh_file" value="true" />
-  <xacro:property name="mesh_file" value="package://rotors_description/meshes/firefly.dae" />
+  <xacro:property name="mesh_file" value="package://rotors_description/meshes/firefly.dae" /> <!-- this need to be changed with NEO mesh file!! -->
   <xacro:property name="mass" value="2.77" /> <!-- [kg] --> <!-- Neo-like params -->
   <xacro:property name="body_width" value="0.1" /> <!-- [m] -->
@@ -40,8 +41,8 @@
   <!-- Property Blocks -->
   <xacro:property name="body_inertia">
-		<inertia ixx="0.0331" ixy="0.0" ixz="0.0" iyy="0.0350" iyz="0.0" izz="0.0605" /> <!-- Neo-like params -->
+		<inertia ixx="0.0331" ixy="0.0" ixz="0.0" iyy="0.0350" iyz="0.0" izz="0.0605" />
 		<!--[kg m^2] [kg m^2] [kg m^2] [kg m^2] [kg m^2] [kg m^2] -->
   </xacro:property>
-  <!-- inertia of a single rotor, assuming it is a cuboid. Height=3mm, width=15mm -->
+  <!-- Inertia of a single rotor, assuming it is a cuboid. Height=3mm, width=15mm -->
   <xacro:property name="rotor_inertia">
     <xacro:box_inertia x="${radius_rotor}" y="0.015" z="0.003" mass="${mass_rotor*rotor_velocity_slowdown_sim}" />

File: rotors_description/urdf/neo_base.xacro (robot description, xacro)
@@ -6,4 +6,5 @@
   Copyright 2015 Janosch Nikolic, ASL, ETH Zurich, Switzerland
   Copyright 2015 Markus Achtelik, ASL, ETH Zurich, Switzerland
+  Copyright 2015 Simone Comari, ASL, ETH Zurich, Switzerland
   Licensed under the Apache License, Version 2.0 (the "License");
   you may not use this file except in compliance with the License.
@@ -16,8 +17,8 @@
   limitations under the License.
 -->
-<robot name="firefly" xmlns:xacro="http://ros.org/wiki/xacro">
+<robot name="neo" xmlns:xacro="http://ros.org/wiki/xacro">
   <xacro:include filename="$(find rotors_description)/urdf/component_snippets.xacro" />
   <!-- Instantiate firefly "mechanics" -->
-  <xacro:include filename="$(find rotors_description)/urdf/firefly_qp.xacro" />
+  <xacro:include filename="$(find rotors_description)/urdf/neo.xacro" />
   <!-- Instantiate a controller. -->
   <xacro:controller_plugin_macro namespace="${namespace}" imu_sub_topic="imu" />
