Commit message: Removing unfinished parts of px4 dummy controller and gazebo mavlink interface. Refactoring gazebo mavlink interface.

File: rotors_description/urdf/ardrone_base.xacro (robot description, xacro)
@@ -8,5 +8,5 @@
   <xacro:if value="$(arg enable_mavlink_interface)">
     <!-- Instantiate mavlink telemetry interface. -->
-    <xacro:mavlink_interface_macro namespace="${namespace}" imu_sub_topic="imu" />
+    <xacro:default_mavlink_interface namespace="${namespace}" imu_sub_topic="imu" />
   </xacro:if>
   <!-- Mount an ADIS16448 IMU. -->

File: rotors_description/urdf/asymmetric_quadrotor_base.xacro (robot description, xacro)
@@ -22,4 +22,8 @@
   <!-- Instantiate a controller. -->
   <xacro:controller_plugin_macro namespace="${namespace}" imu_sub_topic="imu" />
+  <xacro:if value="$(arg enable_mavlink_interface)">
+    <!-- Instantiate mavlink telemetry interface. -->
+    <xacro:default_mavlink_interface namespace="${namespace}" imu_sub_topic="imu" />
+  </xacro:if>
   <!-- Mount an ADIS16448 IMU. -->
   <xacro:default_imu namespace="${namespace}" parent_link="${namespace}/base_link" />

File: rotors_description/urdf/component_snippets.xacro (robot description, xacro)
@@ -246,10 +246,25 @@
   </xacro:macro>
   <!-- Macro to add the mavlink interface. -->
-  <xacro:macro name="mavlink_interface_macro" params="namespace imu_sub_topic">
+  <xacro:macro name="mavlink_interface_macro"
+    params="namespace imu_sub_topic mavlink_pub_topic gps_update_freq
+      reference_magnetic_field_north reference_magnetic_field_east
+      reference_magnetic_field_down reference_latitude reference_longitude
+      reference_altitude">
     <gazebo>
       <plugin name="mavlink_interface" filename="librotors_gazebo_mavlink_interface.so">
         <robotNamespace>${namespace}</robotNamespace>
         <imuSubTopic>${imu_sub_topic}</imuSubTopic>
-        <motorSpeedCommandPubTopic>gazebo/command/motor_speed</motorSpeedCommandPubTopic>
+        <mavlinkHilSensorPubTopic>${mavlink_pub_topic}</mavlinkHilSensorPubTopic>
+	<gpsUpdateFreq>${gps_update_freq}</gpsUpdateFreq> <!-- Frequency of HIL GPS messages [Hz] -->
+        <!-- [Gauss] Below are the North, East, and Down components of the Earth's magnetic field at the reference location.
+             The default reference location is Zurich (lat=+47.3667degN, lon=+8.5500degE, h=+500m, WGS84).
+	     You can obtain the magnetic field strength for your location using the World Magnetic Model:
+             https://www.ngdc.noaa.gov/geomag/WMM/calculators.shtml -->
+        <referenceMagNorth>${reference_magnetic_field_north}</referenceMagNorth>
+        <referenceMagEast>${reference_magnetic_field_east}</referenceMagEast>
+        <referenceMagDown>${reference_magnetic_field_down}</referenceMagDown>
+	<referenceLatitude>${reference_latitude}</referenceLatitude> <!-- the initial latitude [degrees [-90, 90]] -->
+        <referenceLongitude>${reference_longitude}</referenceLongitude> <!-- the initial longitude [degrees [-180, 180]] -->
+        <referenceAltitude>${reference_altitude}</referenceAltitude> <!-- the initial altitude [m] -->
       </plugin>
     </gazebo>
@@ -650,3 +665,17 @@
     </xacro:imu_plugin_macro>
   </xacro:macro>
+  <xacro:macro name="default_mavlink_interface" params="namespace imu_sub_topic">
+    <xacro:mavlink_interface_macro
+      namespace="${namespace}"
+      imu_sub_topic="${imu_sub_topic}"
+      mavlink_pub_topic="mavlink/from"
+      gps_update_freq="5.0"
+      reference_magnetic_field_north="0.21475"
+      reference_magnetic_field_east="0.00797"
+      reference_magnetic_field_down="0.42817"
+      reference_latitude="47.3667"
+      reference_longitude="8.5500"
+      reference_altitude="500.0">
+    </xacro:mavlink_interface_macro>
+  </xacro:macro>
 </robot>

File: rotors_description/urdf/firefly_base.xacro (robot description, xacro)
@@ -24,5 +24,5 @@
   <xacro:if value="$(arg enable_mavlink_interface)">
     <!-- Instantiate mavlink telemetry interface. -->
-    <xacro:mavlink_interface_macro namespace="${namespace}" imu_sub_topic="imu" />
+    <xacro:default_mavlink_interface namespace="${namespace}" imu_sub_topic="imu" />
   </xacro:if>
   <!-- Mount an ADIS16448 IMU. -->

File: rotors_description/urdf/hummingbird_base.xacro (robot description, xacro)
@@ -24,5 +24,5 @@
   <xacro:if value="$(arg enable_mavlink_interface)">
     <!-- Instantiate mavlink telemetry interface. -->
-    <xacro:mavlink_interface_macro namespace="${namespace}" imu_sub_topic="imu" />
+    <xacro:default_mavlink_interface namespace="${namespace}" imu_sub_topic="imu" />
   </xacro:if>
   <!-- Mount an ADIS16448 IMU. -->

File: rotors_description/urdf/iris_base.xacro (robot description, xacro)
@@ -8,5 +8,5 @@
   <xacro:if value="$(arg enable_mavlink_interface)">
     <!-- Instantiate mavlink telemetry interface. -->
-    <xacro:mavlink_interface_macro namespace="${namespace}" imu_sub_topic="imu" />
+    <xacro:default_mavlink_interface namespace="${namespace}" imu_sub_topic="imu" />
   </xacro:if>
   <!-- Mount an ADIS16448 IMU. -->

File: rotors_description/urdf/pelican_base.xacro (robot description, xacro)
@@ -24,5 +24,5 @@
   <xacro:if value="$(arg enable_mavlink_interface)">
     <!-- Instantiate mavlink telemetry interface. -->
-    <xacro:mavlink_interface_macro namespace="${namespace}" imu_sub_topic="imu" />
+    <xacro:default_mavlink_interface namespace="${namespace}" imu_sub_topic="imu" />
   </xacro:if>
   <!-- Mount an ADIS16448 IMU. -->

Commit message: Refactoring mavlink interface plugin more

File: rotors_description/urdf/ardrone_base.xacro (robot description, xacro)
@@ -8,5 +8,5 @@
   <xacro:if value="$(arg enable_mavlink_interface)">
     <!-- Instantiate mavlink telemetry interface. -->
-    <xacro:default_mavlink_interface namespace="${namespace}" imu_sub_topic="imu" />
+    <xacro:default_mavlink_interface namespace="${namespace}" imu_sub_topic="imu" rotor_count="4" />
   </xacro:if>
   <!-- Mount an ADIS16448 IMU. -->

File: rotors_description/urdf/asymmetric_quadrotor_base.xacro (robot description, xacro)
@@ -24,5 +24,5 @@
   <xacro:if value="$(arg enable_mavlink_interface)">
     <!-- Instantiate mavlink telemetry interface. -->
-    <xacro:default_mavlink_interface namespace="${namespace}" imu_sub_topic="imu" />
+    <xacro:default_mavlink_interface namespace="${namespace}" imu_sub_topic="imu" rotor_count="4" />
   </xacro:if>
   <!-- Mount an ADIS16448 IMU. -->

File: rotors_description/urdf/component_snippets.xacro (robot description, xacro)
@@ -247,14 +247,17 @@
   <!-- Macro to add the mavlink interface. -->
   <xacro:macro name="mavlink_interface_macro"
-    params="namespace imu_sub_topic mavlink_pub_topic gps_update_freq
-      reference_magnetic_field_north reference_magnetic_field_east
-      reference_magnetic_field_down reference_latitude reference_longitude
-      reference_altitude">
+    params="namespace mavlink_sub_topic imu_sub_topic mavlink_pub_topic
+      motors_speeds_pub_topic gps_update_freq rotor_count reference_magnetic_field_north
+      reference_magnetic_field_east reference_magnetic_field_down reference_latitude
+      reference_longitude reference_altitude">
     <gazebo>
       <plugin name="mavlink_interface" filename="librotors_gazebo_mavlink_interface.so">
         <robotNamespace>${namespace}</robotNamespace>
+	<mavlinkControlSubTopic>${mavlink_sub_topic}</mavlinkControlSubTopic>
         <imuSubTopic>${imu_sub_topic}</imuSubTopic>
         <mavlinkHilSensorPubTopic>${mavlink_pub_topic}</mavlinkHilSensorPubTopic>
+	<motorSpeedsPubTopic>${motors_speeds_pub_topic}</motorSpeedsPubTopic>
 	<gpsUpdateFreq>${gps_update_freq}</gpsUpdateFreq> <!-- Frequency of HIL GPS messages [Hz] -->
+	<rotorCount>${rotor_count}</rotorCount>
         <!-- [Gauss] Below are the North, East, and Down components of the Earth's magnetic field at the reference location.
              The default reference location is Zurich (lat=+47.3667degN, lon=+8.5500degE, h=+500m, WGS84).
@@ -665,10 +668,13 @@
     </xacro:imu_plugin_macro>
   </xacro:macro>
-  <xacro:macro name="default_mavlink_interface" params="namespace imu_sub_topic">
+  <xacro:macro name="default_mavlink_interface" params="namespace imu_sub_topic rotor_count">
     <xacro:mavlink_interface_macro
       namespace="${namespace}"
+      mavlink_sub_topic="/mavlink/from"
       imu_sub_topic="${imu_sub_topic}"
-      mavlink_pub_topic="mavlink/from"
+      mavlink_pub_topic="/mavlink/to"
+      motors_speeds_pub_topic="command/motor_speed"
       gps_update_freq="5.0"
+      rotor_count="${rotor_count}"
       reference_magnetic_field_north="0.21475"
       reference_magnetic_field_east="0.00797"

File: rotors_description/urdf/firefly_base.xacro (robot description, xacro)
@@ -24,5 +24,5 @@
   <xacro:if value="$(arg enable_mavlink_interface)">
     <!-- Instantiate mavlink telemetry interface. -->
-    <xacro:default_mavlink_interface namespace="${namespace}" imu_sub_topic="imu" />
+    <xacro:default_mavlink_interface namespace="${namespace}" imu_sub_topic="imu" rotor_count="6" />
   </xacro:if>
   <!-- Mount an ADIS16448 IMU. -->

File: rotors_description/urdf/hummingbird_base.xacro (robot description, xacro)
@@ -24,5 +24,5 @@
   <xacro:if value="$(arg enable_mavlink_interface)">
     <!-- Instantiate mavlink telemetry interface. -->
-    <xacro:default_mavlink_interface namespace="${namespace}" imu_sub_topic="imu" />
+    <xacro:default_mavlink_interface namespace="${namespace}" imu_sub_topic="imu" rotor_count="4" />
   </xacro:if>
   <!-- Mount an ADIS16448 IMU. -->

File: rotors_description/urdf/iris_base.xacro (robot description, xacro)
@@ -8,5 +8,5 @@
   <xacro:if value="$(arg enable_mavlink_interface)">
     <!-- Instantiate mavlink telemetry interface. -->
-    <xacro:default_mavlink_interface namespace="${namespace}" imu_sub_topic="imu" />
+    <xacro:default_mavlink_interface namespace="${namespace}" imu_sub_topic="imu" rotor_count="4" />
   </xacro:if>
   <!-- Mount an ADIS16448 IMU. -->

File: rotors_description/urdf/pelican_base.xacro (robot description, xacro)
@@ -24,5 +24,5 @@
   <xacro:if value="$(arg enable_mavlink_interface)">
     <!-- Instantiate mavlink telemetry interface. -->
-    <xacro:default_mavlink_interface namespace="${namespace}" imu_sub_topic="imu" />
+    <xacro:default_mavlink_interface namespace="${namespace}" imu_sub_topic="imu" rotor_count="4" />
   </xacro:if>
   <!-- Mount an ADIS16448 IMU. -->
