Commit message: Adding meshes and URDF components for flaps in Techpod model

File: rotors_description/urdf/techpod.xacro (robot description, xacro)
@@ -20,6 +20,7 @@
   <xacro:property name="PI" value="3.1415926535897931" />
   <!-- Component masses -->
-  <xacro:property name="mass_fuselage" value="2.65" /> <!-- [kg] -->
-  <xacro:property name="mass_aileron" value="0.2" /> <!-- [kg] -->
+  <xacro:property name="mass_fuselage" value="2.05" /> <!-- [kg] -->
+  <xacro:property name="mass_aileron" value="0.1" /> <!-- [kg] -->
+  <xacro:property name="mass_flap" value="0.1" /> <!-- [kg] -->
   <xacro:property name="mass_elevator" value="0.1" /> <!-- [kg] -->
   <xacro:property name="mass_rudder" value="0.1" /> <!-- [kg] -->
@@ -44,4 +45,11 @@
   <xacro:property name="elevator_max_angle" value="0.349066" /> <!-- [rad] -->
   <xacro:property name="elevator_color" value="Blue" />
+  <!-- Flap properties -->
+  <xacro:property name="flap_length" value="0.076" /> <!-- [m] -->
+  <xacro:property name="flap_width" value="0.459" /> <!-- [m] -->
+  <xacro:property name="flap_height" value="0.016" /> <!-- [m] -->
+  <xacro:property name="flap_min_angle" value="0.0" /> <!-- [rad] -->
+  <xacro:property name="flap_max_angle" value="0.0" /> <!-- [rad] -->
+  <xacro:property name="flap_color" value="Yellow" />
   <!-- Rudder properties -->
   <xacro:property name="rudder_length" value="0.129" />
@@ -68,4 +76,8 @@
     <xacro:box_inertia x="${elevator_length}" y="${elevator_width}" z="${elevator_height}" mass="${mass_elevator}" />
   </xacro:property>
+  <!-- Inertia of the flap, assuming it is a cuboid -->
+  <xacro:property name="flap_inertia">
+    <xacro:box_inertia x="${flap_length}" y="${flap_width}" z="${flap_height}" mass="${mass_flap}" />
+  </xacro:property>
   <!-- Inertia of the rudder, assuming it is a cuboid -->
   <xacro:property name="rudder_inertia">
@@ -88,5 +100,5 @@
     use_mesh_file="${use_mesh}"
     mesh_file="package://rotors_description/meshes/techpod/techpod_body.dae">
-    <origin xyz="0 0 0" rpy="${PI} 0 0" />
+    <origin xyz="0 0 0" rpy="0 0 0" />
     <xacro:insert_block name="body_inertia" />
   </xacro:fixed_wing_base_macro>
@@ -106,6 +118,6 @@
     surface_height="${aileron_height}">
     <axis xyz="0 -1 0" />   <!-- Joint axis -->
-    <origin xyz="0.1095 -0.99245 -0.115" rpy="0.0 0.0 0.0" />   <!-- Joint origin -->
-    <origin xyz="0.0 0.0 0.0" rpy="${PI} 0.0 0.0" />   <!-- Link origin -->
+    <origin xyz="0.1095 0.99245 0.115" rpy="0 0 0" />   <!-- Joint origin -->
+    <origin xyz="0 0 0" rpy="0 0 0" />   <!-- Link origin -->
     <xacro:insert_block name="aileron_inertia" />
   </xacro:control_surface>
@@ -124,6 +136,6 @@
     surface_height="${aileron_height}">
     <axis xyz="0 1 0" />   <!-- Joint axis -->
-    <origin xyz="0.1095 0.99245 -0.115" rpy="0.0 0.0 0.0" />   <!-- Joint origin -->
-    <origin xyz="0.0 0.0 0.0" rpy="${PI} 0.0 0.0" />   <!-- Link origin -->
+    <origin xyz="0.1095 -0.99245 0.115" rpy="0 0 0" />   <!-- Joint origin -->
+    <origin xyz="0 0 0" rpy="0 0 0" />   <!-- Link origin -->
     <xacro:insert_block name="aileron_inertia" />
   </xacro:control_surface>
@@ -142,8 +154,45 @@
     surface_width="${elevator_width}"
     surface_height="${elevator_height}">
+    <axis xyz="0 -1 0" />   <!-- Joint axis -->
+    <origin xyz="-0.555 0 0.26" rpy="0 0 0" />   <!-- Joint origin -->
+    <origin xyz="0 0 0" rpy="0 0 0" />   <!-- Link origin -->
+    <xacro:insert_block name="elevator_inertia" />
+  </xacro:control_surface>
+  <!-- Instantiate the flaps -->
+  <xacro:control_surface
+    robot_namespace="${namespace}"
+    surface_name="flap_left"
+    parent="${namespace}/base_link"
+    mass_surface="${mass_flap}"
+    min_angle="${flap_min_angle}"
+    max_angle="${flap_max_angle}"
+    color="${flap_color}"
+    use_mesh_file="${use_mesh}"
+    mesh_file="package://rotors_description/meshes/techpod/techpod_flap_left.dae"
+    surface_length="${flap_length}"
+    surface_width="${flap_width}"
+    surface_height="${flap_height}">
+    <axis xyz="0 -1 0" />   <!-- Joint axis -->
+    <origin xyz="0.101 0.382 0.1185" rpy="0 0 0" />   <!-- Joint origin -->
+    <origin xyz="0 0 0" rpy="0 0 0" />   <!-- Link origin -->
+    <xacro:insert_block name="flap_inertia" />
+  </xacro:control_surface>
+  <xacro:control_surface
+    robot_namespace="${namespace}"
+    surface_name="flap_right"
+    parent="${namespace}/base_link"
+    mass_surface="${mass_flap}"
+    min_angle="${flap_min_angle}"
+    max_angle="${flap_max_angle}"
+    color="${flap_color}"
+    use_mesh_file="${use_mesh}"
+    mesh_file="package://rotors_description/meshes/techpod/techpod_flap_right.dae"
+    surface_length="${flap_length}"
+    surface_width="${flap_width}"
+    surface_height="${flap_height}">
     <axis xyz="0 1 0" />   <!-- Joint axis -->
-    <origin xyz="-0.555 0.0 -0.26" rpy="0.0 0.0 0.0" />   <!-- Joint origin -->
-    <origin xyz="0.0 0.0 0.0" rpy="${PI} 0.0 0.0" />   <!-- Link origin -->
-    <xacro:insert_block name="elevator_inertia" />
+    <origin xyz="0.101 -0.382 0.1185" rpy="0 0 0" />   <!-- Joint origin -->
+    <origin xyz="0 0 0" rpy="0 0 0" />   <!-- Link origin -->
+    <xacro:insert_block name="flap_inertia" />
   </xacro:control_surface>
   <!-- Instantiate the rudder -->
@@ -162,6 +211,6 @@
     surface_height="${rudder_height}">
     <axis xyz="0 0 1" />   <!-- Joint axis -->
-    <origin xyz="-0.428 0.0 0.0" rpy="0.0 0.25 0.0" />   <!-- Joint origin -->
-    <origin xyz="0.0 0.0 0.0" rpy="${PI} -0.25 0.0" />   <!-- Link origin -->
+    <origin xyz="-0.428 0 0" rpy="0 -0.25 0" />   <!-- Joint origin -->
+    <origin xyz="0 0 0" rpy="0 0.25 0" />   <!-- Link origin -->
     <xacro:insert_block name="rudder_inertia" />
   </xacro:control_surface>
@@ -176,5 +225,5 @@
     use_mesh_file="${use_mesh}"
     mesh_file="package://rotors_description/meshes/propeller_${propeller_direction}.dae">
-    <origin xyz="-0.025 0.0 -0.15" rpy="0.0 ${-0.5*PI} 0.0" />
+    <origin xyz="-0.025 0 0.15" rpy="0 ${-0.5*PI} 0" />
     <xacro:insert_block name="propeller_inertia" />
   </xacro:propeller>
