Commit message: Now you could you mav_name:=mockingbird to start the simulation. Mesh for core added

File: rotors_description/urdf/mockingbird.xacro (robot description, xacro)
@@ -16,11 +16,11 @@
   limitations under the License.
 -->
-<robot name="firefly" xmlns:xacro="http://ros.org/wiki/xacro">
+<robot name="mockingbird" xmlns:xacro="http://ros.org/wiki/xacro">
   <!-- Properties -->
   <xacro:property name="namespace" value="$(arg namespace)" />
   <xacro:property name="rotor_velocity_slowdown_sim" value="10" />
   <xacro:property name="use_mesh_file" value="true" />
-  <xacro:property name="mesh_file" value="package://rotors_description/meshes/firefly.dae" />
-  <xacro:property name="mass" value="1.5" /> <!-- [kg] -->
+  <xacro:property name="mesh_file" value="package://rotors_description/meshes/mockingbird_core.dae" />
+  <xacro:property name="mass" value="2" /> <!-- [kg] -->
   <xacro:property name="body_width" value="0.1" /> <!-- [m] -->
   <xacro:property name="body_height" value="0.16" /> <!-- [m] -->

File: rotors_description/urdf/mockingbird_base.xacro (robot description, xacro)
@@ -16,8 +16,8 @@
   limitations under the License.
 -->
-<robot name="firefly" xmlns:xacro="http://ros.org/wiki/xacro">
+<robot name="mockingbird" xmlns:xacro="http://ros.org/wiki/xacro">
   <xacro:include filename="$(find rotors_description)/urdf/component_snippets.xacro" />
   <!-- Instantiate firefly "mechanics" -->
-  <xacro:include filename="$(find rotors_description)/urdf/firefly.xacro" />
+  <xacro:include filename="$(find rotors_description)/urdf/mockingbird.xacro" />
   <!-- Instantiate a controller. -->
   <xacro:controller_plugin_macro namespace="${namespace}" imu_sub_topic="imu" />

File: rotors_description/urdf/multirotor_base.xacro (robot description, xacro)
@@ -132,3 +132,40 @@
     </gazebo>
   </xacro:macro>
+  <!-- Tilting rotorunit link and joint -->
+  <xacro:macro name="rotorunit"
+    params="robot_namespace suffix direction motor_constant moment_constant parent mass_rotor radius_rotor time_constant_up time_constant_down max_rot_velocity motor_number rotor_drag_coefficient rolling_moment_coefficient color use_own_mesh mesh *origin *inertia">
+    <joint name="${robot_namespace}/rotor_${motor_number}_joint" type="continuous">
+      <xacro:insert_block name="origin" />
+      <axis xyz="0 0 1" />
+      <!-- TODO(ff): not currently set because it's not yet supported -->
+      <!-- <limit effort="2000" velocity="${max_rot_velocity}" /> -->
+      <parent link="${parent}" />
+      <child link="${robot_namespace}/rotor_${motor_number}" />
+    </joint>
+    <link name="${robot_namespace}/rotor_${motor_number}">
+      <inertial>
+        <mass value="${mass_rotor}" /> <!-- [kg] -->
+        <xacro:insert_block name="inertia" />
+      </inertial>
+      <visual>
+        <geometry>
+          <!-- <cylinder length="0.005" radius="${radius_rotor}"/> --> <!-- [m] -->
+          <xacro:if value="${use_own_mesh}">
+            <mesh filename="${mesh}"
+              scale="1 1 1" />
+          </xacro:if>
+          <xacro:unless value="${use_own_mesh}">
+            <mesh filename="package://rotors_description/meshes/propeller_${direction}.dae"
+              scale="${radius_rotor} ${radius_rotor} ${radius_rotor}" /> <!-- The propeller meshes have a radius of 1m -->
+            <!-- <box size="${2*radius_rotor} 0.01 0.005"/> -->
+          </xacro:unless>
+        </geometry>
+      </visual>
+      <collision>
+        <geometry>
+          <cylinder length="0.005" radius="${radius_rotor}" /> <!-- [m] -->
+        </geometry>
+      </collision>
+    </link>
+  </xacro:macro>
 </robot>

Commit message: Add the rotorunit whitout transmission to the drone for one axis

File: rotors_description/urdf/mockingbird.xacro (robot description, xacro)
@@ -20,13 +20,16 @@
   <xacro:property name="namespace" value="$(arg namespace)" />
   <xacro:property name="rotor_velocity_slowdown_sim" value="10" />
-  <xacro:property name="use_mesh_file" value="true" />
-  <xacro:property name="mesh_file" value="package://rotors_description/meshes/mockingbird_core.dae" />
-  <xacro:property name="mass" value="2" /> <!-- [kg] -->
+  <xacro:property name="use_mesh_file_core" value="true" />
+  <xacro:property name="use_mesh_file_rotor_unit" value="true" />
+  <xacro:property name="mesh_file_core" value="package://rotors_description/meshes/mockingbird_core.dae" />
+  <xacro:property name="mesh_file_rotor_unit" value="package://rotors_description/meshes/mockingbird_rotorunit.dae" />
+  <xacro:property name="mass_core" value="1.3" /> <!-- [kg] -->
+  <xacro:property name="mass_rotor_unit" value="0.2" /> <!-- [kg] -->
   <xacro:property name="body_width" value="0.1" /> <!-- [m] -->
   <xacro:property name="body_height" value="0.16" /> <!-- [m] -->
   <xacro:property name="mass_rotor" value="0.005" /> <!-- [kg] -->
-  <xacro:property name="arm_length" value="0.215" /> <!-- [m] -->
+  <xacro:property name="arm_length" value="0.256" /> <!-- [m] -->
   <xacro:property name="rotor_offset_top" value="0.037" /> <!-- [m] -->
-  <xacro:property name="radius_rotor" value="0.1" /> <!-- [m] -->
+  <xacro:property name="radius_rotor" value="0.0765" /> <!-- [m] -->
   <xacro:property name="motor_constant" value="8.54858e-06" /> <!-- [kg m/s^2] -->
   <xacro:property name="moment_constant" value="0.016" /> <!-- [m] -->
@@ -51,16 +54,27 @@
   <xacro:multirotor_base_macro
     robot_namespace="${namespace}"
-    mass="${mass}"
+    mass="${mass_core}"
     body_width="${body_width}"
     body_height="${body_height}"
-    use_mesh_file="${use_mesh_file}"
-    mesh_file="${mesh_file}"
+    use_mesh_file="${use_mesh_file_core}"
+    mesh_file="${mesh_file_core}"
     >
     <xacro:insert_block name="body_inertia" />
   </xacro:multirotor_base_macro>
+  <!-- Instantiate tilting rotor_unit -->
+  <xacro:rotor_unit
+    robot_namespace="${namespace}"
+    suffix="front_left"
+    parent="${namespace}/base_link"
+    mass_rotor_unit="${mass_rotor_unit}"
+    motor_number="0"
+    mesh_rotor_unit="${mesh_file_rotor_unit}">
+    <origin xyz="0 ${arm_length} 0" rpy="0 0 1.57079632679" />
+    <xacro:insert_block name="rotor_inertia" />
+  </xacro:rotor_unit>
   <!-- Instantiate rotors -->
   <xacro:vertical_rotor
     robot_namespace="${namespace}"
-    suffix="front_left"
+    suffix="left"
     direction="ccw"
     motor_constant="${motor_constant}"

File: rotors_description/urdf/multirotor_base.xacro (robot description, xacro)
@@ -133,17 +133,17 @@
   </xacro:macro>
   <!-- Tilting rotorunit link and joint -->
-  <xacro:macro name="rotorunit"
-    params="robot_namespace suffix direction motor_constant moment_constant parent mass_rotor radius_rotor time_constant_up time_constant_down max_rot_velocity motor_number rotor_drag_coefficient rolling_moment_coefficient color use_own_mesh mesh *origin *inertia">
-    <joint name="${robot_namespace}/rotor_${motor_number}_joint" type="continuous">
+  <xacro:macro name="rotor_unit"
+    params="robot_namespace suffix mass_rotor_unit parent motor_number mesh_rotor_unit *origin *inertia">
+    <joint name="${robot_namespace}/rotor_unit_${motor_number}_revolutejoint" type="continuous">
       <xacro:insert_block name="origin" />
-      <axis xyz="0 0 1" />
+      <axis xyz="1 0 0" />
       <!-- TODO(ff): not currently set because it's not yet supported -->
       <!-- <limit effort="2000" velocity="${max_rot_velocity}" /> -->
       <parent link="${parent}" />
-      <child link="${robot_namespace}/rotor_${motor_number}" />
+      <child link="${robot_namespace}/rotor_unit_${motor_number}" />
     </joint>
-    <link name="${robot_namespace}/rotor_${motor_number}">
+    <link name="${robot_namespace}/rotor_unit_${motor_number}">
       <inertial>
-        <mass value="${mass_rotor}" /> <!-- [kg] -->
+        <mass value="${mass_rotor_unit}" /> <!-- [kg] -->
         <xacro:insert_block name="inertia" />
       </inertial>
@@ -151,18 +151,11 @@
         <geometry>
           <!-- <cylinder length="0.005" radius="${radius_rotor}"/> --> <!-- [m] -->
-          <xacro:if value="${use_own_mesh}">
-            <mesh filename="${mesh}"
+            <mesh filename="${mesh_rotor_unit}"
               scale="1 1 1" />
-          </xacro:if>
-          <xacro:unless value="${use_own_mesh}">
-            <mesh filename="package://rotors_description/meshes/propeller_${direction}.dae"
-              scale="${radius_rotor} ${radius_rotor} ${radius_rotor}" /> <!-- The propeller meshes have a radius of 1m -->
-            <!-- <box size="${2*radius_rotor} 0.01 0.005"/> -->
-          </xacro:unless>
         </geometry>
       </visual>
       <collision>
         <geometry>
-          <cylinder length="0.005" radius="${radius_rotor}" /> <!-- [m] -->
+          <box size="0.005 0.005 0.005"  /> <!-- [m] -->
         </geometry>
       </collision>

Commit message: Added all rotorunits with transmission to the model

File: rotors_description/urdf/mockingbird.xacro (robot description, xacro)
@@ -36,5 +36,5 @@
   <xacro:property name="time_constant_up" value="0.0125" /> <!-- [s] -->
   <xacro:property name="time_constant_down" value="0.025" /> <!-- [s] -->
-  <xacro:property name="max_rot_velocity" value="838" /> <!-- [rad/s] -->
+  <xacro:property name="max_rot_velocity" value="838" /> <!-- [rad/s] --> <!-- so that it produce 1 kg thrust -->
   <xacro:property name="sin30" value="0.5" />
   <xacro:property name="cos30" value="0.866025403784" />
@@ -65,10 +65,60 @@
   <xacro:rotor_unit
     robot_namespace="${namespace}"
+    suffix="left"
+    parent="${namespace}/base_link"
+    mass_rotor_unit="${mass_rotor_unit}"
+    motor_number="0"
+    mesh_rotor_unit="${mesh_file_rotor_unit}">
+    <origin xyz="${cos30*arm_length} ${sin30*arm_length} 0" rpy="0 0 0.52359877559" />
+    <xacro:insert_block name="rotor_inertia" />
+  </xacro:rotor_unit>
+  <xacro:rotor_unit
+    robot_namespace="${namespace}"
     suffix="front_left"
     parent="${namespace}/base_link"
     mass_rotor_unit="${mass_rotor_unit}"
-    motor_number="0"
+    motor_number="1"
     mesh_rotor_unit="${mesh_file_rotor_unit}">
     <origin xyz="0 ${arm_length} 0" rpy="0 0 1.57079632679" />
+    <xacro:insert_block name="rotor_inertia" />
+  </xacro:rotor_unit>
+  <xacro:rotor_unit
+    robot_namespace="${namespace}"
+    suffix="back_left"
+    parent="${namespace}/base_link"
+    mass_rotor_unit="${mass_rotor_unit}"
+    motor_number="2"
+    mesh_rotor_unit="${mesh_file_rotor_unit}">
+    <origin xyz="-${cos30*arm_length} ${sin30*arm_length} 0" rpy="0 0 2.61799387799" />
+    <xacro:insert_block name="rotor_inertia" />
+  </xacro:rotor_unit>
+  <xacro:rotor_unit
+    robot_namespace="${namespace}"
+    suffix="back_right"
+    parent="${namespace}/base_link"
+    mass_rotor_unit="${mass_rotor_unit}"
+    motor_number="3"
+    mesh_rotor_unit="${mesh_file_rotor_unit}">
+    <origin xyz="-${cos30*arm_length} -${sin30*arm_length} 0" rpy="0 0 3.66519142919" />
+    <xacro:insert_block name="rotor_inertia" />
+  </xacro:rotor_unit>
+  <xacro:rotor_unit
+    robot_namespace="${namespace}"
+    suffix="right"
+    parent="${namespace}/base_link"
+    mass_rotor_unit="${mass_rotor_unit}"
+    motor_number="4"
+    mesh_rotor_unit="${mesh_file_rotor_unit}">
+    <origin xyz="0 -${arm_length} 0" rpy="0 0 4.71238898038" />
+    <xacro:insert_block name="rotor_inertia" />
+  </xacro:rotor_unit>
+  <xacro:rotor_unit
+    robot_namespace="${namespace}"
+    suffix="front_right"
+    parent="${namespace}/base_link"
+    mass_rotor_unit="${mass_rotor_unit}"
+    motor_number="5"
+    mesh_rotor_unit="${mesh_file_rotor_unit}">
+    <origin xyz="${cos30*arm_length} -${sin30*arm_length} 0" rpy="0 0 5.75958653158" />
     <xacro:insert_block name="rotor_inertia" />
   </xacro:rotor_unit>
@@ -80,5 +130,5 @@
     motor_constant="${motor_constant}"
     moment_constant="${moment_constant}"
-    parent="${namespace}/base_link"
+    parent="${namespace}/rotor_unit_0"
     mass_rotor="${mass_rotor}"
     radius_rotor="${radius_rotor}"
@@ -92,5 +142,5 @@
     use_own_mesh="false"
     mesh="">
-    <origin xyz="${cos30*arm_length} ${sin30*arm_length} ${rotor_offset_top}" rpy="0 0 0" />
+    <origin xyz="0 0 ${rotor_offset_top}" rpy="0 0 0" />
     <xacro:insert_block name="rotor_inertia" />
   </xacro:vertical_rotor>
@@ -101,5 +151,5 @@
     motor_constant="${motor_constant}"
     moment_constant="${moment_constant}"
-    parent="${namespace}/base_link"
+    parent="${namespace}/rotor_unit_1"
     mass_rotor="${mass_rotor}"
     radius_rotor="${radius_rotor}"
@@ -113,5 +163,5 @@
     use_own_mesh="false"
     mesh="">
-    <origin xyz="0 ${arm_length} ${rotor_offset_top}" rpy="0 0 0" />
+    <origin xyz="0 0 ${rotor_offset_top}" rpy="0 0 0" />
     <xacro:insert_block name="rotor_inertia" />
   </xacro:vertical_rotor>
@@ -121,5 +171,5 @@
     motor_constant="${motor_constant}"
     moment_constant="${moment_constant}"
-    parent="${namespace}/base_link"
+    parent="${namespace}/rotor_unit_2"
     mass_rotor="${mass_rotor}"
     radius_rotor="${radius_rotor}"
@@ -133,5 +183,5 @@
     use_own_mesh="false"
     mesh="">
-    <origin xyz="-${cos30*arm_length} ${sin30*arm_length} ${rotor_offset_top}" rpy="0 0 0" />
+    <origin xyz="0 0 ${rotor_offset_top}" rpy="0 0 0" />
     <xacro:insert_block name="rotor_inertia" />
   </xacro:vertical_rotor>
@@ -141,5 +191,5 @@
     motor_constant="${motor_constant}"
     moment_constant="${moment_constant}"
-    parent="${namespace}/base_link"
+    parent="${namespace}/rotor_unit_3"
     mass_rotor="${mass_rotor}"
     radius_rotor="${radius_rotor}"
@@ -153,5 +203,5 @@
     use_own_mesh="false"
     mesh="">
-    <origin xyz="-${cos30*arm_length} -${sin30*arm_length} ${rotor_offset_top}" rpy="0 0 0" />
+    <origin xyz="0 0 ${rotor_offset_top}" rpy="0 0 0" />
     <xacro:insert_block name="rotor_inertia" />
   </xacro:vertical_rotor>
@@ -162,5 +212,5 @@
     motor_constant="${motor_constant}"
     moment_constant="${moment_constant}"
-    parent="${namespace}/base_link"
+    parent="${namespace}/rotor_unit_4"
     mass_rotor="${mass_rotor}"
     radius_rotor="${radius_rotor}"
@@ -174,5 +224,5 @@
     use_own_mesh="false"
     mesh="">
-    <origin xyz="0 -${arm_length} ${rotor_offset_top}" rpy="0 0 0" />
+    <origin xyz="0 0 ${rotor_offset_top}" rpy="0 0 0" />
     <xacro:insert_block name="rotor_inertia" />
   </xacro:vertical_rotor>
@@ -183,5 +233,5 @@
     motor_constant="${motor_constant}"
     moment_constant="${moment_constant}"
-    parent="${namespace}/base_link"
+    parent="${namespace}/rotor_unit_5"
     mass_rotor="${mass_rotor}"
     radius_rotor="${radius_rotor}"
@@ -195,5 +245,5 @@
     use_own_mesh="false"
     mesh="">
-    <origin xyz="${cos30*arm_length} -${sin30*arm_length} ${rotor_offset_top}" rpy="0 0 0" />
+    <origin xyz="0 0 ${rotor_offset_top}" rpy="0 0 0" />
     <xacro:insert_block name="rotor_inertia" />
   </xacro:vertical_rotor>

File: rotors_description/urdf/multirotor_base.xacro (robot description, xacro)
@@ -135,5 +135,5 @@
   <xacro:macro name="rotor_unit"
     params="robot_namespace suffix mass_rotor_unit parent motor_number mesh_rotor_unit *origin *inertia">
-    <joint name="${robot_namespace}/rotor_unit_${motor_number}_revolutejoint" type="continuous">
+    <joint name="${robot_namespace}/rotor_unit_${motor_number}_revolutejoint" type="fixed">
       <xacro:insert_block name="origin" />
       <axis xyz="1 0 0" />
@@ -143,4 +143,14 @@
       <child link="${robot_namespace}/rotor_unit_${motor_number}" />
     </joint>
+    <transmission name="${robot_namespace}/rotor_unit_${motor_number}_trans">
+      <type>transmission_interface/SimpleTransmission</type>
+        <joint name="${robot_namespace}/rotor_unit_${motor_number}_revolutejoint">
+          <hardwareInterface>EffortJointInterface</hardwareInterface>
+        </joint>
+        <actuator name="${robot_namespace}/rotor_unit_${motor_number}_tiltmotor">
+          <hardwareInterface>EffortJointInterface</hardwareInterface>
+          <mechanicalReduction>1</mechanicalReduction>
+        </actuator>
+    </transmission>
     <link name="${robot_namespace}/rotor_unit_${motor_number}">
       <inertial>

Commit message: Revolute Joints added with interface in mockingbird.xacro

File: rotors_description/urdf/mockingbird.xacro (robot description, xacro)
@@ -24,11 +24,11 @@
   <xacro:property name="mesh_file_core" value="package://rotors_description/meshes/mockingbird_core.dae" />
   <xacro:property name="mesh_file_rotor_unit" value="package://rotors_description/meshes/mockingbird_rotorunit.dae" />
-  <xacro:property name="mass_core" value="1.3" /> <!-- [kg] -->
-  <xacro:property name="mass_rotor_unit" value="0.2" /> <!-- [kg] -->
+  <xacro:property name="mass_core" value="0.5" /> <!-- [kg] -->
+  <xacro:property name="mass_rotor_unit" value="0.1" /> <!-- [kg] -->
   <xacro:property name="body_width" value="0.1" /> <!-- [m] -->
   <xacro:property name="body_height" value="0.16" /> <!-- [m] -->
   <xacro:property name="mass_rotor" value="0.005" /> <!-- [kg] -->
   <xacro:property name="arm_length" value="0.256" /> <!-- [m] -->
-  <xacro:property name="rotor_offset_top" value="0.037" /> <!-- [m] -->
+  <xacro:property name="rotor_offset_top" value="0.042" /> <!-- [m] -->
   <xacro:property name="radius_rotor" value="0.0765" /> <!-- [m] -->
   <xacro:property name="motor_constant" value="8.54858e-06" /> <!-- [kg m/s^2] -->
@@ -37,4 +37,8 @@
   <xacro:property name="time_constant_down" value="0.025" /> <!-- [s] -->
   <xacro:property name="max_rot_velocity" value="838" /> <!-- [rad/s] --> <!-- so that it produce 1 kg thrust -->
+  <xacro:property name="lower_limit_revolute" value="0" /> <!-- properties of the revolute joint of the tilted axis -->
+  <xacro:property name="upper_limit_revolute" value="0" /> <!-- properties of the revolute joint of the tilted axis -->
+  <xacro:property name="effort_revolute" value="1000" /> <!-- properties of the revolute joint of the tilted axis -->
+  <xacro:property name="velocity_revolute" value="4" /> <!-- properties of the revolute joint of the tilted axis -->
   <xacro:property name="sin30" value="0.5" />
   <xacro:property name="cos30" value="0.866025403784" />
@@ -69,4 +73,8 @@
     mass_rotor_unit="${mass_rotor_unit}"
     motor_number="0"
+    lower_limit="${lower_limit_revolute}"
+    upper_limit="${upper_limit_revolute}"
+    effort="${effort_revolute}"
+    velocity="${velocity_revolute}"
     mesh_rotor_unit="${mesh_file_rotor_unit}">
     <origin xyz="${cos30*arm_length} ${sin30*arm_length} 0" rpy="0 0 0.52359877559" />
@@ -79,4 +87,8 @@
     mass_rotor_unit="${mass_rotor_unit}"
     motor_number="1"
+    lower_limit="${lower_limit_revolute}"
+    upper_limit="${upper_limit_revolute}"
+    effort="${effort_revolute}"
+    velocity="${velocity_revolute}"
     mesh_rotor_unit="${mesh_file_rotor_unit}">
     <origin xyz="0 ${arm_length} 0" rpy="0 0 1.57079632679" />
@@ -89,4 +101,8 @@
     mass_rotor_unit="${mass_rotor_unit}"
     motor_number="2"
+    lower_limit="${lower_limit_revolute}"
+    upper_limit="${upper_limit_revolute}"
+    effort="${effort_revolute}"
+    velocity="${velocity_revolute}"
     mesh_rotor_unit="${mesh_file_rotor_unit}">
     <origin xyz="-${cos30*arm_length} ${sin30*arm_length} 0" rpy="0 0 2.61799387799" />
@@ -99,4 +115,8 @@
     mass_rotor_unit="${mass_rotor_unit}"
     motor_number="3"
+    lower_limit="${lower_limit_revolute}"
+    upper_limit="${upper_limit_revolute}"
+    effort="${effort_revolute}"
+    velocity="${velocity_revolute}"
     mesh_rotor_unit="${mesh_file_rotor_unit}">
     <origin xyz="-${cos30*arm_length} -${sin30*arm_length} 0" rpy="0 0 3.66519142919" />
@@ -109,4 +129,8 @@
     mass_rotor_unit="${mass_rotor_unit}"
     motor_number="4"
+    lower_limit="${lower_limit_revolute}"
+    upper_limit="${upper_limit_revolute}"
+    effort="${effort_revolute}"
+    velocity="${velocity_revolute}"
     mesh_rotor_unit="${mesh_file_rotor_unit}">
     <origin xyz="0 -${arm_length} 0" rpy="0 0 4.71238898038" />
@@ -119,4 +143,8 @@
     mass_rotor_unit="${mass_rotor_unit}"
     motor_number="5"
+    lower_limit="${lower_limit_revolute}"
+    upper_limit="${upper_limit_revolute}"
+    effort="${effort_revolute}"
+    velocity="${velocity_revolute}"
     mesh_rotor_unit="${mesh_file_rotor_unit}">
     <origin xyz="${cos30*arm_length} -${sin30*arm_length} 0" rpy="0 0 5.75958653158" />

File: rotors_description/urdf/multirotor_base.xacro (robot description, xacro)
@@ -134,8 +134,9 @@
   <!-- Tilting rotorunit link and joint -->
   <xacro:macro name="rotor_unit"
-    params="robot_namespace suffix mass_rotor_unit parent motor_number mesh_rotor_unit *origin *inertia">
-    <joint name="${robot_namespace}/rotor_unit_${motor_number}_revolutejoint" type="fixed">
+    params="robot_namespace suffix mass_rotor_unit parent motor_number lower_limit upper_limit effort velocity mesh_rotor_unit *origin *inertia">
+    <joint name="${robot_namespace}/rotor_unit_${motor_number}_revolutejoint" type="revolute">
       <xacro:insert_block name="origin" />
       <axis xyz="1 0 0" />
+       <limit lower="${lower_limit}" upper="${upper_limit}" effort="${effort}" velocity="${velocity}" />
       <!-- TODO(ff): not currently set because it's not yet supported -->
       <!-- <limit effort="2000" velocity="${max_rot_velocity}" /> -->
