Commit message: Fixing small details and removing references to gazebo plugins

File: rotors_description/urdf/fixed_wing_base.xacro (robot description, xacro)
@@ -1,9 +1,5 @@
 <?xml version="1.0"?>
 <!--
-  Copyright 2015 Fadri Furrer, ASL, ETH Zurich, Switzerland
-  Copyright 2015 Michael Burri, ASL, ETH Zurich, Switzerland
-  Copyright 2015 Mina Kamel, ASL, ETH Zurich, Switzerland
-  Copyright 2015 Janosch Nikolic, ASL, ETH Zurich, Switzerland
-  Copyright 2015 Markus Achtelik, ASL, ETH Zurich, Switzerland
+  Copyright 2016 Pavel Vechersky, ASL, ETH Zurich, Switzerland
   Licensed under the Apache License, Version 2.0 (the "License");
   you may not use this file except in compliance with the License.
@@ -29,8 +25,8 @@
       izz="${0.5 * mass * r * r}" />
   </xacro:macro>
-  <!-- Fixed-wing fuselage link -->
+  <!-- Fixed-wing main body link -->
   <xacro:macro name="fixed_wing_base_macro"
     params="robot_namespace mass length width height color use_mesh_file
-      mesh_file reset_model_service_name *origin *inertia">
+      mesh_file *origin *inertia">
     <link name="${robot_namespace}/base_link"></link>
     <joint name="${robot_namespace}/base_joint" type="fixed">
@@ -68,11 +64,4 @@
       </collision>
     </link>
-    <gazebo>
-      <plugin name="${robot_namespace}_base" filename="librotors_gazebo_fixedwing_base_plugin.so">
-        <robotNamespace>${robot_namespace}</robotNamespace>
-        <linkName>${robot_namespace}/base_link</linkName>
-	<resetModelServiceName>${reset_model_service_name}</resetModelServiceName>
-      </plugin>
-    </gazebo>
     <gazebo reference="${robot_namespace}/base_link">
       <material>Gazebo/${color}</material>

File: rotors_description/urdf/techpod.xacro (robot description, xacro)
@@ -25,5 +25,5 @@
   <xacro:property name="mass_rudder" value="0.1" /> <!-- [kg] -->
   <xacro:property name="mass_propeller" value="0.1" /> <!-- [kg] -->
-  <!-- Fuselage properties -->
+  <!-- Main body properties -->
   <xacro:property name="body_length" value="1.088" /> <!-- [m] -->
   <xacro:property name="body_width" value="2.591" /> <!-- [m] -->
@@ -50,11 +50,13 @@
   <xacro:property name="rudder_min_angle" value="-0.349066" />
   <xacro:property name="rudder_max_angle" value="0.349066" />
+  <xacro:property name="rudder_color" value="Orange" />
   <!-- Propeller properties -->
   <xacro:property name="propeller_direction" value="cw" />
   <xacro:property name="propeller_radius" value="0.1" />
   <xacro:property name="propeller_height" value="0.003" />
-  <!-- Inertia of the fuselage -->
+  <xacro:property name="propeller_color" value="Gray" />
+  <!-- Inertia of the main body -->
   <xacro:property name="body_inertia">
-    <xacro:box_inertia x="${body_length}" y="${body_width}" z="${body_height}" mass="${mass_fuselage}" />
+    <inertia ixx="0.16632" ixy="0.0" ixz="0.0755" iyy="0.3899" iyz="0.0" izz="0.5243" />
   </xacro:property>
   <!-- Inertia of the aileron, assuming it is a cuboid -->
@@ -70,5 +72,5 @@
     <xacro:box_inertia x="${rudder_length}" y="${rudder_width}" z="${rudder_height}" mass="${mass_rudder}" />
   </xacro:property>
-  <!-- Inertia of the propeller, assuming it is a cuboid -->
+  <!-- Inertia of the propeller, assuming it is a cylinder -->
   <xacro:property name="propeller_inertia">
     <xacro:cylinder_inertia r="${propeller_radius}" h="${propeller_height}" mass="${mass_propeller*rotor_velocity_slowdown_sim}" />
@@ -85,9 +87,7 @@
     color="${body_color}"
     use_mesh_file="${use_mesh}"
-    mesh_file="package://rotors_description/meshes/techpod/techpod_body.dae"
-    reset_model_service_name="reset_model">
-    <origin xyz="0 0 0" rpy="3.1415926535897931 0 0" />
-    <inertia ixx="${0.1512 * 1.1}" ixy="0.0" ixz="0.0755" iyy="${0.2785 * 1.4}" iyz="0.0" izz="${0.3745 * 1.4}" />
-    <!--<xacro:insert_block name="body_inertia" />-->
+    mesh_file="package://rotors_description/meshes/techpod/techpod_body.dae">
+    <origin xyz="0 0 0" rpy="${PI} 0 0" />
+    <xacro:insert_block name="body_inertia" />
   </xacro:fixed_wing_base_macro>
   <!-- Instantiate the ailerons -->
@@ -155,5 +155,5 @@
     min_angle="${rudder_min_angle}"
     max_angle="${rudder_max_angle}"
-    color="Orange"
+    color="${rudder_color}"
     use_mesh_file="${use_mesh}"
     mesh_file="package://rotors_description/meshes/techpod/techpod_rudder.dae"
@@ -161,7 +161,7 @@
     surface_width="${rudder_width}"
     surface_height="${rudder_height}">
-    <axis xyz="0 0 1" />
-    <origin xyz="-0.428 0.0 0.0" rpy="0.0 0.25 0.0" />
-    <origin xyz="0.0 0.0 0.0" rpy="${PI} -0.25 0.0" />
+    <axis xyz="0 0 1" />   <!-- Joint axis -->
+    <origin xyz="-0.428 0.0 0.0" rpy="0.0 0.25 0.0" />   <!-- Joint origin -->
+    <origin xyz="0.0 0.0 0.0" rpy="${PI} -0.25 0.0" />   <!-- Link origin -->
     <xacro:insert_block name="rudder_inertia" />
   </xacro:control_surface>
@@ -173,8 +173,8 @@
     mass_propeller="${mass_propeller}"
     propeller_radius="${propeller_radius}"
-    color="Green"
+    color="${propeller_color}"
     use_mesh_file="${use_mesh}"
     mesh_file="package://rotors_description/meshes/propeller_${propeller_direction}.dae">
-    <origin xyz="-0.025 0.0 -0.15" rpy="0.0 ${0.5*PI} 0.0" />
+    <origin xyz="-0.025 0.0 -0.15" rpy="0.0 ${-0.5*PI} 0.0" />
     <xacro:insert_block name="propeller_inertia" />
   </xacro:propeller>

Commit message: Parameterizing techpod mesh files and aerodynamic parameters

File: rotors_description/urdf/fixed_wing_base.xacro (robot description, xacro)
@@ -28,5 +28,5 @@
   <xacro:macro name="fixed_wing_base_macro"
     params="robot_namespace mass length width height color use_mesh_file
-      mesh_file *origin *inertia">
+      mesh_file aero_params_yaml *origin *inertia">
     <link name="${robot_namespace}/base_link"></link>
     <joint name="${robot_namespace}/base_joint" type="fixed">
@@ -61,4 +61,12 @@
     <gazebo reference="${robot_namespace}/base_link">
       <material>Gazebo/${color}</material>
+    </gazebo>
+    <!-- Attach fw_dynamics to the base_link -->
+    <gazebo>
+      <plugin filename="librotors_gazebo_fw_dynamics_plugin.so" name="fw_dynamics_plugin">
+        <robotNamespace>${robot_namespace}</robotNamespace>
+        <linkName>${robot_namespace}/base_link</linkName>
+        <aeroParamsYAML>${aero_params_yaml}</aeroParamsYAML>
+      </plugin>
     </gazebo>
   </xacro:macro>

File: rotors_description/urdf/techpod.xacro (robot description, xacro)
@@ -15,4 +15,5 @@
   <!-- Global properties -->
   <xacro:property name="namespace" value="$(arg namespace)" />
+  <xacro:property name="aero_params_yaml_file" value="$(arg yaml_params_yaml_file)" />
   <xacro:property name="rotor_velocity_slowdown_sim" value="10" />
   <xacro:property name="use_mesh" value="true" />
@@ -31,4 +32,5 @@
   <xacro:property name="body_height" value="0.303" /> <!-- [m] -->
   <xacro:property name="body_color" value="Gray" />
+  <xacro:property name="body_mesh_file" value="package://rotors_description/meshes/techpod/techpod_body.dae" />
   <!-- Aileron properties -->
   <xacro:property name="aileron_length" value="0.053" /> <!-- [m] -->
@@ -38,4 +40,6 @@
   <xacro:property name="aileron_max_angle" value="0.349066" /> <!-- [rad] -->
   <xacro:property name="aileron_color" value="Red" />
+  <xacro:property name="aileron_left_mesh_file" value="package://rotors_description/meshes/techpod/techpod_aileron_left.dae" />
+  <xacro:property name="aileron_right_mesh_file" value="package://rotors_description/meshes/techpod/techpod_aileron_right.dae" />
   <!-- Elevator properties -->
   <xacro:property name="elevator_length" value="0.051" /> <!-- [m] -->
@@ -45,4 +49,5 @@
   <xacro:property name="elevator_max_angle" value="0.349066" /> <!-- [rad] -->
   <xacro:property name="elevator_color" value="Blue" />
+  <xacro:property name="elevator_mesh_file" value="package://rotors_description/meshes/techpod/techpod_elevator.dae" />
   <!-- Flap properties -->
   <xacro:property name="flap_length" value="0.076" /> <!-- [m] -->
@@ -52,4 +57,6 @@
   <xacro:property name="flap_max_angle" value="0.0" /> <!-- [rad] -->
   <xacro:property name="flap_color" value="Yellow" />
+  <xacro:property name="flap_left_mesh_file" value="package://rotors_description/meshes/techpod/techpod_flap_left.dae" />
+  <xacro:property name="flap_right_mesh_file" value="package://rotors_description/meshes/techpod/techpod_flap_right.dae" />
   <!-- Rudder properties -->
   <xacro:property name="rudder_length" value="0.129" />
@@ -59,4 +66,5 @@
   <xacro:property name="rudder_max_angle" value="0.349066" />
   <xacro:property name="rudder_color" value="Orange" />
+  <xacro:property name="rudder_mesh_file" value="package://rotors_description/meshes/techpod/techpod_rudder.dae" />
   <!-- Propeller properties -->
   <xacro:property name="propeller_direction" value="cw" />
@@ -64,4 +72,5 @@
   <xacro:property name="propeller_height" value="0.003" />
   <xacro:property name="propeller_color" value="Gray" />
+  <xacro:property name="propeller_mesh_file" value="package://rotors_description/meshes/propeller_${propeller_direction}.dae" />
   <!-- Inertia of the main body -->
   <xacro:property name="body_inertia">
@@ -99,5 +108,6 @@
     color="${body_color}"
     use_mesh_file="${use_mesh}"
-    mesh_file="package://rotors_description/meshes/techpod/techpod_body.dae">
+    mesh_file="${body_mesh_file}"
+    aero_params_yaml="${aero_params_yaml_file}">
     <origin xyz="0 0 0" rpy="0 0 0" />
     <xacro:insert_block name="body_inertia" />
@@ -113,5 +123,5 @@
     color="${aileron_color}"
     use_mesh_file="${use_mesh}"
-    mesh_file="package://rotors_description/meshes/techpod/techpod_aileron_left.dae"
+    mesh_file="${aileron_left_mesh_file}"
     surface_length="${aileron_length}"
     surface_width="${aileron_width}"
@@ -131,5 +141,5 @@
     color="${aileron_color}"
     use_mesh_file="${use_mesh}"
-    mesh_file="package://rotors_description/meshes/techpod/techpod_aileron_right.dae"
+    mesh_file="${aileron_right_mesh_file}"
     surface_length="${aileron_length}"
     surface_width="${aileron_width}"
@@ -150,5 +160,5 @@
     color="${elevator_color}"
     use_mesh_file="${use_mesh}"
-    mesh_file="package://rotors_description/meshes/techpod/techpod_elevator.dae"
+    mesh_file="${elevator_mesh_file}"
     surface_length="${elevator_length}"
     surface_width="${elevator_width}"
@@ -169,5 +179,5 @@
     color="${flap_color}"
     use_mesh_file="${use_mesh}"
-    mesh_file="package://rotors_description/meshes/techpod/techpod_flap_left.dae"
+    mesh_file="${flap_left_mesh_file}"
     surface_length="${flap_length}"
     surface_width="${flap_width}"
@@ -187,5 +197,5 @@
     color="${flap_color}"
     use_mesh_file="${use_mesh}"
-    mesh_file="package://rotors_description/meshes/techpod/techpod_flap_right.dae"
+    mesh_file="${flap_right_mesh_file}"
     surface_length="${flap_length}"
     surface_width="${flap_width}"
@@ -206,5 +216,5 @@
     color="${rudder_color}"
     use_mesh_file="${use_mesh}"
-    mesh_file="package://rotors_description/meshes/techpod/techpod_rudder.dae"
+    mesh_file="${rudder_mesh_file}"
     surface_length="${rudder_length}"
     surface_width="${rudder_width}"
@@ -224,5 +234,5 @@
     color="${propeller_color}"
     use_mesh_file="${use_mesh}"
-    mesh_file="package://rotors_description/meshes/propeller_${propeller_direction}.dae">
+    mesh_file="${propeller_mesh_file}">
     <origin xyz="-0.025 0 0.15" rpy="0 ${-0.5*PI} 0" />
     <xacro:insert_block name="propeller_inertia" />

Commit message: Implementing the rest of parameter parsing and forces + moments calculations

File: rotors_description/urdf/fixed_wing_base.xacro (robot description, xacro)
@@ -28,5 +28,5 @@
   <xacro:macro name="fixed_wing_base_macro"
     params="robot_namespace mass length width height color use_mesh_file
-      mesh_file aero_params_yaml *origin *inertia">
+      mesh_file aero_params_yaml vehicle_params_yaml *origin *inertia">
     <link name="${robot_namespace}/base_link"></link>
     <joint name="${robot_namespace}/base_joint" type="fixed">
@@ -68,4 +68,5 @@
         <linkName>${robot_namespace}/base_link</linkName>
         <aeroParamsYAML>${aero_params_yaml}</aeroParamsYAML>
+        <vehicleParamsYAML>${vehicle_params_yaml}</vehicleParamsYAML>
       </plugin>
     </gazebo>

File: rotors_description/urdf/techpod.xacro (robot description, xacro)
@@ -15,5 +15,6 @@
   <!-- Global properties -->
   <xacro:property name="namespace" value="$(arg namespace)" />
-  <xacro:property name="aero_params_yaml_file" value="$(arg yaml_params_yaml_file)" />
+  <xacro:property name="aero_params_yaml_file" value="$(arg aero_params_yaml_file)" />
+  <xacro:property name="vehicle_params_yaml_file" value="$(arg vehicle_params_yaml_file)" />
   <xacro:property name="rotor_velocity_slowdown_sim" value="10" />
   <xacro:property name="use_mesh" value="true" />
@@ -109,5 +110,6 @@
     use_mesh_file="${use_mesh}"
     mesh_file="${body_mesh_file}"
-    aero_params_yaml="${aero_params_yaml_file}">
+    aero_params_yaml="${aero_params_yaml_file}"
+    vehicle_params_yaml="${vehicle_params_yaml_file}">
     <origin xyz="0 0 0" rpy="0 0 0" />
     <xacro:insert_block name="body_inertia" />

Commit message: Implementing fixed-wing operation with a joystick

File: rotors_description/urdf/fixed_wing_base.xacro (robot description, xacro)
@@ -28,5 +28,6 @@
   <xacro:macro name="fixed_wing_base_macro"
     params="robot_namespace mass length width height color use_mesh_file
-      mesh_file aero_params_yaml vehicle_params_yaml *origin *inertia">
+      mesh_file aero_params_yaml vehicle_params_yaml is_input_joystick
+      *origin *inertia">
     <link name="${robot_namespace}/base_link"></link>
     <joint name="${robot_namespace}/base_joint" type="fixed">
@@ -69,4 +70,5 @@
         <aeroParamsYAML>${aero_params_yaml}</aeroParamsYAML>
         <vehicleParamsYAML>${vehicle_params_yaml}</vehicleParamsYAML>
+        <isInputJoystick>${is_input_joystick}</isInputJoystick>
       </plugin>
     </gazebo>

File: rotors_description/urdf/techpod.xacro (robot description, xacro)
@@ -15,6 +15,4 @@
   <!-- Global properties -->
   <xacro:property name="namespace" value="$(arg namespace)" />
-  <xacro:property name="aero_params_yaml_file" value="$(arg aero_params_yaml_file)" />
-  <xacro:property name="vehicle_params_yaml_file" value="$(arg vehicle_params_yaml_file)" />
   <xacro:property name="rotor_velocity_slowdown_sim" value="10" />
   <xacro:property name="use_mesh" value="true" />
@@ -110,6 +108,7 @@
     use_mesh_file="${use_mesh}"
     mesh_file="${body_mesh_file}"
-    aero_params_yaml="${aero_params_yaml_file}"
-    vehicle_params_yaml="${vehicle_params_yaml_file}">
+    aero_params_yaml="$(arg aero_params_yaml_file)"
+    vehicle_params_yaml="$(arg vehicle_params_yaml_file)"
+    is_input_joystick="$(arg is_input_joystick)">
     <origin xyz="0 0 0" rpy="0 0 0" />
     <xacro:insert_block name="body_inertia" />

Commit message: Minor fixes

File: rotors_description/urdf/fixed_wing_base.xacro (robot description, xacro)
@@ -84,5 +84,5 @@
       <parent link="${parent}" />
       <child link="${robot_namespace}/${surface_name}" />
-      <limit upper="${max_angle}" lower="${min_angle}" effort="0" velocity="0" />
+      <limit upper="0" lower="0" effort="0" velocity="0" />
     </joint>
     <link name="${robot_namespace}/${surface_name}">
