Commit message: Monocular Camera attached to firefly_drone model

File: rotors_description/urdf/firefly_base.xacro (robot description, xacro)
@@ -16,5 +16,6 @@
   limitations under the License.
 -->
-<robot name="firefly" xmlns:xacro="http://ros.org/wiki/xacro">
+<robot name="firefly"
+  xmlns:xacro="http://ros.org/wiki/xacro">
   <xacro:include filename="$(find rotors_description)/urdf/component_snippets.xacro" />
   <!-- Instantiate firefly "mechanics" -->
@@ -34,5 +35,22 @@
   <xacro:default_magnetometer namespace="${namespace}" parent_link="${namespace}/base_link" />
   <xacro:default_pressure_sensor namespace="${namespace}" parent_link="${namespace}/base_link" />
-  <xacro:camera_macro namespace="${namespace}" parent_link="${namespace}/base_link">
+  <xacro:camera_macro
+    namespace="${namespace}"
+    parent_link="${namespace}/base_link"
+    camera_suffix="${namespace}/camera_suffix"
+    frame_rate="${namespace}/frame_rate"
+    horizontal_fov="1.3962634"
+    image_width="752"
+    image_height="480"
+    image_format="L8"
+    min_distance="0.02"
+    max_distance="30"
+    noise_mean="0.0"
+    noise_stddev="0.007"
+    enable_visual="true">
+    <mesh filename="package://rotors_description/meshes/vi_camera.dae" scale="1 1 1" />
+    <!-- <xacro:insert_block name="origin" /> -->
+    <origin xyz="0 0 -0.05" rpy="0 0 0" />
+  </xacro:camera_macro>
   <xacro:if value="$(arg enable_ground_truth)">
     <xacro:ground_truth_imu_and_odometry namespace="${namespace}" parent_link="${namespace}/base_link" />
@@ -40,9 +58,5 @@
   <xacro:if value="$(arg enable_logging)">
     <!-- Instantiate a logger -->
-    <xacro:bag_plugin_macro
-      namespace="${namespace}"
-      bag_file="$(arg log_file)"
-      rotor_velocity_slowdown_sim="${rotor_velocity_slowdown_sim}"
-      wait_to_record_bag="$(arg wait_to_record_bag)" />
+    <xacro:bag_plugin_macro namespace="${namespace}" bag_file="$(arg log_file)" rotor_velocity_slowdown_sim="${rotor_velocity_slowdown_sim}" wait_to_record_bag="$(arg wait_to_record_bag)" />
   </xacro:if>
 </robot>

Commit message: nearthlab payload model created

File: rotors_description/urdf/firefly_base.xacro (robot description, xacro)
@@ -20,4 +20,5 @@
   <xacro:include filename="$(find rotors_description)/urdf/component_snippets.xacro" />
   <xacro:include filename="$(find rotors_description)/urdf/nearthlab_lidar_sensor.xacro" />
+  <xacro:include filename="$(find rotors_description)/urdf/nearthlab_payload.xacro" />
   <!-- Instantiate firefly "mechanics" -->
   <xacro:include filename="$(find rotors_description)/urdf/firefly.xacro" />
@@ -47,11 +48,10 @@
   </xacro:camera_joint_macro>
   <!--LIDAR Sensor Added by bkjung-->
-  <xacro:lidar_macro namespace="${namespace}" parent_link="${namespace}/base_link">
-    <!-- <origin xyz="0 0 -0.07" rpy="0 0 0" /> -->
+  <!-- <xacro:lidar_macro namespace="${namespace}" parent_link="${namespace}/base_link">
     <origin xyz="0 0 -0.035" rpy="0 0 0" />
     <geometry>
       <cylinder length="0.02" radius="0.015" />
     </geometry>
-  </xacro:lidar_macro>
+  </xacro:lidar_macro> -->
   <xacro:if value="$(arg enable_ground_truth)">
     <xacro:ground_truth_imu_and_odometry namespace="${namespace}" parent_link="${namespace}/base_link" />
@@ -61,3 +61,10 @@
     <xacro:bag_plugin_macro namespace="${namespace}" bag_file="$(arg log_file)" rotor_velocity_slowdown_sim="${rotor_velocity_slowdown_sim}" wait_to_record_bag="$(arg wait_to_record_bag)" />
   </xacro:if>
+  <!--Nearthlab Payload-->
+  <xacro:payload_macro namespace="${namespace}" parent_link="${namespace}/base_link" />
+    <origin xyz="0 0 -0.035" rpy="0 0 0" />
+      <geometry>
+        <mesh filename="package://rotors_description/meshes/nearthlab_payload.dae" scale="1 1 1" />
+      </geometry>
+  </xacro:payload_macro>
 </robot>

Commit message: payload heading revised

File: rotors_description/urdf/firefly_base.xacro (robot description, xacro)
@@ -61,9 +61,8 @@
     <xacro:bag_plugin_macro namespace="${namespace}" bag_file="$(arg log_file)" rotor_velocity_slowdown_sim="${rotor_velocity_slowdown_sim}" wait_to_record_bag="$(arg wait_to_record_bag)" />
   </xacro:if>
-  <!--Nearthlab Payload-->
-  <xacro:payload_macro namespace="${namespace}" parent_link="${namespace}/base_link" />
-    <origin xyz="0 0 -0.035" rpy="0 0 0" />
+  <xacro:payload_macro namespace="${namespace}" parent_link="${namespace}/base_link" >
+    <origin xyz="0 0 -0.07" rpy="0 0 0" />
       <geometry>
-        <mesh filename="package://rotors_description/meshes/nearthlab_payload.dae" scale="1 1 1" />
+        <mesh filename="package://rotors_description/meshes/nearthlab_payload.dae" scale="0.0005 0.0005 0.0005" />
       </geometry>
   </xacro:payload_macro>

File: rotors_description/urdf/nearthlab_payload.xacro (robot description, xacro)
@@ -1,3 +1,2 @@
-<!-- copied most of nearthlab_lidar_sensor.xacro-->
 <?xml version="1.0"?>
 <robot xmlns:xacro="http://ros.org/wiki/xacro">
@@ -11,5 +10,5 @@
       </inertial>
       <visual>
-        <origin xyz="0 0 0" rpy="0 0 0" />
+        <origin xyz="0 0 0" rpy="0 ${pi/2} ${pi/2}" />
         <geometry>
           <xacro:insert_block name="geometry" />

Commit message: Nearthlab Windturbine 3D Model (A shape & Y shape) added

File: rotors_description/urdf/firefly_base.xacro (robot description, xacro)
@@ -63,9 +63,9 @@
   </xacro:lidar_macro>
   <!-- Nearthlab Payload -->
-  <!-- <xacro:payload_macro namespace="${namespace}" parent_link="${namespace}/base_link" > -->
-    <!-- <origin xyz="0 0 -0.06" rpy="0 0 0" /> -->
-      <!-- <geometry> -->
-        <!-- <mesh filename="package://rotors_description/meshes/nearthlab_payload.dae" scale="0.0004 0.0004 0.0004" /> -->
-      <!-- </geometry> -->
-  <!-- </xacro:payload_macro> -->
+  <xacro:payload_macro namespace="${namespace}" parent_link="${namespace}/base_link" >
+    <origin xyz="0 0 -0.06" rpy="0 0 0" />
+      <geometry>
+        <mesh filename="package://rotors_description/meshes/nearthlab_payload.dae" scale="0.0004 0.0004 0.0004" />
+      </geometry>
+  </xacro:payload_macro>
 </robot>

Commit message: WindTurbine Model updated

File: rotors_description/urdf/firefly_base.xacro (robot description, xacro)
@@ -21,4 +21,5 @@
   <xacro:include filename="$(find rotors_description)/urdf/nearthlab_lidar_sensor.xacro" />
   <xacro:include filename="$(find rotors_description)/urdf/nearthlab_payload.xacro" />
+  <xacro:include filename="$(find rotors_description)/urdf/nearthlab_windturbine.xacro" />
   <!-- Instantiate firefly "mechanics" -->
   <xacro:include filename="$(find rotors_description)/urdf/firefly.xacro" />
@@ -57,5 +58,6 @@
   <!--LIDAR Sensor-->
   <xacro:lidar_macro namespace="${namespace}" parent_link="${namespace}/base_link">
-    <origin xyz="0 0 -0.035" rpy="0 0 0" />
+    <!-- <origin xyz="0 0 -0.035" rpy="0 0 0" /> -->
+    <origin xyz="0 0 0" rpy="0 0 0" />
     <geometry>
       <cylinder length="0.02" radius="0.015" />
@@ -63,9 +65,16 @@
   </xacro:lidar_macro>
   <!-- Nearthlab Payload -->
-  <xacro:payload_macro namespace="${namespace}" parent_link="${namespace}/base_link" >
+  <!-- <xacro:payload_macro namespace="${namespace}" parent_link="${namespace}/base_link" >
     <origin xyz="0 0 -0.06" rpy="0 0 0" />
       <geometry>
         <mesh filename="package://rotors_description/meshes/nearthlab_payload.dae" scale="0.0004 0.0004 0.0004" />
       </geometry>
-  </xacro:payload_macro>
+  </xacro:payload_macro> -->
+  <!-- Nearthlab Windturbine -->
+  <xacro:windturbine_macro namespace="${namespace}" parent_link="${namespace}/base_link" >
+    <origin xyz="0 0 0" rpy="0 0 0" />
+      <geometry>
+        <mesh filename="package://rotors_description/meshes/nearthlab_windturbine_A_shape.dae" scale="0.05 0.05 0.05" />
+      </geometry>
+  </xacro:windturbine_macro>
 </robot>

File: rotors_description/urdf/nearthlab_lidar_sensor.xacro (robot description, xacro)
@@ -9,12 +9,16 @@
         <inertia ixx="2.1733e-6" ixy="0" ixz="0" iyy="2.1733e-6" iyz="0" izz="1.8e-7" />
       </inertial>
-      <visual>
-        <origin xyz="0 0 0" rpy="0 ${pi/2} 0" />
+      <visual name="visual">
+        <origin xyz="0 0 -0.035" rpy="0 ${pi/2} 0" />
+        <!-- <geometry>
+          <cylinder length="0.02" radius="0.015" />
+        </geometry> -->
         <geometry>
           <xacro:insert_block name="geometry" />
         </geometry>
-        <material name="black">
-          <!-- <script>Gazebo/Black</script> -->
-        </material>
+        <!-- <material>
+          <script>Gazebo/Black</script>
+        </material> -->
+        <material name="black" />
       </visual>
     </link>
@@ -24,11 +28,7 @@
       <child link="${namespace}/lidar_link" />
     </joint>
-    <gazebo reference="${namespace}/lidar_link">
-      <!-- <sensor name="laser" type="ray"> -->
+    <gazebo>
       <sensor type="ray" name="${namespace}_lidar">
         <pose>0 0 0 0 -1.570896 0</pose>
-        <always_on>1</always_on>
-        <update_rate>20</update_rate>
-        <visualize>true</visualize>
         <ray>
           <scan>
@@ -51,9 +51,9 @@
           </noise>
         </ray>
-        <plugin filename="librotors_gazebo_lidar_plugin.so" name="rotors_gazebo_lidar_plugin">
-          <robotNamespace>${namespace}</robotNamespace>
-          <linkName>${namespace}/lidar_link</linkName>
-          <lidarTopic>lidar</lidarTopic>
-        </plugin>
+	      <plugin name="LaserPlugin" filename="librotors_gazebo_lidar_plugin.so"/>
+		    <robotNamespace></robotNamespace>
+        <always_on>1</always_on>
+        <update_rate>20</update_rate>
+        <visualize>true</visualize>
       </sensor>
     </gazebo>

File: rotors_description/urdf/nearthlab_windturbine.xacro (robot description, xacro)
@@ -2,6 +2,6 @@
 <robot xmlns:xacro="http://ros.org/wiki/xacro">
   <xacro:property name="pi" value="3.14159265359" />
-  <xacro:macro name="payload_macro" params="namespace parent_link *origin **geometry">
-    <link name="${namespace}/payload_link">
+  <xacro:macro name="windturbine_macro" params="namespace parent_link *origin **geometry">
+    <link name="${namespace}/windturbine_link">
       <inertial>
         <pose>0 0 0 0 -0 0</pose>
@@ -9,20 +9,20 @@
         <inertia ixx="2.1733e-6" ixy="0" ixz="0" iyy="2.1733e-6" iyz="0" izz="1.8e-7" />
       </inertial>
-      <visual name="visual">
-        <origin xyz="0 0 0" rpy="${pi/2} 0 ${pi/2}" />
+      <visual>
+        <origin xyz="3 0 0" rpy="0 0 0" />
         <geometry>
           <xacro:insert_block name="geometry" />
         </geometry>
-        <material name="black" />
+        <material name="white" />
       </visual>
     </link>
-    <joint name="${namespace}_payload_joint" type="fixed">
+    <joint name="${namespace}_windturbine_joint" type="fixed">
       <xacro:insert_block name="origin" />
       <parent link="${parent_link}" />
-      <child link="${namespace}/payload_link" />
+      <child link="${namespace}/windturbine_link" />
     </joint>
     <gazebo>
       <!-- <sensor name="laser" type="ray"> -->
-      <sensor type="ray" name="${namespace}_payload">
+      <sensor type="ray" name="${namespace}_windturbine">
         <pose>0 0 0 0 -1.570896 0</pose>
         <ray>
