Commit message: add NIVv1 related files

File: rotors_description/urdf/niv1.xacro (robot description, xacro)
@@ -16,32 +16,41 @@
   limitations under the License.
 -->
-<robot name="firefly" xmlns:xacro="http://ros.org/wiki/xacro">
+<robot name="niv1" xmlns:xacro="http://ros.org/wiki/xacro">
   <!-- Properties -->
   <xacro:property name="namespace" value="$(arg namespace)" />
   <xacro:property name="rotor_velocity_slowdown_sim" value="10" />
   <xacro:property name="use_mesh_file" value="true" />
-  <xacro:property name="mesh_file" value="package://rotors_description/meshes/firefly_red.dae" />
-  <xacro:property name="mass" value="1.5" /> <!-- [kg] -->
-  <xacro:property name="body_width" value="0.1" /> <!-- [m] -->
-  <xacro:property name="body_height" value="0.16" /> <!-- [m] -->
-  <xacro:property name="mass_rotor" value="0.005" /> <!-- [kg] -->
-  <xacro:property name="arm_length" value="0.215" /> <!-- [m] -->
-  <xacro:property name="rotor_offset_top" value="0.037" /> <!-- [m] -->
-  <xacro:property name="radius_rotor" value="0.1" /> <!-- [m] -->
-  <xacro:property name="motor_constant" value="8.54858e-06" /> <!-- [kg m/s^2] -->
-  <xacro:property name="moment_constant" value="0.016" /> <!-- [m] -->
-  <xacro:property name="time_constant_up" value="0.0125" /> <!-- [s] -->
-  <xacro:property name="time_constant_down" value="0.025" /> <!-- [s] -->
-  <xacro:property name="max_rot_velocity" value="838" /> <!-- [rad/s] -->
-  <xacro:property name="sin30" value="0.5" />
-  <xacro:property name="cos30" value="0.866025403784" />
-  <xacro:property name="rotor_drag_coefficient" value="8.06428e-05" />
-  <xacro:property name="rolling_moment_coefficient" value="0.000001" />
+  <xacro:property name="mesh_file" value="package://rotors_description/meshes/niv1_body.dae" />
+  <xacro:property name="mass" value="12" /> <!-- [kg] -->
+  <xacro:property name="body_width" value="0.2" /> <!-- [m] -->
+  <xacro:property name="body_height" value="0.2" /> <!-- [m] -->
+  <xacro:property name="mass_rotor" value="0.2" /> <!-- [kg] -->
+  <xacro:property name="arm_length" value="0.636" /> <!-- [m] -->
+  <xacro:property name="rotor_offset_top" value="0.053" /> <!-- [m] -->
+  <xacro:property name="radius_rotor" value="0.3" /> <!-- [m] -->
+  <xacro:property name="motor_constant_for_ros_sim" value="8.54858e-05" /> <!-- [kg m/s^2]  force = real_motor_velocity * real_motor_velocity * motor_constant_-->
+  <xacro:property name="motor_constant_bak" value="0.9e-04" /> <!-- [kg m/s^2]  force = real_motor_velocity * real_motor_velocity * motor_constant_-->
+  <xacro:property name="motor_constant" value="8.9e-05" /> <!-- [kg m/s^2]  force = real_motor_velocity * real_motor_velocity * motor_constant_-->
+  <xacro:property name="moment_constant" value="0.025" /> <!-- [m] math::Vector3 drag_torque(0, 0, -turning_direction_ * force * moment_constant_); -->
+  <xacro:property name="moment_constan_org" value="0.025" /> <!-- [m] math::Vector3 drag_torque(0, 0, -turning_direction_ * force * moment_constant_); -->
+  <xacro:property name="time_constant_up_org" value="0.0125" /> <!-- [s] -->
+  <xacro:property name="time_constant_down_org" value="0.025" /> <!-- [s] -->
+  <xacro:property name="time_constant_up" value="0.00001" /> <!-- [s] -->
+  <xacro:property name="time_constant_down" value="0.00001" /> <!-- [s] -->
+  <xacro:property name="max_rot_velocity" value="1838" /> <!-- [rad/s] -->
+  <xacro:property name="rotor_pos_x" value="0.45" />
+  <xacro:property name="rotor_pos_y" value="0.45" />
+  <xacro:property name="rotor_drag_coefficient" value="8.06428e-05" /> <!-- math::Vector3 air_drag = -std::abs(real_motor_velocity) * rotor_drag_coefficient_ * body_velocity_perpendicular; -->
+  <xacro:property name="rolling_moment_coefficient" value="0.000001" /> <!-- math::Vector3 rolling_moment = -std::abs(real_motor_velocity) * rolling_moment_coefficient_ * body_velocity_perpendicular; -->
   <!-- Property Blocks -->
   <xacro:property name="body_inertia">
-    <inertia ixx="0.0347563" ixy="0.0" ixz="0.0" iyy="0.0458929" iyz="0.0" izz="0.0977" /> <!-- [kg m^2] [kg m^2] [kg m^2] [kg m^2] [kg m^2] [kg m^2] -->
+    <!--
+    <inertia ixx="0.0347563" ixy="0.0" ixz="0.0" iyy="0.0458929" iyz="0.0" izz="0.0977" /> [kg m^2] [kg m^2] [kg m^2] [kg m^2] [kg m^2] [kg m^2] -->
+    <!-- <inertia ixx="0.801" ixy="0.0" ixz="0.0" iyy="0.827" iyz="0.0" izz="1.450" /> -->
+    <inertia ixx="1.5" ixy="0.0" ixz="0.0" iyy="1.5" iyz="0.0" izz="10.0" />
   </xacro:property>
-  <!-- inertia of a single rotor, assuming it is a cuboid. Height=3mm, width=15mm -->
+  <!-- inertia of a single rotor, assuming it is a cuboid. -->
   <xacro:property name="rotor_inertia">
+    <!-- <xacro:box_inertia x="${radius_rotor}" y="0.015" z="0.003" mass="${mass_rotor*rotor_velocity_slowdown_sim}" /> -->
     <xacro:box_inertia x="${radius_rotor}" y="0.015" z="0.003" mass="${mass_rotor*rotor_velocity_slowdown_sim}" />
   </xacro:property>
@@ -60,7 +69,7 @@
   </xacro:multirotor_base_macro>
   <!-- Instantiate rotors -->
-  <xacro:vertical_rotor
+    <xacro:vertical_rotor
     robot_namespace="${namespace}"
-    suffix="front_left"
+    suffix="front_right"
     direction="ccw"
     motor_constant="${motor_constant}"
@@ -75,13 +84,13 @@
     rotor_drag_coefficient="${rotor_drag_coefficient}"
     rolling_moment_coefficient="${rolling_moment_coefficient}"
-    color="Red"
+    color="Grey"
     use_own_mesh="false"
     mesh="">
-    <origin xyz="${cos30*arm_length} ${sin30*arm_length} ${rotor_offset_top}" rpy="0 0 0" />
+     <origin xyz="${rotor_pos_x} -${rotor_pos_y} ${rotor_offset_top}" rpy="0 0 0" />
     <xacro:insert_block name="rotor_inertia" />
   </xacro:vertical_rotor>
   <xacro:vertical_rotor
     robot_namespace="${namespace}"
-    suffix="left"
+    suffix="front_left"
     direction="cw"
     motor_constant="${motor_constant}"
@@ -96,8 +105,8 @@
     rotor_drag_coefficient="${rotor_drag_coefficient}"
     rolling_moment_coefficient="${rolling_moment_coefficient}"
-    color="Blue"
+    color="Grey"
     use_own_mesh="false"
     mesh="">
-    <origin xyz="0 ${arm_length} ${rotor_offset_top}" rpy="0 0 0" />
+    <origin xyz="${rotor_pos_x} ${rotor_pos_y} ${rotor_offset_top}" rpy="0 0 0" />
     <xacro:insert_block name="rotor_inertia" />
   </xacro:vertical_rotor>
@@ -116,8 +125,8 @@
     rotor_drag_coefficient="${rotor_drag_coefficient}"
     rolling_moment_coefficient="${rolling_moment_coefficient}"
-    color="Blue"
+    color="Grey"
     use_own_mesh="false"
     mesh="">
-    <origin xyz="-${cos30*arm_length} ${sin30*arm_length} ${rotor_offset_top}" rpy="0 0 0" />
+    <origin xyz="-${rotor_pos_x} ${rotor_pos_y} ${rotor_offset_top}" rpy="0 0 0" />
     <xacro:insert_block name="rotor_inertia" />
   </xacro:vertical_rotor>
@@ -136,50 +145,8 @@
     rotor_drag_coefficient="${rotor_drag_coefficient}"
     rolling_moment_coefficient="${rolling_moment_coefficient}"
-    color="Blue"
+    color="Grey"
     use_own_mesh="false"
     mesh="">
-    <origin xyz="-${cos30*arm_length} -${sin30*arm_length} ${rotor_offset_top}" rpy="0 0 0" />
-    <xacro:insert_block name="rotor_inertia" />
-  </xacro:vertical_rotor>
-  <xacro:vertical_rotor
-    robot_namespace="${namespace}"
-    suffix="right"
-    direction="ccw"
-    motor_constant="${motor_constant}"
-    moment_constant="${moment_constant}"
-    parent="${namespace}/base_link"
-    mass_rotor="${mass_rotor}"
-    radius_rotor="${radius_rotor}"
-    time_constant_up="${time_constant_up}"
-    time_constant_down="${time_constant_down}"
-    max_rot_velocity="${max_rot_velocity}"
-    motor_number="4"
-    rotor_drag_coefficient="${rotor_drag_coefficient}"
-    rolling_moment_coefficient="${rolling_moment_coefficient}"
-    color="Blue"
-    use_own_mesh="false"
-    mesh="">
-    <origin xyz="0 -${arm_length} ${rotor_offset_top}" rpy="0 0 0" />
-    <xacro:insert_block name="rotor_inertia" />
-  </xacro:vertical_rotor>
-  <xacro:vertical_rotor
-    robot_namespace="${namespace}"
-    suffix="front_right"
-    direction="cw"
-    motor_constant="${motor_constant}"
-    moment_constant="${moment_constant}"
-    parent="${namespace}/base_link"
-    mass_rotor="${mass_rotor}"
-    radius_rotor="${radius_rotor}"
-    time_constant_up="${time_constant_up}"
-    time_constant_down="${time_constant_down}"
-    max_rot_velocity="${max_rot_velocity}"
-    motor_number="5"
-    rotor_drag_coefficient="${rotor_drag_coefficient}"
-    rolling_moment_coefficient="${rolling_moment_coefficient}"
-    color="Red"
-    use_own_mesh="false"
-    mesh="">
-    <origin xyz="${cos30*arm_length} -${sin30*arm_length} ${rotor_offset_top}" rpy="0 0 0" />
+    <origin xyz="-${rotor_pos_x} -${rotor_pos_y} ${rotor_offset_top}" rpy="0 0 0" />
     <xacro:insert_block name="rotor_inertia" />
   </xacro:vertical_rotor>

File: rotors_description/urdf/niv1_base.xacro (robot description, xacro)
@@ -16,5 +16,5 @@
   limitations under the License.
 -->
-<robot name="firefly"
+<robot name="niv1"
   xmlns:xacro="http://ros.org/wiki/xacro">
   <xacro:include filename="$(find rotors_description)/urdf/component_snippets.xacro" />
@@ -22,6 +22,6 @@
   <xacro:include filename="$(find rotors_description)/urdf/nearthlab_payload.xacro" />
   <xacro:include filename="$(find rotors_description)/urdf/nearthlab_windturbine.xacro" />
-  <!-- Instantiate firefly "mechanics" -->
-  <xacro:include filename="$(find rotors_description)/urdf/firefly.xacro" />
+  <!-- Instantiate niv1 "mechanics" -->
+  <xacro:include filename="$(find rotors_description)/urdf/niv1.xacro" />
   <!-- Instantiate a controller. -->
   <xacro:controller_plugin_macro namespace="${namespace}" imu_sub_topic="imu" />
