Commit message: wip adjust conventions to match hardware

File: rotors_description/urdf/dextar_manipulator.xacro (robot description, xacro)
@@ -3,7 +3,9 @@
   <xacro:include filename="$(find rotors_description)/urdf/manipulator_snippets.xacro" />
   <xacro:property name="link_radius" value="0.02"/>
-  <xacro:property name="link1_length" value="0.296"/>
-  <xacro:property name="link2_length" value="0.5"/>
-  <xacro:property name="link0_center_to_center_length" value="0.1"/>
+  <xacro:property name="link1_length" value="0.315"/>
+  <xacro:property name="link2_length" value="0.455"/>
+  <xacro:property name="link0_center_to_center_length" value="0.08"/>
+  <xacro:property name="joint_1_offset" value="2.70"/>
+  <xacro:property name="joint_2_offset" value="0.44"/>
   <xacro:property name="link0_frame">
     <origin xyz="0 0 0" rpy="0 0 0"/>
@@ -53,12 +55,12 @@
           </link>
           <link name="${namespace}/link1_1">
-            <!-- <collision>
-              <origin xyz="0 0 0" rpy="0 0 0"/>
+            <collision>
+              <origin xyz="0 0 0" rpy="3.14 0 0"/>
               <geometry>
                 <mesh filename="package://rotors_description/meshes/dextar_manipulator/link1_1.dae"/>
               </geometry>
-            </collision> -->
-            <visual>
-              <origin xyz="0 0 0" rpy="0 0 0"/>
+            </collision>
+            <visual>
+              <origin xyz="0 0 0" rpy="3.14 0 0"/>
               <geometry>
                 <mesh filename="package://rotors_description/meshes/dextar_manipulator/link1_1.dae"/>
@@ -71,12 +73,12 @@
           </link>
           <link name="${namespace}/link1_2">
-            <!-- <collision>
-              <origin xyz="0 0 0" rpy="0 0 0"/>
+            <collision>
+              <origin xyz="0 0 0" rpy="3.14 0 0"/>
               <geometry>
                 <mesh filename="package://rotors_description/meshes/dextar_manipulator/link1_2.dae"/>
               </geometry>
-            </collision> -->
-            <visual>
-              <origin xyz="0 0 0" rpy="0 0 0"/>
+            </collision>
+            <visual>
+              <origin xyz="0 0 0" rpy="3.14 0 0"/>
               <geometry>
                 <mesh filename="package://rotors_description/meshes/dextar_manipulator/link1_2.dae"/>
@@ -127,49 +129,49 @@
           <xacro:revolute_joint_macro
             namespace="${namespace}"
-            joint_name="delta_manipulator/joint_1"
+            joint_name="dextar_manipulator/joint_1"
             parent_link="${namespace}/manipulator_base_link"
             child_link="${namespace}/link1_1"
-            axis="0 0 -1"
-            friction="0"
-            damping="0.1">
-            <origin xyz="${-link0_center_to_center_length/2} 0 -0.005" rpy="0 0 0"/>
-          </xacro:revolute_joint_macro>
-          <xacro:revolute_joint_macro
-            namespace="${namespace}"
-            joint_name="delta_manipulator/joint_2"
+            axis="0 0 1"
+            friction="0"
+            damping="0.1">
+            <origin xyz="${-link0_center_to_center_length/2} 0 0" rpy="0 0 ${joint_1_offset}"/>
+          </xacro:revolute_joint_macro>
+          <xacro:revolute_joint_macro
+            namespace="${namespace}"
+            joint_name="dextar_manipulator/joint_2"
             parent_link="${namespace}/manipulator_base_link"
             child_link="${namespace}/link1_2"
-            axis="0 0 -1"
-            friction="0"
-            damping="0.1">
-            <origin xyz="${link0_center_to_center_length/2} 0 -0.005" rpy="0 0 0"/>
-          </xacro:revolute_joint_macro>
-          <xacro:revolute_joint_macro
-            namespace="${namespace}"
-            joint_name="delta_manipulator/joint_3"
+            axis="0 0 1"
+            friction="0"
+            damping="0.1">
+            <origin xyz="${link0_center_to_center_length/2} 0 0" rpy="0 0 ${joint_2_offset}"/>
+          </xacro:revolute_joint_macro>
+          <xacro:revolute_joint_macro
+            namespace="${namespace}"
+            joint_name="dextar_manipulator/joint_3"
             parent_link="${namespace}/link1_1"
             child_link="${namespace}/link2_1"
-            axis="0 0 -1"
-            friction="0"
-            damping="0.1">
-            <origin xyz="${link1_length} 0 -0.0145" rpy="0 0 0"/>
-          </xacro:revolute_joint_macro>
-          <xacro:revolute_joint_macro
-            namespace="${namespace}"
-            joint_name="delta_manipulator/joint_4"
+            axis="0 0 1"
+            friction="0"
+            damping="0.1">
+            <origin xyz="${link1_length} 0 0.016" rpy="0 0 0"/>
+          </xacro:revolute_joint_macro>
+          <xacro:revolute_joint_macro
+            namespace="${namespace}"
+            joint_name="dextar_manipulator/joint_4"
             parent_link="${namespace}/link1_2"
             child_link="${namespace}/link2_2"
-            axis="0 0 -1"
-            friction="0"
-            damping="0.1">
-            <origin xyz="${link1_length} 0 -0.0145" rpy="0 0 0"/>
+            axis="0 0 1"
+            friction="0"
+            damping="0.1">
+            <origin xyz="${link1_length} 0 0.016" rpy="0 0 0"/>
           </xacro:revolute_joint_macro>
           <xacro:gazebo_revolute_joint_macro
             namespace="${namespace}"
-            joint_name="delta_manipulator/joint_5"
+            joint_name="dextar_manipulator/joint_5"
             parent_link="${namespace}/link2_1"
             child_link="${namespace}/link2_2"
             pose="${link2_length} 0 0 0 0 0"
-            axis="0 0 -1"
+            axis="0 0 1"
             friction="0"
             damping="0.1"
@@ -193,5 +195,5 @@
           motor_name="X5-4/M1"
           parent_link="${namespace}/manipulator_base_link"
-          actuated_joint="delta_manipulator/joint_1"
+          actuated_joint="dextar_manipulator/joint_1"
           maxTorque="2"
           noLoadSpeed="0.11"
@@ -213,5 +215,5 @@
           visual_scale="1"
           color="Red">
-          <origin xyz="${link0_center_to_center_length/2} 0 0" rpy="3.14 0 1.57"/>
+          <origin xyz="${link0_center_to_center_length/2} 0 0" rpy="0 0 -1.57"/>
           <xacro:insert_block name="generic_servo_inertial"/>
         </xacro:hebi_actuator_plugin>
@@ -220,5 +222,5 @@
           motor_name="X5-4/M2"
           parent_link="${namespace}/manipulator_base_link"
-          actuated_joint="delta_manipulator/joint_2"
+          actuated_joint="dextar_manipulator/joint_2"
           maxTorque="2"
           noLoadSpeed="0.11"
@@ -240,5 +242,5 @@
           visual_scale="1"
           color="Red">
-          <origin xyz="${-link0_center_to_center_length/2} 0 0" rpy="3.14 0 1.57"/>
+          <origin xyz="${-link0_center_to_center_length/2} 0 0" rpy="0 0 -1.57"/>
           <xacro:insert_block name="generic_servo_inertial"/>
         </xacro:hebi_actuator_plugin>
@@ -248,11 +250,11 @@
             <robotNamespace>${namespace}</robotNamespace>
             <initial_configuration>
-              <config joint_name="delta_manipulator/joint_1"  initial_position="-2.7342"/>
-              <config joint_name="delta_manipulator/joint_3"  initial_position=" 1.8625"/>
-              <config joint_name="delta_manipulator/joint_2" initial_position="-0.4074"/>
-              <config joint_name="delta_manipulator/joint_4" initial_position="-1.8625"/>
+              <config joint_name="dextar_manipulator/joint_1"  initial_position=" 0.0"/>
+              <config joint_name="dextar_manipulator/joint_3"  initial_position="-1.8806"/>
+              <config joint_name="dextar_manipulator/joint_2"  initial_position=" 0.0"/>
+              <config joint_name="dextar_manipulator/joint_4"  initial_position="1.8806"/>
             </initial_configuration>
             <loop_closure_joints>
-              <joint joint_name="delta_manipulator/joint_5"/>
+              <joint joint_name="dextar_manipulator/joint_5"/>
             </loop_closure_joints>
           </plugin>

Commit message: fix namespace and joint state publisher for dextar

File: rotors_description/urdf/dextar_manipulator.xacro (robot description, xacro)
@@ -129,5 +129,5 @@
           <xacro:revolute_joint_macro
             namespace="${namespace}"
-            joint_name="dextar_manipulator/joint_1"
+            joint_name="${namespace}/joint_1"
             parent_link="${namespace}/manipulator_base_link"
             child_link="${namespace}/link1_1"
@@ -139,5 +139,5 @@
           <xacro:revolute_joint_macro
             namespace="${namespace}"
-            joint_name="dextar_manipulator/joint_2"
+            joint_name="${namespace}/joint_2"
             parent_link="${namespace}/manipulator_base_link"
             child_link="${namespace}/link1_2"
@@ -149,5 +149,5 @@
           <xacro:revolute_joint_macro
             namespace="${namespace}"
-            joint_name="dextar_manipulator/joint_3"
+            joint_name="${namespace}/joint_3"
             parent_link="${namespace}/link1_1"
             child_link="${namespace}/link2_1"
@@ -159,5 +159,5 @@
           <xacro:revolute_joint_macro
             namespace="${namespace}"
-            joint_name="dextar_manipulator/joint_4"
+            joint_name="${namespace}/joint_4"
             parent_link="${namespace}/link1_2"
             child_link="${namespace}/link2_2"
@@ -169,5 +169,5 @@
           <xacro:gazebo_revolute_joint_macro
             namespace="${namespace}"
-            joint_name="dextar_manipulator/joint_5"
+            joint_name="${namespace}/joint_5"
             parent_link="${namespace}/link2_1"
             child_link="${namespace}/link2_2"
@@ -195,5 +195,5 @@
           motor_name="X5-4/M1"
           parent_link="${namespace}/manipulator_base_link"
-          actuated_joint="dextar_manipulator/joint_1"
+          actuated_joint="${namespace}/joint_1"
           maxTorque="2"
           noLoadSpeed="0.11"
@@ -222,5 +222,5 @@
           motor_name="X5-4/M2"
           parent_link="${namespace}/manipulator_base_link"
-          actuated_joint="dextar_manipulator/joint_2"
+          actuated_joint="${namespace}/joint_2"
           maxTorque="2"
           noLoadSpeed="0.11"
@@ -250,11 +250,11 @@
             <robotNamespace>${namespace}</robotNamespace>
             <initial_configuration>
-              <config joint_name="dextar_manipulator/joint_1"  initial_position=" 0.0"/>
-              <config joint_name="dextar_manipulator/joint_3"  initial_position="-1.8806"/>
-              <config joint_name="dextar_manipulator/joint_2"  initial_position=" 0.0"/>
-              <config joint_name="dextar_manipulator/joint_4"  initial_position="1.8806"/>
+              <config joint_name="${namespace}/joint_1"  initial_position=" 0.0"/>
+              <config joint_name="${namespace}/joint_3"  initial_position="-1.8806"/>
+              <config joint_name="${namespace}/joint_2"  initial_position=" 0.0"/>
+              <config joint_name="${namespace}/joint_4"  initial_position="1.8806"/>
             </initial_configuration>
             <loop_closure_joints>
-              <joint joint_name="dextar_manipulator/joint_5"/>
+              <joint joint_name="${namespace}/joint_5"/>
             </loop_closure_joints>
           </plugin>

File: rotors_description/urdf/manipulator_snippets.xacro (robot description, xacro)
@@ -178,5 +178,6 @@
     <material>Gazebo/${color}</material>
   </gazebo>
-  <joint name="${namespace}/${motor_name}" type="revolute">
+  <!-- name does not contain namespace to match hardware -->
+  <joint name="${motor_name}" type="revolute">
     <parent link="${parent_link}"/>
     <child link="${namespace}/${motor_name}"/>

Commit message: set effort gain and inital joint pos

File: rotors_description/urdf/dextar_manipulator.xacro (robot description, xacro)
@@ -8,4 +8,5 @@
   <xacro:property name="joint_1_offset" value="2.70"/>
   <xacro:property name="joint_2_offset" value="0.44"/>
+  <xacro:property name="joint_34_offset" value="1.9248"/>
   <xacro:property name="link0_frame">
     <origin xyz="0 0 0" rpy="0 0 0"/>
@@ -251,7 +252,7 @@
             <initial_configuration>
               <config joint_name="${namespace}/joint_1"  initial_position=" 0.0"/>
-              <config joint_name="${namespace}/joint_3"  initial_position="-1.8806"/>
+              <config joint_name="${namespace}/joint_3"  initial_position="${-joint_34_offset}"/>
               <config joint_name="${namespace}/joint_2"  initial_position=" 0.0"/>
-              <config joint_name="${namespace}/joint_4"  initial_position="1.8806"/>
+              <config joint_name="${namespace}/joint_4"  initial_position="${ joint_34_offset}"/>
             </initial_configuration>
             <loop_closure_joints>

File: rotors_description/urdf/manipulator_snippets.xacro (robot description, xacro)
@@ -193,6 +193,6 @@
       <position_kp>0.2</position_kp>
       <velocity_kp>0.1</velocity_kp>
-      <effort_kp>0.0</effort_kp>
-      <effort_kd>0.0</effort_kd>
+      <effort_kp>0.04</effort_kp>
+      <effort_kd>0.005</effort_kd>
       <effort_output_lp>0.5</effort_output_lp>
       <effort_D_on_error>false</effort_D_on_error>

Commit message: add force sensor and dummy meshes

File: rotors_description/urdf/dextar_manipulator.xacro (robot description, xacro)
@@ -2,5 +2,5 @@
 <robot xmlns:xacro="http://ros.org/wiki/xacro">
   <xacro:include filename="$(find rotors_description)/urdf/manipulator_snippets.xacro" />
-  <xacro:property name="link_radius" value="0.02"/>
+  <xacro:property name="link_radius" value="0.01"/>
   <xacro:property name="link1_length" value="0.315"/>
   <xacro:property name="link2_length" value="0.455"/>
@@ -56,15 +56,29 @@
           </link>
           <link name="${namespace}/link1_1">
+            <!-- <collision>
+              <origin xyz="0 0 0" rpy="3.14 0 0"/>
+              <geometry>
+                <mesh filename="package://rotors_description/meshes/dextar_manipulator/link1_1.dae"/>
+              </geometry>
+            </collision>
+            <visual>
+              <origin xyz="0 0 0" rpy="3.14 0 0"/>
+              <geometry>
+                <mesh filename="package://rotors_description/meshes/dextar_manipulator/link1_1.dae"/>
+              </geometry>
+            </visual> -->
             <collision>
-              <origin xyz="0 0 0" rpy="3.14 0 0"/>
-              <geometry>
-                <mesh filename="package://rotors_description/meshes/dextar_manipulator/link1_1.dae"/>
-              </geometry>
-            </collision>
-            <visual>
-              <origin xyz="0 0 0" rpy="3.14 0 0"/>
-              <geometry>
-                <mesh filename="package://rotors_description/meshes/dextar_manipulator/link1_1.dae"/>
-              </geometry>
+              <origin rpy="0 1.57 0" xyz="${link1_length/2} 0 0"/>
+              <geometry>
+                <cylinder radius="${link_radius}" length="${link1_length}" />
+              </geometry>
+      	       <material name="white"/>
+            </collision>
+            <visual>
+              <origin rpy="0 1.57 0" xyz="${link1_length/2} 0 0"/>
+              <geometry>
+                <cylinder radius="${link_radius}" length="${link1_length}" />
+              </geometry>
+      	       <material name="white"/>
             </visual>
             <inertial>
@@ -74,15 +88,29 @@
           </link>
           <link name="${namespace}/link1_2">
+            <!-- <collision>
+              <origin xyz="0 0 0" rpy="3.14 0 0"/>
+              <geometry>
+                <mesh filename="package://rotors_description/meshes/dextar_manipulator/link1_2.dae"/>
+              </geometry>
+            </collision>
+            <visual>
+              <origin xyz="0 0 0" rpy="3.14 0 0"/>
+              <geometry>
+                <mesh filename="package://rotors_description/meshes/dextar_manipulator/link1_2.dae"/>
+              </geometry>
+            </visual> -->
             <collision>
-              <origin xyz="0 0 0" rpy="3.14 0 0"/>
-              <geometry>
-                <mesh filename="package://rotors_description/meshes/dextar_manipulator/link1_2.dae"/>
-              </geometry>
-            </collision>
-            <visual>
-              <origin xyz="0 0 0" rpy="3.14 0 0"/>
-              <geometry>
-                <mesh filename="package://rotors_description/meshes/dextar_manipulator/link1_2.dae"/>
-              </geometry>
+              <origin rpy="0 1.57 0" xyz="${link1_length/2} 0 0"/>
+              <geometry>
+                <cylinder radius="${link_radius}" length="${link1_length}" />
+              </geometry>
+      	       <material name="white"/>
+            </collision>
+            <visual>
+              <origin rpy="0 1.57 0" xyz="${link1_length/2} 0 0"/>
+              <geometry>
+                <cylinder radius="${link_radius}" length="${link1_length}" />
+              </geometry>
+      	       <material name="white"/>
             </visual>
             <inertial>
@@ -92,15 +120,29 @@
           </link>
           <link name="${namespace}/link2_1">
+            <!-- <collision>
+              <origin xyz="0 0 0" rpy="0 0 0"/>
+              <geometry>
+                <mesh filename="package://rotors_description/meshes/dextar_manipulator/link2_1.dae"/>
+              </geometry>
+            </collision>
+            <visual>
+              <origin xyz="0 0 0" rpy="0 0 0"/>
+              <geometry>
+                <mesh filename="package://rotors_description/meshes/dextar_manipulator/link2_1.dae"/>
+              </geometry>
+            </visual> -->
             <collision>
-              <origin xyz="0 0 0" rpy="0 0 0"/>
-              <geometry>
-                <mesh filename="package://rotors_description/meshes/dextar_manipulator/link2_1.dae"/>
-              </geometry>
-            </collision>
-            <visual>
-              <origin xyz="0 0 0" rpy="0 0 0"/>
-              <geometry>
-                <mesh filename="package://rotors_description/meshes/dextar_manipulator/link2_1.dae"/>
-              </geometry>
+              <origin rpy="0 1.57 0" xyz="${link1_length/2} 0 0"/>
+              <geometry>
+                <cylinder radius="${link_radius}" length="${link2_length}" />
+              </geometry>
+      	       <material name="white"/>
+            </collision>
+            <visual>
+              <origin rpy="0 1.57 0" xyz="${link2_length/2} 0 0"/>
+              <geometry>
+                <cylinder radius="${link_radius}" length="${link2_length}" />
+              </geometry>
+      	       <material name="white"/>
             </visual>
             <inertial>
@@ -110,15 +152,29 @@
           </link>
           <link name="${namespace}/link2_2">
+            <!-- <collision>
+              <origin xyz="0 0 0" rpy="0 0 0"/>
+              <geometry>
+                <mesh filename="package://rotors_description/meshes/dextar_manipulator/link2_2.dae"/>
+              </geometry>
+            </collision>
+            <visual>
+              <origin xyz="0 0 0" rpy="0 0 0"/>
+              <geometry>
+                <mesh filename="package://rotors_description/meshes/dextar_manipulator/link2_2.dae"/>
+              </geometry>
+            </visual> -->
             <collision>
-              <origin xyz="0 0 0" rpy="0 0 0"/>
-              <geometry>
-                <mesh filename="package://rotors_description/meshes/dextar_manipulator/link2_2.dae"/>
-              </geometry>
-            </collision>
-            <visual>
-              <origin xyz="0 0 0" rpy="0 0 0"/>
-              <geometry>
-                <mesh filename="package://rotors_description/meshes/dextar_manipulator/link2_2.dae"/>
-              </geometry>
+              <origin rpy="0 1.57 0" xyz="${link1_length/2} 0 0"/>
+              <geometry>
+                <cylinder radius="${link_radius}" length="${link2_length}" />
+              </geometry>
+      	       <material name="white"/>
+            </collision>
+            <visual>
+              <origin rpy="0 1.57 0" xyz="${link2_length/2} 0 0"/>
+              <geometry>
+                <cylinder radius="${link_radius}" length="${link2_length}" />
+              </geometry>
+      	       <material name="white"/>
             </visual>
             <inertial>
@@ -273,4 +329,30 @@
           </plugin>
         </gazebo> -->
+        <!-- Instantiate force sensor on end-effector -->
+      	<xacro:force_sensor_plugin_macro
+      		namespace="${namespace}"
+      		force_sensor_suffix="ee"
+      		parent_link="${namespace}/link2_2"
+      		force_sensor_topic="force_sensor"
+      		force_sensor_truth_topic="force_sensor_truth"
+      		wrench_vector_pub_topic="wrench_vector"
+      		parent_frame_id="world"
+      		reference_frame_id="world"
+      		mass_force_sensor="0.001"
+      		lin_force_meas_enabled="true"
+      		torque_meas_enabled="false"
+      		disp_wrench_vector="true"
+      		measurement_divisor="1"
+      		measurement_delay="0"
+      		unknown_delay="0.0"
+      		cutoff_frequency="10.0"
+      		noise_normal_linear_force="0 0 0"
+      		noise_normal_torque="0 0 0"
+      		noise_uniform_linear_force="0 0 0"
+      		noise_uniform_torque="0 0 0" >
+      		<inertia ixx="0.001" ixy="0.0" ixz="0.0" iyy="0.001" iyz="0.0" izz="0.001"/>
+      		<!-- [kg m^2] [kg m^2] [kg m^2] [kg m^2] [kg m^2] [kg m^2] -->
+      		<origin xyz="${link2_length} 0.0 0.0" rpy="1.57 0.0 ${-joint_34_offset-joint_2_offset}"/>
+      	</xacro:force_sensor_plugin_macro>
       </xacro:macro>
     </robot>

Commit message: commit old bugfix in urdf

File: rotors_description/urdf/dextar_manipulator.xacro (robot description, xacro)
@@ -133,5 +133,5 @@
             </visual> -->
             <collision>
-              <origin rpy="0 1.57 0" xyz="${link1_length/2} 0 0"/>
+              <origin rpy="0 1.57 0" xyz="${link2_length/2} 0 0"/>
               <geometry>
                 <cylinder radius="${link_radius}" length="${link2_length}" />
@@ -165,5 +165,5 @@
             </visual> -->
             <collision>
-              <origin rpy="0 1.57 0" xyz="${link1_length/2} 0 0"/>
+              <origin rpy="0 1.57 0" xyz="${link2_length/2} 0 0"/>
               <geometry>
                 <cylinder radius="${link_radius}" length="${link2_length}" />
@@ -337,5 +337,5 @@
       		force_sensor_truth_topic="force_sensor_truth"
       		wrench_vector_pub_topic="wrench_vector"
-      		parent_frame_id="world"
+      		parent_frame_id="${namespace}/link2_2"
       		reference_frame_id="world"
       		mass_force_sensor="0.001"
