Commit message: cosmetics fix in dextar urdf

File: rotors_description/urdf/dextar_manipulator.xacro (robot description, xacro)
@@ -272,5 +272,5 @@
           visual_scale="1"
           color="Red">
-          <origin xyz="${link0_center_to_center_length/2} 0 0" rpy="0 0 -1.57"/>
+          <origin xyz="${-link0_center_to_center_length/2} 0 0" rpy="0 0 -1.57"/>
           <xacro:insert_block name="generic_servo_inertial"/>
         </xacro:hebi_actuator_plugin>
@@ -299,5 +299,5 @@
           visual_scale="1"
           color="Red">
-          <origin xyz="${-link0_center_to_center_length/2} 0 0" rpy="0 0 -1.57"/>
+          <origin xyz="${link0_center_to_center_length/2} 0 0" rpy="0 0 -1.57"/>
           <xacro:insert_block name="generic_servo_inertial"/>
         </xacro:hebi_actuator_plugin>

Commit message: heavy dextar for ff_impedance_control testing

File: rotors_description/urdf/dextar_manipulator.xacro (robot description, xacro)
@@ -26,4 +26,9 @@
         iyy="0.00730949" iyz="0.0"
         izz="0.006364922"/>
+      <!-- heavy manipulator for ff_impedance control testing -->
+      <!-- <mass value="0.1"/> -->
+      <!-- <inertia ixx="${5*0.000948062}" ixy="0.0" ixz="${5*-0.001716204}"
+        iyy="${5*0.00730949}" iyz="0.0"
+        izz="${5*0.006364922}"/> -->
       </xacro:property>
     <xacro:property name="link2_frame">
@@ -35,4 +40,9 @@
         iyy="0.0018644679" iyz="0.0"
         izz="0.0018419229"/>
+      <!-- heavy manipulator for ff_impedance control testing -->
+      <!-- <mass value="0.1"/> -->
+      <!-- <inertia ixx="${5*0.000229511}" ixy="0.0" ixz="${5*0.00000098}"
+        iyy="${5*0.0018644679}" iyz="0.0"
+        izz="${5*0.0018419229}"/> -->
       </xacro:property>
           <!--
