Commit message: Add Gimbal

File: rotors_description/urdf/gimbal_front_v1.xacro (robot description, xacro)
@@ -5,60 +5,71 @@
 <robot xmlns:xacro="http://ros.org/wiki/xacro">
   <xacro:property name="pi" value="3.14159265359" />
-  <xacro:property name="resolution" value="3" />
-  <xacro:property name="sample" value="8" />
-  <xacro:property name="min_angle_deg" value="-24" />
-  <xacro:property name="max_angle_deg" value="24" />
-  <xacro:property name="view_angle_deg" value="${max_angle_deg-min_angle_deg}" />
-  <xacro:property name="slot_angle_deg" value="${(view_angle_deg/sample)/resolution}" />
-  <xacro:macro name="lidar_macro" params="namespace parent_link *origin">
-    <link name="${namespace}/lidar_link">
-      <visual name="visual">
-        <origin xyz="0 0 0" rpy="${pi/2} 0 0" />
+  <xacro:macro name="gimbal_macro" params="namespace parent_link *origin">
+    <link name="${namespace}/gimbal_roll_link">
+      <inertial>
+        <mass value="0.1" />
+        <inertia ixx="0.01" ixy="0.0" ixz="0.0" iyy="0.01" iyz="0.0" izz="0.01" />
+      </inertial>
+      <visual>
+        <origin xyz="0 0 0" rpy="0 ${pi/2} 0" />
         <geometry>
-          <mesh filename="package://rotors_description/meshes/leddarvu.dae" scale="1 1 1" />
+          <cylinder radius="0.02" length="0.02" />
         </geometry>
       </visual>
     </link>
-    <joint name="${namespace}/lidar_joint" type="fixed">
+    <joint name="${namespace}/gimbal_roll_joint" type="continuous">
       <xacro:insert_block name="origin" />
       <parent link="${parent_link}" />
-      <child link="${namespace}/lidar_link" />
+      <child link="${namespace}/gimbal_roll_link" />
+      <axis xyz="1 0 0" />
     </joint>
-    <link name="${namespace}/lidar_optical_link">
+    <link name="${namespace}/gimbal_pitch_link">
+      <inertial>
+        <mass value="0.1" />
+        <inertia ixx="0.01" ixy="0.0" ixz="0.0" iyy="0.01" iyz="0.0" izz="0.01" />
+      </inertial>
+      <visual>
+        <origin xyz="0 0 0" rpy="${pi/2} 0 0" />
+        <geometry>
+          <cylinder radius="0.02" length="0.02" />
+        </geometry>
+      </visual>
     </link>
-    <joint name="${namespace}/lidar_optical_joint" type="fixed">
-      <origin xyz="0.03 0 0" rpy="0 0 0" />
-      <parent link="${namespace}/lidar_link" />
-      <child link="${namespace}/lidar_optical_link" />
+    <joint name="${namespace}/gimbal_pitch_joint" type="continuous">
+      <origin xyz="0.1 0.1 0" rpy="0 0 0" />
+      <parent link="${namespace}/gimbal_roll_link" />
+      <child link="${namespace}/gimbal_pitch_link" />
+      <axis xyz="0 1 0" />
     </joint>
-    <gazebo reference="${namespace}/lidar_optical_link">
-      <sensor type="ray" name="${namespace}_lidar">
-        <pose>0 0 0 0 0 0</pose>
-        <visualize>true</visualize>
-        <update_rate>100</update_rate>
-        <ray>
-          <scan>
-            <horizontal>
-              <samples>${sample}</samples>
-              <resolution>${resolution}</resolution>
-              <min_angle>${(min_angle_deg+(slot_angle_deg/2))/180.0*pi}</min_angle>
-              <max_angle>${(max_angle_deg-(slot_angle_deg/2))/180.0*pi}</max_angle>
-            </horizontal>
-          </scan>
-          <range>
-            <min>0.06</min>
-            <max>25</max>
-            <resolution>0.01</resolution>
-          </range>
-          <noise>
-            <type>gaussian</type>
-            <mean>0.0</mean>
-            <stddev>0.01</stddev>
-          </noise>
-        </ray>
-	      <plugin name="rotors_gazebo_lidar_plugin" filename="librotors_gazebo_lidar_plugin.so"/>
-		    <robotNamespace>${namespace}</robotNamespace>
-        <always_on>1</always_on>
-      </sensor>
+    <link name="${namespace}/gimbal_plate_link">
+      <inertial>
+        <mass value="0.1" />
+        <inertia ixx="0.01" ixy="0.0" ixz="0.0" iyy="0.01" iyz="0.0" izz="0.01" />
+      </inertial>
+      <visual>
+        <origin xyz="0 0 0" rpy="0 0 0" />
+        <geometry>
+          <box size ="0.05 0.1 0.005" />
+        </geometry>
+      </visual>
+    </link>
+    <joint name="${namespace}/gimbal_plate_joint" type="fixed">
+      <origin xyz="0 -0.1 -0.02" rpy="0 0 0" />
+      <parent link="${namespace}/gimbal_pitch_link" />
+      <child link="${namespace}/gimbal_plate_link" />
+    </joint>
+    <gazebo>
+      <plugin name="front_gimbal_plugin" filename="libgazebo_front_gimbal_plugin.so">
+      <robotNamespace>${namespace}</robotNamespace>
+      </plugin>
+    </gazebo>
+    <gazebo reference="${namespace}/gimbal_roll_link">
+      <material>Gazebo/Black</material>
+    </gazebo>
+    <gazebo reference="${namespace}/gimbal_pitch_link">
+      <material>Gazebo/Black</material>
+    </gazebo>
+    <gazebo reference="${namespace}/gimbal_plate_link">
+      <material>Gazebo/Black</material>
     </gazebo>
   </xacro:macro>

File: rotors_description/urdf/leddarvu.xacro (robot description, xacro)
@@ -11,6 +11,6 @@
   <xacro:property name="view_angle_deg" value="${max_angle_deg-min_angle_deg}" />
   <xacro:property name="slot_angle_deg" value="${(view_angle_deg/sample)/resolution}" />
-  <xacro:macro name="lidar_macro" params="namespace parent_link *origin">
-    <link name="${namespace}/lidar_link">
+  <xacro:macro name="lidar_macro" params="namespace parent_link lidar_number *origin">
+    <link name="${namespace}/lidar_link_${lidar_number}">
       <visual name="visual">
         <origin xyz="0 0 0" rpy="${pi/2} 0 0" />
@@ -20,18 +20,18 @@
       </visual>
     </link>
-    <joint name="${namespace}/lidar_joint" type="fixed">
+    <joint name="${namespace}/lidar_joint_${lidar_number}" type="fixed">
       <xacro:insert_block name="origin" />
       <parent link="${parent_link}" />
-      <child link="${namespace}/lidar_link" />
+      <child link="${namespace}/lidar_link_${lidar_number}" />
     </joint>
-    <link name="${namespace}/lidar_optical_link">
+    <link name="${namespace}/lidar_optical_link_${lidar_number}">
     </link>
-    <joint name="${namespace}/lidar_optical_joint" type="fixed">
+    <joint name="${namespace}/lidar_optical_joint_${lidar_number}" type="fixed">
       <origin xyz="0.03 0 0" rpy="0 0 0" />
-      <parent link="${namespace}/lidar_link" />
-      <child link="${namespace}/lidar_optical_link" />
+      <parent link="${namespace}/lidar_link_${lidar_number}" />
+      <child link="${namespace}/lidar_optical_link_${lidar_number}" />
     </joint>
-    <gazebo reference="${namespace}/lidar_optical_link">
-      <sensor type="ray" name="${namespace}_lidar">
+    <gazebo reference="${namespace}/lidar_optical_link_${lidar_number}">
+      <sensor type="ray" name="${namespace}_lidar_${lidar_number}">
         <pose>0 0 0 0 0 0</pose>
         <visualize>true</visualize>
@@ -57,6 +57,8 @@
           </noise>
         </ray>
-	      <plugin name="rotors_gazebo_lidar_plugin" filename="librotors_gazebo_lidar_plugin.so"/>
-		    <robotNamespace>${namespace}</robotNamespace>
+	      <plugin name="rotors_gazebo_lidar_plugin_${lidar_number}" filename="librotors_gazebo_lidar_plugin.so">
+		      <robotNamespace>${namespace}</robotNamespace>
+          <lidarTopic>lidar_${lidar_number}</lidarTopic>
+        </plugin>
         <always_on>1</always_on>
       </sensor>

File: rotors_description/urdf/niv1_base.xacro (robot description, xacro)
@@ -23,8 +23,10 @@
   <!-- Instantiate niv1 "mechanics" -->
   <xacro:include filename="$(find rotors_description)/urdf/niv1.xacro" />
-  <!-- Instantiate a controller. -->
+    <!-- Instantiate a controller. -->
   <xacro:controller_plugin_macro namespace="${namespace}" imu_sub_topic="imu" />
-  <!-- Instantiate a ROS message interface -->
-  <!-- <xacro:ros_interface_plugin_macro namespace="${namespace}" />-->
+  <!-- Instantiate a ROS message interface
+  <xacro:ros_interface_plugin_macro namespace="${namespace}" />
+  -->
+  <xacro:include filename="$(find rotors_description)/urdf/gimbal_front_v1.xacro" />
   <xacro:if value="$(arg enable_mavlink_interface)">
     <!-- Instantiate mavlink telemetry interface. -->
@@ -35,13 +37,20 @@
   <xacro:niv1_magnetometer namespace="${namespace}" parent_link="${namespace}/base_link" />
   <xacro:niv1_pressure_sensor namespace="${namespace}" parent_link="${namespace}/base_link" />
+  <xacro:gimbal_macro namespace="${namespace}" parent_link="${namespace}/base_link" >
+    <origin xyz="0.36 0 0.03" rpy="0 0 0" />
+  </xacro:gimbal_macro>
   <!-- Camera Sensor -->
-  <xacro:camera_macro namespace="${namespace}" parent_link="${namespace}/base_link" camera_suffix="0" frame_rate="30" horizontal_fov="1.448622" image_width="640" image_height="480" image_format="" min_distance="0.02" max_distance="200" noise_mean="0.0" noise_stddev="0.007" enable_visual="true">
+  <xacro:camera_macro namespace="${namespace}" parent_link="${namespace}/gimbal_plate_link" camera_suffix="0" frame_rate="30" horizontal_fov="1.448622" image_width="640" image_height="480" image_format="" min_distance="0.02" max_distance="200" noise_mean="0.0" noise_stddev="0.007" enable_visual="true">
     <mesh filename="package://rotors_description/meshes/csi_camera.dae" scale="1 1 1" />
-    <origin xyz="0.45 0 0.05" rpy="0 0 0" />
+    <origin xyz="0.02 -0.02 0.02" rpy="0 0 0" />
   </xacro:camera_macro>
   <!--LIDAR Sensor-->
-  <xacro:lidar_macro namespace="${namespace}" parent_link="${namespace}/base_link">
+  <xacro:lidar_macro namespace="${namespace}" parent_link="${namespace}/base_link" lidar_number="0">
     <!-- <origin xyz="0 0 -0.035" rpy="0 0 0" /> -->
-    <origin xyz="0.4 0 0" rpy="0 0 0" />
+    <origin xyz="0.34 0 -0.1" rpy="0 0 0" />
+  </xacro:lidar_macro>
+  <xacro:lidar_macro namespace="${namespace}" parent_link="${namespace}/gimbal_plate_link" lidar_number="1">
+    <!-- <origin xyz="0 0 -0.035" rpy="0 0 0" /> -->
+    <origin xyz="0.0 0 -0.025" rpy="0 0 0" />
   </xacro:lidar_macro>
   <!-- Nearthlab Payload -->
