Commit message: adds robot namespace to velodyne xacros

File: rotors_description/urdf/velodyne_HDL_32E.urdf.xacro (robot description, xacro)
@@ -5,8 +5,9 @@
   <gazebo>
     <plugin name="JointController" filename="libgazebo_ros_continous_joint_controller_plugin.so">
-      <joint>${sensor_name}_joint</joint>
-      <default_velocity_limit>100</default_velocity_limit>
-      <spin_frequency_hz>${spin_frequency_hz}</spin_frequency_hz>
-    </plugin>
+        <joint>${sensor_name}_joint</joint>
+	<robot_namespace>${model_name}</robot_namespace>
+	<default_velocity_limit>100</default_velocity_limit>
+        <spin_frequency_hz>${spin_frequency_hz}</spin_frequency_hz>
+      </plugin>
   </gazebo>
   <link name="${lidar_base_frame}">

File: rotors_description/urdf/velodyne_VLP_16.urdf.xacro (robot description, xacro)
@@ -12,5 +12,6 @@
       <plugin name="JointController" filename="libgazebo_ros_continous_joint_controller_plugin.so">
         <joint>${sensor_name}_joint</joint>
-        <default_velocity_limit>100</default_velocity_limit>
+	<robot_namespace>${model_name}</robot_namespace>
+	<default_velocity_limit>100</default_velocity_limit>
         <spin_frequency_hz>${spin_frequency_hz}</spin_frequency_hz>
       </plugin>
