Commit message: fixes vlp-16 namespacing

File: rotors_description/urdf/velodyne_VLP_16.urdf.xacro (robot description, xacro)
@@ -8,19 +8,19 @@
   <xacro:property name="r2" value="0.0516"/>
   <xacro:property name="l2" value="0.0381"/>
-  <xacro:macro name="VLP-16" params="*origin parent:=world sensor_name:=velodyne topic:=/velodyne_points horizontal_angular_resolution_deg:=1.0 spin_frequency_hz:=0.5 lidar_base_frame:=velodyne_base lidar_points_frame:=velodyne_top model_name:=example">
+  <xacro:macro name="VLP-16" params="*origin parent:=world sensor_name:=velodyne topic:=/velodyne_points horizontal_angular_resolution_deg:=1.0 spin_frequency_hz:=0.5 lidar_base_frame:=velodyne_base lidar_points_frame:=velodyne_top namespace:=example min_range:=0.06">
     <gazebo>
       <plugin name="JointController" filename="libgazebo_ros_continous_joint_controller_plugin.so">
-        <joint>${sensor_name}_joint</joint>
-	<robot_namespace>${model_name}</robot_namespace>
-	<default_velocity_limit>100</default_velocity_limit>
+        <joint>${namespace}/${sensor_name}_joint</joint>
+	      <robot_namespace>${namespace}</robot_namespace>
+	      <default_velocity_limit>100</default_velocity_limit>
         <spin_frequency_hz>${spin_frequency_hz}</spin_frequency_hz>
       </plugin>
     </gazebo>
-    <joint name="${lidar_base_frame}_mount_joint" type="fixed">
+    <joint name="${namespace}/${lidar_base_frame}_mount_joint" type="fixed">
       <xacro:insert_block name="origin" />
       <parent link="${parent}"/>
-      <child link="${lidar_base_frame}"/>
+      <child link="${namespace}/${lidar_base_frame}"/>
     </joint>
-    <link name="${lidar_base_frame}">
+    <link name="${namespace}/${lidar_base_frame}">
       <inertial>
         <mass value="${m1}"/>
@@ -30,5 +30,5 @@
                  izz="${0.5 * m1 * (r1*r1)}"/>
       </inertial>
-      <collision name="${lidar_base_frame}_collision">
+      <collision name="${namespace}/${lidar_base_frame}_collision">
         <origin rpy="0 0 0" xyz="0 0 ${l1*0.5}"/>
         <geometry>
@@ -36,5 +36,5 @@
         </geometry>
       </collision>
-      <visual name="${lidar_base_frame}_visual">
+      <visual name="${namespace}/${lidar_base_frame}_visual">
         <origin rpy="0 0 0" xyz="0 0 ${l1*0.5}"/>
         <geometry>
@@ -43,12 +43,12 @@
       </visual>
     </link>
-    <joint name="${sensor_name}_joint" type="continuous">
-      <parent link="${lidar_base_frame}"/>
-      <child link="${lidar_points_frame}"/>
+    <joint name="${namespace}/${sensor_name}_joint" type="continuous">
+      <parent link="${namespace}/${lidar_base_frame}"/>
+      <child link="${namespace}/${lidar_points_frame}"/>
       <origin rpy="0 0 0" xyz="0 0 ${l1+l2*0.5}"/>
       <axis xyz="0 0 1"/>
       <limit effort="100.0" velocity="100.0"/>
     </joint>
-    <link name="${lidar_points_frame}">
+    <link name="${namespace}/${lidar_points_frame}">
       <inertial>
         <mass value="${m2}"/>
@@ -64,5 +64,5 @@
         </geometry>
       </collision>
-      <visual name="${lidar_points_frame}_visual">
+      <visual name="${namespace}/${lidar_points_frame}_visual">
         <origin rpy="0 0 0" xyz="0 0 0"/>
         <geometry>
@@ -71,13 +71,13 @@
       </visual>
     </link>
-    <gazebo reference="${lidar_points_frame}">
+    <gazebo reference="${namespace}/${lidar_points_frame}">
       <material>Gazebo/Black</material>
     </gazebo>
     <joint name="${sensor_name}_joint_hat" type="fixed">
-      <parent link="${lidar_base_frame}"/>
-      <child link="${lidar_base_frame}_hat"/>
+      <parent link="${namespace}/${lidar_base_frame}"/>
+      <child link="${namespace}/${lidar_base_frame}_hat"/>
       <origin rpy="0 0 0" xyz="0 0 ${l1+l2*0.5}"/>
     </joint>
-    <link name="${lidar_base_frame}_hat">
+    <link name="${namespace}/${lidar_base_frame}_hat">
       <inertial>
         <mass value="${m1}"/>
@@ -100,5 +100,5 @@
       </visual>
     </link>
-    <gazebo reference="${lidar_points_frame}">
+    <gazebo reference="${namespace}/${lidar_points_frame}">
       <!-- Add a ray sensor, and give it a name -->
       <sensor type="ray" name="sensor">
@@ -132,5 +132,5 @@
           <range>
             <!-- Minimum distance of the beam -->
-            <min>${r1+0.05}</min>
+            <min>${min_range}</min>
             <!-- Maximum distance of the beam -->
             <max>70</max>
@@ -140,9 +140,9 @@
         </ray>
         <plugin name="gazebo_ros_laser_plugin" filename="libgazebo_ros_laser_plugin.so">
-          <model_name>${model_name}</model_name>
-          <joint_name>${sensor_name}_joint</joint_name>
+          <robot_namespace>${namespace}</robot_namespace>
+          <joint_name>${namespace}/${sensor_name}_joint</joint_name>
           <topic_name>${topic}</topic_name>
           <frame_name>${lidar_points_frame}</frame_name>
-          <min_range>${r1+0.05}</min_range>
+          <min_range>${min_range}</min_range>
           <max_range>70</max_range>
           <gaussian_noise>0.02</gaussian_noise>
