Commit message: Fixed orientation and position of mesh relative to camera center (here, left imager) as per datasheet)

File: rotors_description/urdf/rgbd_base.xacro (robot description, xacro)
@@ -11,5 +11,5 @@
     </collision>
     <visual>
-      <origin xyz="0 0 0" rpy="0 0 0" />
+      <origin xyz="0 -0.0175 0" rpy="${pi/2} 0 ${pi/2}" />
       <geometry>
               <mesh filename="package://rotors_description/meshes/d435_simple.dae" scale="1 1 1" />
@@ -18,5 +18,5 @@
     </visual>
     <inertial>
-      <mass value="100" />
+      <mass value="0" />
       <origin xyz="0 0 0" rpy="0 0 0" />
       <inertia ixx="1" ixy="0" ixz="0" iyy="1" iyz="0" izz="1" />
@@ -109,6 +109,6 @@
       noise_mean="0.0"
       noise_stddev="0.007"
-      enable_visual="false">
-              <mesh filename="package://rotors_description/meshes/d435_simple.dae" scale="1 1 1" />
+      enable_visual="true">
+          <box size="0.01 0.01 0.1" />
         <origin xyz="0.0 0.0 0.0" rpy="0 0 0" />
     </xacro:camera_macro>

Commit message: Cleanup of .xacro file

File: rotors_description/urdf/rgbd_base.xacro (robot description, xacro)
@@ -1,9 +1,12 @@
 <?xml version="1.0"?>
-<robot name="rgbd_camera" xmlns:xacro="http://ros.org/wiki/xacro">
-  <xacro:property name="namespace" value="rgbd_camera" />
+<robot name="$(arg mav_name)" xmlns:xacro="http://ros.org/wiki/xacro">
   <xacro:include filename="$(find rotors_description)/urdf/component_snippets.xacro" />
+  <!-- Note that whenever possible, values from Realsense D435 were used.
+       See Intel Document 337029-004: Intel RealSense TM D400 Series Product Family Datasheet.
+       https://www.intel.com/content/dam/support/us/en/documents/emerging-technologies/intel-realsense-technology/Intel-RealSense-D400-Series-Datasheet.pdf
+  -->
   <link name="rgbd_camera/base_link">
     <collision>
-      <origin xyz="0 0 0" rpy="0 0 0" />
+      <origin xyz="0 -0.0175 0" rpy="${pi/2} 0 ${pi/2}" />
       <geometry>
               <mesh filename="package://rotors_description/meshes/d435_simple.dae" scale="1 1 1" />
@@ -17,13 +20,8 @@
       <material name="black" />
     </visual>
-    <inertial>
-      <mass value="0" />
-      <origin xyz="0 0 0" rpy="0 0 0" />
-      <inertia ixx="1" ixy="0" ixz="0" iyy="1" iyz="0" izz="1" />
-    </inertial>
   </link>
-<!-- Macro to add a depth camera on the VI-sensor. -->
+<!-- Define Macro to add a depth camera using noisy depth plugin  -->
   <xacro:macro name="rgbd_sensor_depth_macro"
-    params="namespace parent_link camera_suffix frame_rate max_range *origin">
+    params="namespace parent_link camera_suffix frame_rate width height fov max_range min_range baseline *origin">
     <link name="${namespace}/camera_${camera_suffix}_link">
       <collision>
@@ -45,5 +43,4 @@
       <limit upper="0" lower="0" effort="0" velocity="0" />
     </joint>
-    <!-- Optical center of camera -->
     <link name="${namespace}/camera_${camera_suffix}_optical_center_link" />
     <joint name="${namespace}/camera_${camera_suffix}_optical_center_joint" type="fixed">
@@ -53,4 +50,23 @@
       <limit upper="0" lower="0" effort="0" velocity="0" />
     </joint>
+    <!-- Call rgb sensor macro-->
+    <!-- RGB sensor has "unlimited ranges"-->
+    <xacro:camera_macro
+            namespace="${namespace}"
+            parent_link="rgbd_camera/base_link"
+            camera_suffix="rgb"
+            frame_rate="${frame_rate}"
+            horizontal_fov="${fov}"
+            image_width="${width}"
+            image_height="${height}"
+            image_format="R8G8B8"
+            min_distance="0.01"
+            max_distance="500"
+            noise_mean="0.0"
+            noise_stddev="0.007"
+            enable_visual="false">
+      <box size="0.01 0.01 0.1" />
+      <origin xyz="0.0 0.0 0.0" rpy="0 0 0" />
+    </xacro:camera_macro>
     <gazebo reference="${namespace}/camera_${camera_suffix}_link">
       <sensor type="depth" name="${namespace}_camera_{camera_suffix}">
@@ -58,12 +74,12 @@
         <update_rate>${frame_rate}</update_rate>
         <camera>
-          <horizontal_fov>1.3962634</horizontal_fov>
+          <horizontal_fov>${fov}</horizontal_fov>
           <image>
             <format>L8</format>
-            <width>640</width>
-            <height>480</height>
+            <width>${width}</width>
+            <height>${height}</height>
           </image>
           <clip>
-            <near>0.01</near>
+            <near>${min_range}</near>
             <far>${max_range}</far>
           </clip>
@@ -72,5 +88,5 @@
           <robotNamespace>${namespace}</robotNamespace>
           <alwaysOn>true</alwaysOn>
-          <baseline>0.11</baseline>
+          <baseline>${baseline}</baseline>
           <updateRate>${frame_rate}</updateRate>
           <cameraName>camera_${camera_suffix}</cameraName>
@@ -90,26 +106,22 @@
     </gazebo>
   </xacro:macro>
-  <!-- Depth Sensor -->
-      <xacro:rgbd_sensor_depth_macro
-        namespace="${namespace}" parent_link="${namespace}/base_link"
-        camera_suffix="depth" frame_rate="30.0" max_range="10.0">
-        <origin xyz="0.0 0.0 0.0" rpy="0 0 0" />
-      </xacro:rgbd_sensor_depth_macro>
-    <xacro:camera_macro
-      namespace="${namespace}"
-      parent_link="${namespace}/base_link"
-      camera_suffix="rgb"
-      frame_rate="30.0"
-      horizontal_fov="1.3962634"
-      image_width="640"
-      image_height="480"
-      image_format="R8G8B8"
-      min_distance="0.02"
-      max_distance="300"
-      noise_mean="0.0"
-      noise_stddev="0.007"
-      enable_visual="false">
-          <box size="0.01 0.01 0.1" />
-        <origin xyz="0.0 0.0 0.0" rpy="0 0 0" />
-    </xacro:camera_macro>
+  <!-- Call depth sensor macro
+    Realsense values -
+      91.2 Deg Horizontal FOV
+      848x480 Optimal depth resolution
+        w 195 mm minimium-z depth
+      5 cm baseline.
+  -->
+  <xacro:rgbd_sensor_depth_macro
+    namespace="${namespace}/rgbd" parent_link="rgbd_camera/base_link"
+    camera_suffix="depth"
+    frame_rate="30.0"
+    fov = "1.59174"
+    baseline = "0.05"
+    width = "848"
+    height = "480"
+    max_range="50.0"
+    min_range="0.195">
+    <origin xyz="0.0 0.0 0.0" rpy="0 0 0" />
+  </xacro:rgbd_sensor_depth_macro>
 </robot>
