Commit message: fix m100 with/without visensor

File: rotors_description/urdf/m100_base.xacro (robot description, xacro)
@@ -41,13 +41,4 @@
       wait_to_record_bag="$(arg wait_to_record_bag)" />
   </xacro:if>
-  <!-- Mount a VI-sensor in front of the Firefly. -->
-  <xacro:vi_sensor_macro
-    namespace="${namespace}/vi_sensor"
-    parent_link="${namespace}/base_link"
-    enable_cameras="true"
-    enable_depth="true"
-    enable_ground_truth="true">
-    <origin xyz="0.15 0.0 -0.05" rpy="0 0.3 0" />
-  </xacro:vi_sensor_macro>
 	<xacro:include filename="$(find rotors_description)/urdf/m100_pccase.xacro" />
   <xacro:pccase_macro
