Commit message: fixes namespaces in os-1 models and related plugins

File: rotors_description/urdf/ouster_os1.urdf.xacro (robot description, xacro)
@@ -8,19 +8,19 @@
   <xacro:property name="r2" value="0.0425"/>
   <xacro:property name="l2" value="0.0305"/>
-  <xacro:macro name="OS-1" params="*origin parent:=world sensor_name:=os1 topic:=/os1_points horizontal_angular_resolution_deg:=0.18 spin_frequency_hz:=10 lidar_base_frame:=os1_base lidar_points_frame:=os1_top model_name:=example min_range:=0.05">
+  <xacro:macro name="OS-1" params="*origin parent:=world sensor_name:=os1 topic:=/os1_points horizontal_angular_resolution_deg:=0.18 spin_frequency_hz:=10 lidar_base_frame:=os1_base lidar_points_frame:=os1_top namespace:=example min_range:=0.05">
     <gazebo>
       <plugin name="JointController" filename="libgazebo_ros_continous_joint_controller_plugin.so">
-        <joint>${sensor_name}_joint</joint>
-	<robot_namespace>${model_name}</robot_namespace>
-	<default_velocity_limit>100</default_velocity_limit>
+        <joint>${namespace}/${sensor_name}_joint</joint>
+	      <robot_namespace>${namespace}</robot_namespace>
+	      <default_velocity_limit>100</default_velocity_limit>
         <spin_frequency_hz>${spin_frequency_hz}</spin_frequency_hz>
       </plugin>
     </gazebo>
-    <joint name="${lidar_base_frame}_mount_joint" type="fixed">
+    <joint name="${namespace}/${lidar_base_frame}_mount_joint" type="fixed">
       <xacro:insert_block name="origin" />
       <parent link="${parent}"/>
-      <child link="${lidar_base_frame}"/>
+      <child link="${namespace}/${lidar_base_frame}"/>
     </joint>
-    <link name="${lidar_base_frame}">
+    <link name="${namespace}/${lidar_base_frame}">
       <inertial>
         <mass value="${m1}"/>
@@ -30,5 +30,5 @@
                  izz="${0.5 * m1 * (r1*r1)}"/>
       </inertial>
-      <collision name="${lidar_base_frame}_collision">
+      <collision name="${namespace}/${lidar_base_frame}_collision">
         <origin rpy="0 0 0" xyz="0 0 ${l1*0.5}"/>
         <geometry>
@@ -36,5 +36,5 @@
         </geometry>
       </collision>
-      <visual name="${lidar_base_frame}_visual">
+      <visual name="${namespace}/${lidar_base_frame}_visual">
         <origin rpy="0 0 0" xyz="0 0 ${l1*0.5}"/>
         <geometry>
@@ -43,12 +43,12 @@
       </visual>
     </link>
-    <joint name="${sensor_name}_joint" type="continuous">
-      <parent link="${lidar_base_frame}"/>
-      <child link="${lidar_points_frame}"/>
+    <joint name="${namespace}/${sensor_name}_joint" type="continuous">
+      <parent link="${namespace}/${lidar_base_frame}"/>
+      <child link="${namespace}/${lidar_points_frame}"/>
       <origin rpy="0 0 0" xyz="0 0 ${l1+l2*0.5}"/>
       <axis xyz="0 0 1"/>
       <limit effort="100.0" velocity="100.0"/>
     </joint>
-    <link name="${lidar_points_frame}">
+    <link name="${namespace}/${lidar_points_frame}">
       <inertial>
         <mass value="${m2}"/>
@@ -64,5 +64,5 @@
         </geometry>
       </collision>
-      <visual name="${lidar_points_frame}_visual">
+      <visual name="${namespace}/${lidar_points_frame}_visual">
         <origin rpy="0 0 0" xyz="0 0 0"/>
         <geometry>
@@ -71,13 +71,13 @@
       </visual>
     </link>
-    <gazebo reference="${lidar_points_frame}">
+    <gazebo reference="${namespace}/${lidar_points_frame}">
       <material>Gazebo/Black</material>
     </gazebo>
     <joint name="${sensor_name}_joint_hat" type="fixed">
-      <parent link="${lidar_base_frame}"/>
-      <child link="${lidar_base_frame}_hat"/>
+      <parent link="${namespace}/${lidar_base_frame}"/>
+      <child link="${namespace}/${lidar_base_frame}_hat"/>
       <origin rpy="0 0 0" xyz="0 0 ${l1+l2*0.5}"/>
     </joint>
-    <link name="${lidar_base_frame}_hat">
+    <link name="${namespace}/${lidar_base_frame}_hat">
       <inertial>
         <mass value="${m1}"/>
@@ -100,5 +100,5 @@
       </visual>
     </link>
-    <gazebo reference="${lidar_points_frame}">
+    <gazebo reference="${namespace}/${lidar_points_frame}">
       <!-- Add a ray sensor, and give it a name -->
       <sensor type="ray" name="sensor">
@@ -140,6 +140,6 @@
         </ray>
         <plugin name="gazebo_ros_laser_plugin" filename="libgazebo_ros_laser_plugin.so">
-          <model_name>${model_name}</model_name>
-          <joint_name>${sensor_name}_joint</joint_name>
+          <robot_namespace>${namespace}</robot_namespace>
+          <joint_name>${namespace}/${sensor_name}_joint</joint_name>
           <topic_name>${topic}</topic_name>
           <frame_name>${lidar_points_frame}</frame_name>

Commit message: adds a different implementation of an os1 plugin
makes it capable of hitting the high spinning frequencies without crashing gazebo. tradeoff is a lack of information between the scans

File: rotors_description/urdf/ouster_os1.urdf.xacro (robot description, xacro)
@@ -8,13 +8,5 @@
   <xacro:property name="r2" value="0.0425"/>
   <xacro:property name="l2" value="0.0305"/>
-  <xacro:macro name="OS-1" params="*origin parent:=world sensor_name:=os1 topic:=/os1_points horizontal_angular_resolution_deg:=0.18 spin_frequency_hz:=10 lidar_base_frame:=os1_base lidar_points_frame:=os1_top namespace:=example min_range:=0.05">
-    <gazebo>
-      <plugin name="JointController" filename="libgazebo_ros_continous_joint_controller_plugin.so">
-        <joint>${namespace}/${sensor_name}_joint</joint>
-	      <robot_namespace>${namespace}</robot_namespace>
-	      <default_velocity_limit>100</default_velocity_limit>
-        <spin_frequency_hz>${spin_frequency_hz}</spin_frequency_hz>
-      </plugin>
-    </gazebo>
+  <xacro:macro name="OS-1" params="*origin parent:=world sensor_name:=os1 topic:=/os1_points spin_frequency_hz:=10 lidar_base_frame:=os1_base lidar_points_frame:=os1_top namespace:=example min_range:=0.05">
     <joint name="${namespace}/${lidar_base_frame}_mount_joint" type="fixed">
       <xacro:insert_block name="origin" />
@@ -43,10 +35,7 @@
       </visual>
     </link>
-    <joint name="${namespace}/${sensor_name}_joint" type="continuous">
+    <joint name="${namespace}/${sensor_name}_joint" type="fixed">
       <parent link="${namespace}/${lidar_base_frame}"/>
       <child link="${namespace}/${lidar_points_frame}"/>
-      <origin rpy="0 0 0" xyz="0 0 ${l1+l2*0.5}"/>
-      <axis xyz="0 0 1"/>
-      <limit effort="100.0" velocity="100.0"/>
     </joint>
     <link name="${namespace}/${lidar_points_frame}">
@@ -105,7 +94,7 @@
         <pose>0 0 0 0 0 0</pose>
         <!-- Enable visualization to see the rays in the GUI -->
-        <visualize>true</visualize>
+        <visualize>false</visualize>
         <!-- Set the update rate of the sensor -->
-        <update_rate>${360.0/horizontal_angular_resolution_deg*spin_frequency_hz}</update_rate>
+        <update_rate>${spin_frequency_hz}</update_rate>
         <ray>
           <noise>
@@ -117,5 +106,5 @@
           <scan>
             <horizontal>
-              <samples>1</samples>
+              <samples>1024</samples>
               <resolution>1</resolution>
               <min_angle>0</min_angle>
@@ -139,7 +128,6 @@
           </range>
         </ray>
-        <plugin name="gazebo_ros_laser_plugin" filename="libgazebo_ros_laser_plugin.so">
+        <plugin name="gazebo_ros_lidar_plugin" filename="librotors_gazebo_os1_plugin.so">
           <robot_namespace>${namespace}</robot_namespace>
-          <joint_name>${namespace}/${sensor_name}_joint</joint_name>
           <topic_name>${topic}</topic_name>
           <frame_name>${lidar_points_frame}</frame_name>

Commit message: Makes the fixed OS-1 the default. Moves the spinning one into a different file

File: rotors_description/urdf/ouster_os1.urdf.xacro (robot description, xacro)
@@ -9,13 +9,5 @@
   <xacro:property name="l2" value="0.0305"/>
   <xacro:include filename="$(find rotors_description)/urdf/multirotor_base.xacro" />
-  <xacro:macro name="OS-1" params="*origin parent:=world sensor_name:=os1 topic:=/os1_points horizontal_angular_resolution_deg:=0.18 spin_frequency_hz:=10 lidar_base_frame:=os1_base lidar_points_frame:=os1_top namespace:=example min_range:=0.05">
-    <gazebo>
-      <plugin name="JointController" filename="libgazebo_ros_continous_joint_controller_plugin.so">
-        <joint>${namespace}/${sensor_name}_joint</joint>
-	      <robot_namespace>${namespace}</robot_namespace>
-	      <default_velocity_limit>100</default_velocity_limit>
-        <spin_frequency_hz>${spin_frequency_hz}</spin_frequency_hz>
-      </plugin>
-    </gazebo>
+  <xacro:macro name="OS-1" params="*origin parent:=world sensor_name:=os1 topic:=/os1_points spin_frequency_hz:=10 lidar_base_frame:=os1_base lidar_points_frame:=os1_top namespace:=example min_range:=0.05">
     <joint name="${namespace}/${lidar_base_frame}_mount_joint" type="fixed">
       <xacro:insert_block name="origin" />
@@ -27,10 +19,7 @@
         <origin rpy="0 0 0" xyz="0 0 ${l1*0.5}"/>
     </xacro:cylinder_link_complete>
-    <joint name="${namespace}/${sensor_name}_joint" type="continuous">
+    <joint name="${namespace}/${sensor_name}_joint" type="fixed">
       <parent link="${namespace}/${lidar_base_frame}"/>
       <child link="${namespace}/${lidar_points_frame}"/>
-      <origin rpy="0 0 0" xyz="0 0 ${l1+l2*0.5}"/>
-      <axis xyz="0 0 1"/>
-      <limit effort="100.0" velocity="100.0"/>
     </joint>
     <xacro:cylinder_link_complete link_name="${namespace}/${lidar_points_frame}"
@@ -55,7 +44,7 @@
         <pose>0 0 0 0 0 0</pose>
         <!-- Enable visualization to see the rays in the GUI -->
-        <visualize>true</visualize>
+        <visualize>false</visualize>
         <!-- Set the update rate of the sensor -->
-        <update_rate>${360.0/horizontal_angular_resolution_deg*spin_frequency_hz}</update_rate>
+        <update_rate>${spin_frequency_hz}</update_rate>
         <ray>
           <noise>
@@ -67,5 +56,5 @@
           <scan>
             <horizontal>
-              <samples>1</samples>
+              <samples>1024</samples>
               <resolution>1</resolution>
               <min_angle>0</min_angle>
@@ -89,7 +78,6 @@
           </range>
         </ray>
-        <plugin name="gazebo_ros_laser_plugin" filename="libgazebo_ros_laser_plugin.so">
+        <plugin name="gazebo_ros_lidar_plugin" filename="librotors_gazebo_os1_plugin.so">
           <robot_namespace>${namespace}</robot_namespace>
-          <joint_name>${namespace}/${sensor_name}_joint</joint_name>
           <topic_name>${topic}</topic_name>
           <frame_name>${lidar_points_frame}</frame_name>

File: rotors_description/urdf/ouster_os1_spinning.urdf.xacro (robot description, xacro)
@@ -1,4 +1,4 @@
 <?xml version="1.0" ?>
-<robot xmlns:xacro="http://www.ros.org/wiki/xacro" name="OS-1">
+<robot xmlns:xacro="http://www.ros.org/wiki/xacro" name="OS-1-spinning">
   <xacro:property name="M_PI" value="3.1415926535897931" />
   <xacro:property name="m1" value="0.15"/>
@@ -8,5 +8,14 @@
   <xacro:property name="r2" value="0.0425"/>
   <xacro:property name="l2" value="0.0305"/>
-  <xacro:macro name="OS-1" params="*origin parent:=world sensor_name:=os1 topic:=/os1_points spin_frequency_hz:=10 lidar_base_frame:=os1_base lidar_points_frame:=os1_top namespace:=example min_range:=0.05">
+  <xacro:include filename="$(find rotors_description)/urdf/multirotor_base.xacro" />
+  <xacro:macro name="OS-1" params="*origin parent:=world sensor_name:=os1 topic:=/os1_points horizontal_angular_resolution_deg:=0.18 spin_frequency_hz:=10 lidar_base_frame:=os1_base lidar_points_frame:=os1_top namespace:=example min_range:=0.05">
+    <gazebo>
+      <plugin name="JointController" filename="libgazebo_ros_continous_joint_controller_plugin.so">
+        <joint>${namespace}/${sensor_name}_joint</joint>
+	      <robot_namespace>${namespace}</robot_namespace>
+	      <default_velocity_limit>100</default_velocity_limit>
+        <spin_frequency_hz>${spin_frequency_hz}</spin_frequency_hz>
+      </plugin>
+    </gazebo>
     <joint name="${namespace}/${lidar_base_frame}_mount_joint" type="fixed">
       <xacro:insert_block name="origin" />
@@ -14,50 +23,19 @@
       <child link="${namespace}/${lidar_base_frame}"/>
     </joint>
-    <link name="${namespace}/${lidar_base_frame}">
-      <inertial>
-        <mass value="${m1}"/>
+    <xacro:cylinder_link_complete link_name="${namespace}/${lidar_base_frame}"
+      mass="${m1}" length="${l1}" radius="${r1}">
         <origin rpy="0 0 0" xyz="0 0 ${l1*0.5}"/>
-        <inertia ixx="${(m1 * (3.0*r1*r1 + l1*l1)) / 12.0}" ixy="0" ixz="0"
-                 iyy="${(m1 * (3.0*r1*r1 + l1*l1)) / 12.0}" iyz="0"
-                 izz="${0.5 * m1 * (r1*r1)}"/>
-      </inertial>
-      <collision name="${namespace}/${lidar_base_frame}_collision">
-        <origin rpy="0 0 0" xyz="0 0 ${l1*0.5}"/>
-        <geometry>
-          <cylinder length="${l1}" radius="${r1}"/>
-        </geometry>
-      </collision>
-      <visual name="${namespace}/${lidar_base_frame}_visual">
-        <origin rpy="0 0 0" xyz="0 0 ${l1*0.5}"/>
-        <geometry>
-          <cylinder length="${l1}" radius="${r1}"/>
-        </geometry>
-      </visual>
-    </link>
-    <joint name="${namespace}/${sensor_name}_joint" type="fixed">
+    </xacro:cylinder_link_complete>
+    <joint name="${namespace}/${sensor_name}_joint" type="continuous">
       <parent link="${namespace}/${lidar_base_frame}"/>
       <child link="${namespace}/${lidar_points_frame}"/>
+      <origin rpy="0 0 0" xyz="0 0 ${l1+l2*0.5}"/>
+      <axis xyz="0 0 1"/>
+      <limit effort="100.0" velocity="100.0"/>
     </joint>
-    <link name="${namespace}/${lidar_points_frame}">
-      <inertial>
-        <mass value="${m2}"/>
+    <xacro:cylinder_link_complete link_name="${namespace}/${lidar_points_frame}"
+      mass="${m2}" length="${l2}" radius="${r2}">
         <origin rpy="0 0 0" xyz="0 0 0"/>
-        <inertia ixx="${(m2 * (3.0*r2*r2 + l2*l2)) / 12.0}" ixy="0" ixz="0"
-                 iyy="${(m2 * (3.0*r2*r2 + l2*l2)) / 12.0}" iyz="0"
-                 izz="${0.5 * m2 * (r2*r2)}"/>
-      </inertial>
-      <collision>
-        <origin rpy="0 0 0" xyz="0 0 0"/>
-        <geometry>
-          <cylinder length="${l2}" radius="${r2}"/>
-        </geometry>
-      </collision>
-      <visual name="${namespace}/${lidar_points_frame}_visual">
-        <origin rpy="0 0 0" xyz="0 0 0"/>
-        <geometry>
-          <cylinder length="${l2}" radius="${r2}"/>
-        </geometry>
-      </visual>
-    </link>
+    </xacro:cylinder_link_complete>
     <gazebo reference="${namespace}/${lidar_points_frame}">
       <material>Gazebo/Black</material>
@@ -68,25 +46,8 @@
       <origin rpy="0 0 0" xyz="0 0 ${l1+l2*0.5}"/>
     </joint>
-    <link name="${namespace}/${lidar_base_frame}_hat">
-      <inertial>
-        <mass value="${m1}"/>
+    <xacro:cylinder_link_complete link_name="${namespace}/${lidar_base_frame}_hat"
+      mass="${m1}" length="${l1}" radius="${r1}">
         <origin rpy="0 0 0" xyz="0 0 ${(l1+l2)*0.5}"/>
-        <inertia ixx="${(m1 * (3.0*r1*r1 + l1*l1)) / 12.0}" ixy="0" ixz="0"
-                 iyy="${(m1 * (3.0*r1*r1 + l1*l1)) / 12.0}" iyz="0"
-                 izz="${0.5 * m1 * (r1*r1)}"/>
-      </inertial>
-      <collision>
-        <origin rpy="0 0 0" xyz="0 0 ${(l1+l2)*0.5}"/>
-        <geometry>
-          <cylinder length="${l1}" radius="${r1}"/>
-        </geometry>
-      </collision>
-      <visual>
-        <origin rpy="0 0 0" xyz="0 0 ${(l1+l2)*0.5}"/>
-        <geometry>
-          <cylinder length="${l1}" radius="${r1}"/>
-        </geometry>
-      </visual>
-    </link>
+    </xacro:cylinder_link_complete>
     <gazebo reference="${namespace}/${lidar_points_frame}">
       <!-- Add a ray sensor, and give it a name -->
@@ -94,7 +55,7 @@
         <pose>0 0 0 0 0 0</pose>
         <!-- Enable visualization to see the rays in the GUI -->
-        <visualize>false</visualize>
+        <visualize>true</visualize>
         <!-- Set the update rate of the sensor -->
-        <update_rate>${spin_frequency_hz}</update_rate>
+        <update_rate>${360.0/horizontal_angular_resolution_deg*spin_frequency_hz}</update_rate>
         <ray>
           <noise>
@@ -106,5 +67,5 @@
           <scan>
             <horizontal>
-              <samples>1024</samples>
+              <samples>1</samples>
               <resolution>1</resolution>
               <min_angle>0</min_angle>
@@ -128,6 +89,7 @@
           </range>
         </ray>
-        <plugin name="gazebo_ros_lidar_plugin" filename="librotors_gazebo_os1_plugin.so">
+        <plugin name="gazebo_ros_laser_plugin" filename="libgazebo_ros_laser_plugin.so">
           <robot_namespace>${namespace}</robot_namespace>
+          <joint_name>${namespace}/${sensor_name}_joint</joint_name>
           <topic_name>${topic}</topic_name>
           <frame_name>${lidar_points_frame}</frame_name>

Commit message: fixes the os-1

File: rotors_description/urdf/ouster_os1.urdf.xacro (robot description, xacro)
@@ -22,4 +22,5 @@
       <parent link="${namespace}/${lidar_base_frame}"/>
       <child link="${namespace}/${lidar_points_frame}"/>
+      <origin rpy="0 0 0" xyz="0 0 ${l1+l2*0.5}"/>
     </joint>
     <xacro:cylinder_link_complete link_name="${namespace}/${lidar_points_frame}"

Commit message: makes number of beams adjustable for the os1

File: rotors_description/urdf/ouster_os1.urdf.xacro (robot description, xacro)
@@ -9,5 +9,5 @@
   <xacro:property name="l2" value="0.0305"/>
   <xacro:include filename="$(find rotors_description)/urdf/multirotor_base.xacro" />
-  <xacro:macro name="OS-1" params="*origin parent:=world sensor_name:=os1 topic:=/os1_points spin_frequency_hz:=10 lidar_base_frame:=os1_base lidar_points_frame:=os1_top namespace:=example min_range:=0.05">
+  <xacro:macro name="OS-1" params="*origin parent:=world sensor_name:=os1 topic:=/os1_points spin_frequency_hz:=10 lidar_base_frame:=os1_base lidar_points_frame:=os1_points namespace:=example min_range:=0.05 n_beams:=64">
     <joint name="${namespace}/${lidar_base_frame}_mount_joint" type="fixed">
       <xacro:insert_block name="origin" />
@@ -63,5 +63,5 @@
             </horizontal>
             <vertical>
-              <samples>64</samples>
+              <samples>${n_beams}</samples>
               <resolution>1</resolution>
               <min_angle>-${16.6*M_PI/180.0}</min_angle>

File: rotors_description/urdf/ouster_os1_spinning.urdf.xacro (robot description, xacro)
@@ -9,5 +9,5 @@
   <xacro:property name="l2" value="0.0305"/>
   <xacro:include filename="$(find rotors_description)/urdf/multirotor_base.xacro" />
-  <xacro:macro name="OS-1-spinning" params="*origin parent:=world sensor_name:=os1 topic:=/os1_points horizontal_angular_resolution_deg:=0.18 spin_frequency_hz:=10 lidar_base_frame:=os1_base lidar_points_frame:=os1_top namespace:=example min_range:=0.05">
+  <xacro:macro name="OS-1-spinning" params="*origin parent:=world sensor_name:=os1 topic:=/os1_points horizontal_angular_resolution_deg:=0.18 spin_frequency_hz:=10 lidar_base_frame:=os1_base lidar_points_frame:=os1_top namespace:=example min_range:=0.05 n_beams:=64">
     <gazebo>
       <plugin name="JointController" filename="libgazebo_ros_continous_joint_controller_plugin.so">
@@ -73,5 +73,5 @@
             </horizontal>
             <vertical>
-              <samples>64</samples>
+              <samples>${n_beams}</samples>
               <resolution>1</resolution>
               <min_angle>-${16.6*M_PI/180.0}</min_angle>
