Commit message: fixes HDL-32 namespaces and demo files

File: rotors_description/urdf/lidar_model.urdf.xacro (robot description, xacro)
@@ -3,5 +3,5 @@
 <robot xmlns:xacro="http://www.ros.org/wiki/xacro" name="lidar_model">
   <xacro:arg name="sensor_name" default="velodyne"/>
-  <xacro:arg name="topic" default="/velodyne_points" />
+  <xacro:arg name="topic" default="velodyne_points" />
   <xacro:arg name="horizontal_angular_resolution_deg" default="1.0" />
   <xacro:arg name="spin_frequency_hz" default="0.5" />
@@ -9,4 +9,5 @@
   <xacro:arg name="lidar_points_frame" default="velodyne_top" />
   <xacro:arg name="world_frame" default="world" />
+  <xacro:arg name="namespace" default="lidar_model" />
   <link name="$(arg world_frame)" />
   <xacro:include filename="$(find rotors_description)/urdf/velodyne_HDL_32E.urdf.xacro"/>
@@ -18,5 +19,5 @@
            lidar_base_frame="$(arg lidar_base_frame)"
            lidar_points_frame="$(arg lidar_points_frame)"
-           model_name="lidar_model">
+           namespace="$(arg namespace)">
     <origin xyz="0 0 0.7" rpy="0 0 0" />
   </HDL-32E>

File: rotors_description/urdf/velodyne_HDL_32E.urdf.xacro (robot description, xacro)
@@ -2,14 +2,14 @@
 <robot xmlns:xacro="http://www.ros.org/wiki/xacro" name="HDL-32E">
   <xacro:property name="M_PI" value="3.1415926535897931" />
-  <xacro:macro name="HDL-32E" params="*origin parent:=world sensor_name:=velodyne topic:=/velodyne_points horizontal_angular_resolution_deg:=1.0 spin_frequency_hz:=0.5 lidar_base_frame:=velodyne_base lidar_points_frame:=velodyne_top model_name:=example">
-  <gazebo>
-    <plugin name="JointController" filename="libgazebo_ros_continous_joint_controller_plugin.so">
-        <joint>${sensor_name}_joint</joint>
-	<robot_namespace>${model_name}</robot_namespace>
-	<default_velocity_limit>100</default_velocity_limit>
+  <xacro:macro name="HDL-32E" params="*origin parent:=world sensor_name:=velodyne topic:=/velodyne_points horizontal_angular_resolution_deg:=1.0 spin_frequency_hz:=0.5 lidar_base_frame:=velodyne_base lidar_points_frame:=velodyne_top namespace:=example min_range:=0.06">
+    <gazebo>
+      <plugin name="JointController" filename="libgazebo_ros_continous_joint_controller_plugin.so">
+        <joint>${namespace}/${sensor_name}_joint</joint>
+	      <robot_namespace>${namespace}</robot_namespace>
+	      <default_velocity_limit>100</default_velocity_limit>
         <spin_frequency_hz>${spin_frequency_hz}</spin_frequency_hz>
       </plugin>
-  </gazebo>
-  <link name="${lidar_base_frame}">
+    </gazebo>
+  <link name="${namespace}/${lidar_base_frame}">
     <inertial>
       <mass value="1.2"/>
@@ -17,5 +17,5 @@
       <inertia ixx="0.001087473" ixy="0" ixz="0" iyy="0.001087473" iyz="0" izz="0.001092437"/>
     </inertial>
-    <collision name="${lidar_base_frame}_collision">
+    <collision name="${namespace}/${lidar_base_frame}_collision">
       <origin rpy="0 0 0" xyz="0 0 0.02933"/>
       <geometry>
@@ -23,5 +23,5 @@
       </geometry>
     </collision>
-    <visual name="${lidar_base_frame}_visual">
+    <visual name="${namespace}/${lidar_base_frame}_visual">
       <origin rpy="0 0 0" xyz="0 0 -0.029335"/>
       <geometry>
@@ -30,5 +30,5 @@
     </visual>
   </link>
-  <link name="${lidar_points_frame}">
+  <link name="${namespace}/${lidar_points_frame}">
     <inertial>
       <mass value="0.1"/>
@@ -49,17 +49,17 @@
     </visual>
   </link>
-  <joint name="${lidar_base_frame}_mount_joint" type="fixed">
+  <joint name="${namespace}/${lidar_base_frame}_mount_joint" type="fixed">
     <xacro:insert_block name="origin" />
     <parent link="${parent}"/>
-    <child link="${lidar_base_frame}"/>
+    <child link="${namespace}/${lidar_base_frame}"/>
   </joint>
-  <joint name="${sensor_name}_joint" type="continuous">
-    <parent link="${lidar_base_frame}"/>
-    <child link="${lidar_points_frame}"/>
+  <joint name="${namespace}/${sensor_name}_joint" type="continuous">
+    <parent link="${namespace}/${lidar_base_frame}"/>
+    <child link="${namespace}/${lidar_points_frame}"/>
     <origin rpy="0 0 0" xyz="0 0 0.05867"/>
     <axis xyz="0 0 1"/>
     <limit effort="100.0" velocity="100.0"/>
   </joint>
-  <gazebo reference="${lidar_points_frame}">
+  <gazebo reference="${namespace}/${lidar_points_frame}">
     <!-- Add a ray sensor, and give it a name -->
     <sensor type="ray" name="sensor">
@@ -93,5 +93,5 @@
         <range>
           <!-- Minimum distance of the beam -->
-          <min>0.05</min>
+          <min>${min_range}</min>
           <!-- Maximum distance of the beam -->
           <max>70</max>
@@ -101,9 +101,9 @@
       </ray>
       <plugin name="gazebo_ros_laser_plugin" filename="libgazebo_ros_laser_plugin.so">
-        <model_name>${model_name}</model_name>
-        <joint_name>${sensor_name}_joint</joint_name>
+        <robot_namespace>${namespace}</robot_namespace>
+        <joint_name>${namespace}/${sensor_name}_joint</joint_name>
         <topic_name>${topic}</topic_name>
         <frame_name>${lidar_points_frame}</frame_name>
-        <min_range>0.05</min_range>
+        <min_range>${min_range}</min_range>
         <max_range>70</max_range>
         <gaussian_noise>0.02</gaussian_noise>

Commit message: fixes the spinning os1. updates xacro ros-link declarations

File: rotors_description/urdf/lidar_model.urdf.xacro (robot description, xacro)
@@ -1,5 +1,5 @@
 <?xml version="1.0"?>
 <!-- Provides a world frame and mounts the lidar sensor to it. -->
-<robot xmlns:xacro="http://www.ros.org/wiki/xacro" name="lidar_model">
+<robot xmlns:xacro="http://ros.org/wiki/xacro" name="lidar_model">
   <xacro:arg name="sensor_name" default="velodyne"/>
   <xacro:arg name="topic" default="velodyne_points" />

File: rotors_description/urdf/ouster_os1.urdf.xacro (robot description, xacro)
@@ -1,4 +1,4 @@
 <?xml version="1.0" ?>
-<robot xmlns:xacro="http://www.ros.org/wiki/xacro" name="OS-1">
+<robot xmlns:xacro="http://ros.org/wiki/xacro" name="OS-1">
   <xacro:property name="M_PI" value="3.1415926535897931" />
   <xacro:property name="m1" value="0.15"/>

File: rotors_description/urdf/ouster_os1_spinning.urdf.xacro (robot description, xacro)
@@ -1,4 +1,4 @@
 <?xml version="1.0" ?>
-<robot xmlns:xacro="http://www.ros.org/wiki/xacro" name="OS-1-spinning">
+<robot xmlns:xacro="http://ros.org/wiki/xacro" name="OS-1-spinning">
   <xacro:property name="M_PI" value="3.1415926535897931" />
   <xacro:property name="m1" value="0.15"/>
@@ -9,5 +9,5 @@
   <xacro:property name="l2" value="0.0305"/>
   <xacro:include filename="$(find rotors_description)/urdf/multirotor_base.xacro" />
-  <xacro:macro name="OS-1" params="*origin parent:=world sensor_name:=os1 topic:=/os1_points horizontal_angular_resolution_deg:=0.18 spin_frequency_hz:=10 lidar_base_frame:=os1_base lidar_points_frame:=os1_top namespace:=example min_range:=0.05">
+  <xacro:macro name="OS-1-spinning" params="*origin parent:=world sensor_name:=os1 topic:=/os1_points horizontal_angular_resolution_deg:=0.18 spin_frequency_hz:=10 lidar_base_frame:=os1_base lidar_points_frame:=os1_top namespace:=example min_range:=0.05">
     <gazebo>
       <plugin name="JointController" filename="libgazebo_ros_continous_joint_controller_plugin.so">

File: rotors_description/urdf/velodyne_HDL_32E.urdf.xacro (robot description, xacro)
@@ -1,4 +1,4 @@
 <?xml version="1.0" ?>
-<robot xmlns:xacro="http://www.ros.org/wiki/xacro" name="HDL-32E">
+<robot xmlns:xacro="http://ros.org/wiki/xacro" name="HDL-32E">
   <xacro:property name="M_PI" value="3.1415926535897931" />
   <xacro:macro name="HDL-32E" params="*origin parent:=world sensor_name:=velodyne topic:=/velodyne_points horizontal_angular_resolution_deg:=1.0 spin_frequency_hz:=0.5 lidar_base_frame:=velodyne_base lidar_points_frame:=velodyne_top namespace:=example min_range:=0.06">

File: rotors_description/urdf/velodyne_VLP_16.urdf.xacro (robot description, xacro)
@@ -1,4 +1,4 @@
 <?xml version="1.0" ?>
-<robot xmlns:xacro="http://www.ros.org/wiki/xacro" name="VLP-16">
+<robot xmlns:xacro="http://ros.org/wiki/xacro" name="VLP-16">
   <xacro:property name="M_PI" value="3.1415926535897931" />
   <xacro:property name="m1" value="0.4"/>

File: rotors_description/urdf/vi_sensor_base.xacro (robot description, xacro)
@@ -1,4 +1,4 @@
 <?xml version="1.0"?>
-<robot name="vi_sensor" xmlns:xacro="http://www.ros.org/wiki/xacro">
+<robot name="vi_sensor" xmlns:xacro="http://ros.org/wiki/xacro">
   <xacro:property name="namespace" value="vi_sensor" />
   <xacro:include filename="$(find rotors_description)/urdf/component_snippets.xacro" />

Commit message: removed ouster noise and changed pitch of lidar

File: rotors_description/urdf/lidar_model.urdf.xacro (robot description, xacro)
@@ -20,5 +20,5 @@
            lidar_points_frame="$(arg lidar_points_frame)"
            namespace="$(arg namespace)">
-    <origin xyz="0 0 0.7" rpy="0 0 0" />
+    <origin xyz="0 0 0.7" rpy="0 0.17 0" />
   </HDL-32E>
 </robot>

File: rotors_description/urdf/ouster_os1.urdf.xacro (robot description, xacro)
@@ -53,5 +53,5 @@
             <type>gaussian</type>
             <mean>0.0</mean>
-            <stddev>0.02</stddev>
+            <stddev>0.0</stddev> <!--TODO 0.02 -->
           </noise>
           <scan>
@@ -85,5 +85,5 @@
           <min_range>${min_range}</min_range>
           <max_range>120</max_range>
-          <gaussian_noise>0.02</gaussian_noise>
+          <gaussian_noise>0.0</gaussian_noise><!--TODO 0.02 -->
         </plugin>
       </sensor>

Commit message: changed lidar orientation

File: rotors_description/urdf/lidar_model.urdf.xacro (robot description, xacro)
@@ -20,5 +20,5 @@
            lidar_points_frame="$(arg lidar_points_frame)"
            namespace="$(arg namespace)">
-    <origin xyz="0 0 0.7" rpy="0 0.17 0" />
+    <origin xyz="0 0 0.7" rpy="0 1.5 0" />
   </HDL-32E>
 </robot>
