Commit message: Progress on flexing-wing techpod
- Added "toy-world" for easy testing
- 500Hz sim rate to simulate stiffer wings (stiffer->faster dynamics->smaller timesteps required)
- Renaming xacros, adding more visual parts + cameras observing the wings

File: rotors_description/urdf/techpod_X_flex.xacro (robot description, xacro)
@@ -12,5 +12,5 @@
   limitations under the License.
 -->
-<robot name="techpod_X" xmlns:xacro="http://ros.org/wiki/xacro">
+<robot name="techpod_X_flex" xmlns:xacro="http://ros.org/wiki/xacro">
   <!-- Global properties -->
   <xacro:property name="namespace" value="$(arg namespace)" />
@@ -21,5 +21,5 @@
   <xacro:property name="PI" value="3.1415926535897931" />
   <!-- Component masses -->
-  <xacro:property name="mass_fuselage" value="2.05" /> <!-- [kg] -->
+  <xacro:property name="mass_fuselage" value="1.8" /> <!-- [kg] -->
   <xacro:property name="mass_aileron" value="0.1" /> <!-- [kg] -->
   <xacro:property name="mass_flap" value="0.1" /> <!-- [kg] -->
@@ -31,5 +31,5 @@
   <xacro:property name="body_width" value="2.591" /> <!-- [m] -->
   <xacro:property name="body_height" value="0.303" /> <!-- [m] -->
-  <xacro:property name="body_color" value="Gray" />
+  <xacro:property name="body_color" value="White" />
   <xacro:property name="body_mesh_file" value="package://rotors_description/meshes/techpod/techpod_body.dae" />
   <!-- Aileron properties -->
@@ -39,5 +39,5 @@
   <xacro:property name="aileron_min_angle" value="-0.349066" /> <!-- [rad] -->
   <xacro:property name="aileron_max_angle" value="0.349066" /> <!-- [rad] -->
-  <xacro:property name="aileron_color" value="Red" />
+  <xacro:property name="aileron_color" value="${body_color}" />
   <xacro:property name="aileron_left_mesh_file" value="package://rotors_description/meshes/techpod/techpod_aileron_left.dae" />
   <xacro:property name="aileron_right_mesh_file" value="package://rotors_description/meshes/techpod/techpod_aileron_right.dae" />
@@ -48,5 +48,5 @@
   <xacro:property name="elevator_min_angle" value="-0.349066" /> <!-- [rad] -->
   <xacro:property name="elevator_max_angle" value="0.349066" /> <!-- [rad] -->
-  <xacro:property name="elevator_color" value="Blue" />
+  <xacro:property name="elevator_color" value="${body_color}" />
   <xacro:property name="elevator_mesh_file" value="package://rotors_description/meshes/techpod/techpod_elevator.dae" />
   <!-- Flap properties -->
@@ -56,5 +56,5 @@
   <xacro:property name="flap_min_angle" value="-0.349066" /> <!-- [rad] -->
   <xacro:property name="flap_max_angle" value="0.349066" /> <!-- [rad] -->
-  <xacro:property name="flap_color" value="Yellow" />
+  <xacro:property name="flap_color" value="${body_color}" />
   <xacro:property name="flap_left_mesh_file" value="package://rotors_description/meshes/techpod/techpod_flap_left.dae" />
   <xacro:property name="flap_right_mesh_file" value="package://rotors_description/meshes/techpod/techpod_flap_right.dae" />
@@ -65,5 +65,5 @@
   <xacro:property name="rudder_min_angle" value="-0.349066" />
   <xacro:property name="rudder_max_angle" value="0.349066" />
-  <xacro:property name="rudder_color" value="Orange" />
+  <xacro:property name="rudder_color" value="Red" />
   <xacro:property name="rudder_mesh_file" value="package://rotors_description/meshes/techpod/techpod_rudder.dae" />
   <!-- Propeller properties -->
@@ -73,4 +73,23 @@
   <xacro:property name="propeller_color" value="Gray" />
   <xacro:property name="propeller_mesh_file" value="package://rotors_description/meshes/propeller_${propeller_direction}.dae" />
+  <!-- Flexing properties -->
+<!--
+<xacro:property name="k1" value="450" />
+<xacro:property name="d1" value="3.5" />
+<xacro:property name="k2" value="140" />
+<xacro:property name="d2" value="1.9" />
+<xacro:property name="k3" value="60" />
+<xacro:property name="d3" value="1.0" />
+<xacro:property name="k4" value="80" />
+<xacro:property name="d4" value="1.2" />
+-->
+<xacro:property name="k1" value="250" />
+<xacro:property name="d1" value="2" />
+<xacro:property name="k2" value="120" />
+<xacro:property name="d2" value="1.0" />
+<xacro:property name="k3" value="30" />
+<xacro:property name="d3" value="0.7" />
+<xacro:property name="k4" value="80" />
+<xacro:property name="d4" value="1.2" />
   <!-- Inertia of the main body -->
   <xacro:property name="body_inertia">
@@ -108,8 +127,80 @@
     color="${body_color}"
     use_mesh_file="${use_mesh}"
-    mesh_file="package://rotors_description/meshes/techpod_X_flex/fuselage.stl">
-    <origin xyz="0.16 0 0.05" rpy="0 0 0" />
+    mesh_file="package://rotors_description/meshes/techpod_X_flex/fuselage_barless.stl">
+    <origin xyz="0.10 0 0.08" rpy="0 0 0" />
     <xacro:insert_block name="body_inertia" />
   </xacro:fixed_wing_base_macro>
+<joint name="${namespace}/dome_joint" type="fixed">
+  <parent link="${namespace}/base_link" />
+  <child link="${namespace}/dome" />
+</joint>
+<link name="${namespace}/dome">
+  <inertial>
+    <mass value="0.001" />
+    <xacro:box_inertia x="0.001" y="0.001" z="0.001" mass="0.001" />
+  </inertial>
+  <visual>
+    <geometry>
+        <mesh filename="package://rotors_description/meshes/techpod_X_flex/dome.stl" scale="1 1 1" />
+    </geometry>
+  </visual>
+</link>
+<gazebo reference="${namespace}/dome">
+  <material>Gazebo/GreyTransparent</material>
+</gazebo>
+<joint name="${namespace}/bar_joint" type="fixed">
+  <parent link="${namespace}/base_link" />
+  <child link="${namespace}/bar" />
+</joint>
+<link name="${namespace}/bar">
+  <inertial>
+    <mass value="0.001" />
+    <xacro:box_inertia x="0.001" y="0.001" z="0.001" mass="0.001" />
+  </inertial>
+  <visual>
+    <geometry>
+        <mesh filename="package://rotors_description/meshes/techpod_X_flex/bar.stl" scale="1 1 1" />
+    </geometry>
+  </visual>
+</link>
+<gazebo reference="${namespace}/bar">
+  <material>Gazebo/Grey</material>
+</gazebo>
+<joint name="${namespace}/cover" type="fixed">
+  <parent link="${namespace}/base_link" />
+  <child link="${namespace}/cover" />
+</joint>
+<link name="${namespace}/cover">
+  <inertial>
+    <mass value="0.001" />
+    <xacro:box_inertia x="0.001" y="0.001" z="0.001" mass="0.001" />
+  </inertial>
+  <visual>
+    <geometry>
+        <mesh filename="package://rotors_description/meshes/techpod_X_flex/cover_hole.stl" scale="1 1 1" />
+    </geometry>
+  </visual>
+</link>
+<gazebo reference="${namespace}/cover">
+   <material>Gazebo/White</material>
+</gazebo>
+<joint name="${namespace}/motor_joint" type="fixed">
+  <parent link="${namespace}/base_link" />
+  <child link="${namespace}/motor" />
+</joint>
+<link name="${namespace}/motor">
+  <inertial>
+    <mass value="0.001" />
+    <xacro:box_inertia x="0.001" y="0.001" z="0.001" mass="0.001" />
+  </inertial>
+  <visual>
+    <geometry>
+        <mesh filename="package://rotors_description/meshes/techpod_X_flex/motor.stl" scale="1 1 1" />
+    </geometry>
+  </visual>
+</link>
+<gazebo reference="${namespace}/motor">
+  <material>Gazebo/Black</material>
+</gazebo>
   <!-- Instantiate flexing wing segments -->
   <xacro:airfoil_segment
@@ -118,6 +209,6 @@
     parent="${namespace}/base_link"
     mass_segment="0.15"
-    k = "150"
-    c = "5"
+    k = "${k1}"
+    c = "${d1}"
     color="${body_color}"
     use_mesh_file="${use_mesh}"
@@ -156,4 +247,6 @@
           <cs name="flap_left">
               <controlJoint>${namespace}/flap_left_1_joint</controlJoint>
+              <fromTopic>true</fromTopic>
+              <csRefTopic>flap_l1_pos</csRefTopic>
               <radToCLift>2</radToCLift>
               <radToCDrag>0.0</radToCDrag>
@@ -170,6 +263,6 @@
   parent="${namespace}/base_link"
   mass_segment="0.15"
-  k = "150"
-  c = "5"
+  k = "${k1}"
+  c = "${d1}"
   color="${body_color}"
   use_mesh_file="${use_mesh}"
@@ -208,4 +301,6 @@
           <cs name="flap_right">
               <controlJoint>${namespace}/flap_right_1_joint</controlJoint>
+              <fromTopic>true</fromTopic>
+              <csRefTopic>flap_r1_pos</csRefTopic>
               <radToCLift>2</radToCLift>
               <radToCDrag>0.0</radToCDrag>
@@ -222,7 +317,7 @@
   parent="${namespace}/wl_1"
   mass_segment="0.1"
-  k = "50"
-  c = "1"
-  color="${body_color}"
+  k = "${k2}"
+  c = "${d2}"
+  color="Red"
   use_mesh_file="${use_mesh}"
   mesh_file="package://rotors_description/meshes/techpod_X_flex/wing_l_2.stl"
@@ -252,4 +347,6 @@
           <cs name="flap_left">
               <controlJoint>${namespace}/flap_left_2_joint</controlJoint>
+              <fromTopic>true</fromTopic>
+              <csRefTopic>flap_l2_pos</csRefTopic>
               <radToCLift>2</radToCLift>
               <radToCDrag>0.0</radToCDrag>
@@ -274,7 +371,7 @@
   parent="${namespace}/wr_1"
   mass_segment="0.1"
-  k = "50"
-  c = "1"
-  color="${body_color}"
+  k = "${k2}"
+  c = "${d2}"
+  color="Red"
   use_mesh_file="${use_mesh}"
   mesh_file="package://rotors_description/meshes/techpod_X_flex/wing_r_2.stl"
@@ -304,4 +401,6 @@
           <cs name="flap_right">
               <controlJoint>${namespace}/flap_right_2_joint</controlJoint>
+              <fromTopic>true</fromTopic>
+              <csRefTopic>flap_r2_pos</csRefTopic>
               <radToCLift>2</radToCLift>
               <radToCDrag>0.0</radToCDrag>
@@ -326,6 +425,6 @@
   parent="${namespace}/wl_2"
   mass_segment="0.1"
-  k = "35"
-  c = "0.015"
+  k = "${k3}"
+  c = "${d3}"
   color="${body_color}"
   use_mesh_file="${use_mesh}"
@@ -356,4 +455,6 @@
           <cs name="aileron_left">
               <controlJoint>${namespace}/aileron_left_joint</controlJoint>
+              <fromTopic>true</fromTopic>
+              <csRefTopic>ail_l_pos</csRefTopic>
               <radToCLift>2</radToCLift>
               <radToCDrag>0.0</radToCDrag>
@@ -378,6 +479,6 @@
   parent="${namespace}/wr_2"
   mass_segment="0.1"
-  k = "35"
-  c = "0.015"
+  k = "${k3}"
+  c = "${d3}"
   color="${body_color}"
   use_mesh_file="${use_mesh}"
@@ -408,4 +509,6 @@
           <cs name="aileron_right">
               <controlJoint>${namespace}/aileron_right_joint</controlJoint>
+              <fromTopic>true</fromTopic>
+              <csRefTopic>ail_r_pos</csRefTopic>
               <radToCLift>2</radToCLift>
               <radToCDrag>0.0</radToCDrag>
@@ -430,6 +533,6 @@
   parent="${namespace}/base_link"
   mass_segment="0.15"
-  k = "50"
-  c = "0.5"
+  k = "${k4}"
+  c = "${d4}"
   color="${body_color}"
   use_mesh_file="${use_mesh}"
@@ -463,4 +566,6 @@
         <cs name="rudder">
             <controlJoint>${namespace}/rudder_joint</controlJoint>
+            <fromTopic>true</fromTopic>
+            <csRefTopic>rudd_pos</csRefTopic>
             <radToCLift>3</radToCLift>
             <radToCDrag>0.0</radToCDrag>
@@ -477,6 +582,6 @@
   parent="${namespace}/vs"
   mass_segment="0.15"
-  k = "35"
-  c = "0.35"
+  k = "${k4}"
+  c = "${d4}"
   color="${body_color}"
   use_mesh_file="${use_mesh}"
@@ -510,4 +615,6 @@
         <cs name="elevator_left">
             <controlJoint>${namespace}/elevator_joint</controlJoint>
+            <fromTopic>true</fromTopic>
+            <csRefTopic>elev_pos</csRefTopic>
             <radToCLift>2</radToCLift>
             <radToCDrag>0.0</radToCDrag>
@@ -529,4 +636,6 @@
         <cs name="elevator_right">
             <controlJoint>${namespace}/elevator_joint</controlJoint>
+            <fromTopic>true</fromTopic>
+            <csRefTopic>elev_pos</csRefTopic>
             <radToCLift>2</radToCLift>
             <radToCDrag>0.0</radToCDrag>
@@ -624,5 +733,5 @@
   min_angle="${flap_min_angle}"
   max_angle="${flap_max_angle}"
-  color="${flap_color}"
+  color="Red"
   use_mesh_file="true"
   mesh_file="package://rotors_description/meshes/techpod_X_flex/flp_l_2.stl"
@@ -662,5 +771,5 @@
 min_angle="${flap_min_angle}"
 max_angle="${flap_max_angle}"
-color="${flap_color}"
+color="Red"
 use_mesh_file="true"
 mesh_file="package://rotors_description/meshes/techpod_X_flex/flp_r_2.stl"
@@ -940,5 +1049,5 @@
         <input_index>4</input_index>
         <input_offset>1</input_offset>
-        <input_scaling>366</input_scaling><!-- max rad/s/2 -->
+        <input_scaling>466</input_scaling><!-- max rad/s/2 -->
         <zero_position_disarmed>0</zero_position_disarmed>
         <zero_position_armed>0</zero_position_armed>
@@ -963,4 +1072,5 @@
         <joint_control_type>servo</joint_control_type>
         <joint_name>${namespace}/aileron_left_joint</joint_name>
+        <gztopic>ail_l_pos</gztopic>
       </channel>
       <channel name="aileron_right">
@@ -972,4 +1082,5 @@
         <joint_control_type>servo</joint_control_type>
         <joint_name>${namespace}/aileron_right_joint</joint_name>
+        <gztopic>ail_r_pos</gztopic>
       </channel>
       <channel name="elevator">
@@ -981,4 +1092,5 @@
         <joint_control_type>servo</joint_control_type>
         <joint_name>${namespace}/elevator_joint</joint_name>
+        <gztopic>elev_pos</gztopic>
       </channel>
       <channel name="rudder">
@@ -990,4 +1102,5 @@
         <joint_control_type>servo</joint_control_type>
         <joint_name>${namespace}/rudder_joint</joint_name>
+        <gztopic>rudd_pos</gztopic>
       </channel>
       <channel name="flap_left_1">
@@ -999,4 +1112,5 @@
         <joint_control_type>servo</joint_control_type>
         <joint_name>${namespace}/flap_left_1_joint</joint_name>
+        <gztopic>flap_l1_pos</gztopic>
       </channel>
       <channel name="flap_left_2">
@@ -1008,4 +1122,5 @@
         <joint_control_type>servo</joint_control_type>
         <joint_name>${namespace}/flap_left_2_joint</joint_name>
+        <gztopic>flap_l2_pos</gztopic>
       </channel>
       <channel name="flap_right_1">
@@ -1017,4 +1132,5 @@
         <joint_control_type>servo</joint_control_type>
         <joint_name>${namespace}/flap_right_1_joint</joint_name>
+        <gztopic>flap_r1_pos</gztopic>
       </channel>
       <channel name="flap_right_2">
@@ -1026,4 +1142,5 @@
         <joint_control_type>servo</joint_control_type>
         <joint_name>${namespace}/flap_right_2_joint</joint_name>
+        <gztopic>flap_r2_pos</gztopic>
       </channel>
     </control_channels>
