Commit message: Major modifications to propulsion plugin compiling
- New architecture where propellers are implemented as structs within plugin
- Outsourcing propeller parameter to yaml
- Flexible amount of props per plugin, dynamic alloc
- Modified way to input yaml files (only indicating base path in higher-level xacros/launch files)

File: rotors_description/urdf/techpod_X.xacro (robot description, xacro)
@@ -17,4 +17,5 @@
   <xacro:property name="rotor_velocity_slowdown_sim" value="10" />
   <xacro:property name="use_mesh" value="true" />
+  <xacro:property name="yaml_path" value="$(arg yaml_path)"/>
   <!-- Constants -->
   <xacro:property name="PI" value="3.1415926535897931" />
@@ -237,4 +238,16 @@
   </xacro:propeller>
   <gazebo>
+    <plugin filename="librotors_gazebo_propulsion_plugin.so" name="propulsion_plugin">
+      <robotNamespace>${namespace}</robotNamespace>
+      <propeller name = "main">
+        <jointName>${namespace}/propeller_joint</jointName>
+        <turnDir>ccw</turnDir>
+        <cp>0 0 0</cp>
+        <propParamsYAML>${yaml_path}/propeller_test.yaml</propParamsYAML>
+        <propSlpStrPubTopic></propSlpStrPubTopic>
+      </propeller>
+    </plugin>
+  </gazebo>
+  <gazebo>
     <plugin filename="librotors_gazebo_aerodynamics_plugin.so" name="aerodynamics_plugin">
       <robotNamespace>${namespace}</robotNamespace>
@@ -257,5 +270,5 @@
           <seg_area>0.028</seg_area>
           <seg_chord>0.16</seg_chord>
-          <aeroParamsYAML>"$(arg airfoil_yaml_file)"</aeroParamsYAML>
+          <aeroParamsYAML>${yaml_path}/airfoil_test.yaml</aeroParamsYAML>
         </segment>
         <segment name="WL2">
@@ -265,5 +278,5 @@
           <seg_area>0.072</seg_area>
           <seg_chord>0.16</seg_chord>
-          <aeroParamsYAML>"$(arg airfoil_yaml_file)"</aeroParamsYAML>
+          <aeroParamsYAML>${yaml_path}/airfoil_test.yaml</aeroParamsYAML>
           <control>
             <cs name="flap_left">
@@ -281,5 +294,5 @@
           <seg_area>0.032</seg_area>
           <seg_chord>0.16</seg_chord>
-          <aeroParamsYAML>"$(arg airfoil_yaml_file)"</aeroParamsYAML>
+          <aeroParamsYAML>${yaml_path}/airfoil_test.yaml</aeroParamsYAML>
         </segment>
         <segment name="WL4">
@@ -289,5 +302,5 @@
           <seg_area>0.056</seg_area>
           <seg_chord>0.16</seg_chord>
-          <aeroParamsYAML>"$(arg airfoil_yaml_file)"</aeroParamsYAML>
+          <aeroParamsYAML>${yaml_path}/airfoil_test.yaml</aeroParamsYAML>
           <control>
             <cs name="aileron_left">
@@ -305,5 +318,5 @@
           <seg_area>0.0192</seg_area>
           <seg_chord>0.16</seg_chord>
-          <aeroParamsYAML>"$(arg airfoil_yaml_file)"</aeroParamsYAML>
+          <aeroParamsYAML>${yaml_path}/airfoil_test.yaml</aeroParamsYAML>
         </segment>
         <segment name="WR1">
@@ -313,5 +326,5 @@
           <seg_area>0.028</seg_area>
           <seg_chord>0.16</seg_chord>
-          <aeroParamsYAML>"$(arg airfoil_yaml_file)"</aeroParamsYAML>
+          <aeroParamsYAML>${yaml_path}/airfoil_test.yaml</aeroParamsYAML>
         </segment>
         <segment name="WR2">
@@ -321,5 +334,5 @@
           <seg_area>0.072</seg_area>
           <seg_chord>0.16</seg_chord>
-          <aeroParamsYAML>"$(arg airfoil_yaml_file)"</aeroParamsYAML>
+          <aeroParamsYAML>${yaml_path}/airfoil_test.yaml</aeroParamsYAML>
           <control>
             <cs name="flap_right">
@@ -337,5 +350,5 @@
           <seg_area>0.032</seg_area>
           <seg_chord>0.16</seg_chord>
-          <aeroParamsYAML>"$(arg airfoil_yaml_file)"</aeroParamsYAML>
+          <aeroParamsYAML>${yaml_path}/airfoil_test.yaml</aeroParamsYAML>
         </segment>
         <segment name="WR4">
@@ -345,5 +358,5 @@
           <seg_area>0.056</seg_area>
           <seg_chord>0.16</seg_chord>
-          <aeroParamsYAML>"$(arg airfoil_yaml_file)"</aeroParamsYAML>
+          <aeroParamsYAML>${yaml_path}/airfoil_test.yaml</aeroParamsYAML>
           <control>
             <cs name="aileron_right">
@@ -361,5 +374,5 @@
           <seg_area>0.0192</seg_area>
           <seg_chord>0.16</seg_chord>
-          <aeroParamsYAML>"$(arg airfoil_yaml_file)"</aeroParamsYAML>
+          <aeroParamsYAML>${yaml_path}/airfoil_test.yaml</aeroParamsYAML>
         </segment>
         <segment name="EL1">
@@ -369,5 +382,5 @@
           <seg_area>0.03</seg_area>
           <seg_chord>0.12</seg_chord>
-          <aeroParamsYAML>"$(arg airfoil_yaml_file)"</aeroParamsYAML>
+          <aeroParamsYAML>${yaml_path}/airfoil_test.yaml</aeroParamsYAML>
           <control>
             <cs name="elevator_left">
@@ -385,5 +398,5 @@
           <seg_area>0.03</seg_area>
           <seg_chord>0.12</seg_chord>
-          <aeroParamsYAML>"$(arg airfoil_yaml_file)"</aeroParamsYAML>
+          <aeroParamsYAML>${yaml_path}/airfoil_test.yaml</aeroParamsYAML>
           <control>
             <cs name="elevator_right">
@@ -401,5 +414,5 @@
           <seg_area>0.03</seg_area>
           <seg_chord>0.12</seg_chord>
-          <aeroParamsYAML>"$(arg airfoil_yaml_file)"</aeroParamsYAML>
+          <aeroParamsYAML>${yaml_path}/airfoil_test.yaml</aeroParamsYAML>
           <control>
             <cs name="rudder">

Commit message: aerodynamics plugin: - visualization of slipstream velocities - fix error in calculation of slipstream radial decay
propulsion plugin:
- cannot use fast spinning link for prop dynamics without aliasing in physics engine, hence
  either slow down as in rotorS or implement own dynamics -> chose the latter
- subscription to motor reference velocity message (no longer querying joint vel)
- first order motor model: gives angular vel and -accel of prop -> calculate and apply
  total mech. moment by prop on parent link (e.g. fuselage), rigid body dynamics...
- Multiple new parameters/variables to replace info provided by joint before...
- typedef, renaming, formatting, commenting

mavlink interface:
- mods to relay motor speed reference on gazebo float32 msg (subscribed by propellers)

uav_parameters:
- some debugging related to yaml parsing - still not working:
node.IsNull = true all the time but file seems to be ok & is found

techpod_X.xacro, propeller_test.yaml:
- adding slisptream to horizontal- and vertical stabilizer
- adjusting tags for modified propulsion plugin

SetupInstructions:
- wyriwyg

File: rotors_description/urdf/techpod_X.xacro (robot description, xacro)
@@ -26,10 +26,10 @@
   <xacro:property name="mass_elevator" value="0.1" /> <!-- [kg] -->
   <xacro:property name="mass_rudder" value="0.1" /> <!-- [kg] -->
-  <xacro:property name="mass_propeller" value="0.1" /> <!-- [kg] -->
+  <xacro:property name="mass_propeller" value="0.01" /> <!-- [kg] -->
   <!-- Main body properties -->
   <xacro:property name="body_length" value="1.088" /> <!-- [m] -->
   <xacro:property name="body_width" value="2.591" /> <!-- [m] -->
   <xacro:property name="body_height" value="0.303" /> <!-- [m] -->
-  <xacro:property name="body_color" value="Gray" />
+  <xacro:property name="body_color" value="White" />
   <xacro:property name="body_mesh_file" value="package://rotors_description/meshes/techpod/techpod_body.dae" />
   <!-- Aileron properties -->
@@ -240,9 +240,11 @@
     <plugin filename="librotors_gazebo_propulsion_plugin.so" name="propulsion_plugin">
       <robotNamespace>${namespace}</robotNamespace>
-      <linkName>${namespace}/base_link</linkName>
       <prop name="P0">
         <jointName>${namespace}/propeller_P0_joint</jointName>
-        <turnDir>ccw</turnDir>
-        <cp>0 0 0</cp>
+        <linkNameParent>${namespace}/base_link</linkNameParent>
+        <cp>-0.025 0 0.15</cp>
+        <axisPosRot>-1 0 0</axisPosRot>
+        <turnDir>cw</turnDir>
+        <speedRefTopic>prop_P0_ref</speedRefTopic>
         <propParamsYAML>${yaml_path}/propeller_test.yaml</propParamsYAML>
         <slpstrTopic>prop0_slpstr</slpstrTopic>
@@ -385,4 +387,7 @@
           <seg_chord>0.12</seg_chord>
           <aeroParamsYAML>${yaml_path}/airfoil_test.yaml</aeroParamsYAML>
+          <indVel name="prop0">
+            <topic>prop0_slpstr</topic>
+          </indVel>
           <control>
             <cs name="elevator_left">
@@ -401,4 +406,7 @@
           <seg_chord>0.12</seg_chord>
           <aeroParamsYAML>${yaml_path}/airfoil_test.yaml</aeroParamsYAML>
+          <indVel name="prop0">
+            <topic>prop0_slpstr</topic>
+          </indVel>
           <control>
             <cs name="elevator_right">
@@ -417,8 +425,11 @@
           <seg_chord>0.12</seg_chord>
           <aeroParamsYAML>${yaml_path}/airfoil_test.yaml</aeroParamsYAML>
+          <indVel name="prop0">
+            <topic>prop0_slpstr</topic>
+          </indVel>
           <control>
             <cs name="rudder">
                 <controlJoint>${namespace}/rudder_joint</controlJoint>
-                <radToCLift>2</radToCLift>
+                <radToCLift>3</radToCLift>
                 <radToCDrag>0.0</radToCDrag>
                 <radToCPitch>0.0</radToCPitch>
@@ -454,10 +465,19 @@
       <channel name="propeller">
         <input_index>4</input_index>
-        <input_offset>0</input_offset>
-        <input_scaling>0</input_scaling>
-        <zero_position_disarmed>0</zero_position_disarmed>
-        <zero_position_armed>0</zero_position_armed>
-        <joint_control_type>servo</joint_control_type>
-        <joint_name></joint_name>
+        <input_offset>1</input_offset>
+        <input_scaling>366</input_scaling><!-- max rad/s/2 -->
+        <zero_position_disarmed>0</zero_position_disarmed>
+        <zero_position_armed>0</zero_position_armed>
+        <joint_control_type>position_gztopic</joint_control_type>
+        <gztopic>prop_P0_ref</gztopic>
+        <!--
+        <joint_name>${namespace}/propeller_P0_joint</joint_name>
+        <joint_control_pid>
+          <p>1</p>
+          <d>0.1</d>
+          <cmdMin>10</cmdMin>
+          <cmdMax>-10</cmdMax>
+        </joint_control_pid>
+        -->
       </channel>
       <channel name="aileron_left">

Commit message: Adjusted setup instructions, temp fix techpod_X to load .yaml files, sim freq info in debug output
- Fixed/extended setup instructions after two student ran into problems during installation.
- Adding a camera to techpod_X somehow resolved the error when parsing yaml files. No idea why yet.
- Printing simulation frequency in debug output to check for real-time rate even if gzclient not running

File: rotors_description/urdf/techpod_X.xacro (robot description, xacro)
@@ -1,3 +1,3 @@
-<?xml version="1.0"?>
+<?xml version="1.0" encoding="UTF-8"?>
 <!--
   Copyright 2016 Pavel Vechersky, ASL, ETH Zurich, Switzerland
@@ -394,5 +394,5 @@
           <seg_area>0.03</seg_area>
           <seg_chord>0.12</seg_chord>
-          <aeroParamsYAML>${yaml_path}/airfoil_test.yaml</aeroParamsYAML>
+          <aeroParamsYAML>${yaml_path}/airfoil_test_2.yaml</aeroParamsYAML>
           <indVel name="prop0">
             <topic>prop_slpstr_0</topic>
@@ -413,5 +413,5 @@
           <seg_area>0.03</seg_area>
           <seg_chord>0.12</seg_chord>
-          <aeroParamsYAML>${yaml_path}/airfoil_test.yaml</aeroParamsYAML>
+          <aeroParamsYAML>${yaml_path}/airfoil_test_2.yaml</aeroParamsYAML>
           <indVel name="prop0">
             <topic>prop_slpstr_0</topic>
@@ -432,5 +432,5 @@
           <seg_area>0.03</seg_area>
           <seg_chord>0.12</seg_chord>
-          <aeroParamsYAML>${yaml_path}/airfoil_test.yaml</aeroParamsYAML>
+          <aeroParamsYAML>${yaml_path}/airfoil_test_2.yaml</aeroParamsYAML>
           <indVel name="prop0">
             <topic>prop_slpstr_0</topic>

File: rotors_description/urdf/techpod_X_base.xacro (robot description, xacro)
@@ -30,9 +30,12 @@
   <xacro:default_pressure_sensor namespace="${namespace}" parent_link="${namespace}/base_link" />
   -->
+  <!--
   <xacro:if value="$(arg enable_ground_truth)">
     <xacro:ground_truth_imu_and_odometry namespace="${namespace}" parent_link="${namespace}/base_link" />
   </xacro:if>
+  -->
   <xacro:if value="$(arg enable_logging)">
     <!-- Instantiate a logger -->
+    <!--
     <xacro:bag_plugin_macro
       namespace="${namespace}"
@@ -40,4 +43,11 @@
       rotor_velocity_slowdown_sim="${rotor_velocity_slowdown_sim}"
       wait_to_record_bag="$(arg wait_to_record_bag)" />
+    -->
   </xacro:if>
+  <xacro:default_camera
+    namespace="${namespace}"
+    parent_link="${namespace}/base_link"
+    camera_suffix="cam_front">
+    <origin xyz="0.465 0 0.05" rpy="0 0.2 0" />
+  </xacro:default_camera>
 </robot>

Commit message: Adding serial device number as parameter which can be passed via launch file - This enables configurable multi-Pixhawk HIL in the future. - Changed name of fw_playground world to 'fw_playground' (instead of 'yosemite')

File: rotors_description/urdf/techpod_X.xacro (robot description, xacro)
@@ -18,4 +18,5 @@
   <xacro:property name="use_mesh" value="true" />
   <xacro:property name="yaml_path" value="$(arg yaml_path)"/>
+  <xacro:property name="serial_device" value="$(arg serial_device)" />
   <!-- Constants -->
   <xacro:property name="PI" value="3.1415926535897931" />
@@ -461,5 +462,5 @@
       <mavlink_udp_port>14560</mavlink_udp_port>
       <serialEnabled>true</serialEnabled>
-      <serialDevice>/dev/ttyACM0</serialDevice>
+      <serialDevice>${serial_device}</serialDevice>
       <baudRate>921600</baudRate>
       <qgc_addr>INADDR_ANY</qgc_addr>
@@ -475,5 +476,5 @@
         <input_index>4</input_index>
         <input_offset>1</input_offset>
-        <input_scaling>366</input_scaling><!-- max rad/s/2 -->
+        <input_scaling>366</input_scaling><!-- max_vel/2  [rad/s]-->
         <zero_position_disarmed>0</zero_position_disarmed>
         <zero_position_armed>0</zero_position_armed>

File: rotors_description/urdf/techpod_X_flex.xacro (robot description, xacro)
@@ -19,4 +19,5 @@
    <xacro:property name="meshes_path" value="package://rotors_description/meshes/techpod_X_flex"/>
    <xacro:property name="yaml_path" value="$(arg yaml_path)" />
+   <xacro:property name="serial_device" value="$(arg serial_device)" />
    <!-- Constants -->
    <xacro:property name="PI" value="3.1415926535897931" />
@@ -989,5 +990,5 @@
          <mavlink_udp_port>14560</mavlink_udp_port>
          <serialEnabled>true</serialEnabled>
-         <serialDevice>/dev/ttyACM0</serialDevice>
+         <serialDevice>${serial_device}</serialDevice>
          <baudRate>921600</baudRate>
          <qgc_addr>INADDR_ANY</qgc_addr>
@@ -1003,6 +1004,5 @@
                <input_index>4</input_index>
                <input_offset>1</input_offset>
-               <input_scaling>466</input_scaling>
-               <!-- max rad/s/2 -->
+               <input_scaling>466</input_scaling><!-- max_vel/2  [rad/s]-->
                <zero_position_disarmed>0</zero_position_disarmed>
                <zero_position_armed>0</zero_position_armed>
