Commit message: Fixing tracking camera once and for all, fix actuator dynamics stated in mavlink interface
gazebo_tracking_camera:
- Separate launch file for tracking camera
- Improved naming
- Tracking camera now controlled via topic (sent by gazebo_mavlink_interface) instead of querying position of some other model in world (which is probably why it didn't work sometimes)

gazebo_mavlink_interface:
- Publishing position topic in mavlink interface which tracking camera can subscribe to.
- Fix typo in case-distinction to simulate the slew-rate constraint of the actuators. (was only active in positive direction)
- Add parsing to optionally specify slew rate and joint control gains in servo mode via xacro/urdf

File: rotors_description/urdf/tracking_cam.xacro (robot description, xacro)
@@ -13,4 +13,6 @@
 -->
 <robot name="tracking_cam" xmlns:xacro="http://ros.org/wiki/xacro">
+    <xacro:property name="namespace" value="$(arg namespace)" />
+    <xacro:property name="target_pos_topic" value="$(arg target_pos_topic)" />
     <xacro:macro name="cylinder_inertia" params="r h mass">
       <inertia ixx="${0.0833333 * mass * (3*r*r + h*h)}" ixy="0.0" ixz="0.0"
@@ -81,5 +83,5 @@
       </gazebo>
     </xacro:macro>
-    <link name="tracking/tripod">
+    <link name="${namespace}/tripod">
       <inertial>
         <mass value="10" />
@@ -100,5 +102,5 @@
       </collision>
     </link>
-    <link name="tracking/panLink">
+    <link name="${namespace}/panLink">
       <inertial>
         <mass value="1e-5" />
@@ -107,5 +109,5 @@
       </inertial>
     </link>
-    <link name="tracking/tiltLink">
+    <link name="${namespace}/tiltLink">
       <inertial>
         <mass value="1e-5" />
@@ -114,23 +116,23 @@
       </inertial>
     </link>
-    <joint name="tracking/pan_joint" type="continuous">
+    <joint name="${namespace}/pan_joint" type="continuous">
       <origin xyz="0 0 1.75" rpy="0 0 0" />
-      <parent link="tracking/tripod" />
-      <child link="tracking/panLink" />
+      <parent link="${namespace}/tripod" />
+      <child link="${namespace}/panLink" />
       <axis xyz="0 0 1" />
     </joint>
-    <joint name="tracking/tilt_joint" type="revolute">
+    <joint name="${namespace}/tilt_joint" type="revolute">
       <origin xyz="0 0 0" rpy="0 0 0" />
-      <parent link="tracking/panLink" />
-      <child link="tracking/tiltLink" />
+      <parent link="${namespace}/panLink" />
+      <child link="${namespace}/tiltLink" />
       <axis xyz="0 -1 0" />
       <limit effort="30" velocity="10.0" lower="-1.56" upper="1.56" />
     </joint>
     <xacro:camera_macro
-      namespace="tracking"
-      parent_link="tracking/tiltLink"
-      camera_suffix="1"
+      namespace="${namespace}"
+      parent_link="${namespace}/tiltLink"
+      camera_suffix="tc"
       frame_rate="30"
-      horizontal_fov="0.1962634"
+      horizontal_fov="0.2962634"
       image_width="1920"
       image_height="1080"
@@ -146,10 +148,9 @@
     <gazebo>
       <plugin filename="librotors_gazebo_tracking_cam_plugin.so" name="tracking_cam_plugin">
-          <panJoint>tracking/pan_joint</panJoint>
-          <tiltJoint>tracking/tilt_joint</tiltJoint>
-          <cameraBaseLink>tracking/tripod</cameraBaseLink>
-          <cameraLink>tracking/tiltLink</cameraLink>
-          <targetLink>$(arg target_link)</targetLink>
-          <targetName>$(arg target_name)</targetName>
+          <panJoint>${namespace}/pan_joint</panJoint>
+          <tiltJoint>${namespace}/tilt_joint</tiltJoint>
+          <cameraBaseLink>${namespace}/tripod</cameraBaseLink>
+          <cameraLink>${namespace}/tiltLink</cameraLink>
+          <targetPosTopic>${target_pos_topic}</targetPosTopic>
       </plugin>
     </gazebo>

Commit message: Make FOV of tracking cam configurable via launch files

File: rotors_description/urdf/tracking_cam.xacro (robot description, xacro)
@@ -15,4 +15,5 @@
     <xacro:property name="namespace" value="$(arg namespace)" />
     <xacro:property name="target_pos_topic" value="$(arg target_pos_topic)" />
+    <xacro:property name="h_fov" value="$(arg h_fov)" />
     <xacro:macro name="cylinder_inertia" params="r h mass">
       <inertia ixx="${0.0833333 * mass * (3*r*r + h*h)}" ixy="0.0" ixz="0.0"
@@ -134,5 +135,5 @@
       camera_suffix="tc"
       frame_rate="30"
-      horizontal_fov="0.2962634"
+      horizontal_fov="${h_fov}"
       image_width="1920"
       image_height="1080"
