Commit message: Propulsion plugin loads w/o errors in gazebo, bug resolving
- forgot to initialize n_props for dynamic alloc :/
- renaming xacro blocks (naming conflict with propeller macro)
- propeller joint naming bug in xacro macro
- yaml loading errors remain, to be solved later

File: rotors_description/urdf/fixed_wing_X_base.xacro (robot description, xacro)
@@ -105,5 +105,5 @@
     params="robot_namespace suffix parent mass_propeller propeller_radius color
       use_mesh_file mesh_file *origin *inertia">
-    <joint name="${robot_namespace}/propeller_{suffix}_joint" type="continuous">
+    <joint name="${robot_namespace}/propeller_${suffix}_joint" type="continuous">
       <xacro:insert_block name="origin" />
       <axis xyz="0 0 1" />

File: rotors_description/urdf/techpod_X.xacro (robot description, xacro)
@@ -227,5 +227,5 @@
   <xacro:propeller
     robot_namespace="${namespace}"
-    suffix=""
+    suffix="main"
     parent="${namespace}/base_link"
     mass_propeller="${mass_propeller}"
@@ -240,11 +240,12 @@
     <plugin filename="librotors_gazebo_propulsion_plugin.so" name="propulsion_plugin">
       <robotNamespace>${namespace}</robotNamespace>
-      <propeller name = "main">
-        <jointName>${namespace}/propeller_joint</jointName>
+      <linkName>${namespace}/base_link</linkName>
+      <prop name="P1">
+        <jointName>${namespace}/propeller_main_joint</jointName>
         <turnDir>ccw</turnDir>
         <cp>0 0 0</cp>
         <propParamsYAML>${yaml_path}/propeller_test.yaml</propParamsYAML>
-        <propSlpStrPubTopic></propSlpStrPubTopic>
-      </propeller>
+        <propSlpStrPubTopic>slipstr</propSlpStrPubTopic>
+      </prop>
     </plugin>
   </gazebo>

Commit message: First attempt to get flexing wings, more cleanup...
- cleanup in aerodynamics plugin
- adding spring damper plugin since setting joint stiffness/damping via urdf didn't work (probably I missed something?)
- added some general model plugin template
- CAD files of wing segments for visual illustration of flexing/bending
- flexing techpod xacro
- install instructions for sim
- todo list for sim
- So far: Sufficient wing-stiffness is hard to model in real time (too fast dynamics for solver) WIP...

File: rotors_description/urdf/fixed_wing_X_base.xacro (robot description, xacro)
@@ -56,9 +56,64 @@
     </gazebo>
   </xacro:macro>
+<!-- Control surface joint and link -->
+<xacro:macro name="airfoil_segment"
+  params="robot_namespace segment_name parent mass_segment k c color use_mesh_file mesh_file segment_length segment_width
+    segment_height *axis *joint_origin *inertia_origin *mesh_origin *inertia ">
+  <joint name="${robot_namespace}/${segment_name}_joint" type="revolute">
+    <xacro:insert_block name="joint_origin" />
+    <xacro:insert_block name="axis" />
+    <parent link="${parent}" />
+    <child link="${robot_namespace}/${segment_name}"/>
+    <limit upper="0.17" lower="-0.17" effort="5000" velocity="50"/>
+  </joint>
+  <link name="${robot_namespace}/${segment_name}">
+    <inertial>
+      <xacro:insert_block name="inertia_origin" />
+      <mass value="${mass_segment}" />
+      <xacro:box_inertia x="${segment_length}" y="${segment_width}" z="${segment_height}" mass="${mass_segment}" />
+    </inertial>
+    <visual>
+      <xacro:insert_block name="mesh_origin" />
+      <geometry>
+        <xacro:if value="${use_mesh_file}">
+          <mesh filename="${mesh_file}" scale="1 1 1" />
+        </xacro:if>
+        <xacro:unless value="${use_mesh_file}">
+          <box size="${segment_length} ${segment_width} ${segment_height}" />
+        </xacro:unless>
+      </geometry>
+    </visual>
+    <collision>
+      <xacro:insert_block name="mesh_origin" />
+      <geometry>
+        <xacro:if value="${use_mesh_file}">
+          <mesh filename="${mesh_file}" scale="1 1 1" />
+        </xacro:if>
+        <xacro:unless value="${use_mesh_file}">
+          <box size="${segment_length} ${segment_width} ${segment_height}" />
+        </xacro:unless>
+      </geometry>
+    </collision>
+  </link>
+  <gazebo reference="${robot_namespace}/${segment_name}">
+    <material>Gazebo/${color}</material>
+  </gazebo>
+  <gazebo reference="${robot_namespace}/${segment_name}_joint">
+    <implicitSpringDamper>true</implicitSpringDamper>
+  </gazebo>
+  <gazebo>
+    <plugin filename="librotors_gazebo_springdamper_plugin.so" name="gazebo_springdamper_plugin">
+      <robotNamespace>${robot_namespace}</robotNamespace>
+      <jointName>${robot_namespace}/${segment_name}_joint</jointName>
+      <damping>${c}</damping>
+      <stiffness>${k}</stiffness>
+    </plugin>
+  </gazebo>
+</xacro:macro>
   <!-- Control surface joint and link -->
   <xacro:macro name="control_surface"
     params="robot_namespace surface_name parent mass_surface min_angle
       max_angle color use_mesh_file mesh_file surface_length surface_width
-      surface_height *axis *joint_origin *link_origin *inertia">
+      surface_height *axis *joint_origin *link_origin *mesh_origin *inertia">
     <joint name="${robot_namespace}/${surface_name}_joint" type="revolute">
       <xacro:insert_block name="joint_origin" />
@@ -75,5 +130,5 @@
       </inertial>
       <visual>
-        <xacro:insert_block name="link_origin" />
+        <xacro:insert_block name="mesh_origin" />
         <geometry>
           <xacro:if value="${use_mesh_file}">
@@ -91,7 +146,9 @@
             <mesh filename="${mesh_file}" scale="1 1 1" />
           </xacro:if>
+          <!--
           <xacro:unless value="${use_mesh_file}">
             <box size="${surface_length} ${surface_width} ${surface_height}" />
           </xacro:unless>
+          -->
         </geometry>
       </collision>
@@ -104,5 +161,5 @@
   <xacro:macro name="propeller"
     params="robot_namespace suffix parent mass_propeller propeller_radius color
-      use_mesh_file mesh_file *origin *inertia">
+      use_mesh_file mesh_file *origin *mesh_origin *inertia">
     <joint name="${robot_namespace}/propeller_${suffix}_joint" type="continuous">
       <xacro:insert_block name="origin" />
@@ -117,12 +174,14 @@
       </inertial>
       <visual>
-        <geometry>
-          <xacro:if value="${use_mesh_file}">
-            <mesh filename="${mesh_file}"
-              scale="${propeller_radius} ${propeller_radius} ${propeller_radius}" />
-          </xacro:if>
+        <xacro:insert_block name="mesh_origin" />
+        <geometry>
+          <xacro:if value="${use_mesh_file}">
+            <mesh filename="${mesh_file}"/>
+          </xacro:if>
+          <!--
           <xacro:unless value="${use_mesh_file}">
             <cylinder length="0.005" radius="${propeller_radius}"/>
           </xacro:unless>
+          -->
         </geometry>
       </visual>
@@ -130,10 +189,11 @@
         <geometry>
           <xacro:if value="${use_mesh_file}">
-            <mesh filename="${mesh_file}"
-              scale="${propeller_radius} ${propeller_radius} ${propeller_radius}" />
-          </xacro:if>
+            <mesh filename="${mesh_file}"/>
+          </xacro:if>
+          <!--
           <xacro:unless value="${use_mesh_file}">
             <cylinder length="0.005" radius="${propeller_radius}"/>
           </xacro:unless>
+          -->
         </geometry>
       </collision>

File: rotors_description/urdf/techpod_X-flex.xacro (robot description, xacro)
@@ -31,5 +31,5 @@
   <xacro:property name="body_width" value="2.591" /> <!-- [m] -->
   <xacro:property name="body_height" value="0.303" /> <!-- [m] -->
-  <xacro:property name="body_color" value="White" />
+  <xacro:property name="body_color" value="Gray" />
   <xacro:property name="body_mesh_file" value="package://rotors_description/meshes/techpod/techpod_body.dae" />
   <!-- Aileron properties -->
@@ -72,5 +72,5 @@
   <xacro:property name="propeller_height" value="0.003" />
   <xacro:property name="propeller_color" value="Gray" />
-  <xacro:property name="propeller_mesh_file" value="package://rotors_description/meshes/techpod/techpod_prop.stl" />
+  <xacro:property name="propeller_mesh_file" value="package://rotors_description/meshes/propeller_${propeller_direction}.dae" />
   <!-- Inertia of the main body -->
   <xacro:property name="body_inertia">
@@ -108,26 +108,452 @@
     color="${body_color}"
     use_mesh_file="${use_mesh}"
-    mesh_file="${body_mesh_file}">
+    mesh_file="package://rotors_description/meshes/techpod_X_flex/fuselage.stl">
     <origin xyz="0.16 0 0.05" rpy="0 0 0" />
     <xacro:insert_block name="body_inertia" />
   </xacro:fixed_wing_base_macro>
+  <!-- Instantiate flexing wing segments -->
+  <xacro:airfoil_segment
+    robot_namespace="${namespace}"
+    segment_name="wl_1"
+    parent="${namespace}/base_link"
+    mass_segment="0.15"
+    k = "150"
+    c = "5"
+    color="${body_color}"
+    use_mesh_file="${use_mesh}"
+    mesh_file="package://rotors_description/meshes/techpod_X_flex/wing_l_1.stl"
+    segment_length="0.1"
+    segment_width="0.4"
+    segment_height="0.02">
+    <axis xyz="1 0 0" />   <!-- Joint axis -->
+    <origin xyz="0 0 0.162" rpy="0 0 0" />   <!-- Joint origin -->
+    <origin xyz="0 0.195 0" rpy="0 0 0" />       <!-- Inertia origin -->
+    <origin xyz="0 0 -0.162" rpy="0 0 0" />  <!-- Mesh origin -->
+    <xacro:insert_block name="aileron_inertia" />
+  </xacro:airfoil_segment>
+<gazebo>
+  <plugin filename="librotors_gazebo_aerodynamics_plugin.so" name="aerodynamics_plugin">
+    <robotNamespace>${namespace}</robotNamespace>
+    <linkName>${namespace}/wl_1</linkName>
+    <aeroForcesVis>aero_force_vis_wl1</aeroForcesVis>
+    <airfoil>
+      <segment name="WL1_1">
+        <forward>1 0 0</forward>
+        <upward>0 0 1</upward>
+        <cp>0 0.1 0</cp>
+        <seg_area>0.016</seg_area>
+        <seg_chord>0.16</seg_chord>
+        <aeroParamsYAML>${yaml_path}/airfoil_test.yaml</aeroParamsYAML>
+      </segment>
+      <segment name="WL1_2">
+        <forward>1 0 0</forward>
+        <upward>0 0 1</upward>
+        <cp>0.0 0.28 0</cp>
+        <seg_area>0.032</seg_area>
+        <seg_chord>0.16</seg_chord>
+        <aeroParamsYAML>${yaml_path}/airfoil_test.yaml</aeroParamsYAML>
+        <control>
+          <cs name="flap_left">
+              <controlJoint>${namespace}/flap_left_1_joint</controlJoint>
+              <radToCLift>2</radToCLift>
+              <radToCDrag>0.0</radToCDrag>
+              <radToCPitch>0.0</radToCPitch>
+          </cs>
+        </control>
+      </segment>
+    </airfoil>
+  </plugin>
+</gazebo>
+<xacro:airfoil_segment
+  robot_namespace="${namespace}"
+  segment_name="wr_1"
+  parent="${namespace}/base_link"
+  mass_segment="0.15"
+  k = "150"
+  c = "5"
+  color="${body_color}"
+  use_mesh_file="${use_mesh}"
+  mesh_file="package://rotors_description/meshes/techpod_X_flex/wing_r_1.stl"
+  segment_length="0.1"
+  segment_width="0.4"
+  segment_height="0.02">
+  <axis xyz="1 0 0" />   <!-- Joint axis -->
+  <origin xyz="0 0 0.162" rpy="0 0 0" />   <!-- Joint origin -->
+  <origin xyz="0 -0.195 0" rpy="0 0 0" />       <!-- Inertia origin -->
+  <origin xyz="0 0 -0.162" rpy="0 0 0" />  <!-- Mesh origin -->
+  <xacro:insert_block name="aileron_inertia" />
+</xacro:airfoil_segment>
+<gazebo>
+  <plugin filename="librotors_gazebo_aerodynamics_plugin.so" name="aerodynamics_plugin">
+    <robotNamespace>${namespace}</robotNamespace>
+    <linkName>${namespace}/wr_1</linkName>
+    <aeroForcesVis>aero_force_vis_wr1</aeroForcesVis>
+    <airfoil>
+      <segment name="WR1_1">
+        <forward>1 0 0</forward>
+        <upward>0 0 1</upward>
+        <cp>0 -0.1 0</cp>
+        <seg_area>0.016</seg_area>
+        <seg_chord>0.16</seg_chord>
+        <aeroParamsYAML>${yaml_path}/airfoil_test.yaml</aeroParamsYAML>
+      </segment>
+      <segment name="WR1_2">
+        <forward>1 0 0</forward>
+        <upward>0 0 1</upward>
+        <cp>0.0 -0.28 0</cp>
+        <seg_area>0.032</seg_area>
+        <seg_chord>0.16</seg_chord>
+        <aeroParamsYAML>${yaml_path}/airfoil_test.yaml</aeroParamsYAML>
+        <control>
+          <cs name="flap_right">
+              <controlJoint>${namespace}/flap_right_1_joint</controlJoint>
+              <radToCLift>2</radToCLift>
+              <radToCDrag>0.0</radToCDrag>
+              <radToCPitch>0.0</radToCPitch>
+          </cs>
+        </control>
+      </segment>
+    </airfoil>
+  </plugin>
+</gazebo>
+<xacro:airfoil_segment
+  robot_namespace="${namespace}"
+  segment_name="wl_2"
+  parent="${namespace}/wl_1"
+  mass_segment="0.1"
+  k = "50"
+  c = "1"
+  color="${body_color}"
+  use_mesh_file="${use_mesh}"
+  mesh_file="package://rotors_description/meshes/techpod_X_flex/wing_l_2.stl"
+  segment_length="0.1"
+  segment_width="0.43"
+  segment_height="0.02">
+  <axis xyz="1 0 0" />   <!-- Joint axis -->
+  <origin xyz="0 0.39 0" rpy="0 0 0" />   <!-- Joint origin -->
+  <origin xyz="0 0.215 0" rpy="0 0 0" />       <!-- Inertia origin -->
+  <origin xyz="0 -0.39 -0.162" rpy="0 0 0" />  <!-- Mesh origin -->
+  <xacro:insert_block name="aileron_inertia" />
+</xacro:airfoil_segment>
+<gazebo>
+  <plugin filename="librotors_gazebo_aerodynamics_plugin.so" name="aerodynamics_plugin">
+    <robotNamespace>${namespace}</robotNamespace>
+    <linkName>${namespace}/wl_2</linkName>
+    <aeroForcesVis>aero_force_vis_wl2</aeroForcesVis>
+    <airfoil>
+      <segment name="WL2_1">
+        <forward>1 0 0</forward>
+        <upward>0 0 1</upward>
+        <cp>0 0.1 0</cp>
+        <seg_area>0.032</seg_area>
+        <seg_chord>0.16</seg_chord>
+        <aeroParamsYAML>${yaml_path}/airfoil_test.yaml</aeroParamsYAML>
+        <control>
+          <cs name="flap_left">
+              <controlJoint>${namespace}/flap_left_2_joint</controlJoint>
+              <radToCLift>2</radToCLift>
+              <radToCDrag>0.0</radToCDrag>
+              <radToCPitch>0.0</radToCPitch>
+          </cs>
+        </control>
+      </segment>
+      <segment name="WL2_2">
+        <forward>1 0 0</forward>
+        <upward>0 0 1</upward>
+        <cp>0.0 0.32 0</cp>
+        <seg_area>0.032</seg_area>
+        <seg_chord>0.16</seg_chord>
+        <aeroParamsYAML>${yaml_path}/airfoil_test.yaml</aeroParamsYAML>
+      </segment>
+    </airfoil>
+  </plugin>
+</gazebo>
+<xacro:airfoil_segment
+  robot_namespace="${namespace}"
+  segment_name="wr_2"
+  parent="${namespace}/wr_1"
+  mass_segment="0.1"
+  k = "50"
+  c = "1"
+  color="${body_color}"
+  use_mesh_file="${use_mesh}"
+  mesh_file="package://rotors_description/meshes/techpod_X_flex/wing_r_2.stl"
+  segment_length="0.1"
+  segment_width="0.43"
+  segment_height="0.02">
+  <axis xyz="1 0 0" />   <!-- Joint axis -->
+  <origin xyz="0 -0.39 0" rpy="0 0 0" />   <!-- Joint origin -->
+  <origin xyz="0 -0.215 0" rpy="0 0 0" />       <!-- Inertia origin -->
+  <origin xyz="0 0.39 -0.162" rpy="0 0 0" />  <!-- Mesh origin -->
+  <xacro:insert_block name="aileron_inertia" />
+</xacro:airfoil_segment>
+<gazebo>
+  <plugin filename="librotors_gazebo_aerodynamics_plugin.so" name="aerodynamics_plugin">
+    <robotNamespace>${namespace}</robotNamespace>
+    <linkName>${namespace}/wr_2</linkName>
+    <aeroForcesVis>aero_force_vis_wr2</aeroForcesVis>
+    <airfoil>
+      <segment name="WR2_1">
+        <forward>1 0 0</forward>
+        <upward>0 0 1</upward>
+        <cp>0 -0.1 0</cp>
+        <seg_area>0.032</seg_area>
+        <seg_chord>0.16</seg_chord>
+        <aeroParamsYAML>${yaml_path}/airfoil_test.yaml</aeroParamsYAML>
+        <control>
+          <cs name="flap_right">
+              <controlJoint>${namespace}/flap_right_2_joint</controlJoint>
+              <radToCLift>2</radToCLift>
+              <radToCDrag>0.0</radToCDrag>
+              <radToCPitch>0.0</radToCPitch>
+          </cs>
+        </control>
+      </segment>
+      <segment name="WR2_2">
+        <forward>1 0 0</forward>
+        <upward>0 0 1</upward>
+        <cp>0.0 -0.32 0</cp>
+        <seg_area>0.032</seg_area>
+        <seg_chord>0.16</seg_chord>
+        <aeroParamsYAML>${yaml_path}/airfoil_test.yaml</aeroParamsYAML>
+      </segment>
+    </airfoil>
+  </plugin>
+</gazebo>
+<xacro:airfoil_segment
+  robot_namespace="${namespace}"
+  segment_name="wl_3"
+  parent="${namespace}/wl_2"
+  mass_segment="0.1"
+  k = "35"
+  c = "0.015"
+  color="${body_color}"
+  use_mesh_file="${use_mesh}"
+  mesh_file="package://rotors_description/meshes/techpod_X_flex/wing_l_3.stl"
+  segment_length="0.1"
+  segment_width="0.5"
+  segment_height="0.02">
+  <axis xyz="1 0 0" />   <!-- Joint axis -->
+  <origin xyz="0 0.43 0" rpy="0 0 0" />   <!-- Joint origin -->
+  <origin xyz="0 0.25 0" rpy="0 0 0" />       <!-- Inertia origin -->
+  <origin xyz="0 -0.82 -0.162" rpy="0 0 0" />  <!-- Mesh origin -->
+  <xacro:insert_block name="aileron_inertia" />
+</xacro:airfoil_segment>
+<gazebo>
+  <plugin filename="librotors_gazebo_aerodynamics_plugin.so" name="aerodynamics_plugin">
+    <robotNamespace>${namespace}</robotNamespace>
+    <linkName>${namespace}/wl_3</linkName>
+    <aeroForcesVis>aero_force_vis_wl3</aeroForcesVis>
+    <airfoil>
+      <segment name="WL3_1">
+        <forward>1 0 0</forward>
+        <upward>0 0 1</upward>
+        <cp>0 0.2 0</cp>
+        <seg_area>0.05</seg_area>
+        <seg_chord>0.16</seg_chord>
+        <aeroParamsYAML>${yaml_path}/airfoil_test.yaml</aeroParamsYAML>
+        <control>
+          <cs name="aileron_left">
+              <controlJoint>${namespace}/aileron_left_joint</controlJoint>
+              <radToCLift>2</radToCLift>
+              <radToCDrag>0.0</radToCDrag>
+              <radToCPitch>0.0</radToCPitch>
+          </cs>
+        </control>
+      </segment>
+      <segment name="WL3_2">
+        <forward>1 0 0</forward>
+        <upward>0 0 1</upward>
+        <cp>0.0 0.4 0</cp>
+        <seg_area>0.016</seg_area>
+        <seg_chord>0.16</seg_chord>
+        <aeroParamsYAML>${yaml_path}/airfoil_test.yaml</aeroParamsYAML>
+      </segment>
+    </airfoil>
+  </plugin>
+</gazebo>
+<xacro:airfoil_segment
+  robot_namespace="${namespace}"
+  segment_name="wr_3"
+  parent="${namespace}/wr_2"
+  mass_segment="0.1"
+  k = "35"
+  c = "0.015"
+  color="${body_color}"
+  use_mesh_file="${use_mesh}"
+  mesh_file="package://rotors_description/meshes/techpod_X_flex/wing_r_3.stl"
+  segment_length="0.1"
+  segment_width="0.5"
+  segment_height="0.02">
+  <axis xyz="1 0 0" />   <!-- Joint axis -->
+  <origin xyz="0 -0.43 0" rpy="0 0 0" />   <!-- Joint origin -->
+  <origin xyz="0 -0.25 0" rpy="0 0 0" />       <!-- Inertia origin -->
+  <origin xyz="0 0.82 -0.162" rpy="0 0 0" />  <!-- Mesh origin -->
+  <xacro:insert_block name="aileron_inertia" />
+</xacro:airfoil_segment>
+<gazebo>
+  <plugin filename="librotors_gazebo_aerodynamics_plugin.so" name="aerodynamics_plugin">
+    <robotNamespace>${namespace}</robotNamespace>
+    <linkName>${namespace}/wr_3</linkName>
+    <aeroForcesVis>aero_force_vis_wr3</aeroForcesVis>
+    <airfoil>
+      <segment name="WR3_1">
+        <forward>1 0 0</forward>
+        <upward>0 0 1</upward>
+        <cp>0 -0.2 0</cp>
+        <seg_area>0.05</seg_area>
+        <seg_chord>0.16</seg_chord>
+        <aeroParamsYAML>${yaml_path}/airfoil_test.yaml</aeroParamsYAML>
+        <control>
+          <cs name="aileron_right">
+              <controlJoint>${namespace}/aileron_right_joint</controlJoint>
+              <radToCLift>2</radToCLift>
+              <radToCDrag>0.0</radToCDrag>
+              <radToCPitch>0.0</radToCPitch>
+          </cs>
+        </control>
+      </segment>
+      <segment name="WR3_2">
+        <forward>1 0 0</forward>
+        <upward>0 0 1</upward>
+        <cp>0.0 -0.4 0</cp>
+        <seg_area>0.016</seg_area>
+        <seg_chord>0.16</seg_chord>
+        <aeroParamsYAML>${yaml_path}/airfoil_test.yaml</aeroParamsYAML>
+      </segment>
+    </airfoil>
+  </plugin>
+</gazebo>
+<xacro:airfoil_segment
+  robot_namespace="${namespace}"
+  segment_name="vs"
+  parent="${namespace}/base_link"
+  mass_segment="0.15"
+  k = "50"
+  c = "0.5"
+  color="${body_color}"
+  use_mesh_file="${use_mesh}"
+  mesh_file="package://rotors_description/meshes/techpod_X_flex/v_stb.stl"
+  segment_length="0.1"
+  segment_width="0.02"
+  segment_height="0.3">
+  <axis xyz="1 0 0" />   <!-- Joint axis -->
+  <origin xyz="-0.618 0 0.031" rpy="0 0 0" />   <!-- Joint origin -->
+  <origin xyz="0 0 0.15" rpy="0 0 0" />       <!-- Inertia origin -->
+  <origin xyz="0.618 0 -0.031" rpy="0 0 0" />  <!-- Mesh origin -->
+  <xacro:insert_block name="aileron_inertia" />
+</xacro:airfoil_segment>
+<gazebo>
+  <plugin filename="librotors_gazebo_aerodynamics_plugin.so" name="aerodynamics_plugin">
+    <robotNamespace>${namespace}</robotNamespace>
+    <linkName>${namespace}/vs</linkName>
+    <aeroForcesVis>aero_force_vis_vs</aeroForcesVis>
+    <airfoil>
+    <segment name="vs">
+      <forward>1 0 0</forward>
+      <upward>0 -1 0</upward>
+      <cp>-0.02 0.0 0.13</cp>
+      <seg_area>0.03</seg_area>
+      <seg_chord>0.12</seg_chord>
+      <aeroParamsYAML>${yaml_path}/airfoil_test.yaml</aeroParamsYAML>
+      <indVel name="prop0">
+        <topic>prop_slpstr_0</topic>
+      </indVel>
+      <control>
+        <cs name="rudder">
+            <controlJoint>${namespace}/rudder_joint</controlJoint>
+            <radToCLift>3</radToCLift>
+            <radToCDrag>0.0</radToCDrag>
+            <radToCPitch>0.0</radToCPitch>
+        </cs>
+      </control>
+    </segment>
+    </airfoil>
+  </plugin>
+</gazebo>
+<xacro:airfoil_segment
+  robot_namespace="${namespace}"
+  segment_name="hs"
+  parent="${namespace}/vs"
+  mass_segment="0.15"
+  k = "35"
+  c = "0.35"
+  color="${body_color}"
+  use_mesh_file="${use_mesh}"
+  mesh_file="package://rotors_description/meshes/techpod_X_flex/h_stb.stl"
+  segment_length="0.1"
+  segment_width="0.4"
+  segment_height="0.02">
+  <axis xyz="1 0 0" />   <!-- Joint axis -->
+  <origin xyz="-0.039 0 0.274" rpy="0 0 0" />   <!-- Joint origin -->
+  <origin xyz="-0.03 0 0" rpy="0 0 0" />       <!-- Inertia origin -->
+  <origin xyz="0.657 0 -0.305" rpy="0 0 0" />  <!-- Mesh origin -->
+  <xacro:insert_block name="aileron_inertia" />
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