Commit message: Timing debug output mavlink, gps ground truth sub for correct magnetometer calc
- fixed_wing_X_base.xacro: some renaming, comment non-base-link collisions for reduced computational compelexity
- comment unused sensors/plugins (magnetometer, pressure sensor)
- add gps-ground truth to mavlink interface (used to look up magnetic field at current (true) position)
- set imu-rate to 250Hz (techpod_X(_flex).xacro)
- timing output to get frequency histogram of sent mavlink messages -> to debug source of timeouts (compare hist with hist from mavlink_receiver on pixhawk -> sim delays vs mavlink delays)

File: rotors_description/urdf/fixed_wing_X_base.xacro (robot description, xacro)
@@ -46,5 +46,5 @@
         </visual>
         <collision>
-          <origin xyz="0 0 0" rpy="0 0 0" />
+          <origin xyz="-0.2 0 0.15" rpy="0 0 0" />
           <geometry>
             <box size="${length} ${width} ${height}" />
@@ -56,8 +56,8 @@
     </gazebo>
   </xacro:macro>
-<!-- Control surface joint and link -->
+<!-- Airfoil segment joint, link and plugin -->
 <xacro:macro name="airfoil_segment"
   params="robot_namespace segment_name parent mass_segment k c color use_mesh_file mesh_file segment_length segment_width
-    segment_height *axis *joint_origin *inertia_origin *mesh_origin *inertia ">
+    segment_height *axis *joint_origin *inertia_origin *vis_coll_origin *inertia ">
   <joint name="${robot_namespace}/${segment_name}_joint" type="revolute">
     <xacro:insert_block name="joint_origin" />
@@ -74,5 +74,5 @@
     </inertial>
     <visual>
-      <xacro:insert_block name="mesh_origin" />
+      <xacro:insert_block name="vis_coll_origin" />
       <geometry>
         <xacro:if value="${use_mesh_file}">
@@ -84,6 +84,7 @@
       </geometry>
     </visual>
+    <!--
     <collision>
-      <xacro:insert_block name="mesh_origin" />
+      <xacro:insert_block name="vis_coll_origin" />
       <geometry>
         <xacro:if value="${use_mesh_file}">
@@ -95,4 +96,5 @@
       </geometry>
     </collision>
+    -->
   </link>
   <gazebo reference="${robot_namespace}/${segment_name}">
@@ -115,5 +117,5 @@
     params="robot_namespace surface_name parent mass_surface min_angle
       max_angle color use_mesh_file mesh_file surface_length surface_width
-      surface_height *axis *joint_origin *link_origin *mesh_origin *inertia">
+      surface_height *axis *joint_origin *link_origin *vis_coll_origin *inertia">
     <joint name="${robot_namespace}/${surface_name}_joint" type="revolute">
       <xacro:insert_block name="joint_origin" />
@@ -130,5 +132,5 @@
       </inertial>
       <visual>
-        <xacro:insert_block name="mesh_origin" />
+        <xacro:insert_block name="vis_coll_origin" />
         <geometry>
           <xacro:if value="${use_mesh_file}">
@@ -140,17 +142,17 @@
         </geometry>
       </visual>
+      <!--
       <collision>
-        <xacro:insert_block name="link_origin" />
+        <xacro:insert_block name="vis_coll_origin" />
         <geometry>
           <xacro:if value="${use_mesh_file}">
             <mesh filename="${mesh_file}" scale="1 1 1" />
           </xacro:if>
-          <!--
           <xacro:unless value="${use_mesh_file}">
             <box size="${surface_length} ${surface_width} ${surface_height}" />
           </xacro:unless>
-          -->
         </geometry>
       </collision>
+      -->
     </link>
     <gazebo reference="${robot_namespace}/${surface_name}">
@@ -161,5 +163,5 @@
   <xacro:macro name="propeller"
     params="robot_namespace suffix parent mass_propeller propeller_radius color
-      use_mesh_file mesh_file *origin *mesh_origin *inertia">
+      use_mesh_file mesh_file *origin *vis_coll_origin *inertia">
     <joint name="${robot_namespace}/propeller_${suffix}_joint" type="continuous">
       <xacro:insert_block name="origin" />
@@ -174,28 +176,27 @@
       </inertial>
       <visual>
-        <xacro:insert_block name="mesh_origin" />
+        <xacro:insert_block name="vis_coll_origin" />
         <geometry>
           <xacro:if value="${use_mesh_file}">
             <mesh filename="${mesh_file}"/>
           </xacro:if>
-          <!--
           <xacro:unless value="${use_mesh_file}">
             <cylinder length="0.005" radius="${propeller_radius}"/>
           </xacro:unless>
-          -->
         </geometry>
       </visual>
+      <!--
       <collision>
+        <xacro:insert_block name="vis_coll_origin" />
         <geometry>
           <xacro:if value="${use_mesh_file}">
             <mesh filename="${mesh_file}"/>
           </xacro:if>
-          <!--
           <xacro:unless value="${use_mesh_file}">
             <cylinder length="0.005" radius="${propeller_radius}"/>
           </xacro:unless>
-          -->
         </geometry>
       </collision>
+      -->
     </link>
     <gazebo reference="${robot_namespace}/propeller_${suffix}">

File: rotors_description/urdf/techpod_X.xacro (robot description, xacro)
@@ -453,6 +453,7 @@
       <protocol_version>2.0</protocol_version>
       <imuSubTopic>/imu</imuSubTopic>
-      <imu_rate>100</imu_rate>
+      <imu_rate>250</imu_rate>
       <gpsSubTopic>/gps</gpsSubTopic>
+      <gpsGtSubTopic>/gps_gt</gpsGtSubTopic>
       <lidarSubTopic></lidarSubTopic>
       <opticalFlowSubTopic></opticalFlowSubTopic>
@@ -465,5 +466,5 @@
       <qgc_udp_port>14550</qgc_udp_port>
       <hil_mode>true</hil_mode>
-      <hil_state_level>true</hil_state_level>
+      <hil_state_level>false</hil_state_level>
       <enable_lockstep>false</enable_lockstep>
       <use_tcp>false</use_tcp>

File: rotors_description/urdf/techpod_X_base.xacro (robot description, xacro)
@@ -22,8 +22,12 @@
     <origin xyz="0 0 0" rpy="0 0 0" />
   </xacro:default_gps>
-  <!-- Mount a magnetometer. -->
+  <!-- Mount a magnetometer. note: mavlink interface already does this based on position from gps-->
+  <!--
   <xacro:default_magnetometer namespace="${namespace}" parent_link="${namespace}/base_link" />
-  <!-- Mount a pressure sensor. -->
+  -->
+  <!-- Mount a pressure sensor. note: mavlink interface already does this -->
+  <!--
   <xacro:default_pressure_sensor namespace="${namespace}" parent_link="${namespace}/base_link" />
+  -->
   <xacro:if value="$(arg enable_ground_truth)">
     <xacro:ground_truth_imu_and_odometry namespace="${namespace}" parent_link="${namespace}/base_link" />

File: rotors_description/urdf/techpod_X_flex.xacro (robot description, xacro)
@@ -1028,6 +1028,7 @@
       <protocol_version>2.0</protocol_version>
       <imuSubTopic>/imu</imuSubTopic>
-      <imu_rate>100</imu_rate>
+      <imu_rate>250</imu_rate>
       <gpsSubTopic>/gps</gpsSubTopic>
+      <gpsGtSubTopic>/gps_gt</gpsGtSubTopic>
       <lidarSubTopic></lidarSubTopic>
       <opticalFlowSubTopic></opticalFlowSubTopic>
@@ -1040,5 +1041,5 @@
       <qgc_udp_port>14550</qgc_udp_port>
       <hil_mode>true</hil_mode>
-      <hil_state_level>true</hil_state_level>
+      <hil_state_level>false</hil_state_level>
       <enable_lockstep>false</enable_lockstep>
       <use_tcp>false</use_tcp>

File: rotors_description/urdf/techpod_X_flex_base.xacro (robot description, xacro)
@@ -24,10 +24,12 @@
   </xacro:default_gps>
   <!-- -->
-  <!-- Mount a magnetometer. -->
+  <!-- Mount a magnetometer. note: mavlink interface already does this based on position from gps-->
+  <!--
   <xacro:default_magnetometer namespace="${namespace}" parent_link="${namespace}/base_link" />
-  <!-- -->
-  <!-- Mount a pressure sensor. -->
+  -->
+  <!-- Mount a pressure sensor. note: mavlink interface already does this -->
+  <!--
   <xacro:default_pressure_sensor namespace="${namespace}" parent_link="${namespace}/base_link" />
-  <!-- -->
+  -->
   <!--
   <xacro:if value="$(arg enable_ground_truth)">

Commit message: Turned out that the custom spring_damper plugin is not required after all (to simulate flexing wings using xacro/urdf)
- There are urdf <dynamics> and <springStiffness> tags that can be used to simulate spring-damper-like joints

File: rotors_description/urdf/fixed_wing_X_base.xacro (robot description, xacro)
@@ -66,4 +66,5 @@
     <child link="${robot_namespace}/${segment_name}"/>
     <limit upper="0.17" lower="-0.17" effort="5000" velocity="50"/>
+    <dynamics damping="${c}"/>
   </joint>
   <link name="${robot_namespace}/${segment_name}">
@@ -103,5 +104,7 @@
   <gazebo reference="${robot_namespace}/${segment_name}_joint">
     <implicitSpringDamper>true</implicitSpringDamper>
+    <springStiffness>${k}</springStiffness>
   </gazebo>
+  <!--
   <gazebo>
     <plugin filename="librotors_gazebo_springdamper_plugin.so" name="gazebo_springdamper_plugin">
@@ -112,4 +115,5 @@
     </plugin>
   </gazebo>
+  -->
 </xacro:macro>
   <!-- Control surface joint and link -->

Commit message: Adding functionality on simulator side for alpha/beta vanes
- Links, joints, aerodynamics
- To Do: Plugin to generate sensor readings (read joint angle and publish with some bias, noise etc.)

File: rotors_description/urdf/fixed_wing_X_base.xacro (robot description, xacro)
@@ -208,3 +208,87 @@
     </gazebo>
   </xacro:macro>
+<!-- Aerodyn. angle vane -->
+<xacro:macro name="angle_vane"
+  params="robot_namespace vane_name type chord arm_cp parent mass_vane
+          color mesh_file *joint_origin *vis_coll_origin *inertia">
+  <joint name="${robot_namespace}/${vane_name}_joint" type="continuous">
+    <xacro:insert_block name="joint_origin" />
+    <xacro:if value="${type=='alpha'}">
+       <axis xyz="0 1 0" />
+     </xacro:if>
+     <xacro:if value="${type=='beta'}">
+       <axis xyz="0 0 -1" />
+     </xacro:if>
+     <parent link="${parent}" />
+     <child link="${robot_namespace}/${vane_name}" />
+     <dynamics friction="0" damping="0.001"/>
+  </joint>
+  <link name="${robot_namespace}/${vane_name}">
+    <inertial>
+      <mass value="${mass_vane}" />
+      <xacro:insert_block name="inertia" />
+    </inertial>
+    <visual>
+      <xacro:insert_block name="vis_coll_origin" />
+      <geometry>
+        <box size="0.1 0.003 0.003" />
+      </geometry>
+    </visual>
+    <visual>
+      <xacro:if value="${type=='alpha'}">
+        <origin xyz="-0.04 0.02 0" rpy="0 0 0" />
+        <geometry>
+          <box size="0.02 0.04 0.002" />
+        </geometry>
+      </xacro:if>
+      <xacro:if value="${type=='beta'}">
+        <origin xyz="-0.04 0 0.02" rpy="0 0 0" />
+        <geometry>
+          <box size="0.02 0.002 0.04" />
+        </geometry>
+      </xacro:if>
+    </visual>
+  </link>
+  <gazebo reference="${robot_namespace}/${vane_name}">
+    <material>Gazebo/${color}</material>
+  </gazebo>
+  <xacro:if value="${type=='alpha'}">
+   <gazebo>
+     <plugin filename="librotors_gazebo_aerodynamics_plugin.so" name="aerodynamics_plugin">
+       <robotNamespace>${namespace}</robotNamespace>
+       <linkName>${robot_namespace}/${vane_name}</linkName>
+        <aeroForcesVis>aero_force_vis_${vane_name}</aeroForcesVis>
+        <airfoil>
+          <segment name="alpha_vane">
+            <forward>1 0 0</forward>
+            <upward>0 0 1</upward>
+            <cp>${-arm_cp} 0 0</cp>
+            <seg_area>${2*chord*chord}</seg_area>
+            <seg_chord>${chord}</seg_chord>
+            <aeroParamsYAML>${yaml_path}/airfoil_test_2.yaml</aeroParamsYAML>
+          </segment>
+        </airfoil>
+      </plugin>
+    </gazebo>
+  </xacro:if>
+  <xacro:if value="${type=='beta'}">
+   <gazebo>
+     <plugin filename="librotors_gazebo_aerodynamics_plugin.so" name="aerodynamics_plugin">
+       <robotNamespace>${namespace}</robotNamespace>
+       <linkName>${robot_namespace}/${vane_name}</linkName>
+        <aeroForcesVis>aero_force_vis_${vane_name}</aeroForcesVis>
+        <airfoil>
+          <segment name="beta_vane">
+            <forward>1 0 0</forward>
+            <upward>0 -1 0</upward>
+            <cp>${-arm_cp} 0 0</cp>
+            <seg_area>${2*chord*chord}</seg_area>
+            <seg_chord>${chord}</seg_chord>
+            <aeroParamsYAML>${yaml_path}/airfoil_test_2.yaml</aeroParamsYAML>
+          </segment>
+        </airfoil>
+      </plugin>
+    </gazebo>
+  </xacro:if>
+</xacro:macro>
 </robot>

File: rotors_description/urdf/techpod_X_flex.xacro (robot description, xacro)
@@ -258,4 +258,18 @@
   </plugin>
 </gazebo>
+  <xacro:angle_vane
+    robot_namespace="${namespace}"
+    vane_name="alpha_1"
+    type="alpha"
+    chord="0.02"
+    arm_cp="0.05"
+    mass_vane="0.02"
+    parent="${namespace}/wl_1"
+    color="Grey"
+    mesh_file="package://rotors_description/meshes/techpod_X_flex/flp_l_1.stl">
+    <origin xyz="0.15 0.35 0.05" rpy="0 0 0" />   <!-- Joint origin -->
+    <origin xyz="0 0 0" rpy="0 0 0" />       <!-- vis_coll origin -->
+    <xacro:box_inertia x="0.1" y="0.02" z="0.02" mass="0.02" />
+  </xacro:angle_vane>
 <xacro:airfoil_segment
   robot_namespace="${namespace}"
@@ -312,4 +326,18 @@
   </plugin>
 </gazebo>
+<xacro:angle_vane
+  robot_namespace="${namespace}"
+  vane_name="beta_1"
+  type="beta"
+  chord="0.02"
+  arm_cp="0.05"
+  mass_vane="0.02"
+  parent="${namespace}/wr_1"
+  color="Grey"
+  mesh_file="package://rotors_description/meshes/techpod_X_flex/flp_l_1.stl">
+  <origin xyz="0.15 -0.35 0.05" rpy="0 0 0" />   <!-- Joint origin -->
+  <origin xyz="0 0 0" rpy="0 0 0" />       <!-- vis_coll origin -->
+  <xacro:box_inertia x="0.1" y="0.02" z="0.02" mass="0.02" />
+</xacro:angle_vane>
 <xacro:airfoil_segment
   robot_namespace="${namespace}"

Commit message: Including new plugins in xacro/world files for testing
- Adding sample payload
- Adding "tracing ribbons" via visual plugin for illustration
- Aerodynamic angle vanes publishing their angle (joint state) to gazebo msg
- New base-link collision geometry to prevent interaction with payload

File: rotors_description/urdf/fixed_wing_X_base.xacro (robot description, xacro)
@@ -24,4 +24,10 @@
       iyy="${0.0833333 * mass * (3*r*r + h*h)}" iyz="0.0"
       izz="${0.5 * mass * r * r}" />
+  </xacro:macro>
+  <!-- Macro for the inertia of a cylinder -->
+  <xacro:macro name="sphere_inertia" params="r mass">
+    <inertia ixx="${0.4 * mass * r*r}" ixy="0.0" ixz="0.0"
+           iyy="${0.4 * mass * r*r}" iyz="0.0"
+           izz="${0.4 * mass * r*r}" />
   </xacro:macro>
   <!-- Fixed-wing main body link -->
@@ -85,5 +91,4 @@
       </geometry>
     </visual>
-    <!--
     <collision>
       <xacro:insert_block name="vis_coll_origin" />
@@ -97,5 +102,4 @@
       </geometry>
     </collision>
-    -->
   </link>
   <gazebo reference="${robot_namespace}/${segment_name}">

File: rotors_description/urdf/techpod_X_flex.xacro (robot description, xacro)
@@ -123,5 +123,5 @@
     mass="${mass_fuselage}"
     length="${body_length}"
-    width="${body_width}"
+    width="0.2"
     height="${body_height}"
     color="${body_color}"
@@ -223,4 +223,61 @@
     <xacro:insert_block name="aileron_inertia" />
   </xacro:airfoil_segment>
+<gazebo reference="${namespace}/base_link">
+  <visual>
+    <plugin name='visual_plugin_base_link' filename='librotors_gazebo_template_visual_plugin.so'/>
+  </visual>
+</gazebo>
+<link name="${namespace}/payload_1">
+  <inertial>
+    <mass value="0.5" />
+    <xacro:sphere_inertia r="0.05" mass="0.5" />
+  </inertial>
+  <visual>
+    <origin xyz="0 0 0" rpy="0 1.5708 0" />
+    <geometry>
+        <cylinder length="0.25" radius="0.03"/>
+    </geometry>
+  </visual>
+  <collision>
+    <origin xyz="0 0 0" rpy="0 1.5708 0" />
+    <geometry>
+        <cylinder length="0.25" radius="0.03"/>
+    </geometry>
+  </collision>
+</link>
+<!--
+<joint name="${namespace}/payload_1_joint" type="revolute">
+  <parent link="${namespace}/wl_2" />
+  <child link="${namespace}/payload_1" />
+  <origin xyz="0.05 0 -0.1" rpy="0 0 0" />
+  <limit upper="0" lower="0" effort="5000" velocity="50"/>
+</joint>
+-->
+<joint name="${namespace}/payload_1_joint" type="floating">
+  <parent link="${namespace}/wl_2" />
+  <child link="${namespace}/payload_1" />
+  <origin xyz="0.05 0 -0.1" rpy="0 0 0" />
+</joint>
+<gazebo reference="${namespace}/payload_1">
+  <visual>
+    <plugin name='visual_plugin_payload_1' filename='librotors_gazebo_template_visual_plugin.so'/>
+  </visual>
+  <material>Gazebo/Orange</material>
+  <mu1>0.2</mu1>
+  <mu2>0.2</mu2>
+  <kp>10000</kp>
+  <kd>1</kd>
+</gazebo>
+<gazebo>
+  <plugin filename="librotors_gazebo_payload_plugin.so" name="payload_plugin_1">
+    <robotNamespace>${namespace}</robotNamespace>
+    <joint>${namespace}/payload_1_joint</joint>
+    <payload>${namespace}/payload_1</payload>
+    <parent>${namespace}/wl_2</parent>
+    <hoistPosParent>0 -0.15 -0.07</hoistPosParent>
+    <hoistPosPayload>0 0 0</hoistPosPayload>
+    <dropTopic>drop_1</dropTopic>
+  </plugin>
+</gazebo>
 <gazebo>
   <plugin filename="librotors_gazebo_aerodynamics_plugin.so" name="aerodynamics_plugin">
@@ -272,4 +329,11 @@
     <xacro:box_inertia x="0.1" y="0.02" z="0.02" mass="0.02" />
   </xacro:angle_vane>
+<gazebo>
+  <plugin filename="librotors_gazebo_vane_plugin.so" name="alpha_1_vane_plugin">
+    <robotNamespace>${namespace}</robotNamespace>
+    <vaneJoint>${namespace}/alpha_1_joint</vaneJoint>
+    <vaneTopic>alpha_1_vane_sensor</vaneTopic>
+  </plugin>
+</gazebo>
 <xacro:airfoil_segment
   robot_namespace="${namespace}"
@@ -340,4 +404,11 @@
   <xacro:box_inertia x="0.1" y="0.02" z="0.02" mass="0.02" />
 </xacro:angle_vane>
+<gazebo>
+  <plugin filename="librotors_gazebo_vane_plugin.so" name="beta_1_vane_plugin">
+    <robotNamespace>${namespace}</robotNamespace>
+    <vaneJoint>${namespace}/beta_1_joint</vaneJoint>
+    <vaneTopic>beta_1_vane_sensor</vaneTopic>
+  </plugin>
+</gazebo>
 <xacro:airfoil_segment
   robot_namespace="${namespace}"
@@ -1173,4 +1244,13 @@
         <gztopic>flap_r2_pos</gztopic>
       </channel>
+      <channel name="payload">
+        <input_index>5</input_index>
+        <input_offset>0</input_offset>
+        <input_scaling>1</input_scaling>
+        <zero_position_disarmed>0</zero_position_disarmed>
+        <zero_position_armed>0</zero_position_armed>
+        <joint_control_type>gz_msg</joint_control_type>
+        <gztopic>drop_1</gztopic>
+      </channel>
     </control_channels>
   </plugin>
