Commit message: Including wind tags in multiple .xacros
- Telling airfoil segments, bodies and propulsion units to watch out for wind...
- Alpha-/Beta vanes also affected by wind
- Adding wind-field *.csvs to test parsing and loading of 3D wind fields (e.g. ones generated by CFD)

File: rotors_description/urdf/fixed_wing_X_base.xacro (robot description, xacro)
@@ -215,5 +215,5 @@
 <!-- Aerodyn. angle vane -->
 <xacro:macro name="angle_vane"
-  params="robot_namespace vane_name type chord arm_cp parent mass_vane
+  params="robot_namespace vane_name type chord arm_cp parent wind_topic mass_vane
           color mesh_file *joint_origin *vis_coll_origin *inertia">
   <joint name="${robot_namespace}/${vane_name}_joint" type="continuous">
@@ -272,4 +272,7 @@
             <seg_chord>${chord}</seg_chord>
             <aeroParamsYAML>${yaml_path}/airfoil_test_2.yaml</aeroParamsYAML>
+            <wind name="wind">
+              <topic>${wind_topic}</topic>
+            </wind>
           </segment>
         </airfoil>
@@ -291,4 +294,7 @@
             <seg_chord>${chord}</seg_chord>
             <aeroParamsYAML>${yaml_path}/airfoil_test_2.yaml</aeroParamsYAML>
+            <wind name="wind">
+              <topic>${wind_topic}</topic>
+            </wind>
           </segment>
         </airfoil>

File: rotors_description/urdf/techpod_TJ.xacro (robot description, xacro)
@@ -254,4 +254,34 @@
   -->
   <gazebo>
+    <plugin filename="librotors_gazebo_wind_beta_plugin.so" name="wind_beta_plugin">
+      <robotNamespace>${namespace}</robotNamespace>
+      <windLayer>
+        <layer name="layer1">
+          <altitude>10</altitude>
+          <windMeanNED>-5 0 0</windMeanNED>
+        </layer>
+        <layer name="layer2">
+          <altitude>25</altitude>
+          <windMeanNED>-6 0 0</windMeanNED>
+        </layer>
+        <layer name="layer3">
+          <altitude>35</altitude>
+          <windMeanNED>-10 0 0</windMeanNED>
+        </layer>
+      </windLayer>
+      <findWind>
+        <query name="q1">
+          <linkName>${namespace}/base_link</linkName>
+          <windTopic>wind_base_link</windTopic>
+        </query>
+      </findWind>
+      <lambdaMin>10</lambdaMin>
+      <lengthScale>725</lengthScale>
+      <fourierNNN>10 10 10</fourierNNN>
+      <sigma>5</sigma>
+      <trnspVelTurbNED>5 0 0</trnspVelTurbNED>
+    </plugin>
+  </gazebo>
+  <gazebo>
     <plugin filename="librotors_gazebo_propulsion_plugin.so" name="propulsion_plugin">
       <robotNamespace>${namespace}</robotNamespace>
@@ -266,4 +296,7 @@
         <slpstrTopic>prop_slpstr_0</slpstrTopic>
         <visTopic>prop_vis_0</visTopic>
+        <wind name="wind">
+          <topic>wind_base_link</topic>
+        </wind>
       </prop>
     </plugin>
@@ -282,4 +315,7 @@
           <upward>0 0 1</upward>
           <cp>0.16 0.0 0.05</cp>
+          <wind name="wind">
+            <topic>wind_base_link</topic>
+          </wind>
         </element>
       </body>
@@ -292,4 +328,7 @@
           <seg_chord>0.194</seg_chord>
           <aeroParamsYAML>${yaml_path}/techpod_TJ_wing.yaml</aeroParamsYAML>
+          <wind name="wind">
+            <topic>wind_base_link</topic>
+          </wind>
         </segment>
         <segment name="WL2">
@@ -300,4 +339,7 @@
           <seg_chord>0.183</seg_chord>
           <aeroParamsYAML>${yaml_path}/techpod_TJ_wing.yaml</aeroParamsYAML>
+          <wind name="wind">
+            <topic>wind_base_link</topic>
+          </wind>
           <control>
             <cs name="flap_left">
@@ -317,4 +359,7 @@
           <seg_chord>0.170</seg_chord>
           <aeroParamsYAML>${yaml_path}/techpod_TJ_wing.yaml</aeroParamsYAML>
+          <wind name="wind">
+            <topic>wind_base_link</topic>
+          </wind>
           <control>
             <cs name="flap_left">
@@ -334,4 +379,7 @@
           <seg_chord>0.157</seg_chord>
           <aeroParamsYAML>${yaml_path}/techpod_TJ_wing.yaml</aeroParamsYAML>
+          <wind name="wind">
+            <topic>wind_base_link</topic>
+          </wind>
         </segment>
         <segment name="WL5">
@@ -342,4 +390,7 @@
           <seg_chord>0.146</seg_chord>
           <aeroParamsYAML>${yaml_path}/techpod_TJ_wing.yaml</aeroParamsYAML>
+          <wind name="wind">
+            <topic>wind_base_link</topic>
+          </wind>
           <control>
             <cs name="aileron_left">
@@ -359,4 +410,7 @@
           <seg_chord>0.136</seg_chord>
           <aeroParamsYAML>${yaml_path}/techpod_TJ_wing.yaml</aeroParamsYAML>
+          <wind name="wind">
+            <topic>wind_base_link</topic>
+          </wind>
           <control>
             <cs name="aileron_left">
@@ -376,4 +430,7 @@
           <seg_chord>0.127</seg_chord>
           <aeroParamsYAML>${yaml_path}/techpod_TJ_wing.yaml</aeroParamsYAML>
+          <wind name="wind">
+            <topic>wind_base_link</topic>
+          </wind>
         </segment>
         <segment name="WR1">
@@ -384,4 +441,7 @@
           <seg_chord>0.194</seg_chord>
           <aeroParamsYAML>${yaml_path}/techpod_TJ_wing.yaml</aeroParamsYAML>
+          <wind name="wind">
+            <topic>wind_base_link</topic>
+          </wind>
         </segment>
         <segment name="WR2">
@@ -392,4 +452,7 @@
           <seg_chord>0.183</seg_chord>
           <aeroParamsYAML>${yaml_path}/techpod_TJ_wing.yaml</aeroParamsYAML>
+          <wind name="wind">
+            <topic>wind_base_link</topic>
+          </wind>
           <control>
             <cs name="flap_right">
@@ -409,4 +472,7 @@
           <seg_chord>0.170</seg_chord>
           <aeroParamsYAML>${yaml_path}/techpod_TJ_wing.yaml</aeroParamsYAML>
+          <wind name="wind">
+            <topic>wind_base_link</topic>
+          </wind>
           <control>
             <cs name="flap_right">
@@ -426,4 +492,7 @@
           <seg_chord>0.157</seg_chord>
           <aeroParamsYAML>${yaml_path}/techpod_TJ_wing.yaml</aeroParamsYAML>
+          <wind name="wind">
+            <topic>wind_base_link</topic>
+          </wind>
         </segment>
         <segment name="WR5">
@@ -434,4 +503,7 @@
           <seg_chord>0.146</seg_chord>
           <aeroParamsYAML>${yaml_path}/techpod_TJ_wing.yaml</aeroParamsYAML>
+          <wind name="wind">
+            <topic>wind_base_link</topic>
+          </wind>
           <control>
             <cs name="aileron_right">
@@ -451,4 +523,7 @@
           <seg_chord>0.136</seg_chord>
           <aeroParamsYAML>${yaml_path}/techpod_TJ_wing.yaml</aeroParamsYAML>
+          <wind name="wind">
+            <topic>wind_base_link</topic>
+          </wind>
           <control>
             <cs name="aileron_right">
@@ -468,4 +543,7 @@
           <seg_chord>0.127</seg_chord>
           <aeroParamsYAML>${yaml_path}/techpod_TJ_wing.yaml</aeroParamsYAML>
+          <wind name="wind">
+            <topic>wind_base_link</topic>
+          </wind>
         </segment>
         <segment name="EL1">
@@ -479,4 +557,7 @@
             <topic>prop_slpstr_0</topic>
           </indVel>
+          <wind name="wind">
+            <topic>wind_base_link</topic>
+          </wind>
           <control>
             <cs name="elevator_left">
@@ -499,4 +580,7 @@
             <topic>prop_slpstr_0</topic>
           </indVel>
+          <wind name="wind">
+            <topic>wind_base_link</topic>
+          </wind>
           <control>
             <cs name="elevator_right">
@@ -519,4 +603,7 @@
             <topic>prop_slpstr_0</topic>
           </indVel>
+          <wind name="wind">
+            <topic>wind_base_link</topic>
+          </wind>
           <control>
             <cs name="rudder">

File: rotors_description/urdf/techpod_X.xacro (robot description, xacro)
@@ -246,4 +246,41 @@
   </xacro:propeller>
   <gazebo>
+    <plugin filename="librotors_gazebo_wind_beta_plugin.so" name="wind_beta_plugin">
+      <robotNamespace>${namespace}</robotNamespace>
+      <windLayer>
+        <layer name="layer1">
+          <altitude>10</altitude>
+          <windMeanNED>-5 0 0</windMeanNED>
+        </layer>
+        <layer name="layer2">
+          <altitude>25</altitude>
+          <windMeanNED>-6 0 0</windMeanNED>
+        </layer>
+        <layer name="layer3">
+          <altitude>35</altitude>
+          <windMeanNED>-10 0 0</windMeanNED>
+        </layer>
+      </windLayer>
+      <!---->
+      <findWind>
+        <query name="q1">
+          <linkName>${namespace}/base_link</linkName>
+          <windTopic>wind_base_link</windTopic>
+        </query>
+      </findWind>
+      <!--
+      <customWindFieldPath>${yaml_path}/../test_wind_field.csv</customWindFieldPath>
+      <windFieldXOffset>100</windFieldXOffset>
+      <windFieldYOffset>100</windFieldYOffset>
+      <windFieldZOffset>0</windFieldZOffset>
+      -->
+      <lambdaMin>10</lambdaMin>
+      <lengthScale>725</lengthScale>
+      <fourierNNN>7 7 7</fourierNNN>
+      <sigma>2</sigma>
+      <trnspVelTurbNED>5 0 0</trnspVelTurbNED>
+    </plugin>
+  </gazebo>
+  <gazebo>
     <plugin filename="librotors_gazebo_propulsion_plugin.so" name="propulsion_plugin">
       <robotNamespace>${namespace}</robotNamespace>
@@ -258,4 +295,7 @@
         <slpstrTopic>prop_slpstr_0</slpstrTopic>
         <visTopic>prop_vis_0</visTopic>
+        <wind name="wind">
+          <topic>wind_base_link</topic>
+        </wind>
       </prop>
     </plugin>
@@ -274,4 +314,7 @@
           <upward>0 0 1</upward>
           <cp>0.2 0.0 0.05</cp>
+          <wind name="wind">
+            <topic>wind_base_link</topic>
+          </wind>
         </element>
       </body>
@@ -284,4 +327,7 @@
           <seg_chord>0.16</seg_chord>
           <aeroParamsYAML>${yaml_path}/airfoil_test.yaml</aeroParamsYAML>
+          <wind name="wind">
+            <topic>wind_base_link</topic>
+          </wind>
         </segment>
         <segment name="WL2">
@@ -292,4 +338,7 @@
           <seg_chord>0.16</seg_chord>
           <aeroParamsYAML>${yaml_path}/airfoil_test.yaml</aeroParamsYAML>
+          <wind name="wind">
+            <topic>wind_base_link</topic>
+          </wind>
           <control>
             <cs name="flap_left">
@@ -308,4 +357,7 @@
           <seg_chord>0.16</seg_chord>
           <aeroParamsYAML>${yaml_path}/airfoil_test.yaml</aeroParamsYAML>
+          <wind name="wind">
+            <topic>wind_base_link</topic>
+          </wind>
         </segment>
         <segment name="WL4">
@@ -316,4 +368,7 @@
           <seg_chord>0.16</seg_chord>
           <aeroParamsYAML>${yaml_path}/airfoil_test.yaml</aeroParamsYAML>
+          <wind name="wind">
+            <topic>wind_base_link</topic>
+          </wind>
           <control>
             <cs name="aileron_left">
@@ -332,4 +387,7 @@
           <seg_chord>0.16</seg_chord>
           <aeroParamsYAML>${yaml_path}/airfoil_test.yaml</aeroParamsYAML>
+          <wind name="wind">
+            <topic>wind_base_link</topic>
+          </wind>
         </segment>
         <segment name="WR1">
@@ -340,4 +398,7 @@
           <seg_chord>0.16</seg_chord>
           <aeroParamsYAML>${yaml_path}/airfoil_test.yaml</aeroParamsYAML>
+          <wind name="wind">
+            <topic>wind_base_link</topic>
+          </wind>
         </segment>
         <segment name="WR2">
@@ -348,4 +409,7 @@
           <seg_chord>0.16</seg_chord>
           <aeroParamsYAML>${yaml_path}/airfoil_test.yaml</aeroParamsYAML>
+          <wind name="wind">
+            <topic>wind_base_link</topic>
+          </wind>
           <control>
             <cs name="flap_right">
@@ -364,4 +428,7 @@
           <seg_chord>0.16</seg_chord>
           <aeroParamsYAML>${yaml_path}/airfoil_test.yaml</aeroParamsYAML>
+          <wind name="wind">
+            <topic>wind_base_link</topic>
+          </wind>
         </segment>
         <segment name="WR4">
@@ -372,4 +439,7 @@
           <seg_chord>0.16</seg_chord>
           <aeroParamsYAML>${yaml_path}/airfoil_test.yaml</aeroParamsYAML>
+          <wind name="wind">
+            <topic>wind_base_link</topic>
+          </wind>
           <control>
             <cs name="aileron_right">
@@ -388,4 +458,7 @@
           <seg_chord>0.16</seg_chord>
           <aeroParamsYAML>${yaml_path}/airfoil_test.yaml</aeroParamsYAML>
+          <wind name="wind">
+            <topic>wind_base_link</topic>
+          </wind>
         </segment>
         <segment name="EL1">
@@ -399,4 +472,7 @@
             <topic>prop_slpstr_0</topic>
           </indVel>
+          <wind name="wind">
+            <topic>wind_base_link</topic>
+          </wind>
           <control>
             <cs name="elevator_left">
@@ -418,4 +494,7 @@
             <topic>prop_slpstr_0</topic>
           </indVel>
+          <wind name="wind">
+            <topic>wind_base_link</topic>
+          </wind>
           <control>
             <cs name="elevator_right">
@@ -437,4 +516,7 @@
             <topic>prop_slpstr_0</topic>
           </indVel>
+          <wind name="wind">
+            <topic>wind_base_link</topic>
+          </wind>
           <control>
             <cs name="rudder">
@@ -448,4 +530,9 @@
       </airfoil>
     </plugin>
+  </gazebo>
+  <gazebo reference="${namespace}/base_link">
+     <visual>
+        <plugin name="visual_plugin_base_link" filename="librotors_gazebo_template_visual_plugin.so" />
+     </visual>
   </gazebo>
   <gazebo>

File: rotors_description/urdf/techpod_X_flex.xacro (robot description, xacro)
@@ -228,4 +228,7 @@
                <seg_chord>0.16</seg_chord>
                <aeroParamsYAML>${yaml_path}/airfoil_test.yaml</aeroParamsYAML>
+               <wind name="wind">
+                 <topic>wind_base_link</topic>
+               </wind>
             </segment>
             <segment name="WL1_2">
@@ -236,4 +239,7 @@
                <seg_chord>0.16</seg_chord>
                <aeroParamsYAML>${yaml_path}/airfoil_test.yaml</aeroParamsYAML>
+               <wind name="wind">
+                 <topic>wind_base_link</topic>
+               </wind>
                <control>
                   <cs name="flap_left">
@@ -282,4 +288,7 @@
                <seg_chord>0.16</seg_chord>
                <aeroParamsYAML>${yaml_path}/airfoil_test.yaml</aeroParamsYAML>
+               <wind name="wind">
+                 <topic>wind_base_link</topic>
+               </wind>
             </segment>
             <segment name="WR1_2">
@@ -290,4 +299,7 @@
                <seg_chord>0.16</seg_chord>
                <aeroParamsYAML>${yaml_path}/airfoil_test.yaml</aeroParamsYAML>
+               <wind name="wind">
+                 <topic>wind_base_link</topic>
+               </wind>
                <control>
                   <cs name="flap_right">
@@ -336,4 +348,7 @@
                <seg_chord>0.16</seg_chord>
                <aeroParamsYAML>${yaml_path}/airfoil_test.yaml</aeroParamsYAML>
+               <wind name="wind">
+                 <topic>wind_base_link</topic>
+               </wind>
                <control>
                   <cs name="flap_left">
@@ -354,4 +369,7 @@
                <seg_chord>0.16</seg_chord>
                <aeroParamsYAML>${yaml_path}/airfoil_test.yaml</aeroParamsYAML>
+               <wind name="wind">
+                 <topic>wind_base_link</topic>
+               </wind>
             </segment>
          </airfoil>
@@ -390,4 +408,7 @@
                <seg_chord>0.16</seg_chord>
                <aeroParamsYAML>${yaml_path}/airfoil_test.yaml</aeroParamsYAML>
+               <wind name="wind">
+                 <topic>wind_base_link</topic>
+               </wind>
                <control>
                   <cs name="flap_right">
@@ -408,4 +429,7 @@
                <seg_chord>0.16</seg_chord>
                <aeroParamsYAML>${yaml_path}/airfoil_test.yaml</aeroParamsYAML>
+               <wind name="wind">
+                 <topic>wind_base_link</topic>
+               </wind>
             </segment>
          </airfoil>
@@ -444,4 +468,7 @@
                <seg_chord>0.16</seg_chord>
                <aeroParamsYAML>${yaml_path}/airfoil_test.yaml</aeroParamsYAML>
+               <wind name="wind">
+                 <topic>wind_base_link</topic>
+               </wind>
                <control>
                   <cs name="aileron_left">
@@ -462,4 +489,7 @@
                <seg_chord>0.16</seg_chord>
                <aeroParamsYAML>${yaml_path}/airfoil_test.yaml</aeroParamsYAML>
+               <wind name="wind">
+                 <topic>wind_base_link</topic>
+               </wind>
             </segment>
          </airfoil>
@@ -498,4 +528,7 @@
                <seg_chord>0.16</seg_chord>
                <aeroParamsYAML>${yaml_path}/airfoil_test.yaml</aeroParamsYAML>
+               <wind name="wind">
+                 <topic>wind_base_link</topic>
+               </wind>
                <control>
                   <cs name="aileron_right">
@@ -516,4 +549,7 @@
                <seg_chord>0.16</seg_chord>
                <aeroParamsYAML>${yaml_path}/airfoil_test.yaml</aeroParamsYAML>
+               <wind name="wind">
+                 <topic>wind_base_link</topic>
+               </wind>
             </segment>
          </airfoil>
@@ -552,4 +588,7 @@
                <seg_chord>0.12</seg_chord>
                <aeroParamsYAML>${yaml_path}/airfoil_test_2.yaml</aeroParamsYAML>
+               <wind name="wind">
+                 <topic>wind_base_link</topic>
+               </wind>
                <indVel name="prop0">
                   <topic>prop_slpstr_0</topic>
@@ -601,4 +640,7 @@
                <seg_chord>0.12</seg_chord>
                <aeroParamsYAML>${yaml_path}/airfoil_test_2.yaml</aeroParamsYAML>
+               <wind name="wind">
+                 <topic>wind_base_link</topic>
+               </wind>
                <indVel name="prop0">
                   <topic>prop_slpstr_0</topic>
@@ -622,4 +664,7 @@
                <seg_chord>0.12</seg_chord>
                <aeroParamsYAML>${yaml_path}/airfoil_test_2.yaml</aeroParamsYAML>
+               <wind name="wind">
+                 <topic>wind_base_link</topic>
+               </wind>
                <indVel name="prop0">
                   <topic>prop_slpstr_0</topic>
@@ -811,4 +856,7 @@
             <slpstrTopic>prop_slpstr_0</slpstrTopic>
             <visTopic>prop_vis_0</visTopic>
+            <wind name="wind">
+              <topic>wind_base_link</topic>
+            </wind>
          </prop>
       </plugin>
@@ -828,4 +876,7 @@
                <upward>0 0 1</upward>
                <cp>0.2 0.0 0.05</cp>
+               <wind name="wind">
+                 <topic>wind_base_link</topic>
+               </wind>
             </element>
          </body>
@@ -840,4 +891,5 @@
       mass_vane="0.02"
       parent="${namespace}/wl_1"
+      wind_topic="wind_base_link"
       color="Grey"
       mesh_file="package://rotors_description/meshes/techpod_X_flex/flp_l_1.stl">
@@ -860,4 +912,5 @@
       mass_vane="0.02"
       parent="${namespace}/wr_1"
+      wind_topic="wind_base_link"
       color="Grey"
       mesh_file="package://rotors_description/meshes/techpod_X_flex/flp_l_1.stl">
@@ -873,6 +926,41 @@
       </plugin>
    </gazebo>
+   <gazebo>
+     <plugin filename="librotors_gazebo_wind_beta_plugin.so" name="wind_beta_plugin">
+       <robotNamespace>${namespace}</robotNamespace>
+       <windLayer>
+         <layer name="layer1">
+           <altitude>10</altitude>
+           <windMeanNED>-5 0 0</windMeanNED>
+         </layer>
+         <layer name="layer2">
+           <altitude>25</altitude>
+           <windMeanNED>-6 0 0</windMeanNED>
+         </layer>
+         <layer name="layer3">
+           <altitude>35</altitude>
+           <windMeanNED>-10 0 0</windMeanNED>
+         </layer>
+       </windLayer>
+       <findWind>
+         <query name="q1">
+           <linkName>${namespace}/base_link</linkName>
+           <windTopic>wind_base_link</windTopic>
+         </query>
+         <!--
+         <query name="q2">
+           <linkName>${namespace}/payload_1</linkName>
+           <windTopic>wind_payload</windTopic>
+         </query>
+         -->
+       </findWind>
+       <lambdaMin>2</lambdaMin>
+       <lengthScale>725</lengthScale>
+       <fourierNNN>10 10 10</fourierNNN>
+       <sigma>5</sigma>
+       <trnspVelTurbNED>-5 0 0</trnspVelTurbNED>
+     </plugin>
+   </gazebo>
    <!-- Tracing ribbon/Visual plugin -->
-   <!--
    <gazebo reference="${namespace}/base_link">
       <visual>
@@ -880,5 +968,5 @@
       </visual>
    </gazebo>
-   -->
+   <!---->
    <!-- Payload -->
    <!--
@@ -941,4 +1029,7 @@
                <seg_chord>0.05</seg_chord>
                <aeroParamsYAML>${yaml_path}/airfoil_test_2.yaml</aeroParamsYAML>
+               <wind name="wind">
+                 <topic>wind_payload</topic>
+               </wind>
             </segment>
             <segment name="VS">
@@ -949,4 +1040,7 @@
                <seg_chord>0.05</seg_chord>
                <aeroParamsYAML>${yaml_path}/airfoil_test_2.yaml</aeroParamsYAML>
+               <wind name="wind">
+                 <topic>wind_payload</topic>
+               </wind>
             </segment>
          </airfoil>
@@ -959,4 +1053,7 @@
                <upward>0 0 1</upward>
                <cp>-0.05 0.0 0</cp>
+               <wind name="wind">
+                 <topic>wind_payload</topic>
+               </wind>
             </element>
          </body>
