Commit message: TJ TechPod version used for Marko 12.08.19

File: rotors_description/urdf/techpod_TJ.xacro (robot description, xacro)
@@ -76,5 +76,5 @@
   <!-- Inertia of the main body -->
   <xacro:property name="body_inertia">
-    <inertia ixx="0.6688" ixy="0.0" ixz="-0.32112" iyy="0.16235" iyz="0.0" izz="0.69364" />
+    <inertia ixx="0.6688" ixy="0.0" ixz="0.0" iyy="0.16235" iyz="0.0" izz="0.69364" />
   </xacro:property>
   <!-- Inertia of the aileron, assuming it is a cuboid -->
@@ -251,6 +251,6 @@
         <jointName>${namespace}/propeller_P0_joint</jointName>
         <linkNameParent>${namespace}/base_link</linkNameParent>
-        <cp>0 0 0.15</cp>
-        <axisPosRot>-1 0 0.035</axisPosRot>
+        <cp>0 0 0.05</cp>
+        <axisPosRot>-1 0 0</axisPosRot>
         <turnDir>cw</turnDir>
         <speedRefTopic>prop_ref_0</speedRefTopic>
@@ -474,5 +474,5 @@
             <cs name="elevator_left">
                 <controlJoint>${namespace}/elevator_joint</controlJoint>
-                <radToCLift>1.2322 0</radToCLift>
+                <radToCLift>1.15 0</radToCLift>
                 <radToCDrag>0 0</radToCDrag>
                 <radToCPitch>0 0</radToCPitch>
@@ -494,5 +494,5 @@
             <cs name="elevator_right">
                 <controlJoint>${namespace}/elevator_joint</controlJoint>
-                <radToCLift>1.2322 0</radToCLift>
+                <radToCLift>1.15 0</radToCLift>
                 <radToCDrag>0 0</radToCDrag>
                 <radToCPitch>0 0</radToCPitch>

Commit message: Major fix of propulsion plugin - center of pressure was wrongly defined relative to cg instead of link frame...

File: rotors_description/urdf/techpod_TJ.xacro (robot description, xacro)
@@ -19,4 +19,5 @@
   <xacro:property name="yaml_path" value="$(arg yaml_path)"/>
   <xacro:property name="serial_device" value="$(arg serial_device)" />
+  <xacro:property name="main_color" value="Orange"/>
   <!-- Constants -->
   <xacro:property name="PI" value="3.1415926535897931" />
@@ -32,5 +33,5 @@
   <xacro:property name="body_width" value="2.591" /> <!-- [m] -->
   <xacro:property name="body_height" value="0.303" /> <!-- [m] -->
-  <xacro:property name="body_color" value="White" />
+  <xacro:property name="body_color" value="${main_color}" />
   <xacro:property name="body_mesh_file" value="package://rotors_description/meshes/techpod/techpod_body.dae" />
   <!-- Aileron properties -->
@@ -40,5 +41,5 @@
   <xacro:property name="aileron_min_angle" value="-0.349066" /> <!-- [rad] -->
   <xacro:property name="aileron_max_angle" value="0.349066" /> <!-- [rad] -->
-  <xacro:property name="aileron_color" value="White" />
+  <xacro:property name="aileron_color" value="${main_color}" />
   <xacro:property name="aileron_left_mesh_file" value="package://rotors_description/meshes/techpod/techpod_aileron_left.dae" />
   <xacro:property name="aileron_right_mesh_file" value="package://rotors_description/meshes/techpod/techpod_aileron_right.dae" />
@@ -49,5 +50,5 @@
   <xacro:property name="elevator_min_angle" value="-0.349066" /> <!-- [rad] -->
   <xacro:property name="elevator_max_angle" value="0.349066" /> <!-- [rad] -->
-  <xacro:property name="elevator_color" value="White" />
+  <xacro:property name="elevator_color" value="${main_color}" />
   <xacro:property name="elevator_mesh_file" value="package://rotors_description/meshes/techpod/techpod_elevator.dae" />
   <!-- Flap properties -->
@@ -57,5 +58,5 @@
   <xacro:property name="flap_min_angle" value="-0.349066" /> <!-- [rad] -->
   <xacro:property name="flap_max_angle" value="0.349066" /> <!-- [rad] -->
-  <xacro:property name="flap_color" value="White" />
+  <xacro:property name="flap_color" value="${main_color}" />
   <xacro:property name="flap_left_mesh_file" value="package://rotors_description/meshes/techpod/techpod_flap_left.dae" />
   <xacro:property name="flap_right_mesh_file" value="package://rotors_description/meshes/techpod/techpod_flap_right.dae" />
@@ -66,5 +67,5 @@
   <xacro:property name="rudder_min_angle" value="-0.349066" />
   <xacro:property name="rudder_max_angle" value="0.349066" />
-  <xacro:property name="rudder_color" value="White" />
+  <xacro:property name="rudder_color" value="${main_color}" />
   <xacro:property name="rudder_mesh_file" value="package://rotors_description/meshes/techpod/techpod_rudder.dae" />
   <!-- Propeller properties -->
@@ -110,5 +111,5 @@
     use_mesh_file="${use_mesh}"
     mesh_file="${body_mesh_file}">
-    <origin xyz="0.16 0 0.05" rpy="0 0 0" />
+    <origin xyz="0.16 0 0.10" rpy="0 0 0" />
     <xacro:insert_block name="body_inertia" />
   </xacro:fixed_wing_base_macro>
@@ -245,4 +246,10 @@
     <xacro:insert_block name="propeller_inertia" />
   </xacro:propeller>
+<!-- Tracing ribbon/Visual plugin -->
+<gazebo reference="${namespace}/base_link">
+   <visual>
+      <plugin name="visual_plugin_base_link" filename="librotors_gazebo_template_visual_plugin.so" />
+   </visual>
+</gazebo>
   <gazebo>
     <plugin filename="librotors_gazebo_propulsion_plugin.so" name="propulsion_plugin">
@@ -251,5 +258,5 @@
         <jointName>${namespace}/propeller_P0_joint</jointName>
         <linkNameParent>${namespace}/base_link</linkNameParent>
-        <cp>0 0 0.05</cp>
+        <cp>0 0 0.15</cp>
         <axisPosRot>-1 0 0</axisPosRot>
         <turnDir>cw</turnDir>

Commit message: Techpod_TJ xacro cleanup

File: rotors_description/urdf/techpod_TJ.xacro (robot description, xacro)
@@ -19,5 +19,5 @@
   <xacro:property name="yaml_path" value="$(arg yaml_path)"/>
   <xacro:property name="serial_device" value="$(arg serial_device)" />
-  <xacro:property name="main_color" value="Orange"/>
+  <xacro:property name="main_color" value="White"/>
   <!-- Constants -->
   <xacro:property name="PI" value="3.1415926535897931" />
@@ -246,10 +246,11 @@
     <xacro:insert_block name="propeller_inertia" />
   </xacro:propeller>
-<!-- Tracing ribbon/Visual plugin -->
-<gazebo reference="${namespace}/base_link">
-   <visual>
-      <plugin name="visual_plugin_base_link" filename="librotors_gazebo_template_visual_plugin.so" />
-   </visual>
-</gazebo>
+  <!-- Tracing ribbon/Visual plugin
+  <gazebo reference="${namespace}/base_link">
+     <visual>
+        <plugin name="visual_plugin_base_link" filename="librotors_gazebo_template_visual_plugin.so" />
+     </visual>
+  </gazebo>
+  -->
   <gazebo>
     <plugin filename="librotors_gazebo_propulsion_plugin.so" name="propulsion_plugin">
@@ -376,96 +377,96 @@
           <aeroParamsYAML>${yaml_path}/techpod_TJ_wing.yaml</aeroParamsYAML>
         </segment>
-  <segment name="WR1">
-    <forward>1 0 0</forward>
-    <upward>0 0 1</upward>
-    <cp>0.175 -0.075 0.115</cp>
-    <seg_area>0.029</seg_area>
-    <seg_chord>0.194</seg_chord>
-    <aeroParamsYAML>${yaml_path}/techpod_TJ_wing.yaml</aeroParamsYAML>
-  </segment>
-  <segment name="WR2">
-    <forward>1 0 0</forward>
-    <upward>0 0 1</upward>
-    <cp>0.172 -0.265 0.115</cp>
-    <seg_area>0.042</seg_area>
-    <seg_chord>0.183</seg_chord>
-    <aeroParamsYAML>${yaml_path}/techpod_TJ_wing.yaml</aeroParamsYAML>
-    <control>
-      <cs name="flap_right">
-          <controlJoint>${namespace}/flap_right_joint</controlJoint>
-          <radToCLift>1.6067 0</radToCLift>
-          <radToCDrag>0.1438 0.8227</radToCDrag>
-          <radToCPitch>0.0898 0</radToCPitch>
-          <radToAoAB>-0.08</radToAoAB>
-      </cs>
-    </control>
-  </segment>
-  <segment name="WR3">
-    <forward>1 0 0</forward>
-    <upward>0 0 1</upward>
-    <cp>0.169 -0.495 0.115</cp>
-    <seg_area>0.039</seg_area>
-    <seg_chord>0.170</seg_chord>
-    <aeroParamsYAML>${yaml_path}/techpod_TJ_wing.yaml</aeroParamsYAML>
-    <control>
-      <cs name="flap_right">
-         <controlJoint>${namespace}/flap_right_joint</controlJoint>
-         <radToCLift>1.6067 0</radToCLift>
-         <radToCDrag>0.1438 0.8227</radToCDrag>
-         <radToCPitch>0.0898 0</radToCPitch>
-         <radToAoAB>-0.08</radToAoAB>
-     </cs>
-    </control>
-  </segment>
-  <segment name="WR4">
-    <forward>1 0 0</forward>
-    <upward>0 0 1</upward>
-    <cp>0.165 -0.715 0.115</cp>
-    <seg_area>0.033</seg_area>
-    <seg_chord>0.157</seg_chord>
-    <aeroParamsYAML>${yaml_path}/techpod_TJ_wing.yaml</aeroParamsYAML>
-  </segment>
-  <segment name="WR5">
-    <forward>1 0 0</forward>
-    <upward>0 0 1</upward>
-    <cp>0.162 -0.907 0.115</cp>
-    <seg_area>0.026</seg_area>
-    <seg_chord>0.146</seg_chord>
-    <aeroParamsYAML>${yaml_path}/techpod_TJ_wing.yaml</aeroParamsYAML>
-    <control>
-      <cs name="aileron_right">
-          <controlJoint>${namespace}/aileron_right_joint</controlJoint>
-          <radToCLift>1.7541 0</radToCLift>
-          <radToCDrag>0.1053 0.6267</radToCDrag>
-          <radToCPitch>-0.1789 0</radToCPitch>
-          <radToAoAB>0.0</radToAoAB>
-      </cs>
-    </control>
-  </segment>
-  <segment name="WR6">
-    <forward>1 0 0</forward>
-    <upward>0 0 1</upward>
-    <cp>0.160 -1.083 0.115</cp>
-    <seg_area>0.024</seg_area>
-    <seg_chord>0.136</seg_chord>
-    <aeroParamsYAML>${yaml_path}/techpod_TJ_wing.yaml</aeroParamsYAML>
-    <control>
-      <cs name="aileron_right">
-         <controlJoint>${namespace}/aileron_right_joint</controlJoint>
-         <radToCLift>1.7541 0</radToCLift>
-         <radToCDrag>0.1053 0.6267</radToCDrag>
-         <radToCPitch>-0.1789 0</radToCPitch>
-         <radToAoAB>0.0</radToAoAB>
-      </cs>
-    </control>
-  </segment>
-  <segment name="WR7">
-    <forward>1 0 0</forward>
-    <upward>0 0 1</upward>
-    <cp>0.157 -1.234 0.115</cp>
-    <seg_area>0.016</seg_area>
-    <seg_chord>0.127</seg_chord>
-    <aeroParamsYAML>${yaml_path}/techpod_TJ_wing.yaml</aeroParamsYAML>
-  </segment>
+        <segment name="WR1">
+          <forward>1 0 0</forward>
+          <upward>0 0 1</upward>
+          <cp>0.175 -0.075 0.115</cp>
+          <seg_area>0.029</seg_area>
+          <seg_chord>0.194</seg_chord>
+          <aeroParamsYAML>${yaml_path}/techpod_TJ_wing.yaml</aeroParamsYAML>
+        </segment>
+        <segment name="WR2">
+          <forward>1 0 0</forward>
+          <upward>0 0 1</upward>
+          <cp>0.172 -0.265 0.115</cp>
+          <seg_area>0.042</seg_area>
+          <seg_chord>0.183</seg_chord>
+          <aeroParamsYAML>${yaml_path}/techpod_TJ_wing.yaml</aeroParamsYAML>
+          <control>
+            <cs name="flap_right">
+                <controlJoint>${namespace}/flap_right_joint</controlJoint>
+                <radToCLift>1.6067 0</radToCLift>
+                <radToCDrag>0.1438 0.8227</radToCDrag>
+                <radToCPitch>0.0898 0</radToCPitch>
+                <radToAoAB>-0.08</radToAoAB>
+            </cs>
+          </control>
+        </segment>
+        <segment name="WR3">
+          <forward>1 0 0</forward>
+          <upward>0 0 1</upward>
+          <cp>0.169 -0.495 0.115</cp>
+          <seg_area>0.039</seg_area>
+          <seg_chord>0.170</seg_chord>
+          <aeroParamsYAML>${yaml_path}/techpod_TJ_wing.yaml</aeroParamsYAML>
+          <control>
+            <cs name="flap_right">
+               <controlJoint>${namespace}/flap_right_joint</controlJoint>
+               <radToCLift>1.6067 0</radToCLift>
+               <radToCDrag>0.1438 0.8227</radToCDrag>
+               <radToCPitch>0.0898 0</radToCPitch>
+               <radToAoAB>-0.08</radToAoAB>
+           </cs>
+          </control>
+        </segment>
+        <segment name="WR4">
+          <forward>1 0 0</forward>
+          <upward>0 0 1</upward>
+          <cp>0.165 -0.715 0.115</cp>
+          <seg_area>0.033</seg_area>
+          <seg_chord>0.157</seg_chord>
+          <aeroParamsYAML>${yaml_path}/techpod_TJ_wing.yaml</aeroParamsYAML>
+        </segment>
+        <segment name="WR5">
+          <forward>1 0 0</forward>
+          <upward>0 0 1</upward>
+          <cp>0.162 -0.907 0.115</cp>
+          <seg_area>0.026</seg_area>
+          <seg_chord>0.146</seg_chord>
+          <aeroParamsYAML>${yaml_path}/techpod_TJ_wing.yaml</aeroParamsYAML>
+          <control>
+            <cs name="aileron_right">
+                <controlJoint>${namespace}/aileron_right_joint</controlJoint>
+                <radToCLift>1.7541 0</radToCLift>
+                <radToCDrag>0.1053 0.6267</radToCDrag>
+                <radToCPitch>-0.1789 0</radToCPitch>
+                <radToAoAB>0.0</radToAoAB>
+            </cs>
+          </control>
+        </segment>
+        <segment name="WR6">
+          <forward>1 0 0</forward>
+          <upward>0 0 1</upward>
+          <cp>0.160 -1.083 0.115</cp>
+          <seg_area>0.024</seg_area>
+          <seg_chord>0.136</seg_chord>
+          <aeroParamsYAML>${yaml_path}/techpod_TJ_wing.yaml</aeroParamsYAML>
+          <control>
+            <cs name="aileron_right">
+               <controlJoint>${namespace}/aileron_right_joint</controlJoint>
+               <radToCLift>1.7541 0</radToCLift>
+               <radToCDrag>0.1053 0.6267</radToCDrag>
+               <radToCPitch>-0.1789 0</radToCPitch>
+               <radToAoAB>0.0</radToAoAB>
+            </cs>
+          </control>
+        </segment>
+        <segment name="WR7">
+          <forward>1 0 0</forward>
+          <upward>0 0 1</upward>
+          <cp>0.157 -1.234 0.115</cp>
+          <seg_area>0.016</seg_area>
+          <seg_chord>0.127</seg_chord>
+          <aeroParamsYAML>${yaml_path}/techpod_TJ_wing.yaml</aeroParamsYAML>
+        </segment>
         <segment name="EL1">
           <forward>1 0 0</forward>

File: rotors_description/urdf/techpod_TJ_base.xacro (robot description, xacro)
@@ -22,27 +22,4 @@
     <origin xyz="0 0 0" rpy="0 0 0" />
   </xacro:default_gps>
-  <!-- Mount a magnetometer. note: mavlink interface already does this based on position from gps-->
-  <!--
-  <xacro:default_magnetometer namespace="${namespace}" parent_link="${namespace}/base_link" />
-  -->
-  <!-- Mount a pressure sensor. note: mavlink interface already does this -->
-  <!--
-  <xacro:default_pressure_sensor namespace="${namespace}" parent_link="${namespace}/base_link" />
-  -->
-  <!--
-  <xacro:if value="$(arg enable_ground_truth)">
-    <xacro:ground_truth_imu_and_odometry namespace="${namespace}" parent_link="${namespace}/base_link" />
-  </xacro:if>
-  -->
-  <xacro:if value="$(arg enable_logging)">
-    <!-- Instantiate a logger -->
-    <!--
-    <xacro:bag_plugin_macro
-      namespace="${namespace}"
-      bag_file="$(arg log_file)"
-      rotor_velocity_slowdown_sim="${rotor_velocity_slowdown_sim}"
-      wait_to_record_bag="$(arg wait_to_record_bag)" />
-    -->
-  </xacro:if>
   <xacro:default_camera
     namespace="${namespace}"

Commit message: Adjusted techpod_TJ according to latest set of sys-ID parameters from 15.08.19

File: rotors_description/urdf/techpod_TJ.xacro (robot description, xacro)
@@ -77,5 +77,5 @@
   <!-- Inertia of the main body -->
   <xacro:property name="body_inertia">
-    <inertia ixx="0.6688" ixy="0.0" ixz="0.0" iyy="0.16235" iyz="0.0" izz="0.69364" />
+    <inertia ixx="0.6688" ixy="0.0" ixz="0.0281" iyy="0.16235" iyz="0.0" izz="0.69364" />
   </xacro:property>
   <!-- Inertia of the aileron, assuming it is a cuboid -->
@@ -303,7 +303,7 @@
             <cs name="flap_left">
                 <controlJoint>${namespace}/flap_left_joint</controlJoint>
-                <radToCLift>1.6067 0</radToCLift>
-                <radToCDrag>0.1438 0.8227</radToCDrag>
-                <radToCPitch>0.0898 0</radToCPitch>
+                <radToCLift>1.6228 0</radToCLift>
+                <radToCDrag>0.1431 0.8085</radToCDrag>
+                <radToCPitch>0.0880 0</radToCPitch>
                 <radToAoAB>-0.08</radToAoAB>
             </cs>
@@ -320,7 +320,7 @@
             <cs name="flap_left">
                <controlJoint>${namespace}/flap_left_joint</controlJoint>
-               <radToCLift>1.6067 0</radToCLift>
-               <radToCDrag>0.1438 0.8227</radToCDrag>
-               <radToCPitch>0.0898 0</radToCPitch>
+               <radToCLift>1.6228 0</radToCLift>
+               <radToCDrag>0.1431 0.8085</radToCDrag>
+               <radToCPitch>0.0880 0</radToCPitch>
                <radToAoAB>-0.08</radToAoAB>
            </cs>
@@ -345,7 +345,7 @@
             <cs name="aileron_left">
                 <controlJoint>${namespace}/aileron_left_joint</controlJoint>
-                <radToCLift>1.7541 0</radToCLift>
-                <radToCDrag>0.1053 0.6267</radToCDrag>
-                <radToCPitch>-0.1789 0</radToCPitch>
+                <radToCLift>1.8386 0</radToCLift>
+                <radToCDrag>0.1053 0.5616</radToCDrag>
+                <radToCPitch>-0.0518 0</radToCPitch>
                 <radToAoAB>0.0</radToAoAB>
             </cs>
@@ -362,7 +362,7 @@
             <cs name="aileron_left">
                <controlJoint>${namespace}/aileron_left_joint</controlJoint>
-               <radToCLift>1.7541 0</radToCLift>
-               <radToCDrag>0.1053 0.6267</radToCDrag>
-               <radToCPitch>-0.1789 0</radToCPitch>
+               <radToCLift>1.8386 0</radToCLift>
+               <radToCDrag>0.1053 0.5616</radToCDrag>
+               <radToCPitch>-0.0518 0</radToCPitch>
                <radToAoAB>0.0</radToAoAB>
             </cs>
@@ -395,7 +395,7 @@
             <cs name="flap_right">
                 <controlJoint>${namespace}/flap_right_joint</controlJoint>
-                <radToCLift>1.6067 0</radToCLift>
-                <radToCDrag>0.1438 0.8227</radToCDrag>
-                <radToCPitch>0.0898 0</radToCPitch>
+                <radToCLift>1.6228 0</radToCLift>
+                <radToCDrag>0.1431 0.8085</radToCDrag>
+                <radToCPitch>0.0880 0</radToCPitch>
                 <radToAoAB>-0.08</radToAoAB>
             </cs>
@@ -412,7 +412,7 @@
             <cs name="flap_right">
                <controlJoint>${namespace}/flap_right_joint</controlJoint>
-               <radToCLift>1.6067 0</radToCLift>
-               <radToCDrag>0.1438 0.8227</radToCDrag>
-               <radToCPitch>0.0898 0</radToCPitch>
+               <radToCLift>1.6228 0</radToCLift>
+               <radToCDrag>0.1431 0.8085</radToCDrag>
+               <radToCPitch>0.0880 0</radToCPitch>
                <radToAoAB>-0.08</radToAoAB>
            </cs>
@@ -437,7 +437,7 @@
             <cs name="aileron_right">
                 <controlJoint>${namespace}/aileron_right_joint</controlJoint>
-                <radToCLift>1.7541 0</radToCLift>
-                <radToCDrag>0.1053 0.6267</radToCDrag>
-                <radToCPitch>-0.1789 0</radToCPitch>
+                <radToCLift>1.8386 0</radToCLift>
+                <radToCDrag>0.1053 0.5616</radToCDrag>
+                <radToCPitch>-0.0518 0</radToCPitch>
                 <radToAoAB>0.0</radToAoAB>
             </cs>
@@ -454,7 +454,7 @@
             <cs name="aileron_right">
                <controlJoint>${namespace}/aileron_right_joint</controlJoint>
-               <radToCLift>1.7541 0</radToCLift>
-               <radToCDrag>0.1053 0.6267</radToCDrag>
-               <radToCPitch>-0.1789 0</radToCPitch>
+               <radToCLift>1.8386 0</radToCLift>
+               <radToCDrag>0.1053 0.5616</radToCDrag>
+               <radToCPitch>-0.0518 0</radToCPitch>
                <radToAoAB>0.0</radToAoAB>
             </cs>
@@ -482,5 +482,5 @@
             <cs name="elevator_left">
                 <controlJoint>${namespace}/elevator_joint</controlJoint>
-                <radToCLift>1.15 0</radToCLift>
+                <radToCLift>1.5676 0</radToCLift>
                 <radToCDrag>0 0</radToCDrag>
                 <radToCPitch>0 0</radToCPitch>
@@ -502,5 +502,5 @@
             <cs name="elevator_right">
                 <controlJoint>${namespace}/elevator_joint</controlJoint>
-                <radToCLift>1.15 0</radToCLift>
+                <radToCLift>1.5676 0</radToCLift>
                 <radToCDrag>0 0</radToCDrag>
                 <radToCPitch>0 0</radToCPitch>
@@ -522,5 +522,5 @@
             <cs name="rudder">
                 <controlJoint>${namespace}/rudder_joint</controlJoint>
-                <radToCLift>2.2459 0</radToCLift>
+                <radToCLift>2.2801 0</radToCLift>
                 <radToCDrag>0 0</radToCDrag>
                 <radToCPitch>0 0</radToCPitch>
