Commit message: Adding ability to enable/disable wind via launch parameters

File: rotors_description/urdf/techpod_TJ.xacro (robot description, xacro)
@@ -20,4 +20,5 @@
   <xacro:property name="serial_device" value="$(arg serial_device)" />
   <xacro:property name="main_color" value="White"/>
+  <xacro:property name="enable_wind" value="$(arg enable_wind)"/>
   <!-- Constants -->
   <xacro:property name="PI" value="3.1415926535897931" />
@@ -253,34 +254,36 @@
   </gazebo>
   -->
-  <gazebo>
-    <plugin filename="librotors_gazebo_wind_beta_plugin.so" name="wind_beta_plugin">
-      <robotNamespace>${namespace}</robotNamespace>
-      <windLayer>
-        <layer name="layer1">
-          <altitude>10</altitude>
-          <windMeanNED>-5 0 0</windMeanNED>
-        </layer>
-        <layer name="layer2">
-          <altitude>25</altitude>
-          <windMeanNED>-6 0 0</windMeanNED>
-        </layer>
-        <layer name="layer3">
-          <altitude>35</altitude>
-          <windMeanNED>-10 0 0</windMeanNED>
-        </layer>
-      </windLayer>
-      <findWind>
-        <query name="q1">
-          <linkName>${namespace}/base_link</linkName>
-          <windTopic>wind_base_link</windTopic>
-        </query>
-      </findWind>
-      <lambdaMin>10</lambdaMin>
-      <lengthScale>725</lengthScale>
-      <fourierNNN>10 10 10</fourierNNN>
-      <sigma>5</sigma>
-      <trnspVelTurbNED>5 0 0</trnspVelTurbNED>
-    </plugin>
-  </gazebo>
+  <xacro:if value="${enable_wind}">
+    <gazebo>
+      <plugin filename="librotors_gazebo_wind_beta_plugin.so" name="wind_beta_plugin">
+        <robotNamespace>${namespace}</robotNamespace>
+        <windLayer>
+          <layer name="layer1">
+            <altitude>10</altitude>
+            <windMeanNED>-5 0 0</windMeanNED>
+          </layer>
+          <layer name="layer2">
+            <altitude>25</altitude>
+            <windMeanNED>-6 0 0</windMeanNED>
+          </layer>
+          <layer name="layer3">
+            <altitude>35</altitude>
+            <windMeanNED>-10 0 0</windMeanNED>
+          </layer>
+        </windLayer>
+        <findWind>
+          <query name="q1">
+            <linkName>${namespace}/base_link</linkName>
+            <windTopic>wind_base_link</windTopic>
+          </query>
+        </findWind>
+        <lambdaMin>10</lambdaMin>
+        <lengthScale>725</lengthScale>
+        <fourierNNN>10 10 10</fourierNNN>
+        <sigma>5</sigma>
+        <trnspVelTurbNED>5 0 0</trnspVelTurbNED>
+      </plugin>
+    </gazebo>
+  </xacro:if>
   <gazebo>
     <plugin filename="librotors_gazebo_propulsion_plugin.so" name="propulsion_plugin">

File: rotors_description/urdf/techpod_TJ_flex.xacro (robot description, xacro)
@@ -20,4 +20,5 @@
    <xacro:property name="yaml_path" value="$(arg yaml_path)" />
    <xacro:property name="serial_device" value="$(arg serial_device)" />
+   <xacro:property name="enable_wind" value="$(arg enable_wind)"/>
    <!-- Constants -->
    <xacro:property name="PI" value="3.1415926535897931" />
@@ -1117,36 +1118,36 @@
    </gazebo>
    <!-- Wind -->
-   <!--
-   <gazebo>
-     <plugin filename="librotors_gazebo_wind_beta_plugin.so" name="wind_beta_plugin">
-       <robotNamespace>${namespace}</robotNamespace>
-       <windLayer>
-         <layer name="layer1">
-           <altitude>10</altitude>
-           <windMeanNED>-5 0 0</windMeanNED>
-         </layer>
-         <layer name="layer2">
-           <altitude>25</altitude>
-           <windMeanNED>-6 0 0</windMeanNED>
-         </layer>
-         <layer name="layer3">
-           <altitude>35</altitude>
-           <windMeanNED>-10 0 0</windMeanNED>
-         </layer>
-       </windLayer>
-       <findWind>
-         <query name="q1">
-           <linkName>${namespace}/base_link</linkName>
-           <windTopic>wind_base_link</windTopic>
-         </query>
-       </findWind>
-       <lambdaMin>2</lambdaMin>
-       <lengthScale>725</lengthScale>
-       <fourierNNN>10 10 10</fourierNNN>
-       <sigma>5</sigma>
-       <trnspVelTurbNED>-5 0 0</trnspVelTurbNED>
-     </plugin>
-   </gazebo>
-   -->
+   <xacro:if value="${enable_wind}">
+     <gazebo>
+       <plugin filename="librotors_gazebo_wind_beta_plugin.so" name="wind_beta_plugin">
+         <robotNamespace>${namespace}</robotNamespace>
+         <windLayer>
+           <layer name="layer1">
+             <altitude>10</altitude>
+             <windMeanNED>-3 0 0</windMeanNED>
+           </layer>
+           <layer name="layer2">
+             <altitude>25</altitude>
+             <windMeanNED>-4 0 0</windMeanNED>
+           </layer>
+           <layer name="layer3">
+             <altitude>35</altitude>
+             <windMeanNED>-5 0 0</windMeanNED>
+           </layer>
+         </windLayer>
+         <findWind>
+           <query name="q1">
+             <linkName>${namespace}/base_link</linkName>
+             <windTopic>wind_base_link</windTopic>
+           </query>
+         </findWind>
+         <lambdaMin>2</lambdaMin>
+         <lengthScale>725</lengthScale>
+         <fourierNNN>10 10 10</fourierNNN>
+         <sigma>3</sigma>
+         <trnspVelTurbNED>-3 0 0</trnspVelTurbNED>
+       </plugin>
+     </gazebo>
+   </xacro:if>
    <!-- Tracing ribbon/Visual plugin -->
    <!--

File: rotors_description/urdf/techpod_X.xacro (robot description, xacro)
@@ -19,4 +19,5 @@
   <xacro:property name="yaml_path" value="$(arg yaml_path)"/>
   <xacro:property name="serial_device" value="$(arg serial_device)" />
+  <xacro:property name="enable_wind" value="$(arg enable_wind)"/>
   <!-- Constants -->
   <xacro:property name="PI" value="3.1415926535897931" />
@@ -245,41 +246,43 @@
     <xacro:insert_block name="propeller_inertia" />
   </xacro:propeller>
-  <gazebo>
-    <plugin filename="librotors_gazebo_wind_beta_plugin.so" name="wind_beta_plugin">
-      <robotNamespace>${namespace}</robotNamespace>
-      <windLayer>
-        <layer name="layer1">
-          <altitude>10</altitude>
-          <windMeanNED>-5 0 0</windMeanNED>
-        </layer>
-        <layer name="layer2">
-          <altitude>25</altitude>
-          <windMeanNED>-6 0 0</windMeanNED>
-        </layer>
-        <layer name="layer3">
-          <altitude>35</altitude>
-          <windMeanNED>-10 0 0</windMeanNED>
-        </layer>
-      </windLayer>
-      <!---->
-      <findWind>
-        <query name="q1">
-          <linkName>${namespace}/base_link</linkName>
-          <windTopic>wind_base_link</windTopic>
-        </query>
-      </findWind>
-      <!--
-      <customWindFieldPath>${yaml_path}/../test_wind_field.csv</customWindFieldPath>
-      <windFieldXOffset>100</windFieldXOffset>
-      <windFieldYOffset>100</windFieldYOffset>
-      <windFieldZOffset>0</windFieldZOffset>
-      -->
-      <lambdaMin>10</lambdaMin>
-      <lengthScale>725</lengthScale>
-      <fourierNNN>7 7 7</fourierNNN>
-      <sigma>2</sigma>
-      <trnspVelTurbNED>5 0 0</trnspVelTurbNED>
-    </plugin>
-  </gazebo>
+  <xacro:if value="${enable_wind}">
+    <gazebo>
+      <plugin filename="librotors_gazebo_wind_beta_plugin.so" name="wind_beta_plugin">
+        <robotNamespace>${namespace}</robotNamespace>
+        <windLayer>
+          <layer name="layer1">
+            <altitude>10</altitude>
+            <windMeanNED>-5 0 0</windMeanNED>
+          </layer>
+          <layer name="layer2">
+            <altitude>25</altitude>
+            <windMeanNED>-6 0 0</windMeanNED>
+          </layer>
+          <layer name="layer3">
+            <altitude>35</altitude>
+            <windMeanNED>-10 0 0</windMeanNED>
+          </layer>
+        </windLayer>
+        <!---->
+        <findWind>
+          <query name="q1">
+            <linkName>${namespace}/base_link</linkName>
+            <windTopic>wind_base_link</windTopic>
+          </query>
+        </findWind>
+        <!--
+        <customWindFieldPath>${yaml_path}/../test_wind_field.csv</customWindFieldPath>
+        <windFieldXOffset>100</windFieldXOffset>
+        <windFieldYOffset>100</windFieldYOffset>
+        <windFieldZOffset>0</windFieldZOffset>
+        -->
+        <lambdaMin>10</lambdaMin>
+        <lengthScale>725</lengthScale>
+        <fourierNNN>7 7 7</fourierNNN>
+        <sigma>2</sigma>
+        <trnspVelTurbNED>5 0 0</trnspVelTurbNED>
+      </plugin>
+    </gazebo>
+  </xacro:if>
   <gazebo>
     <plugin filename="librotors_gazebo_propulsion_plugin.so" name="propulsion_plugin">

File: rotors_description/urdf/techpod_X_flex.xacro (robot description, xacro)
@@ -20,4 +20,5 @@
    <xacro:property name="yaml_path" value="$(arg yaml_path)" />
    <xacro:property name="serial_device" value="$(arg serial_device)" />
+   <xacro:property name="enable_wind" value="$(arg enable_wind)"/>
    <!-- Constants -->
    <xacro:property name="PI" value="3.1415926535897931" />
@@ -926,40 +927,42 @@
       </plugin>
    </gazebo>
-   <gazebo>
-     <plugin filename="librotors_gazebo_wind_beta_plugin.so" name="wind_beta_plugin">
-       <robotNamespace>${namespace}</robotNamespace>
-       <windLayer>
-         <layer name="layer1">
-           <altitude>10</altitude>
-           <windMeanNED>-5 0 0</windMeanNED>
-         </layer>
-         <layer name="layer2">
-           <altitude>25</altitude>
-           <windMeanNED>-6 0 0</windMeanNED>
-         </layer>
-         <layer name="layer3">
-           <altitude>35</altitude>
-           <windMeanNED>-10 0 0</windMeanNED>
-         </layer>
-       </windLayer>
-       <findWind>
-         <query name="q1">
-           <linkName>${namespace}/base_link</linkName>
-           <windTopic>wind_base_link</windTopic>
-         </query>
-         <!--
-         <query name="q2">
-           <linkName>${namespace}/payload_1</linkName>
-           <windTopic>wind_payload</windTopic>
-         </query>
-         -->
-       </findWind>
-       <lambdaMin>2</lambdaMin>
-       <lengthScale>725</lengthScale>
-       <fourierNNN>10 10 10</fourierNNN>
-       <sigma>5</sigma>
-       <trnspVelTurbNED>-5 0 0</trnspVelTurbNED>
-     </plugin>
-   </gazebo>
+   <xacro:if value="${enable_wind}">
+     <gazebo>
+       <plugin filename="librotors_gazebo_wind_beta_plugin.so" name="wind_beta_plugin">
+         <robotNamespace>${namespace}</robotNamespace>
+         <windLayer>
+           <layer name="layer1">
+             <altitude>10</altitude>
+             <windMeanNED>-5 0 0</windMeanNED>
+           </layer>
+           <layer name="layer2">
+             <altitude>25</altitude>
+             <windMeanNED>-6 0 0</windMeanNED>
+           </layer>
+           <layer name="layer3">
+             <altitude>35</altitude>
+             <windMeanNED>-10 0 0</windMeanNED>
+           </layer>
+         </windLayer>
+         <findWind>
+           <query name="q1">
+             <linkName>${namespace}/base_link</linkName>
+             <windTopic>wind_base_link</windTopic>
+           </query>
+           <!--
+           <query name="q2">
+             <linkName>${namespace}/payload_1</linkName>
+             <windTopic>wind_payload</windTopic>
+           </query>
+           -->
+         </findWind>
+         <lambdaMin>2</lambdaMin>
+         <lengthScale>725</lengthScale>
+         <fourierNNN>10 10 10</fourierNNN>
+         <sigma>5</sigma>
+         <trnspVelTurbNED>-5 0 0</trnspVelTurbNED>
+       </plugin>
+     </gazebo>
+   </xacro:if>
    <!-- Tracing ribbon/Visual plugin -->
    <gazebo reference="${namespace}/base_link">
