Commit message: change "voliro" to "omav"

File: rotors_description/urdf/omav.xacro (robot description, xacro)
@@ -18,5 +18,4 @@
 <robot name="$(arg mav_name)" xmlns:xacro="http://ros.org/wiki/xacro">
   <!-- Included URDF Files -->
-  <xacro:include filename="$(find rotors_description)/urdf/multirotor_base.xacro"/>
   <xacro:include filename="$(find rotors_description)/urdf/overactuated_base.xacro"/>
     <!-- Properties -->
@@ -25,6 +24,6 @@
     <xacro:property name="use_mesh_file_core" value="true"/>
     <xacro:property name="use_mesh_file_rotor_unit" value="true"/>
-    <xacro:property name="mesh_file_core" value="package://rotors_description/meshes/voliro/voliroX_core.dae"/>
-    <xacro:property name="mesh_file_tilt_unit" value="package://rotors_description/meshes/voliro/voliroX_tiltarm.dae"/>-->
+    <xacro:property name="mesh_file_core" value="package://rotors_description/meshes/omav/omav_core.dae"/>
+    <xacro:property name="mesh_file_tilt_unit" value="package://rotors_description/meshes/omav/omav_tiltarm.dae"/>-->
     <xacro:property name="mass_core" value="2.30"/>    <!-- [kg] -->
     <xacro:property name="mass_tilt_unit" value="0.277"/>    <!-- [kg] -->

File: rotors_description/urdf/omav_base.xacro (robot description, xacro)
@@ -18,6 +18,6 @@
 <robot name="$(arg mav_name)" xmlns:xacro="http://ros.org/wiki/xacro">
   <xacro:include filename="$(find rotors_description)/urdf/component_snippets.xacro"/>
-  <!-- Instantiate voliro "mechanics". -->
-  <xacro:include filename="$(find rotors_description)/urdf/voliro.xacro"/>
+  <!-- Instantiate OMAV "mechanics". -->
+  <xacro:include filename="$(find rotors_description)/urdf/omav.xacro"/>
   <!-- Instantiate a controller. -->
   <xacro:controller_plugin_macro namespace="${namespace}" imu_sub_topic="imu"/>

Commit message: rename "voliro" to "omav"

File: rotors_description/urdf/omav.xacro (robot description, xacro)
@@ -25,6 +25,6 @@
     <xacro:property name="use_mesh_file_core" value="true"/>
     <xacro:property name="use_mesh_file_rotor_unit" value="true"/>
-    <xacro:property name="mesh_file_core" value="package://rotors_description/meshes/voliro/voliroX_core.dae"/>
-    <xacro:property name="mesh_file_tilt_unit" value="package://rotors_description/meshes/voliro/voliroX_tiltarm.dae"/>-->
+    <xacro:property name="mesh_file_core" value="package://rotors_description/meshes/omav/omav_core.dae"/>
+    <xacro:property name="mesh_file_tilt_unit" value="package://rotors_description/meshes/omav/omav_tiltarm.dae"/>-->
     <xacro:property name="mass_core" value="2.30"/>    <!-- [kg] -->
     <xacro:property name="mass_tilt_unit" value="0.277"/>    <!-- [kg] -->

Commit message: Remove extra ref in xacro file. Update Cf values and CoM offset to 0.

File: rotors_description/urdf/omav.xacro (robot description, xacro)
@@ -18,5 +18,4 @@
 <robot name="$(arg mav_name)" xmlns:xacro="http://ros.org/wiki/xacro">
   <!-- Included URDF Files -->
-  <xacro:include filename="$(find rotors_description)/urdf/multirotor_base.xacro"/>
   <xacro:include filename="$(find rotors_description)/urdf/overactuated_base.xacro"/>
     <!-- Properties -->
@@ -35,6 +34,6 @@
     <xacro:property name="rotor_offset_top" value="0.060"/>    <!-- [m] -->
     <xacro:property name="radius_rotor" value="0.1143"/>    <!-- [m] -->
-    <xacro:property name="motor_constant" value="${8.54858e-06}"/>    <!-- [kg m/s^2] -->
-    <xacro:property name="motor_constant_lower" value="${8.54858e-06}"/>    <!-- [kg m/s^2] -->
+    <xacro:property name="motor_constant" value="${7.2e-06}"/>    <!-- [kg m/s^2] -->
+    <xacro:property name="motor_constant_lower" value="${7.2e-06}"/>    <!-- [kg m/s^2] -->
     <xacro:property name="moment_constant" value="0.015"/>    <!-- [m] -->
     <xacro:property name="moment_constant_lower" value="0.005"/>    <!-- [m] -->
@@ -56,5 +55,5 @@
     <!-- Body Interia / CoM Offset -->
     <xacro:property name="body_inertia_origin">
-      <origin xyz="0 0 -0.05" />
+      <origin xyz="0 0 0" />
     </xacro:property>
     <!-- Rotor unit inertia without the propellor. -->

Commit message: Parametrize pid tilt gains.

File: rotors_description/urdf/omav.xacro (robot description, xacro)
@@ -48,4 +48,7 @@
     <xacro:property name="rotor_drag_coefficient" value="${8.06428e-05}"/>
     <xacro:property name="rolling_moment_coefficient" value="0.000001"/>
+    <xacro:property name="tilt_p_gain" value="1.0"/>
+    <xacro:property name="tilt_i_gain" value="0.0"/>
+    <xacro:property name="tilt_d_gain" value="0.1"/>
     <!-- Property Blocks -->
     <xacro:property name="body_inertia">
@@ -98,5 +101,8 @@
     mesh="propeller"
     mesh_tilt_unit="${mesh_file_tilt_unit}"
-    color="Black">
+    color="Black"
+    p_gain="${tilt_p_gain}"
+    i_gain="${tilt_i_gain}"
+    d_gain="${tilt_d_gain}">
     <origin xyz="0 -${arm_length} 0" rpy="0 0 4.71238898038"/>
     <xacro:insert_block name="rotor_inertia" />
@@ -123,5 +129,8 @@
     mesh="propeller"
     mesh_tilt_unit="${mesh_file_tilt_unit}"
-    color="Black">
+    color="Black"
+    p_gain="${tilt_p_gain}"
+    i_gain="${tilt_i_gain}"
+    d_gain="${tilt_d_gain}">
     <origin xyz="0 ${arm_length} 0" rpy="0 0 1.57079632679"/>
     <xacro:insert_block name="rotor_inertia" />
@@ -148,5 +157,8 @@
     mesh="propeller"
     mesh_tilt_unit="${mesh_file_tilt_unit}"
-    color="Orange">
+    color="Orange"
+    p_gain="${tilt_p_gain}"
+    i_gain="${tilt_i_gain}"
+    d_gain="${tilt_d_gain}">
     <origin xyz="${cos30*arm_length} ${sin30*arm_length} 0" rpy="0 0 0.52359877559"/>
     <xacro:insert_block name="rotor_inertia" />
@@ -172,5 +184,8 @@
     mesh="propeller"
     mesh_tilt_unit="${mesh_file_tilt_unit}"
-    color="DarkGrey">
+    color="DarkGrey"
+    p_gain="${tilt_p_gain}"
+    i_gain="${tilt_i_gain}"
+    d_gain="${tilt_d_gain}">
     <origin xyz="-${cos30*arm_length} -${sin30*arm_length} 0" rpy="0 0 3.66519142919"/>
     <xacro:insert_block name="rotor_inertia" />
@@ -196,5 +211,8 @@
     mesh="propeller"
     mesh_tilt_unit="${mesh_file_tilt_unit}"
-    color="Orange">
+    color="Orange"
+    p_gain="${tilt_p_gain}"
+    i_gain="${tilt_i_gain}"
+    d_gain="${tilt_d_gain}">
     <origin xyz="${cos30*arm_length} -${sin30*arm_length} 0" rpy="0 0 5.75958653158"/>
     <xacro:insert_block name="rotor_inertia" />
@@ -220,5 +238,8 @@
     mesh="propeller"
     mesh_tilt_unit="${mesh_file_tilt_unit}"
-    color="DarkGrey">
+    color="DarkGrey"
+    p_gain="${tilt_p_gain}"
+    i_gain="${tilt_i_gain}"
+    d_gain="${tilt_d_gain}">
     <origin xyz="-${cos30*arm_length} ${sin30*arm_length} 0" rpy="0 0 2.61799387799"/>
     <xacro:insert_block name="rotor_inertia" />

File: rotors_description/urdf/overactuated_base.xacro (robot description, xacro)
@@ -160,5 +160,5 @@
   <!-- Double tilt unit joint and link -->
   <xacro:macro name="double_tilt_unit"
-    params="robot_namespace suffix direction_upper direction_lower motor_constant motor_constant_lower moment_constant moment_constant_lower parent mass_rotor mass_tilt_unit time_constant_up time_constant_down max_rot_velocity rotor_offset_top motor_number rotor_drag_coefficient rolling_moment_coefficient color mesh mesh_tilt_unit *origin *inertia">
+    params="robot_namespace suffix direction_upper direction_lower motor_constant motor_constant_lower moment_constant moment_constant_lower parent mass_rotor mass_tilt_unit time_constant_up time_constant_down max_rot_velocity rotor_offset_top motor_number rotor_drag_coefficient rolling_moment_coefficient color mesh mesh_tilt_unit p_gain i_gain d_gain *origin *inertia">
     <!-- Rotor tilt_unit -->
     <joint name="${robot_namespace}/tilt_unit_${motor_number}_revolutejoint" type="continuous">
@@ -197,7 +197,7 @@
         <motorPositionPubTopic>/tilt_motor_${motor_number}/position</motorPositionPubTopic>
         <joint_control_pid>
-            <p>1.0</p>
-            <i>0.0</i>
-            <d>0.005</d>
+            <p>${p_gain}</p>
+            <i>${i_gain}</i>
+            <d>${d_gain}</d>
             <iMax>1.0</iMax>
             <iMin>-1.0</iMin>
