Commit message: - improved and extended state machine in payload plugin - macro passive payload pick-up hook

File: rotors_description/urdf/techpod_exp_flex.xacro (robot description, xacro)
@@ -17,4 +17,5 @@
    <xacro:include filename="$(find rotors_description)/urdf/rope.xacro" />
    <xacro:include filename="$(find rotors_description)/urdf/hook.xacro" />
+   <xacro:include filename="$(find rotors_description)/urdf/hook_simple.xacro" />
    <!-- Global properties -->
    <xacro:property name="namespace" value="$(arg namespace)" />
@@ -1162,12 +1163,153 @@
    </xacro:if>
    <!-- Tracing ribbon/Visual plugin -->
+   <!---->
+   <gazebo reference="${namespace}/base_link">
+      <visual>
+         <plugin name="visual_plugin_base_link" filename="librotors_gazebo_template_visual_plugin.so" />
+      </visual>
+   </gazebo>
+   <!-- fw challenge payloads -->
+   <xacro:payload_hook_simple namespace="${namespace}">
+   </xacro:payload_hook_simple>
+   <link name="${namespace}/payload_1">
+      <inertial>
+         <origin xyz="0 0 0" rpy="0 0 0" />
+         <mass value="0.25" />
+         <xacro:sphere_inertia r="0.05" mass="0.25" />
+      </inertial>
+      <visual>
+         <origin xyz="0 0 0" rpy="0 0 0" />
+         <geometry>
+            <box size = "0.5 0.5 0.5" />
+         </geometry>
+      </visual>
+      <collision>
+         <origin xyz="0 0 0" rpy="0 0 0" />
+         <geometry>
+            <box size = "0.5 0.5 0.5" />
+         </geometry>
+      </collision>
+   </link>
+   <joint name="${namespace}/payload_1_joint" type="floating">
+      <parent link="${namespace}/payload_hook" />
+      <child link="${namespace}/payload_1" />
+      <origin xyz="-1.5 0 0" rpy="0 0 0" />
+   </joint>
+   <gazebo reference="${namespace}/payload_1">
+      <material>Gazebo/Yellow</material>
+      <mu1>0.2</mu1>
+      <mu2>0.2</mu2>
+      <kp>10000</kp>
+      <kd>1</kd>
+   </gazebo>
+   <gazebo>
+      <plugin filename="librotors_gazebo_payload_plugin.so" name="payload_plugin_1">
+         <robotNamespace>${namespace}</robotNamespace>
+         <joint>${namespace}/payload_1_joint</joint>
+         <payload>${namespace}/payload_1</payload>
+         <parent>${namespace}/payload_hook</parent>
+         <proxRec>true</proxRec>
+         <radiusRec>5</radiusRec>
+         <hoistPosParent>-1.5 0 0</hoistPosParent>
+         <hoistPosPayload>0 0 0</hoistPosPayload>
+         <pickupWorldPosPayload>256.65 43.54 80</pickupWorldPosPayload>
+         <initialState>3</initialState> <!-- 0: attached, 1: falling, 2: teleporting, 3: resting @ pickup pos-->
+         <dropTopic>drop_1</dropTopic>
+      </plugin>
+   </gazebo>
+   <link name="${namespace}/payload_2">
+      <inertial>
+         <origin xyz="0 0 0" rpy="0 0 0" />
+         <mass value="0.25" />
+         <xacro:sphere_inertia r="0.05" mass="0.25" />
+      </inertial>
+      <visual>
+         <origin xyz="0 0 0" rpy="0 0 0" />
+         <geometry>
+            <box size = "0.5 0.5 0.5" />
+         </geometry>
+      </visual>
+      <collision>
+         <origin xyz="0 0 0" rpy="0 0 0" />
+         <geometry>
+            <box size = "0.5 0.5 0.5" />
+         </geometry>
+      </collision>
+   </link>
+   <joint name="${namespace}/payload_2_joint" type="floating">
+      <parent link="${namespace}/payload_hook" />
+      <child link="${namespace}/payload_2" />
+      <origin xyz="-1.5 0 0" rpy="0 0 0" />
+   </joint>
+   <gazebo reference="${namespace}/payload_2">
+      <material>Gazebo/Red</material>
+      <mu1>0.2</mu1>
+      <mu2>0.2</mu2>
+      <kp>10000</kp>
+      <kd>1</kd>
+   </gazebo>
+   <gazebo>
+      <plugin filename="librotors_gazebo_payload_plugin.so" name="payload_plugin_1">
+         <robotNamespace>${namespace}</robotNamespace>
+         <joint>${namespace}/payload_2_joint</joint>
+         <payload>${namespace}/payload_2</payload>
+         <parent>${namespace}/payload_hook</parent>
+         <proxRec>true</proxRec>
+         <radiusRec>5</radiusRec>
+         <hoistPosParent>-1.5 0 0</hoistPosParent>
+         <hoistPosPayload>0 0 0</hoistPosPayload>
+         <pickupWorldPosPayload>246.65 38.54 80</pickupWorldPosPayload>
+         <initialState>3</initialState> <!-- 0: attached, 1: falling, 2: teleporting, 3: resting @ pickup pos-->
+         <dropTopic>drop_1</dropTopic>
+      </plugin>
+   </gazebo>
+   <link name="${namespace}/payload_3">
+      <inertial>
+         <origin xyz="0 0 0" rpy="0 0 0" />
+         <mass value="0.25" />
+         <xacro:sphere_inertia r="0.05" mass="0.25" />
+      </inertial>
+      <visual>
+         <origin xyz="0 0 0" rpy="0 0 0" />
+         <geometry>
+            <box size = "0.5 0.5 0.5" />
+         </geometry>
+      </visual>
+      <collision>
+         <origin xyz="0 0 0" rpy="0 0 0" />
+         <geometry>
+            <box size = "0.5 0.5 0.5" />
+         </geometry>
+      </collision>
+   </link>
+   <joint name="${namespace}/payload_3_joint" type="floating">
+      <parent link="${namespace}/payload_hook" />
+      <child link="${namespace}/payload_3" />
+      <origin xyz="-1.5 0 0" rpy="0 0 0" />
+   </joint>
+   <gazebo reference="${namespace}/payload_3">
+      <material>Gazebo/Blue</material>
+      <mu1>0.2</mu1>
+      <mu2>0.2</mu2>
+      <kp>10000</kp>
+      <kd>1</kd>
+   </gazebo>
+   <gazebo>
+      <plugin filename="librotors_gazebo_payload_plugin.so" name="payload_plugin_1">
+         <robotNamespace>${namespace}</robotNamespace>
+         <joint>${namespace}/payload_3_joint</joint>
+         <payload>${namespace}/payload_3</payload>
+         <parent>${namespace}/payload_hook</parent>
+         <proxRec>true</proxRec>
+         <radiusRec>5</radiusRec>
+         <hoistPosParent>-1.5 0 0</hoistPosParent>
+         <hoistPosPayload>0 0 0</hoistPosPayload>
+         <pickupWorldPosPayload>246.65 48.54 80</pickupWorldPosPayload>
+         <initialState>3</initialState> <!-- 0: attached, 1: falling, 2: teleporting, 3: resting @ pickup pos-->
+         <dropTopic>drop_1</dropTopic>
+      </plugin>
+   </gazebo>
+   <!-- Payload on hook -->
    <!--
-   <gazebo reference="${namespace}/base_link">
-      <visual>
-         <plugin name="visual_plugin_base_link" filename="librotors_gazebo_template_visual_plugin.so" />
-      </visual>
-   </gazebo>
-   -->
-   <!-- Payload on hook -->
    <xacro:payload_hook namespace="${namespace}">
    </xacro:payload_hook>
@@ -1224,5 +1366,5 @@
      <origin xyz="-0.2 0 0" rpy="0 2.356 0" />
    </xacro:default_lidar>
-   <!---->
+   -->
    <!-- Payload on wing -->
    <!--
@@ -1269,4 +1411,6 @@
          <hoistPosParent>0 -0.15 -0.04</hoistPosParent>
          <hoistPosPayload>0 0 0</hoistPosPayload>
+         <teleportBackToAircraft>true</teleportBackToAircraft>
+         <initialState>0</initialState>
          <dropTopic>drop_1</dropTopic>
       </plugin>
@@ -1489,18 +1633,3 @@
       </plugin>
    </gazebo>
-   <!-- Miscellaneous -->
-   <!--
-   <link name="${namespace}/check_coordinates">
-      <inertial>
-         <mass value="0.1" />
-         <xacro:box_inertia x="0.1" y="0.1" z="0.1" mass="0.1" />
-      </inertial>
-   </link>
-   <joint name="${namespace}/check_coordinates_joint" type="revolute">
-     <origin xyz="0.54 0 0.184" rpy="0 0 0" />
-     <parent link="${namespace}/base_link" />
-     <child link="${namespace}/check_coordinates" />
-     <limit upper="0" lower="0" effort="0" velocity="0" />
-   </joint>
-   -->
 </robot>

Commit message: Fixed-wing challenge environment for Juan Nieto's farewell!

File: rotors_description/urdf/techpod_exp_flex.xacro (robot description, xacro)
@@ -158,5 +158,5 @@
    <gazebo reference="${namespace}/dome">
       <material>Gazebo/GreyTransparent</material>
-   </gazebo>-->
+   </gazebo>
    <joint name="${namespace}/bar_joint" type="fixed">
       <parent link="${namespace}/base_link" />
@@ -1163,14 +1163,14 @@
    </xacro:if>
    <!-- Tracing ribbon/Visual plugin -->
-   <!---->
+   <!--
    <gazebo reference="${namespace}/base_link">
       <visual>
          <plugin name="visual_plugin_base_link" filename="librotors_gazebo_template_visual_plugin.so" />
       </visual>
-   </gazebo>
+   </gazebo>-->
    <!-- fw challenge payloads -->
    <xacro:payload_hook_simple namespace="${namespace}">
    </xacro:payload_hook_simple>
-   <link name="${namespace}/payload_1">
+   <link name="${namespace}/soccer_ball_1">
       <inertial>
          <origin xyz="0 0 0" rpy="0 0 0" />
@@ -1181,5 +1181,5 @@
          <origin xyz="0 0 0" rpy="0 0 0" />
          <geometry>
-            <box size = "0.5 0.5 0.5" />
+            <sphere radius = "0.5" />
          </geometry>
       </visual>
@@ -1187,5 +1187,5 @@
          <origin xyz="0 0 0" rpy="0 0 0" />
          <geometry>
-            <box size = "0.5 0.5 0.5" />
+            <sphere radius = "0.5" />
          </geometry>
       </collision>
@@ -1193,9 +1193,9 @@
    <joint name="${namespace}/payload_1_joint" type="floating">
       <parent link="${namespace}/payload_hook" />
-      <child link="${namespace}/payload_1" />
+      <child link="${namespace}/soccer_ball_1" />
       <origin xyz="-1.5 0 0" rpy="0 0 0" />
    </joint>
-   <gazebo reference="${namespace}/payload_1">
-      <material>Gazebo/Yellow</material>
+   <gazebo reference="${namespace}/soccer_ball_1">
+      <material>Gazebo/White</material>
       <mu1>0.2</mu1>
       <mu2>0.2</mu2>
@@ -1207,5 +1207,5 @@
          <robotNamespace>${namespace}</robotNamespace>
          <joint>${namespace}/payload_1_joint</joint>
-         <payload>${namespace}/payload_1</payload>
+         <payload>${namespace}/soccer_ball_1</payload>
          <parent>${namespace}/payload_hook</parent>
          <proxRec>true</proxRec>
@@ -1213,10 +1213,11 @@
          <hoistPosParent>-1.5 0 0</hoistPosParent>
          <hoistPosPayload>0 0 0</hoistPosPayload>
-         <pickupWorldPosPayload>256.65 43.54 80</pickupWorldPosPayload>
+         <pickupWorldPosPayload>22 -306 22.5</pickupWorldPosPayload>
          <initialState>3</initialState> <!-- 0: attached, 1: falling, 2: teleporting, 3: resting @ pickup pos-->
          <dropTopic>drop_1</dropTopic>
-      </plugin>
-   </gazebo>
-   <link name="${namespace}/payload_2">
+         <payloadTrackingTopic>soccer_ball_1</payloadTrackingTopic>
+      </plugin>
+   </gazebo>
+   <link name="${namespace}/soccer_ball_2">
       <inertial>
          <origin xyz="0 0 0" rpy="0 0 0" />
@@ -1227,5 +1228,5 @@
          <origin xyz="0 0 0" rpy="0 0 0" />
          <geometry>
-            <box size = "0.5 0.5 0.5" />
+            <sphere radius = "0.5" />
          </geometry>
       </visual>
@@ -1233,5 +1234,5 @@
          <origin xyz="0 0 0" rpy="0 0 0" />
          <geometry>
-            <box size = "0.5 0.5 0.5" />
+            <sphere radius = "0.5" />
          </geometry>
       </collision>
@@ -1239,8 +1240,50 @@
    <joint name="${namespace}/payload_2_joint" type="floating">
       <parent link="${namespace}/payload_hook" />
-      <child link="${namespace}/payload_2" />
+      <child link="${namespace}/soccer_ball_2" />
       <origin xyz="-1.5 0 0" rpy="0 0 0" />
    </joint>
-   <gazebo reference="${namespace}/payload_2">
+   <gazebo reference="${namespace}/soccer_ball_2">
+      <material>Gazebo/White</material>
+      <mu1>0.2</mu1>
+      <mu2>0.2</mu2>
+      <kp>10000</kp>
+      <kd>1</kd>
+   </gazebo>
+   <gazebo>
+      <plugin filename="librotors_gazebo_payload_plugin.so" name="payload_plugin_1">
+         <robotNamespace>${namespace}</robotNamespace>
+         <joint>${namespace}/payload_2_joint</joint>
+         <payload>${namespace}/soccer_ball_2</payload>
+         <parent>${namespace}/payload_hook</parent>
+         <proxRec>true</proxRec>
+         <radiusRec>5</radiusRec>
+         <hoistPosParent>-1.5 0 0</hoistPosParent>
+         <hoistPosPayload>0 0 0</hoistPosPayload>
+         <pickupWorldPosPayload>-49 -328 22.5</pickupWorldPosPayload>
+         <initialState>3</initialState> <!-- 0: attached, 1: falling, 2: teleporting, 3: resting @ pickup pos-->
+         <dropTopic>drop_1</dropTopic>
+         <payloadTrackingTopic>soccer_ball_2</payloadTrackingTopic>
+      </plugin>
+   </gazebo>
+   <link name="${namespace}/steak_1">
+      <inertial>
+         <origin xyz="0 0 0" rpy="0 0 0" />
+         <mass value="0.25" />
+         <xacro:sphere_inertia r="0.05" mass="0.25" />
+      </inertial>
+      <visual>
+         <origin xyz="0 0 0" rpy="0 0 0" />
+         <geometry>
+           <mesh filename="package://rotors_gazebo/models/fw_challenge/meshes/fw_challenge_grill_steak_a.stl" scale="1 1 1" />
+         </geometry>
+      </visual>
+      <collision>
+         <origin xyz="0 0 0" rpy="0 0 0" />
+         <geometry>
+            <box size = "0.5 0.5 0.5" />
+         </geometry>
+      </collision>
+   </link>
+   <gazebo reference="${namespace}/steak_1">
       <material>Gazebo/Red</material>
       <mu1>0.2</mu1>
@@ -1249,9 +1292,50 @@
       <kd>1</kd>
    </gazebo>
+   <joint name="${namespace}/steak_vis_ab_1_joint" type="fixed">
+      <parent link="${namespace}/steak_1" />
+      <child link="${namespace}/steak_vis_b_1" />
+   </joint>
+   <link name="${namespace}/steak_vis_b_1">
+      <inertial>
+         <mass value="0.001" />
+         <xacro:box_inertia x="0.001" y="0.001" z="0.001" mass="0.001" />
+      </inertial>
+      <visual>
+         <geometry>
+            <mesh filename="package://rotors_gazebo/models/fw_challenge/meshes/fw_challenge_grill_steak_b.stl" scale="1 1 1" />
+         </geometry>
+      </visual>
+   </link>
+   <gazebo reference="${namespace}/steak_vis_b_1">
+      <material>Gazebo/White</material>
+   </gazebo>
+   <joint name="${namespace}/steak_vis_bc_1_joint" type="fixed">
+      <parent link="${namespace}/steak_vis_b_1" />
+      <child link="${namespace}/steak_vis_c_1" />
+   </joint>
+   <link name="${namespace}/steak_vis_c_1">
+      <inertial>
+         <mass value="0.001" />
+         <xacro:box_inertia x="0.001" y="0.001" z="0.001" mass="0.001" />
+      </inertial>
+      <visual>
+         <geometry>
+            <mesh filename="package://rotors_gazebo/models/fw_challenge/meshes/fw_challenge_grill_steak_c.stl" scale="1 1 1" />
+         </geometry>
+      </visual>
+   </link>
+   <gazebo reference="${namespace}/steak_vis_c_1">
+      <material>Gazebo/Red</material>
+   </gazebo>
+   <joint name="${namespace}/payload_3_joint" type="floating">
+      <parent link="${namespace}/payload_hook" />
+      <child link="${namespace}/steak_1" />
+      <origin xyz="-1.5 0 0" rpy="0 0 0" />
+   </joint>
    <gazebo>
       <plugin filename="librotors_gazebo_payload_plugin.so" name="payload_plugin_1">
          <robotNamespace>${namespace}</robotNamespace>
-         <joint>${namespace}/payload_2_joint</joint>
-         <payload>${namespace}/payload_2</payload>
+         <joint>${namespace}/payload_3_joint</joint>
+         <payload>${namespace}/steak_1</payload>
          <parent>${namespace}/payload_hook</parent>
          <proxRec>true</proxRec>
@@ -1259,53 +1343,8 @@
          <hoistPosParent>-1.5 0 0</hoistPosParent>
          <hoistPosPayload>0 0 0</hoistPosPayload>
-         <pickupWorldPosPayload>246.65 38.54 80</pickupWorldPosPayload>
+         <pickupWorldPosPayload>251.65 43.54 80</pickupWorldPosPayload>
          <initialState>3</initialState> <!-- 0: attached, 1: falling, 2: teleporting, 3: resting @ pickup pos-->
          <dropTopic>drop_1</dropTopic>
-      </plugin>
-   </gazebo>
-   <link name="${namespace}/payload_3">
-      <inertial>
-         <origin xyz="0 0 0" rpy="0 0 0" />
-         <mass value="0.25" />
-         <xacro:sphere_inertia r="0.05" mass="0.25" />
-      </inertial>
-      <visual>
-         <origin xyz="0 0 0" rpy="0 0 0" />
-         <geometry>
-            <box size = "0.5 0.5 0.5" />
-         </geometry>
-      </visual>
-      <collision>
-         <origin xyz="0 0 0" rpy="0 0 0" />
-         <geometry>
-            <box size = "0.5 0.5 0.5" />
-         </geometry>
-      </collision>
-   </link>
-   <joint name="${namespace}/payload_3_joint" type="floating">
-      <parent link="${namespace}/payload_hook" />
-      <child link="${namespace}/payload_3" />
-      <origin xyz="-1.5 0 0" rpy="0 0 0" />
-   </joint>
-   <gazebo reference="${namespace}/payload_3">
-      <material>Gazebo/Blue</material>
-      <mu1>0.2</mu1>
-      <mu2>0.2</mu2>
-      <kp>10000</kp>
-      <kd>1</kd>
-   </gazebo>
-   <gazebo>
-      <plugin filename="librotors_gazebo_payload_plugin.so" name="payload_plugin_1">
-         <robotNamespace>${namespace}</robotNamespace>
-         <joint>${namespace}/payload_3_joint</joint>
-         <payload>${namespace}/payload_3</payload>
-         <parent>${namespace}/payload_hook</parent>
-         <proxRec>true</proxRec>
-         <radiusRec>5</radiusRec>
-         <hoistPosParent>-1.5 0 0</hoistPosParent>
-         <hoistPosPayload>0 0 0</hoistPosPayload>
-         <pickupWorldPosPayload>246.65 48.54 80</pickupWorldPosPayload>
-         <initialState>3</initialState> <!-- 0: attached, 1: falling, 2: teleporting, 3: resting @ pickup pos-->
-         <dropTopic>drop_1</dropTopic>
+         <payloadTrackingTopic>steak_1</payloadTrackingTopic>
       </plugin>
    </gazebo>
@@ -1500,5 +1539,5 @@
          <qgc_udp_port>14550</qgc_udp_port>
          <hil_mode>true</hil_mode>
-         <hil_state_level>false</hil_state_level>
+         <hil_state_level>true</hil_state_level>
          <enable_lockstep>false</enable_lockstep>
          <use_tcp>false</use_tcp>
