Commit message: Add windturbine model and cylinder markers on NIV1 model

File: rotors_description/urdf/multirotor_base.xacro (robot description, xacro)
@@ -144,5 +144,5 @@
     <link name="${robot_namespace}/support_${support_number}">
       <inertial>
-        <mass value="0.001" /> <!-- [kg] -->
+        <mass value="0.1" /> [kg]
         <xacro:insert_block name="inertia" />
       </inertial>
@@ -154,5 +154,5 @@
       <collision>
         <geometry>
-          <cylinder length="0.2" radius="0.01" /> <!-- [m] -->
+          <cylinder length="0.1" radius="0.01" /> <!-- [m] -->
         </geometry>
       </collision>
@@ -162,3 +162,33 @@
     </gazebo>
   </xacro:macro>
+  <xacro:macro name="cmarker"
+    params="robot_namespace suffix parent cmarker_number color *origin *inertia">
+    <joint name="${robot_namespace}/cmarker_${cmarker_number}_joint" type="continuous">
+      <xacro:insert_block name="origin" />
+      <axis xyz="0 0 1" />
+      <parent link="${parent}" />
+      <child link="${robot_namespace}/cmarker_${cmarker_number}" />
+    </joint>
+    <link name="${robot_namespace}/cmarker_${cmarker_number}">
+      <inertial>
+        <mass value="0.00001" /> <!-- [kg] -->
+        <xacro:insert_block name="inertia" />
+      </inertial>
+      <visual>
+        <geometry>
+          <cylinder length="0.2" radius="0.018"/> --> <!-- [m] -->
+        </geometry>
+      </visual>
+      <!--
+      <collision>
+        <geometry>
+          <cylinder length="0.2" radius="0.01" />
+        </geometry>
+      </collision>
+      -->
+    </link>
+    <gazebo reference="${robot_namespace}/cmarker_${cmarker_number}">
+      <material>Gazebo/${color}</material>
+    </gazebo>
+  </xacro:macro>
 </robot>

File: rotors_description/urdf/niv1.xacro (robot description, xacro)
@@ -23,18 +23,17 @@
   <xacro:property name="mesh_file" value="package://rotors_description/meshes/niv1_body.dae" />
   <xacro:property name="mass" value="12" /> <!-- [kg] -->
-  <xacro:property name="body_width" value="0.05" /> <!-- [m] -->
-  <xacro:property name="body_height" value="0.05" /> <!-- [m] -->
+  <xacro:property name="body_width" value="0.2" /> <!-- [m] -->
+  <xacro:property name="body_height" value="0.3" /> <!-- [m] -->
   <xacro:property name="mass_rotor" value="0.2" /> <!-- [kg] -->
   <xacro:property name="arm_length" value="0.636" /> <!-- [m] -->
   <xacro:property name="rotor_offset_top" value="0.053" /> <!-- [m] -->
+  <xacro:property name="support_offset_top" value="-0.12" /> <!-- [m] -->
+  <xacro:property name="cmarker_offset_top" value="0.018" /> <!-- [m] -->
   <xacro:property name="radius_rotor" value="0.3" /> <!-- [m] -->
   <xacro:property name="motor_constant_for_ros_sim" value="8.54858e-05" /> <!-- [kg m/s^2]  force = real_motor_velocity * real_motor_velocity * motor_constant_-->
   <xacro:property name="motor_constant" value="1.2e-04" /> <!-- [kg m/s^2]  force = real_motor_velocity * real_motor_velocity * motor_constant_-->
   <xacro:property name="moment_constant" value="0.025" /> <!-- [m] math::Vector3 drag_torque(0, 0, -turning_direction_ * force * moment_constant_); -->
-  <xacro:property name="moment_constan_org" value="0.025" /> <!-- [m] math::Vector3 drag_torque(0, 0, -turning_direction_ * force * moment_constant_); -->
-  <xacro:property name="time_constant_up_org" value="0.0125" /> <!-- [s] -->
-  <xacro:property name="time_constant_down_org" value="0.025" /> <!-- [s] -->
-  <xacro:property name="time_constant_up" value="0.00001" /> <!-- [s] -->
-  <xacro:property name="time_constant_down" value="0.00001" /> <!-- [s] -->
+  <xacro:property name="time_constant_up" value="0.00125" /> <!-- [s] -->
+  <xacro:property name="time_constant_down" value="0.0025" /> <!-- [s] -->
   <xacro:property name="max_rot_velocity" value="1838" /> <!-- [rad/s] -->
   <xacro:property name="rotor_pos_x" value="0.45" />
@@ -59,4 +58,8 @@
     <xacro:box_inertia x="0.03" y="0.03" z="0.2" mass="0.001" />
   </xacro:property>
+  <xacro:property name="cmarker_inertia">
+    <!-- <xacro:box_inertia x="${radius_rotor}" y="0.015" z="0.003" mass="${mass_rotor*rotor_velocity_slowdown_sim}" /> -->
+    <xacro:box_inertia x="0.03" y="0.03" z="0.2" mass="0.001" />
+  </xacro:property>
   <!-- Included URDF Files -->
   <xacro:include filename="$(find rotors_description)/urdf/multirotor_base.xacro" />
@@ -162,6 +165,6 @@
     support_number="0"
     color="Grey">
-     <origin xyz="${rotor_pos_x} -${rotor_pos_y} ${rotor_offset_top-0.2}" rpy="0 0 0" />
-    <xacro:insert_block name="rotor_inertia" />
+     <origin xyz="${rotor_pos_x} -${rotor_pos_y} ${support_offset_top}" rpy="0 0 0" />
+    <xacro:insert_block name="support_inertia" />
   </xacro:support>
   <xacro:support
@@ -171,6 +174,6 @@
     support_number="1"
     color="Grey">
-    <origin xyz="${rotor_pos_x} ${rotor_pos_y} ${rotor_offset_top-0.2}" rpy="0 0 0" />
-    <xacro:insert_block name="rotor_inertia" />
+    <origin xyz="${rotor_pos_x} ${rotor_pos_y} ${support_offset_top}" rpy="0 0 0" />
+    <xacro:insert_block name="support_inertia" />
   </xacro:support>
   <xacro:support robot_namespace="${namespace}"
@@ -179,5 +182,5 @@
     support_number="2"
     color="Grey">
-    <origin xyz="-${rotor_pos_x} ${rotor_pos_y} ${rotor_offset_top-0.2}" rpy="0 0 0" />
+    <origin xyz="-${rotor_pos_x} ${rotor_pos_y} ${support_offset_top}" rpy="0 0 0" />
     <xacro:insert_block name="support_inertia" />
   </xacro:support>
@@ -187,6 +190,41 @@
     support_number="3"
     color="Grey">
-    <origin xyz="-${rotor_pos_x} -${rotor_pos_y} ${rotor_offset_top-0.2}" rpy="0 0 0" />
-    <xacro:insert_block name="support_inertia" />
-  </xacro:support>
+    <origin xyz="-${rotor_pos_x} -${rotor_pos_y} ${support_offset_top}" rpy="0 0 0" />
+    <xacro:insert_block name="support_inertia" />
+  </xacro:support>
+ <!-- Instantiate cylinder marker -->
+    <xacro:cmarker
+    robot_namespace="${namespace}"
+    suffix="front_right"
+    parent="${namespace}/base_link"
+    cmarker_number="0"
+    color="Red">
+    <origin xyz="${rotor_pos_x/2} -${rotor_pos_y} ${cmarker_offset_top}" rpy="0 ${pi/2} 0" />
+    <xacro:insert_block name="cmarker_inertia" />
+  </xacro:cmarker>
+  <xacro:cmarker
+    robot_namespace="${namespace}"
+    suffix="front_left"
+    parent="${namespace}/base_link"
+    cmarker_number="1"
+    color="Red">
+    <origin xyz="${rotor_pos_x/2} ${rotor_pos_y} ${cmarker_offset_top}" rpy="0 ${pi/2} 0" />
+    <xacro:insert_block name="cmarker_inertia" />
+  </xacro:cmarker>
+  <xacro:cmarker robot_namespace="${namespace}"
+    suffix="back_left"
+    parent="${namespace}/base_link"
+    cmarker_number="2"
+    color="White">
+    <origin xyz="-${rotor_pos_x/2} ${rotor_pos_y} ${cmarker_offset_top}" rpy="0 ${pi/2} 0" />
+    <xacro:insert_block name="cmarker_inertia" />
+  </xacro:cmarker>
+  <xacro:cmarker robot_namespace="${namespace}"
+    suffix="back_right"
+    parent="${namespace}/base_link"
+    cmarker_number="3"
+    color="White">
+    <origin xyz="-${rotor_pos_x/2} -${rotor_pos_y} ${cmarker_offset_top}" rpy="0 ${pi/2} 0" />
+    <xacro:insert_block name="cmarker_inertia" />
+  </xacro:cmarker>
 </robot>

Commit message: Make firefly unstatic again

File: rotors_description/urdf/multirotor_base.xacro (robot description, xacro)
@@ -34,11 +34,5 @@
   <xacro:macro name="multirotor_base_macro"
     params="robot_namespace mass body_width body_height use_mesh_file mesh_file *inertia">
-<link name="world" />
     <link name="${robot_namespace}/base_link"></link>
-<joint name="world_joint"  type="fixed">
-    <origin xyz="2 0 1.5" rpy="0 0 0" />
-    <parent link="world"/>
-    <child link="${robot_namespace}/base_link"/>
-</joint>
     <joint name="${robot_namespace}/base_joint" type="fixed">
       <origin xyz="0 0 0" rpy="0 0 0" />

Commit message: Fake no rotor collisions

File: rotors_description/urdf/multirotor_base.xacro (robot description, xacro)
@@ -104,7 +104,7 @@
       </visual>
       <collision>
-        <geometry>
-          <cylinder length="0.005" radius="${radius_rotor}" /> <!-- [m] -->
-        </geometry>
+        <!--<geometry>
+          <cylinder length="0.005" radius="${radius_rotor}" /> <!- [m] ->
+        </geometry>-->
       </collision>
     </link>

Commit message: further parametrization of the lidar models

File: rotors_description/urdf/multirotor_base.xacro (robot description, xacro)
@@ -30,4 +30,37 @@
       <xacro:box_inertia x="${x}" y="${y}" z="${z}" mass="${mass}" />
     </inertial>
+  </xacro:macro>
+  <!-- Macro for the inertia of a cylinder -->
+  <xacro:macro name="cylinder_inertia" params="radius length mass">
+    <inertia ixx="${(mass * (3.0*radius*radius + length*length)) / 12.0}" ixy="0" ixz="0"
+             iyy="${(mass * (3.0*radius*radius + length*length)) / 12.0}" iyz="0"
+             izz="${0.5 * mass * (radius*radius)}"/>
+  </xacro:macro>
+  <!-- Macro for the inertial properties of a cylinder -->
+  <xacro:macro name="cylinder_inertial" params="radius length mass *origin">
+    <inertial>
+      <mass value="${mass}"/>
+      <xacro:insert_block name="origin" />
+      <xacro:cylinder_inertia radius="${radius}" length="${length}" mass="${mass}" />
+    </inertial>
+  </xacro:macro>
+  <xacro:macro name="cylinder_link_complete" params="link_name radius length mass *origin">
+    <link name="${link_name}">
+      <xacro:cylinder_inertial radius="${radius}" length="${length}" mass="${mass}" >
+        <xacro:insert_block name="origin" />
+      </xacro:cylinder_inertial>
+      <collision name="${link_name}_collision">
+        <xacro:insert_block name="origin" />
+        <geometry>
+          <cylinder length="${length}" radius="${radius}"/>
+        </geometry>
+      </collision>
+      <visual name="${link_name}_visual">
+        <xacro:insert_block name="origin" />
+        <geometry>
+          <cylinder length="${length}" radius="${radius}"/>
+        </geometry>
+      </visual>
+    </link>
   </xacro:macro>
   <!-- Main multirotor link -->

File: rotors_description/urdf/ouster_os1.urdf.xacro (robot description, xacro)
@@ -8,4 +8,5 @@
   <xacro:property name="r2" value="0.0425"/>
   <xacro:property name="l2" value="0.0305"/>
+  <xacro:include filename="$(find rotors_description)/urdf/multirotor_base.xacro" />
   <xacro:macro name="OS-1" params="*origin parent:=world sensor_name:=os1 topic:=/os1_points horizontal_angular_resolution_deg:=0.18 spin_frequency_hz:=10 lidar_base_frame:=os1_base lidar_points_frame:=os1_top namespace:=example min_range:=0.05">
     <gazebo>
@@ -22,25 +23,8 @@
       <child link="${namespace}/${lidar_base_frame}"/>
     </joint>
-    <link name="${namespace}/${lidar_base_frame}">
-      <inertial>
-        <mass value="${m1}"/>
+    <xacro:cylinder_link_complete link_name="${namespace}/${lidar_base_frame}"
+      mass="${m1}" length="${l1}" radius="${r1}">
         <origin rpy="0 0 0" xyz="0 0 ${l1*0.5}"/>
-        <inertia ixx="${(m1 * (3.0*r1*r1 + l1*l1)) / 12.0}" ixy="0" ixz="0"
-                 iyy="${(m1 * (3.0*r1*r1 + l1*l1)) / 12.0}" iyz="0"
-                 izz="${0.5 * m1 * (r1*r1)}"/>
-      </inertial>
-      <collision name="${namespace}/${lidar_base_frame}_collision">
-        <origin rpy="0 0 0" xyz="0 0 ${l1*0.5}"/>
-        <geometry>
-          <cylinder length="${l1}" radius="${r1}"/>
-        </geometry>
-      </collision>
-      <visual name="${namespace}/${lidar_base_frame}_visual">
-        <origin rpy="0 0 0" xyz="0 0 ${l1*0.5}"/>
-        <geometry>
-          <cylinder length="${l1}" radius="${r1}"/>
-        </geometry>
-      </visual>
-    </link>
+    </xacro:cylinder_link_complete>
     <joint name="${namespace}/${sensor_name}_joint" type="continuous">
       <parent link="${namespace}/${lidar_base_frame}"/>
@@ -50,25 +34,8 @@
       <limit effort="100.0" velocity="100.0"/>
     </joint>
-    <link name="${namespace}/${lidar_points_frame}">
-      <inertial>
-        <mass value="${m2}"/>
+    <xacro:cylinder_link_complete link_name="${namespace}/${lidar_points_frame}"
+      mass="${m2}" length="${l2}" radius="${r2}">
         <origin rpy="0 0 0" xyz="0 0 0"/>
-        <inertia ixx="${(m2 * (3.0*r2*r2 + l2*l2)) / 12.0}" ixy="0" ixz="0"
-                 iyy="${(m2 * (3.0*r2*r2 + l2*l2)) / 12.0}" iyz="0"
-                 izz="${0.5 * m2 * (r2*r2)}"/>
-      </inertial>
-      <collision>
-        <origin rpy="0 0 0" xyz="0 0 0"/>
-        <geometry>
-          <cylinder length="${l2}" radius="${r2}"/>
-        </geometry>
-      </collision>
-      <visual name="${namespace}/${lidar_points_frame}_visual">
-        <origin rpy="0 0 0" xyz="0 0 0"/>
-        <geometry>
-          <cylinder length="${l2}" radius="${r2}"/>
-        </geometry>
-      </visual>
-    </link>
+    </xacro:cylinder_link_complete>
     <gazebo reference="${namespace}/${lidar_points_frame}">
       <material>Gazebo/Black</material>
@@ -79,25 +46,8 @@
       <origin rpy="0 0 0" xyz="0 0 ${l1+l2*0.5}"/>
     </joint>
-    <link name="${namespace}/${lidar_base_frame}_hat">
-      <inertial>
-        <mass value="${m1}"/>
+    <xacro:cylinder_link_complete link_name="${namespace}/${lidar_base_frame}_hat"
+      mass="${m1}" length="${l1}" radius="${r1}">
         <origin rpy="0 0 0" xyz="0 0 ${(l1+l2)*0.5}"/>
-        <inertia ixx="${(m1 * (3.0*r1*r1 + l1*l1)) / 12.0}" ixy="0" ixz="0"
-                 iyy="${(m1 * (3.0*r1*r1 + l1*l1)) / 12.0}" iyz="0"
-                 izz="${0.5 * m1 * (r1*r1)}"/>
-      </inertial>
-      <collision>
-        <origin rpy="0 0 0" xyz="0 0 ${(l1+l2)*0.5}"/>
-        <geometry>
-          <cylinder length="${l1}" radius="${r1}"/>
-        </geometry>
-      </collision>
-      <visual>
-        <origin rpy="0 0 0" xyz="0 0 ${(l1+l2)*0.5}"/>
-        <geometry>
-          <cylinder length="${l1}" radius="${r1}"/>
-        </geometry>
-      </visual>
-    </link>
+    </xacro:cylinder_link_complete>
     <gazebo reference="${namespace}/${lidar_points_frame}">
       <!-- Add a ray sensor, and give it a name -->

File: rotors_description/urdf/velodyne_VLP_16.urdf.xacro (robot description, xacro)
@@ -8,4 +8,5 @@
   <xacro:property name="r2" value="0.0516"/>
   <xacro:property name="l2" value="0.0381"/>
+  <xacro:include filename="$(find rotors_description)/urdf/multirotor_base.xacro" />
   <xacro:macro name="VLP-16" params="*origin parent:=world sensor_name:=velodyne topic:=/velodyne_points horizontal_angular_resolution_deg:=1.0 spin_frequency_hz:=0.5 lidar_base_frame:=velodyne_base lidar_points_frame:=velodyne_top namespace:=example min_range:=0.06">
     <gazebo>
@@ -22,25 +23,8 @@
       <child link="${namespace}/${lidar_base_frame}"/>
     </joint>
-    <link name="${namespace}/${lidar_base_frame}">
-      <inertial>
-        <mass value="${m1}"/>
+    <xacro:cylinder_link_complete link_name="${namespace}/${lidar_base_frame}"
+      mass="${m1}" length="${l1}" radius="${r1}">
         <origin rpy="0 0 0" xyz="0 0 ${l1*0.5}"/>
-        <inertia ixx="${(m1 * (3.0*r1*r1 + l1*l1)) / 12.0}" ixy="0" ixz="0"
-                 iyy="${(m1 * (3.0*r1*r1 + l1*l1)) / 12.0}" iyz="0"
-                 izz="${0.5 * m1 * (r1*r1)}"/>
-      </inertial>
-      <collision name="${namespace}/${lidar_base_frame}_collision">
-        <origin rpy="0 0 0" xyz="0 0 ${l1*0.5}"/>
-        <geometry>
-          <cylinder length="${l1}" radius="${r1}"/>
-        </geometry>
-      </collision>
-      <visual name="${namespace}/${lidar_base_frame}_visual">
-        <origin rpy="0 0 0" xyz="0 0 ${l1*0.5}"/>
-        <geometry>
-          <cylinder length="${l1}" radius="${r1}"/>
-        </geometry>
-      </visual>
-    </link>
+    </xacro:cylinder_link_complete>
     <joint name="${namespace}/${sensor_name}_joint" type="continuous">
       <parent link="${namespace}/${lidar_base_frame}"/>
@@ -50,25 +34,8 @@
       <limit effort="100.0" velocity="100.0"/>
     </joint>
-    <link name="${namespace}/${lidar_points_frame}">
-      <inertial>
-        <mass value="${m2}"/>
+    <xacro:cylinder_link_complete link_name="${namespace}/${lidar_points_frame}"
+      mass="${m2}" length="${l2}" radius="${r2}">
         <origin rpy="0 0 0" xyz="0 0 0"/>
-        <inertia ixx="${(m2 * (3.0*r2*r2 + l2*l2)) / 12.0}" ixy="0" ixz="0"
-                 iyy="${(m2 * (3.0*r2*r2 + l2*l2)) / 12.0}" iyz="0"
-                 izz="${0.5 * m2 * (r2*r2)}"/>
-      </inertial>
-      <collision>
-        <origin rpy="0 0 0" xyz="0 0 0"/>
-        <geometry>
-          <cylinder length="${l2}" radius="${r2}"/>
-        </geometry>
-      </collision>
-      <visual name="${namespace}/${lidar_points_frame}_visual">
-        <origin rpy="0 0 0" xyz="0 0 0"/>
-        <geometry>
-          <cylinder length="${l2}" radius="${r2}"/>
-        </geometry>
-      </visual>
-    </link>
+    </xacro:cylinder_link_complete>
     <gazebo reference="${namespace}/${lidar_points_frame}">
       <material>Gazebo/Black</material>
@@ -79,25 +46,8 @@
       <origin rpy="0 0 0" xyz="0 0 ${l1+l2*0.5}"/>
     </joint>
-    <link name="${namespace}/${lidar_base_frame}_hat">
-      <inertial>
-        <mass value="${m1}"/>
+    <xacro:cylinder_link_complete link_name="${namespace}/${lidar_base_frame}_hat"
+      mass="${m1}" length="${l1}" radius="${r1}">
         <origin rpy="0 0 0" xyz="0 0 ${(l1+l2)*0.5}"/>
-        <inertia ixx="${(m1 * (3.0*r1*r1 + l1*l1)) / 12.0}" ixy="0" ixz="0"
-                 iyy="${(m1 * (3.0*r1*r1 + l1*l1)) / 12.0}" iyz="0"
-                 izz="${0.5 * m1 * (r1*r1)}"/>
-      </inertial>
-      <collision>
-        <origin rpy="0 0 0" xyz="0 0 ${(l1+l2)*0.5}"/>
-        <geometry>
-          <cylinder length="${l1}" radius="${r1}"/>
-        </geometry>
-      </collision>
-      <visual>
-        <origin rpy="0 0 0" xyz="0 0 ${(l1+l2)*0.5}"/>
-        <geometry>
-          <cylinder length="${l1}" radius="${r1}"/>
-        </geometry>
-      </visual>
-    </link>
+    </xacro:cylinder_link_complete>
     <gazebo reference="${namespace}/${lidar_points_frame}">
       <!-- Add a ray sensor, and give it a name -->

Commit message: Added plugin for collisions to multirotor_base.xacro

File: rotors_description/urdf/multirotor_base.xacro (robot description, xacro)
@@ -30,4 +30,20 @@
       <xacro:box_inertia x="${x}" y="${y}" z="${z}" mass="${mass}" />
     </inertial>
+  </xacro:macro>
+  <!-- Macro for the collision detection plugin -->
+  <xacro:macro name="collision detection plugin" params="ns link_name">
+  <gazebo reference="${link_name}">
+    <sensor name="${link_name}_contact_sensor" type="contact">
+      <always_on>true</always_on>
+      <contact>
+        <!-- Name of the link + '_collision' : check sdf file for exact name -->
+        <collision>${link_name}_collision</collision>
+      </contact>
+      <plugin name="${link_name}_bumper_plugin" filename="libgazebo_ros_bumper.so">
+        <bumperTopicName>${ns}/plugin_collision</bumperTopicName>
+        <frameName>${link_name}</frameName>
+      </plugin>
+    </sensor>
+  </gazebo>
   </xacro:macro>
   <!-- Main multirotor link -->
@@ -131,4 +147,18 @@
       <material>Gazebo/${color}</material>
     </gazebo>
+    <!-- Contact Sensor for the rotor link -->
+    <gazebo reference="${robot_namespace}/rotor_${motor_number}">
+      <sensor name="rotor_${motor_number}_contact_sensor" type="contact">
+        <always_on>true</always_on>
+        <contact>
+            <!-- Name of the link + '_collision' : check sdf file for exact name -->
+          <collision>${robot_namespace}/rotor_${motor_number}_collision</collision>
+        </contact>
+        <plugin name="${robot_namespace}/rotor_${motor_number}_bumper_plugin" filename="libgazebo_ros_bumper.so">
+          <bumperTopicName>${robot_namespace}/plugin_collision</bumperTopicName>
+          <frameName>${robot_namespace}/rotor_${motor_number}</frameName>
+        </plugin>
+      </sensor>
+    </gazebo>
   </xacro:macro>
 </robot>
