Commit message: add offset

File: rotors_description/urdf/delta_manipulator.xacro (robot description, xacro)
@@ -8,5 +8,5 @@
     <xacro:property name="delta_start_index" default="12" />
     <joint name="mounting_joint" type="fixed">
-        <origin xyz="0 0 ${height_offset}" rpy="0.0 0.0 0.0"/>
+        <origin xyz="0 -0.01 -0.077" rpy="0.0 0.0 0.0"/>
         <parent link="${mounting_link}"/>
         <child link="${delta_namespace}/delta_base_link"/>

Commit message: add costumized B_p_D position

File: rotors_description/urdf/delta_manipulator.xacro (robot description, xacro)
@@ -4,9 +4,11 @@
     <xacro:include filename="$(find rotors_description)/urdf/delta_elements.xacro" />
     <xacro:property name="mounting_link" default="world" />
-    <xacro:property name="height_offset" default="-0.07" />
+    <xacro:property name="x_offset" default="-0.0015" />
+    <xacro:property name="y_offset" default="0.0101" />
+    <xacro:property name="z_offset" default="0.07735" />
     <xacro:property name="delta_namespace" default="${delta_namespace}" />
     <xacro:property name="delta_start_index" default="12" />
     <joint name="mounting_joint" type="fixed">
-        <origin xyz="0 -0.01 -0.077" rpy="0.0 0.0 0.0"/>
+        <origin xyz="${x_offset} ${y_offset} ${z_offset}" rpy="0.0 0.0 0.0"/>
         <parent link="${mounting_link}"/>
         <child link="${delta_namespace}/delta_base_link"/>

Commit message: old offset

File: rotors_description/urdf/delta_manipulator.xacro (robot description, xacro)
@@ -4,7 +4,7 @@
     <xacro:include filename="$(find rotors_description)/urdf/delta_elements.xacro" />
     <xacro:property name="mounting_link" default="world" />
-    <xacro:property name="x_offset" default="-0.0015" />
-    <xacro:property name="y_offset" default="0.0101" />
-    <xacro:property name="z_offset" default="0.07735" />
+    <xacro:property name="x_offset" default="-0.0" />
+    <xacro:property name="y_offset" default="0.0" />
+    <xacro:property name="z_offset" default="0.070" />
     <xacro:property name="delta_namespace" default="${delta_namespace}" />
     <xacro:property name="delta_start_index" default="12" />

Commit message: z offset

File: rotors_description/urdf/delta_manipulator.xacro (robot description, xacro)
@@ -4,11 +4,11 @@
     <xacro:include filename="$(find rotors_description)/urdf/delta_elements.xacro" />
     <xacro:property name="mounting_link" default="world" />
-    <xacro:property name="x_offset" default="-0.0" />
+    <xacro:property name="x_offset" default="0.0" />
     <xacro:property name="y_offset" default="0.0" />
-    <xacro:property name="z_offset" default="0.070" />
+    <xacro:property name="height_offset" default="-0.7" />
     <xacro:property name="delta_namespace" default="${delta_namespace}" />
     <xacro:property name="delta_start_index" default="12" />
     <joint name="mounting_joint" type="fixed">
-        <origin xyz="${x_offset} ${y_offset} ${z_offset}" rpy="0.0 0.0 0.0"/>
+        <origin xyz="${x_offset} ${y_offset} ${height_offset}" rpy="0.0 0.0 0.0"/>
         <parent link="${mounting_link}"/>
         <child link="${delta_namespace}/delta_base_link"/>

Commit message: height offset

File: rotors_description/urdf/delta_manipulator.xacro (robot description, xacro)
@@ -6,5 +6,5 @@
     <xacro:property name="x_offset" default="0.0" />
     <xacro:property name="y_offset" default="0.0" />
-    <xacro:property name="height_offset" default="-0.7" />
+    <xacro:property name="height_offset" default="-0.07" />
     <xacro:property name="delta_namespace" default="${delta_namespace}" />
     <xacro:property name="delta_start_index" default="12" />

Commit message: remove x and y offset from file

File: rotors_description/urdf/delta_manipulator.xacro (robot description, xacro)
@@ -4,11 +4,9 @@
     <xacro:include filename="$(find rotors_description)/urdf/delta_elements.xacro" />
     <xacro:property name="mounting_link" default="world" />
-    <xacro:property name="x_offset" default="0.0" />
-    <xacro:property name="y_offset" default="0.0" />
     <xacro:property name="height_offset" default="-0.07" />
     <xacro:property name="delta_namespace" default="${delta_namespace}" />
     <xacro:property name="delta_start_index" default="12" />
     <joint name="mounting_joint" type="fixed">
-        <origin xyz="${x_offset} ${y_offset} ${height_offset}" rpy="0.0 0.0 0.0"/>
+        <origin xyz="$0.0 0.0 ${height_offset}" rpy="0.0 0.0 0.0"/>
         <parent link="${mounting_link}"/>
         <child link="${delta_namespace}/delta_base_link"/>
