Commit message: link length adapted

File: rotors_description/urdf/delta_elements.xacro (robot description, xacro)
@@ -6,9 +6,9 @@
     <xacro:property name="base_plate_height" value="${0.003}" />
     <xacro:property name="base_plate_mass" value="${0.25}" />
-    <xacro:property name="link_proximal_length" value="${0.1558227}" />
+    <xacro:property name="link_proximal_length" value="${0.156}" />
     <xacro:property name="link_proximal_width" value="${0.019}" />
     <xacro:property name="link_proximal_height" value="${0.010}" />
     <xacro:property name="link_proximal_mass" value="${0.041}" />
-    <xacro:property name="link_distal_length" value="${0.2430566}" />
+    <xacro:property name="link_distal_length" value="${0.24}" />
     <xacro:property name="link_distal_radius" value="${0.0024}" />
     <xacro:property name="link_distal_mass" value="${0.020}" />

Commit message: tool plate radius update

File: rotors_description/urdf/delta_elements.xacro (robot description, xacro)
@@ -17,5 +17,5 @@
     <xacro:property name="link_distal_izz" value="${0.5*link_distal_mass*(link_distal_radius+link_distal_radius)}" />
     <xacro:property name="tool_plate_height" value="${0.01}" />
-    <xacro:property name="tool_plate_radius" value="${0.03}" />
+    <xacro:property name="tool_plate_radius" value="${0.038}" />
     <xacro:property name="tool_plate_mass" value="${0.0233}" />
     <xacro:property name="tool_plate_ixx" value="${0.833*tool_plate_mass*(3.0*tool_plate_radius*tool_plate_radius+tool_plate_height*tool_plate_height)}" />
