Commit message: Improved collision for the overactuated base. Split the collision boxes in two. One at the wheels and one at the body. Now the collision box doesn't go so far above the actual body. Hardcoded values. Still need to parametrize..

File: rotors_description/urdf/overactuated_base.xacro (robot description, xacro)
@@ -44,7 +44,13 @@
       </visual>
       <collision>
-        <origin xyz="0 0 0" rpy="0 0 0" />
-        <geometry>
-          <box size="${body_width} ${body_width} ${body_height}" /> <!-- [m] [m] [m] -->
+        <origin xyz="0 0 0.0" rpy="0 0 0" />
+        <geometry>
+          <box size="${body_width} ${body_width} 0.2" /> <!-- [m] [m] [m] -->
+        </geometry>
+      </collision>
+      <collision>
+        <origin xyz="0 0 -0.23" rpy="0 0 0" />
+        <geometry>
+          <box size="0.35 0.35 0.01" /> <!-- [m] [m] [m] -->
         </geometry>
       </collision>

Commit message: removed collision box of body so that end-effector on springs doesn't get caught in there at initialization

File: rotors_description/urdf/overactuated_base.xacro (robot description, xacro)
@@ -43,10 +43,10 @@
         </geometry>
       </visual>
-      <collision>
+      <!-- <collision>
         <origin xyz="0 0 0.0" rpy="0 0 0" />
         <geometry>
-          <box size="${body_width} ${body_width} 0.2" /> <!-- [m] [m] [m] -->
-        </geometry>
-      </collision>
+          <box size="${body_width} ${body_width} 0.2" />
+        </geometry>
+      </collision> -->
       <collision>
         <origin xyz="0 0 -0.23" rpy="0 0 0" />
