Commit message: Added parameter to check if gazebo should use mesh for collision

File: rotors_description/urdf/omav3.xacro (robot description, xacro)
@@ -25,4 +25,5 @@
     <xacro:property name="use_mesh_file_rotor_unit" value="true"/>
     <xacro:property name="mesh_file_core" value="package://rotors_description/meshes/omav/omav3_base.stl"/>
+    <xacro:property name="use_collision_mesh_file" value="true" />
     <xacro:property name="mesh_file_core_collision" value="package://rotors_description/meshes/omav/omav3_base.stl"/>
     <xacro:property name="mesh_file_tilt_unit" value="package://rotors_description/meshes/omav/omav3_tiltarm.stl"/>

File: rotors_description/urdf/omav_snippets.xacro (robot description, xacro)
@@ -19,5 +19,5 @@
   <xacro:include filename="$(find rotors_description)/urdf/multirotor_base.xacro"/>
   <xacro:macro name="omav_base_macro"
-    params="robot_namespace mass body_width body_height use_mesh_file mesh_file collision_mesh_file *origin *inertia *inertia_origin">
+    params="robot_namespace mass body_width body_height use_mesh_file mesh_file use_collision_mesh_file collision_mesh_file *origin *inertia *inertia_origin">
     <link name="${robot_namespace}/base_link"></link>
     <joint name="${robot_namespace}/base_joint" type="fixed">
@@ -46,8 +46,8 @@
         <origin xyz="0 0 0" rpy="0 0 0" />
         <geometry>
-          <xacro:if value="${use_mesh_file}">
+          <xacro:if value="${use_collision_mesh_file}">
             <mesh filename="${collision_mesh_file}" scale="1 1 1" />
           </xacro:if>
-          <xacro:unless value="${use_mesh_file}">
+          <xacro:unless value="${use_collision_mesh_file}">
             <box size="${body_width} ${body_width} ${body_height}"/> <!-- [m] [m] [m] -->
           </xacro:unless>
