Commit message: also adapt firefly moment constant

File: rotors_description/urdf/firefly.xacro (robot description, xacro)
@@ -29,6 +29,6 @@
   <xacro:property name="rotor_offset_top" value="0.037" /> <!-- [m] -->
   <xacro:property name="radius_rotor" value="0.1" /> <!-- [m] -->
-  <xacro:property name="motor_constant" value="8.54858e-06" /> <!-- [kg m/s^2] -->
-  <xacro:property name="moment_constant" value="0.016" /> <!-- [m] -->
+  <xacro:property name="motor_constant" value="8.54858e-06" /> <!-- [kg m] -->
+  <xacro:property name="moment_constant" value="1.3677728e-07" /> <!-- [kg m^2] -->
   <xacro:property name="time_constant_up" value="0.025" /> <!-- [s] -->
   <xacro:property name="time_constant_down" value="0.025" /> <!-- [s] -->

Commit message: Instantaneous motor commands

File: rotors_description/urdf/firefly.xacro (robot description, xacro)
@@ -31,6 +31,6 @@
   <xacro:property name="motor_constant" value="8.54858e-06" /> <!-- [kg m] -->
   <xacro:property name="moment_constant" value="1.3677728e-07" /> <!-- [kg m^2] -->
-  <xacro:property name="time_constant_up" value="0.025" /> <!-- [s] -->
-  <xacro:property name="time_constant_down" value="0.025" /> <!-- [s] -->
+  <xacro:property name="time_constant_up" value="0.0" /> <!-- [s] -->
+  <xacro:property name="time_constant_down" value="0.0" /> <!-- [s] -->
   <xacro:property name="max_rot_velocity" value="838" /> <!-- [rad/s] -->
   <xacro:property name="sin30" value="0.5" />

Commit message: added main body drag

File: rotors_description/urdf/firefly.xacro (robot description, xacro)
@@ -38,4 +38,5 @@
   <xacro:property name="rotor_drag_coefficient" value="0.0176" />
   <xacro:property name="rolling_moment_coefficient" value="0.000001" />
+  <xacro:property name="main_body_drag_coefficient" value="0.002 0.002 0.0" />
   <!-- Property Blocks -->
   <xacro:property name="body_inertia">
@@ -51,4 +52,5 @@
   <xacro:multirotor_base_macro
     robot_namespace="${namespace}"
+    main_body_drag_coefficient="${main_body_drag_coefficient}"
     mass="${mass}"
     body_width="${body_width}"

File: rotors_description/urdf/multirotor_base.xacro (robot description, xacro)
@@ -33,5 +33,5 @@
   <!-- Main multirotor link -->
   <xacro:macro name="multirotor_base_macro"
-    params="robot_namespace mass body_width body_height use_mesh_file mesh_file *inertia">
+    params="robot_namespace main_body_drag_coefficient mass body_width body_height use_mesh_file mesh_file *inertia">
     <link name="${robot_namespace}/base_link"></link>
     <joint name="${robot_namespace}/base_joint" type="fixed">
@@ -70,4 +70,5 @@
         <linkName>${robot_namespace}/base_link</linkName>
         <rotorVelocitySlowdownSim>${rotor_velocity_slowdown_sim}</rotorVelocitySlowdownSim>
+        <mainBodyDragCoefficient>${main_body_drag_coefficient}</mainBodyDragCoefficient>
       </plugin>
     </gazebo>

Commit message: added noise on rotor forces and torques

File: rotors_description/urdf/firefly.xacro (robot description, xacro)
@@ -38,4 +38,6 @@
   <xacro:property name="rotor_drag_coefficient" value="0.0176" />
   <xacro:property name="rolling_moment_coefficient" value="0.000001" />
+  <xacro:property name="forces_noise_density" value="0.01 0.01 0.01" />
+  <xacro:property name="moments_noise_density" value="0.004 0.004 0.002" />
   <xacro:property name="main_body_drag_coefficient" value="0.002 0.002 0.0" />
   <!-- Property Blocks -->
@@ -77,4 +79,6 @@
     rotor_drag_coefficient="${rotor_drag_coefficient}"
     rolling_moment_coefficient="${rolling_moment_coefficient}"
+    forces_noise_density="${forces_noise_density}"
+    moments_noise_density="${moments_noise_density}"
     color="Red"
     use_own_mesh="false"
@@ -98,4 +102,6 @@
     rotor_drag_coefficient="${rotor_drag_coefficient}"
     rolling_moment_coefficient="${rolling_moment_coefficient}"
+    forces_noise_density="${forces_noise_density}"
+    moments_noise_density="${moments_noise_density}"
     color="Blue"
     use_own_mesh="false"
@@ -118,4 +124,6 @@
     rotor_drag_coefficient="${rotor_drag_coefficient}"
     rolling_moment_coefficient="${rolling_moment_coefficient}"
+    forces_noise_density="${forces_noise_density}"
+    moments_noise_density="${moments_noise_density}"
     color="Blue"
     use_own_mesh="false"
@@ -138,4 +146,6 @@
     rotor_drag_coefficient="${rotor_drag_coefficient}"
     rolling_moment_coefficient="${rolling_moment_coefficient}"
+    forces_noise_density="${forces_noise_density}"
+    moments_noise_density="${moments_noise_density}"
     color="Blue"
     use_own_mesh="false"
@@ -159,4 +169,6 @@
     rotor_drag_coefficient="${rotor_drag_coefficient}"
     rolling_moment_coefficient="${rolling_moment_coefficient}"
+    forces_noise_density="${forces_noise_density}"
+    moments_noise_density="${moments_noise_density}"
     color="Blue"
     use_own_mesh="false"
@@ -180,4 +192,6 @@
     rotor_drag_coefficient="${rotor_drag_coefficient}"
     rolling_moment_coefficient="${rolling_moment_coefficient}"
+    forces_noise_density="${forces_noise_density}"
+    moments_noise_density="${moments_noise_density}"
     color="Red"
     use_own_mesh="false"

File: rotors_description/urdf/multirotor_base.xacro (robot description, xacro)
@@ -76,5 +76,5 @@
   <!-- Rotor joint and link -->
   <xacro:macro name="vertical_rotor"
-    params="robot_namespace suffix direction motor_constant moment_constant parent mass_rotor radius_rotor time_constant_up time_constant_down max_rot_velocity motor_number rotor_drag_coefficient rolling_moment_coefficient color use_own_mesh mesh *origin *inertia">
+    params="robot_namespace suffix direction motor_constant moment_constant parent mass_rotor radius_rotor time_constant_up time_constant_down max_rot_velocity motor_number rotor_drag_coefficient rolling_moment_coefficient forces_noise_density moments_noise_density color use_own_mesh mesh *origin *inertia">
     <joint name="${robot_namespace}/rotor_${motor_number}_joint" type="continuous">
       <xacro:insert_block name="origin" />
@@ -127,4 +127,6 @@
         <motorSpeedPubTopic>motor_speed/${motor_number}</motorSpeedPubTopic>
         <rotorVelocitySlowdownSim>${rotor_velocity_slowdown_sim}</rotorVelocitySlowdownSim>
+        <forcesNoiseDensity>${forces_noise_density}</forcesNoiseDensity>
+        <momentsNoiseDensity>${moments_noise_density}</momentsNoiseDensity>
       </plugin>
     </gazebo>

Commit message: final version?

File: rotors_description/urdf/firefly.xacro (robot description, xacro)
@@ -25,5 +25,5 @@
   <xacro:property name="body_width" value="0.1" /> <!-- [m] -->
   <xacro:property name="body_height" value="0.16" /> <!-- [m] -->
-  <xacro:property name="mass_rotor" value="0.005" /> <!-- [kg] -->
+  <xacro:property name="mass_rotor" value="0.006" /> <!-- [kg] -->
   <xacro:property name="arm_length" value="0.215" /> <!-- [m] -->
   <xacro:property name="rotor_offset_top" value="0.037" /> <!-- [m] -->
@@ -39,8 +39,9 @@
   <xacro:property name="rolling_moment_coefficient" value="0.000001" />
   <!--xacro:property name="forces_noise_density" value="0.01 0.01 0.01" /> -->
-  <!--xacro:property name="moments_noise_density" value="0.004 0.004 0.002" /> -->
-  <xacro:property name="forces_noise_density" value="0.01 0.01 0.01" />
-  <xacro:property name="moments_noise_density" value="0.004 0.004 0.004" />
-  <xacro:property name="main_body_drag_coefficient" value="0.002 0.002 0.0" />
+  <!--xacro:property name="moments_noise_density" value="0.001 0.001 0.001" /> -->
+  <xacro:property name="forces_noise_density" value="0.0 0.0 0.0" />
+  <xacro:property name="moments_noise_density" value="0.0 0.0 0.0" />
+  <!--xacro:property name="main_body_drag_coefficient" value="0.0189 0.0189 0.0" /> -->
+  <xacro:property name="main_body_drag_coefficient" value="0.0 0.0 0.0" />
   <!-- Property Blocks -->
   <xacro:property name="body_inertia">
@@ -49,6 +50,6 @@
   <!-- inertia of a single rotor, assuming it is a cuboid. Height=3mm, width=15mm -->
   <xacro:property name="rotor_inertia">
-    <!-- <xacro:box_inertia x="${2 * radius_rotor}" y="0.015" z="0.003" mass="${mass_rotor*rotor_velocity_slowdown_sim}" /> -->
-    <xacro:rotor_disk_inertia rotor_velocity_slowdown_sim="${rotor_velocity_slowdown_sim}" radius="${radius_rotor}" mass="${mass_rotor}" />
+    <xacro:box_inertia x="${2 * radius_rotor}" y="0.015" z="0.003" mass="${mass_rotor*rotor_velocity_slowdown_sim}" />
+  <!--   <xacro:rotor_disk_inertia rotor_velocity_slowdown_sim="${rotor_velocity_slowdown_sim}" radius="${radius_rotor}" mass="${mass_rotor}" /> -->
   </xacro:property>
   <!-- Included URDF Files -->

Commit message: correct model for paper

File: rotors_description/urdf/firefly.xacro (robot description, xacro)
@@ -39,9 +39,8 @@
   <xacro:property name="rolling_moment_coefficient" value="0.000001" />
   <!--xacro:property name="forces_noise_density" value="0.01 0.01 0.01" /> -->
-  <!--xacro:property name="moments_noise_density" value="0.001 0.001 0.001" /> -->
-  <xacro:property name="forces_noise_density" value="0.0 0.0 0.0" />
-  <xacro:property name="moments_noise_density" value="0.0 0.0 0.0" />
-  <!--xacro:property name="main_body_drag_coefficient" value="0.0189 0.0189 0.0" /> -->
-  <xacro:property name="main_body_drag_coefficient" value="0.0 0.0 0.0" />
+  <!--xacro:property name="moments_noise_density" value="0.004 0.004 0.002" /> -->
+  <xacro:property name="forces_noise_density" value="0.01 0.01 0.01" />
+  <xacro:property name="moments_noise_density" value="0.001 0.001 0.001" />
+  <xacro:property name="main_body_drag_coefficient" value="0.0189 0.0189 0.0" />
   <!-- Property Blocks -->
   <xacro:property name="body_inertia">
@@ -50,6 +49,6 @@
   <!-- inertia of a single rotor, assuming it is a cuboid. Height=3mm, width=15mm -->
   <xacro:property name="rotor_inertia">
-    <xacro:box_inertia x="${2 * radius_rotor}" y="0.015" z="0.003" mass="${mass_rotor*rotor_velocity_slowdown_sim}" />
-  <!--   <xacro:rotor_disk_inertia rotor_velocity_slowdown_sim="${rotor_velocity_slowdown_sim}" radius="${radius_rotor}" mass="${mass_rotor}" /> -->
+    <!-- <xacro:box_inertia x="${2 * radius_rotor}" y="0.015" z="0.003" mass="${mass_rotor*rotor_velocity_slowdown_sim}" /> -->
+    <xacro:rotor_disk_inertia rotor_velocity_slowdown_sim="${rotor_velocity_slowdown_sim}" radius="${radius_rotor}" mass="${mass_rotor}" />
   </xacro:property>
   <!-- Included URDF Files -->

Commit message: final values

File: rotors_description/urdf/firefly.xacro (robot description, xacro)
@@ -22,5 +22,5 @@
   <xacro:property name="use_mesh_file" value="true" />
   <xacro:property name="mesh_file" value="package://rotors_description/meshes/firefly.dae" />
-  <xacro:property name="mass" value="1.5" /> <!-- [kg] -->
+  <xacro:property name="mass" value="1.62697" /> <!-- [kg] -->
   <xacro:property name="body_width" value="0.1" /> <!-- [m] -->
   <xacro:property name="body_height" value="0.16" /> <!-- [m] -->
@@ -29,6 +29,6 @@
   <xacro:property name="rotor_offset_top" value="0.037" /> <!-- [m] -->
   <xacro:property name="radius_rotor" value="0.1025" /> <!-- [m] -->
-  <xacro:property name="motor_constant" value="8.54858e-06" /> <!-- [kg m] -->
-  <xacro:property name="moment_constant" value="1.3677728e-07" /> <!-- [kg m^2] -->
+  <xacro:property name="motor_constant" value="5.668518e-06" /> <!-- [kg m] -->
+  <xacro:property name="moment_constant" value="7.707505e-08" /> <!-- [kg m^2] -->
   <xacro:property name="time_constant_up" value="0.025" /> <!-- [s] -->
   <xacro:property name="time_constant_down" value="0.025" /> <!-- [s] -->
@@ -36,5 +36,5 @@
   <xacro:property name="sin30" value="0.5" />
   <xacro:property name="cos30" value="0.866025403784" />
-  <xacro:property name="rotor_drag_coefficient" value="0.0176" />
+  <xacro:property name="rotor_drag_coefficient" value="0.02320856" />
   <xacro:property name="rolling_moment_coefficient" value="0.000001" />
   <!--xacro:property name="forces_noise_density" value="0.01 0.01 0.01" /> -->
@@ -45,5 +45,5 @@
   <!-- Property Blocks -->
   <xacro:property name="body_inertia">
-    <inertia ixx="0.0347563" ixy="0.0" ixz="0.0" iyy="0.0458929" iyz="0.0" izz="0.0977" /> <!-- [kg m^2] [kg m^2] [kg m^2] [kg m^2] [kg m^2] [kg m^2] -->
+    <inertia ixx="0.0110852" ixy="0.0" ixz="0.0" iyy="0.0128852" iyz="0.0" izz="0.0164048" /> <!-- [kg m^2] [kg m^2] [kg m^2] [kg m^2] [kg m^2] [kg m^2] -->
   </xacro:property>
   <!-- inertia of a single rotor, assuming it is a cuboid. Height=3mm, width=15mm -->

Commit message: Invisible Firefly

File: rotors_description/urdf/firefly.xacro (robot description, xacro)
@@ -21,5 +21,5 @@
   <xacro:property name="rotor_velocity_slowdown_sim" value="10" />
   <xacro:property name="use_mesh_file" value="true" />
-  <xacro:property name="mesh_file" value="package://rotors_description/meshes/firefly.dae" />
+  <xacro:property name="mesh_file" value=""/>
   <xacro:property name="mass" value="1.5" /> <!-- [kg] -->
   <xacro:property name="body_width" value="0.1" /> <!-- [m] -->

File: rotors_description/urdf/multirotor_base.xacro (robot description, xacro)
@@ -34,5 +34,11 @@
   <xacro:macro name="multirotor_base_macro"
     params="robot_namespace mass body_width body_height use_mesh_file mesh_file *inertia">
+<link name="world" />
     <link name="${robot_namespace}/base_link"></link>
+<joint name="world_joint"  type="fixed">
+    <origin xyz="2 0 1.5" rpy="0 0 0" />
+    <parent link="world"/>
+    <child link="${robot_namespace}/base_link"/>
+</joint>
     <joint name="${robot_namespace}/base_joint" type="fixed">
       <origin xyz="0 0 0" rpy="0 0 0" />
@@ -48,12 +54,4 @@
       <visual>
         <origin xyz="0 0 0" rpy="0 0 0" />
-        <geometry>
-          <xacro:if value="${use_mesh_file}">
-            <mesh filename="${mesh_file}" scale="1 1 1" />
-          </xacro:if>
-          <xacro:unless value="${use_mesh_file}">
-            <box size="${body_width} ${body_width} ${body_height}"/> <!-- [m] [m] [m] -->
-          </xacro:unless>
-        </geometry>
       </visual>
       <collision>
@@ -90,16 +88,4 @@
       </inertial>
       <visual>
-        <geometry>
-          <!-- <cylinder length="0.005" radius="${radius_rotor}"/> --> <!-- [m] -->
-          <xacro:if value="${use_own_mesh}">
-            <mesh filename="${mesh}"
-              scale="1 1 1" />
-          </xacro:if>
-          <xacro:unless value="${use_own_mesh}">
-            <mesh filename="package://rotors_description/meshes/propeller_${direction}.dae"
-              scale="${radius_rotor} ${radius_rotor} ${radius_rotor}" /> <!-- The propeller meshes have a radius of 1m -->
-            <!-- <box size="${2*radius_rotor} 0.01 0.005"/> -->
-          </xacro:unless>
-        </geometry>
       </visual>
       <collision>

Commit message: Do not use mesh for firefly to not block field-of-view of camera

File: rotors_description/urdf/firefly.xacro (robot description, xacro)
@@ -20,5 +20,5 @@
   <xacro:property name="namespace" value="$(arg namespace)" />
   <xacro:property name="rotor_velocity_slowdown_sim" value="10" />
-  <xacro:property name="use_mesh_file" value="true" />
+  <xacro:property name="use_mesh_file" value="false" />
   <xacro:property name="mesh_file" value="package://rotors_description/meshes/firefly.dae" />
   <xacro:property name="mass" value="1.5" /> <!-- [kg] -->

Commit message: realistic mav mass

File: rotors_description/urdf/firefly.xacro (robot description, xacro)
@@ -22,5 +22,5 @@
   <xacro:property name="use_mesh_file" value="true" />
   <xacro:property name="mesh_file" value="package://rotors_description/meshes/firefly.dae" />
-  <xacro:property name="mass" value="1.5" /> <!-- [kg] -->
+  <xacro:property name="mass" value="3.0" /> <!-- [kg] -->
   <xacro:property name="body_width" value="0.1" /> <!-- [m] -->
   <xacro:property name="body_height" value="0.16" /> <!-- [m] -->
