Commit message: vi_sensor: moved adjusted everything to rotors_simulator
Also added the option to use the vi_sensor as a kinect.

File: rotors_description/urdf/component_snippets.xacro (robot description, xacro)
@@ -116,5 +116,5 @@
   <!-- Macro to add an IMU. -->
   <xacro:macro name="imu_plugin_macro"
-    params="namespace imu_suffix imu_topic
+    params="namespace imu_suffix parent_link imu_topic
       mass_imu_sensor gyroscope_noise_density gyroscopoe_random_walk
       gyroscope_bias_correlation_time gyroscope_turn_on_bias_sigma
@@ -133,5 +133,5 @@
     <joint name="imu${imu_suffix}_joint" type="revolute">
       <xacro:insert_block name="origin" />
-      <parent link="base_link" />
+      <parent link="${parent_link}" />
       <child link="imu${imu_suffix}_link" />
       <limit upper="0" lower="0" effort="0" velocity="0" />
@@ -158,5 +158,5 @@
   <xacro:macro name="odometry_plugin_macro"
     params="
-      namespace odometry_sensor_suffix pose_topic pose_with_covariance_topic
+      namespace odometry_sensor_suffix parent_link pose_topic pose_with_covariance_topic
       position_topic transform_topic odometry_topic parent_frame_id
       mass_odometry_sensor measurement_divisor measurement_delay unknown_delay
@@ -175,5 +175,5 @@
     <!-- odometry joint -->
     <joint name="odometry_sensor${odometry_sensor_suffix}_joint" type="revolute">
-      <parent link="base_link" />
+      <parent link="${parent_link}" />
       <xacro:insert_block name="origin" />
       <child link="odometry_sensor${odometry_sensor_suffix}_link" />
@@ -228,3 +228,86 @@
     </gazebo>
   </xacro:macro>
+  <!-- Macro to add the wind plugin. -->
+  <xacro:macro name="vi_sensor_camera_macro"
+    params="camera_suffix frame_rate">
+    <gazebo reference="camera_${camera_suffix}_link">
+      <sensor type="camera" name="camera_${camera_suffix}">
+        <update_rate>${frame_rate}</update_rate>
+        <camera name="head">
+          <horizontal_fov>1.3962634</horizontal_fov>
+          <image>
+            <width>752</width>
+            <height>480</height>
+            <format>L8</format>
+          </image>
+          <clip>
+            <near>0.02</near>
+            <far>30</far>
+          </clip>
+          <noise>
+            <type>gaussian</type>
+            <!-- Noise is sampled independently per pixel on each frame.
+                 That pixel's noise value is added to each of its color
+                 channels, which at that point lie in the range [0,1]. -->
+            <mean>0.0</mean>
+            <stddev>0.007</stddev>
+          </noise>
+        </camera>
+        <plugin name="camera_${camera_suffix}_controller" filename="libgazebo_ros_camera.so">
+          <alwaysOn>true</alwaysOn>
+          <updateRate>${frame_rate}</updateRate>
+          <cameraName>vi_sensor/camera_${camera_suffix}</cameraName>
+          <imageTopicName>image_raw</imageTopicName>
+          <cameraInfoTopicName>camera_info</cameraInfoTopicName>
+          <frameName>camera_${camera_suffix}_link</frameName>
+          <hackBaseline>0.0</hackBaseline>
+          <distortionK1>0.0</distortionK1>
+          <distortionK2>0.0</distortionK2>
+          <distortionK3>0.0</distortionK3>
+          <distortionT1>0.0</distortionT1>
+          <distortionT2>0.0</distortionT2>
+        </plugin>
+      </sensor>
+      <turnGravityOff>true</turnGravityOff>
+      <material>Gazebo/Blue</material>
+    </gazebo>
+  </xacro:macro>
+  <xacro:macro name="vi_sensor_kinect_macro" params="frame_rate">
+    <gazebo reference="kinect_link">
+      <sensor type="depth" name="vi_sensor_kinect">
+        <always_on>true</always_on>
+        <update_rate>${frame_rate}</update_rate>
+        <camera>
+          <horizontal_fov>2</horizontal_fov>
+          <image>
+            <format>L8</format>
+            <width>640</width>
+            <height>480</height>
+          </image>
+          <clip>
+            <near>0.01</near>
+            <far>100</far>
+          </clip>
+        </camera>
+        <plugin name="kinect" filename="libgazebo_ros_openni_kinect.so">
+          <baseline>0.11</baseline>
+          <alwaysOn>true</alwaysOn>
+          <updateRate>${frame_rate}</updateRate>
+          <cameraName>vi_sensor/kinect</cameraName>
+          <imageTopicName>camera/image_raw</imageTopicName>
+          <cameraInfoTopicName>camera/camera_info</cameraInfoTopicName>
+          <depthImageTopicName>depth/disparity</depthImageTopicName>
+          <depthImageCameraInfoTopicName>depth/camera_info</depthImageCameraInfoTopicName>
+          <pointCloudTopicName>depth/points</pointCloudTopicName>
+          <frameName>kinect_link</frameName>
+          <pointCloudCutoff>0.5</pointCloudCutoff>
+          <distortionK1>0.0</distortionK1>
+          <distortionK2>0.0</distortionK2>
+          <distortionK3>0.0</distortionK3>
+          <distortionT1>0.0</distortionT1>
+          <distortionT2>0.0</distortionT2>
+        </plugin>
+      </sensor>
+    </gazebo>
+  </xacro:macro>
 </robot>

File: rotors_description/urdf/firefly_base.xacro (robot description, xacro)
@@ -30,4 +30,5 @@
     namespace="${namespace}"
     imu_suffix=""
+    parent_link="base_link"
     imu_topic="imu"
     mass_imu_sensor="0.015"
@@ -49,4 +50,5 @@
       namespace="${namespace}"
       imu_suffix="gt"
+      parent_link="base_link"
       imu_topic="ground_truth/imu"
       mass_imu_sensor="0.00001"
@@ -67,4 +69,5 @@
       namespace="${namespace}/ground_truth"
       odometry_sensor_suffix="gt"
+      parent_link="base_link"
       pose_topic="pose"
       pose_with_covariance_topic="pose_with_covariance"

File: rotors_description/urdf/hummingbird_base.xacro (robot description, xacro)
@@ -30,4 +30,5 @@
     namespace="${namespace}"
     imu_suffix=""
+    parent_link="base_link"
     imu_topic="imu"
     mass_imu_sensor="0.015"
@@ -49,4 +50,5 @@
       namespace="${namespace}"
       imu_suffix="gt"
+      parent_link="base_link"
       imu_topic="ground_truth/imu"
       mass_imu_sensor="0.00001"
@@ -67,4 +69,5 @@
       namespace="${namespace}/ground_truth"
       odometry_sensor_suffix="gt"
+      parent_link="base_link"
       pose_topic="pose"
       pose_with_covariance_topic="pose_with_covariance"

File: rotors_description/urdf/vi_sensor.xacro (robot description, xacro)
@@ -2,7 +2,6 @@
 <!-- Revolute-Revolute Manipulator -->
 <robot name="vi_sensor" xmlns:xacro="http://www.ros.org/wiki/xacro">
+  <xacro:property name="namespace" value="vi_sensor" />
   <xacro:property name="PI" value="3.141592654" />
-  <!-- Import all Gazebo-customization elements, including Gazebo colors -->
-  <xacro:include filename="$(find mav_description)/urdf/vi_sensor.gazebo" />
   <!-- Vi Sensor Link -->
   <link name="vi_sensor_link">
@@ -16,5 +15,5 @@
       <origin xyz="0 0 0" rpy="0 0 0" />
       <geometry>
-        <mesh filename="package://mav_description/meshes/vi_sensor.dae" scale="1 1 1" />
+        <mesh filename="package://rotors_description/meshes/vi_sensor.dae" scale="1 1 1" />
       </geometry>
     </visual>
@@ -33,11 +32,4 @@
       </geometry>
     </collision>
-    <!-- <visual>
-      <origin xyz="0 0 0" rpy="0 ${PI/2} 0" />
-      <geometry>
-        <cylinder length="0.01" radius="0.007" />
-      </geometry>
-      <material name="red" />
-    </visual> -->
     <inertial>
       <mass value="1e-5" />
@@ -54,11 +46,4 @@
       </geometry>
     </collision>
-    <!-- <visual>
-      <origin xyz="0 0 0" rpy="0 ${PI/2} 0" />
-      <geometry>
-        <cylinder length="0.01" radius="0.007" />
-      </geometry>
-      <material name="red" />
-    </visual> -->
     <inertial>
       <mass value="1e-5" />
@@ -67,28 +52,8 @@
     </inertial>
   </link>
-  <!-- IMU Link -->
-  <link name="imu_link">
-    <collision>
-      <origin xyz="0 0 0" rpy="0 0 0" />
-      <geometry>
-        <box size="0.009 0.0425 0.024" />
-      </geometry>
-    </collision>
-    <!-- <visual>
-      <origin xyz="0 0 0" rpy="0 0 0" />
-      <geometry>
-        <box size="0.009 0.0425 0.024" />
-      </geometry>
-      <material name="red" />
-    </visual> -->
-    <inertial>
-      <inertia ixx="0.001" ixy="0.0" ixz="0.0" iyy="0.001" iyz="0.0"
-        izz="0.001" />
-      <mass value="1" />  <!-- [kg] -->
-      <origin xyz="0 0 0" rpy="0 0 0" />
-    </inertial>
-  </link>
+  <!-- Kinect Link -->
+  <link name="kinect_link" />
     <!-- Left Camera Joint -->
-  <joint name="camera_left_joint" type="revolute">
+  <joint name="camera_left_joint" type="fixed">
     <origin xyz="0.015 0.055 0.0065" rpy="0 0 0" />
     <parent link="vi_sensor_link" />
@@ -97,5 +62,5 @@
   </joint>
     <!-- Right Camera Joint -->
-  <joint name="camera_right_joint" type="revolute">
+  <joint name="camera_right_joint" type="fixed">
     <origin xyz="0.015 -0.055 0.0065" rpy="0 0 0" />
     <parent link="vi_sensor_link" />
@@ -103,9 +68,9 @@
     <limit upper="0" lower="0" effort="0" velocity="0" />
   </joint>
-  <!-- IMU Joint -->
-  <joint name="imu_joint" type="revolute">
-    <origin xyz="0.015 0 0.0113" rpy="0 0 0" />
+  <!-- Kinect Joint -->
+  <joint name="kinect_joint" type="fixed">
+    <origin xyz="0.015 0 0.0065" rpy="0 0 0" />
     <parent link="vi_sensor_link" />
-    <child link="imu_link" />
+    <child link="kinect_link" />
     <limit upper="0" lower="0" effort="0" velocity="0" />
   </joint>

Commit message: fixed namespaces and mass of vi sensor

File: rotors_description/urdf/component_snippets.xacro (robot description, xacro)
@@ -231,5 +231,5 @@
   <xacro:macro name="vi_sensor_camera_macro"
     params="camera_suffix frame_rate">
-    <gazebo reference="camera_${camera_suffix}_link">
+    <gazebo reference="${namespace}/camera_${camera_suffix}_link">
       <sensor type="camera" name="camera_${camera_suffix}">
         <update_rate>${frame_rate}</update_rate>
@@ -255,7 +255,8 @@
         </camera>
         <plugin name="camera_${camera_suffix}_controller" filename="libgazebo_ros_camera.so">
+          <robotNamespace>${namespace}</robotNamespace>
           <alwaysOn>true</alwaysOn>
           <updateRate>${frame_rate}</updateRate>
-          <cameraName>vi_sensor/camera_${camera_suffix}</cameraName>
+          <cameraName>camera_${camera_suffix}</cameraName>
           <imageTopicName>image_raw</imageTopicName>
           <cameraInfoTopicName>camera_info</cameraInfoTopicName>
@@ -274,5 +275,5 @@
   </xacro:macro>
   <xacro:macro name="vi_sensor_kinect_macro" params="frame_rate">
-    <gazebo reference="kinect_link">
+    <gazebo reference="${namespace}/kinect_link">
       <sensor type="depth" name="vi_sensor_kinect">
         <always_on>true</always_on>
@@ -291,8 +292,9 @@
         </camera>
         <plugin name="kinect" filename="libgazebo_ros_openni_kinect.so">
+          <robotNamespace>${namespace}</robotNamespace>
+          <alwaysOn>true</alwaysOn>
           <baseline>0.11</baseline>
-          <alwaysOn>true</alwaysOn>
           <updateRate>${frame_rate}</updateRate>
-          <cameraName>vi_sensor/kinect</cameraName>
+          <cameraName>kinect</cameraName>
           <imageTopicName>camera/image_raw</imageTopicName>
           <cameraInfoTopicName>camera/camera_info</cameraInfoTopicName>

File: rotors_description/urdf/vi_sensor.xacro (robot description, xacro)
@@ -19,5 +19,5 @@
     </visual>
     <inertial>
-      <mass value="1e-5" />
+      <mass value="0.13" />
       <origin xyz="0 0 0" rpy="0 0 0" />
       <inertia ixx="1e-6" ixy="0" ixz="0" iyy="1e-6" iyz="0" izz="1e-6" />
@@ -25,5 +25,5 @@
   </link>
   <!-- Left Camera Link -->
-  <link name="camera_left_link">
+  <link name="vi_sensor/camera_left_link">
     <collision>
       <origin xyz="0 0 0" rpy="0 0 0" />
@@ -39,5 +39,5 @@
   </link>
   <!-- Right Camera Link -->
-  <link name="camera_right_link">
+  <link name="vi_sensor/camera_right_link">
     <collision>
       <origin xyz="0 0 0" rpy="0 0 0" />
@@ -53,10 +53,10 @@
   </link>
   <!-- Kinect Link -->
-  <link name="kinect_link" />
+  <link name="vi_sensor/kinect_link" />
     <!-- Left Camera Joint -->
   <joint name="camera_left_joint" type="fixed">
     <origin xyz="0.015 0.055 0.0065" rpy="0 0 0" />
     <parent link="vi_sensor_link" />
-    <child link="camera_left_link" />
+    <child link="vi_sensor/camera_left_link" />
     <limit upper="0" lower="0" effort="0" velocity="0" />
   </joint>
@@ -65,5 +65,5 @@
     <origin xyz="0.015 -0.055 0.0065" rpy="0 0 0" />
     <parent link="vi_sensor_link" />
-    <child link="camera_right_link" />
+    <child link="vi_sensor/camera_right_link" />
     <limit upper="0" lower="0" effort="0" velocity="0" />
   </joint>
@@ -72,5 +72,5 @@
     <origin xyz="0.015 0 0.0065" rpy="0 0 0" />
     <parent link="vi_sensor_link" />
-    <child link="kinect_link" />
+    <child link="vi_sensor/kinect_link" />
     <limit upper="0" lower="0" effort="0" velocity="0" />
   </joint>

Commit message: added pelican hovering example

File: rotors_description/urdf/component_snippets.xacro (robot description, xacro)
@@ -116,5 +116,5 @@
   <!-- Macro to add an IMU. -->
   <xacro:macro name="imu_plugin_macro"
-    params="namespace imu_suffix imu_topic
+    params="namespace imu_suffix parent_link imu_topic
       mass_imu_sensor gyroscope_noise_density gyroscopoe_random_walk
       gyroscope_bias_correlation_time gyroscope_turn_on_bias_sigma
@@ -133,5 +133,5 @@
     <joint name="imu${imu_suffix}_joint" type="revolute">
       <xacro:insert_block name="origin" />
-      <parent link="base_link" />
+      <parent link="${parent_link}" />
       <child link="imu${imu_suffix}_link" />
       <limit upper="0" lower="0" effort="0" velocity="0" />
@@ -158,5 +158,5 @@
   <xacro:macro name="odometry_plugin_macro"
     params="
-      namespace odometry_sensor_suffix pose_topic pose_with_covariance_topic
+      namespace odometry_sensor_suffix parent_link pose_topic pose_with_covariance_topic
       position_topic transform_topic odometry_topic parent_frame_id
       mass_odometry_sensor measurement_divisor measurement_delay unknown_delay
@@ -175,5 +175,5 @@
     <!-- odometry joint -->
     <joint name="odometry_sensor${odometry_sensor_suffix}_joint" type="revolute">
-      <parent link="base_link" />
+      <parent link="${parent_link}" />
       <xacro:insert_block name="origin" />
       <child link="odometry_sensor${odometry_sensor_suffix}_link" />

File: rotors_description/urdf/hummingbird.xacro (robot description, xacro)
@@ -1,3 +1,19 @@
 <?xml version="1.0"?>
+<!--
+  Copyright 2015 Fadri Furrer, ASL, ETH Zurich, Switzerland
+  Copyright 2015 Michael Burri, ASL, ETH Zurich, Switzerland
+  Copyright 2015 Mina Kamel, ASL, ETH Zurich, Switzerland
+  Copyright 2015 Janosch Nikolic, ASL, ETH Zurich, Switzerland
+  Copyright 2015 Markus Achtelik, ASL, ETH Zurich, Switzerland
+  Licensed under the Apache License, Version 2.0 (the "License");
+  you may not use this file except in compliance with the License.
+  You may obtain a copy of the License at
+  http://www.apache.org/licenses/LICENSE-2.0
+  Unless required by applicable law or agreed to in writing, software
+  distributed under the License is distributed on an "AS IS" BASIS,
+  WITHOUT WARRANTIES OR CONDITIONS OF ANY KIND, either express or implied.
+  See the License for the specific language governing permissions and
+  limitations under the License.
+-->
 <robot name="hummingbird" xmlns:xacro="http://ros.org/wiki/xacro">
   <!-- Properties (Taken from Novel Dynamic Inversion Architecture Design

File: rotors_description/urdf/pelican_base.xacro (robot description, xacro)
@@ -17,4 +17,91 @@
 -->
 <robot name="pelican" xmlns:xacro="http://ros.org/wiki/xacro">
+  <xacro:include filename="$(find rotors_description)/urdf/component_snippets.xacro" />
+  <!-- Instantiate pelican "mechanics" -->
   <xacro:include filename="$(find rotors_description)/urdf/pelican.xacro" />
+  <!-- Instantiate a controller. -->
+  <xacro:controller_plugin_macro
+    namespace="${namespace}"
+    imu_sub_topic="imu"
+    >
+  </xacro:controller_plugin_macro>
+  <!-- Mount an ADIS16448 IMU. -->
+  <xacro:imu_plugin_macro
+    namespace="${namespace}"
+    imu_suffix=""
+    parent_link="base_link"
+    imu_topic="imu"
+    mass_imu_sensor="0.015"
+    gyroscope_noise_density="0.0003394"
+    gyroscopoe_random_walk="0.000038785"
+    gyroscope_bias_correlation_time="1000.0"
+    gyroscope_turn_on_bias_sigma="0.0087"
+    accelerometer_noise_density="0.004"
+    accelerometer_random_walk="0.006"
+    accelerometer_bias_correlation_time="300.0"
+    accelerometer_turn_on_bias_sigma="0.1960"
+  >
+    <inertia ixx="0.00001" ixy="0.0" ixz="0.0" iyy="0.00001" iyz="0.0" izz="0.00001" />
+    <origin xyz="0 0 0" rpy="0 0 0" />
+  </xacro:imu_plugin_macro>
+  <xacro:if value="$(arg enable_ground_truth)">
+    <!-- Mount an IMU providing ground truth. -->
+    <xacro:imu_plugin_macro
+      namespace="${namespace}"
+      imu_suffix="gt"
+      parent_link="base_link"
+      imu_topic="ground_truth/imu"
+      mass_imu_sensor="0.00001"
+      gyroscope_noise_density="0.0"
+      gyroscopoe_random_walk="0.0"
+      gyroscope_bias_correlation_time="1000.0"
+      gyroscope_turn_on_bias_sigma="0.0"
+      accelerometer_noise_density="0.0"
+      accelerometer_random_walk="0.0"
+      accelerometer_bias_correlation_time="300.0"
+      accelerometer_turn_on_bias_sigma="0.0"
+    >
+      <inertia ixx="0.00001" ixy="0.0" ixz="0.0" iyy="0.00001" iyz="0.0" izz="0.00001" />
+      <origin xyz="0 0 0" rpy="0 0 0" />
+    </xacro:imu_plugin_macro>
+    <!-- Mount a generic odometry sensor providing ground truth. -->
+    <xacro:odometry_plugin_macro
+      namespace="${namespace}/ground_truth"
+      odometry_sensor_suffix="gt"
+      parent_link="base_link"
+      pose_topic="pose"
+      pose_with_covariance_topic="pose_with_covariance"
+      position_topic="position"
+      transform_topic="transform"
+      odometry_topic="odometry"
+      parent_frame_id="world"
+      mass_odometry_sensor="0.00001"
+      measurement_divisor="1"
+      measurement_delay="0"
+      unknown_delay="0.0"
+      noise_normal_position="0 0 0"
+      noise_normal_quaternion="0 0 0"
+      noise_normal_linear_velocity="0 0 0"
+      noise_normal_angular_velocity="0 0 0"
+      noise_uniform_position="0 0 0"
+      noise_uniform_quaternion="0 0 0"
+      noise_uniform_linear_velocity="0 0 0"
+      noise_uniform_angular_velocity="0 0 0"
+      enable_odometry_map="false"
+      odometry_map=""
+      image_scale=""
+    >
+      <inertia ixx="0.00001" ixy="0.0" ixz="0.0" iyy="0.00001" iyz="0.0" izz="0.00001" /> <!-- [kg·m^2] [kg·m^2] [kg·m^2] [kg·m^2] [kg·m^2] [kg·m^2] -->
+      <origin xyz="0.0 0.0 0.0" rpy="0.0 0.0 0.0" />
+    </xacro:odometry_plugin_macro>
+  </xacro:if>
+  <xacro:if value="$(arg enable_logging)">
+    <!-- Instantiate a logger -->
+    <xacro:bag_plugin_macro
+      namespace="${namespace}"
+      bag_file="$(arg log_file)"
+      rotor_velocity_slowdown_sim="${rotor_velocity_slowdown_sim}"
+    >
+    </xacro:bag_plugin_macro>
+  </xacro:if>
 </robot>
