Commit message: attached the vi_sensor to the firefly and modified the component_snippets for it

File: rotors_description/urdf/component_snippets.xacro (robot description, xacro)
@@ -17,4 +17,5 @@
 -->
 <robot xmlns:xacro="http://ros.org/wiki/xacro">
+  <xacro:property name="PI" value="3.141592654" />
   <!-- Macro for the inertial properties of a box -->
   <xacro:macro name="box_inertial" params="x y z mass *origin">
@@ -333,5 +334,5 @@
   </xacro:macro>
   <!-- VI-Sensor Macro -->
-  <xacro:macro name="vi_sensor_macro" params="namespace parent_link *origin">
+  <xacro:macro name="vi_sensor_macro" params="namespace parent_link enable_cameras enable_depth enable_ground_truth *origin">
     <!-- Vi Sensor Link -->
     <link name="${namespace}/vi_sensor_link">
@@ -360,5 +361,5 @@
     </joint>
     <!-- Cameras -->
-    <xacro:if value="$(arg enable_cameras)">
+    <xacro:if value="${enable_cameras}">
       <!-- Left Camera -->
       <xacro:vi_sensor_camera_macro
@@ -375,5 +376,5 @@
     </xacro:if>
     <!-- Depth Sensor -->
-    <xacro:if value="$(arg enable_depth)">
+    <xacro:if value="${enable_depth}">
       <xacro:vi_sensor_depth_macro
         namespace="${namespace}" parent_link="${namespace}/vi_sensor_link"
@@ -383,5 +384,5 @@
     </xacro:if>
     <!-- Groundtruth -->
-    <xacro:if value="$(arg enable_ground_truth)">
+    <xacro:if value="${enable_ground_truth}">
       <!-- Odometry Sensor -->
       <xacro:odometry_plugin_macro

Commit message: added magnetometer skeleton

File: rotors_description/urdf/component_snippets.xacro (robot description, xacro)
@@ -223,4 +223,33 @@
     </gazebo>
   </xacro:macro>
+  <!-- Macro to add a generic magnetometer sensor. -->
+    <xacro:macro name="magnetometer_plugin_macro"
+      params="
+        namespace magnetometer_sensor_suffix parent_link
+          magnetometer_topic parent_frame_id mass_magnetometer_sensor
+ *inertia *origin">
+      <!-- magnetometer link -->
+      <link name="${namespace}/magnetometer_sensor${magnetometer_sensor_suffix}_link">
+        <inertial>
+          <xacro:insert_block name="inertia" />
+          <mass value="${mass_magnetometer_sensor}" />  <!-- [kg] -->
+        </inertial>
+      </link>
+      <!-- magnetometer joint -->
+      <joint name="${namespace}/magnetometer_sensor${magnetometer_sensor_suffix}_joint" type="revolute">
+        <parent link="${parent_link}" />
+        <xacro:insert_block name="origin" />
+        <child link="${namespace}/magnetometer_sensor${magnetometer_sensor_suffix}_link" />
+        <limit upper="0" lower="0" effort="0" velocity="0" />
+      </joint>
+      <gazebo>
+        <plugin filename="librotors_gazebo_magnetometer_plugin.so" name="magnetometer_sensor${magnetometer_sensor_suffix}">
+          <linkName>${namespace}/magnetometer_sensor${magnetometer_sensor_suffix}_link</linkName>
+          <robotNamespace>${namespace}</robotNamespace>
+          <magnetometerTopic>${magnetometer_topic}</magnetometerTopic>
+          <parentFrameId>${parent_frame_id}</parentFrameId>  <!-- Use the scoped link name here. e.g. Model::link. -->
+        </plugin>
+      </gazebo>
+    </xacro:macro>
   <!-- Macro to add the wind plugin. -->
   <xacro:macro name="wind_plugin_macro"

Commit message: fixed old naming of pi

File: rotors_description/urdf/component_snippets.xacro (robot description, xacro)
@@ -280,5 +280,5 @@
     <link name="${namespace}/camera_${camera_suffix}_optical_center_link" />
     <joint name="${namespace}/camera_${camera_suffix}_optical_center_joint" type="fixed">
-      <origin xyz="0 0 0" rpy="${-PI/2} 0 ${-PI/2}" />
+      <origin xyz="0 0 0" rpy="${-pi/2} 0 ${-pi/2}" />
       <parent link="${namespace}/camera_${camera_suffix}_link" />
       <child link="${namespace}/camera_${camera_suffix}_optical_center_link" />

Commit message: Add a full stereo camera instead of 2 monocular cameras.

File: rotors_description/urdf/component_snippets.xacro (robot description, xacro)
@@ -97,4 +97,110 @@
           <frameName>camera_${camera_suffix}_link</frameName>
           <hackBaseline>0.0</hackBaseline>
+          <distortionK1>0.0</distortionK1>
+          <distortionK2>0.0</distortionK2>
+          <distortionK3>0.0</distortionK3>
+          <distortionT1>0.0</distortionT1>
+          <distortionT2>0.0</distortionT2>
+        </plugin>
+      </sensor>
+    </gazebo>
+  </xacro:macro>
+  <!-- Camera joint macro - just the joints, links, and collisions for a single
+       camera. -->
+  <xacro:macro name="camera_joint_macro"
+    params="namespace parent_link camera_suffix enable_visual *geometry *origin" >
+    <link name="${namespace}/camera_${camera_suffix}_link">
+      <collision>
+        <origin xyz="0 0 0" rpy="0 0 0" />
+        <geometry>
+          <xacro:insert_block name="geometry" />
+        </geometry>
+      </collision>
+      <xacro:if value="${enable_visual}">
+        <visual>
+          <origin xyz="0 0 0" rpy="0 0 0" />
+          <geometry>
+            <xacro:insert_block name="geometry" />
+          </geometry>
+          <material name="red" />
+        </visual>
+      </xacro:if>
+      <inertial>
+        <mass value="1e-5" />
+        <origin xyz="0 0 0" rpy="0 0 0" />
+        <inertia ixx="1e-6" ixy="0" ixz="0" iyy="1e-6" iyz="0" izz="1e-6" />
+      </inertial>
+    </link>
+    <joint name="${namespace}/camera_${camera_suffix}_joint" type="fixed">
+      <xacro:insert_block name="origin" />
+      <parent link="${parent_link}" />
+      <child link="${namespace}/camera_${camera_suffix}_link" />
+    </joint>
+  </xacro:macro>
+  <!-- Camera sensor macro - just image parameters. -->
+  <xacro:macro name="camera_sensor_macro"
+    params="camera_suffix horizontal_fov image_width image_height
+      image_format min_distance max_distance noise_mean noise_stddev" >
+    <camera name="${camera_suffix}">
+      <horizontal_fov>${horizontal_fov}</horizontal_fov>
+      <image>
+        <width>${image_width}</width>
+        <height>${image_height}</height>
+        <format>${image_format}</format>
+      </image>
+      <clip>
+        <near>${min_distance}</near>
+        <far>${max_distance}</far>
+      </clip>
+      <noise>
+        <type>gaussian</type>
+        <!-- Noise is sampled independently per pixel on each frame.
+             That pixel's noise value is added to each of its color
+             channels, which at that point lie in the range [0,1]. -->
+        <mean>${noise_mean}</mean>
+        <stddev>${noise_stddev}</stddev>
+      </noise>
+    </camera>
+  </xacro:macro>
+  <!-- Macro to add a multicamera (stereo pair). -->
+  <xacro:macro name="stereo_camera_macro"
+    params="namespace parent_link frame_rate
+      horizontal_fov image_width image_height image_format min_distance
+      max_distance noise_mean noise_stddev enable_visual offset_x baseline_y
+      offset_z">
+    <!-- These are parameters for the left camera link and then the right
+        as well. -->
+    <xacro:camera_joint_macro namespace="${namespace}"
+      parent_link="${parent_link}"
+      camera_suffix="left" enable_visual="${enable_visual}">
+      <origin xyz="${offset_x} ${baseline_y/2} ${offset_z}" rpy="0 0 0" />
+    </xacro:camera_joint_macro>
+    <xacro:camera_joint_macro namespace="${namespace}"
+      parent_link="${parent_link}"
+      camera_suffix="right" enable_visual="${enable_visual}">
+      <origin xyz="{offset_x} ${-baseline_y/2} ${offset_z}" rpy="0 0 0" />
+    </xacro:camera_joint_macro>
+    <!-- Both cameras in the pair are anchored off the left camera frame. -->
+    <gazebo reference="${namespace}/camera_left_link">
+      <sensor type="multicamera" name="stereo_camera">
+        <update_rate>${frame_rate}</update_rate>
+        <!-- Here we set up the individual cameras of the stereo head. -->
+        <xacro:camera_sensor_macro camera_suffix="left"
+            horizontal_fov="${horizontal_fov}" image_width="${image_width}"
+            image_height="${image_height}" image_format="${image_format}"
+            min_distance="${min_distance}" max_distance="${max_distance}"
+            noise_mean="${noise_mean}" noise_stddev="${noise_stddev}">
+        </xacro:camera_joint_macro>
+        <!-- Stereo controller, setting the transforms between the two cameras. -->
+        <plugin name="stereo_camera_controller" filename="libgazebo_ros_multicamera.so">
+          <alwaysOn>true</alwaysOn>
+          <updateRate>0.0</updateRate>
+          <cameraName>camera</cameraName>
+          <imageTopicName>image_raw</imageTopicName>
+          <cameraInfoTopicName>camera_info</cameraInfoTopicName>
+          <frameName>${namespace}/camera_left_link</frameName>
+          <!-- This is unfortunately the way to get correct parameters for the
+               stereo camera. -->
+          <hackBaseline>${baseline_y}</hackBaseline>
           <distortionK1>0.0</distortionK1>
           <distortionK2>0.0</distortionK2>
@@ -253,4 +359,26 @@
       <cylinder length="0.01" radius="0.007" />
       <xacro:insert_block name="origin" />
+    </xacro:camera_macro>
+  </xacro:macro>
+  <!-- Macro to add a VI-sensor camera. -->
+  <xacro:macro name="vi_sensor_stereo_camera_macro"
+    params="namespace parent_link frame_rate offset_x baseline_y offset_z">
+    <xacro:stereo_camera_macro
+      namespace="${namespace}"
+      parent_link="${parent_link}"
+      frame_rate="${frame_rate}"
+      horizontal_fov="1.3962634"
+      image_width="752"
+      image_height="480"
+      image_format="L8"
+      min_distance="0.02"
+      max_distance="30"
+      noise_mean="0.0"
+      noise_stddev="0.007"
+      enable_visual="false"
+      offset_x="${offset_x}"
+      baseline_y="${baseline_y}"
+      offset_z="${offset_z}"
+      <cylinder length="0.01" radius="0.007" />
     </xacro:camera_macro>
   </xacro:macro>
@@ -352,16 +480,22 @@
     <!-- Cameras -->
     <xacro:if value="${enable_cameras}">
+      <!-- Insert stereo pair. -->
+      <xacro:vi_sensor_camera_macro
+        namespace="${namespace}" parent_link="${namespace}/vi_sensor_link"
+        frame_rate="30.0" offset_x="0.015" baseline_y="${0.055*2}"
+        offset_z="0.0065">
+      </xacro:vi_sensor_camera_macro>
       <!-- Left Camera -->
-      <xacro:vi_sensor_camera_macro
+      <!-- <xacro:vi_sensor_camera_macro
         namespace="${namespace}" parent_link="${namespace}/vi_sensor_link"
         camera_suffix="left" frame_rate="30.0">
         <origin xyz="0.015 0.055 0.0065" rpy="0 0 0" />
-      </xacro:vi_sensor_camera_macro>
+      </xacro:vi_sensor_camera_macro> -->
       <!-- Right Camera -->
-      <xacro:vi_sensor_camera_macro namespace="${namespace}"
+      <!-- <xacro:vi_sensor_camera_macro namespace="${namespace}"
         parent_link="${namespace}/vi_sensor_link"
         camera_suffix="right" frame_rate="30.0">
         <origin xyz="0.015 -0.055 0.0065" rpy="0 0 0" />
-      </xacro:vi_sensor_camera_macro>
+      </xacro:vi_sensor_camera_macro> -->
     </xacro:if>
     <!-- Depth Sensor -->

Commit message: Runs properly now. :)

File: rotors_description/urdf/component_snippets.xacro (robot description, xacro)
@@ -109,5 +109,5 @@
        camera. -->
   <xacro:macro name="camera_joint_macro"
-    params="namespace parent_link camera_suffix enable_visual *geometry *origin" >
+    params="namespace parent_link camera_suffix enable_visual *origin *geometry" >
     <link name="${namespace}/camera_${camera_suffix}_link">
       <collision>
@@ -165,8 +165,8 @@
   <!-- Macro to add a multicamera (stereo pair). -->
   <xacro:macro name="stereo_camera_macro"
-    params="namespace parent_link frame_rate
+    params="namespace camera_name parent_link frame_rate
       horizontal_fov image_width image_height image_format min_distance
       max_distance noise_mean noise_stddev enable_visual offset_x baseline_y
-      offset_z">
+      offset_z *geometry">
     <!-- These are parameters for the left camera link and then the right
         as well. -->
@@ -175,13 +175,15 @@
       camera_suffix="left" enable_visual="${enable_visual}">
       <origin xyz="${offset_x} ${baseline_y/2} ${offset_z}" rpy="0 0 0" />
+      <xacro:insert_block name="geometry" />
     </xacro:camera_joint_macro>
     <xacro:camera_joint_macro namespace="${namespace}"
       parent_link="${parent_link}"
       camera_suffix="right" enable_visual="${enable_visual}">
-      <origin xyz="{offset_x} ${-baseline_y/2} ${offset_z}" rpy="0 0 0" />
+      <origin xyz="${offset_x} ${-baseline_y/2} ${offset_z}" rpy="0 0 0" />
+      <xacro:insert_block name="geometry" />
     </xacro:camera_joint_macro>
     <!-- Both cameras in the pair are anchored off the left camera frame. -->
     <gazebo reference="${namespace}/camera_left_link">
-      <sensor type="multicamera" name="stereo_camera">
+      <sensor type="multicamera" name="${namespace}_stereo_camera">
         <update_rate>${frame_rate}</update_rate>
         <!-- Here we set up the individual cameras of the stereo head. -->
@@ -191,10 +193,16 @@
             min_distance="${min_distance}" max_distance="${max_distance}"
             noise_mean="${noise_mean}" noise_stddev="${noise_stddev}">
-        </xacro:camera_joint_macro>
+        </xacro:camera_sensor_macro>
+        <xacro:camera_sensor_macro camera_suffix="right"
+            horizontal_fov="${horizontal_fov}" image_width="${image_width}"
+            image_height="${image_height}" image_format="${image_format}"
+            min_distance="${min_distance}" max_distance="${max_distance}"
+            noise_mean="${noise_mean}" noise_stddev="${noise_stddev}">
+        </xacro:camera_sensor_macro>
         <!-- Stereo controller, setting the transforms between the two cameras. -->
-        <plugin name="stereo_camera_controller" filename="libgazebo_ros_multicamera.so">
+        <plugin name="${namespace}_stereo_camera_controller" filename="libgazebo_ros_multicamera.so">
           <alwaysOn>true</alwaysOn>
           <updateRate>0.0</updateRate>
-          <cameraName>camera</cameraName>
+          <cameraName>${camera_name}</cameraName>
           <imageTopicName>image_raw</imageTopicName>
           <cameraInfoTopicName>camera_info</cameraInfoTopicName>
@@ -361,9 +369,10 @@
     </xacro:camera_macro>
   </xacro:macro>
-  <!-- Macro to add a VI-sensor camera. -->
+  <!-- Macro to add a VI-sensor stereo camera. -->
   <xacro:macro name="vi_sensor_stereo_camera_macro"
     params="namespace parent_link frame_rate offset_x baseline_y offset_z">
     <xacro:stereo_camera_macro
       namespace="${namespace}"
+      camera_name="vi_sensor"
       parent_link="${parent_link}"
       frame_rate="${frame_rate}"
@@ -379,7 +388,7 @@
       offset_x="${offset_x}"
       baseline_y="${baseline_y}"
-      offset_z="${offset_z}"
+      offset_z="${offset_z}" >
       <cylinder length="0.01" radius="0.007" />
-    </xacro:camera_macro>
+    </xacro:stereo_camera_macro>
   </xacro:macro>
   <!-- Macro to add a depth camera on the VI-sensor. -->
@@ -481,9 +490,9 @@
     <xacro:if value="${enable_cameras}">
       <!-- Insert stereo pair. -->
-      <xacro:vi_sensor_camera_macro
+      <xacro:vi_sensor_stereo_camera_macro
         namespace="${namespace}" parent_link="${namespace}/vi_sensor_link"
         frame_rate="30.0" offset_x="0.015" baseline_y="${0.055*2}"
-        offset_z="0.0065">
-      </xacro:vi_sensor_camera_macro>
+        offset_z="0.0065" >
+      </xacro:vi_sensor_stereo_camera_macro>
       <!-- Left Camera -->
       <!-- <xacro:vi_sensor_camera_macro

Commit message: Remove dead code.

File: rotors_description/urdf/component_snippets.xacro (robot description, xacro)
@@ -499,16 +499,4 @@
         offset_z="0.0065" >
       </xacro:vi_sensor_stereo_camera_macro>
-      <!-- Left Camera -->
-      <!-- <xacro:vi_sensor_camera_macro
-        namespace="${namespace}" parent_link="${namespace}/vi_sensor_link"
-        camera_suffix="left" frame_rate="30.0">
-        <origin xyz="0.015 0.055 0.0065" rpy="0 0 0" />
-      </xacro:vi_sensor_camera_macro> -->
-      <!-- Right Camera -->
-      <!-- <xacro:vi_sensor_camera_macro namespace="${namespace}"
-        parent_link="${namespace}/vi_sensor_link"
-        camera_suffix="right" frame_rate="30.0">
-        <origin xyz="0.015 -0.055 0.0065" rpy="0 0 0" />
-      </xacro:vi_sensor_camera_macro> -->
     </xacro:if>
     <!-- Depth Sensor -->

Commit message: Updated names, cleaned up comments.

File: rotors_description/urdf/component_snippets.xacro (robot description, xacro)
@@ -169,6 +169,6 @@
     params="namespace camera_name parent_link frame_rate
       horizontal_fov image_width image_height image_format min_distance
-      max_distance noise_mean noise_stddev enable_visual offset_x baseline_y
-      offset_z *geometry">
+      max_distance noise_mean noise_stddev enable_visual origin_offset_x
+      baseline_y origin_offset_z *geometry">
     <!-- These are parameters for the left camera link and then the right
         as well. -->
@@ -176,5 +176,5 @@
       parent_link="${parent_link}"
       camera_suffix="left" enable_visual="${enable_visual}">
-      <origin xyz="${offset_x} ${baseline_y/2} ${offset_z}" rpy="0 0 0" />
+      <origin xyz="${origin_offset_x} ${baseline_y/2} ${origin_offset_z}" rpy="0 0 0" />
       <xacro:insert_block name="geometry" />
     </xacro:camera_joint_macro>
@@ -182,5 +182,5 @@
       parent_link="${parent_link}"
       camera_suffix="right" enable_visual="${enable_visual}">
-      <origin xyz="${offset_x} ${-baseline_y/2} ${offset_z}" rpy="0 0 0" />
+      <origin xyz="${origin_offset_x} ${-baseline_y/2} ${origin_offset_z}" rpy="0 0 0" />
       <xacro:insert_block name="geometry" />
     </xacro:camera_joint_macro>
@@ -212,6 +212,4 @@
           <cameraInfoTopicName>camera_info</cameraInfoTopicName>
           <frameName>${camera_name}/camera_left_link</frameName>
-          <!-- This is unfortunately the way to get correct parameters for the
-               stereo camera. -->
           <hackBaseline>${baseline_y}</hackBaseline>
           <distortionK1>0.0</distortionK1>
@@ -375,5 +373,5 @@
   <!-- Macro to add a VI-sensor stereo camera. -->
   <xacro:macro name="vi_sensor_stereo_camera_macro"
-    params="namespace parent_link frame_rate offset_x baseline_y offset_z">
+    params="namespace parent_link frame_rate origin_offset_x baseline_y origin_offset_z">
     <xacro:stereo_camera_macro
       namespace="${namespace}"
@@ -390,7 +388,7 @@
       noise_stddev="0.007"
       enable_visual="false"
-      offset_x="${offset_x}"
+      origin_offset_x="${origin_offset_x}"
       baseline_y="${baseline_y}"
-      offset_z="${offset_z}" >
+      origin_offset_z="${origin_offset_z}" >
       <cylinder length="0.01" radius="0.007" />
     </xacro:stereo_camera_macro>
@@ -496,6 +494,6 @@
       <xacro:vi_sensor_stereo_camera_macro
         namespace="${namespace}" parent_link="${namespace}/vi_sensor_link"
-        frame_rate="30.0" offset_x="0.015" baseline_y="${0.055*2}"
-        offset_z="0.0065" >
+        frame_rate="30.0" origin_offset_x="0.015" baseline_y="${0.055*2}"
+        origin_offset_z="0.0065" >
       </xacro:vi_sensor_stereo_camera_macro>
     </xacro:if>

Commit message: Initial Commit for Piksi Sensor Gazebo Plugin

File: rotors_description/urdf/component_snippets.xacro (robot description, xacro)
@@ -326,4 +326,40 @@
           <covarianceImageScale>${image_scale}</covarianceImageScale> <!-- the scale of the image in the gazebo world, if set to 1.0, 1 pixel in the image corresponds to 1 meter in the world -->
         </xacro:if>
+      </plugin>
+    </gazebo>
+  </xacro:macro>
+<!-- Macro to add a Piksi RTK GPS sensor. -->
+  <xacro:macro name="piksi_plugin_macro"
+    params="
+      namespace piksi_sensor_suffix parent_link spp_position_topic rtk_position_topic
+      parent_frame_id mass_piksi publish_ground_truth spp_noise_normal spp_offset
+      rtk_fixed_noise_normal
+      rtk_fixed_offset *inertia *origin">
+    <!-- piksi link -->
+    <link name="${namespace}/piksi_sensor${piksi_sensor_suffix}_link">
+      <inertial>
+        <xacro:insert_block name="inertia" />
+        <mass value="${mass_piksi}" />  <!-- [kg] -->
+      </inertial>
+    </link>
+    <!-- piksi joint -->
+    <joint name="${namespace}/piksi_sensor${piksi_sensor_suffix}_joint" type="revolute">
+      <parent link="${parent_link}" />
+      <xacro:insert_block name="origin" />
+      <child link="${namespace}/piksi_sensor${piksi_sensor_suffix}_link" />
+      <limit upper="0" lower="0" effort="0" velocity="0" />
+    </joint>
+    <gazebo>
+      <plugin filename="librotors_gazebo_piksi_plugin.so" name="piksi_sensor${piksi_sensor_suffix}">
+        <linkName>${namespace}/piksi_sensor${piksi_sensor_suffix}_link</linkName>
+        <robotNamespace>${namespace}</robotNamespace>
+        <sppPositionTopic>${spp_position_topic}</sppPositionTopic>
+	<rtkPositionTopic>${rtk_position_topic}</rtkPositionTopic>
+	<publishGroundTruth>${publish_ground_truth}</publishGroundTruth>
+        <parentFrameId>${parent_frame_id}</parentFrameId> <!-- Use the scoped link name here. e.g. Model::link. -->
+	<sppNoiseNormal>${spp_noise_normal}</sppNoiseNormal> <!-- standard deviation of additive white gaussian noise [m] -->
+	<sppOffset>${spp_offset}</sppOffset> <!-- offset against ground truth for SPP GPS output [m] -->
+        <rtkFixedNoiseNormal>${rtk_fixed_noise_normal}</rtkFixedNoiseNormal> <!-- standard deviation of additive white gaussian noise [m] -->
+	<rtkFixedOffset>${rtk_fixed_offset}</rtkFixedOffset> <!-- offset against ground truth for RTK Fixed GPS output [m] -->
       </plugin>
     </gazebo>
