Commit message: added manipulator with force sensor plugin

File: rotors_description/urdf/component_snippets.xacro (robot description, xacro)
@@ -627,3 +627,66 @@
     </xacro:imu_plugin_macro>
   </xacro:macro>
+	<!-- Macro to add a generic force sensor. -->
+  <xacro:macro name="force_sensor_plugin_macro" params="namespace force_sensor_suffix parent_link force_sensor_topic
+		force_sensor_truth_topic parent_frame_id reference_frame_id mass_force_sensor measurement_divisor	measurement_delay unknown_delay
+		noise_normal_linear_force noise_normal_torque noise_uniform_linear_force noise_uniform_torque *inertia *origin">
+    <!-- force-to-ground link -->
+    <link name="${namespace}/force_sensor_${force_sensor_suffix}_link">
+      <inertial>
+        <xacro:insert_block name="inertia" />
+        <mass value="${mass_force_sensor}" />  <!-- [kg] -->
+      </inertial>
+    </link>
+    <!-- force-to-ground joint -->
+    <joint name="${namespace}/force_sensor_${force_sensor_suffix}_joint" type="revolute">
+      <parent link="${parent_link}" />
+      <xacro:insert_block name="origin" />
+      <child link="${namespace}/force_sensor_${force_sensor_suffix}_link" />
+      <limit upper="0" lower="0" effort="0" velocity="0" />
+    </joint>
+		<!-- force-to-ground plugin -->
+    <gazebo>
+      <plugin filename="librotors_gazebo_force_sensor_plugin.so" name="force_sensor_${force_sensor_suffix}">
+        <linkName>${namespace}/force_sensor_${force_sensor_suffix}_link</linkName>
+        <robotNamespace>${namespace}</robotNamespace>
+        <forceSensorTopic>${force_sensor_topic}</forceSensorTopic>
+        <forceSensorTruthTopic>${force_sensor_truth_topic}</forceSensorTruthTopic>
+        <parentFrameId>${parent_frame_id}</parentFrameId> <!-- Use the scoped link name here. e.g. Model::link. -->
+				<referenceFrameId>${reference_frame_id}</referenceFrameId>
+        <measurementDivisor>${measurement_divisor}</measurementDivisor>
+				<!-- only every (seq % measurementDivisor) == 0 measurement is published [int] -->
+        <measurementDelay>${measurement_delay}</measurementDelay>
+				<!-- time that measurement gets held back before it's published in [simulation cycles (int)] -->
+        <unknownDelay>${unknown_delay}</unknownDelay> <!-- additional delay, that just gets added to the timestamp [s] -->
+        <noiseNormalLinearForce>${noise_normal_linear_force}</noiseNormalLinearForce>
+				<!-- standard deviation of additive white gaussian noise [N] -->
+        <noiseNormalTorque>${noise_normal_torque}</noiseNormalTorque> <!-- standard deviation of additive white gaussian noise [N*m] -->
+        <noiseUniformLinearForce>${noise_uniform_linear_force}</noiseUniformLinearForce> <!-- symmetric bounds of uniform noise [N] -->
+        <noiseUniformTorque>${noise_uniform_torque}</noiseUniformTorque> <!-- symmetric bounds of uniform noise [N*m] -->
+      </plugin>
+    </gazebo>
+  </xacro:macro>
+	<!-- Macro to add a default force-to-ground sensor. -->
+  <xacro:macro name="default_force_sensor" params="namespace suffix link reference_frame">
+		<xacro:force_sensor_plugin_macro
+			namespace="${namespace}/force_sensor_${suffix}"
+			force_sensor_suffix="${suffix}"
+			parent_link="${link}"
+			force_sensor_topic="force_sensor"
+			force_sensor_truth_topic="force_sensor_truth"
+			parent_frame_id="${link}"
+			reference_frame_id="${reference_frame}"
+			mass_force_sensor="0.001"
+			measurement_divisor="1"
+			measurement_delay="0"
+			unknown_delay="0.0"
+			noise_normal_linear_force="0 0 0"
+			noise_normal_torque="0 0 0"
+			noise_uniform_linear_force="0 0 0"
+			noise_uniform_torque="0 0 0" >
+			<inertia ixx="0.001" ixy="0.0" ixz="0.0" iyy="0.001" iyz="0.0" izz="0.001"/>
+			<!-- [kg m^2] [kg m^2] [kg m^2] [kg m^2] [kg m^2] [kg m^2] -->
+			<origin xyz="0.0 0.0 0.0" rpy="0.0 0.0 0.0"/>
+		</xacro:force_sensor_plugin_macro>
+	</xacro:macro>
 </robot>

Commit message: Added the mavlink interface plugin to the iris model via sdf file

File: rotors_description/urdf/component_snippets.xacro (robot description, xacro)
@@ -113,4 +113,14 @@
         <commandRateThrustSubTopic>command/rate</commandRateThrustSubTopic>
         <commandMotorSpeedSubTopic>command/motor_speed</commandMotorSpeedSubTopic>
+        <imuSubTopic>${imu_sub_topic}</imuSubTopic>
+        <motorSpeedCommandPubTopic>gazebo/command/motor_speed</motorSpeedCommandPubTopic>
+      </plugin>
+    </gazebo>
+  </xacro:macro>
+  <!-- Macro to add the mavlink interface. -->
+  <xacro:macro name="mavlink_interface_macro" params="namespace imu_sub_topic">
+    <gazebo>
+      <plugin name="mavlink_interface" filename="librotors_gazebo_mavlink_interface.so">
+        <robotNamespace>${namespace}</robotNamespace>
         <imuSubTopic>${imu_sub_topic}</imuSubTopic>
         <motorSpeedCommandPubTopic>gazebo/command/motor_speed</motorSpeedCommandPubTopic>

File: rotors_description/urdf/iris_base.xacro (robot description, xacro)
@@ -10,4 +10,10 @@
     >
   </xacro:controller_plugin_macro>
+  <!-- Instantiate mavlink telemetry interface. -->
+  <xacro:mavlink_interface_macro
+    namespace="${namespace}"
+    imu_sub_topic="imu"
+    >
+  </xacro:mavlink_interface_macro>
   <!-- Mount an ADIS16448 IMU. -->
   <xacro:imu_plugin_macro

Commit message: added a mesh for the vi_camera and fixed the mesh for the vi_sensor

File: rotors_description/urdf/component_snippets.xacro (robot description, xacro)
@@ -47,5 +47,5 @@
       <xacro:if value="${enable_visual}">
         <visual>
-          <origin xyz="0 0 0" rpy="0 0 0" />
+          <origin xyz="0 0 0" rpy="0 ${pi/2} 0" />
           <geometry>
             <xacro:insert_block name="geometry" />
@@ -366,6 +366,6 @@
       noise_mean="0.0"
       noise_stddev="0.007"
-      enable_visual="false">
-      <cylinder length="0.01" radius="0.007" />
+      enable_visual="true">
+      <mesh filename="package://rotors_description/meshes/vi_camera.dae" scale="1 1 1" />
       <xacro:insert_block name="origin" />
     </xacro:camera_macro>

Commit message: added force sensor to delta_manipulator

File: rotors_description/urdf/component_snippets.xacro (robot description, xacro)
@@ -627,9 +627,15 @@
 	<!-- Macro to add a generic force sensor. -->
   <xacro:macro name="force_sensor_plugin_macro" params="namespace force_sensor_suffix parent_link force_sensor_topic
-		force_sensor_truth_topic parent_frame_id reference_frame_id mass_force_sensor lin_force_meas_enabled torque_meas_enabled
-		measurement_divisor	measurement_delay unknown_delay noise_normal_linear_force noise_normal_torque noise_uniform_linear_force
-		noise_uniform_torque *inertia *origin">
+		force_sensor_truth_topic wrench_vector_pub_topic parent_frame_id reference_frame_id mass_force_sensor lin_force_meas_enabled
+		torque_meas_enabled disp_wrench_vector measurement_divisor	measurement_delay unknown_delay noise_normal_linear_force
+		noise_normal_torque noise_uniform_linear_force noise_uniform_torque *inertia *origin">
     <!-- force-to-ground link -->
     <link name="${namespace}/force_sensor_${force_sensor_suffix}_link">
+			<visual>
+        <origin xyz="0 0 0" rpy="0 0 0" />
+        <geometry>
+          <cylinder length="0.01" radius="0.005" />
+        </geometry>
+      </visual>
       <inertial>
         <xacro:insert_block name="inertia" />
@@ -637,4 +643,7 @@
       </inertial>
     </link>
+		<gazebo reference="${namespace}/force_sensor_${force_sensor_suffix}_link">
+			<material>Gazebo/Yellow</material>
+		</gazebo>
     <!-- force-to-ground joint -->
     <joint name="${namespace}/force_sensor_${force_sensor_suffix}_joint" type="revolute">
@@ -651,8 +660,10 @@
         <forceSensorTopic>${force_sensor_topic}</forceSensorTopic>
         <forceSensorTruthTopic>${force_sensor_truth_topic}</forceSensorTruthTopic>
+				<wrenchVectorTopic>${wrench_vector_pub_topic}</wrenchVectorTopic>
         <parentFrameId>${parent_frame_id}</parentFrameId> <!-- Use the scoped link name here. e.g. Model::link. -->
 				<referenceFrameId>${reference_frame_id}</referenceFrameId>
 				<linForceMeasEnabled>${lin_force_meas_enabled}</linForceMeasEnabled>
 				<torqueMeasEnabled>${torque_meas_enabled}</torqueMeasEnabled>
+				<dispWrenchVector>${disp_wrench_vector}</dispWrenchVector>
         <measurementDivisor>${measurement_divisor}</measurementDivisor>
 				<!-- only every (seq % measurementDivisor) == 0 measurement is published [int] -->
@@ -676,9 +687,11 @@
 			force_sensor_topic="force_sensor"
 			force_sensor_truth_topic="force_sensor_truth"
+			wrench_vector_pub_topic="wrench_vector"
 			parent_frame_id="${link}"
 			reference_frame_id="${reference_frame}"
 			mass_force_sensor="0.001"
-			lin_force_meas_enabled="false"
-			torque_meas_enabled="false"
+			lin_force_meas_enabled="true"
+			torque_meas_enabled="true"
+			disp_wrench_vector="true"
 			measurement_divisor="1"
 			measurement_delay="0"

Commit message: added single wall world for simple demo + fixed force sensor plugin

File: rotors_description/urdf/component_snippets.xacro (robot description, xacro)
@@ -628,14 +628,20 @@
   <xacro:macro name="force_sensor_plugin_macro" params="namespace force_sensor_suffix parent_link force_sensor_topic
 		force_sensor_truth_topic wrench_vector_pub_topic parent_frame_id reference_frame_id mass_force_sensor lin_force_meas_enabled
-		torque_meas_enabled disp_wrench_vector measurement_divisor	measurement_delay unknown_delay noise_normal_linear_force
+		torque_meas_enabled disp_wrench_vector measurement_divisor	measurement_delay unknown_delay cutoff_frequency noise_normal_linear_force
 		noise_normal_torque noise_uniform_linear_force noise_uniform_torque *inertia *origin">
     <!-- force-to-ground link -->
-    <link name="${namespace}/force_sensor_${force_sensor_suffix}_link">
+    <link name="${namespace}/force_sensor_${force_sensor_suffix}">
 			<visual>
         <origin xyz="0 0 0" rpy="0 0 0" />
         <geometry>
-          <cylinder length="0.01" radius="0.005" />
+          <cylinder length="0.05" radius="0.01" />
         </geometry>
       </visual>
+			<collision>
+        <origin xyz="0 0 0" rpy="0 0 0" />
+        <geometry>
+          <cylinder length="0.05" radius="0.01" />
+        </geometry>
+      </collision>
       <inertial>
         <xacro:insert_block name="inertia" />
@@ -643,18 +649,21 @@
       </inertial>
     </link>
-		<gazebo reference="${namespace}/force_sensor_${force_sensor_suffix}_link">
+		<gazebo reference="${namespace}/force_sensor_${force_sensor_suffix}">
 			<material>Gazebo/Yellow</material>
 		</gazebo>
     <!-- force-to-ground joint -->
-    <joint name="${namespace}/force_sensor_${force_sensor_suffix}_joint" type="revolute">
+    <joint name="${namespace}/force_sensor_${force_sensor_suffix}" type="revolute">
       <parent link="${parent_link}" />
       <xacro:insert_block name="origin" />
-      <child link="${namespace}/force_sensor_${force_sensor_suffix}_link" />
+      <child link="${namespace}/force_sensor_${force_sensor_suffix}" />
       <limit upper="0" lower="0" effort="0" velocity="0" />
     </joint>
+		<gazebo reference="${namespace}/force_sensor_${force_sensor_suffix}">
+	    <provideFeedback>true</provideFeedback>
+		</gazebo>
 		<!-- force-to-ground plugin -->
     <gazebo>
       <plugin filename="librotors_gazebo_force_sensor_plugin.so" name="force_sensor_${force_sensor_suffix}">
-        <linkName>${namespace}/force_sensor_${force_sensor_suffix}_link</linkName>
+        <linkName>${namespace}/force_sensor_${force_sensor_suffix}</linkName>
         <robotNamespace>${namespace}</robotNamespace>
         <forceSensorTopic>${force_sensor_topic}</forceSensorTopic>
@@ -671,4 +680,5 @@
 				<!-- time that measurement gets held back before it's published in [simulation cycles (int)] -->
         <unknownDelay>${unknown_delay}</unknownDelay> <!-- additional delay, that just gets added to the timestamp [s] -->
+				<cutoffFrequency>${cutoff_frequency}</cutoffFrequency> <!-- cut-off frequency of first order filter [Hz] -->
         <noiseNormalLinearForce>${noise_normal_linear_force}</noiseNormalLinearForce>
 				<!-- standard deviation of additive white gaussian noise [N] -->
@@ -680,13 +690,13 @@
   </xacro:macro>
 	<!-- Macro to add a default force-to-ground sensor. -->
-  <xacro:macro name="default_force_sensor" params="namespace suffix link reference_frame">
+  <xacro:macro name="default_force_sensor" params="namespace suffix parent_link reference_frame">
 		<xacro:force_sensor_plugin_macro
-			namespace="${namespace}/force_sensor_${suffix}"
+			namespace="${namespace}"
 			force_sensor_suffix="${suffix}"
-			parent_link="${link}"
+			parent_link="${parent_link}"
 			force_sensor_topic="force_sensor"
 			force_sensor_truth_topic="force_sensor_truth"
 			wrench_vector_pub_topic="wrench_vector"
-			parent_frame_id="${link}"
+			parent_frame_id="${parent_link}"
 			reference_frame_id="${reference_frame}"
 			mass_force_sensor="0.001"
@@ -697,4 +707,5 @@
 			measurement_delay="0"
 			unknown_delay="0.0"
+			cutoff_frequency="10.0"
 			noise_normal_linear_force="0 0 0"
 			noise_normal_torque="0 0 0"

Commit message: icra final version

File: rotors_description/urdf/component_snippets.xacro (robot description, xacro)
@@ -613,10 +613,10 @@
       imu_topic="imu"
       mass_imu_sensor="0.015"
-      gyroscope_noise_density="0.0003394"
-      gyroscopoe_random_walk="0.000038785"
+      gyroscope_noise_density="0.0013"
+      gyroscopoe_random_walk="0.000013"
       gyroscope_bias_correlation_time="1000.0"
       gyroscope_turn_on_bias_sigma="0.0087"
-      accelerometer_noise_density="0.004"
-      accelerometer_random_walk="0.006"
+      accelerometer_noise_density="0.0083"
+      accelerometer_random_walk="0.00083"
       accelerometer_bias_correlation_time="300.0"
       accelerometer_turn_on_bias_sigma="0.1960">

File: rotors_description/urdf/firefly.xacro (robot description, xacro)
@@ -31,10 +31,10 @@
   <xacro:property name="motor_constant" value="8.54858e-06" /> <!-- [kg m/s^2] -->
   <xacro:property name="moment_constant" value="0.016" /> <!-- [m] -->
-  <xacro:property name="time_constant_up" value="0.0125" /> <!-- [s] -->
+  <xacro:property name="time_constant_up" value="0.025" /> <!-- [s] -->
   <xacro:property name="time_constant_down" value="0.025" /> <!-- [s] -->
   <xacro:property name="max_rot_velocity" value="838" /> <!-- [rad/s] -->
   <xacro:property name="sin30" value="0.5" />
   <xacro:property name="cos30" value="0.866025403784" />
-  <xacro:property name="rotor_drag_coefficient" value="8.06428e-05" />
+  <xacro:property name="rotor_drag_coefficient" value="0.0176" />
   <xacro:property name="rolling_moment_coefficient" value="0.000001" />
   <!-- Property Blocks -->

Commit message: fix namespace variable
missing $ sign

File: rotors_description/urdf/component_snippets.xacro (robot description, xacro)
@@ -484,5 +484,5 @@
       </inertial>
     </link>
-    <joint name="{namespace}_vi_sensor_joint" type="fixed">
+    <joint name="${namespace}_vi_sensor_joint" type="fixed">
       <xacro:insert_block name="origin" />
       <parent link="${parent_link}" />

Commit message: add optical joint for camera

File: rotors_description/urdf/component_snippets.xacro (robot description, xacro)
@@ -62,4 +62,10 @@
       <parent link="${parent_link}" />
       <child link="${namespace}/camera_${camera_suffix}_link" />
+    </joint>
+    <link name="${namespace}/camera_${camera_suffix}_optical_link" />
+    <joint name="${namespace}/camera_${camera_suffix}_optical_joint" type="fixed" >
+      <origin xyz="0 0 0" rpy="${-pi/2} 0 ${-pi/2}" />
+      <parent link="${namespace}/camera_${camera_suffix}_link" />
+      <child link="${namespace}/camera_${camera_suffix}_optical_link" />
     </joint>
     <gazebo reference="${namespace}/camera_${camera_suffix}_link">

Commit message: added optical link also to stereo camera

File: rotors_description/urdf/component_snippets.xacro (robot description, xacro)
@@ -189,4 +189,10 @@
       <xacro:insert_block name="geometry" />
     </xacro:camera_joint_macro>
+    <link name="${namespace}/camera_left_optical_link" />
+    <joint name="${namespace}/camera_left_optical_joint" type="fixed" >
+      <origin xyz="0 0 0" rpy="${-pi/2} 0 ${-pi/2}" />
+      <parent link="${namespace}/camera_left_link" />
+      <child link="${namespace}/camera_left_optical_link" />
+    </joint>
     <!-- Both cameras in the pair are anchored off the left camera frame. -->
     <gazebo reference="${namespace}/camera_left_link">
