Commit message: Added/modified xacro files for velodyne puck

File: rotors_description/urdf/component_snippets.xacro (robot description, xacro)
@@ -29,4 +29,164 @@
         <rotorVelocitySlowdownSim>${rotor_velocity_slowdown_sim}</rotorVelocitySlowdownSim>
       </plugin>
+    </gazebo>
+  </xacro:macro>
+  <!-- Macro to add a Velodyne Puck -->
+  <xacro:macro name="velodyne_puck_sensor_macro"
+    params="namespace parent_link horizontal_res visualize_scan velodyne_suffix update_rate *origin">
+    <!-- BASE LINK DEFINITION -->
+    <link name="${namespace}/base_link">
+      <collision>
+        <origin xyz="0 0 0" rpy="0 0 0" />
+        <geometry>
+          <cylinder radius="0.05165" length="0.0188" />
+        </geometry>
+      </collision>
+      <visual>
+        <origin xyz="0 0 -0.0094" rpy="0 0 0" />
+        <geometry>
+          <mesh filename="package://rotors_description/meshes/VLP16_base.dae" scale="1 1 1" />
+        </geometry>
+      </visual>
+      <inertial>
+        <mass value="0.05" />
+        <origin xyz="0 0 0" rpy="0 0 0" />
+        <inertia ixx="0.000030623" ixy="0" ixz="0" iyy="0.000030623" iyz="0" izz="0.000091036" />
+      </inertial>
+    </link>
+    <!-- SCANNER SCREEN LINK DEFINITION -->
+    <link name="${namespace}/scan_link">
+      <pose>0 0 0.028 0 0 0</pose>
+      <collision>
+        <origin xyz="0 0 0" rpy="0 0 0" />
+        <geometry>
+          <cylinder radius="0.005165" length="0.0392" />
+        </geometry>
+      </collision>
+      <visual>
+        <origin xyz="0 0 -0.040" rpy="0 0 0" />
+        <geometry>
+          <mesh filename="package://rotors_description/meshes/VLP16_scan.dae" scale="1 1 1" />
+        </geometry>
+      </visual>
+      <inertial>
+        <!-- mass ~ 0.730g. However firefly cannot hover with that mass -->
+        <mass value="0.00730" />
+        <origin xyz="0 0 0" rpy="0 0 0" />
+        <inertia ixx="0.000090623" ixy="0" ixz="0" iyy="0.000090623" iyz="0" izz="0.000091036" />
+      </inertial>
+    </link>
+    <!-- TOP LINK DEFINITION -->
+    <link name="${namespace}/top_link">
+      <pose>0 0 0.056 0 0 0</pose>
+      <collision>
+        <origin xyz="0 0 0" rpy="0 0 0" />
+        <geometry>
+          <cylinder radius="0.0005165" length="0.0147" />
+        </geometry>
+      </collision>
+      <visual>
+        <origin xyz="0 0 -0.068" rpy="0 0 0" />
+        <geometry>
+          <mesh filename="package://rotors_description/meshes/VLP16_top.dae" scale="1 1 1" />
+        </geometry>
+      </visual>
+      <inertial>
+        <mass value="0.05" />
+        <origin xyz="0 0 0" rpy="0 0 0" />
+        <inertia ixx="0.000030623" ixy="0" ixz="0" iyy="0.000030623" iyz="0" izz="0.000031036" />
+      </inertial>
+    </link>
+    <!-- JOINT DEFINITIONS -->
+    <joint name="${parent_link}_to_${namespace}_base" type="fixed">
+      <parent link="${parent_link}"/>
+      <child link="${namespace}/base_link"/>
+      <xacro:insert_block name="origin" />
+    </joint>
+    <joint name="${namespace}_base_to_${namespace}_scan" type="fixed">
+      <parent link="${namespace}/base_link"/>
+      <child link="${namespace}/scan_link"/>
+      <origin xyz="0 0 0.030"  />
+    </joint>
+    <joint name="${namespace}_scan_to_${namespace}_top" type="fixed">
+      <parent link="${namespace}/scan_link"/>
+      <child link="${namespace}/top_link"/>
+      <origin xyz="0 0 0.027"  />
+    </joint>
+    <xacro:block_laser_macro
+      namespace="${namespace}"
+      parent_link="${namespace}/scan_link"
+      visualize_scan="${visualize_scan}"
+      horizontal_fov_min="0"
+      horizontal_fov_max="${2 * pi}"
+      horizontal_samples="900"
+      horizontal_res="${horizontal_res}"
+      vertical_fov_min="${-15 / 360 *  pi}"
+      vertical_fov_max="${ 15 / 360 *  pi}"
+      vertical_samples="16"
+      vertical_res="1.0"
+      update_rate="${update_rate}"
+      range_min="0.10"
+      range_max="100.0"
+      range_res="0.02"
+      topic_name="${namespace}/velodyne_puck${velodyne_suffix}/scan"
+      frame_name="velodyne_puck${velodyne_suffix}"
+      always_on="true"
+      gaussian_noise="0.0009">
+      <origin xyz="0.0 0.0 -0.004645" rpy="0 0 0" />
+    </xacro:block_laser_macro>
+  </xacro:macro>
+  <!-- Macro to add a block laser -->
+  <xacro:macro name="block_laser_macro"
+    params="namespace  parent_link visualize_scan horizontal_fov_min
+    horizontal_fov_max horizontal_samples horizontal_res vertical_fov_min
+    vertical_fov_max vertical_samples vertical_res update_rate range_min
+    range_max range_res topic_name frame_name always_on gaussian_noise *origin">
+    <!-- This model has 3 links : scan, base, top
+         Each has separate visuals and collision blocks as well as inertias.
+         Finally the sensor 'ray' is connected to the 'scan' link.
+    -->
+    <gazebo reference="${parent_link}">
+      <sensor type="ray" name="${namespace}_${frame_name}">
+        <pose>0 0 -0.004645 0 0 0</pose>
+        <always_on>true</always_on>
+        <visualize>${visualize_scan}</visualize>
+        <update_rate>${update_rate}</update_rate>
+        <ray>
+          <!-- Noise is added in the plugin -->
+          <noise>
+            <type>gaussian</type>
+            <mean>0.0</mean>
+            <stddev>0.000</stddev>
+          </noise>
+          <scan>
+            <vertical>
+              <samples>${vertical_samples}</samples>
+              <resolution>1</resolution>
+              <min_angle>${vertical_fov_min}</min_angle>
+              <max_angle>${vertical_fov_max}</max_angle>
+            </vertical>
+            <horizontal>
+              <samples>${horizontal_samples}</samples>
+              <resolution>${horizontal_res}</resolution>
+              <min_angle>${horizontal_fov_min}</min_angle>
+              <max_angle>${horizontal_fov_max}</max_angle>
+            </horizontal>
+          </scan>
+          <range>
+            <min>${range_min}</min>
+            <max>${range_max}</max>
+            <resolution>${range_res}</resolution>
+          </range>
+        </ray>
+        <!-- The plugin declarion should be inside the sensor tag for proper driver behavior -->
+        <plugin name="gazebo_ros_${frame_name}_controller" filename="libgazebo_ros_block_laser.so">
+          <robotNamespace>${namespace}</robotNamespace>
+          <alwaysOn>${always_on}</alwaysOn>
+          <updateRate>${update_rate}</updateRate>
+          <topicName>${topic_name}</topicName>
+          <frameName>${frame_name}</frameName>
+          <gaussianNoise>${gaussian_noise}</gaussianNoise>
+        </plugin>
+      </sensor>
     </gazebo>
   </xacro:macro>

Commit message: some cleanup for final version

File: rotors_description/urdf/component_snippets.xacro (robot description, xacro)
@@ -660,5 +660,5 @@
       gyroscope_bias_correlation_time="1000.0"
       gyroscope_turn_on_bias_sigma="0.0087"
-      accelerometer_noise_density="0.0083"
+      accelerometer_noise_density="0.083"
       accelerometer_random_walk="0.00083"
       accelerometer_bias_correlation_time="300.0"

File: rotors_description/urdf/firefly.xacro (robot description, xacro)
@@ -28,5 +28,5 @@
   <xacro:property name="arm_length" value="0.215" /> <!-- [m] -->
   <xacro:property name="rotor_offset_top" value="0.037" /> <!-- [m] -->
-  <xacro:property name="radius_rotor" value="0.1" /> <!-- [m] -->
+  <xacro:property name="radius_rotor" value="0.1025" /> <!-- [m] -->
   <xacro:property name="motor_constant" value="8.54858e-06" /> <!-- [kg m] -->
   <xacro:property name="moment_constant" value="1.3677728e-07" /> <!-- [kg m^2] -->
@@ -38,6 +38,8 @@
   <xacro:property name="rotor_drag_coefficient" value="0.0176" />
   <xacro:property name="rolling_moment_coefficient" value="0.000001" />
+  <!--xacro:property name="forces_noise_density" value="0.01 0.01 0.01" /> -->
+  <!--xacro:property name="moments_noise_density" value="0.004 0.004 0.002" /> -->
   <xacro:property name="forces_noise_density" value="0.01 0.01 0.01" />
-  <xacro:property name="moments_noise_density" value="0.004 0.004 0.002" />
+  <xacro:property name="moments_noise_density" value="0.004 0.004 0.004" />
   <xacro:property name="main_body_drag_coefficient" value="0.002 0.002 0.0" />
   <!-- Property Blocks -->
@@ -47,5 +49,6 @@
   <!-- inertia of a single rotor, assuming it is a cuboid. Height=3mm, width=15mm -->
   <xacro:property name="rotor_inertia">
-    <xacro:box_inertia x="${radius_rotor}" y="0.015" z="0.003" mass="${mass_rotor*rotor_velocity_slowdown_sim}" />
+    <!-- <xacro:box_inertia x="${2 * radius_rotor}" y="0.015" z="0.003" mass="${mass_rotor*rotor_velocity_slowdown_sim}" /> -->
+    <xacro:rotor_disk_inertia rotor_velocity_slowdown_sim="${rotor_velocity_slowdown_sim}" radius="${radius_rotor}" mass="${mass_rotor}" />
   </xacro:property>
   <!-- Included URDF Files -->

File: rotors_description/urdf/multirotor_base.xacro (robot description, xacro)
@@ -22,4 +22,12 @@
       iyy="${0.0833333 * mass * (x*x + z*z)}" iyz="0.0"
       izz="${0.0833333 * mass * (x*x + y*y)}" />
+  </xacro:macro>
+  <!-- Macro for the rotor inertia, we approximate it with a cylinder of zero height.
+  Because the angular velocity slow down of the rotor speed mainly has an influence
+  on the inertia in z we adapt the inertia -->
+  <xacro:macro name="rotor_disk_inertia" params="rotor_velocity_slowdown_sim radius mass">
+    <inertia ixx="${0.25 * mass * (radius*radius)}" ixy="0.0" ixz="0.0"
+      iyy="${0.25 * mass * (radius*radius)}" iyz="0.0"
+      izz="${0.5 * mass * (radius*radius)*rotor_velocity_slowdown_sim}" />
   </xacro:macro>
   <!-- Macro for the inertial properties of a box -->

Commit message: Adding a macro for magnetometer component

File: rotors_description/urdf/component_snippets.xacro (robot description, xacro)
@@ -315,5 +315,5 @@
     </gazebo>
   </xacro:macro>
-<!-- Macro to add a generic odometry sensor. -->
+  <!-- Macro to add a generic odometry sensor. -->
   <xacro:macro name="odometry_plugin_macro"
     params="
@@ -367,4 +367,64 @@
         </xacro:if>
       </plugin>
+    </gazebo>
+  </xacro:macro>
+  <!-- Macro to add a magnetometer. -->
+  <xacro:macro name="magnetometer_plugin_macro"
+    params="namespace magnetometer_suffix parent_link magnetometer_topic
+      mass_magnetometer_sensor noise_normal_mag_x noise_normal_mag_bias_x
+      noise_normal_mag_y noise_normal_mag_bias_y noise_normal_mag_z
+      noise_normal_mag_bias_z *inertia *origin">
+    <!-- Magnetometer link -->
+    <link name="${namespace}/magnetometer${magnetometer_suffix}_link">
+      <inertial>
+        <xacro:insert_block name="inertia" />
+        <mass value="${mass_magnetometer_sensor}" />  <!-- [kg] -->
+        <origin xyz="0 0 0" rpy="0 0 0" />
+      </inertial>
+    </link>
+    <!-- Magnetometer joint -->
+    <joint name="${namespace}/magnetometer${magnetometer_suffix}_joint" type="revolute">
+      <xacro:insert_block name="origin" />
+      <parent link="${parent_link}" />
+      <child link="${namespace}/magnetometer${magnetometer_suffix}_link" />
+      <limit upper="0" lower="0" effort="0" velocity="0" />
+    </joint>
+    <gazebo reference="${namespace}/magnetometer${magnetometer_suffix}_link">
+      <sensor type="magnetometer" name="${namespace}/magnetometer${magnetometer_suffix}">
+        <pose>0 0 0 0 0 0</pose>
+        <visualize>0</visualize>
+        <always_on>1</always_on>
+        <magnetometer>
+          <x>
+            <noise type="gaussian">
+              <mean>0.0</mean>
+              <stddev>${noise_normal_mag_x}</stddev>
+              <bias_mean>0.0</bias_mean>
+              <bias_stddev>${noise_normal_mag_bias_x}</bias_stddev>
+            </noise>
+          </x>
+          <y>
+            <noise type="gaussian">
+              <mean>0.0</mean>
+              <stddev>${noise_normal_mag_y}</stddev>
+              <bias_mean>0.0</bias_mean>
+              <bias_stddev>${noise_normal_mag_bias_y}</bias_stddev>
+            </noise>
+          </y>
+          <z>
+            <noise type="gaussian">
+              <mean>0.0</mean>
+              <stddev>${noise_normal_mag_z}</stddev>
+              <bias_mean>0.0</bias_mean>
+              <bias_stddev>${noise_normal_mag_bias_z}</bias_stddev>
+            </noise>
+          </z>
+        </magnetometer>
+        <plugin filename="librotors_gazebo_magnetometer_plugin.so" name="rotors_gazebo_magnetometer${magnetometer_suffix}_plugin">
+          <robotNamespace>${namespace}</robotNamespace> <!-- (string, required): ros namespace in which the messages are published -->
+          <linkName>${namespace}/magnetometer${magnetometer_suffix}_link</linkName> <!-- (string, required): name of the body which holds the magnetometer sensor -->
+          <magnetometerTopic>${magnetometer_topic}</magnetometerTopic> <!-- (string): name of the sensor output topic and prefix of service names (defaults to magnetic_field) -->
+        </plugin>
+      </sensor>
     </gazebo>
   </xacro:macro>
@@ -669,4 +729,21 @@
     </xacro:imu_plugin_macro>
   </xacro:macro>
+  <xacro:macro name="default_magnetometer" params="namespace parent_link">
+    <xacro:magnetometer_plugin_macro
+      namespace="${namespace}"
+      magnetometer_suffix=""
+      parent_link="${parent_link}"
+      magnetometer_topic="magnetic_field"
+      mass_magnetometer_sensor="0.015"
+      noise_normal_mag_x="0.0"
+      noise_normal_mag_bias_x="0.0"
+      noise_normal_mag_y="0.0"
+      noise_normal_mag_bias_y="0.0"
+      noise_normal_mag_z="0.0"
+      noise_normal_mag_bias_z="0.0">
+      <inertia ixx="0.00001" ixy="0.0" ixz="0.0" iyy="0.00001" iyz="0.0" izz="0.00001" />
+      <origin xyz="0 0 0" rpy="0 0 0" />
+    </xacro:magnetometer_plugin_macro>
+  </xacro:macro>
   <xacro:macro name="default_mavlink_interface" params="namespace imu_sub_topic rotor_count">
     <xacro:mavlink_interface_macro

Commit message: Adding GPS to components snipets and mounting it on a fixed-wing Techpod model

File: rotors_description/urdf/component_snippets.xacro (robot description, xacro)
@@ -367,4 +367,81 @@
         </xacro:if>
       </plugin>
+    </gazebo>
+  </xacro:macro>
+  <!-- Macro to add a GPS sensor. -->
+  <xacro:macro name="gps_plugin_macro"
+    params="namespace gps_suffix parent_link gps_topic ground_speed_topic
+      mass_gps_sensor horizontal_pos_std_dev vertical_pos_std_dev
+      horizontal_vel_std_dev vertical_vel_std_dev *inertia *origin">
+    <!-- GPS link -->
+    <link name="${namespace}/gps${gps_suffix}_link">
+      <inertial>
+        <xacro:insert_block name="inertia" />
+        <mass value="${mass_gps_sensor}" />  <!-- [kg] -->
+        <origin xyz="0 0 0" rpy="0 0 0" />
+      </inertial>
+    </link>
+    <!-- GPS joint -->
+    <joint name="${namespace}/gps${gps_suffix}_joint" type="revolute">
+      <xacro:insert_block name="origin" />
+      <parent link="${parent_link}" />
+      <child link="${namespace}/gps${gps_suffix}_link" />
+      <limit upper="0" lower="0" effort="0" velocity="0" />
+    </joint>
+    <gazebo reference="${namespace}/gps${gps_suffix}_link">
+      <sensor type="gps" name="${namespace}_gps${gps_suffix}">
+        <pose>0 0 0 0 0 0</pose>
+        <visualize>0</visualize>
+        <always_on>1</always_on>
+        <update_rate>5</update_rate>
+        <gps>
+          <position_sensing>
+            <horizontal>
+              <noise type="gaussian">
+                <mean>0.0</mean>
+                <stddev>${horizontal_pos_std_dev}</stddev>
+                <bias_mean>0.0</bias_mean>
+                <bias_stddev>0.0</bias_stddev>
+              </noise>
+            </horizontal>
+            <vertical>
+              <noise type="gaussian">
+                <mean>0.0</mean>
+                <stddev>${vertical_pos_std_dev}</stddev>
+                <bias_mean>0.0</bias_mean>
+                <bias_stddev>0.0</bias_stddev>
+              </noise>
+            </vertical>
+          </position_sensing>
+          <velocity_sensing>
+            <horizontal>
+              <noise type="gaussian">
+                <mean>0.0</mean>
+                <stddev>${horizontal_vel_std_dev}</stddev>
+                <bias_mean>0.0</bias_mean>
+                <bias_stddev>0.0</bias_stddev>
+              </noise>
+            </horizontal>
+            <vertical>
+              <noise type="gaussian">
+                <mean>0.0</mean>
+                <stddev>${vertical_vel_std_dev}</stddev>
+                <bias_mean>0.0</bias_mean>
+                <bias_stddev>0.0</bias_stddev>
+              </noise>
+            </vertical>
+          </velocity_sensing>
+        </gps>
+        <plugin filename="librotors_gazebo_gps_plugin.so" name="rotors_gazebo_gps${gps_suffix}_plugin">
+          <robotNamespace>${namespace}</robotNamespace> <!-- (string, required): ros namespace in which the messages are published -->
+          <linkName>${namespace}/gps${gps_suffix}_link</linkName> <!-- (string, required): name of the body which holds the GPS sensor -->
+          <gpsTopic>${gps_topic}</gpsTopic> <!-- (string): name of the sensor output topic and prefix of service names (defaults to 'gps') -->
+          <groundSpeedTopic>${ground_speed_topic}</groundSpeedTopic> <!-- (string): name of the ground speed output topic (defaults to 'ground_speed') -->
+          <horPosStdDev>${horizontal_pos_std_dev}</horPosStdDev> <!-- standard deviation for horizontal position noise [m] -->
+          <verPosStdDev>${vertical_pos_std_dev}</verPosStdDev> <!-- standard deviation for vertical position noise [m] -->
+          <horVelStdDev>${horizontal_vel_std_dev}</horVelStdDev> <!-- standard deviation for horizontal speed noise [m/s] -->
+          <verVelStdDev>${vertical_vel_std_dev}</verVelStdDev> <!-- standard deviation for vertical speed noise [m/s] -->
+        </plugin>
+      </sensor>
     </gazebo>
   </xacro:macro>
@@ -706,4 +783,21 @@
     </xacro:imu_plugin_macro>
   </xacro:macro>
+  <xacro:macro name="default_gps" params="namespace parent_link">
+    <!-- Default GPS. -->
+    <xacro:gps_plugin_macro
+      namespace="${namespace}"
+      gps_suffix=""
+      parent_link="${parent_link}"
+      gps_topic="gps"
+      ground_speed_topic="ground_speed"
+      mass_gps_sensor="0.015"
+      horizontal_pos_std_dev="3.0"
+      vertical_pos_std_dev="6.0"
+      horizontal_vel_std_dev="0.1"
+      vertical_vel_std_dev="0.1">
+      <inertia ixx="0.00001" ixy="0.0" ixz="0.0" iyy="0.00001" iyz="0.0" izz="0.00001" />
+      <origin xyz="0 0 0" rpy="0 0 0" />
+    </xacro:gps_plugin_macro>
+  </xacro:macro>
   <xacro:macro name="default_magnetometer" params="namespace parent_link">
     <!-- ADIS16448 Magnetometer. -->

File: rotors_description/urdf/techpod_base.xacro (robot description, xacro)
@@ -18,4 +18,6 @@
   <!-- Mount an ADIS16448 IMU. -->
   <xacro:default_imu namespace="${namespace}" parent_link="${namespace}/base_link" />
+  <!-- Mount a GPS. -->
+  <xacro:default_gps namespace="${namespace}" parent_link="${namespace}/base_link" />
   <!-- Mount a magnetometer. -->
   <xacro:default_magnetometer namespace="${namespace}" parent_link="${namespace}/base_link" />

Commit message: Gazebo is now outputting debug messages to the console (verbose mode is turned on through launch file).

File: rotors_description/urdf/component_snippets.xacro (robot description, xacro)
@@ -237,4 +237,17 @@
     <gazebo>
       <plugin name="controller_interface" filename="librotors_gazebo_controller_interface.so">
+        <robotNamespace>${namespace}</robotNamespace>
+        <commandAttitudeThrustSubTopic>command/attitude</commandAttitudeThrustSubTopic>
+        <commandRateThrustSubTopic>command/rate</commandRateThrustSubTopic>
+        <commandMotorSpeedSubTopic>command/motor_speed</commandMotorSpeedSubTopic>
+        <imuSubTopic>${imu_sub_topic}</imuSubTopic>
+        <motorSpeedCommandPubTopic>gazebo/command/motor_speed</motorSpeedCommandPubTopic>
+      </plugin>
+    </gazebo>
+  </xacro:macro>
+  <!-- ==================== MSG INTERFACE MACRO ====================== -->
+  <xacro:macro name="msg_interface_macro" params="namespace imu_sub_topic">
+    <gazebo>
+      <plugin name="msg_interface" filename="librotors_gazebo_msg_interface.so">
         <robotNamespace>${namespace}</robotNamespace>
         <commandAttitudeThrustSubTopic>command/attitude</commandAttitudeThrustSubTopic>

Commit message: New Gazebo message interface plugin is loading correctly when hover sim is launched.

File: rotors_description/urdf/component_snippets.xacro (robot description, xacro)
@@ -247,7 +247,7 @@
   </xacro:macro>
   <!-- ==================== MSG INTERFACE MACRO ====================== -->
-  <xacro:macro name="msg_interface_macro" params="namespace imu_sub_topic">
+  <xacro:macro name="msg_interface_plugin_macro" params="namespace imu_sub_topic">
     <gazebo>
-      <plugin name="msg_interface" filename="librotors_gazebo_msg_interface.so">
+      <plugin name="msg_interface_plugin" filename="librotors_gazebo_msg_interface_plugin.so">
         <robotNamespace>${namespace}</robotNamespace>
         <commandAttitudeThrustSubTopic>command/attitude</commandAttitudeThrustSubTopic>

File: rotors_description/urdf/firefly_base.xacro (robot description, xacro)
@@ -22,4 +22,6 @@
   <!-- Instantiate a controller. -->
   <xacro:controller_plugin_macro namespace="${namespace}" imu_sub_topic="imu" />
+  <!-- Instantiate a message interface -->
+  <xacro:msg_interface_plugin_macro namespace="${namespace}" imu_sub_topic="imu" />
   <xacro:if value="$(arg enable_mavlink_interface)">
     <!-- Instantiate mavlink telemetry interface. -->
@@ -39,3 +41,5 @@
       wait_to_record_bag="$(arg wait_to_record_bag)" />
   </xacro:if>
+  <!-- Create a interface to send/receive messages to the outside world -->
+  <xacro:msg_interface_plugin />
 </robot>
