Commit message: Fixed issue with topic name differences between IMU/GPS plugins and the interface plugin.

File: rotors_description/urdf/component_snippets.xacro (robot description, xacro)
@@ -247,5 +247,5 @@
   </xacro:macro>
   <!-- ==================== MSG INTERFACE MACRO ====================== -->
-  <xacro:macro name="msg_interface_plugin_macro" params="namespace imu_sub_topic">
+  <xacro:macro name="msg_interface_plugin_macro" params="namespace imu_sub_topic gps_sub_topic">
     <gazebo>
       <plugin name="msg_interface_plugin" filename="librotors_gazebo_msg_interface_plugin.so">
@@ -255,4 +255,5 @@
         <commandMotorSpeedSubTopic>command/motor_speed</commandMotorSpeedSubTopic>
         <imuSubTopic>${imu_sub_topic}</imuSubTopic>
+        <gpsSubTopic>${gps_sub_topic}</gpsSubTopic>
         <motorSpeedCommandPubTopic>gazebo/command/motor_speed</motorSpeedCommandPubTopic>
       </plugin>

File: rotors_description/urdf/firefly_base.xacro (robot description, xacro)
@@ -22,6 +22,6 @@
   <!-- Instantiate a controller. -->
   <xacro:controller_plugin_macro namespace="${namespace}" imu_sub_topic="imu" />
-  <!-- Instantiate a message interface -->
-  <xacro:msg_interface_plugin_macro namespace="${namespace}" imu_sub_topic="imu" />
+  <!-- Instantiate a ROS message interface -->
+  <xacro:msg_interface_plugin_macro namespace="${namespace}" imu_sub_topic="imu" gps_sub_topic="gps" />
   <xacro:if value="$(arg enable_mavlink_interface)">
     <!-- Instantiate mavlink telemetry interface. -->

Commit message: Changed the name of the robot location GPS message to nav_sat_fix (since there is more than one GPS message type).

File: rotors_description/urdf/component_snippets.xacro (robot description, xacro)
@@ -247,5 +247,5 @@
   </xacro:macro>
   <!-- ==================== MSG INTERFACE MACRO ====================== -->
-  <xacro:macro name="msg_interface_plugin_macro" params="namespace imu_sub_topic gps_sub_topic">
+  <xacro:macro name="msg_interface_plugin_macro" params="namespace imu_sub_topic nav_sat_fix_sub_topic">
     <gazebo>
       <plugin name="msg_interface_plugin" filename="librotors_gazebo_msg_interface_plugin.so">
@@ -255,5 +255,5 @@
         <commandMotorSpeedSubTopic>command/motor_speed</commandMotorSpeedSubTopic>
         <imuSubTopic>${imu_sub_topic}</imuSubTopic>
-        <gpsSubTopic>${gps_sub_topic}</gpsSubTopic>
+        <navSatFixSubTopic>${nav_sat_fix_sub_topic}</navSatFixSubTopic>
         <motorSpeedCommandPubTopic>gazebo/command/motor_speed</motorSpeedCommandPubTopic>
       </plugin>

File: rotors_description/urdf/firefly_base.xacro (robot description, xacro)
@@ -23,5 +23,5 @@
   <xacro:controller_plugin_macro namespace="${namespace}" imu_sub_topic="imu" />
   <!-- Instantiate a ROS message interface -->
-  <xacro:msg_interface_plugin_macro namespace="${namespace}" imu_sub_topic="imu" gps_sub_topic="gps" />
+  <xacro:msg_interface_plugin_macro namespace="${namespace}" imu_sub_topic="imu" nav_sat_fix_sub_topic="nav_sat_fix" />
   <xacro:if value="$(arg enable_mavlink_interface)">
     <!-- Instantiate mavlink telemetry interface. -->

Commit message: ROS message interface plugin now converts magnetic field messages and publishes to ROS.

File: rotors_description/urdf/component_snippets.xacro (robot description, xacro)
@@ -247,5 +247,5 @@
   </xacro:macro>
   <!-- ==================== MSG INTERFACE MACRO ====================== -->
-  <xacro:macro name="msg_interface_plugin_macro" params="namespace imu_sub_topic nav_sat_fix_sub_topic">
+  <xacro:macro name="msg_interface_plugin_macro" params="namespace imu_sub_topic magnetic_field_sub_topic nav_sat_fix_sub_topic">
     <gazebo>
       <plugin name="msg_interface_plugin" filename="librotors_gazebo_msg_interface_plugin.so">
@@ -255,4 +255,5 @@
         <commandMotorSpeedSubTopic>command/motor_speed</commandMotorSpeedSubTopic>
         <imuSubTopic>${imu_sub_topic}</imuSubTopic>
+        <magneticFieldSubTopic>${magnetic_field_sub_topic}</magneticFieldSubTopic>
         <navSatFixSubTopic>${nav_sat_fix_sub_topic}</navSatFixSubTopic>
         <motorSpeedCommandPubTopic>gazebo/command/motor_speed</motorSpeedCommandPubTopic>

File: rotors_description/urdf/firefly_base.xacro (robot description, xacro)
@@ -23,5 +23,5 @@
   <xacro:controller_plugin_macro namespace="${namespace}" imu_sub_topic="imu" />
   <!-- Instantiate a ROS message interface -->
-  <xacro:msg_interface_plugin_macro namespace="${namespace}" imu_sub_topic="imu" nav_sat_fix_sub_topic="nav_sat_fix" />
+  <xacro:msg_interface_plugin_macro namespace="${namespace}" imu_sub_topic="imu" magnetic_field_sub_topic="magnetic_field" nav_sat_fix_sub_topic="nav_sat_fix" />
   <xacro:if value="$(arg enable_mavlink_interface)">
     <!-- Instantiate mavlink telemetry interface. -->

Commit message: Renamed gazebo_msg_interface_plugin to gazebo_ros_interface_plugin, closes #324.

File: rotors_description/urdf/component_snippets.xacro (robot description, xacro)
@@ -246,8 +246,10 @@
     </gazebo>
   </xacro:macro>
-  <!-- ==================== MSG INTERFACE MACRO ====================== -->
-  <xacro:macro name="msg_interface_plugin_macro" params="namespace imu_sub_topic magnetic_field_sub_topic nav_sat_fix_sub_topic">
+  <!-- =============================================================== -->
+  <!-- ==================== ROS INTERFACE MACRO ====================== -->
+  <!-- =============================================================== -->
+  <xacro:macro name="ros_interface_plugin_macro" params="namespace imu_sub_topic magnetic_field_sub_topic nav_sat_fix_sub_topic">
     <gazebo>
-      <plugin name="msg_interface_plugin" filename="librotors_gazebo_msg_interface_plugin.so">
+      <plugin name="ros_interface_plugin" filename="librotors_gazebo_ros_interface_plugin.so">
         <robotNamespace>${namespace}</robotNamespace>
         <commandAttitudeThrustSubTopic>command/attitude</commandAttitudeThrustSubTopic>

File: rotors_description/urdf/firefly_base.xacro (robot description, xacro)
@@ -23,5 +23,5 @@
   <xacro:controller_plugin_macro namespace="${namespace}" imu_sub_topic="imu" />
   <!-- Instantiate a ROS message interface -->
-  <xacro:msg_interface_plugin_macro namespace="${namespace}" imu_sub_topic="imu" magnetic_field_sub_topic="magnetic_field" nav_sat_fix_sub_topic="nav_sat_fix" />
+  <xacro:ros_interface_plugin_macro namespace="${namespace}" imu_sub_topic="imu" magnetic_field_sub_topic="magnetic_field" nav_sat_fix_sub_topic="nav_sat_fix" />
   <xacro:if value="$(arg enable_mavlink_interface)">
     <!-- Instantiate mavlink telemetry interface. -->
@@ -42,4 +42,4 @@
   </xacro:if>
   <!-- Create a interface to send/receive messages to the outside world -->
-  <xacro:msg_interface_plugin />
+  <!--<xacro:msg_interface_plugin />-->
 </robot>

Commit message: ROS interface plugin publishing actuators and link state messages to ROS platform

File: rotors_description/urdf/component_snippets.xacro (robot description, xacro)
@@ -249,5 +249,5 @@
   <!-- ==================== ROS INTERFACE MACRO ====================== -->
   <!-- =============================================================== -->
-  <xacro:macro name="ros_interface_plugin_macro" params="namespace imu_sub_topic magnetic_field_sub_topic nav_sat_fix_sub_topic">
+  <xacro:macro name="ros_interface_plugin_macro" params="namespace actuators_sub_topic imu_sub_topic joint_state_sub_topic magnetic_field_sub_topic nav_sat_fix_sub_topic">
     <gazebo>
       <plugin name="ros_interface_plugin" filename="librotors_gazebo_ros_interface_plugin.so">
@@ -256,5 +256,7 @@
         <commandRateThrustSubTopic>command/rate</commandRateThrustSubTopic>
         <commandMotorSpeedSubTopic>command/motor_speed</commandMotorSpeedSubTopic>
+        <actuatorsSubTopic>${actuators_sub_topic}</actuatorsSubTopic>
         <imuSubTopic>${imu_sub_topic}</imuSubTopic>
+        <jointStateSubTopic>${joint_state_sub_topic}</jointStateSubTopic>
         <magneticFieldSubTopic>${magnetic_field_sub_topic}</magneticFieldSubTopic>
         <navSatFixSubTopic>${nav_sat_fix_sub_topic}</navSatFixSubTopic>

File: rotors_description/urdf/firefly_base.xacro (robot description, xacro)
@@ -23,5 +23,11 @@
   <xacro:controller_plugin_macro namespace="${namespace}" imu_sub_topic="imu" />
   <!-- Instantiate a ROS message interface -->
-  <xacro:ros_interface_plugin_macro namespace="${namespace}" imu_sub_topic="imu" magnetic_field_sub_topic="magnetic_field" nav_sat_fix_sub_topic="nav_sat_fix" />
+  <xacro:ros_interface_plugin_macro
+  		namespace="${namespace}"
+  		actuators_sub_topic="actuators"
+  		imu_sub_topic="imu"
+  		joint_state_sub_topic="joint_state"
+  		magnetic_field_sub_topic="magnetic_field"
+  		nav_sat_fix_sub_topic="nav_sat_fix" />
   <xacro:if value="$(arg enable_mavlink_interface)">
     <!-- Instantiate mavlink telemetry interface. -->

Commit message: Odometry message now being captured by ROS interface plugin and published to ROS framework. Hovering example now works again.

File: rotors_description/urdf/component_snippets.xacro (robot description, xacro)
@@ -249,5 +249,7 @@
   <!-- ==================== ROS INTERFACE MACRO ====================== -->
   <!-- =============================================================== -->
-  <xacro:macro name="ros_interface_plugin_macro" params="namespace actuators_sub_topic imu_sub_topic joint_state_sub_topic magnetic_field_sub_topic nav_sat_fix_sub_topic">
+  <xacro:macro
+  		name="ros_interface_plugin_macro"
+  		params="namespace actuators_sub_topic imu_sub_topic joint_state_sub_topic magnetic_field_sub_topic nav_sat_fix_sub_topic odometry_sub_topic">
     <gazebo>
       <plugin name="ros_interface_plugin" filename="librotors_gazebo_ros_interface_plugin.so">
@@ -261,4 +263,5 @@
         <magneticFieldSubTopic>${magnetic_field_sub_topic}</magneticFieldSubTopic>
         <navSatFixSubTopic>${nav_sat_fix_sub_topic}</navSatFixSubTopic>
+        <odometrySubTopic>${odometry_sub_topic}</odometrySubTopic>
         <motorSpeedCommandPubTopic>gazebo/command/motor_speed</motorSpeedCommandPubTopic>
       </plugin>

File: rotors_description/urdf/firefly_base.xacro (robot description, xacro)
@@ -29,5 +29,6 @@
   		joint_state_sub_topic="joint_state"
   		magnetic_field_sub_topic="magnetic_field"
-  		nav_sat_fix_sub_topic="nav_sat_fix" />
+  		nav_sat_fix_sub_topic="nav_sat_fix"
+  		odometry_sub_topic="odometry_sensor1/odometry" />
   <xacro:if value="$(arg enable_mavlink_interface)">
     <!-- Instantiate mavlink telemetry interface. -->

Commit message: The ROS interface plugin is now attached to a static model in the world rather than being attahed to the firefly MAV.

File: rotors_description/urdf/component_snippets.xacro (robot description, xacro)
@@ -249,5 +249,5 @@
   <!-- ==================== ROS INTERFACE MACRO ====================== -->
   <!-- =============================================================== -->
-  <xacro:macro
+  <!-- <xacro:macro
   		name="ros_interface_plugin_macro"
   		params="namespace">
@@ -257,6 +257,8 @@
       </plugin>
     </gazebo>
-  </xacro:macro>
-  <!-- Macro to add the mavlink interface. -->
+  </xacro:macro>-->
+  <!-- =============================================================== -->
+  <!-- ================== MAVLINK INTERFACE MACRO ==================== -->
+  <!-- =============================================================== -->
   <xacro:macro name="mavlink_interface_macro"
     params="namespace mavlink_sub_topic imu_sub_topic mavlink_pub_topic

File: rotors_description/urdf/firefly_base.xacro (robot description, xacro)
@@ -23,5 +23,5 @@
   <xacro:controller_plugin_macro namespace="${namespace}" imu_sub_topic="imu" />
   <!-- Instantiate a ROS message interface -->
-  <xacro:ros_interface_plugin_macro namespace="${namespace}" />
+  <!-- <xacro:ros_interface_plugin_macro namespace="${namespace}" />-->
   <xacro:if value="$(arg enable_mavlink_interface)">
     <!-- Instantiate mavlink telemetry interface. -->

Commit message: Lidar Model developed by new .xacro file

File: rotors_description/urdf/component_snippets.xacro (robot description, xacro)
@@ -114,5 +114,5 @@
        camera. -->
   <xacro:macro name="camera_joint_macro"
-    params="namespace parent_link camera_suffix enable_visual *origin *geometry" >
+    params="namespace parent_link camera_suffix enable_visual *origin **geometry" >
     <link name="${namespace}/camera_${camera_suffix}_link">
       <collision>

File: rotors_description/urdf/firefly_base.xacro (robot description, xacro)
@@ -19,4 +19,5 @@
   xmlns:xacro="http://ros.org/wiki/xacro">
   <xacro:include filename="$(find rotors_description)/urdf/component_snippets.xacro" />
+  <xacro:include filename="$(find rotors_description)/urdf/nearthlab_lidar_sensor.xacro" />
   <!-- Instantiate firefly "mechanics" -->
   <xacro:include filename="$(find rotors_description)/urdf/firefly.xacro" />
@@ -35,22 +36,24 @@
   <xacro:default_magnetometer namespace="${namespace}" parent_link="${namespace}/base_link" />
   <xacro:default_pressure_sensor namespace="${namespace}" parent_link="${namespace}/base_link" />
-  <xacro:camera_macro
-    namespace="${namespace}"
-    parent_link="${namespace}/base_link"
-    camera_suffix="${namespace}/camera_suffix"
-    frame_rate="${namespace}/frame_rate"
-    horizontal_fov="1.3962634"
-    image_width="752"
-    image_height="480"
-    image_format="L8"
-    min_distance="0.02"
-    max_distance="30"
-    noise_mean="0.0"
-    noise_stddev="0.007"
-    enable_visual="true">
+  <xacro:camera_macro namespace="${namespace}" parent_link="${namespace}/base_link" camera_suffix="${namespace}/camera_suffix" frame_rate="${namespace}/frame_rate" horizontal_fov="1.3962634" image_width="752" image_height="480" image_format="L8" min_distance="0.02" max_distance="30" noise_mean="0.0" noise_stddev="0.007" enable_visual="true">
+  <!-- <xacro:camera_macro namespace="${namespace}" parent_link="${namespace}/base_link" camera_suffix="camera_suffix" frame_rate="${namespace}/frame_rate" horizontal_fov="1.3962634" image_width="752" image_height="480" image_format="L8" min_distance="0.02" max_distance="30" noise_mean="0.0" noise_stddev="0.007" enable_visual="true"> -->
     <mesh filename="package://rotors_description/meshes/vi_camera.dae" scale="1 1 1" />
     <!-- <xacro:insert_block name="origin" /> -->
-    <origin xyz="0 0 -0.05" rpy="0 0 0" />
+    <origin xyz="0 0 -0.04" rpy="0 0 0" />
   </xacro:camera_macro>
+  <xacro:camera_joint_macro namespace="${namespace}" parent_link="${namespace}/base_link" camera_suffix="${namespace}/camera_joint" enable_visual="true">
+  <!-- <xacro:camera_joint_macro namespace="${namespace}" parent_link="${namespace}/base_link" camera_suffix="${namespace}/camear_joint_suffix" enable_visual="true"> -->
+    <origin xyz="0 0 -0.015" rpy="0 0 0" />
+    <geometry>
+      <cylinder length="0.02" radius="0.006" />
+    </geometry>
+  </xacro:camera_joint_macro>
+  <!--LIDAR Sensor Added by bkjung-->
+  <xacro:lidar_macro namespace="${namespace}" parent_link="${namespace}/base_link">
+    <origin xyz="0 0 -0.07" rpy="0 0 0" />
+    <geometry>
+      <cylinder length="0.02" radius="0.015" />
+    </geometry>
+  </xacro:lidar_macro>
   <xacro:if value="$(arg enable_ground_truth)">
     <xacro:ground_truth_imu_and_odometry namespace="${namespace}" parent_link="${namespace}/base_link" />

Commit message: lidar & camera postion/heading revised

File: rotors_description/urdf/component_snippets.xacro (robot description, xacro)
@@ -46,5 +46,6 @@
       <xacro:if value="${enable_visual}">
         <visual>
-          <origin xyz="0 0 0" rpy="0 ${pi/2} 0" />
+          <!-- <origin xyz="0 0 0" rpy="0 ${pi/2} 0" /> -->
+          <origin xyz="0 0 0" rpy="0 ${pi} 0" />
           <geometry>
             <xacro:insert_block name="geometry" />

File: rotors_description/urdf/firefly_base.xacro (robot description, xacro)
@@ -36,12 +36,9 @@
   <xacro:default_magnetometer namespace="${namespace}" parent_link="${namespace}/base_link" />
   <xacro:default_pressure_sensor namespace="${namespace}" parent_link="${namespace}/base_link" />
-  <xacro:camera_macro namespace="${namespace}" parent_link="${namespace}/base_link" camera_suffix="${namespace}/camera_suffix" frame_rate="${namespace}/frame_rate" horizontal_fov="1.3962634" image_width="752" image_height="480" image_format="L8" min_distance="0.02" max_distance="30" noise_mean="0.0" noise_stddev="0.007" enable_visual="true">
-  <!-- <xacro:camera_macro namespace="${namespace}" parent_link="${namespace}/base_link" camera_suffix="camera_suffix" frame_rate="${namespace}/frame_rate" horizontal_fov="1.3962634" image_width="752" image_height="480" image_format="L8" min_distance="0.02" max_distance="30" noise_mean="0.0" noise_stddev="0.007" enable_visual="true"> -->
+  <!-- <xacro:camera_macro namespace="${namespace}" parent_link="${namespace}/base_link" camera_suffix="${namespace}/camera_suffix" frame_rate="${namespace}/frame_rate" horizontal_fov="1.3962634" image_width="752" image_height="480" image_format="L8" min_distance="0.02" max_distance="30" noise_mean="0.0" noise_stddev="0.007" enable_visual="true">
     <mesh filename="package://rotors_description/meshes/vi_camera.dae" scale="1 1 1" />
-    <!-- <xacro:insert_block name="origin" /> -->
-    <origin xyz="0 0 -0.04" rpy="0 0 0" />
-  </xacro:camera_macro>
+    <origin xyz="0 0 -0.035" rpy="0 0 0" />
+  </xacro:camera_macro> -->
   <xacro:camera_joint_macro namespace="${namespace}" parent_link="${namespace}/base_link" camera_suffix="${namespace}/camera_joint" enable_visual="true">
-  <!-- <xacro:camera_joint_macro namespace="${namespace}" parent_link="${namespace}/base_link" camera_suffix="${namespace}/camear_joint_suffix" enable_visual="true"> -->
     <origin xyz="0 0 -0.015" rpy="0 0 0" />
     <geometry>
@@ -51,5 +48,6 @@
   <!--LIDAR Sensor Added by bkjung-->
   <xacro:lidar_macro namespace="${namespace}" parent_link="${namespace}/base_link">
-    <origin xyz="0 0 -0.07" rpy="0 0 0" />
+    <!-- <origin xyz="0 0 -0.07" rpy="0 0 0" /> -->
+    <origin xyz="0 0 -0.035" rpy="0 0 0" />
     <geometry>
       <cylinder length="0.02" radius="0.015" />
