Commit message: developing lidar

File: rotors_description/urdf/component_snippets.xacro (robot description, xacro)
@@ -47,5 +47,6 @@
         <visual>
           <!-- <origin xyz="0 0 0" rpy="0 ${pi/2} 0" /> -->
-          <origin xyz="0 0 0" rpy="0 ${pi} 0" />
+          <!-- <origin xyz="0 0 0" rpy="0 ${pi} 0" /> -->
+          <origin xyz="0.01 0 0" rpy="0 ${pi/2} 0" />
           <geometry>
             <xacro:insert_block name="geometry" />

File: rotors_description/urdf/firefly_base.xacro (robot description, xacro)
@@ -37,8 +37,4 @@
   <xacro:default_magnetometer namespace="${namespace}" parent_link="${namespace}/base_link" />
   <xacro:default_pressure_sensor namespace="${namespace}" parent_link="${namespace}/base_link" />
-  <!-- <xacro:camera_macro namespace="${namespace}" parent_link="${namespace}/base_link" camera_suffix="${namespace}/camera_suffix" frame_rate="${namespace}/frame_rate" horizontal_fov="1.3962634" image_width="752" image_height="480" image_format="L8" min_distance="0.02" max_distance="30" noise_mean="0.0" noise_stddev="0.007" enable_visual="true">
-    <mesh filename="package://rotors_description/meshes/vi_camera.dae" scale="1 1 1" />
-    <origin xyz="0 0 -0.035" rpy="0 0 0" />
-  </xacro:camera_macro> -->
   <xacro:camera_joint_macro namespace="${namespace}" parent_link="${namespace}/base_link" camera_suffix="${namespace}/camera_joint" enable_visual="true">
     <origin xyz="0 0 -0.015" rpy="0 0 0" />
@@ -47,11 +43,9 @@
     </geometry>
   </xacro:camera_joint_macro>
-  <!--LIDAR Sensor Added by bkjung-->
-  <!-- <xacro:lidar_macro namespace="${namespace}" parent_link="${namespace}/base_link">
+  <!-- Camera Sensor-->
+  <xacro:camera_macro namespace="${namespace}" parent_link="${namespace}/base_link" camera_suffix="${namespace}/camera_suffix" frame_rate="${namespace}/frame_rate" horizontal_fov="1.3962634" image_width="752" image_height="480" image_format="L8" min_distance="0.02" max_distance="30" noise_mean="0.0" noise_stddev="0.007" enable_visual="true">
+    <mesh filename="package://rotors_description/meshes/vi_camera.dae" scale="1 1 1" />
     <origin xyz="0 0 -0.035" rpy="0 0 0" />
-    <geometry>
-      <cylinder length="0.02" radius="0.015" />
-    </geometry>
-  </xacro:lidar_macro> -->
+  </xacro:camera_macro>
   <xacro:if value="$(arg enable_ground_truth)">
     <xacro:ground_truth_imu_and_odometry namespace="${namespace}" parent_link="${namespace}/base_link" />
@@ -61,9 +55,17 @@
     <xacro:bag_plugin_macro namespace="${namespace}" bag_file="$(arg log_file)" rotor_velocity_slowdown_sim="${rotor_velocity_slowdown_sim}" wait_to_record_bag="$(arg wait_to_record_bag)" />
   </xacro:if>
-  <xacro:payload_macro namespace="${namespace}" parent_link="${namespace}/base_link" >
-    <origin xyz="0 0 -0.07" rpy="0 0 0" />
-      <geometry>
-        <mesh filename="package://rotors_description/meshes/nearthlab_payload.dae" scale="0.0005 0.0005 0.0005" />
-      </geometry>
-  </xacro:payload_macro>
+  <!--LIDAR Sensor-->
+  <xacro:lidar_macro namespace="${namespace}" parent_link="${namespace}/base_link">
+    <origin xyz="0 0 -0.035" rpy="0 0 0" />
+    <geometry>
+      <cylinder length="0.02" radius="0.015" />
+    </geometry>
+  </xacro:lidar_macro>
+  <!-- Nearthlab Payload -->
+  <!-- <xacro:payload_macro namespace="${namespace}" parent_link="${namespace}/base_link" > -->
+    <!-- <origin xyz="0 0 -0.06" rpy="0 0 0" /> -->
+      <!-- <geometry> -->
+        <!-- <mesh filename="package://rotors_description/meshes/nearthlab_payload.dae" scale="0.0004 0.0004 0.0004" /> -->
+      <!-- </geometry> -->
+  <!-- </xacro:payload_macro> -->
 </robot>

File: rotors_description/urdf/nearthlab_lidar_sensor.xacro (robot description, xacro)
@@ -24,8 +24,11 @@
       <child link="${namespace}/lidar_link" />
     </joint>
-    <gazebo>
+    <gazebo reference="${namespace}/lidar_link">
       <!-- <sensor name="laser" type="ray"> -->
       <sensor type="ray" name="${namespace}_lidar">
         <pose>0 0 0 0 -1.570896 0</pose>
+        <always_on>1</always_on>
+        <update_rate>20</update_rate>
+        <visualize>true</visualize>
         <ray>
           <scan>
@@ -48,9 +51,9 @@
           </noise>
         </ray>
-        <plugin name="LaserPlugin" filename="librotors_gazebo_lidar_plugin.so"/>
-        <robotNamespace></robotNamespace>
-        <always_on>1</always_on>
-        <update_rate>20</update_rate>
-        <visualize>true</visualize>
+        <plugin filename="librotors_gazebo_lidar_plugin.so" name="rotors_gazebo_lidar_plugin">
+          <robotNamespace>${namespace}</robotNamespace>
+          <linkName>${namespace}/lidar_link</linkName>
+          <lidarTopic>lidar</lidarTopic>
+        </plugin>
       </sensor>
     </gazebo>

File: rotors_description/urdf/nearthlab_payload.xacro (robot description, xacro)
@@ -10,5 +10,5 @@
       </inertial>
       <visual>
-        <origin xyz="0 0 0" rpy="0 ${pi/2} ${pi/2}" />
+        <origin xyz="0 0 0" rpy="${pi/2} ${pi/2} ${pi/2}" />
         <geometry>
           <xacro:insert_block name="geometry" />

Commit message: Crazyflie IMU and the complementary filter have been added
The Crazyflie IMU (MPU-9250) and the default state estimator (the complementary filter) have been added in the loop

File: rotors_description/urdf/component_snippets.xacro (robot description, xacro)
@@ -6,4 +6,6 @@
   Copyright 2015 Janosch Nikolic, ASL, ETH Zurich, Switzerland
   Copyright 2015 Markus Achtelik, ASL, ETH Zurich, Switzerland
+  Copyright 2018 Giuseppe Silano, University of Sannio in Benevento, Italy
+  Copyright 2018 Luigi Iannelli, University of Sannio in Benevento, Italy
   Licensed under the Apache License, Version 2.0 (the "License");
   you may not use this file except in compliance with the License.
@@ -831,4 +833,24 @@
     </xacro:imu_plugin_macro>
   </xacro:macro>
+  <xacro:macro name="crazyflie2_imu" params="namespace parent_link">
+    <!-- Mount an MPU-9250 IMU. -->
+    <xacro:imu_plugin_macro
+      namespace="${namespace}"
+      imu_suffix=""
+      parent_link="${parent_link}"
+      imu_topic="imu"
+      mass_imu_sensor="0.00001"
+      gyroscope_noise_density="0.000175"
+      gyroscope_random_walk="0.0105"
+      gyroscope_bias_correlation_time="1000.0"
+      gyroscope_turn_on_bias_sigma= "0.09"
+      accelerometer_noise_density="0.003"
+      accelerometer_random_walk="0.18"
+      accelerometer_bias_correlation_time="300.0"
+      accelerometer_turn_on_bias_sigma="0.588">
+      <inertia ixx="0.00001" ixy="0.0" ixz="0.0" iyy="0.00001" iyz="0.0" izz="0.00001" />
+      <origin xyz="0 0 0" rpy="0 0 0" />
+    </xacro:imu_plugin_macro>
+  </xacro:macro>
   <xacro:macro name="default_gps" params="namespace parent_link">
     <!-- Default GPS. -->

File: rotors_description/urdf/crazyflie2_base.xacro (robot description, xacro)
@@ -25,22 +25,6 @@
     <xacro:default_mavlink_interface namespace="${namespace}" imu_sub_topic="imu" rotor_count="4" />
   </xacro:if>
-  <!-- Mount an MPU-9250 IMU.
-  <xacro:imu_plugin_macro
-      namespace="${namespace}"
-      imu_suffix=""
-      parent_link="${namespace}/base_link"
-      imu_topic="imu"
-      mass_imu_sensor="0.00001"
-      gyroscope_noise_density=""
-      gyroscope_random_walk=""
-      gyroscope_bias_correlation_time=""
-      gyroscope_turn_on_bias_sigma=""
-      accelerometer_noise_density=""
-      accelerometer_random_walk=""
-      accelerometer_bias_correlation_time=""
-      accelerometer_turn_on_bias_sigma="">
-      <inertia ixx="0.00001" ixy="0.0" ixz="0.0" iyy="0.00001" iyz="0.0" izz="0.00001" />
-      <origin xyz="0 0 0" rpy="0 0 0" />
-    </xacro:imu_plugin_macro> -->
+  <!-- Mount an MPU-9250 IMU. -->
+  <xacro:crazyflie2_imu namespace="${namespace}" parent_link="${namespace}/base_link" />
   <xacro:if value="$(arg enable_ground_truth)">
     <xacro:ground_truth_imu_and_odometry namespace="${namespace}" parent_link="${namespace}/base_link" />

Commit message: Air resistance simulation codes are added

File: rotors_description/urdf/component_snippets.xacro (robot description, xacro)
@@ -897,3 +897,87 @@
     </xacro:mavlink_interface_macro>
   </xacro:macro>
+<xacro:macro name="niv1_imu" params="namespace parent_link">
+    <!-- ADIS16448 IMU. -->
+    <xacro:imu_plugin_macro
+      namespace="${namespace}"
+      imu_suffix=""
+      parent_link="${parent_link}"
+      imu_topic="imu"
+      mass_imu_sensor="0.015"
+      gyroscope_noise_density="0.0003394"
+      gyroscope_random_walk="0.000038785"
+      gyroscope_bias_correlation_time="1000.0"
+      gyroscope_turn_on_bias_sigma="0.0"
+      accelerometer_noise_density="0.0004"
+      accelerometer_random_walk="0.0006"
+      accelerometer_bias_correlation_time="300.0"
+      accelerometer_turn_on_bias_sigma="0.0">
+      <inertia ixx="0.00001" ixy="0.0" ixz="0.0" iyy="0.00001" iyz="0.0" izz="0.00001" />
+      <origin xyz="0 0 0.05" rpy="0 0 0" />
+    </xacro:imu_plugin_macro>
+  </xacro:macro>
+  <xacro:macro name="niv1_gps" params="namespace parent_link">
+    <!-- Default GPS. -->
+    <xacro:gps_plugin_macro
+      namespace="${namespace}"
+      gps_suffix=""
+      parent_link="${parent_link}"
+      gps_topic="gps"
+      ground_speed_topic="ground_speed"
+      mass_gps_sensor="0.015"
+      horizontal_pos_std_dev="3.0"
+      vertical_pos_std_dev="6.0"
+      horizontal_vel_std_dev="0.1"
+      vertical_vel_std_dev="0.1">
+      <inertia ixx="0.00001" ixy="0.0" ixz="0.0" iyy="0.00001" iyz="0.0" izz="0.00001" />
+      <origin xyz="0 0 0" rpy="0 0 0" />
+    </xacro:gps_plugin_macro>
+  </xacro:macro>
+  <xacro:macro name="niv1_magnetometer" params="namespace parent_link">
+    <!-- ADIS16448 Magnetometer. -->
+    <xacro:magnetometer_plugin_macro
+      namespace="${namespace}"
+      magnetometer_suffix=""
+      parent_link="${parent_link}"
+      magnetometer_topic="magnetic_field"
+      mass_magnetometer_sensor="0.015"
+      ref_mag_north="0.000021493"
+      ref_mag_east="0.000000815"
+      ref_mag_down="0.000042795"
+      noise_normal="0.000000080 0.000000080 0.000000080"
+      noise_uniform_initial_bias="0.000000400 0.000000400 0.000000400">
+      <inertia ixx="0.00001" ixy="0.0" ixz="0.0" iyy="0.00001" iyz="0.0" izz="0.00001" />
+      <origin xyz="0 0 0" rpy="0 0 0" />
+    </xacro:magnetometer_plugin_macro>
+  </xacro:macro>
+  <xacro:macro name="niv1_pressure_sensor" params="namespace parent_link">
+    <xacro:pressure_sensor_plugin_macro
+      namespace="${namespace}"
+      pressure_sensor_suffix=""
+      parent_link="${parent_link}"
+      pressure_topic="air_pressure"
+      mass_pressure_sensor="0.015"
+      reference_altitude="500.0"
+      pressure_variance="0.0">
+      <inertia ixx="0.00001" ixy="0.0" ixz="0.0" iyy="0.00001" iyz="0.0" izz="0.00001" />
+      <origin xyz="0 0 0" rpy="0 0 0" />
+    </xacro:pressure_sensor_plugin_macro>
+  </xacro:macro>
+  <xacro:macro name="default_mavlink_interface" params="namespace imu_sub_topic rotor_count">
+    <xacro:mavlink_interface_macro
+      namespace="${namespace}"
+      mavlink_sub_topic="/mavlink/from"
+      imu_sub_topic="${imu_sub_topic}"
+      mavlink_pub_topic="/mavlink/to"
+      motors_speeds_pub_topic="gazebo/command/motor_speed"
+      gps_update_freq="5.0"
+      rotor_count="${rotor_count}"
+      reference_magnetic_field_north="0.21475"
+      reference_magnetic_field_east="0.00797"
+      reference_magnetic_field_down="0.42817"
+      reference_latitude="47.3667"
+      reference_longitude="8.5500"
+      reference_altitude="500.0">
+    </xacro:mavlink_interface_macro>
+  </xacro:macro>
 </robot>

File: rotors_description/urdf/multirotor_base.xacro (robot description, xacro)
@@ -70,4 +70,6 @@
         <linkName>${robot_namespace}/base_link</linkName>
         <rotorVelocitySlowdownSim>${rotor_velocity_slowdown_sim}</rotorVelocitySlowdownSim>
+        <angularAirResistance>${angular_air_resistance}</angularAirResistance>
+        <linearAirResistance>${linear_air_resistance}</linearAirResistance>
       </plugin>
     </gazebo>
@@ -132,3 +134,31 @@
     </gazebo>
   </xacro:macro>
+  <xacro:macro name="support"
+    params="robot_namespace suffix parent support_number color *origin *inertia">
+    <joint name="${robot_namespace}/support_${support_number}_joint" type="continuous">
+      <xacro:insert_block name="origin" />
+      <axis xyz="0 0 1" />
+      <parent link="${parent}" />
+      <child link="${robot_namespace}/support_${support_number}" />
+    </joint>
+    <link name="${robot_namespace}/support_${support_number}">
+      <inertial>
+        <mass value="0.001" /> <!-- [kg] -->
+        <xacro:insert_block name="inertia" />
+      </inertial>
+      <visual>
+        <geometry>
+          <cylinder length="0.2" radius="0.01"/> --> <!-- [m] -->
+        </geometry>
+      </visual>
+      <collision>
+        <geometry>
+          <cylinder length="0.2" radius="0.01" /> <!-- [m] -->
+        </geometry>
+      </collision>
+    </link>
+    <gazebo reference="${robot_namespace}/support_${support_number}">
+      <material>Gazebo/${color}</material>
+    </gazebo>
+  </xacro:macro>
 </robot>

File: rotors_description/urdf/niv1.xacro (robot description, xacro)
@@ -23,6 +23,6 @@
   <xacro:property name="mesh_file" value="package://rotors_description/meshes/niv1_body.dae" />
   <xacro:property name="mass" value="12" /> <!-- [kg] -->
-  <xacro:property name="body_width" value="0.2" /> <!-- [m] -->
-  <xacro:property name="body_height" value="0.2" /> <!-- [m] -->
+  <xacro:property name="body_width" value="0.05" /> <!-- [m] -->
+  <xacro:property name="body_height" value="0.05" /> <!-- [m] -->
   <xacro:property name="mass_rotor" value="0.2" /> <!-- [kg] -->
   <xacro:property name="arm_length" value="0.636" /> <!-- [m] -->
@@ -30,6 +30,5 @@
   <xacro:property name="radius_rotor" value="0.3" /> <!-- [m] -->
   <xacro:property name="motor_constant_for_ros_sim" value="8.54858e-05" /> <!-- [kg m/s^2]  force = real_motor_velocity * real_motor_velocity * motor_constant_-->
-  <xacro:property name="motor_constant_bak" value="0.9e-04" /> <!-- [kg m/s^2]  force = real_motor_velocity * real_motor_velocity * motor_constant_-->
-  <xacro:property name="motor_constant" value="8.9e-05" /> <!-- [kg m/s^2]  force = real_motor_velocity * real_motor_velocity * motor_constant_-->
+  <xacro:property name="motor_constant" value="1.2e-04" /> <!-- [kg m/s^2]  force = real_motor_velocity * real_motor_velocity * motor_constant_-->
   <xacro:property name="moment_constant" value="0.025" /> <!-- [m] math::Vector3 drag_torque(0, 0, -turning_direction_ * force * moment_constant_); -->
   <xacro:property name="moment_constan_org" value="0.025" /> <!-- [m] math::Vector3 drag_torque(0, 0, -turning_direction_ * force * moment_constant_); -->
@@ -43,10 +42,11 @@
   <xacro:property name="rotor_drag_coefficient" value="8.06428e-05" /> <!-- math::Vector3 air_drag = -std::abs(real_motor_velocity) * rotor_drag_coefficient_ * body_velocity_perpendicular; -->
   <xacro:property name="rolling_moment_coefficient" value="0.000001" /> <!-- math::Vector3 rolling_moment = -std::abs(real_motor_velocity) * rolling_moment_coefficient_ * body_velocity_perpendicular; -->
+  <xacro:property name="angular_air_resistance" value="0.01" />
+  <xacro:property name="linear_air_resistance" value="0.001" />
   <!-- Property Blocks -->
   <xacro:property name="body_inertia">
     <!--
     <inertia ixx="0.0347563" ixy="0.0" ixz="0.0" iyy="0.0458929" iyz="0.0" izz="0.0977" /> [kg m^2] [kg m^2] [kg m^2] [kg m^2] [kg m^2] [kg m^2] -->
-    <!-- <inertia ixx="0.801" ixy="0.0" ixz="0.0" iyy="0.827" iyz="0.0" izz="1.450" /> -->
-    <inertia ixx="1.5" ixy="0.0" ixz="0.0" iyy="1.5" iyz="0.0" izz="10.0" />
+    <inertia ixx="0.801" ixy="0.0" ixz="0.0" iyy="0.827" iyz="0.0" izz="1.450" />
   </xacro:property>
   <!-- inertia of a single rotor, assuming it is a cuboid. -->
@@ -54,4 +54,8 @@
     <!-- <xacro:box_inertia x="${radius_rotor}" y="0.015" z="0.003" mass="${mass_rotor*rotor_velocity_slowdown_sim}" /> -->
     <xacro:box_inertia x="${radius_rotor}" y="0.015" z="0.003" mass="${mass_rotor*rotor_velocity_slowdown_sim}" />
+  </xacro:property>
+  <xacro:property name="support_inertia">
+    <!-- <xacro:box_inertia x="${radius_rotor}" y="0.015" z="0.003" mass="${mass_rotor*rotor_velocity_slowdown_sim}" /> -->
+    <xacro:box_inertia x="0.03" y="0.03" z="0.2" mass="0.001" />
   </xacro:property>
   <!-- Included URDF Files -->
@@ -151,3 +155,38 @@
     <xacro:insert_block name="rotor_inertia" />
   </xacro:vertical_rotor>
+ <!-- Instantiate support -->
+    <xacro:support
+    robot_namespace="${namespace}"
+    suffix="front_right"
+    parent="${namespace}/base_link"
+    support_number="0"
+    color="Grey">
+     <origin xyz="${rotor_pos_x} -${rotor_pos_y} ${rotor_offset_top-0.2}" rpy="0 0 0" />
+    <xacro:insert_block name="rotor_inertia" />
+  </xacro:support>
+  <xacro:support
+    robot_namespace="${namespace}"
+    suffix="front_left"
+    parent="${namespace}/base_link"
+    support_number="1"
+    color="Grey">
+    <origin xyz="${rotor_pos_x} ${rotor_pos_y} ${rotor_offset_top-0.2}" rpy="0 0 0" />
+    <xacro:insert_block name="rotor_inertia" />
+  </xacro:support>
+  <xacro:support robot_namespace="${namespace}"
+    suffix="back_left"
+    parent="${namespace}/base_link"
+    support_number="2"
+    color="Grey">
+    <origin xyz="-${rotor_pos_x} ${rotor_pos_y} ${rotor_offset_top-0.2}" rpy="0 0 0" />
+    <xacro:insert_block name="support_inertia" />
+  </xacro:support>
+  <xacro:support robot_namespace="${namespace}"
+    suffix="back_right"
+    parent="${namespace}/base_link"
+    support_number="3"
+    color="Grey">
+    <origin xyz="-${rotor_pos_x} -${rotor_pos_y} ${rotor_offset_top-0.2}" rpy="0 0 0" />
+    <xacro:insert_block name="support_inertia" />
+  </xacro:support>
 </robot>

File: rotors_description/urdf/niv1_base.xacro (robot description, xacro)
@@ -30,12 +30,12 @@
   <xacro:if value="$(arg enable_mavlink_interface)">
     <!-- Instantiate mavlink telemetry interface. -->
-    <xacro:default_mavlink_interface namespace="${namespace}" imu_sub_topic="imu" rotor_count="6" />
+    <xacro:niv1_mavlink_interface namespace="${namespace}" imu_sub_topic="imu" rotor_count="6" />
   </xacro:if>
   <!-- Mount an ADIS16448 IMU. -->
-  <xacro:default_imu namespace="${namespace}" parent_link="${namespace}/base_link" />
+  <xacro:niv1_imu namespace="${namespace}" parent_link="${namespace}/base_link" />
   <!-- Added by bkjung -->
-  <xacro:default_gps namespace="${namespace}" parent_link="${namespace}/base_link" />
-  <xacro:default_magnetometer namespace="${namespace}" parent_link="${namespace}/base_link" />
-  <xacro:default_pressure_sensor namespace="${namespace}" parent_link="${namespace}/base_link" />
+  <xacro:niv1_gps namespace="${namespace}" parent_link="${namespace}/base_link" />
+  <xacro:niv1_magnetometer namespace="${namespace}" parent_link="${namespace}/base_link" />
+  <xacro:niv1_pressure_sensor namespace="${namespace}" parent_link="${namespace}/base_link" />
   <xacro:camera_joint_macro namespace="${namespace}" parent_link="${namespace}/base_link" camera_suffix="${namespace}/camera_joint" enable_visual="true">
     <origin xyz="0 0 -0.015" rpy="0 0 0" />

File: rotors_description/urdf/niv1_sim.xacro (robot description, xacro)
@@ -45,6 +45,6 @@
     <!--
     <inertia ixx="0.0347563" ixy="0.0" ixz="0.0" iyy="0.0458929" iyz="0.0" izz="0.0977" /> [kg m^2] [kg m^2] [kg m^2] [kg m^2] [kg m^2] [kg m^2] -->
-    <!-- <inertia ixx="0.801" ixy="0.0" ixz="0.0" iyy="0.827" iyz="0.0" izz="1.450" /> -->
-    <inertia ixx="1.5" ixy="0.0" ixz="0.0" iyy="1.5" iyz="0.0" izz="10.0" />
+    <inertia ixx="0.801" ixy="0.0" ixz="0.0" iyy="0.827" iyz="0.0" izz="1.450" />
+    <!--<inertia ixx="1.5" ixy="0.0" ixz="0.0" iyy="1.5" iyz="0.0" izz="10.0" /> -->
   </xacro:property>
   <!-- inertia of a single rotor, assuming it is a cuboid. -->

File: rotors_description/urdf/niv1_sim_base.xacro (robot description, xacro)
@@ -30,12 +30,12 @@
   <xacro:if value="$(arg enable_mavlink_interface)">
     <!-- Instantiate mavlink telemetry interface. -->
-    <xacro:default_mavlink_interface namespace="${namespace}" imu_sub_topic="imu" rotor_count="6" />
+    <xacro:niv1_mavlink_interface namespace="${namespace}" imu_sub_topic="imu" rotor_count="6" />
   </xacro:if>
   <!-- Mount an ADIS16448 IMU. -->
-  <xacro:default_imu namespace="${namespace}" parent_link="${namespace}/base_link" />
+  <xacro:niv1_imu namespace="${namespace}" parent_link="${namespace}/base_link" />
   <!-- Added by bkjung -->
-  <xacro:default_gps namespace="${namespace}" parent_link="${namespace}/base_link" />
-  <xacro:default_magnetometer namespace="${namespace}" parent_link="${namespace}/base_link" />
-  <xacro:default_pressure_sensor namespace="${namespace}" parent_link="${namespace}/base_link" />
+  <xacro:niv1_gps namespace="${namespace}" parent_link="${namespace}/base_link" />
+  <xacro:niv1_magnetometer namespace="${namespace}" parent_link="${namespace}/base_link" />
+  <xacro:niv1_pressure_sensor namespace="${namespace}" parent_link="${namespace}/base_link" />
   <xacro:camera_joint_macro namespace="${namespace}" parent_link="${namespace}/base_link" camera_suffix="${namespace}/camera_joint" enable_visual="true">
     <origin xyz="0 0 -0.015" rpy="0 0 0" />
