Commit message: working backup

File: rotors_description/urdf/component_snippets.xacro (robot description, xacro)
@@ -926,8 +926,8 @@
       ground_speed_topic="ground_speed"
       mass_gps_sensor="0.015"
-      horizontal_pos_std_dev="3.0"
-      vertical_pos_std_dev="6.0"
-      horizontal_vel_std_dev="0.1"
-      vertical_vel_std_dev="0.1">
+      horizontal_pos_std_dev="0.0"
+      vertical_pos_std_dev="0.0"
+      horizontal_vel_std_dev="0.0"
+      vertical_vel_std_dev="0.0">
       <inertia ixx="0.00001" ixy="0.0" ixz="0.0" iyy="0.00001" iyz="0.0" izz="0.00001" />
       <origin xyz="0 0 0" rpy="0 0 0" />

File: rotors_description/urdf/nearthlab_lidar_sensor.xacro (robot description, xacro)
@@ -2,23 +2,17 @@
 <robot xmlns:xacro="http://ros.org/wiki/xacro">
   <xacro:property name="pi" value="3.14159265359" />
-  <xacro:macro name="lidar_macro" params="namespace parent_link *origin **geometry">
+  <xacro:macro name="lidar_macro" params="namespace parent_link *origin">
     <link name="${namespace}/lidar_link">
       <inertial>
-        <pose>0 0 0 0 -0 0</pose>
+        <pose>0 0 0 0 0 0</pose>
         <mass value="0.01" />
         <inertia ixx="2.1733e-6" ixy="0" ixz="0" iyy="2.1733e-6" iyz="0" izz="1.8e-7" />
       </inertial>
       <visual name="visual">
-        <origin xyz="0 0 -0.035" rpy="0 ${pi/2} 0" />
-        <!-- <geometry>
+        <origin xyz="0 0 0" rpy="0 ${pi/2} 0" />
+        <geometry>
           <cylinder length="0.02" radius="0.015" />
-        </geometry> -->
-        <geometry>
-          <xacro:insert_block name="geometry" />
         </geometry>
-        <!-- <material>
-          <script>Gazebo/Black</script>
-        </material> -->
-        <material name="black" />
+        <material name="Grey" />
       </visual>
     </link>
@@ -28,14 +22,16 @@
       <child link="${namespace}/lidar_link" />
     </joint>
-    <gazebo>
+    <gazebo reference="${namespace}/lidar_link">
       <sensor type="ray" name="${namespace}_lidar">
-        <pose>0 0 0 0 -1.570896 0</pose>
+        <pose>0 0 0 0 0 0</pose>
+        <visualize>true</visualize>
+        <update_rate>100</update_rate>
         <ray>
           <scan>
             <horizontal>
-              <samples>1</samples>
+              <samples>8</samples>
               <resolution>1</resolution>
-              <min_angle>-0</min_angle>
-              <max_angle>0</max_angle>
+              <min_angle>${-24.0/180.0*pi}</min_angle>
+              <max_angle>${ 24.0/180.0*pi}</max_angle>
             </horizontal>
           </scan>
@@ -51,9 +47,7 @@
           </noise>
         </ray>
-	      <plugin name="LaserPlugin" filename="librotors_gazebo_lidar_plugin.so"/>
-		    <robotNamespace></robotNamespace>
+	      <plugin name="rotors_gazebo_lidar_plugin" filename="librotors_gazebo_lidar_plugin.so"/>
+		    <robotNamespace>${namespace}</robotNamespace>
         <always_on>1</always_on>
-        <update_rate>20</update_rate>
-        <visualize>true</visualize>
       </sensor>
     </gazebo>

File: rotors_description/urdf/niv1_base.xacro (robot description, xacro)
@@ -30,5 +30,5 @@
   <xacro:if value="$(arg enable_mavlink_interface)">
     <!-- Instantiate mavlink telemetry interface. -->
-    <xacro:niv1_mavlink_interface namespace="${namespace}" imu_sub_topic="imu" rotor_count="6" />
+    <xacro:niv1_mavlink_interface namespace="${namespace}" imu_sub_topic="imu" rotor_count="4" />
   </xacro:if>
   <!-- Mount an ADIS16448 IMU. -->
@@ -44,9 +44,10 @@
     </geometry>
   </xacro:camera_joint_macro>
-  <!-- Camera Sensor-->
+  <!-- Camera Sensor
   <xacro:camera_macro namespace="${namespace}" parent_link="${namespace}/base_link" camera_suffix="${namespace}/camera_suffix" frame_rate="${namespace}/frame_rate" horizontal_fov="1.3962634" image_width="752" image_height="480" image_format="L8" min_distance="0.02" max_distance="30" noise_mean="0.0" noise_stddev="0.007" enable_visual="true">
     <mesh filename="package://rotors_description/meshes/vi_camera.dae" scale="1 1 1" />
     <origin xyz="0 0 -0.035" rpy="0 0 0" />
   </xacro:camera_macro>
+  -->
   <xacro:if value="$(arg enable_ground_truth)">
     <xacro:ground_truth_imu_and_odometry namespace="${namespace}" parent_link="${namespace}/base_link" />
@@ -59,8 +60,5 @@
   <xacro:lidar_macro namespace="${namespace}" parent_link="${namespace}/base_link">
     <!-- <origin xyz="0 0 -0.035" rpy="0 0 0" /> -->
-    <origin xyz="0 0 0" rpy="0 0 0" />
-    <geometry>
-      <cylinder length="0.02" radius="0.015" />
-    </geometry>
+    <origin xyz="0.6 0 0" rpy="0 0 0" />
   </xacro:lidar_macro>
   <!-- Nearthlab Payload -->
@@ -71,11 +69,3 @@
       </geometry>
   </xacro:payload_macro> -->
-  <!-- Nearthlab Windturbine
-  <xacro:windturbine_macro namespace="${namespace}" parent_link="${namespace}/base_link" >
-    <origin xyz="0 0 0" rpy="0 0 0" />
-      <geometry>
-        <mesh filename="package://rotors_description/meshes/nearthlab_windturbine_A_shape.dae" scale="0.05 0.05 0.05" />
-      </geometry>
-  </xacro:windturbine_macro>
-  -->
 </robot>

Commit message: ATTI and GP mode flight success!

File: rotors_description/urdf/component_snippets.xacro (robot description, xacro)
@@ -905,14 +905,14 @@
       imu_topic="imu"
       mass_imu_sensor="0.015"
-      gyroscope_noise_density="0.0003394"
-      gyroscope_random_walk="0.000038785"
+      gyroscope_noise_density="0.0"
+      gyroscope_random_walk="0.0"
       gyroscope_bias_correlation_time="1000.0"
       gyroscope_turn_on_bias_sigma="0.0"
-      accelerometer_noise_density="0.0004"
-      accelerometer_random_walk="0.0006"
+      accelerometer_noise_density="0.0"
+      accelerometer_random_walk="0.0"
       accelerometer_bias_correlation_time="300.0"
       accelerometer_turn_on_bias_sigma="0.0">
       <inertia ixx="0.00001" ixy="0.0" ixz="0.0" iyy="0.00001" iyz="0.0" izz="0.00001" />
-      <origin xyz="0 0 0.05" rpy="0 0 0" />
+      <origin xyz="0 0 0" rpy="0 0 0" />
     </xacro:imu_plugin_macro>
   </xacro:macro>

File: rotors_description/urdf/niv1.xacro (robot description, xacro)
@@ -33,4 +33,5 @@
   <xacro:property name="motor_constant_for_ros_sim" value="8.54858e-05" /> <!-- [kg m/s^2]  force = real_motor_velocity * real_motor_velocity * motor_constant_-->
   <xacro:property name="motor_constant" value="1.2e-04" /> <!-- [kg m/s^2]  force = real_motor_velocity * real_motor_velocity * motor_constant_-->
+  <xacro:property name="moment_constant_org" value="0.025" /> <!-- [m] math::Vector3 drag_torque(0, 0, -turning_direction_ * force * moment_constant_); -->
   <xacro:property name="moment_constant" value="0.025" /> <!-- [m] math::Vector3 drag_torque(0, 0, -turning_direction_ * force * moment_constant_); -->
   <xacro:property name="time_constant_up" value="0.00125" /> <!-- [s] -->

Commit message: Add noise at IMU and GPS. Lidar plugin is implemented

File: rotors_description/urdf/component_snippets.xacro (robot description, xacro)
@@ -905,10 +905,10 @@
       imu_topic="imu"
       mass_imu_sensor="0.015"
-      gyroscope_noise_density="0.0"
-      gyroscope_random_walk="0.0"
+      gyroscope_noise_density="0.0003394"
+      gyroscope_random_walk="0.000038785"
       gyroscope_bias_correlation_time="1000.0"
-      gyroscope_turn_on_bias_sigma="0.0"
-      accelerometer_noise_density="0.0"
-      accelerometer_random_walk="0.0"
+      gyroscope_turn_on_bias_sigma="0.0087"
+      accelerometer_noise_density="0.004"
+      accelerometer_random_walk="0.006"
       accelerometer_bias_correlation_time="300.0"
       accelerometer_turn_on_bias_sigma="0.0">
@@ -926,8 +926,8 @@
       ground_speed_topic="ground_speed"
       mass_gps_sensor="0.015"
-      horizontal_pos_std_dev="0.0"
-      vertical_pos_std_dev="0.0"
-      horizontal_vel_std_dev="0.0"
-      vertical_vel_std_dev="0.0">
+      horizontal_pos_std_dev="0.01"
+      vertical_pos_std_dev="0.01"
+      horizontal_vel_std_dev="0.001"
+      vertical_vel_std_dev="0.001">
       <inertia ixx="0.00001" ixy="0.0" ixz="0.0" iyy="0.00001" iyz="0.0" izz="0.00001" />
       <origin xyz="0 0 0" rpy="0 0 0" />

File: rotors_description/urdf/nearthlab_lidar_sensor.xacro (robot description, xacro)
@@ -2,4 +2,10 @@
 <robot xmlns:xacro="http://ros.org/wiki/xacro">
   <xacro:property name="pi" value="3.14159265359" />
+  <xacro:property name="resolution" value="3" />
+  <xacro:property name="sample" value="8" />
+  <xacro:property name="min_angle_deg" value="-24" />
+  <xacro:property name="max_angle_deg" value="24" />
+  <xacro:property name="view_angle_deg" value="${max_angle_deg-min_angle_deg}" />
+  <xacro:property name="slot_angle_deg" value="${(view_angle_deg/sample)/resolution}" />
   <xacro:macro name="lidar_macro" params="namespace parent_link *origin">
     <link name="${namespace}/lidar_link">
@@ -30,8 +36,8 @@
           <scan>
             <horizontal>
-              <samples>8</samples>
-              <resolution>1</resolution>
-              <min_angle>${-24.0/180.0*pi}</min_angle>
-              <max_angle>${ 24.0/180.0*pi}</max_angle>
+              <samples>${sample}</samples>
+              <resolution>${resolution}</resolution>
+              <min_angle>${(min_angle_deg+(slot_angle_deg/2))/180.0*pi}</min_angle>
+              <max_angle>${(max_angle_deg-(slot_angle_deg/2))/180.0*pi}</max_angle>
             </horizontal>
           </scan>

Commit message: Add windturbine model

File: rotors_description/urdf/component_snippets.xacro (robot description, xacro)
@@ -46,11 +46,8 @@
       <xacro:if value="${enable_visual}">
         <visual>
-          <!-- <origin xyz="0 0 0" rpy="0 ${pi/2} 0" /> -->
-          <!-- <origin xyz="0 0 0" rpy="0 ${pi} 0" /> -->
-          <origin xyz="0.01 0 0" rpy="0 ${pi/2} 0" />
+          <origin xyz="0 0 0" rpy="0 0 0" />
           <geometry>
             <xacro:insert_block name="geometry" />
           </geometry>
-          <material name="red" />
         </visual>
       </xacro:if>
@@ -68,9 +65,9 @@
     <link name="${namespace}/camera_${camera_suffix}_optical_link" />
     <joint name="${namespace}/camera_${camera_suffix}_optical_joint" type="fixed" >
-      <origin xyz="0 0 0" rpy="${-pi/2} 0 ${-pi/2}" />
+      <origin xyz="0.02 0 0" rpy="0 0 0" />
       <parent link="${namespace}/camera_${camera_suffix}_link" />
       <child link="${namespace}/camera_${camera_suffix}_optical_link" />
     </joint>
-    <gazebo reference="${namespace}/camera_${camera_suffix}_link">
+    <gazebo reference="${namespace}/camera_${camera_suffix}_optical_link">
       <sensor type="camera" name="${namespace}_camera_${camera_suffix}">
         <update_rate>${frame_rate}</update_rate>

File: rotors_description/urdf/gimbal_front_v1.xacro (robot description, xacro)
@@ -1,3 +1,6 @@
 <?xml version="1.0"?>
+<!--
+  Copyright 2018 Nearthalb Inc.
+-->
 <robot xmlns:xacro="http://ros.org/wiki/xacro">
   <xacro:property name="pi" value="3.14159265359" />
@@ -10,23 +13,24 @@
   <xacro:macro name="lidar_macro" params="namespace parent_link *origin">
     <link name="${namespace}/lidar_link">
-      <inertial>
-        <pose>0 0 0 0 0 0</pose>
-        <mass value="0.01" />
-        <inertia ixx="2.1733e-6" ixy="0" ixz="0" iyy="2.1733e-6" iyz="0" izz="1.8e-7" />
-      </inertial>
       <visual name="visual">
-        <origin xyz="0 0 0" rpy="0 ${pi/2} 0" />
+        <origin xyz="0 0 0" rpy="${pi/2} 0 0" />
         <geometry>
-          <cylinder length="0.02" radius="0.015" />
+          <mesh filename="package://rotors_description/meshes/leddarvu.dae" scale="1 1 1" />
         </geometry>
-        <material name="Grey" />
       </visual>
     </link>
-    <joint name="${namespace}_lidar_joint" type="fixed">
+    <joint name="${namespace}/lidar_joint" type="fixed">
       <xacro:insert_block name="origin" />
       <parent link="${parent_link}" />
       <child link="${namespace}/lidar_link" />
     </joint>
-    <gazebo reference="${namespace}/lidar_link">
+    <link name="${namespace}/lidar_optical_link">
+    </link>
+    <joint name="${namespace}/lidar_optical_joint" type="fixed">
+      <origin xyz="0.03 0 0" rpy="0 0 0" />
+      <parent link="${namespace}/lidar_link" />
+      <child link="${namespace}/lidar_optical_link" />
+    </joint>
+    <gazebo reference="${namespace}/lidar_optical_link">
       <sensor type="ray" name="${namespace}_lidar">
         <pose>0 0 0 0 0 0</pose>

File: rotors_description/urdf/niv1.xacro (robot description, xacro)
@@ -19,5 +19,5 @@
   <!-- Properties -->
   <xacro:property name="namespace" value="$(arg namespace)" />
-  <xacro:property name="rotor_velocity_slowdown_sim" value="10" />
+  <xacro:property name="rotor_velocity_slowdown_sim" value="30" />
   <xacro:property name="use_mesh_file" value="true" />
   <xacro:property name="mesh_file" value="package://rotors_description/meshes/niv1_body.dae" />
@@ -42,5 +42,5 @@
   <xacro:property name="rotor_drag_coefficient" value="8.06428e-05" /> <!-- math::Vector3 air_drag = -std::abs(real_motor_velocity) * rotor_drag_coefficient_ * body_velocity_perpendicular; -->
   <xacro:property name="rolling_moment_coefficient" value="0.000001" /> <!-- math::Vector3 rolling_moment = -std::abs(real_motor_velocity) * rolling_moment_coefficient_ * body_velocity_perpendicular; -->
-  <xacro:property name="angular_air_resistance" value="0.01" />
+  <xacro:property name="angular_air_resistance" value="0.015" />
   <xacro:property name="linear_air_resistance" value="0.001" />
   <!-- Property Blocks -->

File: rotors_description/urdf/niv1_base.xacro (robot description, xacro)
@@ -19,7 +19,6 @@
   xmlns:xacro="http://ros.org/wiki/xacro">
   <xacro:include filename="$(find rotors_description)/urdf/component_snippets.xacro" />
-  <xacro:include filename="$(find rotors_description)/urdf/nearthlab_lidar_sensor.xacro" />
+  <xacro:include filename="$(find rotors_description)/urdf/leddarvu.xacro" />
   <xacro:include filename="$(find rotors_description)/urdf/nearthlab_payload.xacro" />
-  <xacro:include filename="$(find rotors_description)/urdf/nearthlab_windturbine.xacro" />
   <!-- Instantiate niv1 "mechanics" -->
   <xacro:include filename="$(find rotors_description)/urdf/niv1.xacro" />
@@ -32,33 +31,17 @@
     <xacro:niv1_mavlink_interface namespace="${namespace}" imu_sub_topic="imu" rotor_count="4" />
   </xacro:if>
-  <!-- Mount an ADIS16448 IMU. -->
   <xacro:niv1_imu namespace="${namespace}" parent_link="${namespace}/base_link" />
-  <!-- Added by bkjung -->
   <xacro:niv1_gps namespace="${namespace}" parent_link="${namespace}/base_link" />
   <xacro:niv1_magnetometer namespace="${namespace}" parent_link="${namespace}/base_link" />
   <xacro:niv1_pressure_sensor namespace="${namespace}" parent_link="${namespace}/base_link" />
-  <xacro:camera_joint_macro namespace="${namespace}" parent_link="${namespace}/base_link" camera_suffix="${namespace}/camera_joint" enable_visual="true">
-    <origin xyz="0 0 -0.015" rpy="0 0 0" />
-    <geometry>
-      <cylinder length="0.02" radius="0.006" />
-    </geometry>
-  </xacro:camera_joint_macro>
-  <!-- Camera Sensor
-  <xacro:camera_macro namespace="${namespace}" parent_link="${namespace}/base_link" camera_suffix="${namespace}/camera_suffix" frame_rate="${namespace}/frame_rate" horizontal_fov="1.3962634" image_width="752" image_height="480" image_format="L8" min_distance="0.02" max_distance="30" noise_mean="0.0" noise_stddev="0.007" enable_visual="true">
-    <mesh filename="package://rotors_description/meshes/vi_camera.dae" scale="1 1 1" />
-    <origin xyz="0 0 -0.035" rpy="0 0 0" />
+  <!-- Camera Sensor -->
+  <xacro:camera_macro namespace="${namespace}" parent_link="${namespace}/base_link" camera_suffix="0" frame_rate="30" horizontal_fov="1.448622" image_width="640" image_height="480" image_format="" min_distance="0.02" max_distance="200" noise_mean="0.0" noise_stddev="0.007" enable_visual="true">
+    <mesh filename="package://rotors_description/meshes/csi_camera.dae" scale="1 1 1" />
+    <origin xyz="0.45 0 0.05" rpy="0 0 0" />
   </xacro:camera_macro>
-  -->
-  <xacro:if value="$(arg enable_ground_truth)">
-    <xacro:ground_truth_imu_and_odometry namespace="${namespace}" parent_link="${namespace}/base_link" />
-  </xacro:if>
-  <xacro:if value="$(arg enable_logging)">
-    <!-- Instantiate a logger -->
-    <xacro:bag_plugin_macro namespace="${namespace}" bag_file="$(arg log_file)" rotor_velocity_slowdown_sim="${rotor_velocity_slowdown_sim}" wait_to_record_bag="$(arg wait_to_record_bag)" />
-  </xacro:if>
   <!--LIDAR Sensor-->
   <xacro:lidar_macro namespace="${namespace}" parent_link="${namespace}/base_link">
     <!-- <origin xyz="0 0 -0.035" rpy="0 0 0" /> -->
-    <origin xyz="0.6 0 0" rpy="0 0 0" />
+    <origin xyz="0.4 0 0" rpy="0 0 0" />
   </xacro:lidar_macro>
   <!-- Nearthlab Payload -->
@@ -69,3 +52,10 @@
       </geometry>
   </xacro:payload_macro> -->
+  <xacro:if value="$(arg enable_ground_truth)">
+    <xacro:ground_truth_imu_and_odometry namespace="${namespace}" parent_link="${namespace}/base_link" />
+  </xacro:if>
+  <xacro:if value="$(arg enable_logging)">
+    <!-- Instantiate a logger -->
+    <xacro:bag_plugin_macro namespace="${namespace}" bag_file="$(arg log_file)" rotor_velocity_slowdown_sim="${rotor_velocity_slowdown_sim}" wait_to_record_bag="$(arg wait_to_record_bag)" />
+  </xacro:if>
 </robot>

Commit message: 8 Hz camera, 40 max depth, smaller firefly

File: rotors_description/urdf/component_snippets.xacro (robot description, xacro)
@@ -698,6 +698,6 @@
       <xacro:vi_sensor_stereo_camera_macro
         namespace="${namespace}" parent_link="${namespace}/vi_sensor_link"
-        frame_rate="30.0" origin_offset_x="0.015" baseline_y="${0.055*2}"
-        origin_offset_z="0.0065" max_range="30.0">
+        frame_rate="8.0" origin_offset_x="0.015" baseline_y="${0.055*2}"
+        origin_offset_z="0.0065" max_range="40.0">
       </xacro:vi_sensor_stereo_camera_macro>
     </xacro:if>
@@ -706,5 +706,5 @@
       <xacro:vi_sensor_depth_macro
         namespace="${namespace}" parent_link="${namespace}/vi_sensor_link"
-        camera_suffix="depth" frame_rate="30.0" max_range="30.0">
+        camera_suffix="depth" frame_rate="8.0" max_range="40.0">
         <origin xyz="0.015 0.055 0.0065" rpy="0 0 0" />
       </xacro:vi_sensor_depth_macro>

File: rotors_description/urdf/firefly.xacro (robot description, xacro)
@@ -23,6 +23,6 @@
   <xacro:property name="mesh_file" value="package://rotors_description/meshes/firefly.dae" />
   <xacro:property name="mass" value="1.5" /> <!-- [kg] -->
-  <xacro:property name="body_width" value="0.1" /> <!-- [m] -->
-  <xacro:property name="body_height" value="0.16" /> <!-- [m] -->
+  <xacro:property name="body_width" value="0.05" /> <!-- [m] -->
+  <xacro:property name="body_height" value="0.08" /> <!-- [m] -->
   <xacro:property name="mass_rotor" value="0.005" /> <!-- [kg] -->
   <xacro:property name="arm_length" value="0.215" /> <!-- [m] -->

Commit message: Tune again firefly for planning simulation

File: rotors_description/urdf/component_snippets.xacro (robot description, xacro)
@@ -564,6 +564,6 @@
       image_height="480"
       image_format="L8"
-      min_distance="0.02"
-      max_distance="30"
+      min_distance="0.001"
+      max_distance="40"
       noise_mean="0.0"
       noise_stddev="0.007"
@@ -586,5 +586,5 @@
       image_height="480"
       image_format="L8"
-      min_distance="0.02"
+      min_distance="0.001"
       max_distance="${max_range}"
       noise_mean="0.0"

File: rotors_description/urdf/firefly.xacro (robot description, xacro)
@@ -23,6 +23,6 @@
   <xacro:property name="mesh_file" value="package://rotors_description/meshes/firefly.dae" />
   <xacro:property name="mass" value="1.5" /> <!-- [kg] -->
-  <xacro:property name="body_width" value="0.05" /> <!-- [m] -->
-  <xacro:property name="body_height" value="0.08" /> <!-- [m] -->
+  <xacro:property name="body_width" value="0.10" /> <!-- [m] -->
+  <xacro:property name="body_height" value="0.16" /> <!-- [m] -->
   <xacro:property name="mass_rotor" value="0.005" /> <!-- [kg] -->
   <xacro:property name="arm_length" value="0.215" /> <!-- [m] -->

File: rotors_description/urdf/multirotor_base.xacro (robot description, xacro)
@@ -104,6 +104,6 @@
       </visual>
       <collision>
-        <!--<geometry>
-          <cylinder length="0.005" radius="${radius_rotor}" /> <!- [m] ->
+<!--        <geometry>
+          <cylinder length="0.001" radius="0.001" /> <!- [m] ->
         </geometry>-->
       </collision>

Commit message: modelify paper changes

File: rotors_description/urdf/component_snippets.xacro (robot description, xacro)
@@ -528,5 +528,5 @@
       frame_rate="${frame_rate}"
       horizontal_fov="1.3962634"
-      image_width="752"
+      image_width="640"
       image_height="480"
       image_format="L8"
@@ -549,5 +549,5 @@
       frame_rate="${frame_rate}"
       horizontal_fov="1.3962634"
-      image_width="752"
+      image_width="640"
       image_height="480"
       image_format="L8"
@@ -600,5 +600,5 @@
           <horizontal_fov>2</horizontal_fov>
           <image>
-            <format>L8</format>
+            <format>R8G8B8</format>
             <width>640</width>
             <height>480</height>
@@ -615,7 +615,7 @@
           <updateRate>${frame_rate}</updateRate>
           <cameraName>camera_${camera_suffix}</cameraName>
-          <imageTopicName>camera/image_raw</imageTopicName>
-          <cameraInfoTopicName>camera/camera_info</cameraInfoTopicName>
-          <depthImageTopicName>depth/disparity</depthImageTopicName>
+          <imageTopicName>rgb/image_raw</imageTopicName>
+          <cameraInfoTopicName>rgb/camera_info</cameraInfoTopicName>
+          <depthImageTopicName>depth/image_raw</depthImageTopicName>
           <depthImageCameraInfoTopicName>depth/camera_info</depthImageCameraInfoTopicName>
           <pointCloudTopicName>depth/points</pointCloudTopicName>
@@ -649,5 +649,5 @@
       </visual>
       <inertial>
-        <mass value="0.13" />
+        <mass value="0.005" />
         <origin xyz="0 0 0" rpy="0 0 0" />
         <inertia ixx="1e-6" ixy="0" ixz="0" iyy="1e-6" iyz="0" izz="1e-6" />
@@ -672,5 +672,5 @@
       <xacro:vi_sensor_depth_macro
         namespace="${namespace}" parent_link="${namespace}/vi_sensor_link"
-        camera_suffix="depth" frame_rate="30.0" max_range="10.0">
+        camera_suffix="depth" frame_rate="5.0" max_range="10.0">
         <origin xyz="0.015 0.055 0.0065" rpy="0 0 0" />
       </xacro:vi_sensor_depth_macro>
