Commit message: Pull request synchronized with the latest CrazyS release

File: rotors_description/urdf/component_snippets.xacro (robot description, xacro)
@@ -293,6 +293,6 @@
   <xacro:macro name="imu_plugin_macro"
     params="namespace imu_suffix parent_link imu_topic
-      mass_imu_sensor gyroscope_noise_density gyroscope_random_walk
-      gyroscope_bias_correlation_time gyroscope_turn_on_bias_sigma
+      mass_imu_sensor measurement_divisor measurement_delay gyroscope_noise_density
+      gyroscope_random_walk gyroscope_bias_correlation_time gyroscope_turn_on_bias_sigma
       accelerometer_noise_density accelerometer_random_walk
       accelerometer_bias_correlation_time accelerometer_turn_on_bias_sigma
@@ -321,4 +321,6 @@
         <imuTopic>${imu_topic}</imuTopic> <!-- (string): name of the sensor output topic and prefix of service names (defaults to imu) -->
         <gyroscopeNoiseDensity>${gyroscope_noise_density}</gyroscopeNoiseDensity> <!-- Gyroscope noise density (two-sided spectrum) [rad/s/sqrt(Hz)] -->
+        <measurementDivisor>${measurement_divisor}</measurementDivisor> <!-- only every (seq % measurementDivisor) == 0 measurement is published [int] -->
+        <measurementDelay>${measurement_delay}</measurementDelay> <!-- time that measurement gets held back before it's published in [simulation cycles (int)] -->
         <gyroscopeRandomWalk>${gyroscope_random_walk}</gyroscopeRandomWalk> <!-- Gyroscope bias random walk [rad/s/s/sqrt(Hz)] -->
         <gyroscopeBiasCorrelationTime>${gyroscope_bias_correlation_time}</gyroscopeBiasCorrelationTime> <!-- Gyroscope bias correlation time constant [s] -->
@@ -750,4 +752,6 @@
       parent_link="${namespace}/vi_sensor_link"
       imu_topic="imu"
+      measurement_delay="0"
+      measurement_divisor="1"
       mass_imu_sensor="0.015"
       gyroscope_noise_density="0.0003394"
@@ -770,4 +774,6 @@
       parent_link="${parent_link}"
       imu_topic="ground_truth/imu"
+      measurement_delay="0"
+      measurement_divisor="1"
       mass_imu_sensor="0.00001"
       gyroscope_noise_density="0.0"
@@ -820,4 +826,6 @@
       parent_link="${parent_link}"
       imu_topic="imu"
+      measurement_delay="0"
+      measurement_divisor="1"
       mass_imu_sensor="0.015"
       gyroscope_noise_density="0.0003394"
@@ -833,4 +841,35 @@
     </xacro:imu_plugin_macro>
   </xacro:macro>
+  <xacro:macro name="crazyflie2_odometry" params="namespace parent_link">
+      <xacro:odometry_plugin_macro
+        namespace="${namespace}"
+        odometry_sensor_suffix=""
+        parent_link="${parent_link}"
+        pose_topic="pose"
+        pose_with_covariance_topic="pose_with_covariance"
+        position_topic="position"
+        transform_topic="transform"
+        odometry_topic="odometry"
+        parent_frame_id="world"
+        child_frame_id="${namespace}/base_link"
+        mass_odometry_sensor="0.00001"
+        measurement_divisor="10"
+        measurement_delay="0"
+        unknown_delay="0.0"
+        noise_normal_position="0 0 0"
+        noise_normal_quaternion="0 0 0"
+        noise_normal_linear_velocity="0 0 0"
+        noise_normal_angular_velocity="0 0 0"
+        noise_uniform_position="0 0 0"
+        noise_uniform_quaternion="0 0 0"
+        noise_uniform_linear_velocity="0 0 0"
+        noise_uniform_angular_velocity="0 0 0"
+        enable_odometry_map="false"
+        odometry_map=""
+        image_scale="">
+        <inertia ixx="0.00001" ixy="0.0" ixz="0.0" iyy="0.00001" iyz="0.0" izz="0.00001" /> <!-- [kg m^2] [kg m^2] [kg m^2] [kg m^2] [kg m^2] [kg m^2] -->
+        <origin xyz="0.0 0.0 0.0" rpy="0.0 0.0 0.0" />
+      </xacro:odometry_plugin_macro>
+  </xacro:macro>
   <xacro:macro name="crazyflie2_imu" params="namespace parent_link">
     <!-- Mount an MPU-9250 IMU. -->
@@ -840,4 +879,6 @@
       parent_link="${parent_link}"
       imu_topic="imu"
+      measurement_delay="0"
+      measurement_divisor="1"
       mass_imu_sensor="0.00001"
       gyroscope_noise_density="0.000175"

File: rotors_description/urdf/crazyflie2.xacro (robot description, xacro)
@@ -16,4 +16,5 @@
 -->
 <robot name="crazyflie2" xmlns:xacro="http://ros.org/wiki/xacro">
+  <!-- Properties (Taken from Novel Dynamic Inversion Architecture Design for Quadrocopter Control by Jian Wang et al.) -->
   <xacro:property name="namespace" value="$(arg mav_name)" />
   <xacro:property name="rotor_velocity_slowdown_sim" value="50" />
@@ -29,4 +30,5 @@
   <xacro:property name="sin45" value="0.707106781186" />
   <xacro:property name="cos45" value="0.707106781186" />
+  <!-- Forster's -->
   <xacro:property name="motor_constant" value="1.28192e-08" /> <!-- [kg m/s^2] -->
   <xacro:property name="moment_constant" value="5.964552e-03" /> <!-- [m] -->

File: rotors_description/urdf/crazyflie2_base.xacro (robot description, xacro)
@@ -21,10 +21,16 @@
   <!-- Instantiate a controller. -->
   <xacro:controller_plugin_macro namespace="${namespace}" imu_sub_topic="imu" />
+  <!-- Enable the MAVLink interface. It is useful for the HIL (Hardware-in-the-loop) tests -->
   <xacro:if value="$(arg enable_mavlink_interface)">
     <!-- Instantiate mavlink telemetry interface. -->
     <xacro:default_mavlink_interface namespace="${namespace}" imu_sub_topic="imu" rotor_count="4" />
   </xacro:if>
-  <!-- Mount an MPU-9250 IMU. -->
-  <xacro:crazyflie2_imu namespace="${namespace}" parent_link="${namespace}/base_link" />
+  <!-- Mount an MPU-9250 IMU if the state estimator is enabled, otherwise the virtual odometry sensor is used. -->
+  <xacro:if value="$(arg enable_state_estimator)">
+    <xacro:crazyflie2_imu namespace="${namespace}" parent_link="${namespace}/base_link" />
+  </xacro:if>
+  <!-- Mount a generic odometry sensor. -->
+  <xacro:crazyflie2_odometry namespace="${namespace}" parent_link="${namespace}/base_link" />
+  <!-- Mount a generic odometry sensor employed as ground truth -->
   <xacro:if value="$(arg enable_ground_truth)">
     <xacro:ground_truth_imu_and_odometry namespace="${namespace}" parent_link="${namespace}/base_link" />

Commit message: GPS plugin modification for hil_gps msg data, camera xacro mods
- New GPS message (copied from PX4 sitl_gazebo). Allows to communicate data used for hil_gps mavlink msg
- According mods to gps plugin (advertise, publish SITLGps with (optional) simulated delay and customized rate), similar to sitl_gazebo gps plugin
- Adjust xacro gps blocks (two plugins for one sensor to enable publication of both noisy+delayed and ground truth data)
- debug camera macro... WIP

File: rotors_description/urdf/component_snippets.xacro (robot description, xacro)
@@ -111,4 +111,75 @@
     </gazebo>
   </xacro:macro>
+  <!-- Macro to add a camera. 2 -->
+  <xacro:macro name="camera_macro_2"
+    params="namespace parent_link camera_suffix frame_rate
+      horizontal_fov image_width image_height image_format min_distance
+      max_distance noise_mean noise_stddev enable_visual *geometry *origin">
+    <link name="${namespace}/camera_${camera_suffix}_link">
+    <collision>
+      <origin xyz="0 0 0" rpy="0 0 0" />
+      <geometry>
+        <xacro:insert_block name="geometry" />
+      </geometry>
+    </collision>
+    <xacro:if value="${enable_visual}">
+      <visual>
+        <origin xyz="0 0 0" rpy="0 ${pi/2} 0" />
+        <geometry>
+          <xacro:insert_block name="geometry" />
+        </geometry>
+        <material name="red" />
+      </visual>
+    </xacro:if>
+      <inertial>
+        <mass value="1e-5" />
+        <origin xyz="0 0 0" rpy="0 0 0" />
+        <inertia ixx="1e-6" ixy="0" ixz="0" iyy="1e-6" iyz="0" izz="1e-6" />
+      </inertial>
+    </link>
+    <joint name="${namespace}/camera_${camera_suffix}_joint" type="revolute">
+      <xacro:insert_block name="origin" />
+      <parent link="${parent_link}" />
+      <child link="${namespace}/camera_${camera_suffix}_link" />
+      <limit upper="0" lower="0" effort="0" velocity="0" />
+    </joint>
+    <gazebo reference="${namespace}/camera_${camera_suffix}_link">
+      <sensor type="camera" name="${namespace}_camera_${camera_suffix}">
+        <update_rate>${frame_rate}</update_rate>
+        <camera name="head">
+          <horizontal_fov>${horizontal_fov}</horizontal_fov>
+          <image>
+            <width>${image_width}</width>
+            <height>${image_height}</height>
+            <format>${image_format}</format>
+          </image>
+          <clip>
+            <near>${min_distance}</near>
+            <far>${max_distance}</far>
+          </clip>
+          <noise>
+            <type>gaussian</type>
+            <mean>${noise_mean}</mean>
+            <stddev>${noise_stddev}</stddev>
+          </noise>
+        </camera>
+        <plugin name="${namespace}_camera_${camera_suffix}_controller" filename="libgazebo_ros_camera.so">
+          <robotNamespace>${namespace}</robotNamespace>
+          <alwaysOn>true</alwaysOn>
+          <updateRate>${frame_rate}</updateRate>
+          <cameraName>camera_${camera_suffix}</cameraName>
+          <imageTopicName>image_raw</imageTopicName>
+          <cameraInfoTopicName>camera_info</cameraInfoTopicName>
+          <frameName>camera_${camera_suffix}_link</frameName>
+          <hackBaseline>0.7</hackBaseline>
+          <distortionK1>0.0</distortionK1>
+          <distortionK2>0.0</distortionK2>
+          <distortionK3>0.0</distortionK3>
+          <distortionT1>0.0</distortionT1>
+          <distortionT2>0.0</distortionT2>
+        </plugin>
+      </sensor>
+    </gazebo>
+  </xacro:macro>
   <!-- Camera joint macro - just the joints, links, and collisions for a single
        camera. -->
@@ -387,5 +458,5 @@
     params="namespace gps_suffix parent_link gps_topic ground_speed_topic
       mass_gps_sensor horizontal_pos_std_dev vertical_pos_std_dev
-      horizontal_vel_std_dev vertical_vel_std_dev *inertia *origin">
+      horizontal_vel_std_dev vertical_vel_std_dev enable_delay *inertia *origin">
     <!-- GPS link -->
     <link name="${namespace}/gps${gps_suffix}_link">
@@ -456,4 +527,6 @@
           <horVelStdDev>${horizontal_vel_std_dev}</horVelStdDev> <!-- standard deviation for horizontal speed noise [m/s] -->
           <verVelStdDev>${vertical_vel_std_dev}</verVelStdDev> <!-- standard deviation for vertical speed noise [m/s] -->
+          <enableDelay>${enable_delay}</enableDelay>
+          <!--<rqstFwdToRos>${rqst_fwd_to_ros}</rqstFwdToRos>-->
         </plugin>
       </sensor>
@@ -831,6 +904,25 @@
     </xacro:imu_plugin_macro>
   </xacro:macro>
-  <xacro:macro name="default_gps" params="namespace parent_link">
-    <!-- Default GPS. -->
+  <xacro:macro name="default_camera" params="namespace parent_link camera_suffix *origin">
+    <xacro:camera_macro_2
+      namespace="${namespace}"
+      parent_link="${parent_link}"
+      camera_suffix="${camera_suffix}"
+      frame_rate="30"
+      horizontal_fov="1.3962634"
+      image_width="752"
+      image_height="480"
+      image_format="L8"
+      min_distance="0.02"
+      max_distance="8000"
+      noise_mean="0.0"
+      noise_stddev="0.007"
+      enable_visual="true">
+      <mesh filename="package://rotors_description/meshes/vi_camera.dae" scale="1 1 1" />
+      <xacro:insert_block name="origin" />
+    </xacro:camera_macro_2>
+  </xacro:macro>
+  <xacro:macro name="default_gps" params="namespace parent_link *origin">
+    <!-- Default GPS including ground truth GPS -->
     <xacro:gps_plugin_macro
       namespace="${namespace}"
@@ -843,7 +935,23 @@
       vertical_pos_std_dev="6.0"
       horizontal_vel_std_dev="0.1"
-      vertical_vel_std_dev="0.1">
+      vertical_vel_std_dev="0.1"
+      enable_delay = "true">
       <inertia ixx="0.00001" ixy="0.0" ixz="0.0" iyy="0.00001" iyz="0.0" izz="0.00001" />
-      <origin xyz="0 0 0" rpy="0 0 0" />
+      <xacro:insert_block name="origin" />
+    </xacro:gps_plugin_macro>
+    <xacro:gps_plugin_macro
+      namespace="${namespace}"
+      gps_suffix="_gt"
+      parent_link="${parent_link}"
+      gps_topic="gps_gt"
+      ground_speed_topic="ground_speed_gt"
+      mass_gps_sensor="0.001"
+      horizontal_pos_std_dev="0.0"
+      vertical_pos_std_dev="0.0"
+      horizontal_vel_std_dev="0.0"
+      vertical_vel_std_dev="0.0"
+      enable_delay = "false">
+      <inertia ixx="0.00001" ixy="0.0" ixz="0.0" iyy="0.00001" iyz="0.0" izz="0.00001" />
+      <xacro:insert_block name="origin" />
     </xacro:gps_plugin_macro>
   </xacro:macro>

File: rotors_description/urdf/techpod_base.xacro (robot description, xacro)
@@ -16,8 +16,30 @@
   <!-- Instantiate fixed wing "mechanics" -->
   <xacro:include filename="$(find rotors_description)/urdf/techpod.xacro" />
+  <!--
+  <xacro:default_camera
+    namespace="${namespace}"
+    parent_link="${namespace}/base_link"
+    camera_suffix="cam_left">
+    <origin xyz="0.3 0.1 0.075" rpy="0 0.1 1.75" />
+  </xacro:default_camera>
+  <xacro:default_camera
+    namespace="${namespace}"
+    parent_link="${namespace}/base_link"
+    camera_suffix="cam_right">
+    <origin xyz="0.3 -0.1 0.075" rpy="0 0.1 -1.75" />
+  </xacro:default_camera>
+  <xacro:default_camera
+    namespace="${namespace}"
+    parent_link="${namespace}/base_link"
+    camera_suffix="cam_front">
+    <origin xyz="0.5 0 0.06" rpy="0 -0.2 0" />
+  </xacro:default_camera>
+  -->
   <!-- Mount an ADIS16448 IMU. -->
   <xacro:default_imu namespace="${namespace}" parent_link="${namespace}/base_link" />
   <!-- Mount a GPS. -->
-  <xacro:default_gps namespace="${namespace}" parent_link="${namespace}/base_link" />
+  <xacro:default_gps namespace="${namespace}" parent_link="${namespace}/base_link" >
+    <origin xyz="0 0 0" rpy="0 0 0" />
+  </xacro:default_gps>
   <!-- Mount a magnetometer. -->
   <xacro:default_magnetometer namespace="${namespace}" parent_link="${namespace}/base_link" />

Commit message: Add macro for gazebo-imu based imu plugin
- Fix camera collision frames
- Increase GPS update rate to 10Hz to reduce timeouts on pixhawk side

File: rotors_description/urdf/component_snippets.xacro (robot description, xacro)
@@ -39,5 +39,5 @@
     <link name="${namespace}/camera_${camera_suffix}_link">
       <collision>
-        <origin xyz="0 0 0" rpy="0 0 0" />
+        <origin xyz="0 0 0" rpy="0 ${pi/2} 0" />
         <geometry>
           <xacro:insert_block name="geometry" />
@@ -117,10 +117,12 @@
       max_distance noise_mean noise_stddev enable_visual *geometry *origin">
     <link name="${namespace}/camera_${camera_suffix}_link">
+    <!--
     <collision>
-      <origin xyz="0 0 0" rpy="0 0 0" />
+      <origin xyz="0 0 0" rpy="0 ${pi/2} 0" />
       <geometry>
         <xacro:insert_block name="geometry" />
       </geometry>
     </collision>
+    -->
     <xacro:if value="${enable_visual}">
       <visual>
@@ -400,4 +402,51 @@
     </gazebo>
   </xacro:macro>
+  <!-- Macro to add an IMU (using Gazebo IMU) -->
+  <xacro:macro name="imu_s_plugin_macro"
+  params="namespace imu_suffix parent_link imu_topic
+    mass_imu_sensor *inertia *origin">
+  <!-- IMU link -->
+  <link name="${namespace}/imu${imu_suffix}_link">
+    <inertial>
+      <xacro:insert_block name="inertia" />
+      <mass value="${mass_imu_sensor}" />  <!-- [kg] -->
+      <origin xyz="0 0 0" rpy="0 0 0" />
+    </inertial>
+  </link>
+  <!-- IMU joint -->
+  <joint name="${namespace}/imu${imu_suffix}_joint" type="revolute">
+    <xacro:insert_block name="origin" />
+    <parent link="${parent_link}" />
+    <child link="${namespace}/imu${imu_suffix}_link" />
+    <limit upper="0" lower="0" effort="0" velocity="0" />
+  </joint>
+  <gazebo reference="${namespace}/imu${imu_suffix}_link">
+    <gravity>true</gravity>
+    <sensor name="imu_sensor" type="imu">
+      <pose>0 0 0 0 0 0</pose>
+      <always_on>true</always_on>
+      <visualize>true</visualize>
+      <topic>__default_topic__</topic>
+      <update_rate>100</update_rate>
+      <imu>
+        <angular_velocity>
+          <x></x>
+          <y></y>
+          <y></y>
+        </angular_velocity>
+        <linear_acceleration>
+          <x></x>
+          <y></y>
+          <y></y>
+        </linear_acceleration>
+      </imu>
+      <plugin filename="librotors_gazebo_imu_s_plugin.so" name="rotors_gazebo_imu_s_plugin">
+        <robotNamespace>${namespace}</robotNamespace> <!-- (string, required): ros namespace in which the messages are published -->
+        <linkName>${namespace}/imu${imu_suffix}_link</linkName> <!-- (string, required): name of the body which holds the IMU sensor -->
+        <imuTopic>${imu_topic}</imuTopic> <!-- (string): name of the sensor output topic and prefix of service names (defaults to imu) -->
+      </plugin>
+    </sensor>
+  </gazebo>
+  </xacro:macro>
   <!-- Macro to add a generic odometry sensor. -->
   <xacro:macro name="odometry_plugin_macro"
@@ -479,5 +528,5 @@
         <visualize>0</visualize>
         <always_on>1</always_on>
-        <update_rate>5</update_rate>
+        <update_rate>10</update_rate>
         <gps>
           <position_sensing>
