Commit message: Modified state-machine for payload-reset in payload plugin, new features of techpod_X_flex (payload with aerod., payload on rope...)
- Payload plugin: During reload/resetting of payload, first "beam" payload to desired pose before activating joint forces
- techpod_X_flex: Tail camera, payload camera, payload aerodynamics, payload on rope (all commented). Formatting.
- rope.xacro: Xacro macro to simulate a rope (multiple cylindrical links connected by ball joints, aerodynamic forces acting on rope)
- fixed_wing_X_base.xacro: Added parameter to control wing flexing properties (on/off), minor mods to nomenclature
- component_snippets.xacro: More compact inertial properties, minor changes to camera macro parameters

File: rotors_description/urdf/component_snippets.xacro (robot description, xacro)
@@ -18,4 +18,14 @@
 <robot xmlns:xacro="http://ros.org/wiki/xacro">
   <xacro:property name="pi" value="3.14159265359" />
+  <!-- Macro for the inertia of a box -->
+  <xacro:macro name="box_inertia" params="x y z mass">
+    <inertia ixx="${0.0833333 * mass * (y*y + z*z)}" ixy="0.0" ixz="0.0"
+      iyy="${0.0833333 * mass * (x*x + z*z)}" iyz="0.0"
+      izz="${0.0833333 * mass * (x*x + y*y)}" />
+  </xacro:macro>
+  <!-- Macro for the inertia of a cube -->
+  <xacro:macro name="cube_inertia" params="l mass">
+    <xacro:box_inertia x="${l}" y="${l}" z="${l}" mass="${mass}" />
+  </xacro:macro>
   <!-- Macro to add logging to a bag file. -->
   <xacro:macro name="bag_plugin_macro"
@@ -115,5 +125,5 @@
     params="namespace parent_link camera_suffix frame_rate
       horizontal_fov image_width image_height image_format min_distance
-      max_distance noise_mean noise_stddev enable_visual *geometry *origin">
+      max_distance noise_mean noise_stddev mass enable_visual *geometry *inertia *origin">
     <link name="${namespace}/camera_${camera_suffix}_link">
     <!--
@@ -135,7 +145,7 @@
     </xacro:if>
       <inertial>
-        <mass value="1e-5" />
-        <origin xyz="0 0 0" rpy="0 0 0" />
-        <inertia ixx="1e-6" ixy="0" ixz="0" iyy="1e-6" iyz="0" izz="1e-6" />
+        <mass value="${mass}" />
+        <origin xyz="0 0 0" rpy="0 0 0" />
+        <xacro:insert_block name="inertia" />
       </inertial>
     </link>
@@ -322,5 +332,6 @@
   <!-- ==================== ROS INTERFACE MACRO ====================== -->
   <!-- =============================================================== -->
-  <!-- <xacro:macro
+  <!--
+  <xacro:macro
   		name="ros_interface_plugin_macro"
   		params="namespace">
@@ -330,5 +341,6 @@
       </plugin>
     </gazebo>
-  </xacro:macro>-->
+  </xacro:macro>
+  -->
   <!-- =============================================================== -->
   <!-- ================== MAVLINK INTERFACE MACRO ==================== -->
@@ -930,5 +942,5 @@
       odometry_map=""
       image_scale="">
-      <inertia ixx="0.00001" ixy="0.0" ixz="0.0" iyy="0.00001" iyz="0.0" izz="0.00001" /> <!-- [kg m^2] [kg m^2] [kg m^2] [kg m^2] [kg m^2] [kg m^2] -->
+      <xacro:cube_inertia l="0.001" mass="0.00001" /> <!-- [kg m^2] [kg m^2] [kg m^2] [kg m^2] [kg m^2] [kg m^2] -->
       <origin xyz="0.0 0.0 0.0" rpy="0.0 0.0 0.0" />
     </xacro:odometry_plugin_macro>
@@ -950,5 +962,5 @@
       accelerometer_bias_correlation_time="300.0"
       accelerometer_turn_on_bias_sigma="0.1960">
-      <inertia ixx="0.00001" ixy="0.0" ixz="0.0" iyy="0.00001" iyz="0.0" izz="0.00001" />
+      <xacro:cube_inertia l="0.02" mass="0.015" />
       <origin xyz="0 0 0" rpy="0 0 0" />
     </xacro:imu_plugin_macro>
@@ -968,6 +980,8 @@
       noise_mean="0.0"
       noise_stddev="0.007"
+      mass = "0.01"
       enable_visual="true">
       <mesh filename="package://rotors_description/meshes/vi_camera.dae" scale="1 1 1" />
+      <xacro:cube_inertia l="0.02" mass="0.01" />
       <xacro:insert_block name="origin" />
     </xacro:camera_macro_2>
@@ -987,5 +1001,5 @@
       vertical_vel_std_dev="0.1"
       enable_delay = "true">
-      <inertia ixx="0.00001" ixy="0.0" ixz="0.0" iyy="0.00001" iyz="0.0" izz="0.00001" />
+      <xacro:cube_inertia l="0.02" mass="0.015" />
       <xacro:insert_block name="origin" />
     </xacro:gps_plugin_macro>
@@ -1002,5 +1016,5 @@
       vertical_vel_std_dev="0.0"
       enable_delay = "false">
-      <inertia ixx="0.00001" ixy="0.0" ixz="0.0" iyy="0.00001" iyz="0.0" izz="0.00001" />
+      <xacro:cube_inertia l="0.02" mass="0.001" />
       <xacro:insert_block name="origin" />
     </xacro:gps_plugin_macro>
@@ -1019,5 +1033,5 @@
       noise_normal="0.000000080 0.000000080 0.000000080"
       noise_uniform_initial_bias="0.000000400 0.000000400 0.000000400">
-      <inertia ixx="0.00001" ixy="0.0" ixz="0.0" iyy="0.00001" iyz="0.0" izz="0.00001" />
+      <xacro:cube_inertia l="0.02" mass="0.015" />
       <origin xyz="0 0 0" rpy="0 0 0" />
     </xacro:magnetometer_plugin_macro>
@@ -1032,5 +1046,5 @@
       reference_altitude="500.0"
       pressure_variance="0.0">
-      <inertia ixx="0.00001" ixy="0.0" ixz="0.0" iyy="0.00001" iyz="0.0" izz="0.00001" />
+      <xacro:cube_inertia l="0.002" mass="0.015" />
       <origin xyz="0 0 0" rpy="0 0 0" />
     </xacro:pressure_sensor_plugin_macro>

File: rotors_description/urdf/fixed_wing_X_base.xacro (robot description, xacro)
@@ -25,5 +25,5 @@
       izz="${0.5 * mass * r * r}" />
   </xacro:macro>
-  <!-- Macro for the inertia of a cylinder -->
+  <!-- Macro for the inertia of a sphere -->
   <xacro:macro name="sphere_inertia" params="r mass">
     <inertia ixx="${0.4 * mass * r*r}" ixy="0.0" ixz="0.0"
@@ -64,14 +64,29 @@
 <!-- Airfoil segment joint, link and plugin -->
 <xacro:macro name="airfoil_segment"
-  params="robot_namespace segment_name parent mass_segment k c color use_mesh_file mesh_file segment_length segment_width
+  params="robot_namespace segment_name parent mass_segment do_flex k c color use_mesh_file mesh_file segment_length segment_width
     segment_height *axis *joint_origin *inertia_origin *vis_coll_origin *inertia ">
-  <joint name="${robot_namespace}/${segment_name}_joint" type="revolute">
-    <xacro:insert_block name="joint_origin" />
-    <xacro:insert_block name="axis" />
-    <parent link="${parent}" />
-    <child link="${robot_namespace}/${segment_name}"/>
-    <limit upper="0.17" lower="-0.17" effort="5000" velocity="50"/>
-    <dynamics damping="${c}"/>
-  </joint>
+  <xacro:if value="${do_flex}">
+    <joint name="${robot_namespace}/${segment_name}_joint" type="revolute">
+      <xacro:insert_block name="joint_origin" />
+      <xacro:insert_block name="axis" />
+      <parent link="${parent}" />
+      <child link="${robot_namespace}/${segment_name}"/>
+      <limit upper="0.17" lower="-0.17" effort="5000" velocity="50"/>
+      <dynamics damping="${c}"/>
+    </joint>
+    <gazebo reference="${robot_namespace}/${segment_name}_joint">
+      <implicitSpringDamper>true</implicitSpringDamper>
+      <springStiffness>${k}</springStiffness>
+    </gazebo>
+  </xacro:if>
+  <xacro:unless value="${do_flex}">
+    <joint name="${robot_namespace}/${segment_name}_joint" type="revolute">
+      <xacro:insert_block name="joint_origin" />
+      <xacro:insert_block name="axis" />
+      <parent link="${parent}" />
+      <child link="${robot_namespace}/${segment_name}"/>
+      <limit upper="0" lower="-0" effort="5000" velocity="50"/>
+    </joint>
+  </xacro:unless>
   <link name="${robot_namespace}/${segment_name}">
     <inertial>
@@ -106,18 +121,4 @@
     <material>Gazebo/${color}</material>
   </gazebo>
-  <gazebo reference="${robot_namespace}/${segment_name}_joint">
-    <implicitSpringDamper>true</implicitSpringDamper>
-    <springStiffness>${k}</springStiffness>
-  </gazebo>
-  <!--
-  <gazebo>
-    <plugin filename="librotors_gazebo_springdamper_plugin.so" name="gazebo_springdamper_plugin">
-      <robotNamespace>${robot_namespace}</robotNamespace>
-      <jointName>${robot_namespace}/${segment_name}_joint</jointName>
-      <damping>${c}</damping>
-      <stiffness>${k}</stiffness>
-    </plugin>
-  </gazebo>
-  -->
 </xacro:macro>
   <!-- Control surface joint and link -->
@@ -125,5 +126,5 @@
     params="robot_namespace surface_name parent mass_surface min_angle
       max_angle color use_mesh_file mesh_file surface_length surface_width
-      surface_height *axis *joint_origin *link_origin *vis_coll_origin *inertia">
+      surface_height *axis *joint_origin *inertia_origin *vis_coll_origin *inertia">
     <joint name="${robot_namespace}/${surface_name}_joint" type="revolute">
       <xacro:insert_block name="joint_origin" />
@@ -135,5 +136,5 @@
     <link name="${robot_namespace}/${surface_name}">
       <inertial>
-        <xacro:insert_block name="link_origin" />
+        <xacro:insert_block name="inertia_origin" />
         <mass value="${mass_surface}" />
         <xacro:insert_block name="inertia" />
