Commit message: Modified state-machine for payload-reset in payload plugin, new features of techpod_X_flex (payload with aerod., payload on rope...)
- Payload plugin: During reload/resetting of payload, first "beam" payload to desired pose before activating joint forces
- techpod_X_flex: Tail camera, payload camera, payload aerodynamics, payload on rope (all commented). Formatting.
- rope.xacro: Xacro macro to simulate a rope (multiple cylindrical links connected by ball joints, aerodynamic forces acting on rope)
- fixed_wing_X_base.xacro: Added parameter to control wing flexing properties (on/off), minor mods to nomenclature
- component_snippets.xacro: More compact inertial properties, minor changes to camera macro parameters

File: rotors_description/urdf/techpod_X_flex.xacro (robot description, xacro)
@@ -1,3 +1,3 @@
-<?xml version="1.0"?>
+<?xml version="1.0" encoding="UTF-8"?>
 <!--
   Copyright 2016 Pavel Vechersky, ASL, ETH Zurich, Switzerland
@@ -12,1247 +12,1093 @@
   limitations under the License.
 -->
-<robot name="techpod_X_flex" xmlns:xacro="http://ros.org/wiki/xacro">
-  <!-- Global properties -->
-  <xacro:property name="namespace" value="$(arg namespace)" />
-  <xacro:property name="rotor_velocity_slowdown_sim" value="10" />
-  <xacro:property name="use_mesh" value="true" />
-  <xacro:property name="yaml_path" value="$(arg yaml_path)"/>
-  <!-- Constants -->
-  <xacro:property name="PI" value="3.1415926535897931" />
-  <!-- Component masses -->
-  <xacro:property name="mass_fuselage" value="1.8" /> <!-- [kg] -->
-  <xacro:property name="mass_aileron" value="0.1" /> <!-- [kg] -->
-  <xacro:property name="mass_flap" value="0.1" /> <!-- [kg] -->
-  <xacro:property name="mass_elevator" value="0.1" /> <!-- [kg] -->
-  <xacro:property name="mass_rudder" value="0.1" /> <!-- [kg] -->
-  <xacro:property name="mass_propeller" value="0.01" /> <!-- [kg] -->
-  <!-- Main body properties -->
-  <xacro:property name="body_length" value="1.088" /> <!-- [m] -->
-  <xacro:property name="body_width" value="2.591" /> <!-- [m] -->
-  <xacro:property name="body_height" value="0.303" /> <!-- [m] -->
-  <xacro:property name="body_color" value="White" />
-  <xacro:property name="body_mesh_file" value="package://rotors_description/meshes/techpod/techpod_body.dae" />
-  <!-- Aileron properties -->
-  <xacro:property name="aileron_length" value="0.053" /> <!-- [m] -->
-  <xacro:property name="aileron_width" value="0.349" /> <!-- [m] -->
-  <xacro:property name="aileron_height" value="0.013" /> <!-- [m] -->
-  <xacro:property name="aileron_min_angle" value="-0.349066" /> <!-- [rad] -->
-  <xacro:property name="aileron_max_angle" value="0.349066" /> <!-- [rad] -->
-  <xacro:property name="aileron_color" value="${body_color}" />
-  <xacro:property name="aileron_left_mesh_file" value="package://rotors_description/meshes/techpod/techpod_aileron_left.dae" />
-  <xacro:property name="aileron_right_mesh_file" value="package://rotors_description/meshes/techpod/techpod_aileron_right.dae" />
-  <!-- Elevator properties -->
-  <xacro:property name="elevator_length" value="0.051" /> <!-- [m] -->
-  <xacro:property name="elevator_width" value="0.457" /> <!-- [m] -->
-  <xacro:property name="elevator_height" value="0.012" /> <!-- [m] -->
-  <xacro:property name="elevator_min_angle" value="-0.349066" /> <!-- [rad] -->
-  <xacro:property name="elevator_max_angle" value="0.349066" /> <!-- [rad] -->
-  <xacro:property name="elevator_color" value="${body_color}" />
-  <xacro:property name="elevator_mesh_file" value="package://rotors_description/meshes/techpod/techpod_elevator.dae" />
-  <!-- Flap properties -->
-  <xacro:property name="flap_length" value="0.076" /> <!-- [m] -->
-  <xacro:property name="flap_width" value="0.459" /> <!-- [m] -->
-  <xacro:property name="flap_height" value="0.016" /> <!-- [m] -->
-  <xacro:property name="flap_min_angle" value="-0.349066" /> <!-- [rad] -->
-  <xacro:property name="flap_max_angle" value="0.349066" /> <!-- [rad] -->
-  <xacro:property name="flap_color" value="${body_color}" />
-  <xacro:property name="flap_left_mesh_file" value="package://rotors_description/meshes/techpod/techpod_flap_left.dae" />
-  <xacro:property name="flap_right_mesh_file" value="package://rotors_description/meshes/techpod/techpod_flap_right.dae" />
-  <!-- Rudder properties -->
-  <xacro:property name="rudder_length" value="0.129" />
-  <xacro:property name="rudder_width" value="0.018" />
-  <xacro:property name="rudder_height" value="0.241" />
-  <xacro:property name="rudder_min_angle" value="-0.349066" />
-  <xacro:property name="rudder_max_angle" value="0.349066" />
-  <xacro:property name="rudder_color" value="Red" />
-  <xacro:property name="rudder_mesh_file" value="package://rotors_description/meshes/techpod/techpod_rudder.dae" />
-  <!-- Propeller properties -->
-  <xacro:property name="propeller_direction" value="cw" />
-  <xacro:property name="propeller_radius" value="0.1" />
-  <xacro:property name="propeller_height" value="0.003" />
-  <xacro:property name="propeller_color" value="Gray" />
-  <xacro:property name="propeller_mesh_file" value="package://rotors_description/meshes/propeller_${propeller_direction}.dae" />
-  <!-- Flexing properties -->
-<!--
-<xacro:property name="k1" value="450" />
-<xacro:property name="d1" value="3.5" />
-<xacro:property name="k2" value="140" />
-<xacro:property name="d2" value="1.9" />
-<xacro:property name="k3" value="60" />
-<xacro:property name="d3" value="1.0" />
-<xacro:property name="k4" value="80" />
-<xacro:property name="d4" value="1.2" />
--->
-<xacro:property name="k1" value="250" />
-<xacro:property name="d1" value="2" />
-<xacro:property name="k2" value="120" />
-<xacro:property name="d2" value="1.0" />
-<xacro:property name="k3" value="30" />
-<xacro:property name="d3" value="0.7" />
-<xacro:property name="k4" value="80" />
-<xacro:property name="d4" value="1.2" />
-  <!-- Inertia of the main body -->
-  <xacro:property name="body_inertia">
-    <inertia ixx="0.16632" ixy="0.0" ixz="0.0755" iyy="0.3899" iyz="0.0" izz="0.5243" />
-  </xacro:property>
-  <!-- Inertia of the aileron, assuming it is a cuboid -->
-  <xacro:property name="aileron_inertia">
-    <xacro:box_inertia x="${aileron_length}" y="${aileron_width}" z="${aileron_height}" mass="${mass_aileron}" />
-  </xacro:property>
-  <!-- Inertia of the elevator, assuming it is a cuboid -->
-  <xacro:property name="elevator_inertia">
-    <xacro:box_inertia x="${elevator_length}" y="${elevator_width}" z="${elevator_height}" mass="${mass_elevator}" />
-  </xacro:property>
-  <!-- Inertia of the flap, assuming it is a cuboid -->
-  <xacro:property name="flap_inertia">
-    <xacro:box_inertia x="${flap_length}" y="${flap_width}" z="${flap_height}" mass="${mass_flap}" />
-  </xacro:property>
-  <!-- Inertia of the rudder, assuming it is a cuboid -->
-  <xacro:property name="rudder_inertia">
-    <xacro:box_inertia x="${rudder_length}" y="${rudder_width}" z="${rudder_height}" mass="${mass_rudder}" />
-  </xacro:property>
-  <!-- Inertia of the propeller, assuming it is a cylinder -->
-  <xacro:property name="propeller_inertia">
-    <xacro:cylinder_inertia r="${propeller_radius}" h="${propeller_height}" mass="${mass_propeller*rotor_velocity_slowdown_sim}" />
-  </xacro:property>
-  <!-- Included URDF Files -->
-  <xacro:include filename="$(find rotors_description)/urdf/fixed_wing_X_base.xacro" />
-  <!-- Instantiate fixed_wing_base_macro once -->
-  <xacro:fixed_wing_base_macro
-    robot_namespace="${namespace}"
-    mass="${mass_fuselage}"
-    length="${body_length}"
-    width="0.2"
-    height="${body_height}"
-    color="${body_color}"
-    use_mesh_file="${use_mesh}"
-    mesh_file="package://rotors_description/meshes/techpod_X_flex/fuselage_barless.stl">
-    <origin xyz="0.10 0 0.08" rpy="0 0 0" />
-    <xacro:insert_block name="body_inertia" />
-  </xacro:fixed_wing_base_macro>
-<joint name="${namespace}/dome_joint" type="fixed">
-  <parent link="${namespace}/base_link" />
-  <child link="${namespace}/dome" />
-</joint>
-<link name="${namespace}/dome">
-  <inertial>
-    <mass value="0.001" />
-    <xacro:box_inertia x="0.001" y="0.001" z="0.001" mass="0.001" />
-  </inertial>
-  <visual>
-    <geometry>
-        <mesh filename="package://rotors_description/meshes/techpod_X_flex/dome.stl" scale="1 1 1" />
-    </geometry>
-  </visual>
-</link>
-<gazebo reference="${namespace}/dome">
-  <material>Gazebo/GreyTransparent</material>
-</gazebo>
-<joint name="${namespace}/bar_joint" type="fixed">
-  <parent link="${namespace}/base_link" />
-  <child link="${namespace}/bar" />
-</joint>
-<link name="${namespace}/bar">
-  <inertial>
-    <mass value="0.001" />
-    <xacro:box_inertia x="0.001" y="0.001" z="0.001" mass="0.001" />
-  </inertial>
-  <visual>
-    <geometry>
-        <mesh filename="package://rotors_description/meshes/techpod_X_flex/bar.stl" scale="1 1 1" />
-    </geometry>
-  </visual>
-</link>
-<gazebo reference="${namespace}/bar">
-  <material>Gazebo/Grey</material>
-</gazebo>
-<joint name="${namespace}/cover" type="fixed">
-  <parent link="${namespace}/base_link" />
-  <child link="${namespace}/cover" />
-</joint>
-<link name="${namespace}/cover">
-  <inertial>
-    <mass value="0.001" />
-    <xacro:box_inertia x="0.001" y="0.001" z="0.001" mass="0.001" />
-  </inertial>
-  <visual>
-    <geometry>
-        <mesh filename="package://rotors_description/meshes/techpod_X_flex/cover_hole.stl" scale="1 1 1" />
-    </geometry>
-  </visual>
-</link>
-<gazebo reference="${namespace}/cover">
-   <material>Gazebo/White</material>
-</gazebo>
-<joint name="${namespace}/motor_joint" type="fixed">
-  <parent link="${namespace}/base_link" />
-  <child link="${namespace}/motor" />
-</joint>
-<link name="${namespace}/motor">
-  <inertial>
-    <mass value="0.001" />
-    <xacro:box_inertia x="0.001" y="0.001" z="0.001" mass="0.001" />
-  </inertial>
-  <visual>
-    <geometry>
-        <mesh filename="package://rotors_description/meshes/techpod_X_flex/motor.stl" scale="1 1 1" />
-    </geometry>
-  </visual>
-</link>
-<gazebo reference="${namespace}/motor">
-  <material>Gazebo/Black</material>
-</gazebo>
-  <!-- Instantiate flexing wing segments -->
-  <xacro:airfoil_segment
-    robot_namespace="${namespace}"
-    segment_name="wl_1"
-    parent="${namespace}/base_link"
-    mass_segment="0.15"
-    k = "${k1}"
-    c = "${d1}"
-    color="${body_color}"
-    use_mesh_file="${use_mesh}"
-    mesh_file="package://rotors_description/meshes/techpod_X_flex/wing_l_1.stl"
-    segment_length="0.1"
-    segment_width="0.4"
-    segment_height="0.02">
-    <axis xyz="1 0 0" />   <!-- Joint axis -->
-    <origin xyz="0 0 0.162" rpy="0 0 0" />   <!-- Joint origin -->
-    <origin xyz="0 0.195 0" rpy="0 0 0" />       <!-- Inertia origin -->
-    <origin xyz="0 0 -0.162" rpy="0 0 0" />  <!-- Mesh origin -->
-    <xacro:insert_block name="aileron_inertia" />
-  </xacro:airfoil_segment>
-<gazebo reference="${namespace}/base_link">
-  <visual>
-    <plugin name='visual_plugin_base_link' filename='librotors_gazebo_template_visual_plugin.so'/>
-  </visual>
-</gazebo>
-<link name="${namespace}/payload_1">
-  <inertial>
-    <mass value="0.5" />
-    <xacro:sphere_inertia r="0.05" mass="0.5" />
-  </inertial>
-  <visual>
-    <origin xyz="0 0 0" rpy="0 1.5708 0" />
-    <geometry>
-        <cylinder length="0.25" radius="0.03"/>
-    </geometry>
-  </visual>
-  <collision>
-    <origin xyz="0 0 0" rpy="0 1.5708 0" />
-    <geometry>
-        <cylinder length="0.25" radius="0.03"/>
-    </geometry>
-  </collision>
-</link>
-<!--
-<joint name="${namespace}/payload_1_joint" type="revolute">
-  <parent link="${namespace}/wl_2" />
-  <child link="${namespace}/payload_1" />
-  <origin xyz="0.05 0 -0.1" rpy="0 0 0" />
-  <limit upper="0" lower="0" effort="5000" velocity="50"/>
-</joint>
--->
-<joint name="${namespace}/payload_1_joint" type="floating">
-  <parent link="${namespace}/wl_2" />
-  <child link="${namespace}/payload_1" />
-  <origin xyz="0.05 0 -0.1" rpy="0 0 0" />
-</joint>
-<gazebo reference="${namespace}/payload_1">
-  <visual>
-    <plugin name='visual_plugin_payload_1' filename='librotors_gazebo_template_visual_plugin.so'/>
-  </visual>
-  <material>Gazebo/Orange</material>
-  <mu1>0.2</mu1>
-  <mu2>0.2</mu2>
-  <kp>10000</kp>
-  <kd>1</kd>
-</gazebo>
-<gazebo>
-  <plugin filename="librotors_gazebo_payload_plugin.so" name="payload_plugin_1">
-    <robotNamespace>${namespace}</robotNamespace>
-    <joint>${namespace}/payload_1_joint</joint>
-    <payload>${namespace}/payload_1</payload>
-    <parent>${namespace}/wl_2</parent>
-    <hoistPosParent>0 -0.15 -0.07</hoistPosParent>
-    <hoistPosPayload>0 0 0</hoistPosPayload>
-    <dropTopic>drop_1</dropTopic>
-  </plugin>
-</gazebo>
-<gazebo>
-  <plugin filename="librotors_gazebo_aerodynamics_plugin.so" name="aerodynamics_plugin">
-    <robotNamespace>${namespace}</robotNamespace>
-    <linkName>${namespace}/wl_1</linkName>
-    <aeroForcesVis>aero_force_vis_wl1</aeroForcesVis>
-    <airfoil>
-      <segment name="WL1_1">
-        <forward>1 0 0</forward>
-        <upward>0 0 1</upward>
-        <cp>0 0.1 0</cp>
-        <seg_area>0.016</seg_area>
-        <seg_chord>0.16</seg_chord>
-        <aeroParamsYAML>${yaml_path}/airfoil_test.yaml</aeroParamsYAML>
-      </segment>
-      <segment name="WL1_2">
-        <forward>1 0 0</forward>
-        <upward>0 0 1</upward>
-        <cp>0.0 0.28 0</cp>
-        <seg_area>0.032</seg_area>
-        <seg_chord>0.16</seg_chord>
-        <aeroParamsYAML>${yaml_path}/airfoil_test.yaml</aeroParamsYAML>
-        <control>
-          <cs name="flap_left">
-              <controlJoint>${namespace}/flap_left_1_joint</controlJoint>
-              <fromTopic>true</fromTopic>
-              <csRefTopic>flap_l1_pos</csRefTopic>
-              <radToCLift>2</radToCLift>
-              <radToCDrag>0.0</radToCDrag>
-              <radToCPitch>0.0</radToCPitch>
-          </cs>
-        </control>
-      </segment>
-    </airfoil>
-  </plugin>
-</gazebo>
-  <xacro:angle_vane
-    robot_namespace="${namespace}"
-    vane_name="alpha_1"
-    type="alpha"
-    chord="0.02"
-    arm_cp="0.05"
-    mass_vane="0.02"
-    parent="${namespace}/wl_1"
-    color="Grey"
-    mesh_file="package://rotors_description/meshes/techpod_X_flex/flp_l_1.stl">
-    <origin xyz="0.15 0.35 0.05" rpy="0 0 0" />   <!-- Joint origin -->
-    <origin xyz="0 0 0" rpy="0 0 0" />       <!-- vis_coll origin -->
-    <xacro:box_inertia x="0.1" y="0.02" z="0.02" mass="0.02" />
-  </xacro:angle_vane>
-<gazebo>
-  <plugin filename="librotors_gazebo_vane_plugin.so" name="alpha_1_vane_plugin">
-    <robotNamespace>${namespace}</robotNamespace>
-    <vaneJoint>${namespace}/alpha_1_joint</vaneJoint>
-    <vaneTopic>alpha_1_vane_sensor</vaneTopic>
-  </plugin>
-</gazebo>
-<xacro:airfoil_segment
-  robot_namespace="${namespace}"
-  segment_name="wr_1"
-  parent="${namespace}/base_link"
-  mass_segment="0.15"
-  k = "${k1}"
-  c = "${d1}"
-  color="${body_color}"
-  use_mesh_file="${use_mesh}"
-  mesh_file="package://rotors_description/meshes/techpod_X_flex/wing_r_1.stl"
-  segment_length="0.1"
-  segment_width="0.4"
-  segment_height="0.02">
-  <axis xyz="1 0 0" />   <!-- Joint axis -->
-  <origin xyz="0 0 0.162" rpy="0 0 0" />   <!-- Joint origin -->
-  <origin xyz="0 -0.195 0" rpy="0 0 0" />       <!-- Inertia origin -->
-  <origin xyz="0 0 -0.162" rpy="0 0 0" />  <!-- Mesh origin -->
-  <xacro:insert_block name="aileron_inertia" />
-</xacro:airfoil_segment>
-<gazebo>
-  <plugin filename="librotors_gazebo_aerodynamics_plugin.so" name="aerodynamics_plugin">
-    <robotNamespace>${namespace}</robotNamespace>
-    <linkName>${namespace}/wr_1</linkName>
-    <aeroForcesVis>aero_force_vis_wr1</aeroForcesVis>
-    <airfoil>
-      <segment name="WR1_1">
-        <forward>1 0 0</forward>
-        <upward>0 0 1</upward>
-        <cp>0 -0.1 0</cp>
-        <seg_area>0.016</seg_area>
-        <seg_chord>0.16</seg_chord>
-        <aeroParamsYAML>${yaml_path}/airfoil_test.yaml</aeroParamsYAML>
-      </segment>
-      <segment name="WR1_2">
-        <forward>1 0 0</forward>
-        <upward>0 0 1</upward>
-        <cp>0.0 -0.28 0</cp>
-        <seg_area>0.032</seg_area>
-        <seg_chord>0.16</seg_chord>
-        <aeroParamsYAML>${yaml_path}/airfoil_test.yaml</aeroParamsYAML>
-        <control>
-          <cs name="flap_right">
-              <controlJoint>${namespace}/flap_right_1_joint</controlJoint>
-              <fromTopic>true</fromTopic>
-              <csRefTopic>flap_r1_pos</csRefTopic>
-              <radToCLift>2</radToCLift>
-              <radToCDrag>0.0</radToCDrag>
-              <radToCPitch>0.0</radToCPitch>
-          </cs>
-        </control>
-      </segment>
-    </airfoil>
-  </plugin>
-</gazebo>
-<xacro:angle_vane
-  robot_namespace="${namespace}"
-  vane_name="beta_1"
-  type="beta"
-  chord="0.02"
-  arm_cp="0.05"
-  mass_vane="0.02"
-  parent="${namespace}/wr_1"
-  color="Grey"
-  mesh_file="package://rotors_description/meshes/techpod_X_flex/flp_l_1.stl">
-  <origin xyz="0.15 -0.35 0.05" rpy="0 0 0" />   <!-- Joint origin -->
-  <origin xyz="0 0 0" rpy="0 0 0" />       <!-- vis_coll origin -->
-  <xacro:box_inertia x="0.1" y="0.02" z="0.02" mass="0.02" />
-</xacro:angle_vane>
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
File: rotors_description/urdf/techpod_X_flex_base.xacro (robot description, xacro)
@@ -12,5 +12,5 @@
   limitations under the License.
 -->
-<robot name="techpod_X" xmlns:xacro="http://ros.org/wiki/xacro">
+<robot name="techpod_X_flex" xmlns:xacro="http://ros.org/wiki/xacro">
   <xacro:include filename="$(find rotors_description)/urdf/component_snippets.xacro" />
   <!-- Instantiate fixed wing "mechanics" -->
@@ -18,10 +18,8 @@
   <!-- Mount an ADIS16448 IMU. -->
   <xacro:default_imu namespace="${namespace}" parent_link="${namespace}/base_link" />
-  <!-- -->
   <!-- Mount a GPS. -->
   <xacro:default_gps namespace="${namespace}" parent_link="${namespace}/base_link" >
     <origin xyz="0 0 0" rpy="0 0 0" />
   </xacro:default_gps>
-  <!-- -->
   <!-- Mount a magnetometer. note: mavlink interface already does this based on position from gps-->
   <!--
@@ -65,3 +63,19 @@
     <origin xyz="0.35 0 0.11" rpy="0 0.2 0" />
   </xacro:default_camera>
+  <!--
+  <xacro:default_camera
+    namespace="${namespace}"
+    parent_link="${namespace}/base_link"
+    camera_suffix="cam_aft">
+    <origin xyz="-0.7 0 0.02" rpy="0 0.4 3.14" />
+  </xacro:default_camera>
+  -->
+  <!--
+  <xacro:default_camera
+    namespace="${namespace}"
+    parent_link="${namespace}/payload_1"
+    camera_suffix="cam_payload">
+    <origin xyz="0.125 0 0" rpy="0 0 0" />
+  </xacro:default_camera>
+  -->
 </robot>
