Commit message: Adding origin tag to default IMU
- Adjusting IMU and GPS positions in all techpod models

File: rotors_description/urdf/component_snippets.xacro (robot description, xacro)
@@ -1018,5 +1018,5 @@
     </xacro:odometry_plugin_macro>
   </xacro:macro>
-  <xacro:macro name="default_imu" params="namespace parent_link">
+  <xacro:macro name="default_imu" params="namespace parent_link *origin">
     <!-- ADIS16448 IMU. -->
     <xacro:imu_plugin_macro
@@ -1035,5 +1035,5 @@
       accelerometer_turn_on_bias_sigma="0.1960">
       <xacro:cube_inertia l="0.02" mass="0.015" />
-      <origin xyz="0 0 0" rpy="0 0 0" />
+      <xacro:insert_block name="origin" />
     </xacro:imu_plugin_macro>
   </xacro:macro>

File: rotors_description/urdf/fixed_wing_X_base.xacro (robot description, xacro)
@@ -62,64 +62,64 @@
     </gazebo>
   </xacro:macro>
-<!-- Airfoil segment joint, link and plugin -->
-<xacro:macro name="airfoil_segment"
-  params="robot_namespace segment_name parent mass_segment do_flex k c color use_mesh_file mesh_file segment_length segment_width
-    segment_height *axis *joint_origin *inertia_origin *vis_coll_origin *inertia ">
-  <xacro:if value="${do_flex}">
-    <joint name="${robot_namespace}/${segment_name}_joint" type="revolute">
-      <xacro:insert_block name="joint_origin" />
-      <xacro:insert_block name="axis" />
-      <parent link="${parent}" />
-      <child link="${robot_namespace}/${segment_name}"/>
-      <limit upper="0.17" lower="-0.17" effort="5000" velocity="50"/>
-      <dynamics damping="${c}"/>
-    </joint>
-    <gazebo reference="${robot_namespace}/${segment_name}_joint">
-      <implicitSpringDamper>true</implicitSpringDamper>
-      <springStiffness>${k}</springStiffness>
-    </gazebo>
-  </xacro:if>
-  <xacro:unless value="${do_flex}">
-    <joint name="${robot_namespace}/${segment_name}_joint" type="revolute">
-      <xacro:insert_block name="joint_origin" />
-      <xacro:insert_block name="axis" />
-      <parent link="${parent}" />
-      <child link="${robot_namespace}/${segment_name}"/>
-      <limit upper="0" lower="-0" effort="5000" velocity="50"/>
-    </joint>
-  </xacro:unless>
-  <link name="${robot_namespace}/${segment_name}">
-    <inertial>
-      <xacro:insert_block name="inertia_origin" />
-      <mass value="${mass_segment}" />
-      <xacro:box_inertia x="${segment_length}" y="${segment_width}" z="${segment_height}" mass="${mass_segment}" />
-    </inertial>
-    <visual>
-      <xacro:insert_block name="vis_coll_origin" />
-      <geometry>
-        <xacro:if value="${use_mesh_file}">
-          <mesh filename="${mesh_file}" scale="1 1 1" />
-        </xacro:if>
-        <xacro:unless value="${use_mesh_file}">
-          <box size="${segment_length} ${segment_width} ${segment_height}" />
-        </xacro:unless>
-      </geometry>
-    </visual>
-    <collision>
-      <xacro:insert_block name="vis_coll_origin" />
-      <geometry>
-        <xacro:if value="${use_mesh_file}">
-          <mesh filename="${mesh_file}" scale="1 1 1" />
-        </xacro:if>
-        <xacro:unless value="${use_mesh_file}">
-          <box size="${segment_length} ${segment_width} ${segment_height}" />
-        </xacro:unless>
-      </geometry>
-    </collision>
-  </link>
-  <gazebo reference="${robot_namespace}/${segment_name}">
-    <material>Gazebo/${color}</material>
-  </gazebo>
-</xacro:macro>
+  <!-- Airfoil segment joint, link and plugin -->
+  <xacro:macro name="airfoil_segment"
+    params="robot_namespace segment_name parent mass_segment do_flex k c color use_mesh_file mesh_file segment_length segment_width
+      segment_height *axis *joint_origin *inertia_origin *vis_coll_origin *inertia ">
+    <xacro:if value="${do_flex}">
+      <joint name="${robot_namespace}/${segment_name}_joint" type="revolute">
+        <xacro:insert_block name="joint_origin" />
+        <xacro:insert_block name="axis" />
+        <parent link="${parent}" />
+        <child link="${robot_namespace}/${segment_name}"/>
+        <limit upper="0.17" lower="-0.17" effort="5000" velocity="50"/>
+        <dynamics damping="${c}"/>
+      </joint>
+      <gazebo reference="${robot_namespace}/${segment_name}_joint">
+        <implicitSpringDamper>true</implicitSpringDamper>
+        <springStiffness>${k}</springStiffness>
+      </gazebo>
+    </xacro:if>
+    <xacro:unless value="${do_flex}">
+      <joint name="${robot_namespace}/${segment_name}_joint" type="revolute">
+        <xacro:insert_block name="joint_origin" />
+        <xacro:insert_block name="axis" />
+        <parent link="${parent}" />
+        <child link="${robot_namespace}/${segment_name}"/>
+        <limit upper="0" lower="-0" effort="5000" velocity="50"/>
+      </joint>
+    </xacro:unless>
+    <link name="${robot_namespace}/${segment_name}">
+      <inertial>
+        <xacro:insert_block name="inertia_origin" />
+        <mass value="${mass_segment}" />
+        <xacro:box_inertia x="${segment_length}" y="${segment_width}" z="${segment_height}" mass="${mass_segment}" />
+      </inertial>
+      <visual>
+        <xacro:insert_block name="vis_coll_origin" />
+        <geometry>
+          <xacro:if value="${use_mesh_file}">
+            <mesh filename="${mesh_file}" scale="1 1 1" />
+          </xacro:if>
+          <xacro:unless value="${use_mesh_file}">
+            <box size="${segment_length} ${segment_width} ${segment_height}" />
+          </xacro:unless>
+        </geometry>
+      </visual>
+      <collision>
+        <xacro:insert_block name="vis_coll_origin" />
+        <geometry>
+          <xacro:if value="${use_mesh_file}">
+            <mesh filename="${mesh_file}" scale="1 1 1" />
+          </xacro:if>
+          <xacro:unless value="${use_mesh_file}">
+            <box size="${segment_length} ${segment_width} ${segment_height}" />
+          </xacro:unless>
+        </geometry>
+      </collision>
+    </link>
+    <gazebo reference="${robot_namespace}/${segment_name}">
+      <material>Gazebo/${color}</material>
+    </gazebo>
+  </xacro:macro>
   <!-- Control surface joint and link -->
   <xacro:macro name="control_surface"
@@ -213,93 +213,93 @@
     </gazebo>
   </xacro:macro>
-<!-- Aerodyn. angle vane -->
-<xacro:macro name="angle_vane"
-  params="robot_namespace vane_name type chord arm_cp parent wind_topic mass_vane
-          color mesh_file *joint_origin *vis_coll_origin *inertia">
-  <joint name="${robot_namespace}/${vane_name}_joint" type="continuous">
-    <xacro:insert_block name="joint_origin" />
+  <!-- Aerodyn. angle vane -->
+  <xacro:macro name="angle_vane"
+    params="robot_namespace vane_name type chord arm_cp parent wind_topic mass_vane
+            color mesh_file *joint_origin *vis_coll_origin *inertia">
+    <joint name="${robot_namespace}/${vane_name}_joint" type="continuous">
+      <xacro:insert_block name="joint_origin" />
+      <xacro:if value="${type=='alpha'}">
+         <axis xyz="0 1 0" />
+       </xacro:if>
+       <xacro:if value="${type=='beta'}">
+         <axis xyz="0 0 -1" />
+       </xacro:if>
+       <parent link="${parent}" />
+       <child link="${robot_namespace}/${vane_name}" />
+       <dynamics friction="0" damping="0.001"/>
+    </joint>
+    <link name="${robot_namespace}/${vane_name}">
+      <inertial>
+        <mass value="${mass_vane}" />
+        <xacro:insert_block name="inertia" />
+      </inertial>
+      <visual>
+        <xacro:insert_block name="vis_coll_origin" />
+        <geometry>
+          <box size="0.1 0.003 0.003" />
+        </geometry>
+      </visual>
+      <visual>
+        <xacro:if value="${type=='alpha'}">
+          <origin xyz="-0.04 0.02 0" rpy="0 0 0" />
+          <geometry>
+            <box size="0.02 0.04 0.002" />
+          </geometry>
+        </xacro:if>
+        <xacro:if value="${type=='beta'}">
+          <origin xyz="-0.04 0 0.02" rpy="0 0 0" />
+          <geometry>
+            <box size="0.02 0.002 0.04" />
+          </geometry>
+        </xacro:if>
+      </visual>
+    </link>
+    <gazebo reference="${robot_namespace}/${vane_name}">
+      <material>Gazebo/${color}</material>
+    </gazebo>
     <xacro:if value="${type=='alpha'}">
-       <axis xyz="0 1 0" />
-     </xacro:if>
-     <xacro:if value="${type=='beta'}">
-       <axis xyz="0 0 -1" />
-     </xacro:if>
-     <parent link="${parent}" />
-     <child link="${robot_namespace}/${vane_name}" />
-     <dynamics friction="0" damping="0.001"/>
-  </joint>
-  <link name="${robot_namespace}/${vane_name}">
-    <inertial>
-      <mass value="${mass_vane}" />
-      <xacro:insert_block name="inertia" />
-    </inertial>
-    <visual>
-      <xacro:insert_block name="vis_coll_origin" />
-      <geometry>
-        <box size="0.1 0.003 0.003" />
-      </geometry>
-    </visual>
-    <visual>
-      <xacro:if value="${type=='alpha'}">
-        <origin xyz="-0.04 0.02 0" rpy="0 0 0" />
-        <geometry>
-          <box size="0.02 0.04 0.002" />
-        </geometry>
-      </xacro:if>
-      <xacro:if value="${type=='beta'}">
-        <origin xyz="-0.04 0 0.02" rpy="0 0 0" />
-        <geometry>
-          <box size="0.02 0.002 0.04" />
-        </geometry>
-      </xacro:if>
-    </visual>
-  </link>
-  <gazebo reference="${robot_namespace}/${vane_name}">
-    <material>Gazebo/${color}</material>
-  </gazebo>
-  <xacro:if value="${type=='alpha'}">
-   <gazebo>
-     <plugin filename="librotors_gazebo_aerodynamics_plugin.so" name="aerodynamics_plugin">
-       <robotNamespace>${namespace}</robotNamespace>
-       <linkName>${robot_namespace}/${vane_name}</linkName>
-        <aeroForcesVis>aero_force_vis_${vane_name}</aeroForcesVis>
-        <airfoil>
-          <segment name="alpha_vane">
-            <forward>1 0 0</forward>
-            <upward>0 0 1</upward>
-            <cp>${-arm_cp} 0 0</cp>
-            <seg_area>${2*chord*chord}</seg_area>
-            <seg_chord>${chord}</seg_chord>
-            <aeroParamsYAML>${yaml_path}/airfoil_test_2.yaml</aeroParamsYAML>
-            <wind name="wind">
-              <topic>${wind_topic}</topic>
-            </wind>
-          </segment>
-        </airfoil>
-      </plugin>
-    </gazebo>
-  </xacro:if>
-  <xacro:if value="${type=='beta'}">
-   <gazebo>
-     <plugin filename="librotors_gazebo_aerodynamics_plugin.so" name="aerodynamics_plugin">
-       <robotNamespace>${namespace}</robotNamespace>
-       <linkName>${robot_namespace}/${vane_name}</linkName>
-        <aeroForcesVis>aero_force_vis_${vane_name}</aeroForcesVis>
-        <airfoil>
-          <segment name="beta_vane">
-            <forward>1 0 0</forward>
-            <upward>0 -1 0</upward>
-            <cp>${-arm_cp} 0 0</cp>
-            <seg_area>${2*chord*chord}</seg_area>
-            <seg_chord>${chord}</seg_chord>
-            <aeroParamsYAML>${yaml_path}/airfoil_test_2.yaml</aeroParamsYAML>
-            <wind name="wind">
-              <topic>${wind_topic}</topic>
-            </wind>
-          </segment>
-        </airfoil>
-      </plugin>
-    </gazebo>
-  </xacro:if>
-</xacro:macro>
+     <gazebo>
+       <plugin filename="librotors_gazebo_aerodynamics_plugin.so" name="aerodynamics_plugin">
+         <robotNamespace>${namespace}</robotNamespace>
+         <linkName>${robot_namespace}/${vane_name}</linkName>
+          <aeroForcesVis>aero_force_vis_${vane_name}</aeroForcesVis>
+          <airfoil>
+            <segment name="alpha_vane">
+              <forward>1 0 0</forward>
+              <upward>0 0 1</upward>
+              <cp>${-arm_cp} 0 0</cp>
+              <seg_area>${2*chord*chord}</seg_area>
+              <seg_chord>${chord}</seg_chord>
+              <aeroParamsYAML>${yaml_path}/airfoil_test_2.yaml</aeroParamsYAML>
+              <wind name="wind">
+                <topic>${wind_topic}</topic>
+              </wind>
+            </segment>
+          </airfoil>
+        </plugin>
+      </gazebo>
+    </xacro:if>
+    <xacro:if value="${type=='beta'}">
+     <gazebo>
+       <plugin filename="librotors_gazebo_aerodynamics_plugin.so" name="aerodynamics_plugin">
+         <robotNamespace>${namespace}</robotNamespace>
+         <linkName>${robot_namespace}/${vane_name}</linkName>
+          <aeroForcesVis>aero_force_vis_${vane_name}</aeroForcesVis>
+          <airfoil>
+            <segment name="beta_vane">
+              <forward>1 0 0</forward>
+              <upward>0 -1 0</upward>
+              <cp>${-arm_cp} 0 0</cp>
+              <seg_area>${2*chord*chord}</seg_area>
+              <seg_chord>${chord}</seg_chord>
+              <aeroParamsYAML>${yaml_path}/airfoil_test_2.yaml</aeroParamsYAML>
+              <wind name="wind">
+                <topic>${wind_topic}</topic>
+              </wind>
+            </segment>
+          </airfoil>
+        </plugin>
+      </gazebo>
+    </xacro:if>
+  </xacro:macro>
 </robot>

File: rotors_description/urdf/techpod_TJ_base.xacro (robot description, xacro)
@@ -17,8 +17,10 @@
   <xacro:include filename="$(find rotors_description)/urdf/techpod_TJ.xacro" />
   <!-- Mount an ADIS16448 IMU. -->
-  <xacro:default_imu namespace="${namespace}" parent_link="${namespace}/base_link" />
+  <xacro:default_imu namespace="${namespace}" parent_link="${namespace}/base_link" >
+    <origin xyz="0.3 -0.01 0.023" rpy="0 0 0" />
+  </xacro:default_imu>
   <!-- Mount a GPS. -->
   <xacro:default_gps namespace="${namespace}" parent_link="${namespace}/base_link" >
-    <origin xyz="0 0 0" rpy="0 0 0" />
+    <origin xyz="0.22 0 0.143" rpy="0 0 0" />
   </xacro:default_gps>
   <xacro:default_camera

File: rotors_description/urdf/techpod_TJ_flex_base.xacro (robot description, xacro)
@@ -17,11 +17,11 @@
   <xacro:include filename="$(find rotors_description)/urdf/techpod_TJ_flex.xacro" />
   <!-- Mount an ADIS16448 IMU. -->
-  <xacro:default_imu namespace="${namespace}" parent_link="${namespace}/base_link" />
-  <!---->
+  <xacro:default_imu namespace="${namespace}" parent_link="${namespace}/base_link" >
+    <origin xyz="0.14 -0.01 0.07" rpy="0 0 0" />
+  </xacro:default_imu>
   <!-- Mount a GPS. -->
   <xacro:default_gps namespace="${namespace}" parent_link="${namespace}/base_link" >
-    <origin xyz="0 0 0" rpy="0 0 0" />
+    <origin xyz="0.06 0 0.19" rpy="0 0 0" />
   </xacro:default_gps>
-  <!---->
   <!-- Mount a magnetometer. note: mavlink interface already does this based on position from gps-->
   <!--
@@ -32,5 +32,4 @@
   <xacro:default_pressure_sensor namespace="${namespace}" parent_link="${namespace}/base_link" />
   -->
-  <!--
   <xacro:default_camera
     namespace="${namespace}"
@@ -45,9 +44,9 @@
     <origin xyz="0.21 -0.045 0.145" rpy="0 -0.1 -2.2" />
   </xacro:default_camera>
-  -->
+  <!---->
   <xacro:camera_macro_2
     namespace="${namespace}"
     parent_link="${namespace}/base_link"
-    camera_suffix="fpv_lowres"
+    camera_suffix="3pv_lowres"
     frame_rate="60"
     horizontal_fov="1.3962634"
@@ -60,10 +59,9 @@
     noise_stddev="0.007"
     mass = "0.01"
-    enable_visual="true">
+    enable_visual="false">
     <mesh filename="package://rotors_description/meshes/vi_camera.dae" scale="1 1 1" />
     <xacro:cube_inertia l="0.02" mass="0.01" />
-    <origin xyz="0.34 0 0.135" rpy="0 0.2 0" />
+    <origin xyz="-2 0 0.5" rpy="0 0.2 0" />
   </xacro:camera_macro_2>
-  <!---->
   <xacro:asl_mono_vi_1
     namespace="${namespace}"
@@ -111,51 +109,4 @@
     <origin xyz="-0.0083 -0.0177 -0.0469" rpy="-3.1363 -0.0648 1.5500" />
   </xacro:asl_mono_vi_1>
-<!--
-<xacro:asl_mono_vi_1
-  namespace="${namespace}"
-  parent_link="${namespace}/base_link"
-  suffix="center"
-  fps="30"
-  h_fov="1.3514"
-  imu_topic="adis/data_raw"
-  acc_nd="0.0"
-  acc_rw="0.0"
-  gyr_nd="0.0"
-  gyr_rw="0.0">
-  <origin xyz="0.35 0 0.11" rpy="0 0.3 0" />
-  <origin xyz="-0.0014 0.0146 -0.1175" rpy="-3.1228 -1.1414 -1.6129" />
-  <origin xyz="-0.0014 0.0146 -0.1175" rpy="-3.1228 -1.1414 -1.6129" />
-</xacro:asl_mono_vi_1>
-<xacro:asl_mono_vi_1
-  namespace="${namespace}"
-  parent_link="${namespace}/wl_3"
-  suffix="left"
-  fps="30"
-  h_fov="1.3560"
-  imu_topic="camImu0/data_raw"
-  acc_nd="0.0"
-  acc_rw="0.0"
-  gyr_nd="0.0"
-  gyr_rw="0.0">
-  <origin xyz="0.05 0.38 0.025" rpy="0 0.3 0" />
-  <origin xyz="-0.0264 0.0061 -0.0331" rpy="3.1298 0.0029 1.5626" />
-  <origin xyz="-0.0264 0.0061 -0.0331" rpy="3.1298 0.0029 1.5626" />
-</xacro:asl_mono_vi_1>
-<xacro:asl_mono_vi_1
-  namespace="${namespace}"
-  parent_link="${namespace}/wr_3"
-  suffix="right"
-  fps="30"
-  h_fov="1.3626"
-  imu_topic="camImu1/data_raw"
-  acc_nd="0.0"
-  acc_rw="0.0"
-  gyr_nd="0.0"
-  gyr_rw="0.0">
-  <origin xyz="0.05 -0.38 0.025" rpy="0 0.3 0" />
-  <origin xyz="-0.0083 -0.0177 -0.0469" rpy="-3.1363 -0.0648 1.5500" />
-  <origin xyz="-0.0083 -0.0177 -0.0469" rpy="-3.1363 -0.0648 1.5500" />
-</xacro:asl_mono_vi_1>
--->
   <!--
   <xacro:default_camera

File: rotors_description/urdf/techpod_X_base.xacro (robot description, xacro)
@@ -17,8 +17,10 @@
   <xacro:include filename="$(find rotors_description)/urdf/techpod_X.xacro" />
   <!-- Mount an ADIS16448 IMU. -->
-  <xacro:default_imu namespace="${namespace}" parent_link="${namespace}/base_link" />
+  <xacro:default_imu namespace="${namespace}" parent_link="${namespace}/base_link" >
+    <origin xyz="0.3 -0.01 0.023" rpy="0 0 0" />
+  </xacro:default_imu>
   <!-- Mount a GPS. -->
   <xacro:default_gps namespace="${namespace}" parent_link="${namespace}/base_link" >
-    <origin xyz="0 0 0" rpy="0 0 0" />
+    <origin xyz="0.22 0 0.143" rpy="0 0 0" />
   </xacro:default_gps>
   <!-- Mount a magnetometer. note: mavlink interface already does this based on position from gps-->

File: rotors_description/urdf/techpod_X_flex_base.xacro (robot description, xacro)
@@ -17,8 +17,10 @@
   <xacro:include filename="$(find rotors_description)/urdf/techpod_X_flex.xacro" />
   <!-- Mount an ADIS16448 IMU. -->
-  <xacro:default_imu namespace="${namespace}" parent_link="${namespace}/base_link" />
+  <xacro:default_imu namespace="${namespace}" parent_link="${namespace}/base_link" >
+    <origin xyz="0.14 -0.01 0.07" rpy="0 0 0" />
+  </xacro:default_imu>
   <!-- Mount a GPS. -->
   <xacro:default_gps namespace="${namespace}" parent_link="${namespace}/base_link" >
-    <origin xyz="0 0 0" rpy="0 0 0" />
+    <origin xyz="0.06 0 0.19" rpy="0 0 0" />
   </xacro:default_gps>
   <!-- Mount a magnetometer. note: mavlink interface already does this based on position from gps-->

Commit message: Updated imu, motor_constant, odometry_update rate so that it is more close to the reality.

File: rotors_description/urdf/component_snippets.xacro (robot description, xacro)
@@ -819,5 +819,5 @@
       imu_topic="imu"
       mass_imu_sensor="0.015"
-      gyroscope_noise_density="0.0003394"
+      gyroscope_noise_density="0.00005366563"
       gyroscope_random_walk="0.000038785"
       gyroscope_bias_correlation_time="1000.0"

File: rotors_description/urdf/overactuated_base.xacro (robot description, xacro)
@@ -197,4 +197,8 @@
         <motorPositionPubTopic>/tilt_motor_${motor_number}/position</motorPositionPubTopic>
         <motorForcePubTopic>/tilt_motor_${motor_number}/force</motorForcePubTopic>
+        <!-- Relationship between the p, d gain and the closed-loop dynamics behaviour of the system:
+        It behaves like a second-order system in the frequency domain: Y(s) = U(s)*(ds + p)/(Is**2 + ds + p)
+        Y(s) is the Laplace transform of the actual tilt motor angle and U(s) is the one of the tilt motor angle command, p and d are the gains, I is the inertia of the link.
+         -->
         <joint_control_pid>
             <p>0.11</p>

File: rotors_description/urdf/voliro.xacro (robot description, xacro)
@@ -35,6 +35,6 @@
     <xacro:property name="rotor_offset_top" value="0.060"/>    <!-- [m] -->
     <xacro:property name="radius_rotor" value="0.1143"/>    <!-- [m] -->
-    <xacro:property name="motor_constant" value="${8.54858e-06}"/>    <!-- [kg m/s^2] -->
-    <xacro:property name="motor_constant_lower" value="${8.54858e-06}"/>    <!-- [kg m/s^2] -->
+    <xacro:property name="motor_constant" value="${7.24858e-06}"/>    <!-- [kg m/s^2] -->
+    <xacro:property name="motor_constant_lower" value="${7.24858e-06}"/>    <!-- [kg m/s^2] -->
     <xacro:property name="moment_constant" value="0.015"/>    <!-- [m] -->
     <xacro:property name="moment_constant_lower" value="0.005"/>    <!-- [m] -->
