Commit message: Miscellaneous, mostly refactoring
- techpod_TJ_flex: Refactoring
- lidar plugin: Publish to custom topic if desired + info printing
- fw_playground: Minor refactoring
- fixed_wing_X_base: Minor refactoring, get rid of unused arguments of vane macro
- component snippets: lidar_plugin_macro, ideal_imu macro, default_odometry macro, default_lidar macro, asl_mono_vi_1 odometry topic renaming
- rope.xacro: Adding prefixes to links
- inertias.xacro: all kind of inertia macros...

File: rotors_description/urdf/component_snippets.xacro (robot description, xacro)
@@ -598,4 +598,62 @@
     </gazebo>
   </xacro:macro>
+  <!-- Macro to add a single-ray LIDAR. -->
+  <xacro:macro name="lidar_plugin_macro"
+    params="namespace lidar_suffix mass_lidar_sensor
+            parent_link lidar_topic n_hrz n_vrt
+            rng_min rng_max ang_min_hrz ang_max_hrz
+            ang_min_vrt ang_max_vrt noise_std *inertia *origin">
+    <!-- LIDAR link -->
+    <link name="${namespace}/lidar${lidar_suffix}_link">
+      <inertial>
+        <xacro:insert_block name="inertia" />
+        <mass value="${mass_lidar_sensor}" />  <!-- [kg] -->
+        <origin xyz="0 0 0" rpy="0 0 0" />
+      </inertial>
+    </link>
+    <!-- LIDAR joint -->
+    <joint name="${namespace}/lidar${lidar_suffix}_joint" type="revolute">
+      <xacro:insert_block name="origin" />
+      <parent link="${parent_link}" />
+      <child link="${namespace}/lidar${lidar_suffix}_link" />
+      <limit upper="0" lower="0" effort="0" velocity="0" />
+    </joint>
+    <gazebo reference="${namespace}/lidar${lidar_suffix}_link">
+      <sensor type="ray" name="${namespace}_lidar${lidar_suffix}">
+        <pose>0 0 0 0 0 0</pose>
+        <visualize>1</visualize>
+        <always_on>1</always_on>
+        <ray>
+          <scan>
+            <horizontal>
+              <samples>${n_hrz}</samples>
+              <resolution>1</resolution>
+              <min_angle>${ang_min_hrz}</min_angle>
+              <max_angle>${ang_max_hrz}</max_angle>
+            </horizontal>
+            <vertical>
+              <samples>${n_vrt}</samples>
+              <resolution>1</resolution>
+              <min_angle>${ang_min_vrt}</min_angle>
+              <max_angle>${ang_max_vrt}</max_angle>
+            </vertical>
+          </scan>
+          <range>
+            <min>${rng_min}</min>
+            <max>${rng_max}</max>
+          </range>
+          <noise>
+            <type>gaussian</type>
+            <mean>0</mean>
+            <stddev>${noise_std}</stddev>
+          </noise>
+        </ray>
+        <plugin filename="librotors_gazebo_lidar_plugin.so" name="rotors_gazebo_lidar${lidar_suffix}_plugin">
+          <robotNamespace>${namespace}</robotNamespace>
+          <lidarTopic>${lidar_topic}</lidarTopic>
+        </plugin>
+      </sensor>
+    </gazebo>
+  </xacro:macro>
   <!-- Macro to add a magnetometer. -->
   <xacro:macro name="magnetometer_plugin_macro"
@@ -942,7 +1000,7 @@
       parent_link="${namespace}/camera_${suffix}_optical_link"
       pose_topic="cam_${suffix}/pose"
-      pose_with_covariance_topic="t1"
-      position_topic="t2"
-      transform_topic="t3"
+      pose_with_covariance_topic="cam_${suffix}/t1"
+      position_topic="cam_${suffix}/t2"
+      transform_topic="cam_${suffix}/t3"
       odometry_topic="cam_${suffix}/odometry"
       parent_frame_id="world"
@@ -1038,4 +1096,23 @@
     </xacro:imu_plugin_macro>
   </xacro:macro>
+  <xacro:macro name="ideal_imu" params="namespace parent_link *origin">
+    <xacro:imu_plugin_macro
+      namespace="${namespace}"
+      imu_suffix=""
+      parent_link="${parent_link}"
+      imu_topic="imu"
+      mass_imu_sensor="0.015"
+      gyroscope_noise_density="0.0"
+      gyroscope_random_walk="0.0"
+      gyroscope_bias_correlation_time="10000.0"
+      gyroscope_turn_on_bias_sigma="0.0"
+      accelerometer_noise_density="0.0"
+      accelerometer_random_walk="0.0"
+      accelerometer_bias_correlation_time="10000.0"
+      accelerometer_turn_on_bias_sigma="0.0">
+      <xacro:cube_inertia l="0.02" mass="0.015" />
+      <xacro:insert_block name="origin" />
+    </xacro:imu_plugin_macro>
+  </xacro:macro>
   <xacro:macro name="default_camera" params="namespace parent_link camera_suffix *origin">
     <xacro:camera_macro_2
@@ -1092,4 +1169,35 @@
     </xacro:gps_plugin_macro>
   </xacro:macro>
+  <xacro:macro name="default_odometry" params="namespace parent_link">
+    <xacro:odometry_plugin_macro
+      namespace="${namespace}"
+      odometry_sensor_suffix="gt"
+      parent_link="${parent_link}"
+      pose_topic="ground_truth/pose"
+      pose_with_covariance_topic="ground_truth/pose_with_covariance"
+      position_topic="ground_truth/position"
+      transform_topic="ground_truth/transform"
+      odometry_topic="ground_truth/odometry"
+      parent_frame_id="world"
+      child_frame_id="${namespace}/base_link"
+      mass_odometry_sensor="0.00001"
+      measurement_divisor="1"
+      measurement_delay="0"
+      unknown_delay="0.0"
+      noise_normal_position="0 0 0"
+      noise_normal_quaternion="0 0 0"
+      noise_normal_linear_velocity="0 0 0"
+      noise_normal_angular_velocity="0 0 0"
+      noise_uniform_position="0 0 0"
+      noise_uniform_quaternion="0 0 0"
+      noise_uniform_linear_velocity="0 0 0"
+      noise_uniform_angular_velocity="0 0 0"
+      enable_odometry_map="false"
+      odometry_map=""
+      image_scale="">
+      <xacro:cube_inertia l="0.001" mass="0.00001" /> <!-- [kg m^2] [kg m^2] [kg m^2] [kg m^2] [kg m^2] [kg m^2] -->
+      <origin xyz="0.0 0.0 0.0" rpy="0.0 0.0 0.0" />
+    </xacro:odometry_plugin_macro>
+  </xacro:macro>
   <xacro:macro name="default_magnetometer" params="namespace parent_link">
     <!-- ADIS16448 Magnetometer. -->
@@ -1139,3 +1247,23 @@
     </xacro:mavlink_interface_macro>
   </xacro:macro>
+  <xacro:macro name="default_lidar" params="namespace parent_link *origin">
+    <xacro:lidar_plugin_macro
+      namespace="${namespace}"
+      lidar_suffix=""
+      mass_lidar_sensor="0.05"
+      parent_link="${parent_link}"
+      lidar_topic="lidar_lite_v3"
+      n_hrz="1"
+      n_vrt="1"
+      rng_min="0.05"
+      rng_max="40"
+      ang_min_hrz="0.01"
+      ang_max_hrz="-0.01"
+      ang_min_vrt="0.01"
+      ang_max_vrt="-0.01"
+      noise_std="0.015">
+      <xacro:cube_inertia l="0.02" mass="0.05" />
+      <xacro:insert_block name="origin" />
+    </xacro:lidar_plugin_macro>
+  </xacro:macro>
 </robot>

File: rotors_description/urdf/fixed_wing_X_base.xacro (robot description, xacro)
@@ -216,5 +216,5 @@
   <xacro:macro name="angle_vane"
     params="robot_namespace vane_name type chord arm_cp parent wind_topic mass_vane
-            color mesh_file *joint_origin *vis_coll_origin *inertia">
+            color *joint_origin *inertia">
     <joint name="${robot_namespace}/${vane_name}_joint" type="continuous">
       <xacro:insert_block name="joint_origin" />
@@ -227,5 +227,5 @@
        <parent link="${parent}" />
        <child link="${robot_namespace}/${vane_name}" />
-       <dynamics friction="0" damping="0.001"/>
+       <dynamics friction="0" damping="0.00001"/>
     </joint>
     <link name="${robot_namespace}/${vane_name}">
@@ -235,5 +235,4 @@
       </inertial>
       <visual>
-        <xacro:insert_block name="vis_coll_origin" />
         <geometry>
           <box size="0.1 0.003 0.003" />

File: rotors_description/urdf/rope.xacro (robot description, xacro)
@@ -26,8 +26,8 @@
   </xacro:macro>
   <!-- Macro for adding a rope -->
-  <xacro:macro name="rope" params="n length dia mass damping parent color *joint_origin">
+  <xacro:macro name="rope" params="n length dia mass damping parent color prefix *joint_origin">
        <xacro:property name="seg_len" value="${length/n}"/>
        <xacro:property name="seg_mass" value="${mass/n}"/>
-       <link name="rope_seg_${n-1}">
+       <link name="${prefix}_rope_seg_${n-1}">
          <inertial>
            <origin xyz="0 0 ${seg_len/2}" rpy="0 0 0" />
@@ -45,6 +45,6 @@
           <plugin filename="librotors_gazebo_aerodynamics_plugin.so" name="aerodynamics_plugin">
              <robotNamespace></robotNamespace>
-             <linkName>rope_seg_${n-1}</linkName>
-             <aeroForcesVis>aero_force_rope_${n-1}</aeroForcesVis>
+             <linkName>${prefix}_rope_seg_${n-1}</linkName>
+             <aeroForcesVis>${prefix}_aero_force_rope_${n-1}</aeroForcesVis>
              <body>
                 <element>
@@ -59,22 +59,23 @@
           </plugin>
        </gazebo>
-       <gazebo reference="rope_seg_${n-1}">
+       <gazebo reference="${prefix}_rope_seg_${n-1}">
          <material>Gazebo/${color}</material>
        </gazebo>
        <xacro:rope_joint
          parent="${parent}"
-         child="rope_seg_${n-1}"
+         child="${prefix}_rope_seg_${n-1}"
          name="p_${n-1}"
-         c="${damping}">
+         c="${damping}"
+         prefix="${prefix}">
          <xacro:insert_block name="joint_origin" />
        </xacro:rope_joint>
        <xacro:if value="${n-1}">
-          <xacro:add_seg n="${n-2}" dia="${dia}" seg_len="${seg_len}" seg_mass="${seg_mass}" color="${color}" damping="${damping}" parent="rope_seg_${n-1}"/>
+          <xacro:add_seg n="${n-2}" dia="${dia}" seg_len="${seg_len}" seg_mass="${seg_mass}" color="${color}" damping="${damping}" parent="rope_seg_${n-1}" prefix="${prefix}"/>
        </xacro:if>
        <!-- add payload -->
-       <link name="rope_payload">
+       <link name="${prefix}_rope_payload">
          <inertial>
            <origin xyz="0 0 0" rpy="0 0 0" />
-           <mass value="0.2" />
+           <mass value="0.1" />
            <xacro:sphere_inertia r="0.1" mass="0.2"/>
          </inertial>
@@ -92,5 +93,5 @@
          </collision>
        </link>
-       <gazebo reference="rope_payload">
+       <gazebo reference="${prefix}_rope_payload">
           <visual>
              <plugin name="visual_plugin_rope_payload" filename="librotors_gazebo_template_visual_plugin.so" />
@@ -105,6 +106,6 @@
           <plugin filename="librotors_gazebo_aerodynamics_plugin.so" name="aerodynamics_plugin">
              <robotNamespace></robotNamespace>
-             <linkName>rope_payload</linkName>
-             <aeroForcesVis>aero_force_rope_payload</aeroForcesVis>
+             <linkName>${prefix}_rope_payload</linkName>
+             <aeroForcesVis>${prefix}_aero_force_rope_payload</aeroForcesVis>
              <body>
                 <element>
@@ -120,13 +121,14 @@
        </gazebo>
        <xacro:rope_joint
-         parent="rope_seg_0"
-         child="rope_payload"
+         parent="${prefix}_rope_seg_0"
+         child="${prefix}_rope_payload"
          name="0_pyld"
-         c="0.5">
+         c="0.5"
+         prefix="${prefix}">
          <origin xyz="0 0 ${seg_len}" rpy="0 0 1.57"/>
        </xacro:rope_joint>
   </xacro:macro>
-  <xacro:macro name="add_seg" params="n dia seg_len seg_mass color damping parent">
-       <link name="rope_seg_${n}">
+  <xacro:macro name="add_seg" params="n dia seg_len seg_mass color damping parent prefix">
+       <link name="${prefix}_rope_seg_${n}">
          <inertial>
            <origin xyz="0 0 ${seg_len/2}" rpy="0 0 0" />
@@ -141,5 +143,5 @@
          </visual>
        </link>
-       <gazebo reference="rope_seg_${n}">
+       <gazebo reference="${prefix}_rope_seg_${n}">
          <material>Gazebo/${color}</material>
        </gazebo>
@@ -147,6 +149,6 @@
           <plugin filename="librotors_gazebo_aerodynamics_plugin.so" name="aerodynamics_plugin">
              <robotNamespace></robotNamespace>
-             <linkName>rope_seg_${n}</linkName>
-             <aeroForcesVis>aero_force_rope_${n}</aeroForcesVis>
+             <linkName>${prefix}_rope_seg_${n}</linkName>
+             <aeroForcesVis>${prefix}_aero_force_rope_${n}</aeroForcesVis>
              <body>
                 <element>
@@ -162,15 +164,16 @@
        </gazebo>
        <xacro:rope_joint
-           parent="rope_seg_${n+1}"
-           child="rope_seg_${n}"
+           parent="${prefix}_rope_seg_${n+1}"
+           child="${prefix}_rope_seg_${n}"
            name="${n+1}_${n}"
-           c="${damping}">
+           c="${damping}"
+           prefix="${prefix}">
            <origin xyz="0 0 ${seg_len}" rpy="0 0 0"/>
        </xacro:rope_joint>
        <xacro:if value="${n}">
-          <xacro:add_seg n="${n-1}" dia="${dia}" seg_len="${seg_len}" seg_mass="${seg_mass}" color="${color}" damping="${damping}" parent="rope_seg_${n}"/>
+          <xacro:add_seg n="${n-1}" dia="${dia}" seg_len="${seg_len}" seg_mass="${seg_mass}" color="${color}" damping="${damping}" parent="rope_seg_${n}" prefix="${prefix}"/>
        </xacro:if>
   </xacro:macro>
-  <xacro:macro name="rope_joint" params="parent child name c *joint_origin">
+  <xacro:macro name="rope_joint" params="parent child name c prefix *joint_origin">
        <!--
        <joint name="rj_${name}_a" type="continuous">
@@ -222,16 +225,16 @@
        </gazebo>
        -->
-       <joint name="rj_${name}_a" type="continuous">
+       <joint name="${prefix}_rj_${name}_a" type="continuous">
          <xacro:insert_block name="joint_origin" />
          <axis xyz="1 0 0"/>
          <parent link="${parent}" />
-         <child link="rl_${name}_a"/>
-         <dynamics damping="${c}"/>
-       </joint>
-       <gazebo reference="rj_${name}_a">
-         <implicitSpringDamper>true</implicitSpringDamper>
-         <springStiffness>0</springStiffness>
-       </gazebo>
-       <link name="rl_${name}_a">
+         <child link="${prefix}_rl_${name}_a"/>
+         <dynamics damping="${c}"/>
+       </joint>
+       <gazebo reference="${prefix}_rj_${name}_a">
+         <implicitSpringDamper>true</implicitSpringDamper>
+         <springStiffness>0</springStiffness>
+       </gazebo>
+       <link name="${prefix}_rl_${name}_a">
          <inertial>
            <origin xyz="0 0 0" rpy="0 0 0"/>
@@ -240,12 +243,12 @@
          </inertial>
        </link>
-       <joint name="rj_${name}_b" type="continuous">
+       <joint name="${prefix}_rj_${name}_b" type="continuous">
          <origin xyz="0 0 0" rpy="0 0 0"/>
          <axis xyz="0 1 0"/>
-         <parent link="rl_${name}_a" />
+         <parent link="${prefix}_rl_${name}_a" />
          <child link="${child}"/>
          <dynamics damping="${c}"/>
        </joint>
-       <gazebo reference="rj_${name}_b">
+       <gazebo reference="${prefix}_rj_${name}_b">
          <implicitSpringDamper>true</implicitSpringDamper>
          <springStiffness>0</springStiffness>
