Commit message: Miscellaneous, mostly refactoring
- techpod_TJ_flex: Refactoring
- lidar plugin: Publish to custom topic if desired + info printing
- fw_playground: Minor refactoring
- fixed_wing_X_base: Minor refactoring, get rid of unused arguments of vane macro
- component snippets: lidar_plugin_macro, ideal_imu macro, default_odometry macro, default_lidar macro, asl_mono_vi_1 odometry topic renaming
- rope.xacro: Adding prefixes to links
- inertias.xacro: all kind of inertia macros...

File: rotors_description/urdf/techpod_TJ_flex.xacro (robot description, xacro)
@@ -13,4 +13,6 @@
 -->
 <robot xmlns:xacro="http://ros.org/wiki/xacro" name="techpod_TJ_flex">
+   <!-- Include URDF files -->
+   <xacro:include filename="$(find rotors_description)/urdf/fixed_wing_X_base.xacro" />
    <!-- Global properties -->
    <xacro:property name="namespace" value="$(arg namespace)" />
@@ -23,12 +25,4 @@
    <!-- Constants -->
    <xacro:property name="PI" value="3.1415926535897931" />
-   <!-- Component masses -->
-   <!--<xacro:property name="mass_fuselage" value="2.124" />--><!-- [kg] -->
-   <xacro:property name="mass_fuselage" value="1.984" />
-   <xacro:property name="mass_aileron" value="0.01" /><!-- [kg] -->
-   <xacro:property name="mass_flap" value="0.01" /><!-- [kg] -->
-   <xacro:property name="mass_elevator" value="0.01" /><!-- [kg] -->
-   <xacro:property name="mass_rudder" value="0.01" /><!-- [kg] -->
-   <xacro:property name="mass_propeller" value="0.01" /><!-- [kg] -->
    <!-- Main body properties -->
    <xacro:property name="body_length" value="1.088" /><!-- [m] -->
@@ -36,5 +30,4 @@
    <xacro:property name="body_height" value="0.303" /><!-- [m] -->
    <xacro:property name="body_color" value="White" />
-   <xacro:property name="body_mesh_file" value="package://rotors_description/meshes/techpod/techpod_body.dae" />
    <!-- Aileron properties -->
    <xacro:property name="aileron_length" value="0.15" /><!-- [m] -->
@@ -44,6 +37,4 @@
    <xacro:property name="aileron_max_angle" value="0.349066" /><!-- [rad] -->
    <xacro:property name="aileron_color" value="${body_color}" />
-   <xacro:property name="aileron_left_mesh_file" value="package://rotors_description/meshes/techpod/techpod_aileron_left.dae" />
-   <xacro:property name="aileron_right_mesh_file" value="package://rotors_description/meshes/techpod/techpod_aileron_right.dae" />
    <!-- Elevator properties -->
    <xacro:property name="elevator_length" value="0.15" /><!-- [m] -->
@@ -53,5 +44,4 @@
    <xacro:property name="elevator_max_angle" value="0.349066" /><!-- [rad] -->
    <xacro:property name="elevator_color" value="${body_color}" />
-   <xacro:property name="elevator_mesh_file" value="package://rotors_description/meshes/techpod/techpod_elevator.dae" />
    <!-- Flap properties -->
    <xacro:property name="flap_length" value="0.18" /><!-- [m] -->
@@ -61,6 +51,4 @@
    <xacro:property name="flap_max_angle" value="0.349066" /><!-- [rad] -->
    <xacro:property name="flap_color" value="${body_color}" />
-   <xacro:property name="flap_left_mesh_file" value="package://rotors_description/meshes/techpod/techpod_flap_left.dae" />
-   <xacro:property name="flap_right_mesh_file" value="package://rotors_description/meshes/techpod/techpod_flap_right.dae" />
    <!-- Rudder properties -->
    <xacro:property name="rudder_length" value="0.13" />
@@ -70,5 +58,4 @@
    <xacro:property name="rudder_max_angle" value="0.349066" />
    <xacro:property name="rudder_color" value="${body_color}" />
-   <xacro:property name="rudder_mesh_file" value="package://rotors_description/meshes/techpod/techpod_rudder.dae" />
    <!-- Propeller properties -->
    <xacro:property name="propeller_direction" value="cw" />
@@ -76,5 +63,4 @@
    <xacro:property name="propeller_height" value="0.003" />
    <xacro:property name="propeller_color" value="Gray" />
-   <xacro:property name="propeller_mesh_file" value="package://rotors_description/meshes/propeller_${propeller_direction}.dae" />
    <!-- Flexing properties -->
    <xacro:property name="k1" value="375" />
@@ -86,13 +72,35 @@
    <xacro:property name="k4" value="120" />
    <xacro:property name="d4" value="1.8" />
-   <!-- Inertia of the main body -->
    <!--
-   <xacro:property name="body_inertia">
-      <inertia ixx="0.16632" ixy="0.0" ixz="0.0755" iyy="0.3899" iyz="0.0" izz="0.5243" />
-   </xacro:property>
-   -->
-   <xacro:property name="body_inertia">
+   Inertial properties - do not change without considering link-tree, i.e.:
+   From System Identification, we obtain total mass m_tot and total inertia J_tot
+   wrt cg. For the Techpod, these are:
+   m_tot = 3.124 kg
+   J_tot = [ixx=0.6688, iyy=0.1623, izz=0.6936, ixz=0.0281] kgm^2  (wrt cg, FLU frame)
+   r_cg = [0, 0, 0.097] (cg position in baselink frame (FLU))
+   Considering the masses and positions of all leaf-links (root = baselink), we
+   calculate mass and inertia of the baselink s.t. the overall inertial properties
+   defined above are matched (ignoring the link-centric inertias of the links as
+   they are deliberately set to very small values...). With the link masses set below
+   and in the segment macros, we get for the baselink:
+   m_base_link = 1.984 kg
+   J_base_link = [ixx=0.1686, iyy=0.0498, izz=0.1100, ixz=0.0013]   (wrt cg, FLU frame)
+   r_cg_base_link = [0.0684, 0, 0.0511] (cg position in baselink frame (FLU))
+  -->
+   <xacro:property name="m_base_link" value="1.984" />
+   <xacro:property name="J_base_link">
      <inertia ixx="0.1686" ixy="0.0" ixz="0.0013" iyy="0.0498" iyz="0.0" izz="0.1100" />
    </xacro:property>
+   <xacro:property name="r_cg_base_link">
+      <!--<origin xyz="0.09 0 0.147" rpy="0 0 0" />-->
+      <origin xyz="0.068 0 ${0.051+0.05}" rpy="0 0 0" />
+   </xacro:property>
+   <!-- the following masses are deliberately small to get neglectable inertias,
+        basically 'dummy inertias'-->
+   <xacro:property name="mass_aileron" value="0.01" /><!-- [kg] -->
+   <xacro:property name="mass_flap" value="0.01" /><!-- [kg] -->
+   <xacro:property name="mass_elevator" value="0.01" /><!-- [kg] -->
+   <xacro:property name="mass_rudder" value="0.01" /><!-- [kg] -->
+   <xacro:property name="mass_propeller" value="0.01" /><!-- [kg] -->
    <!-- Inertia of the aileron, assuming it is a cuboid -->
    <xacro:property name="aileron_inertia">
@@ -112,13 +120,13 @@
    </xacro:property>
    <!-- Inertia of the propeller, assuming it is a cylinder -->
+   <!-- Note: Keep it small as possible, this is as well just a dummy inertia,
+        gyroscopic effects are simulated in propulsion plugin with the mass
+        specified in the propeller's *.yaml file-->
    <xacro:property name="propeller_inertia">
-      <xacro:cylinder_inertia r="${propeller_radius}" h="${propeller_height}" mass="${mass_propeller*rotor_velocity_slowdown_sim}" />
+      <xacro:cylinder_inertia r="${propeller_radius}" h="${propeller_height}" mass="${mass_propeller}" />
    </xacro:property>
-   <!-- Include URDF files -->
-   <xacro:include filename="$(find rotors_description)/urdf/fixed_wing_X_base.xacro" />
-   <xacro:include filename="$(find rotors_description)/urdf/rope.xacro" />
    <!-- Instantiate fixed_wing_base_macro once and adding fuselage parts -->
    <xacro:fixed_wing_base_macro robot_namespace="${namespace}"
-      mass="${mass_fuselage}"
+      mass="${m_base_link}"
       length="${body_length}"
       width="0.2"
@@ -127,7 +135,6 @@
       use_mesh_file="true"
       mesh_file="package://rotors_description/meshes/techpod_X_flex/fuselage_barless.stl">
-      <!--<origin xyz="0.09 0 0.147" rpy="0 0 0" />-->
-      <origin xyz="0.068 0 ${0.051+0.05}" rpy="0 0 0" />
-      <xacro:insert_block name="body_inertia" />
+      <xacro:insert_block name="r_cg_base_link" />
+      <xacro:insert_block name="J_base_link" />
    </xacro:fixed_wing_base_macro>
    <joint name="${namespace}/dome_joint" type="fixed">
@@ -226,18 +233,4 @@
       <material>Gazebo/Grey</material>
    </gazebo>
-   <!--
-   <link name="${namespace}/check_coordinates">
-      <inertial>
-         <mass value="0.1" />
-         <xacro:box_inertia x="0.1" y="0.1" z="0.1" mass="0.1" />
-      </inertial>
-   </link>
-   <joint name="${namespace}/check_coordinates_joint" type="revolute">
-     <origin xyz="0.54 0 0.184" rpy="0 0 0" />
-     <parent link="${namespace}/base_link" />
-     <child link="${namespace}/check_coordinates" />
-     <limit upper="0" lower="0" effort="0" velocity="0" />
-   </joint>
-   -->
    <!-- Instantiate (flexing) wing segments -->
    <xacro:airfoil_segment robot_namespace="${namespace}"
@@ -1071,8 +1064,6 @@
       parent="${namespace}/wl_1"
       wind_topic="wind_base_link"
-      color="Grey"
-      mesh_file="package://rotors_description/meshes/techpod_X_flex/flp_l_1.stl">
+      color="Grey">
       <origin xyz="0.15 0.345 0.05" rpy="0 0 0" /><!-- Joint origin -->
-      <origin xyz="0 0 0" rpy="0 0 0" /><!-- vis_coll origin -->
       <xacro:box_inertia x="0.1" y="0.02" z="0.02" mass="0.02" />
    </xacro:angle_vane>
@@ -1104,8 +1095,6 @@
       parent="${namespace}/wr_1"
       wind_topic="wind_base_link"
-      color="Grey"
-      mesh_file="package://rotors_description/meshes/techpod_X_flex/flp_l_1.stl">
+      color="Grey">
       <origin xyz="0.15 -0.34 0.057" rpy="0 0 0" /><!-- Joint origin -->
-      <origin xyz="0 0 0" rpy="0 0 0" /><!-- vis_coll origin -->
       <xacro:box_inertia x="0.1" y="0.02" z="0.02" mass="0.02" />
    </xacro:angle_vane>
@@ -1170,116 +1159,4 @@
      </gazebo>
    </xacro:if>
-   <!-- Tracing ribbon/Visual plugin -->
-   <!--
-   <gazebo reference="${namespace}/base_link">
-      <visual>
-         <plugin name="visual_plugin_base_link" filename="librotors_gazebo_template_visual_plugin.so" />
-      </visual>
-   </gazebo>
-   -->
-   <!-- Payload -->
-   <!--
-   <link name="${namespace}/payload_1">
-      <inertial>
-         <origin xyz="0.07 0 0" rpy="0 0 0" />
-         <mass value="0.25" />
-         <xacro:sphere_inertia r="0.05" mass="0.25" />
-      </inertial>
-      <visual>
-         <origin xyz="0.07 0 0" rpy="0 0 0" />
-         <geometry>
-            <mesh filename="package://rotors_description/meshes/payloads/payload.stl" scale="0.012 0.012 0.012" />
-         </geometry>
-      </visual>
-      <collision>
-         <origin xyz="0.01 0 0" rpy="0 0 0" />
-         <geometry>
-            <box size = "0.25 0.12 0.05" />
-         </geometry>
-      </collision>
-   </link>
-   <joint name="${namespace}/payload_1_joint" type="floating">
-      <parent link="${namespace}/wl_2" />
-      <child link="${namespace}/payload_1" />
-      <origin xyz="0 0 0" rpy="0 0 0" />
-   </joint>
-   <gazebo reference="${namespace}/payload_1">
-      <visual>
-         <plugin name="visual_plugin_payload_1" filename="librotors_gazebo_template_visual_plugin.so" />
-      </visual>
-      <material>Gazebo/Orange</material>
-      <mu1>0.2</mu1>
-      <mu2>0.2</mu2>
-      <kp>10000</kp>
-      <kd>1</kd>
-   </gazebo>
-   <gazebo>
-      <plugin filename="librotors_gazebo_payload_plugin.so" name="payload_plugin_1">
-         <robotNamespace>${namespace}</robotNamespace>
-         <joint>${namespace}/payload_1_joint</joint>
-         <payload>${namespace}/payload_1</payload>
-         <parent>${namespace}/wl_2</parent>
-         <hoistPosParent>0 -0.15 -0.04</hoistPosParent>
-         <hoistPosPayload>0 0 0</hoistPosPayload>
-         <dropTopic>drop_1</dropTopic>
-      </plugin>
-   </gazebo>
-   <gazebo>
-      <plugin filename="librotors_gazebo_aerodynamics_plugin.so" name="aerodynamics_plugin">
-         <robotNamespace>${namespace}</robotNamespace>
-         <linkName>${namespace}/payload_1</linkName>
-         <aeroForcesVis>aero_force_vis_payload_1</aeroForcesVis>
-         <airfoil>
-            <segment name="HS">
-               <forward>1 0 0</forward>
-               <upward>0 0 1</upward>
-               <cp>-0.15 0 0</cp>
-               <seg_area>0.005</seg_area>
-               <seg_chord>0.05</seg_chord>
-               <aeroParamsYAML>${yaml_path}/airfoil_test_2.yaml</aeroParamsYAML>
-               <wind name="wind">
-                 <topic>wind_payload</topic>
-               </wind>
-            </segment>
-            <segment name="VS">
-               <forward>1 0 0</forward>
-               <upward>0 -1 0</upward>
-               <cp>-0.15 0 0</cp>
-               <seg_area>0.005</seg_area>
-               <seg_chord>0.05</seg_chord>
-               <aeroParamsYAML>${yaml_path}/airfoil_test_2.yaml</aeroParamsYAML>
-               <wind name="wind">
-                 <topic>wind_payload</topic>
-               </wind>
-            </segment>
-         </airfoil>
-         <body>
-            <element>
-               <aBdyXX>0.0028</aBdyXX>
-               <aBdyYY>0.015</aBdyYY>
-               <aBdyZZ>0.015</aBdyZZ>
-               <forward>1 0 0</forward>
-               <upward>0 0 1</upward>
-               <cp>-0.05 0.0 0</cp>
-               <wind name="wind">
-                 <topic>wind_payload</topic>
-               </wind>
-            </element>
-         </body>
-      </plugin>
-   </gazebo>
-   -->
-   <!-- Payload on rope -->
-   <!--
-   <xacro:rope n="20"
-      length="10"
-      dia="0.01"
-      mass="0.05"
-      damping="10"
-      parent="${namespace}/base_link"
-      color="Red">
-      <origin xyz="-0.15 0 0.02" rpy="0 -1.57 0" />
-   </xacro:rope>
-   -->
    <!-- Mavlink interface -->
    <gazebo>
@@ -1322,4 +1199,13 @@
                <joint_control_type>gz_msg</joint_control_type>
                <gztopic>prop_ref_0</gztopic>
+            </channel>
+            <channel name="propeller_anim">
+               <input_index>4</input_index>
+               <input_offset>1</input_offset>
+               <input_scaling>20</input_scaling><!-- rdps_slope/2  [rad/s]-->
+               <zero_position_disarmed>0</zero_position_disarmed>
+               <zero_position_armed>0</zero_position_armed>
+               <joint_control_type>velocity</joint_control_type>
+               <joint_name>${namespace}/propeller_P0_joint</joint_name>
             </channel>
             <channel name="aileron_left">
@@ -1403,15 +1289,21 @@
                <gztopic>flap_r2_pos</gztopic>
             </channel>
-            <channel name="payload">
-               <input_index>8</input_index>
-               <input_offset>0</input_offset>
-               <input_scaling>1</input_scaling>
-               <zero_position_disarmed>0</zero_position_disarmed>
-               <zero_position_armed>0</zero_position_armed>
-               <joint_control_type>gz_msg</joint_control_type>
-               <gztopic>drop_1</gztopic>
-            </channel>
          </control_channels>
       </plugin>
    </gazebo>
+   <!-- Miscellaneous -->
+   <!--
+   <link name="${namespace}/check_coordinates">
+      <inertial>
+         <mass value="0.1" />
+         <xacro:box_inertia x="0.1" y="0.1" z="0.1" mass="0.1" />
+      </inertial>
+   </link>
+   <joint name="${namespace}/check_coordinates_joint" type="revolute">
+     <origin xyz="0.54 0 0.184" rpy="0 0 0" />
+     <parent link="${namespace}/base_link" />
+     <child link="${namespace}/check_coordinates" />
+     <limit upper="0" lower="0" effort="0" velocity="0" />
+   </joint>
+   -->
 </robot>

File: rotors_description/urdf/techpod_TJ_flex_base.xacro (robot description, xacro)
@@ -32,25 +32,12 @@
   <xacro:default_pressure_sensor namespace="${namespace}" parent_link="${namespace}/base_link" />
   -->
-  <xacro:default_camera
-    namespace="${namespace}"
-    parent_link="${namespace}/base_link"
-    camera_suffix="fus_left">
-    <origin xyz="0.21 0.045 0.145" rpy="0 -0.1 2.2" />
-  </xacro:default_camera>
-  <xacro:default_camera
-    namespace="${namespace}"
-    parent_link="${namespace}/base_link"
-    camera_suffix="fus_right">
-    <origin xyz="0.21 -0.045 0.145" rpy="0 -0.1 -2.2" />
-  </xacro:default_camera>
-  <!---->
   <xacro:camera_macro_2
     namespace="${namespace}"
     parent_link="${namespace}/base_link"
-    camera_suffix="3pv_lowres"
+    camera_suffix="3pv"
     frame_rate="60"
     horizontal_fov="1.3962634"
-    image_width="188"
-    image_height="120"
+    image_width="752"
+    image_height="480"
     image_format="L8"
     min_distance="0.02"
@@ -64,50 +51,20 @@
     <origin xyz="-2 0 0.5" rpy="0 0.2 0" />
   </xacro:camera_macro_2>
-  <!--
-  <xacro:asl_mono_vi_1
+  <!-- Trinocular Setup -->
+  <!-- Camera Fuselage Left -->
+  <xacro:default_camera
     namespace="${namespace}"
     parent_link="${namespace}/base_link"
-    suffix="center"
-    fps="30"
-    h_fov="1.3514"
-    imu_topic="adis/data_raw"
-    acc_nd="0.0100"
-    acc_rw="0.0020"
-    gyr_nd="0.0050"
-    gyr_rw="0.00004">
-    <origin xyz="0.35 0 0.11" rpy="0 0.3 0" />
-    <origin xyz="-0.0014 0.0146 -0.1175" rpy="-3.1228 -1.1414 -1.6129" />
-    <origin xyz="-0.0014 0.0146 -0.1175" rpy="-3.1228 -1.1414 -1.6129" />
-  </xacro:asl_mono_vi_1>
-  <xacro:asl_mono_vi_1
+    camera_suffix="fus_left">
+    <origin xyz="0.21 0.045 0.145" rpy="0 -0.1 2.2" />
+  </xacro:default_camera>
+  <!-- Camera Fuselage Right -->
+  <xacro:default_camera
     namespace="${namespace}"
-    parent_link="${namespace}/wl_3"
-    suffix="left"
-    fps="30"
-    h_fov="1.3560"
-    imu_topic="camImu0/data_raw"
-    acc_nd="0.1006"
-    acc_rw="0.0040"
-    gyr_nd="0.0258"
-    gyr_rw="0.0007">
-    <origin xyz="0.05 0.38 0.025" rpy="0 0.3 0" />
-    <origin xyz="-0.0264 0.0061 -0.0331" rpy="3.1298 0.0029 1.5626" />
-    <origin xyz="-0.0264 0.0061 -0.0331" rpy="3.1298 0.0029 1.5626" />
-  </xacro:asl_mono_vi_1>
-  <xacro:asl_mono_vi_1
-    namespace="${namespace}"
-    parent_link="${namespace}/wr_3"
-    suffix="right"
-    fps="30"
-    h_fov="1.3626"
-    imu_topic="camImu1/data_raw"
-    acc_nd="0.1006"
-    acc_rw="0.0040"
-    gyr_nd="0.0258"
-    gyr_rw="0.0007">
-    <origin xyz="0.05 -0.38 0.025" rpy="0 0.3 0" />
-    <origin xyz="-0.0083 -0.0177 -0.0469" rpy="-3.1363 -0.0648 1.5500" />
-    <origin xyz="-0.0083 -0.0177 -0.0469" rpy="-3.1363 -0.0648 1.5500" />
-  </xacro:asl_mono_vi_1>-->
+    parent_link="${namespace}/base_link"
+    camera_suffix="fus_right">
+    <origin xyz="0.21 -0.045 0.145" rpy="0 -0.1 -2.2" />
+  </xacro:default_camera>
+  <!-- Camera/IMU Fuselage Center -->
   <xacro:asl_mono_vi_1
     namespace="${namespace}"
@@ -125,4 +82,5 @@
     <origin xyz="0 0 0" rpy="0 0 0" />
   </xacro:asl_mono_vi_1>
+  <!-- Camera/IMU Wing Left -->
   <xacro:asl_mono_vi_1
     namespace="${namespace}"
@@ -140,4 +98,5 @@
     <origin xyz="0 0 0" rpy="0 0 0" />
   </xacro:asl_mono_vi_1>
+  <!-- Camera/IMU Wing Right -->
   <xacro:asl_mono_vi_1
     namespace="${namespace}"
@@ -155,19 +114,3 @@
     <origin xyz="0 0 0" rpy="0 0 0" />
   </xacro:asl_mono_vi_1>
-  <!--
-  <xacro:default_camera
-    namespace="${namespace}"
-    parent_link="${namespace}/base_link"
-    camera_suffix="cam_aft">
-    <origin xyz="-0.7 0 0.02" rpy="0 0.4 3.14" />
-  </xacro:default_camera>
-  -->
-  <!--
-  <xacro:default_camera
-    namespace="${namespace}"
-    parent_link="${namespace}/payload_1"
-    camera_suffix="cam_payload">
-    <origin xyz="0.125 0 0" rpy="0 0 0" />
-  </xacro:default_camera>
-  -->
 </robot>

Commit message: Add PX4 GPS plugin which does not use gazebo gps sensor

File: rotors_description/urdf/component_snippets.xacro (robot description, xacro)
@@ -598,4 +598,43 @@
     </gazebo>
   </xacro:macro>
+  <!-- Macro to add a GPS sensor. -->
+  <xacro:macro name="gps_plugin_px4_macro"
+    params="namespace gps_suffix parent_link gps_topic
+      mass_gps_sensor Noise XYRandomWalk ZRandomWalk XYNoiseDensity
+      ZNoiseDensity VXYNoiseDensity VZNoiseDensity *inertia *origin">
+    <!-- GPS link -->
+    <link name="${namespace}/gps${gps_suffix}_link">
+      <inertial>
+        <xacro:insert_block name="inertia" />
+        <mass value="${mass_gps_sensor}" />  <!-- [kg] -->
+        <origin xyz="0 0 0" rpy="0 0 0" />
+      </inertial>
+    </link>
+    <!-- GPS joint -->
+    <joint name="${namespace}/gps${gps_suffix}_joint" type="revolute">
+      <xacro:insert_block name="origin" />
+      <parent link="${parent_link}" />
+      <child link="${namespace}/gps${gps_suffix}_link" />
+      <limit upper="0" lower="0" effort="0" velocity="0" />
+    </joint>
+    <gazebo reference="${namespace}/gps${gps_suffix}_link">
+      <sensor type="gps" name="${namespace}_gps${gps_suffix}">
+        <pose>0 0 0 0 0 0</pose>
+        <visualize>0</visualize>
+        <always_on>1</always_on>
+        <plugin filename="librotors_gazebo_gps_plugin_px4.so" name="rotors_gazebo_gps${gps_suffix}_plugin_px4">
+          <robotNamespace>${namespace}</robotNamespace> <!-- (string, required): ros namespace in which the messages are published -->
+          <gpsTopic>${gps_topic}</gpsTopic> <!-- (string): name of the sensor output topic and prefix of service names (defaults to 'gps') -->
+          <gpsNoise>${Noise}</gpsNoise>
+          <gpsXYRandomWalk>${XYRandomWalk}</gpsXYRandomWalk>
+          <gpsZRandomWalk>${ZRandomWalk}</gpsZRandomWalk>
+          <gpsXYNoiseDensity>${XYNoiseDensity}</gpsXYNoiseDensity>
+          <gpsZNoiseDensity>${ZNoiseDensity}</gpsZNoiseDensity>
+          <gpsVXYNoiseDensity>${VXYNoiseDensity}</gpsVXYNoiseDensity>
+          <gpsVZNoiseDensity>${VZNoiseDensity}</gpsVZNoiseDensity>
+        </plugin>
+      </sensor>
+    </gazebo>
+  </xacro:macro>
   <!-- Macro to add a single-ray LIDAR. -->
   <xacro:macro name="lidar_plugin_macro"
@@ -1169,4 +1208,23 @@
     </xacro:gps_plugin_macro>
   </xacro:macro>
+  <xacro:macro name="default_gps_px4" params="namespace parent_link *origin">
+    <!-- Default px4 GPS -->
+    <xacro:gps_plugin_px4_macro
+      namespace="${namespace}"
+      gps_suffix=""
+      parent_link="${parent_link}"
+      gps_topic="gps"
+      mass_gps_sensor="0.015"
+      Noise="1"
+      XYRandomWalk="1.0"
+      ZRandomWalk="4.0"
+      XYNoiseDensity="0.0002"
+      ZNoiseDensity="0.0004"
+      VXYNoiseDensity="0.2"
+      VZNoiseDensity="0.4">
+      <xacro:cube_inertia l="0.02" mass="0.015" />
+      <xacro:insert_block name="origin" />
+    </xacro:gps_plugin_px4_macro>
+  </xacro:macro>
   <xacro:macro name="default_odometry" params="namespace parent_link">
     <xacro:odometry_plugin_macro

File: rotors_description/urdf/techpod_sitl_base.xacro (robot description, xacro)
@@ -21,7 +21,7 @@
   </xacro:default_imu>
   <!-- Mount a GPS. -->
-  <xacro:default_gps namespace="${namespace}" parent_link="${namespace}/base_link" >
+  <xacro:default_gps_px4 namespace="${namespace}" parent_link="${namespace}/base_link" >
     <origin xyz="0.06 0 0.19" rpy="0 0 0" />
-  </xacro:default_gps>
+  </xacro:default_gps_px4>
   <!-- Mount a magnetometer. note: mavlink interface already does this based on position from gps-->
   <!--
