Commit message: Revert "Add PX4 GPS plugin which does not use gazebo gps sensor"
This reverts commit 16925fb16947729911b1a037ef168c2c406bad14.

File: rotors_description/urdf/component_snippets.xacro (robot description, xacro)
@@ -598,43 +598,4 @@
     </gazebo>
   </xacro:macro>
-  <!-- Macro to add a GPS sensor. -->
-  <xacro:macro name="gps_plugin_px4_macro"
-    params="namespace gps_suffix parent_link gps_topic
-      mass_gps_sensor Noise XYRandomWalk ZRandomWalk XYNoiseDensity
-      ZNoiseDensity VXYNoiseDensity VZNoiseDensity *inertia *origin">
-    <!-- GPS link -->
-    <link name="${namespace}/gps${gps_suffix}_link">
-      <inertial>
-        <xacro:insert_block name="inertia" />
-        <mass value="${mass_gps_sensor}" />  <!-- [kg] -->
-        <origin xyz="0 0 0" rpy="0 0 0" />
-      </inertial>
-    </link>
-    <!-- GPS joint -->
-    <joint name="${namespace}/gps${gps_suffix}_joint" type="revolute">
-      <xacro:insert_block name="origin" />
-      <parent link="${parent_link}" />
-      <child link="${namespace}/gps${gps_suffix}_link" />
-      <limit upper="0" lower="0" effort="0" velocity="0" />
-    </joint>
-    <gazebo reference="${namespace}/gps${gps_suffix}_link">
-      <sensor type="gps" name="${namespace}_gps${gps_suffix}">
-        <pose>0 0 0 0 0 0</pose>
-        <visualize>0</visualize>
-        <always_on>1</always_on>
-        <plugin filename="librotors_gazebo_gps_plugin_px4.so" name="rotors_gazebo_gps${gps_suffix}_plugin_px4">
-          <robotNamespace>${namespace}</robotNamespace> <!-- (string, required): ros namespace in which the messages are published -->
-          <gpsTopic>${gps_topic}</gpsTopic> <!-- (string): name of the sensor output topic and prefix of service names (defaults to 'gps') -->
-          <gpsNoise>${Noise}</gpsNoise>
-          <gpsXYRandomWalk>${XYRandomWalk}</gpsXYRandomWalk>
-          <gpsZRandomWalk>${ZRandomWalk}</gpsZRandomWalk>
-          <gpsXYNoiseDensity>${XYNoiseDensity}</gpsXYNoiseDensity>
-          <gpsZNoiseDensity>${ZNoiseDensity}</gpsZNoiseDensity>
-          <gpsVXYNoiseDensity>${VXYNoiseDensity}</gpsVXYNoiseDensity>
-          <gpsVZNoiseDensity>${VZNoiseDensity}</gpsVZNoiseDensity>
-        </plugin>
-      </sensor>
-    </gazebo>
-  </xacro:macro>
   <!-- Macro to add a single-ray LIDAR. -->
   <xacro:macro name="lidar_plugin_macro"
@@ -1208,23 +1169,4 @@
     </xacro:gps_plugin_macro>
   </xacro:macro>
-  <xacro:macro name="default_gps_px4" params="namespace parent_link *origin">
-    <!-- Default px4 GPS -->
-    <xacro:gps_plugin_px4_macro
-      namespace="${namespace}"
-      gps_suffix=""
-      parent_link="${parent_link}"
-      gps_topic="gps"
-      mass_gps_sensor="0.015"
-      Noise="1"
-      XYRandomWalk="1.0"
-      ZRandomWalk="4.0"
-      XYNoiseDensity="0.0002"
-      ZNoiseDensity="0.0004"
-      VXYNoiseDensity="0.2"
-      VZNoiseDensity="0.4">
-      <xacro:cube_inertia l="0.02" mass="0.015" />
-      <xacro:insert_block name="origin" />
-    </xacro:gps_plugin_px4_macro>
-  </xacro:macro>
   <xacro:macro name="default_odometry" params="namespace parent_link">
     <xacro:odometry_plugin_macro

File: rotors_description/urdf/techpod_sitl_base.xacro (robot description, xacro)
@@ -21,7 +21,7 @@
   </xacro:default_imu>
   <!-- Mount a GPS. -->
-  <xacro:default_gps_px4 namespace="${namespace}" parent_link="${namespace}/base_link" >
+  <xacro:default_gps namespace="${namespace}" parent_link="${namespace}/base_link" >
     <origin xyz="0.06 0 0.19" rpy="0 0 0" />
-  </xacro:default_gps_px4>
+  </xacro:default_gps>
   <!-- Mount a magnetometer. note: mavlink interface already does this based on position from gps-->
   <!--

Commit message: init

File: rotors_description/urdf/component_snippets.xacro (robot description, xacro)
@@ -50,5 +50,7 @@
             <xacro:insert_block name="geometry" />
           </geometry>
-          <material name="red" />
+          <material name="red">
+            <color rgba="0.8 0 0 1"/>
+          </material>
         </visual>
       </xacro:if>
@@ -128,5 +130,7 @@
             <xacro:insert_block name="geometry" />
           </geometry>
-          <material name="red" />
+          <material name="red">
+            <color rgba="0.8 0 0 1"/>
+          </material>
         </visual>
       </xacro:if>
@@ -895,3 +899,95 @@
     </xacro:mavlink_interface_macro>
   </xacro:macro>
+  <!-- RGBD SENSOR MACROS  -->
+  <!--_____________________________________________________________________________________________________-->
+  <xacro:macro name="rgbd_sensor_macro"
+    params="namespace parent_link camera_suffix frame_rate width height fov max_range min_range baseline noise_mean noise_stddev enable_visual *geometry *origin">
+    <link name="${namespace}/camera_${camera_suffix}_link">
+      <collision>
+        <origin xyz="0 0 0" rpy="0 0 0" />
+        <geometry>
+          <xacro:insert_block name="geometry" />
+        </geometry>
+      </collision>
+      <xacro:if value="${enable_visual}">
+        <visual>
+          <origin xyz="0 0 0" rpy="0 ${pi/2} 0" />
+          <geometry>
+            <xacro:insert_block name="geometry" />
+          </geometry>
+          <material name="red">
+            <color rgba="0.8 0 0 1"/>
+          </material>
+        </visual>
+      </xacro:if>
+      <inertial>
+        <mass value="1e-5" />
+        <origin xyz="0 0 0" rpy="0 0 0" />
+        <inertia ixx="1e-6" ixy="0" ixz="0" iyy="1e-6" iyz="0" izz="1e-6" />
+      </inertial>
+    </link>
+    <joint name="${namespace}/camera_${camera_suffix}_joint" type="fixed">
+      <xacro:insert_block name="origin" />
+      <parent link="${parent_link}" />
+      <child link="${namespace}/camera_${camera_suffix}_link" />
+      <limit upper="0" lower="0" effort="0" velocity="0" />
+    </joint>
+    <link name="${namespace}/camera_${camera_suffix}_optical_center_link" />
+    <joint name="${namespace}/camera_${camera_suffix}_optical_center_joint" type="fixed">
+      <origin xyz="0 0 0" rpy="${-pi/2} 0 ${-pi/2}" />
+      <parent link="${namespace}/camera_${camera_suffix}_link" />
+      <child link="${namespace}/camera_${camera_suffix}_optical_center_link" />
+      <limit upper="0" lower="0" effort="0" velocity="0" />
+    </joint>
+    <gazebo reference="${namespace}/camera_${camera_suffix}_link">
+      <sensor type="depth" name="${namespace}_camera_{camera_suffix}">
+        <always_on>true</always_on>
+        <update_rate>${frame_rate}</update_rate>
+        <camera>
+          <horizontal_fov>${fov}</horizontal_fov>
+          <image>
+            <format>R8G8B8</format>
+            <width>${width}</width>
+            <height>${height}</height>
+          </image>
+          <clip>
+            <near>${min_range}</near>
+            <far>${max_range}</far>
+          </clip>
+          <noise>
+            <type>gaussian</type>
+            <!-- Noise is sampled independently per pixel on each frame.
+                 That pixel's noise value is added to each of its color
+                 channels, which at that point lie in the range [0,1]. -->
+            <mean>${noise_mean}</mean>
+            <stddev>${noise_stddev}</stddev>
+          </noise>
+        </camera>
+        <plugin name="${namespace}_camera_{camera_suffix}" filename="librotors_gazebo_noisydepth_plugin.so">
+          <robotNamespace>${namespace}</robotNamespace>
+          <alwaysOn>true</alwaysOn>
+          <baseline>${baseline}</baseline>
+          <updateRate>${frame_rate}</updateRate>
+          <cameraName>camera_${camera_suffix}</cameraName>
+          <horizontal_fov>${fov}</horizontal_fov>
+          <depthNoiseModelName>D435</depthNoiseModelName>
+          <depthNoiseMinDist>0.02</depthNoiseMinDist>
+          <depthNoiseMaxDist>50.0</depthNoiseMaxDist>
+          <D435NoiseSubpixelErr>0.25</D435NoiseSubpixelErr>
+          <D435MaxStdev>3</D435MaxStdev>
+          <imageTopicName>camera/color/image_raw</imageTopicName>
+          <cameraInfoTopicName>camera/color/camera_info</cameraInfoTopicName>
+          <depthImageTopicName>camera/depth/image_raw</depthImageTopicName>
+          <depthImageCameraInfoTopicName>camera/depth/camera_info</depthImageCameraInfoTopicName>
+          <pointCloudTopicName>camera/depth/points</pointCloudTopicName>
+          <frameName>camera_${camera_suffix}_optical_center_link</frameName>
+          <distortionK1>0.0</distortionK1>
+          <distortionK2>0.0</distortionK2>
+          <distortionK3>0.0</distortionK3>
+          <distortionT1>0.0</distortionT1>
+          <distortionT2>0.0</distortionT2>
+        </plugin>
+      </sensor>
+    </gazebo>
+  </xacro:macro>
 </robot>

Commit message: some world changes

File: rotors_description/urdf/component_snippets.xacro (robot description, xacro)
@@ -911,10 +911,10 @@
       </collision>
       <xacro:if value="${enable_visual}">
-        <visual>
-          <origin xyz="0 0 0" rpy="0 ${pi/2} 0" />
-          <geometry>
-            <xacro:insert_block name="geometry" />
-          </geometry>
-          <material name="red">
+          <visual>
+            <origin xyz="0 0 0" rpy="0 ${pi/2} 0" />
+            <geometry>
+              <xacro:insert_block name="geometry" />
+            </geometry>
+            <material name="red">
             <color rgba="0.8 0 0 1"/>
           </material>
@@ -981,5 +981,5 @@
           <depthImageCameraInfoTopicName>camera/depth/camera_info</depthImageCameraInfoTopicName>
           <pointCloudTopicName>camera/depth/points</pointCloudTopicName>
-          <frameName>camera_${camera_suffix}_optical_center_link</frameName>
+          <frameName>${namespace}/camera_${camera_suffix}_optical_center_link</frameName>
           <distortionK1>0.0</distortionK1>
           <distortionK2>0.0</distortionK2>

Commit message: delete obsolete, enable running the simulation

File: rotors_description/urdf/component_snippets.xacro (robot description, xacro)
@@ -245,16 +245,4 @@
     </gazebo>
   </xacro:macro>
-  <!-- =============================================================== -->
-  <!-- ==================== ROS INTERFACE MACRO ====================== -->
-  <!-- =============================================================== -->
-  <!-- <xacro:macro
-  		name="ros_interface_plugin_macro"
-  		params="namespace">
-    <gazebo>
-      <plugin name="ros_interface_plugin" filename="librotors_gazebo_ros_interface_plugin.so">
-        <robotNamespace>${namespace}</robotNamespace>
-      </plugin>
-    </gazebo>
-  </xacro:macro>-->
   <!-- =============================================================== -->
   <!-- ================== MAVLINK INTERFACE MACRO ==================== -->

Commit message: drone scaling and odometry noise used for gazebo simulation

File: rotors_description/urdf/component_snippets.xacro (robot description, xacro)
@@ -799,8 +799,8 @@
       measurement_delay="0"
       unknown_delay="0.0"
-      noise_normal_position="0 0 0"
-      noise_normal_quaternion="0 0 0"
-      noise_normal_linear_velocity="0 0 0"
-      noise_normal_angular_velocity="0 0 0"
+      noise_normal_position="0.008 0.008 0.008"
+      noise_normal_quaternion="0.0001 0.0001 0.0001"
+      noise_normal_linear_velocity="0.0005 0.0005 0.0005"
+      noise_normal_angular_velocity="0.0003 0.0003 0.0003"
       noise_uniform_position="0 0 0"
       noise_uniform_quaternion="0 0 0"

File: rotors_description/urdf/omav_snippets.xacro (robot description, xacro)
@@ -33,8 +33,10 @@
       </inertial>
       <visual>
-        <origin xyz="0 0 0" rpy="0 0 0" />
+        <!-- <origin xyz="0.21 0 -0.08" rpy="0 0 0" /> -->
+        <origin xyz="0.21 0 -0.08" rpy="0 0 0" />
         <geometry>
           <xacro:if value="${use_mesh_file}">
-            <mesh filename="${mesh_file}" scale="1 1 1" />
+            <!-- <mesh filename="${mesh_file}" scale="0.11 0.11 0.11" /> -->
+            <mesh filename="${mesh_file}" scale="0.11 0.11 0.11" />
           </xacro:if>
           <xacro:unless value="${use_mesh_file}">
@@ -44,8 +46,8 @@
       </visual>
       <collision>
-        <origin xyz="0 0 0" rpy="0 0 0" />
+        <origin xyz="0.21 0 -0.08" rpy="0 0 0" />
         <geometry>
           <xacro:if value="${use_collision_mesh_file}">
-            <mesh filename="${collision_mesh_file}" scale="1 1 1" />
+            <mesh filename="${collision_mesh_file}" scale="0.11 0.11 0.11" />
           </xacro:if>
           <xacro:unless value="${use_collision_mesh_file}">
