Commit message: Only actuator free tilt units in omav_snippets (former version in overactuated_base).

File: rotors_description/urdf/omav_snippets.xacro (robot description, xacro)
@@ -87,103 +87,4 @@
   </xacro:macro>
   <!-- Tilting rotor unit link and joint. -->
-  <xacro:macro name="single_tilt_unit"
-    params="robot_namespace suffix direction motor_constant moment_constant parent mass_rotor mass_tilt_unit time_constant_up time_constant_down max_rot_velocity rotor_offset_top motor_number rotor_drag_coefficient rolling_moment_coefficient color mesh mesh_tilt_unit p_gain i_gain d_gain *origin *inertia">
-    <!-- Rotor tilt_unit -->
-    <joint name="${robot_namespace}/tilt_unit_${motor_number}_revolutejoint" type="continuous">
-      <xacro:insert_block name="origin" />
-      <axis xyz="1 0 0" />
-      <parent link="${parent}" />
-      <child link="${namespace}/tilt_unit_${motor_number}" />
-    </joint>
-    <link name="${namespace}/tilt_unit_${motor_number}">
-      <inertial>
-        <mass value="${mass_tilt_unit}" /> <!-- [kg] -->
-        <xacro:insert_block name="tilt_unit_inertia" />
-      </inertial>
-      <visual>
-        <geometry>
-            <mesh filename="${mesh_tilt_unit}"
-              scale="1 1 1" />
-        </geometry>
-      </visual>
-      <collision>
-        <geometry>
-          <box size="0.005 0.005 0.005"  /> <!-- [m] -->
-        </geometry>
-      </collision>
-    </link>
-    <gazebo>
-      <plugin name="${suffix}_tilt_unit_model" filename="librotors_gazebo_motor_model.so">
-        <robotNamespace>${robot_namespace}</robotNamespace>
-        <jointName>${namespace}/tilt_unit_${motor_number}_revolutejoint</jointName>
-        <linkName>${namespace}/tilt_unit_${motor_number}</linkName>
-        <turningDirection>ccw</turningDirection>
-        <motorType>position</motorType>
-        <commandSubTopic>/gazebo/command/motor_speed</commandSubTopic>
-        <motorNumber>${motor_number+6}</motorNumber>
-        <motorSpeedPubTopic>/tilt_motor_${motor_number}/velocity</motorSpeedPubTopic>
-        <motorPositionPubTopic>/tilt_motor_${motor_number}/position</motorPositionPubTopic>
-        <joint_control_pid>
-            <p>${p_gain}</p>
-            <i>${i_gain}</i>
-            <d>${d_gain}</d>
-            <iMax>1.0</iMax>
-            <iMin>-1.0</iMin>
-            <cmdMax>2.0</cmdMax>
-            <cmdMin>-2.0</cmdMin>
-        </joint_control_pid>
-      </plugin>
-    </gazebo>
-    <gazebo reference="${namespace}/tilt_unit_${motor_number}">
-      <material>Gazebo/White</material>
-    </gazebo>
-    <!-- Rotor -->
-    <joint name="rotor_${motor_number}_joint" type="continuous">
-      <origin xyz="0 0 ${rotor_offset_top}" rpy="0 0 0" />
-      <axis xyz="0 0 1" />
-      <parent link="${namespace}/tilt_unit_${motor_number}" />
-      <child link="rotor_${motor_number}" />
-    </joint>
-    <link name="rotor_${motor_number}">
-      <inertial>
-        <mass value="${mass_rotor}" /> <!-- [kg] -->
-        <xacro:insert_block name="inertia" />
-      </inertial>
-      <visual>
-        <geometry>
-          <mesh filename="package://rotors_description/meshes/${mesh}_${direction}.dae"
-            scale="${radius_rotor} ${radius_rotor} ${radius_rotor}" />
-        </geometry>
-      </visual>
-      <collision>
-        <geometry>
-          <cylinder length="0.005" radius="${radius_rotor}" /> <!-- [m] -->
-        </geometry>
-      </collision>
-    </link>
-    <gazebo>
-      <plugin name="${suffix}_motor_model" filename="librotors_gazebo_motor_model.so">
-        <robotNamespace>${robot_namespace}</robotNamespace>
-        <jointName>rotor_${motor_number}_joint</jointName>
-        <linkName>rotor_${motor_number}</linkName>
-        <turningDirection>${direction}</turningDirection>
-        <timeConstantUp>${time_constant_up}</timeConstantUp>
-        <timeConstantDown>${time_constant_down}</timeConstantDown>
-        <maxRotVelocity>${max_rot_velocity}</maxRotVelocity>
-        <motorConstant>${motor_constant}</motorConstant>
-        <momentConstant>${moment_constant}</momentConstant>
-        <commandSubTopic>/gazebo/command/motor_speed</commandSubTopic>
-        <motorNumber>${motor_number}</motorNumber>
-        <rotorDragCoefficient>${rotor_drag_coefficient}</rotorDragCoefficient>
-        <rollingMomentCoefficient>${rolling_moment_coefficient}</rollingMomentCoefficient>
-        <motorSpeedPubTopic>/motor_speed/${motor_number}</motorSpeedPubTopic>
-        <rotorVelocitySlowdownSim>${rotor_velocity_slowdown_sim}</rotorVelocitySlowdownSim>
-      </plugin>
-    </gazebo>
-    <gazebo reference="rotor_${motor_number}">
-      <material>Gazebo/${color}</material>
-    </gazebo>
-  </xacro:macro>
-  <!-- Tilting rotor unit link and joint. -->
   <xacro:macro name="single_tilt_unit_minimal"
     params="robot_namespace direction parent mass_rotor mass_tilt_unit rotor_offset_top motor_number color mesh mesh_tilt_unit *origin *inertia">
@@ -246,7 +147,7 @@
     </gazebo>
   </xacro:macro>
-  <!-- Double tilt unit joint and link -->
-  <xacro:macro name="double_tilt_unit"
-    params="robot_namespace suffix direction_upper direction_lower motor_constant motor_constant_lower moment_constant moment_constant_lower parent mass_rotor mass_tilt_unit time_constant_up time_constant_down max_rot_velocity rotor_offset_top motor_number rotor_drag_coefficient rolling_moment_coefficient color mesh mesh_tilt_unit p_gain i_gain d_gain *origin *inertia">
+   <!-- Tilting double rotor unit link and joint. -->
+  <xacro:macro name="double_tilt_unit_minimal"
+    params="robot_namespace direction_upper direction_lower parent mass_rotor mass_tilt_unit rotor_offset_top motor_number lower_start_index color mesh mesh_tilt_unit *origin *inertia">
     <!-- Rotor tilt_unit -->
     <joint name="${robot_namespace}/tilt_unit_${motor_number}_revolutejoint" type="continuous">
@@ -256,4 +157,7 @@
       <child link="${namespace}/tilt_unit_${motor_number}" />
     </joint>
+    <gazebo reference="${robot_namespace}/tilt_unit_${motor_number}_revolutejoint">
+      <provideFeedback>true</provideFeedback>
+    </gazebo>
     <link name="${namespace}/tilt_unit_${motor_number}">
       <inertial>
@@ -273,26 +177,4 @@
       </collision>
     </link>
-    <gazebo>
-      <plugin name="${suffix}_tilt_unit_model" filename="librotors_gazebo_motor_model.so">
-        <robotNamespace>${robot_namespace}</robotNamespace>
-        <jointName>${namespace}/tilt_unit_${motor_number}_revolutejoint</jointName>
-        <linkName>${namespace}/tilt_unit_${motor_number}</linkName>
-        <turningDirection>ccw</turningDirection>
-        <motorType>position</motorType>
-        <commandSubTopic>/gazebo/command/motor_speed</commandSubTopic>
-        <motorNumber>${motor_number+12}</motorNumber>
-        <motorSpeedPubTopic>/tilt_motor_${motor_number}/velocity</motorSpeedPubTopic>
-        <motorPositionPubTopic>/tilt_motor_${motor_number}/position</motorPositionPubTopic>
-        <joint_control_pid>
-            <p>${p_gain}</p>
-            <i>${i_gain}</i>
-            <d>${d_gain}</d>
-            <iMax>1.0</iMax>
-            <iMin>-1.0</iMin>
-            <cmdMax>2.0</cmdMax>
-            <cmdMin>-2.0</cmdMin>
-        </joint_control_pid>
-      </plugin>
-    </gazebo>
     <gazebo reference="${namespace}/tilt_unit_${motor_number}">
       <material>Gazebo/White</material>
@@ -322,34 +204,15 @@
       </collision>
     </link>
-    <gazebo>
-      <plugin name="${suffix}_upper_motor_model" filename="librotors_gazebo_motor_model.so">
-        <robotNamespace>${robot_namespace}</robotNamespace>
-        <jointName>rotor_${motor_number}_joint</jointName>
-        <linkName>rotor_${motor_number}</linkName>
-        <turningDirection>${direction_upper}</turningDirection>
-        <timeConstantUp>${time_constant_up}</timeConstantUp>
-        <timeConstantDown>${time_constant_down}</timeConstantDown>
-        <maxRotVelocity>${max_rot_velocity}</maxRotVelocity>
-        <motorConstant>${motor_constant}</motorConstant>
-        <momentConstant>${moment_constant}</momentConstant>
-        <commandSubTopic>/gazebo/command/motor_speed</commandSubTopic>
-        <motorNumber>${motor_number}</motorNumber>
-        <rotorDragCoefficient>${rotor_drag_coefficient}</rotorDragCoefficient>
-        <rollingMomentCoefficient>${rolling_moment_coefficient}</rollingMomentCoefficient>
-        <motorSpeedPubTopic>/motor_speed/${motor_number}_upper</motorSpeedPubTopic>
-        <rotorVelocitySlowdownSim>${rotor_velocity_slowdown_sim}</rotorVelocitySlowdownSim>
-      </plugin>
-    </gazebo>
     <gazebo reference="rotor_${motor_number}">
       <material>Gazebo/${color}</material>
     </gazebo>
     <!-- Lower Rotor -->
-    <joint name="rotor_${motor_number+6}_joint" type="continuous">
+    <joint name="rotor_${motor_number+lower_start_index}_joint" type="continuous">
       <origin xyz="0 0 ${-rotor_offset_top}" rpy="0 0 0" />
       <axis xyz="0 0 1" />
       <parent link="${namespace}/tilt_unit_${motor_number}" />
-      <child link="rotor_${motor_number+6}" />
-    </joint>
-    <link name="rotor_${motor_number+6}">
+      <child link="rotor_${motor_number+lower_start_index}" />
+    </joint>
+    <link name="rotor_${motor_number+lower_start_index}">
       <inertial>
         <mass value="${mass_rotor}" /> <!-- [kg] -->
@@ -368,24 +231,5 @@
       </collision>
     </link>
-    <gazebo>
-      <plugin name="${suffix}_lower_motor_model" filename="librotors_gazebo_motor_model.so">
-        <robotNamespace>${robot_namespace}</robotNamespace>
-        <jointName>rotor_${motor_number+6}_joint</jointName>
-        <linkName>rotor_${motor_number+6}</linkName>
-        <turningDirection>${direction_lower}</turningDirection>
-        <timeConstantUp>${time_constant_up}</timeConstantUp>
-        <timeConstantDown>${time_constant_down}</timeConstantDown>
-        <maxRotVelocity>${max_rot_velocity}</maxRotVelocity>
-        <motorConstant>${motor_constant_lower}</motorConstant>
-        <momentConstant>${moment_constant_lower}</momentConstant>
-        <commandSubTopic>/gazebo/command/motor_speed</commandSubTopic>
-        <motorNumber>${motor_number+6}</motorNumber>
-        <rotorDragCoefficient>${rotor_drag_coefficient}</rotorDragCoefficient>
-        <rollingMomentCoefficient>${rolling_moment_coefficient}</rollingMomentCoefficient>
-        <motorSpeedPubTopic>/motor_speed/${motor_number}_lower</motorSpeedPubTopic>
-        <rotorVelocitySlowdownSim>${rotor_velocity_slowdown_sim}</rotorVelocitySlowdownSim>
-      </plugin>
-    </gazebo>
-    <gazebo reference="rotor_${motor_number+6}">
+    <gazebo reference="rotor_${motor_number+lower_start_index}">
       <material>Gazebo/${color}</material>
     </gazebo>

Commit message: model loading automatic

File: rotors_description/urdf/omav_snippets.xacro (robot description, xacro)
@@ -93,4 +93,6 @@
       <xacro:insert_block name="origin" />
       <axis xyz="1 0 0" />
+      <!--dynamics damping="0.035" friction="0" /-->
+      <dynamics damping="0.0" friction="0" />
       <parent link="${parent}" />
       <child link="${namespace}/tilt_unit_${motor_number}" />

Commit message: new damping values, using p control

File: rotors_description/urdf/omav_snippets.xacro (robot description, xacro)
@@ -93,6 +93,5 @@
       <xacro:insert_block name="origin" />
       <axis xyz="1 0 0" />
-      <!--dynamics damping="0.035" friction="0" /-->
-      <dynamics damping="0.0" friction="0" />
+      <dynamics damping="0.035" friction="0" />
       <parent link="${parent}" />
       <child link="${namespace}/tilt_unit_${motor_number}" />
